File: cubesat-fcu/fcu-mem.sch (KiCad schematic (older format))
At the start: 6 parts, among them U4 74HC573#SOIC, U5 74HC573#SOIC, U6 IS61C5128AL-10TLI

Commit message: Broke everything
Parts:
- removed U4, U5: 74HC573#SOIC, Package_SO:TSSOP-20_4.4x6.5mm_P0.65mm, symbol yktsat-common:74HC573#SOIC
- added U? (x2): 74HC573#SOIC, Package_SO:TSSOP-20_4.4x6.5mm_P0.65mm, symbol yktsat-common:74HC573#SOIC
Connections:
- net +3V3-A: now also U?.20 (VCC), U?.20 (VCC)
- net FCU_ALE1: now also U?.11 (LE)
- net FCU_ALE2: now also U?.11 (LE)
- net GND: now also U?.1 (~OE), U?.1 (~OE), U?.10 (GND), U?.10 (GND)
- net PK0: now also U?.2 (D0), U?.2 (D0)
- net PK1: now also U?.3 (D1), U?.3 (D1)
- net PK2: now also U?.4 (D2), U?.4 (D2)
- net PK3: now also U?.5 (D3)
- net PK4: now also U?.6 (D4)
- net PK5: now also U?.7 (D5)
- net PK6: now also U?.8 (D6)
- net PK7: now also U?.9 (D7)
- net at U6.41 (A18): now also U?.17 (Q2)
- net at U6.40 (A17): now also U?.18 (Q1)
- net at U6.39 (A16): now also U?.19 (Q0)
- net at U6.38 (A15): now also U?.12 (Q7)
- net at U6.30 (A14): now also U?.13 (Q6)
- net at U6.29 (A13): now also U?.14 (Q5)
- net at U6.28 (A12): now also U?.15 (Q4)
- net at U6.27 (A11): now also U?.16 (Q3)
- net at U6.26 (A10): now also U?.17 (Q2)
- net at U6.20 (A9): now also U?.18 (Q1)
- net at U6.19 (A8): now also U?.19 (Q0)
Changed lines of the file:
@@
 $Descr A4 11693 8268
 encoding utf-8
-Sheet 4 4
+Sheet 4 5
 Title "Yktsat FCU SRAM Module"
 Date "2020-03-29"
@@
 Comment4 ""
 $EndDescr
-$Comp
-L yktsat-common:74HC573#SOIC U?
-U 1 1 5E800EE2
-P 4500 6050
-AR Path="/5E800EE2" Ref="U?"  Part="1"
-AR Path="/5E7F1954/5E800EE2" Ref="U5"  Part="1"
-F 0 "U5" H 4725 7367 50  0000 C CNN
-F 1 "74HC573#SOIC" H 4725 7276 50  0000 C CNN
-F 2 "Package_SO:TSSOP-20_4.4x6.5mm_P0.65mm" H 5400 5900 50  0001 C CNN
-F 3 "http://www.farnell.com/datasheets/2030238.pdf" H 4500 6300 50  0001 C CNN
-	1    4500 6050
-	1    0    0    -1
-$EndComp
-$Comp
-L yktsat-common:74HC573#SOIC U?
-U 1 1 5E800EE8
-P 4500 4650
-AR Path="/5E800EE8" Ref="U?"  Part="1"
-AR Path="/5E7F1954/5E800EE8" Ref="U4"  Part="1"
-F 0 "U4" H 4725 5967 50  0000 C CNN
-F 1 "74HC573#SOIC" H 4725 5876 50  0000 C CNN
-F 2 "Package_SO:TSSOP-20_4.4x6.5mm_P0.65mm" H 5400 4500 50  0001 C CNN
-F 3 "http://www.farnell.com/datasheets/2030238.pdf" H 4500 4900 50  0001 C CNN
-	1    4500 4650
-	1    0    0    -1
-$EndComp
-$Comp
-L yktsat-common:+3V3-A #PWR0101
-U 1 1 5E830280
-P 7000 1650
-F 0 "#PWR0101" H 7000 1500 50  0001 C CNN
-F 1 "+3V3-A" H 7015 1823 50  0000 C CNN
-F 2 "" H 7000 1650 50  0001 C CNN
-F 3 "" H 7000 1650 50  0001 C CNN
-	1    7000 1650
-	1    0    0    -1
-$EndComp
 $Comp
 L power:GND #PWR0111
@@
 Wire Wire Line
 	5150 4450 5050 4450
-$Comp
-L yktsat-common:+3V3-A #PWR0117
-U 1 1 5E844DE0
-P 5150 5850
-F 0 "#PWR0117" H 5150 5700 50  0001 C CNN
-F 1 "+3V3-A" V 5200 5850 50  0000 C CNN
-F 2 "" H 5150 5850 50  0001 C CNN
-F 3 "" H 5150 5850 50  0001 C CNN
-	1    5150 5850
-	1    0    0    -1
-$EndComp
 Wire Wire Line
 	5150 5850 5050 5850
@@
 F 3 "http://www.issi.com/WW/pdf/61-64C5128AL.pdf" H 7000 3450 50  0001 C CNN
 	1    7000 3450
-	1    0    0    -1
-$EndComp
-$Comp
-L yktsat-common:+3V3-A #PWR0116
-U 1 1 5E8426E1
-P 5150 4400
-F 0 "#PWR0116" H 5150 4250 50  0001 C CNN
-F 1 "+3V3-A" V 5200 4400 50  0000 C CNN
-F 2 "" H 5150 4400 50  0001 C CNN
-F 3 "" H 5150 4400 50  0001 C CNN
-	1    5150 4400
 	1    0    0    -1
 $EndComp
@@
 Wire Bus Line
 	3600 2250 3050 2250
+Text Label 3100 2250 0    50   ~ 0
+PK[0..7]
+Text HLabel 3050 2250 0    50   Input ~ 0
+PK[0..7]
 Wire Bus Line
 	8450 2250 8450 2950
 Wire Bus Line
 	3600 2250 3600 5100
-Text Label 3100 2250 0    50   ~ 0
-PK[0..7]
-Text HLabel 3050 2250 0    50   Input ~ 0
-PK[0..7]
+$Comp
+L yktsat-common:+3V3-A #PWR?
+U 1 1 5E82F2F9
+P 7000 1650
+F 0 "#PWR?" H 7000 1500 50  0001 C CNN
+F 1 "+3V3-A" H 7015 1823 50  0000 C CNN
+F 2 "" H 7000 1650 50  0001 C CNN
+F 3 "" H 7000 1650 50  0001 C CNN
+	1    7000 1650
+	1    0    0    -1
+$EndComp
+$Comp
+L yktsat-common:+3V3-A #PWR?
+U 1 1 5E82FDB1
+P 5150 4400
+F 0 "#PWR?" H 5150 4250 50  0001 C CNN
+F 1 "+3V3-A" H 5165 4573 50  0000 C CNN
+F 2 "" H 5150 4400 50  0001 C CNN
+F 3 "" H 5150 4400 50  0001 C CNN
+	1    5150 4400
+	1    0    0    -1
+$EndComp
+$Comp
+L yktsat-common:+3V3-A #PWR?
+U 1 1 5E830FFC
+P 5150 5850
+F 0 "#PWR?" H 5150 5700 50  0001 C CNN
+F 1 "+3V3-A" H 5165 6023 50  0000 C CNN
+F 2 "" H 5150 5850 50  0001 C CNN
+F 3 "" H 5150 5850 50  0001 C CNN
+	1    5150 5850
+	1    0    0    -1
+$EndComp
+$Comp
+L yktsat-common:74HC573#SOIC U?
+U 1 1 5E841AC9
+P 4500 4650
+F 0 "U?" H 4725 5967 50  0000 C CNN
+F 1 "74HC573#SOIC" H 4725 5876 50  0000 C CNN
+F 2 "Package_SO:TSSOP-20_4.4x6.5mm_P0.65mm" H 5400 4500 50  0001 C CNN
+F 3 "" H 4500 4900 50  0001 C CNN
+	1    4500 4650
+	1    0    0    -1
+$EndComp
+$Comp
+L yktsat-common:74HC573#SOIC U?
+U 1 1 5E842DB1
+P 4500 6050
+F 0 "U?" H 4725 7367 50  0000 C CNN
+F 1 "74HC573#SOIC" H 4725 7276 50  0000 C CNN
+F 2 "Package_SO:TSSOP-20_4.4x6.5mm_P0.65mm" H 5400 5900 50  0001 C CNN
+F 3 "" H 4500 6300 50  0001 C CNN
+	1    4500 6050
+	1    0    0    -1
+$EndComp
 $EndSCHEMATC
