File: cubesat-fcu/fcu-mram.sch (KiCad schematic (older format))
At the start: 0 parts

Commit message: Broke everything
Parts:
- added U?: MR25H128A, Package_DFN_QFN:DFN-8-1EP_6x5mm_P1.27mm_EP2x2mm, symbol yktsat-common:MR25H128A
Changed lines of the file:
@@
 $Descr A4 11693 8268
 encoding utf-8
-Sheet 1 1
+Sheet 5 5
 Title ""
 Date ""
@@
 Comment4 ""
 $EndDescr
+$Comp
+L yktsat-common:MR25H128A U?
+U 1 1 5E83DB63
+P 5600 4350
+F 0 "U?" H 6050 5417 50  0000 C CNN
+F 1 "MR25H128A" H 6050 5326 50  0000 C CNN
+F 2 "Package_DFN_QFN:DFN-8-1EP_6x5mm_P1.27mm_EP2x2mm" H 6750 4200 50  0001 C CNN
+F 3 "https://ru.mouser.com/datasheet/2/144/MR25H128A_Datasheet-1219034.pdf" H 5600 4350 50  0001 C CNN
+	1    5600 4350
+	1    0    0    -1
+$EndComp
 $EndSCHEMATC
