File: ykts-payload/_autosave-ykts-payload-mcu.sch (KiCad schematic (older format))
At the start: 77 parts, among them J3 AVR-JTAG-10, J4 AVR-ISP-6, J5 Conn_01x03_Male, U10 PCA9534BS3,118, U11 PCA9534BS3,118, U12 PCA9534BS3,118, U13 PCA9534BS3,118, U4 ATmega2560-16AU, U5 74HC4051BQ,115, U7 74HC4051BQ,115, U8 74HC4051BQ,115, U9 74HC4051BQ,115, Y1 8 MHz

Commit message: Add nodes
Changed lines of the file:
@@
-$EndSheet
-$Sheet
-S 500  13500 1500 500
-U 63801AEE
-F0 "MCU Node2" 50
-F1 "ykts-mcu-node1.sch" 50
 $EndSheet
 $Sheet
@@
 F1 "ykts-mcu-node15.sch" 50
 $EndSheet
+$Sheet
+S 500  13500 1500 500
+U 63801AEE
+F0 "MCU Node2" 50
+F1 "ykts-mcu-node2.sch" 50
+$EndSheet
 $EndSCHEMATC
