File: ykts-payload/_autosave-ykts-payload-mcu.sch (KiCad schematic (older format))
At the start: 101 parts, among them J3 AVR-JTAG-10, J4 Conn_01x07_Female, J5 Conn_01x03_Female, J6 Micro_SD_Card, J7 AVR-ISP-6, J8 Conn_01x03_Male, U10 74HC4051BQ,115, U11 74HC4051BQ,115, U12 74HC4051BQ,115, U13 PCA9534BS3,118, U4 PCA9534BS3,118, U5 PCA9534BS3,118, U6 ATmega2560-16AU, U7 AMS1117-3.3, U8 PCA9534BS3,118, U9 74HC4051BQ,115, Y2 8 MHz

Commit message: Update PCB
Parts:
- added R47: 1K, Resistor_SMD:R_0402_1005Metric, symbol Device:R_Small
- renumbered R47 to R48, R48 to R49, R49 to R50, R50 to R51, R51 to R52, R52 to R53, R53 to R54, R54 to R55, R55 to R56, R56 to R57, R57 to R58, R58 to R59, R59 to R60, R60 to R61, R61 to R62, R62 to R63, R63 to R64, R64 to R65, R65 to R66, R66 to R67, R67 to R68, R68 to R69, R69 to R70, R70 to R71, R71 to R72, R72 to R73
Connections:
- net GEIGER_EN: now also R47.2; no longer U6.74 (PA4)
- new net: R47.1, U6.74 (PA4)
Changed lines of the file:
@@
 P 11100 1350
 AR Path="/61584717" Ref="R?"  Part="1"
-AR Path="/6174477C/61584717" Ref="R59"  Part="1"
-F 0 "R59" V 10904 1350 50  0000 C CNN
+AR Path="/6174477C/61584717" Ref="R60"  Part="1"
+F 0 "R60" V 10904 1350 50  0000 C CNN
 F 1 "33K" V 10995 1350 50  0000 C CNN
 F 2 "Resistor_SMD:R_0402_1005Metric" H 11100 1350 50  0001 C CNN
@@
 P 11100 3100
 AR Path="/61597144" Ref="R?"  Part="1"
-AR Path="/6174477C/61597144" Ref="R60"  Part="1"
-F 0 "R60" V 10904 3100 50  0000 C CNN
+AR Path="/6174477C/61597144" Ref="R61"  Part="1"
+F 0 "R61" V 10904 3100 50  0000 C CNN
 F 1 "33K" V 10995 3100 50  0000 C CNN
 F 2 "Resistor_SMD:R_0402_1005Metric" H 11100 3100 50  0001 C CNN
@@
 P 13800 1350
 AR Path="/6159EB55" Ref="R?"  Part="1"
-AR Path="/6174477C/6159EB55" Ref="R64"  Part="1"
-F 0 "R64" V 13604 1350 50  0000 C CNN
+AR Path="/6174477C/6159EB55" Ref="R65"  Part="1"
+F 0 "R65" V 13604 1350 50  0000 C CNN
 F 1 "33K" V 13695 1350 50  0000 C CNN
 F 2 "Resistor_SMD:R_0402_1005Metric" H 13800 1350 50  0001 C CNN
@@
 P 13800 3100
 AR Path="/6159EB86" Ref="R?"  Part="1"
-AR Path="/6174477C/6159EB86" Ref="R65"  Part="1"
-F 0 "R65" V 13604 3100 50  0000 C CNN
+AR Path="/6174477C/6159EB86" Ref="R66"  Part="1"
+F 0 "R66" V 13604 3100 50  0000 C CNN
 F 1 "33K" V 13695 3100 50  0000 C CNN
 F 2 "Resistor_SMD:R_0402_1005Metric" H 13800 3100 50  0001 C CNN
@@
 P 10550 6600
 AR Path="/6165476D" Ref="R?"  Part="1"
-AR Path="/6174477C/6165476D" Ref="R52"  Part="1"
-F 0 "R52" V 10354 6600 50  0000 C CNN
+AR Path="/6174477C/6165476D" Ref="R53"  Part="1"
+F 0 "R53" V 10354 6600 50  0000 C CNN
 F 1 "JMP" V 10445 6600 50  0000 C CNN
 F 2 "Resistor_SMD:R_0402_1005Metric" H 10550 6600 50  0001 C CNN
@@
 P 10350 6700
 AR Path="/61654D72" Ref="R?"  Part="1"
-AR Path="/6174477C/61654D72" Ref="R51"  Part="1"
-F 0 "R51" V 10154 6700 50  0000 C CNN
+AR Path="/6174477C/61654D72" Ref="R52"  Part="1"
+F 0 "R52" V 10154 6700 50  0000 C CNN
 F 1 "JMP" V 10245 6700 50  0000 C CNN
 F 2 "Resistor_SMD:R_0402_1005Metric" H 10350 6700 50  0001 C CNN
@@
 P 10750 6500
 AR Path="/6164472D" Ref="R?"  Part="1"
-AR Path="/6174477C/6164472D" Ref="R53"  Part="1"
-F 0 "R53" V 10554 6500 50  0000 C CNN
+AR Path="/6174477C/6164472D" Ref="R54"  Part="1"
+F 0 "R54" V 10554 6500 50  0000 C CNN
 F 1 "JMP" V 10645 6500 50  0000 C CNN
 F 2 "Resistor_SMD:R_0402_1005Metric" H 10750 6500 50  0001 C CNN
@@
 P 11050 6900
 AR Path="/6167FC40" Ref="R?"  Part="1"
-AR Path="/6174477C/6167FC40" Ref="R58"  Part="1"
-F 0 "R58" V 10854 6900 50  0000 C CNN
+AR Path="/6174477C/6167FC40" Ref="R59"  Part="1"
+F 0 "R59" V 10854 6900 50  0000 C CNN
 F 1 "10K" V 10945 6900 50  0000 C CNN
 F 2 "Resistor_SMD:R_0402_1005Metric" H 11050 6900 50  0001 C CNN
@@
 P 10950 7100
 AR Path="/6168072B" Ref="R?"  Part="1"
-AR Path="/6174477C/6168072B" Ref="R56"  Part="1"
-F 0 "R56" V 10754 7100 50  0000 C CNN
+AR Path="/6174477C/6168072B" Ref="R57"  Part="1"
+F 0 "R57" V 10754 7100 50  0000 C CNN
 F 1 "10K" V 10845 7100 50  0000 C CNN
 F 2 "Resistor_SMD:R_0402_1005Metric" H 10950 7100 50  0001 C CNN
@@
 P 10850 7300
 AR Path="/61680B52" Ref="R?"  Part="1"
-AR Path="/6174477C/61680B52" Ref="R54"  Part="1"
-F 0 "R54" V 10654 7300 50  0000 C CNN
+AR Path="/6174477C/61680B52" Ref="R55"  Part="1"
+F 0 "R55" V 10654 7300 50  0000 C CNN
 F 1 "10K" V 10745 7300 50  0000 C CNN
 F 2 "Resistor_SMD:R_0402_1005Metric" H 10850 7300 50  0001 C CNN
@@
 P 11050 5750
 AR Path="/616EDD64" Ref="R?"  Part="1"
-AR Path="/6174477C/616EDD64" Ref="R57"  Part="1"
-F 0 "R57" V 10854 5750 50  0000 C CNN
+AR Path="/6174477C/616EDD64" Ref="R58"  Part="1"
+F 0 "R58" V 10854 5750 50  0000 C CNN
 F 1 "10K" V 10945 5750 50  0000 C CNN
 F 2 "Resistor_SMD:R_0402_1005Metric" H 11050 5750 50  0001 C CNN
@@
 P 10950 5550
 AR Path="/616EE4AA" Ref="R?"  Part="1"
-AR Path="/6174477C/616EE4AA" Ref="R55"  Part="1"
-F 0 "R55" V 10754 5550 50  0000 C CNN
+AR Path="/6174477C/616EE4AA" Ref="R56"  Part="1"
+F 0 "R56" V 10754 5550 50  0000 C CNN
 F 1 "10K" V 10845 5550 50  0000 C CNN
 F 2 "Resistor_SMD:R_0402_1005Metric" H 10950 5550 50  0001 C CNN
@@
 P 13550 6600
 AR Path="/6171D25B" Ref="R?"  Part="1"
-AR Path="/6174477C/6171D25B" Ref="R62"  Part="1"
-F 0 "R62" V 13354 6600 50  0000 C CNN
+AR Path="/6174477C/6171D25B" Ref="R63"  Part="1"
+F 0 "R63" V 13354 6600 50  0000 C CNN
 F 1 "JMP" V 13445 6600 50  0000 C CNN
 F 2 "Resistor_SMD:R_0402_1005Metric" H 13550 6600 50  0001 C CNN
@@
 P 13350 6700
 AR Path="/6171D261" Ref="R?"  Part="1"
-AR Path="/6174477C/6171D261" Ref="R61"  Part="1"
-F 0 "R61" V 13154 6700 50  0000 C CNN
+AR Path="/6174477C/6171D261" Ref="R62"  Part="1"
+F 0 "R62" V 13154 6700 50  0000 C CNN
 F 1 "JMP" V 13245 6700 50  0000 C CNN
 F 2 "Resistor_SMD:R_0402_1005Metric" H 13350 6700 50  0001 C CNN
@@
 P 13750 6500
 AR Path="/6171D269" Ref="R?"  Part="1"
-AR Path="/6174477C/6171D269" Ref="R63"  Part="1"
-F 0 "R63" V 13554 6500 50  0000 C CNN
+AR Path="/6174477C/6171D269" Ref="R64"  Part="1"
+F 0 "R64" V 13554 6500 50  0000 C CNN
 F 1 "JMP" V 13645 6500 50  0000 C CNN
 F 2 "Resistor_SMD:R_0402_1005Metric" H 13750 6500 50  0001 C CNN
@@
 P 14050 6900
 AR Path="/6171D27D" Ref="R?"  Part="1"
-AR Path="/6174477C/6171D27D" Ref="R70"  Part="1"
-F 0 "R70" V 13854 6900 50  0000 C CNN
+AR Path="/6174477C/6171D27D" Ref="R71"  Part="1"
+F 0 "R71" V 13854 6900 50  0000 C CNN
 F 1 "10K" V 13945 6900 50  0000 C CNN
 F 2 "Resistor_SMD:R_0402_1005Metric" H 14050 6900 50  0001 C CNN
@@
 P 13950 7100
 AR Path="/6171D283" Ref="R?"  Part="1"
-AR Path="/6174477C/6171D283" Ref="R68"  Part="1"
-F 0 "R68" V 13754 7100 50  0000 C CNN
+AR Path="/6174477C/6171D283" Ref="R69"  Part="1"
+F 0 "R69" V 13754 7100 50  0000 C CNN
 F 1 "10K" V 13845 7100 50  0000 C CNN
 F 2 "Resistor_SMD:R_0402_1005Metric" H 13950 7100 50  0001 C CNN
@@
 P 13850 7300
 AR Path="/6171D289" Ref="R?"  Part="1"
-AR Path="/6174477C/6171D289" Ref="R66"  Part="1"
-F 0 "R66" V 13654 7300 50  0000 C CNN
+AR Path="/6174477C/6171D289" Ref="R67"  Part="1"
+F 0 "R67" V 13654 7300 50  0000 C CNN
 F 1 "10K" V 13745 7300 50  0000 C CNN
 F 2 "Resistor_SMD:R_0402_1005Metric" H 13850 7300 50  0001 C CNN
@@
 P 14050 5750
 AR Path="/6171D2B5" Ref="R?"  Part="1"
-AR Path="/6174477C/6171D2B5" Ref="R69"  Part="1"
-F 0 "R69" V 13854 5750 50  0000 C CNN
+AR Path="/6174477C/6171D2B5" Ref="R70"  Part="1"
+F 0 "R70" V 13854 5750 50  0000 C CNN
 F 1 "10K" V 13945 5750 50  0000 C CNN
 F 2 "Resistor_SMD:R_0402_1005Metric" H 14050 5750 50  0001 C CNN
@@
 P 13950 5550
 AR Path="/6171D2BB" Ref="R?"  Part="1"
-AR Path="/6174477C/6171D2BB" Ref="R67"  Part="1"
-F 0 "R67" V 13754 5550 50  0000 C CNN
+AR Path="/6174477C/6171D2BB" Ref="R68"  Part="1"
+F 0 "R68" V 13754 5550 50  0000 C CNN
 F 1 "10K" V 13845 5550 50  0000 C CNN
 F 2 "Resistor_SMD:R_0402_1005Metric" H 13950 5550 50  0001 C CNN
@@
 P 14750 9550
 AR Path="/61B92498" Ref="R?"  Part="1"
-AR Path="/6174477C/61B92498" Ref="R71"  Part="1"
-F 0 "R71" V 14554 9550 50  0000 C CNN
+AR Path="/6174477C/61B92498" Ref="R72"  Part="1"
+F 0 "R72" V 14554 9550 50  0000 C CNN
 F 1 "1K" V 14645 9550 50  0000 C CNN
 F 2 "Resistor_SMD:R_0402_1005Metric" H 14750 9550 50  0001 C CNN
@@
 P 15450 9550
 AR Path="/61BF2AF0" Ref="R?"  Part="1"
-AR Path="/6174477C/61BF2AF0" Ref="R72"  Part="1"
-F 0 "R72" V 15254 9550 50  0000 C CNN
+AR Path="/6174477C/61BF2AF0" Ref="R73"  Part="1"
+F 0 "R73" V 15254 9550 50  0000 C CNN
 F 1 "1K" V 15345 9550 50  0000 C CNN
 F 2 "Resistor_SMD:R_0402_1005Metric" H 15450 9550 50  0001 C CNN
@@
 P 10250 8650
 AR Path="/61D9999C" Ref="R?"  Part="1"
-AR Path="/6174477C/61D9999C" Ref="R47"  Part="1"
-F 0 "R47" V 10054 8650 50  0000 C CNN
+AR Path="/6174477C/61D9999C" Ref="R48"  Part="1"
+F 0 "R48" V 10054 8650 50  0000 C CNN
 F 1 "1M" V 10145 8650 50  0000 C CNN
 F 2 "Resistor_SMD:R_0603_1608Metric" H 10250 8650 50  0001 C CNN
@@
 P 10250 8900
 AR Path="/61E1E7C4" Ref="R?"  Part="1"
-AR Path="/6174477C/61E1E7C4" Ref="R48"  Part="1"
-F 0 "R48" V 10054 8900 50  0000 C CNN
+AR Path="/6174477C/61E1E7C4" Ref="R49"  Part="1"
+F 0 "R49" V 10054 8900 50  0000 C CNN
 F 1 "1M" V 10145 8900 50  0000 C CNN
 F 2 "Resistor_SMD:R_0603_1608Metric" H 10250 8900 50  0001 C CNN
@@
 P 10250 9150
 AR Path="/61E3F9BE" Ref="R?"  Part="1"
-AR Path="/6174477C/61E3F9BE" Ref="R49"  Part="1"
-F 0 "R49" V 10054 9150 50  0000 C CNN
+AR Path="/6174477C/61E3F9BE" Ref="R50"  Part="1"
+F 0 "R50" V 10054 9150 50  0000 C CNN
 F 1 "1M" V 10145 9150 50  0000 C CNN
 F 2 "Resistor_SMD:R_0603_1608Metric" H 10250 9150 50  0001 C CNN
@@
 P 10250 9400
 AR Path="/61E6091E" Ref="R?"  Part="1"
-AR Path="/6174477C/61E6091E" Ref="R50"  Part="1"
-F 0 "R50" V 10054 9400 50  0000 C CNN
+AR Path="/6174477C/61E6091E" Ref="R51"  Part="1"
+F 0 "R51" V 10054 9400 50  0000 C CNN
 F 1 "1M" V 10145 9400 50  0000 C CNN
 F 2 "Resistor_SMD:R_0603_1608Metric" H 10250 9400 50  0001 C CNN
@@
 Wire Wire Line
 	4200 9250 4050 9250
-Text Label 8250 2400 0    50   ~ 0
+Text Label 8550 2400 0    50   ~ 0
 GEIGER_EN
-Wire Wire Line
-	8250 2400 7900 2400
 Text Label 4350 9450 0    50   ~ 0
 GEIGER_EN
@@
 	-1   0    0    1
 $EndComp
+$Comp
+L Device:R_Small R?
+U 1 1 65A83E0A
+P 8400 2400
+AR Path="/65A83E0A" Ref="R?"  Part="1"
+AR Path="/6174477C/65A83E0A" Ref="R47"  Part="1"
+F 0 "R47" V 8204 2400 50  0000 C CNN
+F 1 "1K" V 8295 2400 50  0000 C CNN
+F 2 "Resistor_SMD:R_0402_1005Metric" H 8400 2400 50  0001 C CNN
+F 3 "~" H 8400 2400 50  0001 C CNN
+	1    8400 2400
+	0    -1   -1   0
+$EndComp
+Wire Wire Line
+	7900 2400 8300 2400
+Wire Wire Line
+	8500 2400 8550 2400
 $EndSCHEMATC
