File: ykts-payload/_autosave-ykts-payload.kicad_pcb (KiCad board)
At the start: 2 copper layers, 79 parts, among them J1 PC/104 Connector, U1 AMS1117-3.3, U10 PCA9534BS3,118, U11 PCA9534BS3,118, U12 PCA9534BS3,118, U13 PCA9534BS3,118, U14 ATmega328PB-MU, U15 ATmega328PB-MU, U16 ATmega328PB-MU, U17 ATmega328PB-MU, U18 ATmega328PB-MU, U19 ATmega328PB-MU, U2 MCP2515-xST, U20 ATmega328PB-MU, U21 ATmega328PB-MU, U22 ATmega328PB-MU, U23 ATmega328PB-MU, U24 ATmega328PB-MU, U25 ATmega328PB-MU, U26 ATmega328PB-MU, U27 ATmega328PB-MU, U28 ATmega328PB-MU, U29 ATmega328PB-MU, U3 TJA1051T-3, U4 ATmega2560-16AU, U5 74HC4051BQ,115, U6 INA3221AIRGVR, U7 74HC4051BQ,115, U8 74HC4051BQ,115, U9 74HC4051BQ,115, Y1 8 MHz, Y2 12MHz

Commit message: Add nodes
Parts:
- removed C1, C2, C22, C32: 22pF, Capacitor_SMD:C_0402_1005Metric
- removed C10, C17, C3, C6, C8: 100nF, Capacitor_SMD:C_0603_1608Metric
- removed C11, C20, C21, C31, C33, C34: 100nF, Capacitor_SMD:C_0402_1005Metric
- removed C16: 10nF, Capacitor_SMD:C_0402_1005Metric
- removed C18: 10uF, Capacitor_Tantalum_SMD:CP_EIA-3216-10_Kemet-I
- removed C35, C36, C4, C9: 22uF, Capacitor_Tantalum_SMD:CP_EIA-3216-10_Kemet-I
- removed C5: 10uF, Capacitor_SMD:C_0603_1608Metric
- removed C7: 22uF, Capacitor_SMD:C_0603_1608Metric
- removed CH1, CH2, CL1, CL2: 50pF, Capacitor_SMD:C_0402_1005Metric
- removed D1: Generic, Diode_SMD:D_SOD-323
- removed D2: TVS1, Diode_SMD:D_SOD-323
- removed D3: TVS2, Diode_SMD:D_SOD-323
- removed FL1: DLW21SN921SK2, Inductor_SMD:L_CommonModeChoke_Coilcraft_0805USB
- removed J1: PC/104 Connector, Connector_PinSocket_2.54mm:PinSocket_2x32_P2.54mm_Vertical
- removed L5: Ferrite, Inductor_SMD:L_1206_3216Metric
- removed R1, R2: 1K, Resistor_SMD:R_0402_1005Metric
- removed R10, R7, R8, R9: 4.7K, Resistor_SMD:R_0402_1005Metric
- removed R19, R22, R23: 0.1, Resistor_SMD:R_2512_6332Metric
- removed R20, R21, R3, R4, R5, R6: 10K, Resistor_SMD:R_0402_1005Metric
- removed U1: AMS1117-3.3, Package_TO_SOT_SMD:SOT-223-3_TabPin2
- removed U10, U11, U12, U13: PCA9534BS3,118, Package_DFN_QFN:HVQFN-16-1EP_3x3mm_P0.5mm_EP1.5x1.5mm
- removed U14, U15, U16, U17, U18, U19, U20, U21, U22, U23, U24, U25, U26, U27, U28, U29: ATmega328PB-MU, Package_DFN_QFN:QFN-32-1EP_5x5mm_P0.5mm_EP3.1x3.1mm
- removed U2: MCP2515-xST, Package_SO:TSSOP-20_4.4x6.5mm_P0.65mm
- removed U3: TJA1051T-3, Package_SO:SOIC-8_3.9x4.9mm_P1.27mm
- removed U4: ATmega2560-16AU, Package_QFP:TQFP-100_14x14mm_P0.5mm
- removed U5, U7, U8, U9: 74HC4051BQ,115, 74hc4051:QFN50P250X350X100-17N-D
- removed U6: INA3221AIRGVR, Package_DFN_QFN:QFN-16-1EP_4x4mm_P0.65mm_EP2.1x2.1mm
- removed Y1: 8 MHz, Crystal:Crystal_SMD_5032-4Pin_5.0x3.2mm
- removed Y2: 12MHz, Crystal:Crystal_SMD_5032-4Pin_5.0x3.2mm
