File: ykts-payload/ykts-mcu-node10.sch (KiCad schematic (older format))
At the start: 12 parts

Commit message: Update nodes
Parts:
- D15: renamed from D?; value NODE0_STATUSLED -> NODE10_STATUSLED
- gave numbers to parts that had none: 11
Connections:
- net NODE0_PWR renamed NODE10_PWR
- net NODE0_RESET renamed NODE10_RESET
- net NODE0_RX renamed NODE10_RX
- net NODE0_TX renamed NODE10_TX
Other:
- note added: "MCU Node 10"
- note removed: "MCU Node 0"
Changed lines of the file:
@@
 AR Path="/6174477C/638385BA/6391686F" Ref="U?"  Part="1"
 AR Path="/6174477C/638DF11D/6391686F" Ref="U?"  Part="1"
-AR Path="/6174477C/638DF11F/6391686F" Ref="U?"  Part="1"
-F 0 "U?" H 6100 2711 50  0000 C CNN
+AR Path="/6174477C/638DF11F/6391686F" Ref="U23"  Part="1"
+F 0 "U23" H 6100 2711 50  0000 C CNN
 F 1 "ATmega328PB-MU" H 6100 2620 50  0000 C CNN
 F 2 "Package_DFN_QFN:QFN-32-1EP_5x5mm_P0.5mm_EP3.1x3.1mm" H 6100 4300 50  0001 C CIN
@@
 AR Path="/6174477C/638385BA/63916878" Ref="SW?"  Part="1"
 AR Path="/6174477C/638DF11D/63916878" Ref="SW?"  Part="1"
-AR Path="/6174477C/638DF11F/63916878" Ref="SW?"  Part="1"
-F 0 "SW?" H 3500 2631 50  0000 C CNN
+AR Path="/6174477C/638DF11F/63916878" Ref="SW10"  Part="1"
+F 0 "SW10" H 3500 2631 50  0000 C CNN
 F 1 "ADG802BRT" H 3500 2540 50  0000 C CNN
 F 2 "Package_TO_SOT_SMD:SOT-23-6" H 3500 2500 50  0001 C CNN
@@
 AR Path="/6174477C/638385BA/63916879" Ref="C?"  Part="1"
 AR Path="/6174477C/638DF11D/63916879" Ref="C?"  Part="1"
-AR Path="/6174477C/638DF11F/63916879" Ref="C?"  Part="1"
-F 0 "C?" H 4292 2646 50  0000 L CNN
+AR Path="/6174477C/638DF11F/63916879" Ref="C64"  Part="1"
+F 0 "C64" H 4292 2646 50  0000 L CNN
 F 1 "1uF" H 4292 2555 50  0000 L CNN
 F 2 "Capacitor_SMD:C_0603_1608Metric" H 4200 2600 50  0001 C CNN
@@
 AR Path="/6174477C/638385BA/6391687A" Ref="C?"  Part="1"
 AR Path="/6174477C/638DF11D/6391687A" Ref="C?"  Part="1"
-AR Path="/6174477C/638DF11F/6391687A" Ref="C?"  Part="1"
-F 0 "C?" H 4642 2646 50  0000 L CNN
+AR Path="/6174477C/638DF11F/6391687A" Ref="C65"  Part="1"
+F 0 "C65" H 4642 2646 50  0000 L CNN
 F 1 "100nF" H 4642 2555 50  0000 L CNN
 F 2 "Capacitor_SMD:C_0402_1005Metric" H 4550 2600 50  0001 C CNN
@@
 AR Path="/6174477C/638385BA/6391687B" Ref="#PWR?"  Part="1"
 AR Path="/6174477C/638DF11D/6391687B" Ref="#PWR?"  Part="1"
-AR Path="/6174477C/638DF11F/6391687B" Ref="#PWR?"  Part="1"
-F 0 "#PWR?" H 3500 2600 50  0001 C CNN
+AR Path="/6174477C/638DF11F/6391687B" Ref="#PWR0247"  Part="1"
+F 0 "#PWR0247" H 3500 2600 50  0001 C CNN
 F 1 "GND" H 3505 2677 50  0000 C CNN
 F 2 "" H 3500 2850 50  0001 C CNN
@@
 AR Path="/6174477C/638385BA/6386F03C" Ref="C?"  Part="1"
 AR Path="/6174477C/638DF11D/6386F03C" Ref="C?"  Part="1"
-AR Path="/6174477C/638DF11F/6386F03C" Ref="C?"  Part="1"
-F 0 "C?" H 8100 4600 50  0000 L CNN
+AR Path="/6174477C/638DF11F/6386F03C" Ref="C67"  Part="1"
+F 0 "C67" H 8100 4600 50  0000 L CNN
 F 1 "22pF" H 8100 4500 50  0000 L CNN
 F 2 "Capacitor_SMD:C_0402_1005Metric" H 8400 4550 50  0001 C CNN
@@
 AR Path="/6174477C/638385BA/63916884" Ref="C?"  Part="1"
 AR Path="/6174477C/638DF11D/63916884" Ref="C?"  Part="1"
-AR Path="/6174477C/638DF11F/63916884" Ref="C?"  Part="1"
-F 0 "C?" H 8100 4600 50  0000 L CNN
+AR Path="/6174477C/638DF11F/63916884" Ref="C66"  Part="1"
+F 0 "C66" H 8100 4600 50  0000 L CNN
 F 1 "22pF" H 8100 4500 50  0000 L CNN
 F 2 "Capacitor_SMD:C_0402_1005Metric" H 8000 4550 50  0001 C CNN
@@
 AR Path="/6174477C/638385BA/6391687F" Ref="#PWR?"  Part="1"
 AR Path="/6174477C/638DF11D/6391687F" Ref="#PWR?"  Part="1"
-AR Path="/6174477C/638DF11F/6391687F" Ref="#PWR?"  Part="1"
-F 0 "#PWR?" H 8400 4450 50  0001 C CNN
+AR Path="/6174477C/638DF11F/6391687F" Ref="#PWR0248"  Part="1"
+F 0 "#PWR0248" H 8400 4450 50  0001 C CNN
 F 1 "GND" H 8405 4527 50  0000 C CNN
 F 2 "" H 8400 4700 50  0001 C CNN
@@
 AR Path="/6174477C/638385BA/63916880" Ref="#PWR?"  Part="1"
 AR Path="/6174477C/638DF11D/63916880" Ref="#PWR?"  Part="1"
-AR Path="/6174477C/638DF11F/63916880" Ref="#PWR?"  Part="1"
-F 0 "#PWR?" H 8000 4450 50  0001 C CNN
+AR Path="/6174477C/638DF11F/63916880" Ref="#PWR0249"  Part="1"
+F 0 "#PWR0249" H 8000 4450 50  0001 C CNN
 F 1 "GND" H 8005 4527 50  0000 C CNN
 F 2 "" H 8000 4700 50  0001 C CNN
@@
 	8400 4700 8400 4650
 Text Label 7050 4600 0    50   ~ 0
-NODE0_RESET
+NODE10_RESET
 $Comp
 L Device:Crystal_GND24_Small Y?
@@
 AR Path="/6174477C/638385BA/6386F034" Ref="Y?"  Part="1"
 AR Path="/6174477C/638DF11D/6386F034" Ref="Y?"  Part="1"
-AR Path="/6174477C/638DF11F/6386F034" Ref="Y?"  Part="1"
-F 0 "Y?" H 8450 4350 50  0000 L CNN
+AR Path="/6174477C/638DF11F/6386F034" Ref="Y12"  Part="1"
+F 0 "Y12" H 8450 4350 50  0000 L CNN
 F 1 "8 MHz" H 8450 4250 50  0000 L CNN
 F 2 "Crystal:Crystal_SMD_2520-4Pin_2.5x2.0mm" H 8200 4300 50  0001 C CNN
@@
 AR Path="/6174477C/638385BA/6391687D" Ref="#PWR?"  Part="1"
 AR Path="/6174477C/638DF11D/6391687D" Ref="#PWR?"  Part="1"
-AR Path="/6174477C/638DF11F/6391687D" Ref="#PWR?"  Part="1"
-F 0 "#PWR?" H 8200 3950 50  0001 C CNN
+AR Path="/6174477C/638DF11F/6391687D" Ref="#PWR0250"  Part="1"
+F 0 "#PWR0250" H 8200 3950 50  0001 C CNN
 F 1 "GND" H 8205 4027 50  0000 C CNN
 F 2 "" H 8200 4200 50  0001 C CNN
@@
 AR Path="/6174477C/638385BA/63916870" Ref="#PWR?"  Part="1"
 AR Path="/6174477C/638DF11D/63916870" Ref="#PWR?"  Part="1"
-AR Path="/6174477C/638DF11F/63916870" Ref="#PWR?"  Part="1"
-F 0 "#PWR?" H 8200 4150 50  0001 C CNN
+AR Path="/6174477C/638DF11F/63916870" Ref="#PWR0251"  Part="1"
+F 0 "#PWR0251" H 8200 4150 50  0001 C CNN
 F 1 "GND" H 8205 4227 50  0000 C CNN
 F 2 "" H 8200 4400 50  0001 C CNN
@@
 AR Path="/6174477C/638385BA/6386EE39" Ref="R?"  Part="1"
 AR Path="/6174477C/638DF11D/6386EE39" Ref="R?"  Part="1"
-AR Path="/6174477C/638DF11F/6386EE39" Ref="R?"  Part="1"
-F 0 "R?" V 6754 4400 50  0000 C CNN
+AR Path="/6174477C/638DF11F/6386EE39" Ref="R86"  Part="1"
+F 0 "R86" V 6754 4400 50  0000 C CNN
 F 1 "20K" V 6845 4400 50  0000 C CNN
 F 2 "Resistor_SMD:R_0402_1005Metric" H 6950 4400 50  0001 C CNN
@@
 $EndComp
 Text GLabel 2700 2450 0    50   Input ~ 0
-NODE0_PWR
+NODE10_PWR
 Text GLabel 3900 3650 0    50   Input ~ 0
-NODE0_RESET
+NODE10_RESET
 Text GLabel 3900 3750 0    50   Input ~ 0
-NODE0_RX
+NODE10_RX
 Text GLabel 3900 3850 0    50   Input ~ 0
-NODE0_TX
+NODE10_TX
 $Comp
 L yktsat-common:+5V_A #PWR?
@@
 AR Path="/6174477C/638385BA/6386F03F" Ref="#PWR?"  Part="1"
 AR Path="/6174477C/638DF11D/6386F03F" Ref="#PWR?"  Part="1"
-AR Path="/6174477C/638DF11F/6386F03F" Ref="#PWR?"  Part="1"
-F 0 "#PWR?" H 3500 1650 50  0001 C CNN
+AR Path="/6174477C/638DF11F/6386F03F" Ref="#PWR0252"  Part="1"
+F 0 "#PWR0252" H 3500 1650 50  0001 C CNN
 F 1 "+5V_A" H 3515 1973 50  0000 C CNN
 F 2 "" H 3500 1800 50  0001 C CNN
@@
 AR Path="/6174477C/638385BA/63916881" Ref="#PWR?"  Part="1"
 AR Path="/6174477C/638DF11D/63916881" Ref="#PWR?"  Part="1"
-AR Path="/6174477C/638DF11F/63916881" Ref="#PWR?"  Part="1"
-F 0 "#PWR?" H 4550 2600 50  0001 C CNN
+AR Path="/6174477C/638DF11F/63916881" Ref="#PWR0253"  Part="1"
+F 0 "#PWR0253" H 4550 2600 50  0001 C CNN
 F 1 "GND" H 4555 2677 50  0000 C CNN
 F 2 "" H 4550 2850 50  0001 C CNN
@@
 AR Path="/6174477C/638385BA/63916875" Ref="R?"  Part="1"
 AR Path="/6174477C/638DF11D/63916875" Ref="R?"  Part="1"
-AR Path="/6174477C/638DF11F/63916875" Ref="R?"  Part="1"
-F 0 "R?" V 8004 3950 50  0000 C CNN
+AR Path="/6174477C/638DF11F/63916875" Ref="R87"  Part="1"
+F 0 "R87" V 8004 3950 50  0000 C CNN
 F 1 "1M" V 8095 3950 50  0000 C CNN
 F 2 "Resistor_SMD:R_0402_1005Metric" H 8200 3950 50  0001 C CNN
@@
 AR Path="/6174477C/638385BA/63916876" Ref="J?"  Part="1"
 AR Path="/6174477C/638DF11D/63916876" Ref="J?"  Part="1"
-AR Path="/6174477C/638DF11F/63916876" Ref="J?"  Part="1"
-F 0 "J?" H 3770 5146 50  0000 R CNN
+AR Path="/6174477C/638DF11F/63916876" Ref="J15"  Part="1"
+F 0 "J15" H 3770 5146 50  0000 R CNN
 F 1 "AVR-ISP-6" H 3770 5055 50  0000 R CNN
 F 2 "Connector_PinHeader_2.54mm:PinHeader_2x03_P2.54mm_Vertical" V 3850 5100 50  0001 C CNN
@@
 AR Path="/6174477C/638385BA/63916877" Ref="#PWR?"  Part="1"
 AR Path="/6174477C/638DF11D/63916877" Ref="#PWR?"  Part="1"
-AR Path="/6174477C/638DF11F/63916877" Ref="#PWR?"  Part="1"
-F 0 "#PWR?" H 4200 5300 50  0001 C CNN
+AR Path="/6174477C/638DF11F/63916877" Ref="#PWR0254"  Part="1"
+F 0 "#PWR0254" H 4200 5300 50  0001 C CNN
 F 1 "GND" H 4205 5377 50  0000 C CNN
 F 2 "" H 4200 5550 50  0001 C CNN
@@
 AR Path="/6174477C/638385BA/6386EE3F" Ref="D?"  Part="1"
 AR Path="/6174477C/638DF11D/6386EE3F" Ref="D?"  Part="1"
-AR Path="/6174477C/638DF11F/6386EE3F" Ref="D?"  Part="1"
-F 0 "D?" V 8439 2682 50  0000 R CNN
-F 1 "NODE0_STATUSLED" V 8348 2682 50  0000 R CNN
+AR Path="/6174477C/638DF11F/6386EE3F" Ref="D15"  Part="1"
+F 0 "D15" V 8439 2682 50  0000 R CNN
+F 1 "NODE10_STATUSLED" V 8348 2682 50  0000 R CNN
 F 2 "LED_SMD:LED_0402_1005Metric" H 8400 2800 50  0001 C CNN
 F 3 "~" H 8400 2800 50  0001 C CNN
@@
 AR Path="/6174477C/638385BA/6386F047" Ref="R?"  Part="1"
 AR Path="/6174477C/638DF11D/6386F047" Ref="R?"  Part="1"
-AR Path="/6174477C/638DF11F/6386F047" Ref="R?"  Part="1"
-F 0 "R?" V 8204 3150 50  0000 C CNN
+AR Path="/6174477C/638DF11F/6386F047" Ref="R88"  Part="1"
+F 0 "R88" V 8204 3150 50  0000 C CNN
 F 1 "1K" V 8295 3150 50  0000 C CNN
 F 2 "Resistor_SMD:R_0402_1005Metric" H 8400 3150 50  0001 C CNN
@@
 AR Path="/6174477C/638385BA/6386F048" Ref="#PWR?"  Part="1"
 AR Path="/6174477C/638DF11D/6386F048" Ref="#PWR?"  Part="1"
-AR Path="/6174477C/638DF11F/6386F048" Ref="#PWR?"  Part="1"
-F 0 "#PWR?" H 8400 3100 50  0001 C CNN
+AR Path="/6174477C/638DF11F/6386F048" Ref="#PWR0255"  Part="1"
+F 0 "#PWR0255" H 8400 3100 50  0001 C CNN
 F 1 "GND" H 8405 3177 50  0000 C CNN
 F 2 "" H 8400 3350 50  0001 C CNN
@@
 AR Path="/6174477C/638385BA/63916871" Ref="#PWR?"  Part="1"
 AR Path="/6174477C/638DF11D/63916871" Ref="#PWR?"  Part="1"
-AR Path="/6174477C/638DF11F/63916871" Ref="#PWR?"  Part="1"
-F 0 "#PWR?" H 6100 5800 50  0001 C CNN
+AR Path="/6174477C/638DF11F/63916871" Ref="#PWR0256"  Part="1"
+F 0 "#PWR0256" H 6100 5800 50  0001 C CNN
 F 1 "GND" H 6105 5877 50  0000 C CNN
 F 2 "" H 6100 6050 50  0001 C CNN
@@
 	4200 3750 3900 3750
 Text Label 4200 3650 0    50   ~ 0
-NODE0_RESET
+NODE10_RESET
 Wire Wire Line
 	4200 3650 3900 3650
 Text Notes 5700 950  0    100  ~ 0
-MCU Node 0
+MCU Node 10
 Wire Wire Line
 	2700 2450 3100 2450
@@
 ISP_RESET
 Text Label 4200 3550 0    50   ~ 0
-NODE0_RESET
+NODE10_RESET
 Wire Wire Line
 	4200 3550 3900 3550
