File: ykts-payload/ykts-mcu-node10.sch (KiCad schematic (older format))
At the start: 12 parts, among them J23 AVR-ISP-6, SW11 ADG802BRT, U22 ATmega328PB-MU, Y15 8 MHz

Commit message: Revision B2
Hierarchal sheets for nodes
Partial PCB layout
Parts:
- renumbered C79 to C81, C80 to C82, C81 to C83, C82 to C84, U22 to U24
Changed lines of the file:
@@
 Sheet 13 18
 Title "YktSat Payload Module"
-Date "2021-10-22"
-Rev "B0"
+Date "2021-10-26"
+Rev "B1"
 Comp "Sakha Aerospace Systems, LLC"
 Comment1 ""
@@
 AR Path="/6174477C/6572958C/65833EEB" Ref="U?"  Part="1"
 AR Path="/6174477C/6577909A/65833EEB" Ref="U?"  Part="1"
-AR Path="/6174477C/6577909E/65833EEB" Ref="U22"  Part="1"
-F 0 "U22" H 6100 2711 50  0000 C CNN
+AR Path="/6174477C/6577909E/65833EEB" Ref="U24"  Part="1"
+F 0 "U24" H 6100 2711 50  0000 C CNN
 F 1 "ATmega328PB-MU" H 6100 2620 50  0000 C CNN
 F 2 "Package_DFN_QFN:QFN-32-1EP_5x5mm_P0.5mm_EP3.1x3.1mm" H 6100 4300 50  0001 C CIN
@@
 AR Path="/6174477C/6572958C/65833DB6" Ref="C?"  Part="1"
 AR Path="/6174477C/6577909A/65833DB6" Ref="C?"  Part="1"
-AR Path="/6174477C/6577909E/65833DB6" Ref="C79"  Part="1"
-F 0 "C79" H 4442 2646 50  0000 L CNN
+AR Path="/6174477C/6577909E/65833DB6" Ref="C81"  Part="1"
+F 0 "C81" H 4442 2646 50  0000 L CNN
 F 1 "1uF" H 4442 2555 50  0000 L CNN
 F 2 "Capacitor_SMD:C_0603_1608Metric" H 4350 2600 50  0001 C CNN
@@
 AR Path="/6174477C/6572958C/63916676" Ref="C?"  Part="1"
 AR Path="/6174477C/6577909A/63916676" Ref="C?"  Part="1"
-AR Path="/6174477C/6577909E/63916676" Ref="C80"  Part="1"
-F 0 "C80" H 4792 2646 50  0000 L CNN
+AR Path="/6174477C/6577909E/63916676" Ref="C82"  Part="1"
+F 0 "C82" H 4792 2646 50  0000 L CNN
 F 1 "100nF" H 4792 2555 50  0000 L CNN
 F 2 "Capacitor_SMD:C_0402_1005Metric" H 4700 2600 50  0001 C CNN
@@
 AR Path="/6174477C/6572958C/65833DE7" Ref="#PWR?"  Part="1"
 AR Path="/6174477C/6577909A/65833DE7" Ref="#PWR?"  Part="1"
-AR Path="/6174477C/6577909E/65833DE7" Ref="#PWR0205"  Part="1"
-F 0 "#PWR0205" H 3500 2600 50  0001 C CNN
+AR Path="/6174477C/6577909E/65833DE7" Ref="#PWR0209"  Part="1"
+F 0 "#PWR0209" H 3500 2600 50  0001 C CNN
 F 1 "GND" H 3505 2677 50  0000 C CNN
 F 2 "" H 3500 2850 50  0001 C CNN
@@
 AR Path="/6174477C/6572958C/6386EE32" Ref="C?"  Part="1"
 AR Path="/6174477C/6577909A/6386EE32" Ref="C?"  Part="1"
-AR Path="/6174477C/6577909E/6386EE32" Ref="C82"  Part="1"
-F 0 "C82" H 8100 4600 50  0000 L CNN
+AR Path="/6174477C/6577909E/6386EE32" Ref="C84"  Part="1"
+F 0 "C84" H 8100 4600 50  0000 L CNN
 F 1 "22pF" H 8100 4500 50  0000 L CNN
 F 2 "Capacitor_SMD:C_0402_1005Metric" H 8400 4550 50  0001 C CNN
@@
 AR Path="/6174477C/6572958C/65833E93" Ref="C?"  Part="1"
 AR Path="/6174477C/6577909A/65833E93" Ref="C?"  Part="1"
-AR Path="/6174477C/6577909E/65833E93" Ref="C81"  Part="1"
-F 0 "C81" H 8100 4600 50  0000 L CNN
+AR Path="/6174477C/6577909E/65833E93" Ref="C83"  Part="1"
+F 0 "C83" H 8100 4600 50  0000 L CNN
 F 1 "22pF" H 8100 4500 50  0000 L CNN
 F 2 "Capacitor_SMD:C_0402_1005Metric" H 8000 4550 50  0001 C CNN
@@
 AR Path="/6174477C/6572958C/65833EA4" Ref="#PWR?"  Part="1"
 AR Path="/6174477C/6577909A/65833EA4" Ref="#PWR?"  Part="1"
-AR Path="/6174477C/6577909E/65833EA4" Ref="#PWR0213"  Part="1"
-F 0 "#PWR0213" H 8400 4450 50  0001 C CNN
+AR Path="/6174477C/6577909E/65833EA4" Ref="#PWR0217"  Part="1"
+F 0 "#PWR0217" H 8400 4450 50  0001 C CNN
 F 1 "GND" H 8405 4527 50  0000 C CNN
 F 2 "" H 8400 4700 50  0001 C CNN
@@
 AR Path="/6174477C/6572958C/65833EB4" Ref="#PWR?"  Part="1"
 AR Path="/6174477C/6577909A/65833EB4" Ref="#PWR?"  Part="1"
-AR Path="/6174477C/6577909E/65833EB4" Ref="#PWR0209"  Part="1"
-F 0 "#PWR0209" H 8000 4450 50  0001 C CNN
+AR Path="/6174477C/6577909E/65833EB4" Ref="#PWR0213"  Part="1"
+F 0 "#PWR0213" H 8000 4450 50  0001 C CNN
 F 1 "GND" H 8005 4527 50  0000 C CNN
 F 2 "" H 8000 4700 50  0001 C CNN
@@
 AR Path="/6174477C/6572958C/65833E05" Ref="#PWR?"  Part="1"
 AR Path="/6174477C/6577909A/65833E05" Ref="#PWR?"  Part="1"
-AR Path="/6174477C/6577909E/65833E05" Ref="#PWR0210"  Part="1"
-F 0 "#PWR0210" H 8200 3950 50  0001 C CNN
+AR Path="/6174477C/6577909E/65833E05" Ref="#PWR0214"  Part="1"
+F 0 "#PWR0214" H 8200 3950 50  0001 C CNN
 F 1 "GND" H 8205 4027 50  0000 C CNN
 F 2 "" H 8200 4200 50  0001 C CNN
@@
 AR Path="/6174477C/6572958C/65833E0F" Ref="#PWR?"  Part="1"
 AR Path="/6174477C/6577909A/65833E0F" Ref="#PWR?"  Part="1"
-AR Path="/6174477C/6577909E/65833E0F" Ref="#PWR0211"  Part="1"
-F 0 "#PWR0211" H 8200 4150 50  0001 C CNN
+AR Path="/6174477C/6577909E/65833E0F" Ref="#PWR0215"  Part="1"
+F 0 "#PWR0215" H 8200 4150 50  0001 C CNN
 F 1 "GND" H 8205 4227 50  0000 C CNN
 F 2 "" H 8200 4400 50  0001 C CNN
@@
 AR Path="/6174477C/6572958C/65833E1C" Ref="#PWR?"  Part="1"
 AR Path="/6174477C/6577909A/65833E1C" Ref="#PWR?"  Part="1"
-AR Path="/6174477C/6577909E/65833E1C" Ref="#PWR0204"  Part="1"
-F 0 "#PWR0204" H 3500 1650 50  0001 C CNN
+AR Path="/6174477C/6577909E/65833E1C" Ref="#PWR0208"  Part="1"
+F 0 "#PWR0208" H 3500 1650 50  0001 C CNN
 F 1 "+5V_A" H 3515 1973 50  0000 C CNN
 F 2 "" H 3500 1800 50  0001 C CNN
@@
 AR Path="/6174477C/6572958C/65833E2C" Ref="#PWR?"  Part="1"
 AR Path="/6174477C/6577909A/65833E2C" Ref="#PWR?"  Part="1"
-AR Path="/6174477C/6577909E/65833E2C" Ref="#PWR0207"  Part="1"
-F 0 "#PWR0207" H 4700 2600 50  0001 C CNN
+AR Path="/6174477C/6577909E/65833E2C" Ref="#PWR0211"  Part="1"
+F 0 "#PWR0211" H 4700 2600 50  0001 C CNN
 F 1 "GND" H 4705 2677 50  0000 C CNN
 F 2 "" H 4700 2850 50  0001 C CNN
@@
 AR Path="/6174477C/6572958C/65833E5F" Ref="#PWR?"  Part="1"
 AR Path="/6174477C/6577909A/65833E5F" Ref="#PWR?"  Part="1"
-AR Path="/6174477C/6577909E/65833E5F" Ref="#PWR0206"  Part="1"
-F 0 "#PWR0206" H 4200 5300 50  0001 C CNN
+AR Path="/6174477C/6577909E/65833E5F" Ref="#PWR0210"  Part="1"
+F 0 "#PWR0210" H 4200 5300 50  0001 C CNN
 F 1 "GND" H 4205 5377 50  0000 C CNN
 F 2 "" H 4200 5550 50  0001 C CNN
@@
 AR Path="/6174477C/6572958C/65833EEE" Ref="#PWR?"  Part="1"
 AR Path="/6174477C/6577909A/65833EEE" Ref="#PWR?"  Part="1"
-AR Path="/6174477C/6577909E/65833EEE" Ref="#PWR0212"  Part="1"
-F 0 "#PWR0212" H 8400 3100 50  0001 C CNN
+AR Path="/6174477C/6577909E/65833EEE" Ref="#PWR0216"  Part="1"
+F 0 "#PWR0216" H 8400 3100 50  0001 C CNN
 F 1 "GND" H 8405 3177 50  0000 C CNN
 F 2 "" H 8400 3350 50  0001 C CNN
@@
 AR Path="/6174477C/6572958C/65833DC7" Ref="#PWR?"  Part="1"
 AR Path="/6174477C/6577909A/65833DC7" Ref="#PWR?"  Part="1"
-AR Path="/6174477C/6577909E/65833DC7" Ref="#PWR0208"  Part="1"
-F 0 "#PWR0208" H 6100 5800 50  0001 C CNN
+AR Path="/6174477C/6577909E/65833DC7" Ref="#PWR0212"  Part="1"
+F 0 "#PWR0212" H 6100 5800 50  0001 C CNN
 F 1 "GND" H 6105 5877 50  0000 C CNN
 F 2 "" H 6100 6050 50  0001 C CNN
