File: ykts-payload/ykts-mcu-node12.sch (KiCad schematic (older format))
At the start: 12 parts

Commit message: Update nodes
Parts:
- D17: renamed from D?; value NODE0_STATUSLED -> NODE12_STATUSLED
- gave numbers to parts that had none: 11
Connections:
- net NODE0_PWR renamed NODE12_PWR
- net NODE0_RESET renamed NODE12_RESET
- net NODE0_RX renamed NODE12_RX
- net NODE0_TX renamed NODE12_TX
Other:
- note added: "MCU Node 12"
- note removed: "MCU Node 0"
Changed lines of the file:
@@
 AR Path="/6174477C/63801AEE/63916A79" Ref="U?"  Part="1"
 AR Path="/6174477C/638385B6/63916A79" Ref="U?"  Part="1"
-AR Path="/6174477C/638DF123/63916A79" Ref="U?"  Part="1"
-F 0 "U?" H 6100 2711 50  0000 C CNN
+AR Path="/6174477C/638DF123/63916A79" Ref="U25"  Part="1"
+F 0 "U25" H 6100 2711 50  0000 C CNN
 F 1 "ATmega328PB-MU" H 6100 2620 50  0000 C CNN
 F 2 "Package_DFN_QFN:QFN-32-1EP_5x5mm_P0.5mm_EP3.1x3.1mm" H 6100 4300 50  0001 C CIN
@@
 AR Path="/6174477C/63801AEE/6386EF30" Ref="SW?"  Part="1"
 AR Path="/6174477C/638385B6/6386EF30" Ref="SW?"  Part="1"
-AR Path="/6174477C/638DF123/6386EF30" Ref="SW?"  Part="1"
-F 0 "SW?" H 3500 2631 50  0000 C CNN
+AR Path="/6174477C/638DF123/6386EF30" Ref="SW12"  Part="1"
+F 0 "SW12" H 3500 2631 50  0000 C CNN
 F 1 "ADG802BRT" H 3500 2540 50  0000 C CNN
 F 2 "Package_TO_SOT_SMD:SOT-23-6" H 3500 2500 50  0001 C CNN
@@
 AR Path="/6174477C/63801AEE/6386EF31" Ref="C?"  Part="1"
 AR Path="/6174477C/638385B6/6386EF31" Ref="C?"  Part="1"
-AR Path="/6174477C/638DF123/6386EF31" Ref="C?"  Part="1"
-F 0 "C?" H 4292 2646 50  0000 L CNN
+AR Path="/6174477C/638DF123/6386EF31" Ref="C72"  Part="1"
+F 0 "C72" H 4292 2646 50  0000 L CNN
 F 1 "1uF" H 4292 2555 50  0000 L CNN
 F 2 "Capacitor_SMD:C_0603_1608Metric" H 4200 2600 50  0001 C CNN
@@
 AR Path="/6174477C/63801AEE/63916A75" Ref="C?"  Part="1"
 AR Path="/6174477C/638385B6/63916A75" Ref="C?"  Part="1"
-AR Path="/6174477C/638DF123/63916A75" Ref="C?"  Part="1"
-F 0 "C?" H 4642 2646 50  0000 L CNN
+AR Path="/6174477C/638DF123/63916A75" Ref="C73"  Part="1"
+F 0 "C73" H 4642 2646 50  0000 L CNN
 F 1 "100nF" H 4642 2555 50  0000 L CNN
 F 2 "Capacitor_SMD:C_0402_1005Metric" H 4550 2600 50  0001 C CNN
@@
 AR Path="/6174477C/63801AEE/6386EF33" Ref="#PWR?"  Part="1"
 AR Path="/6174477C/638385B6/6386EF33" Ref="#PWR?"  Part="1"
-AR Path="/6174477C/638DF123/6386EF33" Ref="#PWR?"  Part="1"
-F 0 "#PWR?" H 3500 2600 50  0001 C CNN
+AR Path="/6174477C/638DF123/6386EF33" Ref="#PWR0267"  Part="1"
+F 0 "#PWR0267" H 3500 2600 50  0001 C CNN
 F 1 "GND" H 3505 2677 50  0000 C CNN
 F 2 "" H 3500 2850 50  0001 C CNN
@@
 AR Path="/6174477C/63801AEE/6386EF34" Ref="C?"  Part="1"
 AR Path="/6174477C/638385B6/6386EF34" Ref="C?"  Part="1"
-AR Path="/6174477C/638DF123/6386EF34" Ref="C?"  Part="1"
-F 0 "C?" H 8100 4600 50  0000 L CNN
+AR Path="/6174477C/638DF123/6386EF34" Ref="C75"  Part="1"
+F 0 "C75" H 8100 4600 50  0000 L CNN
 F 1 "22pF" H 8100 4500 50  0000 L CNN
 F 2 "Capacitor_SMD:C_0402_1005Metric" H 8400 4550 50  0001 C CNN
@@
 AR Path="/6174477C/63801AEE/6386EF3A" Ref="C?"  Part="1"
 AR Path="/6174477C/638385B6/6386EF3A" Ref="C?"  Part="1"
-AR Path="/6174477C/638DF123/6386EF3A" Ref="C?"  Part="1"
-F 0 "C?" H 8100 4600 50  0000 L CNN
+AR Path="/6174477C/638DF123/6386EF3A" Ref="C74"  Part="1"
+F 0 "C74" H 8100 4600 50  0000 L CNN
 F 1 "22pF" H 8100 4500 50  0000 L CNN
 F 2 "Capacitor_SMD:C_0402_1005Metric" H 8000 4550 50  0001 C CNN
@@
 AR Path="/6174477C/63801AEE/6386EF3B" Ref="#PWR?"  Part="1"
 AR Path="/6174477C/638385B6/6386EF3B" Ref="#PWR?"  Part="1"
-AR Path="/6174477C/638DF123/6386EF3B" Ref="#PWR?"  Part="1"
-F 0 "#PWR?" H 8400 4450 50  0001 C CNN
+AR Path="/6174477C/638DF123/6386EF3B" Ref="#PWR0268"  Part="1"
+F 0 "#PWR0268" H 8400 4450 50  0001 C CNN
 F 1 "GND" H 8405 4527 50  0000 C CNN
 F 2 "" H 8400 4700 50  0001 C CNN
@@
 AR Path="/6174477C/63801AEE/6386EF3C" Ref="#PWR?"  Part="1"
 AR Path="/6174477C/638385B6/6386EF3C" Ref="#PWR?"  Part="1"
-AR Path="/6174477C/638DF123/6386EF3C" Ref="#PWR?"  Part="1"
-F 0 "#PWR?" H 8000 4450 50  0001 C CNN
+AR Path="/6174477C/638DF123/6386EF3C" Ref="#PWR0269"  Part="1"
+F 0 "#PWR0269" H 8000 4450 50  0001 C CNN
 F 1 "GND" H 8005 4527 50  0000 C CNN
 F 2 "" H 8000 4700 50  0001 C CNN
@@
 	8400 4700 8400 4650
 Text Label 7050 4600 0    50   ~ 0
-NODE0_RESET
+NODE12_RESET
 $Comp
 L Device:Crystal_GND24_Small Y?
@@
 AR Path="/6174477C/63801AEE/6386EF3D" Ref="Y?"  Part="1"
 AR Path="/6174477C/638385B6/6386EF3D" Ref="Y?"  Part="1"
-AR Path="/6174477C/638DF123/6386EF3D" Ref="Y?"  Part="1"
-F 0 "Y?" H 8450 4350 50  0000 L CNN
+AR Path="/6174477C/638DF123/6386EF3D" Ref="Y14"  Part="1"
+F 0 "Y14" H 8450 4350 50  0000 L CNN
 F 1 "8 MHz" H 8450 4250 50  0000 L CNN
 F 2 "Crystal:Crystal_SMD_2520-4Pin_2.5x2.0mm" H 8200 4300 50  0001 C CNN
@@
 AR Path="/6174477C/63801AEE/63760B1F" Ref="#PWR?"  Part="1"
 AR Path="/6174477C/638385B6/63760B1F" Ref="#PWR?"  Part="1"
-AR Path="/6174477C/638DF123/63760B1F" Ref="#PWR?"  Part="1"
-F 0 "#PWR?" H 8200 3950 50  0001 C CNN
+AR Path="/6174477C/638DF123/63760B1F" Ref="#PWR0270"  Part="1"
+F 0 "#PWR0270" H 8200 3950 50  0001 C CNN
 F 1 "GND" H 8205 4027 50  0000 C CNN
 F 2 "" H 8200 4200 50  0001 C CNN
@@
 AR Path="/6174477C/63801AEE/63760B25" Ref="#PWR?"  Part="1"
 AR Path="/6174477C/638385B6/63760B25" Ref="#PWR?"  Part="1"
-AR Path="/6174477C/638DF123/63760B25" Ref="#PWR?"  Part="1"
-F 0 "#PWR?" H 8200 4150 50  0001 C CNN
+AR Path="/6174477C/638DF123/63760B25" Ref="#PWR0271"  Part="1"
+F 0 "#PWR0271" H 8200 4150 50  0001 C CNN
 F 1 "GND" H 8205 4227 50  0000 C CNN
 F 2 "" H 8200 4400 50  0001 C CNN
@@
 AR Path="/6174477C/63801AEE/63916A8A" Ref="R?"  Part="1"
 AR Path="/6174477C/638385B6/63916A8A" Ref="R?"  Part="1"
-AR Path="/6174477C/638DF123/63916A8A" Ref="R?"  Part="1"
-F 0 "R?" V 6754 4400 50  0000 C CNN
+AR Path="/6174477C/638DF123/63916A8A" Ref="R92"  Part="1"
+F 0 "R92" V 6754 4400 50  0000 C CNN
 F 1 "20K" V 6845 4400 50  0000 C CNN
 F 2 "Resistor_SMD:R_0402_1005Metric" H 6950 4400 50  0001 C CNN
@@
 $EndComp
 Text GLabel 2700 2450 0    50   Input ~ 0
-NODE0_PWR
+NODE12_PWR
 Text GLabel 3900 3650 0    50   Input ~ 0
-NODE0_RESET
+NODE12_RESET
 Text GLabel 3900 3750 0    50   Input ~ 0
-NODE0_RX
+NODE12_RX
 Text GLabel 3900 3850 0    50   Input ~ 0
-NODE0_TX
+NODE12_TX
 $Comp
 L yktsat-common:+5V_A #PWR?
@@
 AR Path="/6174477C/63801AEE/6376D72E" Ref="#PWR?"  Part="1"
 AR Path="/6174477C/638385B6/6376D72E" Ref="#PWR?"  Part="1"
-AR Path="/6174477C/638DF123/6376D72E" Ref="#PWR?"  Part="1"
-F 0 "#PWR?" H 3500 1650 50  0001 C CNN
+AR Path="/6174477C/638DF123/6376D72E" Ref="#PWR0272"  Part="1"
+F 0 "#PWR0272" H 3500 1650 50  0001 C CNN
 F 1 "+5V_A" H 3515 1973 50  0000 C CNN
 F 2 "" H 3500 1800 50  0001 C CNN
@@
 AR Path="/6174477C/63801AEE/63916A7A" Ref="#PWR?"  Part="1"
 AR Path="/6174477C/638385B6/63916A7A" Ref="#PWR?"  Part="1"
-AR Path="/6174477C/638DF123/63916A7A" Ref="#PWR?"  Part="1"
-F 0 "#PWR?" H 4550 2600 50  0001 C CNN
+AR Path="/6174477C/638DF123/63916A7A" Ref="#PWR0273"  Part="1"
+F 0 "#PWR0273" H 4550 2600 50  0001 C CNN
 F 1 "GND" H 4555 2677 50  0000 C CNN
 F 2 "" H 4550 2850 50  0001 C CNN
@@
 AR Path="/6174477C/63801AEE/638383BE" Ref="R?"  Part="1"
 AR Path="/6174477C/638385B6/638383BE" Ref="R?"  Part="1"
-AR Path="/6174477C/638DF123/638383BE" Ref="R?"  Part="1"
-F 0 "R?" V 8004 3950 50  0000 C CNN
+AR Path="/6174477C/638DF123/638383BE" Ref="R93"  Part="1"
+F 0 "R93" V 8004 3950 50  0000 C CNN
 F 1 "1M" V 8095 3950 50  0000 C CNN
 F 2 "Resistor_SMD:R_0402_1005Metric" H 8200 3950 50  0001 C CNN
@@
 AR Path="/6174477C/63801AEE/638383BF" Ref="J?"  Part="1"
 AR Path="/6174477C/638385B6/638383BF" Ref="J?"  Part="1"
-AR Path="/6174477C/638DF123/638383BF" Ref="J?"  Part="1"
-F 0 "J?" H 3770 5146 50  0000 R CNN
+AR Path="/6174477C/638DF123/638383BF" Ref="J17"  Part="1"
+F 0 "J17" H 3770 5146 50  0000 R CNN
 F 1 "AVR-ISP-6" H 3770 5055 50  0000 R CNN
 F 2 "Connector_PinHeader_2.54mm:PinHeader_2x03_P2.54mm_Vertical" V 3850 5100 50  0001 C CNN
@@
 AR Path="/6174477C/63801AEE/638383C0" Ref="#PWR?"  Part="1"
 AR Path="/6174477C/638385B6/638383C0" Ref="#PWR?"  Part="1"
-AR Path="/6174477C/638DF123/638383C0" Ref="#PWR?"  Part="1"
-F 0 "#PWR?" H 4200 5300 50  0001 C CNN
+AR Path="/6174477C/638DF123/638383C0" Ref="#PWR0274"  Part="1"
+F 0 "#PWR0274" H 4200 5300 50  0001 C CNN
 F 1 "GND" H 4205 5377 50  0000 C CNN
 F 2 "" H 4200 5550 50  0001 C CNN
@@
 AR Path="/6174477C/63801AEE/638383C1" Ref="D?"  Part="1"
 AR Path="/6174477C/638385B6/638383C1" Ref="D?"  Part="1"
-AR Path="/6174477C/638DF123/638383C1" Ref="D?"  Part="1"
-F 0 "D?" V 8439 2682 50  0000 R CNN
-F 1 "NODE0_STATUSLED" V 8348 2682 50  0000 R CNN
+AR Path="/6174477C/638DF123/638383C1" Ref="D17"  Part="1"
+F 0 "D17" V 8439 2682 50  0000 R CNN
+F 1 "NODE12_STATUSLED" V 8348 2682 50  0000 R CNN
 F 2 "LED_SMD:LED_0402_1005Metric" H 8400 2800 50  0001 C CNN
 F 3 "~" H 8400 2800 50  0001 C CNN
@@
 AR Path="/6174477C/63801AEE/638383C2" Ref="R?"  Part="1"
 AR Path="/6174477C/638385B6/638383C2" Ref="R?"  Part="1"
-AR Path="/6174477C/638DF123/638383C2" Ref="R?"  Part="1"
-F 0 "R?" V 8204 3150 50  0000 C CNN
+AR Path="/6174477C/638DF123/638383C2" Ref="R94"  Part="1"
+F 0 "R94" V 8204 3150 50  0000 C CNN
 F 1 "1K" V 8295 3150 50  0000 C CNN
 F 2 "Resistor_SMD:R_0402_1005Metric" H 8400 3150 50  0001 C CNN
@@
 AR Path="/6174477C/63801AEE/63916A80" Ref="#PWR?"  Part="1"
 AR Path="/6174477C/638385B6/63916A80" Ref="#PWR?"  Part="1"
-AR Path="/6174477C/638DF123/63916A80" Ref="#PWR?"  Part="1"
-F 0 "#PWR?" H 8400 3100 50  0001 C CNN
+AR Path="/6174477C/638DF123/63916A80" Ref="#PWR0275"  Part="1"
+F 0 "#PWR0275" H 8400 3100 50  0001 C CNN
 F 1 "GND" H 8405 3177 50  0000 C CNN
 F 2 "" H 8400 3350 50  0001 C CNN
@@
 AR Path="/6174477C/63801AEE/6386EF38" Ref="#PWR?"  Part="1"
 AR Path="/6174477C/638385B6/6386EF38" Ref="#PWR?"  Part="1"
-AR Path="/6174477C/638DF123/6386EF38" Ref="#PWR?"  Part="1"
-F 0 "#PWR?" H 6100 5800 50  0001 C CNN
+AR Path="/6174477C/638DF123/6386EF38" Ref="#PWR0276"  Part="1"
+F 0 "#PWR0276" H 6100 5800 50  0001 C CNN
 F 1 "GND" H 6105 5877 50  0000 C CNN
 F 2 "" H 6100 6050 50  0001 C CNN
@@
 	4200 3750 3900 3750
 Text Label 4200 3650 0    50   ~ 0
-NODE0_RESET
+NODE12_RESET
 Wire Wire Line
 	4200 3650 3900 3650
 Text Notes 5700 950  0    100  ~ 0
-MCU Node 0
+MCU Node 12
 Wire Wire Line
 	2700 2450 3100 2450
@@
 ISP_RESET
 Text Label 4200 3550 0    50   ~ 0
-NODE0_RESET
+NODE12_RESET
 Wire Wire Line
 	4200 3550 3900 3550
