File: ykts-payload/ykts-mcu-node12.sch (KiCad schematic (older format))
At the start: 12 parts, among them J25 AVR-ISP-6, SW13 ADG802BRT, U24 ATmega328PB-MU, Y17 8 MHz

Commit message: Revision B2
Hierarchal sheets for nodes
Partial PCB layout
Parts:
- renumbered C87 to C89, C88 to C90, C89 to C91, C90 to C92, U24 to U26
Changed lines of the file:
@@
 Sheet 15 18
 Title "YktSat Payload Module"
-Date "2021-10-22"
-Rev "B0"
+Date "2021-10-26"
+Rev "B1"
 Comp "Sakha Aerospace Systems, LLC"
 Comment1 ""
@@
 AR Path="/6174477C/6572958C/65833EDF" Ref="U?"  Part="1"
 AR Path="/6174477C/6577909A/65833EDF" Ref="U?"  Part="1"
-AR Path="/6174477C/657790A2/65833EDF" Ref="U24"  Part="1"
-F 0 "U24" H 6100 2711 50  0000 C CNN
+AR Path="/6174477C/657790A2/65833EDF" Ref="U26"  Part="1"
+F 0 "U26" H 6100 2711 50  0000 C CNN
 F 1 "ATmega328PB-MU" H 6100 2620 50  0000 C CNN
 F 2 "Package_DFN_QFN:QFN-32-1EP_5x5mm_P0.5mm_EP3.1x3.1mm" H 6100 4300 50  0001 C CIN
@@
 AR Path="/6174477C/6572958C/65833DBA" Ref="C?"  Part="1"
 AR Path="/6174477C/6577909A/65833DBA" Ref="C?"  Part="1"
-AR Path="/6174477C/657790A2/65833DBA" Ref="C87"  Part="1"
-F 0 "C87" H 4442 2646 50  0000 L CNN
+AR Path="/6174477C/657790A2/65833DBA" Ref="C89"  Part="1"
+F 0 "C89" H 4442 2646 50  0000 L CNN
 F 1 "1uF" H 4442 2555 50  0000 L CNN
 F 2 "Capacitor_SMD:C_0603_1608Metric" H 4350 2600 50  0001 C CNN
@@
 AR Path="/6174477C/6572958C/65833ED5" Ref="C?"  Part="1"
 AR Path="/6174477C/6577909A/65833ED5" Ref="C?"  Part="1"
-AR Path="/6174477C/657790A2/65833ED5" Ref="C88"  Part="1"
-F 0 "C88" H 4792 2646 50  0000 L CNN
+AR Path="/6174477C/657790A2/65833ED5" Ref="C90"  Part="1"
+F 0 "C90" H 4792 2646 50  0000 L CNN
 F 1 "100nF" H 4792 2555 50  0000 L CNN
 F 2 "Capacitor_SMD:C_0402_1005Metric" H 4700 2600 50  0001 C CNN
@@
 AR Path="/6174477C/6572958C/65833DED" Ref="#PWR?"  Part="1"
 AR Path="/6174477C/6577909A/65833DED" Ref="#PWR?"  Part="1"
-AR Path="/6174477C/657790A2/65833DED" Ref="#PWR0225"  Part="1"
-F 0 "#PWR0225" H 3500 2600 50  0001 C CNN
+AR Path="/6174477C/657790A2/65833DED" Ref="#PWR0229"  Part="1"
+F 0 "#PWR0229" H 3500 2600 50  0001 C CNN
 F 1 "GND" H 3505 2677 50  0000 C CNN
 F 2 "" H 3500 2850 50  0001 C CNN
@@
 AR Path="/6174477C/6572958C/65833DF7" Ref="C?"  Part="1"
 AR Path="/6174477C/6577909A/65833DF7" Ref="C?"  Part="1"
-AR Path="/6174477C/657790A2/65833DF7" Ref="C90"  Part="1"
-F 0 "C90" H 8100 4600 50  0000 L CNN
+AR Path="/6174477C/657790A2/65833DF7" Ref="C92"  Part="1"
+F 0 "C92" H 8100 4600 50  0000 L CNN
 F 1 "22pF" H 8100 4500 50  0000 L CNN
 F 2 "Capacitor_SMD:C_0402_1005Metric" H 8400 4550 50  0001 C CNN
@@
 AR Path="/6174477C/6572958C/65833E9F" Ref="C?"  Part="1"
 AR Path="/6174477C/6577909A/65833E9F" Ref="C?"  Part="1"
-AR Path="/6174477C/657790A2/65833E9F" Ref="C89"  Part="1"
-F 0 "C89" H 8100 4600 50  0000 L CNN
+AR Path="/6174477C/657790A2/65833E9F" Ref="C91"  Part="1"
+F 0 "C91" H 8100 4600 50  0000 L CNN
 F 1 "22pF" H 8100 4500 50  0000 L CNN
 F 2 "Capacitor_SMD:C_0402_1005Metric" H 8000 4550 50  0001 C CNN
@@
 AR Path="/6174477C/6572958C/65833EA3" Ref="#PWR?"  Part="1"
 AR Path="/6174477C/6577909A/65833EA3" Ref="#PWR?"  Part="1"
-AR Path="/6174477C/657790A2/65833EA3" Ref="#PWR0233"  Part="1"
-F 0 "#PWR0233" H 8400 4450 50  0001 C CNN
+AR Path="/6174477C/657790A2/65833EA3" Ref="#PWR0237"  Part="1"
+F 0 "#PWR0237" H 8400 4450 50  0001 C CNN
 F 1 "GND" H 8405 4527 50  0000 C CNN
 F 2 "" H 8400 4700 50  0001 C CNN
@@
 AR Path="/6174477C/6572958C/65833EB9" Ref="#PWR?"  Part="1"
 AR Path="/6174477C/6577909A/65833EB9" Ref="#PWR?"  Part="1"
-AR Path="/6174477C/657790A2/65833EB9" Ref="#PWR0229"  Part="1"
-F 0 "#PWR0229" H 8000 4450 50  0001 C CNN
+AR Path="/6174477C/657790A2/65833EB9" Ref="#PWR0233"  Part="1"
+F 0 "#PWR0233" H 8000 4450 50  0001 C CNN
 F 1 "GND" H 8005 4527 50  0000 C CNN
 F 2 "" H 8000 4700 50  0001 C CNN
@@
 AR Path="/6174477C/6572958C/65833E00" Ref="#PWR?"  Part="1"
 AR Path="/6174477C/6577909A/65833E00" Ref="#PWR?"  Part="1"
-AR Path="/6174477C/657790A2/65833E00" Ref="#PWR0230"  Part="1"
-F 0 "#PWR0230" H 8200 3950 50  0001 C CNN
+AR Path="/6174477C/657790A2/65833E00" Ref="#PWR0234"  Part="1"
+F 0 "#PWR0234" H 8200 3950 50  0001 C CNN
 F 1 "GND" H 8205 4027 50  0000 C CNN
 F 2 "" H 8200 4200 50  0001 C CNN
@@
 AR Path="/6174477C/6572958C/65833E15" Ref="#PWR?"  Part="1"
 AR Path="/6174477C/6577909A/65833E15" Ref="#PWR?"  Part="1"
-AR Path="/6174477C/657790A2/65833E15" Ref="#PWR0231"  Part="1"
-F 0 "#PWR0231" H 8200 4150 50  0001 C CNN
+AR Path="/6174477C/657790A2/65833E15" Ref="#PWR0235"  Part="1"
+F 0 "#PWR0235" H 8200 4150 50  0001 C CNN
 F 1 "GND" H 8205 4227 50  0000 C CNN
 F 2 "" H 8200 4400 50  0001 C CNN
@@
 AR Path="/6174477C/6572958C/65833E23" Ref="#PWR?"  Part="1"
 AR Path="/6174477C/6577909A/65833E23" Ref="#PWR?"  Part="1"
-AR Path="/6174477C/657790A2/65833E23" Ref="#PWR0224"  Part="1"
-F 0 "#PWR0224" H 3500 1650 50  0001 C CNN
+AR Path="/6174477C/657790A2/65833E23" Ref="#PWR0228"  Part="1"
+F 0 "#PWR0228" H 3500 1650 50  0001 C CNN
 F 1 "+5V_A" H 3515 1973 50  0000 C CNN
 F 2 "" H 3500 1800 50  0001 C CNN
@@
 AR Path="/6174477C/6572958C/65833E34" Ref="#PWR?"  Part="1"
 AR Path="/6174477C/6577909A/65833E34" Ref="#PWR?"  Part="1"
-AR Path="/6174477C/657790A2/65833E34" Ref="#PWR0227"  Part="1"
-F 0 "#PWR0227" H 4700 2600 50  0001 C CNN
+AR Path="/6174477C/657790A2/65833E34" Ref="#PWR0231"  Part="1"
+F 0 "#PWR0231" H 4700 2600 50  0001 C CNN
 F 1 "GND" H 4705 2677 50  0000 C CNN
 F 2 "" H 4700 2850 50  0001 C CNN
@@
 AR Path="/6174477C/6572958C/65833E57" Ref="#PWR?"  Part="1"
 AR Path="/6174477C/6577909A/65833E57" Ref="#PWR?"  Part="1"
-AR Path="/6174477C/657790A2/65833E57" Ref="#PWR0226"  Part="1"
-F 0 "#PWR0226" H 4200 5300 50  0001 C CNN
+AR Path="/6174477C/657790A2/65833E57" Ref="#PWR0230"  Part="1"
+F 0 "#PWR0230" H 4200 5300 50  0001 C CNN
 F 1 "GND" H 4205 5377 50  0000 C CNN
 F 2 "" H 4200 5550 50  0001 C CNN
@@
 AR Path="/6174477C/6572958C/65833EF5" Ref="#PWR?"  Part="1"
 AR Path="/6174477C/6577909A/65833EF5" Ref="#PWR?"  Part="1"
-AR Path="/6174477C/657790A2/65833EF5" Ref="#PWR0232"  Part="1"
-F 0 "#PWR0232" H 8400 3100 50  0001 C CNN
+AR Path="/6174477C/657790A2/65833EF5" Ref="#PWR0236"  Part="1"
+F 0 "#PWR0236" H 8400 3100 50  0001 C CNN
 F 1 "GND" H 8405 3177 50  0000 C CNN
 F 2 "" H 8400 3350 50  0001 C CNN
@@
 AR Path="/6174477C/6572958C/65833DC1" Ref="#PWR?"  Part="1"
 AR Path="/6174477C/6577909A/65833DC1" Ref="#PWR?"  Part="1"
-AR Path="/6174477C/657790A2/65833DC1" Ref="#PWR0228"  Part="1"
-F 0 "#PWR0228" H 6100 5800 50  0001 C CNN
+AR Path="/6174477C/657790A2/65833DC1" Ref="#PWR0232"  Part="1"
+F 0 "#PWR0232" H 6100 5800 50  0001 C CNN
 F 1 "GND" H 6105 5877 50  0000 C CNN
 F 2 "" H 6100 6050 50  0001 C CNN
