File: ykts-payload/ykts-mcu-node14.sch (KiCad schematic (older format))
At the start: 12 parts

Commit message: Update nodes
Parts:
- D19: renamed from D?; value NODE0_STATUSLED -> NODE14_STATUSLED
- gave numbers to parts that had none: 11
Connections:
- net NODE0_PWR renamed NODE14_PWR
- net NODE0_RESET renamed NODE14_RESET
- net NODE0_RX renamed NODE14_RX
- net NODE0_TX renamed NODE14_TX
Other:
- note added: "MCU Node 14"
- note removed: "MCU Node 0"
Changed lines of the file:
@@
 AR Path="/6174477C/638385B8/63916C85" Ref="U?"  Part="1"
 AR Path="/6174477C/638385BA/63916C85" Ref="U?"  Part="1"
-AR Path="/6174477C/638DF127/63916C85" Ref="U?"  Part="1"
-F 0 "U?" H 6100 2711 50  0000 C CNN
+AR Path="/6174477C/638DF127/63916C85" Ref="U27"  Part="1"
+F 0 "U27" H 6100 2711 50  0000 C CNN
 F 1 "ATmega328PB-MU" H 6100 2620 50  0000 C CNN
 F 2 "Package_DFN_QFN:QFN-32-1EP_5x5mm_P0.5mm_EP3.1x3.1mm" H 6100 4300 50  0001 C CIN
@@
 AR Path="/6174477C/638385B8/6386F13B" Ref="SW?"  Part="1"
 AR Path="/6174477C/638385BA/6386F13B" Ref="SW?"  Part="1"
-AR Path="/6174477C/638DF127/6386F13B" Ref="SW?"  Part="1"
-F 0 "SW?" H 3500 2631 50  0000 C CNN
+AR Path="/6174477C/638DF127/6386F13B" Ref="SW14"  Part="1"
+F 0 "SW14" H 3500 2631 50  0000 C CNN
 F 1 "ADG802BRT" H 3500 2540 50  0000 C CNN
 F 2 "Package_TO_SOT_SMD:SOT-23-6" H 3500 2500 50  0001 C CNN
@@
 AR Path="/6174477C/638385B8/63916C7C" Ref="C?"  Part="1"
 AR Path="/6174477C/638385BA/63916C7C" Ref="C?"  Part="1"
-AR Path="/6174477C/638DF127/63916C7C" Ref="C?"  Part="1"
-F 0 "C?" H 4292 2646 50  0000 L CNN
+AR Path="/6174477C/638DF127/63916C7C" Ref="C80"  Part="1"
+F 0 "C80" H 4292 2646 50  0000 L CNN
 F 1 "1uF" H 4292 2555 50  0000 L CNN
 F 2 "Capacitor_SMD:C_0603_1608Metric" H 4200 2600 50  0001 C CNN
@@
 AR Path="/6174477C/638385B8/638383B2" Ref="C?"  Part="1"
 AR Path="/6174477C/638385BA/638383B2" Ref="C?"  Part="1"
-AR Path="/6174477C/638DF127/638383B2" Ref="C?"  Part="1"
-F 0 "C?" H 4642 2646 50  0000 L CNN
+AR Path="/6174477C/638DF127/638383B2" Ref="C81"  Part="1"
+F 0 "C81" H 4642 2646 50  0000 L CNN
 F 1 "100nF" H 4642 2555 50  0000 L CNN
 F 2 "Capacitor_SMD:C_0402_1005Metric" H 4550 2600 50  0001 C CNN
@@
 AR Path="/6174477C/638385B8/63916C7E" Ref="#PWR?"  Part="1"
 AR Path="/6174477C/638385BA/63916C7E" Ref="#PWR?"  Part="1"
-AR Path="/6174477C/638DF127/63916C7E" Ref="#PWR?"  Part="1"
-F 0 "#PWR?" H 3500 2600 50  0001 C CNN
+AR Path="/6174477C/638DF127/63916C7E" Ref="#PWR0287"  Part="1"
+F 0 "#PWR0287" H 3500 2600 50  0001 C CNN
 F 1 "GND" H 3505 2677 50  0000 C CNN
 F 2 "" H 3500 2850 50  0001 C CNN
@@
 AR Path="/6174477C/638385B8/638383B4" Ref="C?"  Part="1"
 AR Path="/6174477C/638385BA/638383B4" Ref="C?"  Part="1"
-AR Path="/6174477C/638DF127/638383B4" Ref="C?"  Part="1"
-F 0 "C?" H 8100 4600 50  0000 L CNN
+AR Path="/6174477C/638DF127/638383B4" Ref="C83"  Part="1"
+F 0 "C83" H 8100 4600 50  0000 L CNN
 F 1 "22pF" H 8100 4500 50  0000 L CNN
 F 2 "Capacitor_SMD:C_0402_1005Metric" H 8400 4550 50  0001 C CNN
@@
 AR Path="/6174477C/638385B8/63916C80" Ref="C?"  Part="1"
 AR Path="/6174477C/638385BA/63916C80" Ref="C?"  Part="1"
-AR Path="/6174477C/638DF127/63916C80" Ref="C?"  Part="1"
-F 0 "C?" H 8100 4600 50  0000 L CNN
+AR Path="/6174477C/638DF127/63916C80" Ref="C82"  Part="1"
+F 0 "C82" H 8100 4600 50  0000 L CNN
 F 1 "22pF" H 8100 4500 50  0000 L CNN
 F 2 "Capacitor_SMD:C_0402_1005Metric" H 8000 4550 50  0001 C CNN
@@
 AR Path="/6174477C/638385B8/6386EE34" Ref="#PWR?"  Part="1"
 AR Path="/6174477C/638385BA/6386EE34" Ref="#PWR?"  Part="1"
-AR Path="/6174477C/638DF127/6386EE34" Ref="#PWR?"  Part="1"
-F 0 "#PWR?" H 8400 4450 50  0001 C CNN
+AR Path="/6174477C/638DF127/6386EE34" Ref="#PWR0288"  Part="1"
+F 0 "#PWR0288" H 8400 4450 50  0001 C CNN
 F 1 "GND" H 8405 4527 50  0000 C CNN
 F 2 "" H 8400 4700 50  0001 C CNN
@@
 AR Path="/6174477C/638385B8/63916C82" Ref="#PWR?"  Part="1"
 AR Path="/6174477C/638385BA/63916C82" Ref="#PWR?"  Part="1"
-AR Path="/6174477C/638DF127/63916C82" Ref="#PWR?"  Part="1"
-F 0 "#PWR?" H 8000 4450 50  0001 C CNN
+AR Path="/6174477C/638DF127/63916C82" Ref="#PWR0289"  Part="1"
+F 0 "#PWR0289" H 8000 4450 50  0001 C CNN
 F 1 "GND" H 8005 4527 50  0000 C CNN
 F 2 "" H 8000 4700 50  0001 C CNN
@@
 	8400 4700 8400 4650
 Text Label 7050 4600 0    50   ~ 0
-NODE0_RESET
+NODE14_RESET
 $Comp
 L Device:Crystal_GND24_Small Y?
@@
 AR Path="/6174477C/638385B8/63760B19" Ref="Y?"  Part="1"
 AR Path="/6174477C/638385BA/63760B19" Ref="Y?"  Part="1"
-AR Path="/6174477C/638DF127/63760B19" Ref="Y?"  Part="1"
-F 0 "Y?" H 8450 4350 50  0000 L CNN
+AR Path="/6174477C/638DF127/63760B19" Ref="Y16"  Part="1"
+F 0 "Y16" H 8450 4350 50  0000 L CNN
 F 1 "8 MHz" H 8450 4250 50  0000 L CNN
 F 2 "Crystal:Crystal_SMD_2520-4Pin_2.5x2.0mm" H 8200 4300 50  0001 C CNN
@@
 AR Path="/6174477C/638385B8/63916C8A" Ref="#PWR?"  Part="1"
 AR Path="/6174477C/638385BA/63916C8A" Ref="#PWR?"  Part="1"
-AR Path="/6174477C/638DF127/63916C8A" Ref="#PWR?"  Part="1"
-F 0 "#PWR?" H 8200 3950 50  0001 C CNN
+AR Path="/6174477C/638DF127/63916C8A" Ref="#PWR0290"  Part="1"
+F 0 "#PWR0290" H 8200 3950 50  0001 C CNN
 F 1 "GND" H 8205 4027 50  0000 C CNN
 F 2 "" H 8200 4200 50  0001 C CNN
@@
 AR Path="/6174477C/638385B8/6386F141" Ref="#PWR?"  Part="1"
 AR Path="/6174477C/638385BA/6386F141" Ref="#PWR?"  Part="1"
-AR Path="/6174477C/638DF127/6386F141" Ref="#PWR?"  Part="1"
-F 0 "#PWR?" H 8200 4150 50  0001 C CNN
+AR Path="/6174477C/638DF127/6386F141" Ref="#PWR0291"  Part="1"
+F 0 "#PWR0291" H 8200 4150 50  0001 C CNN
 F 1 "GND" H 8205 4227 50  0000 C CNN
 F 2 "" H 8200 4400 50  0001 C CNN
@@
 AR Path="/6174477C/638385B8/6386F147" Ref="R?"  Part="1"
 AR Path="/6174477C/638385BA/6386F147" Ref="R?"  Part="1"
-AR Path="/6174477C/638DF127/6386F147" Ref="R?"  Part="1"
-F 0 "R?" V 6754 4400 50  0000 C CNN
+AR Path="/6174477C/638DF127/6386F147" Ref="R98"  Part="1"
+F 0 "R98" V 6754 4400 50  0000 C CNN
 F 1 "20K" V 6845 4400 50  0000 C CNN
 F 2 "Resistor_SMD:R_0402_1005Metric" H 6950 4400 50  0001 C CNN
@@
 $EndComp
 Text GLabel 2700 2450 0    50   Input ~ 0
-NODE0_PWR
+NODE14_PWR
 Text GLabel 3900 3650 0    50   Input ~ 0
-NODE0_RESET
+NODE14_RESET
 Text GLabel 3900 3750 0    50   Input ~ 0
-NODE0_RX
+NODE14_RX
 Text GLabel 3900 3850 0    50   Input ~ 0
-NODE0_TX
+NODE14_TX
 $Comp
 L yktsat-common:+5V_A #PWR?
@@
 AR Path="/6174477C/638385B8/6386F142" Ref="#PWR?"  Part="1"
 AR Path="/6174477C/638385BA/6386F142" Ref="#PWR?"  Part="1"
-AR Path="/6174477C/638DF127/6386F142" Ref="#PWR?"  Part="1"
-F 0 "#PWR?" H 3500 1650 50  0001 C CNN
+AR Path="/6174477C/638DF127/6386F142" Ref="#PWR0292"  Part="1"
+F 0 "#PWR0292" H 3500 1650 50  0001 C CNN
 F 1 "+5V_A" H 3515 1973 50  0000 C CNN
 F 2 "" H 3500 1800 50  0001 C CNN
@@
 AR Path="/6174477C/638385B8/6386F148" Ref="#PWR?"  Part="1"
 AR Path="/6174477C/638385BA/6386F148" Ref="#PWR?"  Part="1"
-AR Path="/6174477C/638DF127/6386F148" Ref="#PWR?"  Part="1"
-F 0 "#PWR?" H 4550 2600 50  0001 C CNN
+AR Path="/6174477C/638DF127/6386F148" Ref="#PWR0293"  Part="1"
+F 0 "#PWR0293" H 4550 2600 50  0001 C CNN
 F 1 "GND" H 4555 2677 50  0000 C CNN
 F 2 "" H 4550 2850 50  0001 C CNN
@@
 AR Path="/6174477C/638385B8/63916C86" Ref="R?"  Part="1"
 AR Path="/6174477C/638385BA/63916C86" Ref="R?"  Part="1"
-AR Path="/6174477C/638DF127/63916C86" Ref="R?"  Part="1"
-F 0 "R?" V 8004 3950 50  0000 C CNN
+AR Path="/6174477C/638DF127/63916C86" Ref="R99"  Part="1"
+F 0 "R99" V 8004 3950 50  0000 C CNN
 F 1 "1M" V 8095 3950 50  0000 C CNN
 F 2 "Resistor_SMD:R_0402_1005Metric" H 8200 3950 50  0001 C CNN
@@
 AR Path="/6174477C/638385B8/63916C87" Ref="J?"  Part="1"
 AR Path="/6174477C/638385BA/63916C87" Ref="J?"  Part="1"
-AR Path="/6174477C/638DF127/63916C87" Ref="J?"  Part="1"
-F 0 "J?" H 3770 5146 50  0000 R CNN
+AR Path="/6174477C/638DF127/63916C87" Ref="J19"  Part="1"
+F 0 "J19" H 3770 5146 50  0000 R CNN
 F 1 "AVR-ISP-6" H 3770 5055 50  0000 R CNN
 F 2 "Connector_PinHeader_2.54mm:PinHeader_2x03_P2.54mm_Vertical" V 3850 5100 50  0001 C CNN
@@
 AR Path="/6174477C/638385B8/63916C88" Ref="#PWR?"  Part="1"
 AR Path="/6174477C/638385BA/63916C88" Ref="#PWR?"  Part="1"
-AR Path="/6174477C/638DF127/63916C88" Ref="#PWR?"  Part="1"
-F 0 "#PWR?" H 4200 5300 50  0001 C CNN
+AR Path="/6174477C/638DF127/63916C88" Ref="#PWR0294"  Part="1"
+F 0 "#PWR0294" H 4200 5300 50  0001 C CNN
 F 1 "GND" H 4205 5377 50  0000 C CNN
 F 2 "" H 4200 5550 50  0001 C CNN
@@
 AR Path="/6174477C/638385B8/63916C90" Ref="D?"  Part="1"
 AR Path="/6174477C/638385BA/63916C90" Ref="D?"  Part="1"
-AR Path="/6174477C/638DF127/63916C90" Ref="D?"  Part="1"
-F 0 "D?" V 8439 2682 50  0000 R CNN
-F 1 "NODE0_STATUSLED" V 8348 2682 50  0000 R CNN
+AR Path="/6174477C/638DF127/63916C90" Ref="D19"  Part="1"
+F 0 "D19" V 8439 2682 50  0000 R CNN
+F 1 "NODE14_STATUSLED" V 8348 2682 50  0000 R CNN
 F 2 "LED_SMD:LED_0402_1005Metric" H 8400 2800 50  0001 C CNN
 F 3 "~" H 8400 2800 50  0001 C CNN
@@
 AR Path="/6174477C/638385B8/6386EE40" Ref="R?"  Part="1"
 AR Path="/6174477C/638385BA/6386EE40" Ref="R?"  Part="1"
-AR Path="/6174477C/638DF127/6386EE40" Ref="R?"  Part="1"
-F 0 "R?" V 8204 3150 50  0000 C CNN
+AR Path="/6174477C/638DF127/6386EE40" Ref="R100"  Part="1"
+F 0 "R100" V 8204 3150 50  0000 C CNN
 F 1 "1K" V 8295 3150 50  0000 C CNN
 F 2 "Resistor_SMD:R_0402_1005Metric" H 8400 3150 50  0001 C CNN
@@
 AR Path="/6174477C/638385B8/63916C84" Ref="#PWR?"  Part="1"
 AR Path="/6174477C/638385BA/63916C84" Ref="#PWR?"  Part="1"
-AR Path="/6174477C/638DF127/63916C84" Ref="#PWR?"  Part="1"
-F 0 "#PWR?" H 8400 3100 50  0001 C CNN
+AR Path="/6174477C/638DF127/63916C84" Ref="#PWR0295"  Part="1"
+F 0 "#PWR0295" H 8400 3100 50  0001 C CNN
 F 1 "GND" H 8405 3177 50  0000 C CNN
 F 2 "" H 8400 3350 50  0001 C CNN
@@
 AR Path="/6174477C/638385B8/63916C8D" Ref="#PWR?"  Part="1"
 AR Path="/6174477C/638385BA/63916C8D" Ref="#PWR?"  Part="1"
-AR Path="/6174477C/638DF127/63916C8D" Ref="#PWR?"  Part="1"
-F 0 "#PWR?" H 6100 5800 50  0001 C CNN
+AR Path="/6174477C/638DF127/63916C8D" Ref="#PWR0296"  Part="1"
+F 0 "#PWR0296" H 6100 5800 50  0001 C CNN
 F 1 "GND" H 6105 5877 50  0000 C CNN
 F 2 "" H 6100 6050 50  0001 C CNN
@@
 	4200 3750 3900 3750
 Text Label 4200 3650 0    50   ~ 0
-NODE0_RESET
+NODE14_RESET
 Wire Wire Line
 	4200 3650 3900 3650
 Text Notes 5700 950  0    100  ~ 0
-MCU Node 0
+MCU Node 14
 Wire Wire Line
 	2700 2450 3100 2450
@@
 ISP_RESET
 Text Label 4200 3550 0    50   ~ 0
-NODE0_RESET
+NODE14_RESET
 Wire Wire Line
 	4200 3550 3900 3550
