File: ykts-payload/ykts-mcu-node14.sch (KiCad schematic (older format))
At the start: 12 parts, among them J27 AVR-ISP-6, SW15 ADG802BRT, U26 ATmega328PB-MU, Y19 8 MHz

Commit message: Revision B2
Hierarchal sheets for nodes
Partial PCB layout
Parts:
- renumbered C98 to C100, C95 to C97, C96 to C98, C97 to C99, U26 to U28
Changed lines of the file:
@@
 Sheet 17 18
 Title "YktSat Payload Module"
-Date "2021-10-22"
-Rev "B0"
+Date "2021-10-26"
+Rev "B1"
 Comp "Sakha Aerospace Systems, LLC"
 Comment1 ""
@@
 AR Path="/6174477C/6572958C/65833EE2" Ref="U?"  Part="1"
 AR Path="/6174477C/6577909A/65833EE2" Ref="U?"  Part="1"
-AR Path="/6174477C/657790A6/65833EE2" Ref="U26"  Part="1"
-F 0 "U26" H 6100 2711 50  0000 C CNN
+AR Path="/6174477C/657790A6/65833EE2" Ref="U28"  Part="1"
+F 0 "U28" H 6100 2711 50  0000 C CNN
 F 1 "ATmega328PB-MU" H 6100 2620 50  0000 C CNN
 F 2 "Package_DFN_QFN:QFN-32-1EP_5x5mm_P0.5mm_EP3.1x3.1mm" H 6100 4300 50  0001 C CIN
@@
 AR Path="/6174477C/6572958C/6375CEE6" Ref="C?"  Part="1"
 AR Path="/6174477C/6577909A/6375CEE6" Ref="C?"  Part="1"
-AR Path="/6174477C/657790A6/6375CEE6" Ref="C95"  Part="1"
-F 0 "C95" H 4442 2646 50  0000 L CNN
+AR Path="/6174477C/657790A6/6375CEE6" Ref="C97"  Part="1"
+F 0 "C97" H 4442 2646 50  0000 L CNN
 F 1 "1uF" H 4442 2555 50  0000 L CNN
 F 2 "Capacitor_SMD:C_0603_1608Metric" H 4350 2600 50  0001 C CNN
@@
 AR Path="/6174477C/6572958C/65833ECF" Ref="C?"  Part="1"
 AR Path="/6174477C/6577909A/65833ECF" Ref="C?"  Part="1"
-AR Path="/6174477C/657790A6/65833ECF" Ref="C96"  Part="1"
-F 0 "C96" H 4792 2646 50  0000 L CNN
+AR Path="/6174477C/657790A6/65833ECF" Ref="C98"  Part="1"
+F 0 "C98" H 4792 2646 50  0000 L CNN
 F 1 "100nF" H 4792 2555 50  0000 L CNN
 F 2 "Capacitor_SMD:C_0402_1005Metric" H 4700 2600 50  0001 C CNN
@@
 AR Path="/6174477C/6572958C/65833DE4" Ref="#PWR?"  Part="1"
 AR Path="/6174477C/6577909A/65833DE4" Ref="#PWR?"  Part="1"
-AR Path="/6174477C/657790A6/65833DE4" Ref="#PWR0245"  Part="1"
-F 0 "#PWR0245" H 3500 2600 50  0001 C CNN
+AR Path="/6174477C/657790A6/65833DE4" Ref="#PWR0249"  Part="1"
+F 0 "#PWR0249" H 3500 2600 50  0001 C CNN
 F 1 "GND" H 3505 2677 50  0000 C CNN
 F 2 "" H 3500 2850 50  0001 C CNN
@@
 AR Path="/6174477C/6572958C/65833DFB" Ref="C?"  Part="1"
 AR Path="/6174477C/6577909A/65833DFB" Ref="C?"  Part="1"
-AR Path="/6174477C/657790A6/65833DFB" Ref="C98"  Part="1"
-F 0 "C98" H 8100 4600 50  0000 L CNN
+AR Path="/6174477C/657790A6/65833DFB" Ref="C100"  Part="1"
+F 0 "C100" H 8100 4600 50  0000 L CNN
 F 1 "22pF" H 8100 4500 50  0000 L CNN
 F 2 "Capacitor_SMD:C_0402_1005Metric" H 8400 4550 50  0001 C CNN
@@
 AR Path="/6174477C/6572958C/65833E9A" Ref="C?"  Part="1"
 AR Path="/6174477C/6577909A/65833E9A" Ref="C?"  Part="1"
-AR Path="/6174477C/657790A6/65833E9A" Ref="C97"  Part="1"
-F 0 "C97" H 8100 4600 50  0000 L CNN
+AR Path="/6174477C/657790A6/65833E9A" Ref="C99"  Part="1"
+F 0 "C99" H 8100 4600 50  0000 L CNN
 F 1 "22pF" H 8100 4500 50  0000 L CNN
 F 2 "Capacitor_SMD:C_0402_1005Metric" H 8000 4550 50  0001 C CNN
@@
 AR Path="/6174477C/6572958C/65833EA9" Ref="#PWR?"  Part="1"
 AR Path="/6174477C/6577909A/65833EA9" Ref="#PWR?"  Part="1"
-AR Path="/6174477C/657790A6/65833EA9" Ref="#PWR0253"  Part="1"
-F 0 "#PWR0253" H 8400 4450 50  0001 C CNN
+AR Path="/6174477C/657790A6/65833EA9" Ref="#PWR0257"  Part="1"
+F 0 "#PWR0257" H 8400 4450 50  0001 C CNN
 F 1 "GND" H 8405 4527 50  0000 C CNN
 F 2 "" H 8400 4700 50  0001 C CNN
@@
 AR Path="/6174477C/6572958C/65833EBD" Ref="#PWR?"  Part="1"
 AR Path="/6174477C/6577909A/65833EBD" Ref="#PWR?"  Part="1"
-AR Path="/6174477C/657790A6/65833EBD" Ref="#PWR0249"  Part="1"
-F 0 "#PWR0249" H 8000 4450 50  0001 C CNN
+AR Path="/6174477C/657790A6/65833EBD" Ref="#PWR0253"  Part="1"
+F 0 "#PWR0253" H 8000 4450 50  0001 C CNN
 F 1 "GND" H 8005 4527 50  0000 C CNN
 F 2 "" H 8000 4700 50  0001 C CNN
@@
 AR Path="/6174477C/6572958C/65833DFE" Ref="#PWR?"  Part="1"
 AR Path="/6174477C/6577909A/65833DFE" Ref="#PWR?"  Part="1"
-AR Path="/6174477C/657790A6/65833DFE" Ref="#PWR0250"  Part="1"
-F 0 "#PWR0250" H 8200 3950 50  0001 C CNN
+AR Path="/6174477C/657790A6/65833DFE" Ref="#PWR0254"  Part="1"
+F 0 "#PWR0254" H 8200 3950 50  0001 C CNN
 F 1 "GND" H 8205 4027 50  0000 C CNN
 F 2 "" H 8200 4200 50  0001 C CNN
@@
 AR Path="/6174477C/6572958C/65833E12" Ref="#PWR?"  Part="1"
 AR Path="/6174477C/6577909A/65833E12" Ref="#PWR?"  Part="1"
-AR Path="/6174477C/657790A6/65833E12" Ref="#PWR0251"  Part="1"
-F 0 "#PWR0251" H 8200 4150 50  0001 C CNN
+AR Path="/6174477C/657790A6/65833E12" Ref="#PWR0255"  Part="1"
+F 0 "#PWR0255" H 8200 4150 50  0001 C CNN
 F 1 "GND" H 8205 4227 50  0000 C CNN
 F 2 "" H 8200 4400 50  0001 C CNN
@@
 AR Path="/6174477C/6572958C/65833E27" Ref="#PWR?"  Part="1"
 AR Path="/6174477C/6577909A/65833E27" Ref="#PWR?"  Part="1"
-AR Path="/6174477C/657790A6/65833E27" Ref="#PWR0244"  Part="1"
-F 0 "#PWR0244" H 3500 1650 50  0001 C CNN
+AR Path="/6174477C/657790A6/65833E27" Ref="#PWR0248"  Part="1"
+F 0 "#PWR0248" H 3500 1650 50  0001 C CNN
 F 1 "+5V_A" H 3515 1973 50  0000 C CNN
 F 2 "" H 3500 1800 50  0001 C CNN
@@
 AR Path="/6174477C/6572958C/65833E35" Ref="#PWR?"  Part="1"
 AR Path="/6174477C/6577909A/65833E35" Ref="#PWR?"  Part="1"
-AR Path="/6174477C/657790A6/65833E35" Ref="#PWR0247"  Part="1"
-F 0 "#PWR0247" H 4700 2600 50  0001 C CNN
+AR Path="/6174477C/657790A6/65833E35" Ref="#PWR0251"  Part="1"
+F 0 "#PWR0251" H 4700 2600 50  0001 C CNN
 F 1 "GND" H 4705 2677 50  0000 C CNN
 F 2 "" H 4700 2850 50  0001 C CNN
@@
 AR Path="/6174477C/6572958C/65833E58" Ref="#PWR?"  Part="1"
 AR Path="/6174477C/6577909A/65833E58" Ref="#PWR?"  Part="1"
-AR Path="/6174477C/657790A6/65833E58" Ref="#PWR0246"  Part="1"
-F 0 "#PWR0246" H 4200 5300 50  0001 C CNN
+AR Path="/6174477C/657790A6/65833E58" Ref="#PWR0250"  Part="1"
+F 0 "#PWR0250" H 4200 5300 50  0001 C CNN
 F 1 "GND" H 4205 5377 50  0000 C CNN
 F 2 "" H 4200 5550 50  0001 C CNN
@@
 AR Path="/6174477C/6572958C/65833EF0" Ref="#PWR?"  Part="1"
 AR Path="/6174477C/6577909A/65833EF0" Ref="#PWR?"  Part="1"
-AR Path="/6174477C/657790A6/65833EF0" Ref="#PWR0252"  Part="1"
-F 0 "#PWR0252" H 8400 3100 50  0001 C CNN
+AR Path="/6174477C/657790A6/65833EF0" Ref="#PWR0256"  Part="1"
+F 0 "#PWR0256" H 8400 3100 50  0001 C CNN
 F 1 "GND" H 8405 3177 50  0000 C CNN
 F 2 "" H 8400 3350 50  0001 C CNN
@@
 AR Path="/6174477C/6572958C/6379A741" Ref="#PWR?"  Part="1"
 AR Path="/6174477C/6577909A/6379A741" Ref="#PWR?"  Part="1"
-AR Path="/6174477C/657790A6/6379A741" Ref="#PWR0248"  Part="1"
-F 0 "#PWR0248" H 6100 5800 50  0001 C CNN
+AR Path="/6174477C/657790A6/6379A741" Ref="#PWR0252"  Part="1"
+F 0 "#PWR0252" H 6100 5800 50  0001 C CNN
 F 1 "GND" H 6105 5877 50  0000 C CNN
 F 2 "" H 6100 6050 50  0001 C CNN
