File: ykts-payload/ykts-mcu-node15.sch (KiCad schematic (older format))
At the start: 12 parts

Commit message: Update nodes
Parts:
- removed C?: 22pF, Capacitor_SMD:C_0402_1005Metric, symbol Device:C_Small
- removed C?: 1uF, Capacitor_SMD:C_0603_1608Metric, symbol Device:C_Small
- removed C?: 100nF, Capacitor_SMD:C_0402_1005Metric, symbol Device:C_Small
- removed D?: NODE0_STATUSLED, LED_SMD:LED_0402_1005Metric, symbol Device:LED
- removed J?: AVR-ISP-6, Connector_PinHeader_2.54mm:PinHeader_2x03_P2.54mm_Vertical, symbol Connector:AVR-ISP-6
- removed R?: 1M, Resistor_SMD:R_0402_1005Metric, symbol Device:R_Small
- removed SW?: ADG802BRT, Package_TO_SOT_SMD:SOT-23-6, symbol yktsat-common:ADG802BRT
- removed U?: ATmega328PB-MU, Package_DFN_QFN:QFN-32-1EP_5x5mm_P0.5mm_EP3.1x3.1mm, symbol MCU_Microchip_ATmega:ATmega328PB-MU
- added C84: 1uF, Capacitor_SMD:C_0603_1608Metric, symbol Device:C_Small
- added C85: 100nF, Capacitor_SMD:C_0402_1005Metric, symbol Device:C_Small
- added C86: 22pF, Capacitor_SMD:C_0402_1005Metric, symbol Device:C_Small
- added D20: NODE15_STATUSLED, LED_SMD:LED_0402_1005Metric, symbol Device:LED
- added J20: AVR-ISP-6, Connector_PinHeader_2.54mm:PinHeader_2x03_P2.54mm_Vertical, symbol Connector:AVR-ISP-6
- added R102: 1M, Resistor_SMD:R_0402_1005Metric, symbol Device:R_Small
- added SW15: ADG802BRT, Package_TO_SOT_SMD:SOT-23-6, symbol yktsat-common:ADG802BRT
- added U28: ATmega328PB-MU, Package_DFN_QFN:QFN-32-1EP_5x5mm_P0.5mm_EP3.1x3.1mm, symbol MCU_Microchip_ATmega:ATmega328PB-MU
- gave numbers to parts that had none: 4
Connections:
- net +5V_A: now also C84.1, C85.1, D20.2 (A), SW15.3 (S), SW15.6 (VDD), U28.18 (AVCC), U28.20 (AREF), U28.4 (VCC)
- net GND: now also C84.2, C85.2, C86.2, J20.6 (GND), SW15.3 (S), U28.21 (GND), U28.33 (GND), U28.5 (GND)
- net ISP_MISO: now also J20.1 (MISO), U28.16 (PB4)
- net ISP_MOSI: now also J20.4 (MOSI), U28.15 (PB3)
- net ISP_SCK: now also J20.3 (SCK), U28.17 (PB5)
- net at Y17.3: now also C86.1, R102.2, U28.8 (XTAL2/PB7)
- net at C87.1, Y17.1: now also R102.1, U28.7 (XTAL1/PB6)
- net at R103.2: now also D20.1 (K)
- net NODE0_RESET renamed NODE15_RESET
- net NODE15_RESET: now also J20.5 (~RST), U28.29 (~RESET~/PC6)
- new net NODE15_PWR: SW15.4 (IN)
- new net NODE15_RX: U28.31 (PD1)
- new net NODE15_TX: U28.30 (PD0)
Other:
- note added: "MCU Node 15"
- note removed: "MCU Node 0"
