File: ykts-payload/ykts-mcu-node15.sch (KiCad schematic (older format))
At the start: 12 parts, among them J28 AVR-ISP-6, SW16 ADG802BRT, U27 ATmega328PB-MU, Y20 8 MHz

Commit message: Revision B2
Hierarchal sheets for nodes
Partial PCB layout
Parts:
- renumbered C99 to C101, C100 to C102, C101 to C103, C102 to C104, U27 to U29
Changed lines of the file:
@@
 Sheet 18 18
 Title "YktSat Payload Module"
-Date "2021-10-22"
-Rev "B0"
+Date "2021-10-26"
+Rev "B1"
 Comp "Sakha Aerospace Systems, LLC"
 Comment1 ""
@@
 AR Path="/6174477C/6572958C/65833EE4" Ref="U?"  Part="1"
 AR Path="/6174477C/6577909A/65833EE4" Ref="U?"  Part="1"
-AR Path="/6174477C/657790A8/65833EE4" Ref="U27"  Part="1"
-F 0 "U27" H 6100 2711 50  0000 C CNN
+AR Path="/6174477C/657790A8/65833EE4" Ref="U29"  Part="1"
+F 0 "U29" H 6100 2711 50  0000 C CNN
 F 1 "ATmega328PB-MU" H 6100 2620 50  0000 C CNN
 F 2 "Package_DFN_QFN:QFN-32-1EP_5x5mm_P0.5mm_EP3.1x3.1mm" H 6100 4300 50  0001 C CIN
@@
 AR Path="/6174477C/6572958C/65833DB5" Ref="C?"  Part="1"
 AR Path="/6174477C/6577909A/65833DB5" Ref="C?"  Part="1"
-AR Path="/6174477C/657790A8/65833DB5" Ref="C99"  Part="1"
-F 0 "C99" H 4442 2646 50  0000 L CNN
+AR Path="/6174477C/657790A8/65833DB5" Ref="C101"  Part="1"
+F 0 "C101" H 4442 2646 50  0000 L CNN
 F 1 "1uF" H 4442 2555 50  0000 L CNN
 F 2 "Capacitor_SMD:C_0603_1608Metric" H 4350 2600 50  0001 C CNN
@@
 AR Path="/6174477C/6572958C/65833EDD" Ref="C?"  Part="1"
 AR Path="/6174477C/6577909A/65833EDD" Ref="C?"  Part="1"
-AR Path="/6174477C/657790A8/65833EDD" Ref="C100"  Part="1"
-F 0 "C100" H 4792 2646 50  0000 L CNN
+AR Path="/6174477C/657790A8/65833EDD" Ref="C102"  Part="1"
+F 0 "C102" H 4792 2646 50  0000 L CNN
 F 1 "100nF" H 4792 2555 50  0000 L CNN
 F 2 "Capacitor_SMD:C_0402_1005Metric" H 4700 2600 50  0001 C CNN
@@
 AR Path="/6174477C/6572958C/65833DE8" Ref="#PWR?"  Part="1"
 AR Path="/6174477C/6577909A/65833DE8" Ref="#PWR?"  Part="1"
-AR Path="/6174477C/657790A8/65833DE8" Ref="#PWR0255"  Part="1"
-F 0 "#PWR0255" H 3500 2600 50  0001 C CNN
+AR Path="/6174477C/657790A8/65833DE8" Ref="#PWR0259"  Part="1"
+F 0 "#PWR0259" H 3500 2600 50  0001 C CNN
 F 1 "GND" H 3505 2677 50  0000 C CNN
 F 2 "" H 3500 2850 50  0001 C CNN
@@
 AR Path="/6174477C/6572958C/65833DF9" Ref="C?"  Part="1"
 AR Path="/6174477C/6577909A/65833DF9" Ref="C?"  Part="1"
-AR Path="/6174477C/657790A8/65833DF9" Ref="C102"  Part="1"
-F 0 "C102" H 8100 4600 50  0000 L CNN
+AR Path="/6174477C/657790A8/65833DF9" Ref="C104"  Part="1"
+F 0 "C104" H 8100 4600 50  0000 L CNN
 F 1 "22pF" H 8100 4500 50  0000 L CNN
 F 2 "Capacitor_SMD:C_0402_1005Metric" H 8400 4550 50  0001 C CNN
@@
 AR Path="/6174477C/6572958C/6391666C" Ref="C?"  Part="1"
 AR Path="/6174477C/6577909A/6391666C" Ref="C?"  Part="1"
-AR Path="/6174477C/657790A8/6391666C" Ref="C101"  Part="1"
-F 0 "C101" H 8100 4600 50  0000 L CNN
+AR Path="/6174477C/657790A8/6391666C" Ref="C103"  Part="1"
+F 0 "C103" H 8100 4600 50  0000 L CNN
 F 1 "22pF" H 8100 4500 50  0000 L CNN
 F 2 "Capacitor_SMD:C_0402_1005Metric" H 8000 4550 50  0001 C CNN
@@
 AR Path="/6174477C/6572958C/65833EA7" Ref="#PWR?"  Part="1"
 AR Path="/6174477C/6577909A/65833EA7" Ref="#PWR?"  Part="1"
-AR Path="/6174477C/657790A8/65833EA7" Ref="#PWR0263"  Part="1"
-F 0 "#PWR0263" H 8400 4450 50  0001 C CNN
+AR Path="/6174477C/657790A8/65833EA7" Ref="#PWR0267"  Part="1"
+F 0 "#PWR0267" H 8400 4450 50  0001 C CNN
 F 1 "GND" H 8405 4527 50  0000 C CNN
 F 2 "" H 8400 4700 50  0001 C CNN
@@
 AR Path="/6174477C/6572958C/65833EB1" Ref="#PWR?"  Part="1"
 AR Path="/6174477C/6577909A/65833EB1" Ref="#PWR?"  Part="1"
-AR Path="/6174477C/657790A8/65833EB1" Ref="#PWR0259"  Part="1"
-F 0 "#PWR0259" H 8000 4450 50  0001 C CNN
+AR Path="/6174477C/657790A8/65833EB1" Ref="#PWR0263"  Part="1"
+F 0 "#PWR0263" H 8000 4450 50  0001 C CNN
 F 1 "GND" H 8005 4527 50  0000 C CNN
 F 2 "" H 8000 4700 50  0001 C CNN
@@
 AR Path="/6174477C/6572958C/65833E03" Ref="#PWR?"  Part="1"
 AR Path="/6174477C/6577909A/65833E03" Ref="#PWR?"  Part="1"
-AR Path="/6174477C/657790A8/65833E03" Ref="#PWR0260"  Part="1"
-F 0 "#PWR0260" H 8200 3950 50  0001 C CNN
+AR Path="/6174477C/657790A8/65833E03" Ref="#PWR0264"  Part="1"
+F 0 "#PWR0264" H 8200 3950 50  0001 C CNN
 F 1 "GND" H 8205 4027 50  0000 C CNN
 F 2 "" H 8200 4200 50  0001 C CNN
@@
 AR Path="/6174477C/6572958C/65833E17" Ref="#PWR?"  Part="1"
 AR Path="/6174477C/6577909A/65833E17" Ref="#PWR?"  Part="1"
-AR Path="/6174477C/657790A8/65833E17" Ref="#PWR0261"  Part="1"
-F 0 "#PWR0261" H 8200 4150 50  0001 C CNN
+AR Path="/6174477C/657790A8/65833E17" Ref="#PWR0265"  Part="1"
+F 0 "#PWR0265" H 8200 4150 50  0001 C CNN
 F 1 "GND" H 8205 4227 50  0000 C CNN
 F 2 "" H 8200 4400 50  0001 C CNN
@@
 AR Path="/6174477C/6572958C/65833E1F" Ref="#PWR?"  Part="1"
 AR Path="/6174477C/6577909A/65833E1F" Ref="#PWR?"  Part="1"
-AR Path="/6174477C/657790A8/65833E1F" Ref="#PWR0254"  Part="1"
-F 0 "#PWR0254" H 3500 1650 50  0001 C CNN
+AR Path="/6174477C/657790A8/65833E1F" Ref="#PWR0258"  Part="1"
+F 0 "#PWR0258" H 3500 1650 50  0001 C CNN
 F 1 "+5V_A" H 3515 1973 50  0000 C CNN
 F 2 "" H 3500 1800 50  0001 C CNN
@@
 AR Path="/6174477C/6572958C/65833E2F" Ref="#PWR?"  Part="1"
 AR Path="/6174477C/6577909A/65833E2F" Ref="#PWR?"  Part="1"
-AR Path="/6174477C/657790A8/65833E2F" Ref="#PWR0257"  Part="1"
-F 0 "#PWR0257" H 4700 2600 50  0001 C CNN
+AR Path="/6174477C/657790A8/65833E2F" Ref="#PWR0261"  Part="1"
+F 0 "#PWR0261" H 4700 2600 50  0001 C CNN
 F 1 "GND" H 4705 2677 50  0000 C CNN
 F 2 "" H 4700 2850 50  0001 C CNN
@@
 AR Path="/6174477C/6572958C/65833E5B" Ref="#PWR?"  Part="1"
 AR Path="/6174477C/6577909A/65833E5B" Ref="#PWR?"  Part="1"
-AR Path="/6174477C/657790A8/65833E5B" Ref="#PWR0256"  Part="1"
-F 0 "#PWR0256" H 4200 5300 50  0001 C CNN
+AR Path="/6174477C/657790A8/65833E5B" Ref="#PWR0260"  Part="1"
+F 0 "#PWR0260" H 4200 5300 50  0001 C CNN
 F 1 "GND" H 4205 5377 50  0000 C CNN
 F 2 "" H 4200 5550 50  0001 C CNN
@@
 AR Path="/6174477C/6572958C/65833EF3" Ref="#PWR?"  Part="1"
 AR Path="/6174477C/6577909A/65833EF3" Ref="#PWR?"  Part="1"
-AR Path="/6174477C/657790A8/65833EF3" Ref="#PWR0262"  Part="1"
-F 0 "#PWR0262" H 8400 3100 50  0001 C CNN
+AR Path="/6174477C/657790A8/65833EF3" Ref="#PWR0266"  Part="1"
+F 0 "#PWR0266" H 8400 3100 50  0001 C CNN
 F 1 "GND" H 8405 3177 50  0000 C CNN
 F 2 "" H 8400 3350 50  0001 C CNN
@@
 AR Path="/6174477C/6572958C/65833DCF" Ref="#PWR?"  Part="1"
 AR Path="/6174477C/6577909A/65833DCF" Ref="#PWR?"  Part="1"
-AR Path="/6174477C/657790A8/65833DCF" Ref="#PWR0258"  Part="1"
-F 0 "#PWR0258" H 6100 5800 50  0001 C CNN
+AR Path="/6174477C/657790A8/65833DCF" Ref="#PWR0262"  Part="1"
+F 0 "#PWR0262" H 6100 5800 50  0001 C CNN
 F 1 "GND" H 6105 5877 50  0000 C CNN
 F 2 "" H 6100 6050 50  0001 C CNN
