File: ykts-payload/ykts-mcu-node3.sch (KiCad schematic (older format))
At the start: 12 parts

Commit message: Update nodes
Parts:
- D8: renamed from D?; value NODE0_STATUSLED -> NODE3_STATUSLED
- gave numbers to parts that had none: 11
Connections:
- net NODE0_PWR renamed NODE3_PWR
- net NODE0_RESET renamed NODE3_RESET
- net NODE0_RX renamed NODE3_RX
- net NODE0_TX renamed NODE3_TX
Other:
- note added: "MCU Node 3"
- note removed: "MCU Node 0"
