File: ykts-payload/ykts-mcu-node3.sch (KiCad schematic (older format))
At the start: 12 parts, among them J8 AVR-ISP-6, SW3 ADG802BRT, U16 ATmega328PB-MU, Y5 8 MHz

Commit message: Fixed annotations & sheet ordering
Parts:
- renumbered C30 to C40, C37 to C41, C38 to C42, C39 to C43, D8 to D12, J8 to J11, R65 to R78, R66 to R79, R67 to R80, SW3 to SW4, U16 to U17, Y5 to Y6

Commit message: Revision A2
Added debug power
Basic ESD protection on UART
MCP Reset from MCU
Parts:
- renumbered D12 to D11, J11 to J12, R78 to R82, R79 to R83, R80 to R84
Changed lines of the file:
@@
 $Descr A4 11693 8268
 encoding utf-8
-Sheet 5 18
+Sheet 6 18
 Title "YktSat Payload Module"
-Date "2021-10-02"
-Rev "A1"
+Date "2021-10-03"
+Rev "A2"
 Comp "Sakha Aerospace Systems, LLC"
 Comment1 ""
@@
 AR Path="/6174477C/637564E2/63916566" Ref="#PWR?"  Part="1"
 AR Path="/6174477C/637CB186/63916566" Ref="#PWR?"  Part="1"
-AR Path="/6174477C/63801AF0/63916566" Ref="#PWR0119"  Part="1"
+AR Path="/6174477C/63801AF0/63916566" Ref="#PWR0121"  Part="1"
 AR Path="/6174477C/638385BC/63916566" Ref="#PWR?"  Part="1"
 AR Path="/6174477C/638DF121/63916566" Ref="#PWR?"  Part="1"
-F 0 "#PWR0119" H 3500 2600 50  0001 C CNN
+F 0 "#PWR0121" H 3500 2600 50  0001 C CNN
 F 1 "GND" H 3505 2677 50  0000 C CNN
 F 2 "" H 3500 2850 50  0001 C CNN
@@
 AR Path="/6174477C/637564E2/63916569" Ref="#PWR?"  Part="1"
 AR Path="/6174477C/637CB186/63916569" Ref="#PWR?"  Part="1"
-AR Path="/6174477C/63801AF0/63916569" Ref="#PWR0127"  Part="1"
+AR Path="/6174477C/63801AF0/63916569" Ref="#PWR0129"  Part="1"
 AR Path="/6174477C/638385BC/63916569" Ref="#PWR?"  Part="1"
 AR Path="/6174477C/638DF121/63916569" Ref="#PWR?"  Part="1"
-F 0 "#PWR0127" H 8400 4450 50  0001 C CNN
+F 0 "#PWR0129" H 8400 4450 50  0001 C CNN
 F 1 "GND" H 8405 4527 50  0000 C CNN
 F 2 "" H 8400 4700 50  0001 C CNN
@@
 AR Path="/6174477C/637564E2/6391697C" Ref="#PWR?"  Part="1"
 AR Path="/6174477C/637CB186/6391697C" Ref="#PWR?"  Part="1"
-AR Path="/6174477C/63801AF0/6391697C" Ref="#PWR0123"  Part="1"
+AR Path="/6174477C/63801AF0/6391697C" Ref="#PWR0125"  Part="1"
 AR Path="/6174477C/638385BC/6391697C" Ref="#PWR?"  Part="1"
 AR Path="/6174477C/638DF121/6391697C" Ref="#PWR?"  Part="1"
-F 0 "#PWR0123" H 8000 4450 50  0001 C CNN
+F 0 "#PWR0125" H 8000 4450 50  0001 C CNN
 F 1 "GND" H 8005 4527 50  0000 C CNN
 F 2 "" H 8000 4700 50  0001 C CNN
@@
 AR Path="/6174477C/637564E2/63916986" Ref="#PWR?"  Part="1"
 AR Path="/6174477C/637CB186/63916986" Ref="#PWR?"  Part="1"
-AR Path="/6174477C/63801AF0/63916986" Ref="#PWR0124"  Part="1"
+AR Path="/6174477C/63801AF0/63916986" Ref="#PWR0126"  Part="1"
 AR Path="/6174477C/638385BC/63916986" Ref="#PWR?"  Part="1"
 AR Path="/6174477C/638DF121/63916986" Ref="#PWR?"  Part="1"
-F 0 "#PWR0124" H 8200 3950 50  0001 C CNN
+F 0 "#PWR0126" H 8200 3950 50  0001 C CNN
 F 1 "GND" H 8205 4027 50  0000 C CNN
 F 2 "" H 8200 4200 50  0001 C CNN
@@
 AR Path="/6174477C/637564E2/63916987" Ref="#PWR?"  Part="1"
 AR Path="/6174477C/637CB186/63916987" Ref="#PWR?"  Part="1"
-AR Path="/6174477C/63801AF0/63916987" Ref="#PWR0125"  Part="1"
+AR Path="/6174477C/63801AF0/63916987" Ref="#PWR0127"  Part="1"
 AR Path="/6174477C/638385BC/63916987" Ref="#PWR?"  Part="1"
 AR Path="/6174477C/638DF121/63916987" Ref="#PWR?"  Part="1"
-F 0 "#PWR0125" H 8200 4150 50  0001 C CNN
+F 0 "#PWR0127" H 8200 4150 50  0001 C CNN
 F 1 "GND" H 8205 4227 50  0000 C CNN
 F 2 "" H 8200 4400 50  0001 C CNN
@@
 AR Path="/6174477C/637564E2/63760B3D" Ref="R?"  Part="1"
 AR Path="/6174477C/637CB186/63760B3D" Ref="R?"  Part="1"
-AR Path="/6174477C/63801AF0/63760B3D" Ref="R78"  Part="1"
+AR Path="/6174477C/63801AF0/63760B3D" Ref="R82"  Part="1"
 AR Path="/6174477C/638385BC/63760B3D" Ref="R?"  Part="1"
 AR Path="/6174477C/638DF121/63760B3D" Ref="R?"  Part="1"
-F 0 "R78" V 6754 4400 50  0000 C CNN
+F 0 "R82" V 6754 4400 50  0000 C CNN
 F 1 "20K" V 6845 4400 50  0000 C CNN
 F 2 "Resistor_SMD:R_0402_1005Metric" H 6950 4400 50  0001 C CNN
@@
 AR Path="/6174477C/637564E2/6386EF37" Ref="#PWR?"  Part="1"
 AR Path="/6174477C/637CB186/6386EF37" Ref="#PWR?"  Part="1"
-AR Path="/6174477C/63801AF0/6386EF37" Ref="#PWR0118"  Part="1"
+AR Path="/6174477C/63801AF0/6386EF37" Ref="#PWR0120"  Part="1"
 AR Path="/6174477C/638385BC/6386EF37" Ref="#PWR?"  Part="1"
 AR Path="/6174477C/638DF121/6386EF37" Ref="#PWR?"  Part="1"
-F 0 "#PWR0118" H 3500 1650 50  0001 C CNN
+F 0 "#PWR0120" H 3500 1650 50  0001 C CNN
 F 1 "+5V_A" H 3515 1973 50  0000 C CNN
 F 2 "" H 3500 1800 50  0001 C CNN
@@
 AR Path="/6174477C/637564E2/6391697D" Ref="#PWR?"  Part="1"
 AR Path="/6174477C/637CB186/6391697D" Ref="#PWR?"  Part="1"
-AR Path="/6174477C/63801AF0/6391697D" Ref="#PWR0121"  Part="1"
+AR Path="/6174477C/63801AF0/6391697D" Ref="#PWR0123"  Part="1"
 AR Path="/6174477C/638385BC/6391697D" Ref="#PWR?"  Part="1"
 AR Path="/6174477C/638DF121/6391697D" Ref="#PWR?"  Part="1"
-F 0 "#PWR0121" H 4550 2600 50  0001 C CNN
+F 0 "#PWR0123" H 4550 2600 50  0001 C CNN
 F 1 "GND" H 4555 2677 50  0000 C CNN
 F 2 "" H 4550 2850 50  0001 C CNN
@@
 AR Path="/6174477C/637564E2/63916983" Ref="R?"  Part="1"
 AR Path="/6174477C/637CB186/63916983" Ref="R?"  Part="1"
-AR Path="/6174477C/63801AF0/63916983" Ref="R79"  Part="1"
+AR Path="/6174477C/63801AF0/63916983" Ref="R83"  Part="1"
 AR Path="/6174477C/638385BC/63916983" Ref="R?"  Part="1"
 AR Path="/6174477C/638DF121/63916983" Ref="R?"  Part="1"
-F 0 "R79" V 8004 3950 50  0000 C CNN
+F 0 "R83" V 8004 3950 50  0000 C CNN
 F 1 "1M" V 8095 3950 50  0000 C CNN
 F 2 "Resistor_SMD:R_0402_1005Metric" H 8200 3950 50  0001 C CNN
@@
 AR Path="/6174477C/637564E2/63916984" Ref="J?"  Part="1"
 AR Path="/6174477C/637CB186/63916984" Ref="J?"  Part="1"
-AR Path="/6174477C/63801AF0/63916984" Ref="J11"  Part="1"
+AR Path="/6174477C/63801AF0/63916984" Ref="J12"  Part="1"
 AR Path="/6174477C/638385BC/63916984" Ref="J?"  Part="1"
 AR Path="/6174477C/638DF121/63916984" Ref="J?"  Part="1"
-F 0 "J11" H 3770 5146 50  0000 R CNN
+F 0 "J12" H 3770 5146 50  0000 R CNN
 F 1 "AVR-ISP-6" H 3770 5055 50  0000 R CNN
 F 2 "Connector_PinHeader_2.54mm:PinHeader_2x03_P2.54mm_Vertical" V 3850 5100 50  0001 C CNN
@@
 AR Path="/6174477C/637564E2/63916577" Ref="#PWR?"  Part="1"
 AR Path="/6174477C/637CB186/63916577" Ref="#PWR?"  Part="1"
-AR Path="/6174477C/63801AF0/63916577" Ref="#PWR0120"  Part="1"
+AR Path="/6174477C/63801AF0/63916577" Ref="#PWR0122"  Part="1"
 AR Path="/6174477C/638385BC/63916577" Ref="#PWR?"  Part="1"
 AR Path="/6174477C/638DF121/63916577" Ref="#PWR?"  Part="1"
-F 0 "#PWR0120" H 4200 5300 50  0001 C CNN
+F 0 "#PWR0122" H 4200 5300 50  0001 C CNN
 F 1 "GND" H 4205 5377 50  0000 C CNN
 F 2 "" H 4200 5550 50  0001 C CNN
@@
 AR Path="/6174477C/637564E2/63796EF3" Ref="D?"  Part="1"
 AR Path="/6174477C/637CB186/63796EF3" Ref="D?"  Part="1"
-AR Path="/6174477C/63801AF0/63796EF3" Ref="D12"  Part="1"
+AR Path="/6174477C/63801AF0/63796EF3" Ref="D11"  Part="1"
 AR Path="/6174477C/638385BC/63796EF3" Ref="D?"  Part="1"
 AR Path="/6174477C/638DF121/63796EF3" Ref="D?"  Part="1"
-F 0 "D12" V 8439 2682 50  0000 R CNN
+F 0 "D11" V 8439 2682 50  0000 R CNN
 F 1 "NODE3_STATUSLED" V 8348 2682 50  0000 R CNN
 F 2 "LED_SMD:LED_0402_1005Metric" H 8400 2800 50  0001 C CNN
@@
 AR Path="/6174477C/637564E2/63916975" Ref="R?"  Part="1"
 AR Path="/6174477C/637CB186/63916975" Ref="R?"  Part="1"
-AR Path="/6174477C/63801AF0/63916975" Ref="R80"  Part="1"
+AR Path="/6174477C/63801AF0/63916975" Ref="R84"  Part="1"
 AR Path="/6174477C/638385BC/63916975" Ref="R?"  Part="1"
 AR Path="/6174477C/638DF121/63916975" Ref="R?"  Part="1"
-F 0 "R80" V 8204 3150 50  0000 C CNN
+F 0 "R84" V 8204 3150 50  0000 C CNN
 F 1 "1K" V 8295 3150 50  0000 C CNN
 F 2 "Resistor_SMD:R_0402_1005Metric" H 8400 3150 50  0001 C CNN
@@
 AR Path="/6174477C/637564E2/6391656F" Ref="#PWR?"  Part="1"
 AR Path="/6174477C/637CB186/6391656F" Ref="#PWR?"  Part="1"
-AR Path="/6174477C/63801AF0/6391656F" Ref="#PWR0126"  Part="1"
+AR Path="/6174477C/63801AF0/6391656F" Ref="#PWR0128"  Part="1"
 AR Path="/6174477C/638385BC/6391656F" Ref="#PWR?"  Part="1"
 AR Path="/6174477C/638DF121/6391656F" Ref="#PWR?"  Part="1"
-F 0 "#PWR0126" H 8400 3100 50  0001 C CNN
+F 0 "#PWR0128" H 8400 3100 50  0001 C CNN
 F 1 "GND" H 8405 3177 50  0000 C CNN
 F 2 "" H 8400 3350 50  0001 C CNN
@@
 AR Path="/6174477C/637564E2/6386EE42" Ref="#PWR?"  Part="1"
 AR Path="/6174477C/637CB186/6386EE42" Ref="#PWR?"  Part="1"
-AR Path="/6174477C/63801AF0/6386EE42" Ref="#PWR0122"  Part="1"
+AR Path="/6174477C/63801AF0/6386EE42" Ref="#PWR0124"  Part="1"
 AR Path="/6174477C/638385BC/6386EE42" Ref="#PWR?"  Part="1"
 AR Path="/6174477C/638DF121/6386EE42" Ref="#PWR?"  Part="1"
-F 0 "#PWR0122" H 6100 5800 50  0001 C CNN
+F 0 "#PWR0124" H 6100 5800 50  0001 C CNN
 F 1 "GND" H 6105 5877 50  0000 C CNN
 F 2 "" H 6100 6050 50  0001 C CNN

Commit message: Fix git
Connections:
- net +5V_A: no longer C40.1, C41.1, D11.2 (A), R82.2, U17.18 (AVCC), U17.20 (AREF), U17.4 (VCC)
- net at SW4.1 (D): now also C40.1, C41.1, D11.2 (A), R82.2, U17.18 (AVCC), U17.20 (AREF), U17.4 (VCC)

Commit message: Change node ISP connector footprint
Parts:
- J12: footprint Connector_PinHeader_2.54mm:PinHeader_2x03_P2.54mm_Vertical -> Connector_PinHeader_1.27mm:PinHeader_2x03_P1.27mm_Vertical_SMD
Changed lines of the file:
@@
 F 0 "J12" H 3770 5146 50  0000 R CNN
 F 1 "AVR-ISP-6" H 3770 5055 50  0000 R CNN
-F 2 "Connector_PinHeader_2.54mm:PinHeader_2x03_P2.54mm_Vertical" V 3850 5100 50  0001 C CNN
+F 2 "Connector_PinHeader_1.27mm:PinHeader_2x03_P1.27mm_Vertical_SMD" V 3850 5100 50  0001 C CNN
 F 3 " ~" H 2825 4500 50  0001 C CNN
 	1    4100 5050

Commit message: Revision B0
Added second supervisor, mega2560 -> mega128a
Parts:
- renumbered C40 to C51, C41 to C52, C42 to C53, C43 to C54, D11 to D13, J12 to J16, R82 to R60, R83 to R61, R84 to R62, U17 to U15, Y6 to Y8
Changed lines of the file:
@@
 Sheet 6 18
 Title "YktSat Payload Module"
-Date "2021-10-03"
-Rev "A3"
+Date "2021-10-22"
+Rev "B0"
 Comp "Sakha Aerospace Systems, LLC"
 Comment1 ""
@@
 AR Path="/6174477C/6572958C/65833EE7" Ref="U?"  Part="1"
 AR Path="/6174477C/6577909A/65833EE7" Ref="U?"  Part="1"
-AR Path="/6174477C/656DAE2C/65833EE7" Ref="U17"  Part="1"
-F 0 "U17" H 6100 2711 50  0000 C CNN
+AR Path="/6174477C/656DAE2C/65833EE7" Ref="U15"  Part="1"
+F 0 "U15" H 6100 2711 50  0000 C CNN
 F 1 "ATmega328PB-MU" H 6100 2620 50  0000 C CNN
 F 2 "Package_DFN_QFN:QFN-32-1EP_5x5mm_P0.5mm_EP3.1x3.1mm" H 6100 4300 50  0001 C CIN
@@
 AR Path="/6174477C/6572958C/65833DC0" Ref="C?"  Part="1"
 AR Path="/6174477C/6577909A/65833DC0" Ref="C?"  Part="1"
-AR Path="/6174477C/656DAE2C/65833DC0" Ref="C40"  Part="1"
-F 0 "C40" H 4442 2646 50  0000 L CNN
+AR Path="/6174477C/656DAE2C/65833DC0" Ref="C51"  Part="1"
+F 0 "C51" H 4442 2646 50  0000 L CNN
 F 1 "1uF" H 4442 2555 50  0000 L CNN
 F 2 "Capacitor_SMD:C_0603_1608Metric" H 4350 2600 50  0001 C CNN
@@
 AR Path="/6174477C/6572958C/65833ED4" Ref="C?"  Part="1"
 AR Path="/6174477C/6577909A/65833ED4" Ref="C?"  Part="1"
-AR Path="/6174477C/656DAE2C/65833ED4" Ref="C41"  Part="1"
-F 0 "C41" H 4792 2646 50  0000 L CNN
+AR Path="/6174477C/656DAE2C/65833ED4" Ref="C52"  Part="1"
+F 0 "C52" H 4792 2646 50  0000 L CNN
 F 1 "100nF" H 4792 2555 50  0000 L CNN
 F 2 "Capacitor_SMD:C_0402_1005Metric" H 4700 2600 50  0001 C CNN
@@
 AR Path="/6174477C/6572958C/6386EE31" Ref="#PWR?"  Part="1"
 AR Path="/6174477C/6577909A/6386EE31" Ref="#PWR?"  Part="1"
-AR Path="/6174477C/656DAE2C/6386EE31" Ref="#PWR0121"  Part="1"
-F 0 "#PWR0121" H 3500 2600 50  0001 C CNN
+AR Path="/6174477C/656DAE2C/6386EE31" Ref="#PWR0135"  Part="1"
+F 0 "#PWR0135" H 3500 2600 50  0001 C CNN
 F 1 "GND" H 3505 2677 50  0000 C CNN
 F 2 "" H 3500 2850 50  0001 C CNN
@@
 AR Path="/6174477C/6572958C/65833DF2" Ref="C?"  Part="1"
 AR Path="/6174477C/6577909A/65833DF2" Ref="C?"  Part="1"
-AR Path="/6174477C/656DAE2C/65833DF2" Ref="C43"  Part="1"
-F 0 "C43" H 8100 4600 50  0000 L CNN
+AR Path="/6174477C/656DAE2C/65833DF2" Ref="C54"  Part="1"
+F 0 "C54" H 8100 4600 50  0000 L CNN
 F 1 "22pF" H 8100 4500 50  0000 L CNN
 F 2 "Capacitor_SMD:C_0402_1005Metric" H 8400 4550 50  0001 C CNN
@@
 AR Path="/6174477C/6572958C/65833E99" Ref="C?"  Part="1"
 AR Path="/6174477C/6577909A/65833E99" Ref="C?"  Part="1"
-AR Path="/6174477C/656DAE2C/65833E99" Ref="C42"  Part="1"
-F 0 "C42" H 8100 4600 50  0000 L CNN
+AR Path="/6174477C/656DAE2C/65833E99" Ref="C53"  Part="1"
+F 0 "C53" H 8100 4600 50  0000 L CNN
 F 1 "22pF" H 8100 4500 50  0000 L CNN
 F 2 "Capacitor_SMD:C_0402_1005Metric" H 8000 4550 50  0001 C CNN
@@
 AR Path="/6174477C/6572958C/65833EA8" Ref="#PWR?"  Part="1"
 AR Path="/6174477C/6577909A/65833EA8" Ref="#PWR?"  Part="1"
-AR Path="/6174477C/656DAE2C/65833EA8" Ref="#PWR0129"  Part="1"
-F 0 "#PWR0129" H 8400 4450 50  0001 C CNN
+AR Path="/6174477C/656DAE2C/65833EA8" Ref="#PWR0143"  Part="1"
+F 0 "#PWR0143" H 8400 4450 50  0001 C CNN
 F 1 "GND" H 8405 4527 50  0000 C CNN
 F 2 "" H 8400 4700 50  0001 C CNN
@@
 AR Path="/6174477C/6572958C/65833EB5" Ref="#PWR?"  Part="1"
 AR Path="/6174477C/6577909A/65833EB5" Ref="#PWR?"  Part="1"
-AR Path="/6174477C/656DAE2C/65833EB5" Ref="#PWR0125"  Part="1"
-F 0 "#PWR0125" H 8000 4450 50  0001 C CNN
+AR Path="/6174477C/656DAE2C/65833EB5" Ref="#PWR0139"  Part="1"
+F 0 "#PWR0139" H 8000 4450 50  0001 C CNN
 F 1 "GND" H 8005 4527 50  0000 C CNN
 F 2 "" H 8000 4700 50  0001 C CNN
@@
 AR Path="/6174477C/6572958C/65833EC2" Ref="Y?"  Part="1"
 AR Path="/6174477C/6577909A/65833EC2" Ref="Y?"  Part="1"
-AR Path="/6174477C/656DAE2C/65833EC2" Ref="Y6"  Part="1"
-F 0 "Y6" H 8450 4350 50  0000 L CNN
+AR Path="/6174477C/656DAE2C/65833EC2" Ref="Y8"  Part="1"
+F 0 "Y8" H 8450 4350 50  0000 L CNN
 F 1 "8 MHz" H 8450 4250 50  0000 L CNN
 F 2 "Crystal:Crystal_SMD_2520-4Pin_2.5x2.0mm" H 8200 4300 50  0001 C CNN
@@
 AR Path="/6174477C/6572958C/65833E0B" Ref="#PWR?"  Part="1"
 AR Path="/6174477C/6577909A/65833E0B" Ref="#PWR?"  Part="1"
-AR Path="/6174477C/656DAE2C/65833E0B" Ref="#PWR0126"  Part="1"
-F 0 "#PWR0126" H 8200 3950 50  0001 C CNN
+AR Path="/6174477C/656DAE2C/65833E0B" Ref="#PWR0140"  Part="1"
+F 0 "#PWR0140" H 8200 3950 50  0001 C CNN
 F 1 "GND" H 8205 4027 50  0000 C CNN
 F 2 "" H 8200 4200 50  0001 C CNN
@@
 AR Path="/6174477C/6572958C/65833E14" Ref="#PWR?"  Part="1"
 AR Path="/6174477C/6577909A/65833E14" Ref="#PWR?"  Part="1"
-AR Path="/6174477C/656DAE2C/65833E14" Ref="#PWR0127"  Part="1"
-F 0 "#PWR0127" H 8200 4150 50  0001 C CNN
+AR Path="/6174477C/656DAE2C/65833E14" Ref="#PWR0141"  Part="1"
+F 0 "#PWR0141" H 8200 4150 50  0001 C CNN
 F 1 "GND" H 8205 4227 50  0000 C CNN
 F 2 "" H 8200 4400 50  0001 C CNN
@@
 AR Path="/6174477C/6572958C/638383BB" Ref="R?"  Part="1"
 AR Path="/6174477C/6577909A/638383BB" Ref="R?"  Part="1"
-AR Path="/6174477C/656DAE2C/638383BB" Ref="R82"  Part="1"
-F 0 "R82" V 6754 4400 50  0000 C CNN
+AR Path="/6174477C/656DAE2C/638383BB" Ref="R60"  Part="1"
+F 0 "R60" V 6754 4400 50  0000 C CNN
 F 1 "20K" V 6845 4400 50  0000 C CNN
 F 2 "Resistor_SMD:R_0402_1005Metric" H 6950 4400 50  0001 C CNN
@@
 AR Path="/6174477C/6572958C/65833E1B" Ref="#PWR?"  Part="1"
 AR Path="/6174477C/6577909A/65833E1B" Ref="#PWR?"  Part="1"
-AR Path="/6174477C/656DAE2C/65833E1B" Ref="#PWR0120"  Part="1"
-F 0 "#PWR0120" H 3500 1650 50  0001 C CNN
+AR Path="/6174477C/656DAE2C/65833E1B" Ref="#PWR0134"  Part="1"
+F 0 "#PWR0134" H 3500 1650 50  0001 C CNN
 F 1 "+5V_A" H 3515 1973 50  0000 C CNN
 F 2 "" H 3500 1800 50  0001 C CNN
@@
 AR Path="/6174477C/6572958C/65833E2D" Ref="#PWR?"  Part="1"
 AR Path="/6174477C/6577909A/65833E2D" Ref="#PWR?"  Part="1"
-AR Path="/6174477C/656DAE2C/65833E2D" Ref="#PWR0123"  Part="1"
-F 0 "#PWR0123" H 4700 2600 50  0001 C CNN
+AR Path="/6174477C/656DAE2C/65833E2D" Ref="#PWR0137"  Part="1"
+F 0 "#PWR0137" H 4700 2600 50  0001 C CNN
 F 1 "GND" H 4705 2677 50  0000 C CNN
 F 2 "" H 4700 2850 50  0001 C CNN
@@
 AR Path="/6174477C/6572958C/65833E3B" Ref="R?"  Part="1"
 AR Path="/6174477C/6577909A/65833E3B" Ref="R?"  Part="1"
-AR Path="/6174477C/656DAE2C/65833E3B" Ref="R83"  Part="1"
-F 0 "R83" V 8004 3950 50  0000 C CNN
+AR Path="/6174477C/656DAE2C/65833E3B" Ref="R61"  Part="1"
+F 0 "R61" V 8004 3950 50  0000 C CNN
 F 1 "1M" V 8095 3950 50  0000 C CNN
 F 2 "Resistor_SMD:R_0402_1005Metric" H 8200 3950 50  0001 C CNN
@@
 AR Path="/6174477C/6572958C/65833E55" Ref="J?"  Part="1"
 AR Path="/6174477C/6577909A/65833E55" Ref="J?"  Part="1"
-AR Path="/6174477C/656DAE2C/65833E55" Ref="J12"  Part="1"
-F 0 "J12" H 3770 5146 50  0000 R CNN
+AR Path="/6174477C/656DAE2C/65833E55" Ref="J16"  Part="1"
+F 0 "J16" H 3770 5146 50  0000 R CNN
 F 1 "AVR-ISP-6" H 3770 5055 50  0000 R CNN
 F 2 "Connector_PinHeader_1.27mm:PinHeader_2x03_P1.27mm_Vertical_SMD" V 3850 5100 50  0001 C CNN
@@
 AR Path="/6174477C/6572958C/65833E63" Ref="#PWR?"  Part="1"
 AR Path="/6174477C/6577909A/65833E63" Ref="#PWR?"  Part="1"
-AR Path="/6174477C/656DAE2C/65833E63" Ref="#PWR0122"  Part="1"
-F 0 "#PWR0122" H 4200 5300 50  0001 C CNN
+AR Path="/6174477C/656DAE2C/65833E63" Ref="#PWR0136"  Part="1"
+F 0 "#PWR0136" H 4200 5300 50  0001 C CNN
 F 1 "GND" H 4205 5377 50  0000 C CNN
 F 2 "" H 4200 5550 50  0001 C CNN
@@
 AR Path="/6174477C/6572958C/65833E66" Ref="D?"  Part="1"
 AR Path="/6174477C/6577909A/65833E66" Ref="D?"  Part="1"
-AR Path="/6174477C/656DAE2C/65833E66" Ref="D11"  Part="1"
-F 0 "D11" V 8439 2682 50  0000 R CNN
+AR Path="/6174477C/656DAE2C/65833E66" Ref="D13"  Part="1"
+F 0 "D13" V 8439 2682 50  0000 R CNN
 F 1 "NODE3_STATUSLED" V 8348 2682 50  0000 R CNN
 F 2 "LED_SMD:LED_0402_1005Metric" H 8400 2800 50  0001 C CNN
@@
 AR Path="/6174477C/6572958C/65833E7D" Ref="R?"  Part="1"
 AR Path="/6174477C/6577909A/65833E7D" Ref="R?"  Part="1"
-AR Path="/6174477C/656DAE2C/65833E7D" Ref="R84"  Part="1"
-F 0 "R84" V 8204 3150 50  0000 C CNN
+AR Path="/6174477C/656DAE2C/65833E7D" Ref="R62"  Part="1"
+F 0 "R62" V 8204 3150 50  0000 C CNN
 F 1 "1K" V 8295 3150 50  0000 C CNN
 F 2 "Resistor_SMD:R_0402_1005Metric" H 8400 3150 50  0001 C CNN
@@
 AR Path="/6174477C/6572958C/65833EF9" Ref="#PWR?"  Part="1"
 AR Path="/6174477C/6577909A/65833EF9" Ref="#PWR?"  Part="1"
-AR Path="/6174477C/656DAE2C/65833EF9" Ref="#PWR0128"  Part="1"
-F 0 "#PWR0128" H 8400 3100 50  0001 C CNN
+AR Path="/6174477C/656DAE2C/65833EF9" Ref="#PWR0142"  Part="1"
+F 0 "#PWR0142" H 8400 3100 50  0001 C CNN
 F 1 "GND" H 8405 3177 50  0000 C CNN
 F 2 "" H 8400 3350 50  0001 C CNN
@@
 AR Path="/6174477C/6572958C/65833DCE" Ref="#PWR?"  Part="1"
 AR Path="/6174477C/6577909A/65833DCE" Ref="#PWR?"  Part="1"
-AR Path="/6174477C/656DAE2C/65833DCE" Ref="#PWR0124"  Part="1"
-F 0 "#PWR0124" H 6100 5800 50  0001 C CNN
+AR Path="/6174477C/656DAE2C/65833DCE" Ref="#PWR0138"  Part="1"
+F 0 "#PWR0138" H 6100 5800 50  0001 C CNN
 F 1 "GND" H 6105 5877 50  0000 C CNN
 F 2 "" H 6100 6050 50  0001 C CNN
