File: ykts-payload/ykts-mcu-node3.sch (KiCad schematic (older format))
At the start: 12 parts, among them J16 AVR-ISP-6, SW4 ADG802BRT, U15 ATmega328PB-MU, Y8 8 MHz

Commit message: Revision B2
Hierarchal sheets for nodes
Partial PCB layout
Parts:
- renumbered C51 to C53, C52 to C54, C53 to C55, C54 to C56, U15 to U17
Changed lines of the file:
@@
 Sheet 6 18
 Title "YktSat Payload Module"
-Date "2021-10-22"
-Rev "B0"
+Date "2021-10-26"
+Rev "B1"
 Comp "Sakha Aerospace Systems, LLC"
 Comment1 ""
@@
 AR Path="/6174477C/6572958C/65833EE7" Ref="U?"  Part="1"
 AR Path="/6174477C/6577909A/65833EE7" Ref="U?"  Part="1"
-AR Path="/6174477C/656DAE2C/65833EE7" Ref="U15"  Part="1"
-F 0 "U15" H 6100 2711 50  0000 C CNN
+AR Path="/6174477C/656DAE2C/65833EE7" Ref="U17"  Part="1"
+F 0 "U17" H 6100 2711 50  0000 C CNN
 F 1 "ATmega328PB-MU" H 6100 2620 50  0000 C CNN
 F 2 "Package_DFN_QFN:QFN-32-1EP_5x5mm_P0.5mm_EP3.1x3.1mm" H 6100 4300 50  0001 C CIN
@@
 AR Path="/6174477C/6572958C/65833DC0" Ref="C?"  Part="1"
 AR Path="/6174477C/6577909A/65833DC0" Ref="C?"  Part="1"
-AR Path="/6174477C/656DAE2C/65833DC0" Ref="C51"  Part="1"
-F 0 "C51" H 4442 2646 50  0000 L CNN
+AR Path="/6174477C/656DAE2C/65833DC0" Ref="C53"  Part="1"
+F 0 "C53" H 4442 2646 50  0000 L CNN
 F 1 "1uF" H 4442 2555 50  0000 L CNN
 F 2 "Capacitor_SMD:C_0603_1608Metric" H 4350 2600 50  0001 C CNN
@@
 AR Path="/6174477C/6572958C/65833ED4" Ref="C?"  Part="1"
 AR Path="/6174477C/6577909A/65833ED4" Ref="C?"  Part="1"
-AR Path="/6174477C/656DAE2C/65833ED4" Ref="C52"  Part="1"
-F 0 "C52" H 4792 2646 50  0000 L CNN
+AR Path="/6174477C/656DAE2C/65833ED4" Ref="C54"  Part="1"
+F 0 "C54" H 4792 2646 50  0000 L CNN
 F 1 "100nF" H 4792 2555 50  0000 L CNN
 F 2 "Capacitor_SMD:C_0402_1005Metric" H 4700 2600 50  0001 C CNN
@@
 AR Path="/6174477C/6572958C/6386EE31" Ref="#PWR?"  Part="1"
 AR Path="/6174477C/6577909A/6386EE31" Ref="#PWR?"  Part="1"
-AR Path="/6174477C/656DAE2C/6386EE31" Ref="#PWR0135"  Part="1"
-F 0 "#PWR0135" H 3500 2600 50  0001 C CNN
+AR Path="/6174477C/656DAE2C/6386EE31" Ref="#PWR0139"  Part="1"
+F 0 "#PWR0139" H 3500 2600 50  0001 C CNN
 F 1 "GND" H 3505 2677 50  0000 C CNN
 F 2 "" H 3500 2850 50  0001 C CNN
@@
 AR Path="/6174477C/6572958C/65833DF2" Ref="C?"  Part="1"
 AR Path="/6174477C/6577909A/65833DF2" Ref="C?"  Part="1"
-AR Path="/6174477C/656DAE2C/65833DF2" Ref="C54"  Part="1"
-F 0 "C54" H 8100 4600 50  0000 L CNN
+AR Path="/6174477C/656DAE2C/65833DF2" Ref="C56"  Part="1"
+F 0 "C56" H 8100 4600 50  0000 L CNN
 F 1 "22pF" H 8100 4500 50  0000 L CNN
 F 2 "Capacitor_SMD:C_0402_1005Metric" H 8400 4550 50  0001 C CNN
@@
 AR Path="/6174477C/6572958C/65833E99" Ref="C?"  Part="1"
 AR Path="/6174477C/6577909A/65833E99" Ref="C?"  Part="1"
-AR Path="/6174477C/656DAE2C/65833E99" Ref="C53"  Part="1"
-F 0 "C53" H 8100 4600 50  0000 L CNN
+AR Path="/6174477C/656DAE2C/65833E99" Ref="C55"  Part="1"
+F 0 "C55" H 8100 4600 50  0000 L CNN
 F 1 "22pF" H 8100 4500 50  0000 L CNN
 F 2 "Capacitor_SMD:C_0402_1005Metric" H 8000 4550 50  0001 C CNN
@@
 AR Path="/6174477C/6572958C/65833EA8" Ref="#PWR?"  Part="1"
 AR Path="/6174477C/6577909A/65833EA8" Ref="#PWR?"  Part="1"
-AR Path="/6174477C/656DAE2C/65833EA8" Ref="#PWR0143"  Part="1"
-F 0 "#PWR0143" H 8400 4450 50  0001 C CNN
+AR Path="/6174477C/656DAE2C/65833EA8" Ref="#PWR0147"  Part="1"
+F 0 "#PWR0147" H 8400 4450 50  0001 C CNN
 F 1 "GND" H 8405 4527 50  0000 C CNN
 F 2 "" H 8400 4700 50  0001 C CNN
@@
 AR Path="/6174477C/6572958C/65833EB5" Ref="#PWR?"  Part="1"
 AR Path="/6174477C/6577909A/65833EB5" Ref="#PWR?"  Part="1"
-AR Path="/6174477C/656DAE2C/65833EB5" Ref="#PWR0139"  Part="1"
-F 0 "#PWR0139" H 8000 4450 50  0001 C CNN
+AR Path="/6174477C/656DAE2C/65833EB5" Ref="#PWR0143"  Part="1"
+F 0 "#PWR0143" H 8000 4450 50  0001 C CNN
 F 1 "GND" H 8005 4527 50  0000 C CNN
 F 2 "" H 8000 4700 50  0001 C CNN
@@
 AR Path="/6174477C/6572958C/65833E0B" Ref="#PWR?"  Part="1"
 AR Path="/6174477C/6577909A/65833E0B" Ref="#PWR?"  Part="1"
-AR Path="/6174477C/656DAE2C/65833E0B" Ref="#PWR0140"  Part="1"
-F 0 "#PWR0140" H 8200 3950 50  0001 C CNN
+AR Path="/6174477C/656DAE2C/65833E0B" Ref="#PWR0144"  Part="1"
+F 0 "#PWR0144" H 8200 3950 50  0001 C CNN
 F 1 "GND" H 8205 4027 50  0000 C CNN
 F 2 "" H 8200 4200 50  0001 C CNN
@@
 AR Path="/6174477C/6572958C/65833E14" Ref="#PWR?"  Part="1"
 AR Path="/6174477C/6577909A/65833E14" Ref="#PWR?"  Part="1"
-AR Path="/6174477C/656DAE2C/65833E14" Ref="#PWR0141"  Part="1"
-F 0 "#PWR0141" H 8200 4150 50  0001 C CNN
+AR Path="/6174477C/656DAE2C/65833E14" Ref="#PWR0145"  Part="1"
+F 0 "#PWR0145" H 8200 4150 50  0001 C CNN
 F 1 "GND" H 8205 4227 50  0000 C CNN
 F 2 "" H 8200 4400 50  0001 C CNN
@@
 AR Path="/6174477C/6572958C/65833E1B" Ref="#PWR?"  Part="1"
 AR Path="/6174477C/6577909A/65833E1B" Ref="#PWR?"  Part="1"
-AR Path="/6174477C/656DAE2C/65833E1B" Ref="#PWR0134"  Part="1"
-F 0 "#PWR0134" H 3500 1650 50  0001 C CNN
+AR Path="/6174477C/656DAE2C/65833E1B" Ref="#PWR0138"  Part="1"
+F 0 "#PWR0138" H 3500 1650 50  0001 C CNN
 F 1 "+5V_A" H 3515 1973 50  0000 C CNN
 F 2 "" H 3500 1800 50  0001 C CNN
@@
 AR Path="/6174477C/6572958C/65833E2D" Ref="#PWR?"  Part="1"
 AR Path="/6174477C/6577909A/65833E2D" Ref="#PWR?"  Part="1"
-AR Path="/6174477C/656DAE2C/65833E2D" Ref="#PWR0137"  Part="1"
-F 0 "#PWR0137" H 4700 2600 50  0001 C CNN
+AR Path="/6174477C/656DAE2C/65833E2D" Ref="#PWR0141"  Part="1"
+F 0 "#PWR0141" H 4700 2600 50  0001 C CNN
 F 1 "GND" H 4705 2677 50  0000 C CNN
 F 2 "" H 4700 2850 50  0001 C CNN
@@
 AR Path="/6174477C/6572958C/65833E63" Ref="#PWR?"  Part="1"
 AR Path="/6174477C/6577909A/65833E63" Ref="#PWR?"  Part="1"
-AR Path="/6174477C/656DAE2C/65833E63" Ref="#PWR0136"  Part="1"
-F 0 "#PWR0136" H 4200 5300 50  0001 C CNN
+AR Path="/6174477C/656DAE2C/65833E63" Ref="#PWR0140"  Part="1"
+F 0 "#PWR0140" H 4200 5300 50  0001 C CNN
 F 1 "GND" H 4205 5377 50  0000 C CNN
 F 2 "" H 4200 5550 50  0001 C CNN
@@
 AR Path="/6174477C/6572958C/65833EF9" Ref="#PWR?"  Part="1"
 AR Path="/6174477C/6577909A/65833EF9" Ref="#PWR?"  Part="1"
-AR Path="/6174477C/656DAE2C/65833EF9" Ref="#PWR0142"  Part="1"
-F 0 "#PWR0142" H 8400 3100 50  0001 C CNN
+AR Path="/6174477C/656DAE2C/65833EF9" Ref="#PWR0146"  Part="1"
+F 0 "#PWR0146" H 8400 3100 50  0001 C CNN
 F 1 "GND" H 8405 3177 50  0000 C CNN
 F 2 "" H 8400 3350 50  0001 C CNN
@@
 AR Path="/6174477C/6572958C/65833DCE" Ref="#PWR?"  Part="1"
 AR Path="/6174477C/6577909A/65833DCE" Ref="#PWR?"  Part="1"
-AR Path="/6174477C/656DAE2C/65833DCE" Ref="#PWR0138"  Part="1"
-F 0 "#PWR0138" H 6100 5800 50  0001 C CNN
+AR Path="/6174477C/656DAE2C/65833DCE" Ref="#PWR0142"  Part="1"
+F 0 "#PWR0142" H 6100 5800 50  0001 C CNN
 F 1 "GND" H 6105 5877 50  0000 C CNN
 F 2 "" H 6100 6050 50  0001 C CNN
