File: ykts-payload/ykts-mcu-node4.sch (KiCad schematic (older format))
At the start: 12 parts

Commit message: Update nodes
Parts:
- D9: renamed from D?; value NODE0_STATUSLED -> NODE4_STATUSLED
- gave numbers to parts that had none: 11
Connections:
- net NODE0_PWR renamed NODE4_PWR
- net NODE0_RESET renamed NODE4_RESET
- net NODE0_RX renamed NODE4_RX
- net NODE0_TX renamed NODE4_TX
Other:
- note added: "MCU Node 4"
- note removed: "MCU Node 0"
