File: ykts-payload/ykts-mcu-node4.sch (KiCad schematic (older format))
At the start: 12 parts, among them J9 AVR-ISP-6, SW4 ADG802BRT, U17 ATmega328PB-MU, Y6 8 MHz

Commit message: Fixed annotations & sheet ordering
Parts:
- renumbered C40 to C44, C41 to C45, C42 to C46, C43 to C47, D9 to D13, J9 to J12, R68 to R81, R69 to R82, R70 to R83, SW4 to SW5, U17 to U18, Y6 to Y7

Commit message: Revision A2
Added debug power
Basic ESD protection on UART
MCP Reset from MCU
Parts:
- renumbered D13 to D12, J12 to J13, R81 to R85, R82 to R86, R83 to R87
Changed lines of the file:
@@
 $Descr A4 11693 8268
 encoding utf-8
-Sheet 6 18
+Sheet 7 18
 Title "YktSat Payload Module"
-Date "2021-10-02"
-Rev "A1"
+Date "2021-10-03"
+Rev "A2"
 Comp "Sakha Aerospace Systems, LLC"
 Comment1 ""
@@
 AR Path="/6174477C/637CB186/63916A83" Ref="#PWR?"  Part="1"
 AR Path="/6174477C/63801AEE/63916A83" Ref="#PWR?"  Part="1"
-AR Path="/6174477C/638385B6/63916A83" Ref="#PWR0129"  Part="1"
+AR Path="/6174477C/638385B6/63916A83" Ref="#PWR0131"  Part="1"
 AR Path="/6174477C/638DF123/63916A83" Ref="#PWR?"  Part="1"
-F 0 "#PWR0129" H 3500 2600 50  0001 C CNN
+F 0 "#PWR0131" H 3500 2600 50  0001 C CNN
 F 1 "GND" H 3505 2677 50  0000 C CNN
 F 2 "" H 3500 2850 50  0001 C CNN
@@
 AR Path="/6174477C/637CB186/63916A87" Ref="#PWR?"  Part="1"
 AR Path="/6174477C/63801AEE/63916A87" Ref="#PWR?"  Part="1"
-AR Path="/6174477C/638385B6/63916A87" Ref="#PWR0137"  Part="1"
+AR Path="/6174477C/638385B6/63916A87" Ref="#PWR0139"  Part="1"
 AR Path="/6174477C/638DF123/63916A87" Ref="#PWR?"  Part="1"
-F 0 "#PWR0137" H 8400 4450 50  0001 C CNN
+F 0 "#PWR0139" H 8400 4450 50  0001 C CNN
 F 1 "GND" H 8405 4527 50  0000 C CNN
 F 2 "" H 8400 4700 50  0001 C CNN
@@
 AR Path="/6174477C/637CB186/63916A88" Ref="#PWR?"  Part="1"
 AR Path="/6174477C/63801AEE/63916A88" Ref="#PWR?"  Part="1"
-AR Path="/6174477C/638385B6/63916A88" Ref="#PWR0133"  Part="1"
+AR Path="/6174477C/638385B6/63916A88" Ref="#PWR0135"  Part="1"
 AR Path="/6174477C/638DF123/63916A88" Ref="#PWR?"  Part="1"
-F 0 "#PWR0133" H 8000 4450 50  0001 C CNN
+F 0 "#PWR0135" H 8000 4450 50  0001 C CNN
 F 1 "GND" H 8005 4527 50  0000 C CNN
 F 2 "" H 8000 4700 50  0001 C CNN
@@
 AR Path="/6174477C/637CB186/63916A76" Ref="#PWR?"  Part="1"
 AR Path="/6174477C/63801AEE/63916A76" Ref="#PWR?"  Part="1"
-AR Path="/6174477C/638385B6/63916A76" Ref="#PWR0134"  Part="1"
+AR Path="/6174477C/638385B6/63916A76" Ref="#PWR0136"  Part="1"
 AR Path="/6174477C/638DF123/63916A76" Ref="#PWR?"  Part="1"
-F 0 "#PWR0134" H 8200 3950 50  0001 C CNN
+F 0 "#PWR0136" H 8200 3950 50  0001 C CNN
 F 1 "GND" H 8205 4027 50  0000 C CNN
 F 2 "" H 8200 4200 50  0001 C CNN
@@
 AR Path="/6174477C/637CB186/63916A77" Ref="#PWR?"  Part="1"
 AR Path="/6174477C/63801AEE/63916A77" Ref="#PWR?"  Part="1"
-AR Path="/6174477C/638385B6/63916A77" Ref="#PWR0135"  Part="1"
+AR Path="/6174477C/638385B6/63916A77" Ref="#PWR0137"  Part="1"
 AR Path="/6174477C/638DF123/63916A77" Ref="#PWR?"  Part="1"
-F 0 "#PWR0135" H 8200 4150 50  0001 C CNN
+F 0 "#PWR0137" H 8200 4150 50  0001 C CNN
 F 1 "GND" H 8205 4227 50  0000 C CNN
 F 2 "" H 8200 4400 50  0001 C CNN
@@
 AR Path="/6174477C/637CB186/6386EF3E" Ref="R?"  Part="1"
 AR Path="/6174477C/63801AEE/6386EF3E" Ref="R?"  Part="1"
-AR Path="/6174477C/638385B6/6386EF3E" Ref="R81"  Part="1"
+AR Path="/6174477C/638385B6/6386EF3E" Ref="R85"  Part="1"
 AR Path="/6174477C/638DF123/6386EF3E" Ref="R?"  Part="1"
-F 0 "R81" V 6754 4400 50  0000 C CNN
+F 0 "R85" V 6754 4400 50  0000 C CNN
 F 1 "20K" V 6845 4400 50  0000 C CNN
 F 2 "Resistor_SMD:R_0402_1005Metric" H 6950 4400 50  0001 C CNN
@@
 AR Path="/6174477C/637CB186/63916A78" Ref="#PWR?"  Part="1"
 AR Path="/6174477C/63801AEE/63916A78" Ref="#PWR?"  Part="1"
-AR Path="/6174477C/638385B6/63916A78" Ref="#PWR0128"  Part="1"
+AR Path="/6174477C/638385B6/63916A78" Ref="#PWR0130"  Part="1"
 AR Path="/6174477C/638DF123/63916A78" Ref="#PWR?"  Part="1"
-F 0 "#PWR0128" H 3500 1650 50  0001 C CNN
+F 0 "#PWR0130" H 3500 1650 50  0001 C CNN
 F 1 "+5V_A" H 3515 1973 50  0000 C CNN
 F 2 "" H 3500 1800 50  0001 C CNN
@@
 AR Path="/6174477C/637CB186/638383BD" Ref="#PWR?"  Part="1"
 AR Path="/6174477C/63801AEE/638383BD" Ref="#PWR?"  Part="1"
-AR Path="/6174477C/638385B6/638383BD" Ref="#PWR0131"  Part="1"
+AR Path="/6174477C/638385B6/638383BD" Ref="#PWR0133"  Part="1"
 AR Path="/6174477C/638DF123/638383BD" Ref="#PWR?"  Part="1"
-F 0 "#PWR0131" H 4550 2600 50  0001 C CNN
+F 0 "#PWR0133" H 4550 2600 50  0001 C CNN
 F 1 "GND" H 4555 2677 50  0000 C CNN
 F 2 "" H 4550 2850 50  0001 C CNN
@@
 AR Path="/6174477C/637CB186/63916A7B" Ref="R?"  Part="1"
 AR Path="/6174477C/63801AEE/63916A7B" Ref="R?"  Part="1"
-AR Path="/6174477C/638385B6/63916A7B" Ref="R82"  Part="1"
+AR Path="/6174477C/638385B6/63916A7B" Ref="R86"  Part="1"
 AR Path="/6174477C/638DF123/63916A7B" Ref="R?"  Part="1"
-F 0 "R82" V 8004 3950 50  0000 C CNN
+F 0 "R86" V 8004 3950 50  0000 C CNN
 F 1 "1M" V 8095 3950 50  0000 C CNN
 F 2 "Resistor_SMD:R_0402_1005Metric" H 8200 3950 50  0001 C CNN
@@
 AR Path="/6174477C/637CB186/63916A7C" Ref="J?"  Part="1"
 AR Path="/6174477C/63801AEE/63916A7C" Ref="J?"  Part="1"
-AR Path="/6174477C/638385B6/63916A7C" Ref="J12"  Part="1"
+AR Path="/6174477C/638385B6/63916A7C" Ref="J13"  Part="1"
 AR Path="/6174477C/638DF123/63916A7C" Ref="J?"  Part="1"
-F 0 "J12" H 3770 5146 50  0000 R CNN
+F 0 "J13" H 3770 5146 50  0000 R CNN
 F 1 "AVR-ISP-6" H 3770 5055 50  0000 R CNN
 F 2 "Connector_PinHeader_2.54mm:PinHeader_2x03_P2.54mm_Vertical" V 3850 5100 50  0001 C CNN
@@
 AR Path="/6174477C/637CB186/63916A7D" Ref="#PWR?"  Part="1"
 AR Path="/6174477C/63801AEE/63916A7D" Ref="#PWR?"  Part="1"
-AR Path="/6174477C/638385B6/63916A7D" Ref="#PWR0130"  Part="1"
+AR Path="/6174477C/638385B6/63916A7D" Ref="#PWR0132"  Part="1"
 AR Path="/6174477C/638DF123/63916A7D" Ref="#PWR?"  Part="1"
-F 0 "#PWR0130" H 4200 5300 50  0001 C CNN
+F 0 "#PWR0132" H 4200 5300 50  0001 C CNN
 F 1 "GND" H 4205 5377 50  0000 C CNN
 F 2 "" H 4200 5550 50  0001 C CNN
@@
 AR Path="/6174477C/637CB186/63916A7E" Ref="D?"  Part="1"
 AR Path="/6174477C/63801AEE/63916A7E" Ref="D?"  Part="1"
-AR Path="/6174477C/638385B6/63916A7E" Ref="D13"  Part="1"
+AR Path="/6174477C/638385B6/63916A7E" Ref="D12"  Part="1"
 AR Path="/6174477C/638DF123/63916A7E" Ref="D?"  Part="1"
-F 0 "D13" V 8439 2682 50  0000 R CNN
+F 0 "D12" V 8439 2682 50  0000 R CNN
 F 1 "NODE4_STATUSLED" V 8348 2682 50  0000 R CNN
 F 2 "LED_SMD:LED_0402_1005Metric" H 8400 2800 50  0001 C CNN
@@
 AR Path="/6174477C/637CB186/63916A7F" Ref="R?"  Part="1"
 AR Path="/6174477C/63801AEE/63916A7F" Ref="R?"  Part="1"
-AR Path="/6174477C/638385B6/63916A7F" Ref="R83"  Part="1"
+AR Path="/6174477C/638385B6/63916A7F" Ref="R87"  Part="1"
 AR Path="/6174477C/638DF123/63916A7F" Ref="R?"  Part="1"
-F 0 "R83" V 8204 3150 50  0000 C CNN
+F 0 "R87" V 8204 3150 50  0000 C CNN
 F 1 "1K" V 8295 3150 50  0000 C CNN
 F 2 "Resistor_SMD:R_0402_1005Metric" H 8400 3150 50  0001 C CNN
@@
 AR Path="/6174477C/637CB186/638383C3" Ref="#PWR?"  Part="1"
 AR Path="/6174477C/63801AEE/638383C3" Ref="#PWR?"  Part="1"
-AR Path="/6174477C/638385B6/638383C3" Ref="#PWR0136"  Part="1"
+AR Path="/6174477C/638385B6/638383C3" Ref="#PWR0138"  Part="1"
 AR Path="/6174477C/638DF123/638383C3" Ref="#PWR?"  Part="1"
-F 0 "#PWR0136" H 8400 3100 50  0001 C CNN
+F 0 "#PWR0138" H 8400 3100 50  0001 C CNN
 F 1 "GND" H 8405 3177 50  0000 C CNN
 F 2 "" H 8400 3350 50  0001 C CNN
@@
 AR Path="/6174477C/637CB186/63916A85" Ref="#PWR?"  Part="1"
 AR Path="/6174477C/63801AEE/63916A85" Ref="#PWR?"  Part="1"
-AR Path="/6174477C/638385B6/63916A85" Ref="#PWR0132"  Part="1"
+AR Path="/6174477C/638385B6/63916A85" Ref="#PWR0134"  Part="1"
 AR Path="/6174477C/638DF123/63916A85" Ref="#PWR?"  Part="1"
-F 0 "#PWR0132" H 6100 5800 50  0001 C CNN
+F 0 "#PWR0134" H 6100 5800 50  0001 C CNN
 F 1 "GND" H 6105 5877 50  0000 C CNN
 F 2 "" H 6100 6050 50  0001 C CNN

Commit message: Fix git
Connections:
- net +5V_A: no longer C44.1, C45.1, D12.2 (A), R85.2, U18.18 (AVCC), U18.20 (AREF), U18.4 (VCC)
- net at SW5.1 (D): now also C44.1, C45.1, D12.2 (A), R85.2, U18.18 (AVCC), U18.20 (AREF), U18.4 (VCC)

Commit message: Change node ISP connector footprint
Parts:
- J13: footprint Connector_PinHeader_2.54mm:PinHeader_2x03_P2.54mm_Vertical -> Connector_PinHeader_1.27mm:PinHeader_2x03_P1.27mm_Vertical_SMD
Changed lines of the file:
@@
 F 0 "J13" H 3770 5146 50  0000 R CNN
 F 1 "AVR-ISP-6" H 3770 5055 50  0000 R CNN
-F 2 "Connector_PinHeader_2.54mm:PinHeader_2x03_P2.54mm_Vertical" V 3850 5100 50  0001 C CNN
+F 2 "Connector_PinHeader_1.27mm:PinHeader_2x03_P1.27mm_Vertical_SMD" V 3850 5100 50  0001 C CNN
 F 3 " ~" H 2825 4500 50  0001 C CNN
 	1    4100 5050

Commit message: Revision B0
Added second supervisor, mega2560 -> mega128a
Parts:
- renumbered C44 to C55, C45 to C56, C46 to C57, C47 to C58, D12 to D14, J13 to J17, R85 to R63, R86 to R64, R87 to R65, U18 to U16, Y7 to Y9

Commit message: Revision B2
Hierarchal sheets for nodes
Partial PCB layout
Parts:
- renumbered C55 to C57, C56 to C58, C57 to C59, C58 to C60, U16 to U18
Changed lines of the file:
@@
 Sheet 7 18
 Title "YktSat Payload Module"
-Date "2021-10-22"
-Rev "B0"
+Date "2021-10-26"
+Rev "B1"
 Comp "Sakha Aerospace Systems, LLC"
 Comment1 ""
@@
 AR Path="/6174477C/6568C69E/65833EE0" Ref="U?"  Part="1"
 AR Path="/6174477C/656DAE2A/65833EE0" Ref="U?"  Part="1"
-AR Path="/6174477C/65729588/65833EE0" Ref="U16"  Part="1"
+AR Path="/6174477C/65729588/65833EE0" Ref="U18"  Part="1"
 AR Path="/6174477C/6572958C/65833EE0" Ref="U?"  Part="1"
 AR Path="/6174477C/6577909A/65833EE0" Ref="U?"  Part="1"
-F 0 "U16" H 6100 2711 50  0000 C CNN
+F 0 "U18" H 6100 2711 50  0000 C CNN
 F 1 "ATmega328PB-MU" H 6100 2620 50  0000 C CNN
 F 2 "Package_DFN_QFN:QFN-32-1EP_5x5mm_P0.5mm_EP3.1x3.1mm" H 6100 4300 50  0001 C CIN
@@
 AR Path="/6174477C/6568C69E/65833DBE" Ref="C?"  Part="1"
 AR Path="/6174477C/656DAE2A/65833DBE" Ref="C?"  Part="1"
-AR Path="/6174477C/65729588/65833DBE" Ref="C55"  Part="1"
+AR Path="/6174477C/65729588/65833DBE" Ref="C57"  Part="1"
 AR Path="/6174477C/6572958C/65833DBE" Ref="C?"  Part="1"
 AR Path="/6174477C/6577909A/65833DBE" Ref="C?"  Part="1"
-F 0 "C55" H 4442 2646 50  0000 L CNN
+F 0 "C57" H 4442 2646 50  0000 L CNN
 F 1 "1uF" H 4442 2555 50  0000 L CNN
 F 2 "Capacitor_SMD:C_0603_1608Metric" H 4350 2600 50  0001 C CNN
@@
 AR Path="/6174477C/6568C69E/65833ED3" Ref="C?"  Part="1"
 AR Path="/6174477C/656DAE2A/65833ED3" Ref="C?"  Part="1"
-AR Path="/6174477C/65729588/65833ED3" Ref="C56"  Part="1"
+AR Path="/6174477C/65729588/65833ED3" Ref="C58"  Part="1"
 AR Path="/6174477C/6572958C/65833ED3" Ref="C?"  Part="1"
 AR Path="/6174477C/6577909A/65833ED3" Ref="C?"  Part="1"
-F 0 "C56" H 4792 2646 50  0000 L CNN
+F 0 "C58" H 4792 2646 50  0000 L CNN
 F 1 "100nF" H 4792 2555 50  0000 L CNN
 F 2 "Capacitor_SMD:C_0402_1005Metric" H 4700 2600 50  0001 C CNN
@@
 AR Path="/6174477C/6568C69E/65833DEB" Ref="#PWR?"  Part="1"
 AR Path="/6174477C/656DAE2A/65833DEB" Ref="#PWR?"  Part="1"
-AR Path="/6174477C/65729588/65833DEB" Ref="#PWR0145"  Part="1"
+AR Path="/6174477C/65729588/65833DEB" Ref="#PWR0149"  Part="1"
 AR Path="/6174477C/6572958C/65833DEB" Ref="#PWR?"  Part="1"
 AR Path="/6174477C/6577909A/65833DEB" Ref="#PWR?"  Part="1"
-F 0 "#PWR0145" H 3500 2600 50  0001 C CNN
+F 0 "#PWR0149" H 3500 2600 50  0001 C CNN
 F 1 "GND" H 3505 2677 50  0000 C CNN
 F 2 "" H 3500 2850 50  0001 C CNN
@@
 AR Path="/6174477C/6568C69E/65833DF1" Ref="C?"  Part="1"
 AR Path="/6174477C/656DAE2A/65833DF1" Ref="C?"  Part="1"
-AR Path="/6174477C/65729588/65833DF1" Ref="C58"  Part="1"
+AR Path="/6174477C/65729588/65833DF1" Ref="C60"  Part="1"
 AR Path="/6174477C/6572958C/65833DF1" Ref="C?"  Part="1"
 AR Path="/6174477C/6577909A/65833DF1" Ref="C?"  Part="1"
-F 0 "C58" H 8100 4600 50  0000 L CNN
+F 0 "C60" H 8100 4600 50  0000 L CNN
 F 1 "22pF" H 8100 4500 50  0000 L CNN
 F 2 "Capacitor_SMD:C_0402_1005Metric" H 8400 4550 50  0001 C CNN
@@
 AR Path="/6174477C/6568C69E/65833E98" Ref="C?"  Part="1"
 AR Path="/6174477C/656DAE2A/65833E98" Ref="C?"  Part="1"
-AR Path="/6174477C/65729588/65833E98" Ref="C57"  Part="1"
+AR Path="/6174477C/65729588/65833E98" Ref="C59"  Part="1"
 AR Path="/6174477C/6572958C/65833E98" Ref="C?"  Part="1"
 AR Path="/6174477C/6577909A/65833E98" Ref="C?"  Part="1"
-F 0 "C57" H 8100 4600 50  0000 L CNN
+F 0 "C59" H 8100 4600 50  0000 L CNN
 F 1 "22pF" H 8100 4500 50  0000 L CNN
 F 2 "Capacitor_SMD:C_0402_1005Metric" H 8000 4550 50  0001 C CNN
@@
 AR Path="/6174477C/6568C69E/65833EAB" Ref="#PWR?"  Part="1"
 AR Path="/6174477C/656DAE2A/65833EAB" Ref="#PWR?"  Part="1"
-AR Path="/6174477C/65729588/65833EAB" Ref="#PWR0153"  Part="1"
+AR Path="/6174477C/65729588/65833EAB" Ref="#PWR0157"  Part="1"
 AR Path="/6174477C/6572958C/65833EAB" Ref="#PWR?"  Part="1"
 AR Path="/6174477C/6577909A/65833EAB" Ref="#PWR?"  Part="1"
-F 0 "#PWR0153" H 8400 4450 50  0001 C CNN
+F 0 "#PWR0157" H 8400 4450 50  0001 C CNN
 F 1 "GND" H 8405 4527 50  0000 C CNN
 F 2 "" H 8400 4700 50  0001 C CNN
@@
 AR Path="/6174477C/6568C69E/65833EBF" Ref="#PWR?"  Part="1"
 AR Path="/6174477C/656DAE2A/65833EBF" Ref="#PWR?"  Part="1"
-AR Path="/6174477C/65729588/65833EBF" Ref="#PWR0149"  Part="1"
+AR Path="/6174477C/65729588/65833EBF" Ref="#PWR0153"  Part="1"
 AR Path="/6174477C/6572958C/65833EBF" Ref="#PWR?"  Part="1"
 AR Path="/6174477C/6577909A/65833EBF" Ref="#PWR?"  Part="1"
-F 0 "#PWR0149" H 8000 4450 50  0001 C CNN
+F 0 "#PWR0153" H 8000 4450 50  0001 C CNN
 F 1 "GND" H 8005 4527 50  0000 C CNN
 F 2 "" H 8000 4700 50  0001 C CNN
@@
 AR Path="/6174477C/6568C69E/65833E07" Ref="#PWR?"  Part="1"
 AR Path="/6174477C/656DAE2A/65833E07" Ref="#PWR?"  Part="1"
-AR Path="/6174477C/65729588/65833E07" Ref="#PWR0150"  Part="1"
+AR Path="/6174477C/65729588/65833E07" Ref="#PWR0154"  Part="1"
 AR Path="/6174477C/6572958C/65833E07" Ref="#PWR?"  Part="1"
 AR Path="/6174477C/6577909A/65833E07" Ref="#PWR?"  Part="1"
-F 0 "#PWR0150" H 8200 3950 50  0001 C CNN
+F 0 "#PWR0154" H 8200 3950 50  0001 C CNN
 F 1 "GND" H 8205 4027 50  0000 C CNN
 F 2 "" H 8200 4200 50  0001 C CNN
@@
 AR Path="/6174477C/6568C69E/65833E1A" Ref="#PWR?"  Part="1"
 AR Path="/6174477C/656DAE2A/65833E1A" Ref="#PWR?"  Part="1"
-AR Path="/6174477C/65729588/65833E1A" Ref="#PWR0151"  Part="1"
+AR Path="/6174477C/65729588/65833E1A" Ref="#PWR0155"  Part="1"
 AR Path="/6174477C/6572958C/65833E1A" Ref="#PWR?"  Part="1"
 AR Path="/6174477C/6577909A/65833E1A" Ref="#PWR?"  Part="1"
-F 0 "#PWR0151" H 8200 4150 50  0001 C CNN
+F 0 "#PWR0155" H 8200 4150 50  0001 C CNN
 F 1 "GND" H 8205 4227 50  0000 C CNN
 F 2 "" H 8200 4400 50  0001 C CNN
@@
 AR Path="/6174477C/6568C69E/65833E1E" Ref="#PWR?"  Part="1"
 AR Path="/6174477C/656DAE2A/65833E1E" Ref="#PWR?"  Part="1"
-AR Path="/6174477C/65729588/65833E1E" Ref="#PWR0144"  Part="1"
+AR Path="/6174477C/65729588/65833E1E" Ref="#PWR0148"  Part="1"
 AR Path="/6174477C/6572958C/65833E1E" Ref="#PWR?"  Part="1"
 AR Path="/6174477C/6577909A/65833E1E" Ref="#PWR?"  Part="1"
-F 0 "#PWR0144" H 3500 1650 50  0001 C CNN
+F 0 "#PWR0148" H 3500 1650 50  0001 C CNN
 F 1 "+5V_A" H 3515 1973 50  0000 C CNN
 F 2 "" H 3500 1800 50  0001 C CNN
@@
 AR Path="/6174477C/6568C69E/65833E31" Ref="#PWR?"  Part="1"
 AR Path="/6174477C/656DAE2A/65833E31" Ref="#PWR?"  Part="1"
-AR Path="/6174477C/65729588/65833E31" Ref="#PWR0147"  Part="1"
+AR Path="/6174477C/65729588/65833E31" Ref="#PWR0151"  Part="1"
 AR Path="/6174477C/6572958C/65833E31" Ref="#PWR?"  Part="1"
 AR Path="/6174477C/6577909A/65833E31" Ref="#PWR?"  Part="1"
-F 0 "#PWR0147" H 4700 2600 50  0001 C CNN
+F 0 "#PWR0151" H 4700 2600 50  0001 C CNN
 F 1 "GND" H 4705 2677 50  0000 C CNN
 F 2 "" H 4700 2850 50  0001 C CNN
@@
 AR Path="/6174477C/6568C69E/65833E64" Ref="#PWR?"  Part="1"
 AR Path="/6174477C/656DAE2A/65833E64" Ref="#PWR?"  Part="1"
-AR Path="/6174477C/65729588/65833E64" Ref="#PWR0146"  Part="1"
+AR Path="/6174477C/65729588/65833E64" Ref="#PWR0150"  Part="1"
 AR Path="/6174477C/6572958C/65833E64" Ref="#PWR?"  Part="1"
 AR Path="/6174477C/6577909A/65833E64" Ref="#PWR?"  Part="1"
-F 0 "#PWR0146" H 4200 5300 50  0001 C CNN
+F 0 "#PWR0150" H 4200 5300 50  0001 C CNN
 F 1 "GND" H 4205 5377 50  0000 C CNN
 F 2 "" H 4200 5550 50  0001 C CNN
@@
 AR Path="/6174477C/6568C69E/65833EFB" Ref="#PWR?"  Part="1"
 AR Path="/6174477C/656DAE2A/65833EFB" Ref="#PWR?"  Part="1"
-AR Path="/6174477C/65729588/65833EFB" Ref="#PWR0152"  Part="1"
+AR Path="/6174477C/65729588/65833EFB" Ref="#PWR0156"  Part="1"
 AR Path="/6174477C/6572958C/65833EFB" Ref="#PWR?"  Part="1"
 AR Path="/6174477C/6577909A/65833EFB" Ref="#PWR?"  Part="1"
-F 0 "#PWR0152" H 8400 3100 50  0001 C CNN
+F 0 "#PWR0156" H 8400 3100 50  0001 C CNN
 F 1 "GND" H 8405 3177 50  0000 C CNN
 F 2 "" H 8400 3350 50  0001 C CNN
@@
 AR Path="/6174477C/6568C69E/65833DCD" Ref="#PWR?"  Part="1"
 AR Path="/6174477C/656DAE2A/65833DCD" Ref="#PWR?"  Part="1"
-AR Path="/6174477C/65729588/65833DCD" Ref="#PWR0148"  Part="1"
+AR Path="/6174477C/65729588/65833DCD" Ref="#PWR0152"  Part="1"
 AR Path="/6174477C/6572958C/65833DCD" Ref="#PWR?"  Part="1"
 AR Path="/6174477C/6577909A/65833DCD" Ref="#PWR?"  Part="1"
-F 0 "#PWR0148" H 6100 5800 50  0001 C CNN
+F 0 "#PWR0152" H 6100 5800 50  0001 C CNN
 F 1 "GND" H 6105 5877 50  0000 C CNN
 F 2 "" H 6100 6050 50  0001 C CNN
