File: ykts-payload/ykts-mcu-node5.sch (KiCad schematic (older format))
At the start: 12 parts

Commit message: Update nodes
Parts:
- D10: renamed from D?; value NODE0_STATUSLED -> NODE5_STATUSLED
- gave numbers to parts that had none: 11
Connections:
- net NODE0_PWR renamed NODE5_PWR
- net NODE0_RESET renamed NODE5_RESET
- net NODE0_RX renamed NODE5_RX
- net NODE0_TX renamed NODE5_TX
Other:
- note added: "MCU Node 5"
- note removed: "MCU Node 0"
