File: ykts-payload/ykts-mcu-node5.sch (KiCad schematic (older format))
At the start: 12 parts, among them J10 AVR-ISP-6, SW5 ADG802BRT, U18 ATmega328PB-MU, Y7 8 MHz

Commit message: Fixed annotations & sheet ordering
Parts:
- renumbered C44 to C48, C45 to C49, C46 to C50, C47 to C51, D10 to D14, J10 to J13, R71 to R84, R72 to R85, R73 to R86, SW5 to SW6, U18 to U19, Y7 to Y8

Commit message: Revision A2
Added debug power
Basic ESD protection on UART
MCP Reset from MCU
Parts:
- renumbered D14 to D13, J13 to J14, R84 to R88, R85 to R89, R86 to R90
Changed lines of the file:
@@
 $Descr A4 11693 8268
 encoding utf-8
-Sheet 7 18
+Sheet 8 18
 Title "YktSat Payload Module"
-Date "2021-10-02"
-Rev "A1"
+Date "2021-10-03"
+Rev "A2"
 Comp "Sakha Aerospace Systems, LLC"
 Comment1 ""
@@
 AR Path="/6174477C/63801AF0/6386F13E" Ref="#PWR?"  Part="1"
 AR Path="/6174477C/63801AEE/6386F13E" Ref="#PWR?"  Part="1"
-AR Path="/6174477C/638385B8/6386F13E" Ref="#PWR0139"  Part="1"
+AR Path="/6174477C/638385B8/6386F13E" Ref="#PWR0141"  Part="1"
 AR Path="/6174477C/638385BA/6386F13E" Ref="#PWR?"  Part="1"
 AR Path="/6174477C/638DF125/6386F13E" Ref="#PWR?"  Part="1"
-F 0 "#PWR0139" H 3500 2600 50  0001 C CNN
+F 0 "#PWR0141" H 3500 2600 50  0001 C CNN
 F 1 "GND" H 3505 2677 50  0000 C CNN
 F 2 "" H 3500 2850 50  0001 C CNN
@@
 AR Path="/6174477C/63801AF0/63916B8A" Ref="#PWR?"  Part="1"
 AR Path="/6174477C/63801AEE/63916B8A" Ref="#PWR?"  Part="1"
-AR Path="/6174477C/638385B8/63916B8A" Ref="#PWR0147"  Part="1"
+AR Path="/6174477C/638385B8/63916B8A" Ref="#PWR0149"  Part="1"
 AR Path="/6174477C/638385BA/63916B8A" Ref="#PWR?"  Part="1"
 AR Path="/6174477C/638DF125/63916B8A" Ref="#PWR?"  Part="1"
-F 0 "#PWR0147" H 8400 4450 50  0001 C CNN
+F 0 "#PWR0149" H 8400 4450 50  0001 C CNN
 F 1 "GND" H 8405 4527 50  0000 C CNN
 F 2 "" H 8400 4700 50  0001 C CNN
@@
 AR Path="/6174477C/63801AF0/6386F146" Ref="#PWR?"  Part="1"
 AR Path="/6174477C/63801AEE/6386F146" Ref="#PWR?"  Part="1"
-AR Path="/6174477C/638385B8/6386F146" Ref="#PWR0143"  Part="1"
+AR Path="/6174477C/638385B8/6386F146" Ref="#PWR0145"  Part="1"
 AR Path="/6174477C/638385BA/6386F146" Ref="#PWR?"  Part="1"
 AR Path="/6174477C/638DF125/6386F146" Ref="#PWR?"  Part="1"
-F 0 "#PWR0143" H 8000 4450 50  0001 C CNN
+F 0 "#PWR0145" H 8000 4450 50  0001 C CNN
 F 1 "GND" H 8005 4527 50  0000 C CNN
 F 2 "" H 8000 4700 50  0001 C CNN
@@
 AR Path="/6174477C/63801AF0/63916B7C" Ref="#PWR?"  Part="1"
 AR Path="/6174477C/63801AEE/63916B7C" Ref="#PWR?"  Part="1"
-AR Path="/6174477C/638385B8/63916B7C" Ref="#PWR0144"  Part="1"
+AR Path="/6174477C/638385B8/63916B7C" Ref="#PWR0146"  Part="1"
 AR Path="/6174477C/638385BA/63916B7C" Ref="#PWR?"  Part="1"
 AR Path="/6174477C/638DF125/63916B7C" Ref="#PWR?"  Part="1"
-F 0 "#PWR0144" H 8200 3950 50  0001 C CNN
+F 0 "#PWR0146" H 8200 3950 50  0001 C CNN
 F 1 "GND" H 8205 4027 50  0000 C CNN
 F 2 "" H 8200 4200 50  0001 C CNN
@@
 AR Path="/6174477C/63801AF0/63916B80" Ref="#PWR?"  Part="1"
 AR Path="/6174477C/63801AEE/63916B80" Ref="#PWR?"  Part="1"
-AR Path="/6174477C/638385B8/63916B80" Ref="#PWR0145"  Part="1"
+AR Path="/6174477C/638385B8/63916B80" Ref="#PWR0147"  Part="1"
 AR Path="/6174477C/638385BA/63916B80" Ref="#PWR?"  Part="1"
 AR Path="/6174477C/638DF125/63916B80" Ref="#PWR?"  Part="1"
-F 0 "#PWR0145" H 8200 4150 50  0001 C CNN
+F 0 "#PWR0147" H 8200 4150 50  0001 C CNN
 F 1 "GND" H 8205 4227 50  0000 C CNN
 F 2 "" H 8200 4400 50  0001 C CNN
@@
 AR Path="/6174477C/63801AF0/6386F044" Ref="R?"  Part="1"
 AR Path="/6174477C/63801AEE/6386F044" Ref="R?"  Part="1"
-AR Path="/6174477C/638385B8/6386F044" Ref="R84"  Part="1"
+AR Path="/6174477C/638385B8/6386F044" Ref="R88"  Part="1"
 AR Path="/6174477C/638385BA/6386F044" Ref="R?"  Part="1"
 AR Path="/6174477C/638DF125/6386F044" Ref="R?"  Part="1"
-F 0 "R84" V 6754 4400 50  0000 C CNN
+F 0 "R88" V 6754 4400 50  0000 C CNN
 F 1 "20K" V 6845 4400 50  0000 C CNN
 F 2 "Resistor_SMD:R_0402_1005Metric" H 6950 4400 50  0001 C CNN
@@
 AR Path="/6174477C/63801AF0/638383BC" Ref="#PWR?"  Part="1"
 AR Path="/6174477C/63801AEE/638383BC" Ref="#PWR?"  Part="1"
-AR Path="/6174477C/638385B8/638383BC" Ref="#PWR0138"  Part="1"
+AR Path="/6174477C/638385B8/638383BC" Ref="#PWR0140"  Part="1"
 AR Path="/6174477C/638385BA/638383BC" Ref="#PWR?"  Part="1"
 AR Path="/6174477C/638DF125/638383BC" Ref="#PWR?"  Part="1"
-F 0 "#PWR0138" H 3500 1650 50  0001 C CNN
+F 0 "#PWR0140" H 3500 1650 50  0001 C CNN
 F 1 "+5V_A" H 3515 1973 50  0000 C CNN
 F 2 "" H 3500 1800 50  0001 C CNN
@@
 AR Path="/6174477C/63801AF0/6386EE3B" Ref="#PWR?"  Part="1"
 AR Path="/6174477C/63801AEE/6386EE3B" Ref="#PWR?"  Part="1"
-AR Path="/6174477C/638385B8/6386EE3B" Ref="#PWR0141"  Part="1"
+AR Path="/6174477C/638385B8/6386EE3B" Ref="#PWR0143"  Part="1"
 AR Path="/6174477C/638385BA/6386EE3B" Ref="#PWR?"  Part="1"
 AR Path="/6174477C/638DF125/6386EE3B" Ref="#PWR?"  Part="1"
-F 0 "#PWR0141" H 4550 2600 50  0001 C CNN
+F 0 "#PWR0143" H 4550 2600 50  0001 C CNN
 F 1 "GND" H 4555 2677 50  0000 C CNN
 F 2 "" H 4550 2850 50  0001 C CNN
@@
 AR Path="/6174477C/63801AF0/6378772A" Ref="R?"  Part="1"
 AR Path="/6174477C/63801AEE/6378772A" Ref="R?"  Part="1"
-AR Path="/6174477C/638385B8/6378772A" Ref="R85"  Part="1"
+AR Path="/6174477C/638385B8/6378772A" Ref="R89"  Part="1"
 AR Path="/6174477C/638385BA/6378772A" Ref="R?"  Part="1"
 AR Path="/6174477C/638DF125/6378772A" Ref="R?"  Part="1"
-F 0 "R85" V 8004 3950 50  0000 C CNN
+F 0 "R89" V 8004 3950 50  0000 C CNN
 F 1 "1M" V 8095 3950 50  0000 C CNN
 F 2 "Resistor_SMD:R_0402_1005Metric" H 8200 3950 50  0001 C CNN
@@
 AR Path="/6174477C/63801AF0/63916B79" Ref="J?"  Part="1"
 AR Path="/6174477C/63801AEE/63916B79" Ref="J?"  Part="1"
-AR Path="/6174477C/638385B8/63916B79" Ref="J13"  Part="1"
+AR Path="/6174477C/638385B8/63916B79" Ref="J14"  Part="1"
 AR Path="/6174477C/638385BA/63916B79" Ref="J?"  Part="1"
 AR Path="/6174477C/638DF125/63916B79" Ref="J?"  Part="1"
-F 0 "J13" H 3770 5146 50  0000 R CNN
+F 0 "J14" H 3770 5146 50  0000 R CNN
 F 1 "AVR-ISP-6" H 3770 5055 50  0000 R CNN
 F 2 "Connector_PinHeader_2.54mm:PinHeader_2x03_P2.54mm_Vertical" V 3850 5100 50  0001 C CNN
@@
 AR Path="/6174477C/63801AF0/6378E8B1" Ref="#PWR?"  Part="1"
 AR Path="/6174477C/63801AEE/6378E8B1" Ref="#PWR?"  Part="1"
-AR Path="/6174477C/638385B8/6378E8B1" Ref="#PWR0140"  Part="1"
+AR Path="/6174477C/638385B8/6378E8B1" Ref="#PWR0142"  Part="1"
 AR Path="/6174477C/638385BA/6378E8B1" Ref="#PWR?"  Part="1"
 AR Path="/6174477C/638DF125/6378E8B1" Ref="#PWR?"  Part="1"
-F 0 "#PWR0140" H 4200 5300 50  0001 C CNN
+F 0 "#PWR0142" H 4200 5300 50  0001 C CNN
 F 1 "GND" H 4205 5377 50  0000 C CNN
 F 2 "" H 4200 5550 50  0001 C CNN
@@
 AR Path="/6174477C/63801AF0/63916B84" Ref="D?"  Part="1"
 AR Path="/6174477C/63801AEE/63916B84" Ref="D?"  Part="1"
-AR Path="/6174477C/638385B8/63916B84" Ref="D14"  Part="1"
+AR Path="/6174477C/638385B8/63916B84" Ref="D13"  Part="1"
 AR Path="/6174477C/638385BA/63916B84" Ref="D?"  Part="1"
 AR Path="/6174477C/638DF125/63916B84" Ref="D?"  Part="1"
-F 0 "D14" V 8439 2682 50  0000 R CNN
+F 0 "D13" V 8439 2682 50  0000 R CNN
 F 1 "NODE5_STATUSLED" V 8348 2682 50  0000 R CNN
 F 2 "LED_SMD:LED_0402_1005Metric" H 8400 2800 50  0001 C CNN
@@
 AR Path="/6174477C/63801AF0/63916B8C" Ref="R?"  Part="1"
 AR Path="/6174477C/63801AEE/63916B8C" Ref="R?"  Part="1"
-AR Path="/6174477C/638385B8/63916B8C" Ref="R86"  Part="1"
+AR Path="/6174477C/638385B8/63916B8C" Ref="R90"  Part="1"
 AR Path="/6174477C/638385BA/63916B8C" Ref="R?"  Part="1"
 AR Path="/6174477C/638DF125/63916B8C" Ref="R?"  Part="1"
-F 0 "R86" V 8204 3150 50  0000 C CNN
+F 0 "R90" V 8204 3150 50  0000 C CNN
 F 1 "1K" V 8295 3150 50  0000 C CNN
 F 2 "Resistor_SMD:R_0402_1005Metric" H 8400 3150 50  0001 C CNN
@@
 AR Path="/6174477C/63801AF0/63916B8D" Ref="#PWR?"  Part="1"
 AR Path="/6174477C/63801AEE/63916B8D" Ref="#PWR?"  Part="1"
-AR Path="/6174477C/638385B8/63916B8D" Ref="#PWR0146"  Part="1"
+AR Path="/6174477C/638385B8/63916B8D" Ref="#PWR0148"  Part="1"
 AR Path="/6174477C/638385BA/63916B8D" Ref="#PWR?"  Part="1"
 AR Path="/6174477C/638DF125/63916B8D" Ref="#PWR?"  Part="1"
-F 0 "#PWR0146" H 8400 3100 50  0001 C CNN
+F 0 "#PWR0148" H 8400 3100 50  0001 C CNN
 F 1 "GND" H 8405 3177 50  0000 C CNN
 F 2 "" H 8400 3350 50  0001 C CNN
@@
 AR Path="/6174477C/63801AF0/63916B81" Ref="#PWR?"  Part="1"
 AR Path="/6174477C/63801AEE/63916B81" Ref="#PWR?"  Part="1"
-AR Path="/6174477C/638385B8/63916B81" Ref="#PWR0142"  Part="1"
+AR Path="/6174477C/638385B8/63916B81" Ref="#PWR0144"  Part="1"
 AR Path="/6174477C/638385BA/63916B81" Ref="#PWR?"  Part="1"
 AR Path="/6174477C/638DF125/63916B81" Ref="#PWR?"  Part="1"
-F 0 "#PWR0142" H 6100 5800 50  0001 C CNN
+F 0 "#PWR0144" H 6100 5800 50  0001 C CNN
 F 1 "GND" H 6105 5877 50  0000 C CNN
 F 2 "" H 6100 6050 50  0001 C CNN

Commit message: Fix git
Connections:
- net +5V_A: no longer C48.1, C49.1, D13.2 (A), R88.2, U19.18 (AVCC), U19.20 (AREF), U19.4 (VCC)
- net at SW6.1 (D): now also C48.1, C49.1, D13.2 (A), R88.2, U19.18 (AVCC), U19.20 (AREF), U19.4 (VCC)

Commit message: Change node ISP connector footprint
Parts:
- J14: footprint Connector_PinHeader_2.54mm:PinHeader_2x03_P2.54mm_Vertical -> Connector_PinHeader_1.27mm:PinHeader_2x03_P1.27mm_Vertical_SMD
Changed lines of the file:
@@
 F 0 "J14" H 3770 5146 50  0000 R CNN
 F 1 "AVR-ISP-6" H 3770 5055 50  0000 R CNN
-F 2 "Connector_PinHeader_2.54mm:PinHeader_2x03_P2.54mm_Vertical" V 3850 5100 50  0001 C CNN
+F 2 "Connector_PinHeader_1.27mm:PinHeader_2x03_P1.27mm_Vertical_SMD" V 3850 5100 50  0001 C CNN
 F 3 " ~" H 2825 4500 50  0001 C CNN
 	1    4100 5050

Commit message: Revision B0
Added second supervisor, mega2560 -> mega128a
Parts:
- renumbered C48 to C59, C49 to C60, C50 to C61, C51 to C62, D13 to D15, J14 to J18, R88 to R66, R89 to R67, R90 to R68, U19 to U17, Y8 to Y10
Changed lines of the file:
@@
 Sheet 8 18
 Title "YktSat Payload Module"
-Date "2021-10-03"
-Rev "A3"
+Date "2021-10-22"
+Rev "B0"
 Comp "Sakha Aerospace Systems, LLC"
 Comment1 ""
@@
 AR Path="/6174477C/6572958C/65833EE8" Ref="U?"  Part="1"
 AR Path="/6174477C/6577909A/65833EE8" Ref="U?"  Part="1"
-AR Path="/6174477C/6572958A/65833EE8" Ref="U19"  Part="1"
-F 0 "U19" H 6100 2711 50  0000 C CNN
+AR Path="/6174477C/6572958A/65833EE8" Ref="U17"  Part="1"
+F 0 "U17" H 6100 2711 50  0000 C CNN
 F 1 "ATmega328PB-MU" H 6100 2620 50  0000 C CNN
 F 2 "Package_DFN_QFN:QFN-32-1EP_5x5mm_P0.5mm_EP3.1x3.1mm" H 6100 4300 50  0001 C CIN
@@
 AR Path="/6174477C/6572958C/65833DBD" Ref="C?"  Part="1"
 AR Path="/6174477C/6577909A/65833DBD" Ref="C?"  Part="1"
-AR Path="/6174477C/6572958A/65833DBD" Ref="C48"  Part="1"
-F 0 "C48" H 4442 2646 50  0000 L CNN
+AR Path="/6174477C/6572958A/65833DBD" Ref="C59"  Part="1"
+F 0 "C59" H 4442 2646 50  0000 L CNN
 F 1 "1uF" H 4442 2555 50  0000 L CNN
 F 2 "Capacitor_SMD:C_0603_1608Metric" H 4350 2600 50  0001 C CNN
@@
 AR Path="/6174477C/6572958C/65833ED6" Ref="C?"  Part="1"
 AR Path="/6174477C/6577909A/65833ED6" Ref="C?"  Part="1"
-AR Path="/6174477C/6572958A/65833ED6" Ref="C49"  Part="1"
-F 0 "C49" H 4792 2646 50  0000 L CNN
+AR Path="/6174477C/6572958A/65833ED6" Ref="C60"  Part="1"
+F 0 "C60" H 4792 2646 50  0000 L CNN
 F 1 "100nF" H 4792 2555 50  0000 L CNN
 F 2 "Capacitor_SMD:C_0402_1005Metric" H 4700 2600 50  0001 C CNN
@@
 AR Path="/6174477C/6572958C/65833DEC" Ref="#PWR?"  Part="1"
 AR Path="/6174477C/6577909A/65833DEC" Ref="#PWR?"  Part="1"
-AR Path="/6174477C/6572958A/65833DEC" Ref="#PWR0141"  Part="1"
-F 0 "#PWR0141" H 3500 2600 50  0001 C CNN
+AR Path="/6174477C/6572958A/65833DEC" Ref="#PWR0155"  Part="1"
+F 0 "#PWR0155" H 3500 2600 50  0001 C CNN
 F 1 "GND" H 3505 2677 50  0000 C CNN
 F 2 "" H 3500 2850 50  0001 C CNN
@@
 AR Path="/6174477C/6572958C/65833DF4" Ref="C?"  Part="1"
 AR Path="/6174477C/6577909A/65833DF4" Ref="C?"  Part="1"
-AR Path="/6174477C/6572958A/65833DF4" Ref="C51"  Part="1"
-F 0 "C51" H 8100 4600 50  0000 L CNN
+AR Path="/6174477C/6572958A/65833DF4" Ref="C62"  Part="1"
+F 0 "C62" H 8100 4600 50  0000 L CNN
 F 1 "22pF" H 8100 4500 50  0000 L CNN
 F 2 "Capacitor_SMD:C_0402_1005Metric" H 8400 4550 50  0001 C CNN
@@
 AR Path="/6174477C/6572958C/65833E9B" Ref="C?"  Part="1"
 AR Path="/6174477C/6577909A/65833E9B" Ref="C?"  Part="1"
-AR Path="/6174477C/6572958A/65833E9B" Ref="C50"  Part="1"
-F 0 "C50" H 8100 4600 50  0000 L CNN
+AR Path="/6174477C/6572958A/65833E9B" Ref="C61"  Part="1"
+F 0 "C61" H 8100 4600 50  0000 L CNN
 F 1 "22pF" H 8100 4500 50  0000 L CNN
 F 2 "Capacitor_SMD:C_0402_1005Metric" H 8000 4550 50  0001 C CNN
@@
 AR Path="/6174477C/6572958C/65833EA2" Ref="#PWR?"  Part="1"
 AR Path="/6174477C/6577909A/65833EA2" Ref="#PWR?"  Part="1"
-AR Path="/6174477C/6572958A/65833EA2" Ref="#PWR0149"  Part="1"
-F 0 "#PWR0149" H 8400 4450 50  0001 C CNN
+AR Path="/6174477C/6572958A/65833EA2" Ref="#PWR0163"  Part="1"
+F 0 "#PWR0163" H 8400 4450 50  0001 C CNN
 F 1 "GND" H 8405 4527 50  0000 C CNN
 F 2 "" H 8400 4700 50  0001 C CNN
@@
 AR Path="/6174477C/6572958C/65833EBE" Ref="#PWR?"  Part="1"
 AR Path="/6174477C/6577909A/65833EBE" Ref="#PWR?"  Part="1"
-AR Path="/6174477C/6572958A/65833EBE" Ref="#PWR0145"  Part="1"
-F 0 "#PWR0145" H 8000 4450 50  0001 C CNN
+AR Path="/6174477C/6572958A/65833EBE" Ref="#PWR0159"  Part="1"
+F 0 "#PWR0159" H 8000 4450 50  0001 C CNN
 F 1 "GND" H 8005 4527 50  0000 C CNN
 F 2 "" H 8000 4700 50  0001 C CNN
@@
 AR Path="/6174477C/6572958C/65833EC1" Ref="Y?"  Part="1"
 AR Path="/6174477C/6577909A/65833EC1" Ref="Y?"  Part="1"
-AR Path="/6174477C/6572958A/65833EC1" Ref="Y8"  Part="1"
-F 0 "Y8" H 8450 4350 50  0000 L CNN
+AR Path="/6174477C/6572958A/65833EC1" Ref="Y10"  Part="1"
+F 0 "Y10" H 8450 4350 50  0000 L CNN
 F 1 "8 MHz" H 8450 4250 50  0000 L CNN
 F 2 "Crystal:Crystal_SMD_2520-4Pin_2.5x2.0mm" H 8200 4300 50  0001 C CNN
@@
 AR Path="/6174477C/6572958C/65833DFD" Ref="#PWR?"  Part="1"
 AR Path="/6174477C/6577909A/65833DFD" Ref="#PWR?"  Part="1"
-AR Path="/6174477C/6572958A/65833DFD" Ref="#PWR0146"  Part="1"
-F 0 "#PWR0146" H 8200 3950 50  0001 C CNN
+AR Path="/6174477C/6572958A/65833DFD" Ref="#PWR0160"  Part="1"
+F 0 "#PWR0160" H 8200 3950 50  0001 C CNN
 F 1 "GND" H 8205 4027 50  0000 C CNN
 F 2 "" H 8200 4200 50  0001 C CNN
@@
 AR Path="/6174477C/6572958C/65833E13" Ref="#PWR?"  Part="1"
 AR Path="/6174477C/6577909A/65833E13" Ref="#PWR?"  Part="1"
-AR Path="/6174477C/6572958A/65833E13" Ref="#PWR0147"  Part="1"
-F 0 "#PWR0147" H 8200 4150 50  0001 C CNN
+AR Path="/6174477C/6572958A/65833E13" Ref="#PWR0161"  Part="1"
+F 0 "#PWR0161" H 8200 4150 50  0001 C CNN
 F 1 "GND" H 8205 4227 50  0000 C CNN
 F 2 "" H 8200 4400 50  0001 C CNN
@@
 AR Path="/6174477C/6572958C/65833DD7" Ref="R?"  Part="1"
 AR Path="/6174477C/6577909A/65833DD7" Ref="R?"  Part="1"
-AR Path="/6174477C/6572958A/65833DD7" Ref="R88"  Part="1"
-F 0 "R88" V 6754 4400 50  0000 C CNN
+AR Path="/6174477C/6572958A/65833DD7" Ref="R66"  Part="1"
+F 0 "R66" V 6754 4400 50  0000 C CNN
 F 1 "20K" V 6845 4400 50  0000 C CNN
 F 2 "Resistor_SMD:R_0402_1005Metric" H 6950 4400 50  0001 C CNN
@@
 AR Path="/6174477C/6572958C/65833E1D" Ref="#PWR?"  Part="1"
 AR Path="/6174477C/6577909A/65833E1D" Ref="#PWR?"  Part="1"
-AR Path="/6174477C/6572958A/65833E1D" Ref="#PWR0140"  Part="1"
-F 0 "#PWR0140" H 3500 1650 50  0001 C CNN
+AR Path="/6174477C/6572958A/65833E1D" Ref="#PWR0154"  Part="1"
+F 0 "#PWR0154" H 3500 1650 50  0001 C CNN
 F 1 "+5V_A" H 3515 1973 50  0000 C CNN
 F 2 "" H 3500 1800 50  0001 C CNN
@@
 AR Path="/6174477C/6572958C/65833E38" Ref="#PWR?"  Part="1"
 AR Path="/6174477C/6577909A/65833E38" Ref="#PWR?"  Part="1"
-AR Path="/6174477C/6572958A/65833E38" Ref="#PWR0143"  Part="1"
-F 0 "#PWR0143" H 4700 2600 50  0001 C CNN
+AR Path="/6174477C/6572958A/65833E38" Ref="#PWR0157"  Part="1"
+F 0 "#PWR0157" H 4700 2600 50  0001 C CNN
 F 1 "GND" H 4705 2677 50  0000 C CNN
 F 2 "" H 4700 2850 50  0001 C CNN
@@
 AR Path="/6174477C/6572958C/65833E41" Ref="R?"  Part="1"
 AR Path="/6174477C/6577909A/65833E41" Ref="R?"  Part="1"
-AR Path="/6174477C/6572958A/65833E41" Ref="R89"  Part="1"
-F 0 "R89" V 8004 3950 50  0000 C CNN
+AR Path="/6174477C/6572958A/65833E41" Ref="R67"  Part="1"
+F 0 "R67" V 8004 3950 50  0000 C CNN
 F 1 "1M" V 8095 3950 50  0000 C CNN
 F 2 "Resistor_SMD:R_0402_1005Metric" H 8200 3950 50  0001 C CNN
@@
 AR Path="/6174477C/6572958C/65833E49" Ref="J?"  Part="1"
 AR Path="/6174477C/6577909A/65833E49" Ref="J?"  Part="1"
-AR Path="/6174477C/6572958A/65833E49" Ref="J14"  Part="1"
-F 0 "J14" H 3770 5146 50  0000 R CNN
+AR Path="/6174477C/6572958A/65833E49" Ref="J18"  Part="1"
+F 0 "J18" H 3770 5146 50  0000 R CNN
 F 1 "AVR-ISP-6" H 3770 5055 50  0000 R CNN
 F 2 "Connector_PinHeader_1.27mm:PinHeader_2x03_P1.27mm_Vertical_SMD" V 3850 5100 50  0001 C CNN
@@
 AR Path="/6174477C/6572958C/65833E59" Ref="#PWR?"  Part="1"
 AR Path="/6174477C/6577909A/65833E59" Ref="#PWR?"  Part="1"
-AR Path="/6174477C/6572958A/65833E59" Ref="#PWR0142"  Part="1"
-F 0 "#PWR0142" H 4200 5300 50  0001 C CNN
+AR Path="/6174477C/6572958A/65833E59" Ref="#PWR0156"  Part="1"
+F 0 "#PWR0156" H 4200 5300 50  0001 C CNN
 F 1 "GND" H 4205 5377 50  0000 C CNN
 F 2 "" H 4200 5550 50  0001 C CNN
@@
 AR Path="/6174477C/6572958C/65833E6A" Ref="D?"  Part="1"
 AR Path="/6174477C/6577909A/65833E6A" Ref="D?"  Part="1"
-AR Path="/6174477C/6572958A/65833E6A" Ref="D13"  Part="1"
-F 0 "D13" V 8439 2682 50  0000 R CNN
+AR Path="/6174477C/6572958A/65833E6A" Ref="D15"  Part="1"
+F 0 "D15" V 8439 2682 50  0000 R CNN
 F 1 "NODE5_STATUSLED" V 8348 2682 50  0000 R CNN
 F 2 "LED_SMD:LED_0402_1005Metric" H 8400 2800 50  0001 C CNN
@@
 AR Path="/6174477C/6572958C/65833E82" Ref="R?"  Part="1"
 AR Path="/6174477C/6577909A/65833E82" Ref="R?"  Part="1"
-AR Path="/6174477C/6572958A/65833E82" Ref="R90"  Part="1"
-F 0 "R90" V 8204 3150 50  0000 C CNN
+AR Path="/6174477C/6572958A/65833E82" Ref="R68"  Part="1"
+F 0 "R68" V 8204 3150 50  0000 C CNN
 F 1 "1K" V 8295 3150 50  0000 C CNN
 F 2 "Resistor_SMD:R_0402_1005Metric" H 8400 3150 50  0001 C CNN
@@
 AR Path="/6174477C/6572958C/6391667E" Ref="#PWR?"  Part="1"
 AR Path="/6174477C/6577909A/6391667E" Ref="#PWR?"  Part="1"
-AR Path="/6174477C/6572958A/6391667E" Ref="#PWR0148"  Part="1"
-F 0 "#PWR0148" H 8400 3100 50  0001 C CNN
+AR Path="/6174477C/6572958A/6391667E" Ref="#PWR0162"  Part="1"
+F 0 "#PWR0162" H 8400 3100 50  0001 C CNN
 F 1 "GND" H 8405 3177 50  0000 C CNN
 F 2 "" H 8400 3350 50  0001 C CNN
@@
 AR Path="/6174477C/6572958C/65833DCC" Ref="#PWR?"  Part="1"
 AR Path="/6174477C/6577909A/65833DCC" Ref="#PWR?"  Part="1"
-AR Path="/6174477C/6572958A/65833DCC" Ref="#PWR0144"  Part="1"
-F 0 "#PWR0144" H 6100 5800 50  0001 C CNN
+AR Path="/6174477C/6572958A/65833DCC" Ref="#PWR0158"  Part="1"
+F 0 "#PWR0158" H 6100 5800 50  0001 C CNN
 F 1 "GND" H 6105 5877 50  0000 C CNN
 F 2 "" H 6100 6050 50  0001 C CNN
