File: ykts-payload/ykts-mcu-node5.sch (KiCad schematic (older format))
At the start: 12 parts, among them J18 AVR-ISP-6, SW6 ADG802BRT, U17 ATmega328PB-MU, Y10 8 MHz

Commit message: Revision B2
Hierarchal sheets for nodes
Partial PCB layout
Parts:
- renumbered C59 to C61, C60 to C62, C61 to C63, C62 to C64, U17 to U19
Changed lines of the file:
@@
 Sheet 8 18
 Title "YktSat Payload Module"
-Date "2021-10-22"
-Rev "B0"
+Date "2021-10-26"
+Rev "B1"
 Comp "Sakha Aerospace Systems, LLC"
 Comment1 ""
@@
 AR Path="/6174477C/6572958C/65833EE8" Ref="U?"  Part="1"
 AR Path="/6174477C/6577909A/65833EE8" Ref="U?"  Part="1"
-AR Path="/6174477C/6572958A/65833EE8" Ref="U17"  Part="1"
-F 0 "U17" H 6100 2711 50  0000 C CNN
+AR Path="/6174477C/6572958A/65833EE8" Ref="U19"  Part="1"
+F 0 "U19" H 6100 2711 50  0000 C CNN
 F 1 "ATmega328PB-MU" H 6100 2620 50  0000 C CNN
 F 2 "Package_DFN_QFN:QFN-32-1EP_5x5mm_P0.5mm_EP3.1x3.1mm" H 6100 4300 50  0001 C CIN
@@
 AR Path="/6174477C/6572958C/65833DBD" Ref="C?"  Part="1"
 AR Path="/6174477C/6577909A/65833DBD" Ref="C?"  Part="1"
-AR Path="/6174477C/6572958A/65833DBD" Ref="C59"  Part="1"
-F 0 "C59" H 4442 2646 50  0000 L CNN
+AR Path="/6174477C/6572958A/65833DBD" Ref="C61"  Part="1"
+F 0 "C61" H 4442 2646 50  0000 L CNN
 F 1 "1uF" H 4442 2555 50  0000 L CNN
 F 2 "Capacitor_SMD:C_0603_1608Metric" H 4350 2600 50  0001 C CNN
@@
 AR Path="/6174477C/6572958C/65833ED6" Ref="C?"  Part="1"
 AR Path="/6174477C/6577909A/65833ED6" Ref="C?"  Part="1"
-AR Path="/6174477C/6572958A/65833ED6" Ref="C60"  Part="1"
-F 0 "C60" H 4792 2646 50  0000 L CNN
+AR Path="/6174477C/6572958A/65833ED6" Ref="C62"  Part="1"
+F 0 "C62" H 4792 2646 50  0000 L CNN
 F 1 "100nF" H 4792 2555 50  0000 L CNN
 F 2 "Capacitor_SMD:C_0402_1005Metric" H 4700 2600 50  0001 C CNN
@@
 AR Path="/6174477C/6572958C/65833DEC" Ref="#PWR?"  Part="1"
 AR Path="/6174477C/6577909A/65833DEC" Ref="#PWR?"  Part="1"
-AR Path="/6174477C/6572958A/65833DEC" Ref="#PWR0155"  Part="1"
-F 0 "#PWR0155" H 3500 2600 50  0001 C CNN
+AR Path="/6174477C/6572958A/65833DEC" Ref="#PWR0159"  Part="1"
+F 0 "#PWR0159" H 3500 2600 50  0001 C CNN
 F 1 "GND" H 3505 2677 50  0000 C CNN
 F 2 "" H 3500 2850 50  0001 C CNN
@@
 AR Path="/6174477C/6572958C/65833DF4" Ref="C?"  Part="1"
 AR Path="/6174477C/6577909A/65833DF4" Ref="C?"  Part="1"
-AR Path="/6174477C/6572958A/65833DF4" Ref="C62"  Part="1"
-F 0 "C62" H 8100 4600 50  0000 L CNN
+AR Path="/6174477C/6572958A/65833DF4" Ref="C64"  Part="1"
+F 0 "C64" H 8100 4600 50  0000 L CNN
 F 1 "22pF" H 8100 4500 50  0000 L CNN
 F 2 "Capacitor_SMD:C_0402_1005Metric" H 8400 4550 50  0001 C CNN
@@
 AR Path="/6174477C/6572958C/65833E9B" Ref="C?"  Part="1"
 AR Path="/6174477C/6577909A/65833E9B" Ref="C?"  Part="1"
-AR Path="/6174477C/6572958A/65833E9B" Ref="C61"  Part="1"
-F 0 "C61" H 8100 4600 50  0000 L CNN
+AR Path="/6174477C/6572958A/65833E9B" Ref="C63"  Part="1"
+F 0 "C63" H 8100 4600 50  0000 L CNN
 F 1 "22pF" H 8100 4500 50  0000 L CNN
 F 2 "Capacitor_SMD:C_0402_1005Metric" H 8000 4550 50  0001 C CNN
@@
 AR Path="/6174477C/6572958C/65833EA2" Ref="#PWR?"  Part="1"
 AR Path="/6174477C/6577909A/65833EA2" Ref="#PWR?"  Part="1"
-AR Path="/6174477C/6572958A/65833EA2" Ref="#PWR0163"  Part="1"
-F 0 "#PWR0163" H 8400 4450 50  0001 C CNN
+AR Path="/6174477C/6572958A/65833EA2" Ref="#PWR0167"  Part="1"
+F 0 "#PWR0167" H 8400 4450 50  0001 C CNN
 F 1 "GND" H 8405 4527 50  0000 C CNN
 F 2 "" H 8400 4700 50  0001 C CNN
@@
 AR Path="/6174477C/6572958C/65833EBE" Ref="#PWR?"  Part="1"
 AR Path="/6174477C/6577909A/65833EBE" Ref="#PWR?"  Part="1"
-AR Path="/6174477C/6572958A/65833EBE" Ref="#PWR0159"  Part="1"
-F 0 "#PWR0159" H 8000 4450 50  0001 C CNN
+AR Path="/6174477C/6572958A/65833EBE" Ref="#PWR0163"  Part="1"
+F 0 "#PWR0163" H 8000 4450 50  0001 C CNN
 F 1 "GND" H 8005 4527 50  0000 C CNN
 F 2 "" H 8000 4700 50  0001 C CNN
@@
 AR Path="/6174477C/6572958C/65833DFD" Ref="#PWR?"  Part="1"
 AR Path="/6174477C/6577909A/65833DFD" Ref="#PWR?"  Part="1"
-AR Path="/6174477C/6572958A/65833DFD" Ref="#PWR0160"  Part="1"
-F 0 "#PWR0160" H 8200 3950 50  0001 C CNN
+AR Path="/6174477C/6572958A/65833DFD" Ref="#PWR0164"  Part="1"
+F 0 "#PWR0164" H 8200 3950 50  0001 C CNN
 F 1 "GND" H 8205 4027 50  0000 C CNN
 F 2 "" H 8200 4200 50  0001 C CNN
@@
 AR Path="/6174477C/6572958C/65833E13" Ref="#PWR?"  Part="1"
 AR Path="/6174477C/6577909A/65833E13" Ref="#PWR?"  Part="1"
-AR Path="/6174477C/6572958A/65833E13" Ref="#PWR0161"  Part="1"
-F 0 "#PWR0161" H 8200 4150 50  0001 C CNN
+AR Path="/6174477C/6572958A/65833E13" Ref="#PWR0165"  Part="1"
+F 0 "#PWR0165" H 8200 4150 50  0001 C CNN
 F 1 "GND" H 8205 4227 50  0000 C CNN
 F 2 "" H 8200 4400 50  0001 C CNN
@@
 AR Path="/6174477C/6572958C/65833E1D" Ref="#PWR?"  Part="1"
 AR Path="/6174477C/6577909A/65833E1D" Ref="#PWR?"  Part="1"
-AR Path="/6174477C/6572958A/65833E1D" Ref="#PWR0154"  Part="1"
-F 0 "#PWR0154" H 3500 1650 50  0001 C CNN
+AR Path="/6174477C/6572958A/65833E1D" Ref="#PWR0158"  Part="1"
+F 0 "#PWR0158" H 3500 1650 50  0001 C CNN
 F 1 "+5V_A" H 3515 1973 50  0000 C CNN
 F 2 "" H 3500 1800 50  0001 C CNN
@@
 AR Path="/6174477C/6572958C/65833E38" Ref="#PWR?"  Part="1"
 AR Path="/6174477C/6577909A/65833E38" Ref="#PWR?"  Part="1"
-AR Path="/6174477C/6572958A/65833E38" Ref="#PWR0157"  Part="1"
-F 0 "#PWR0157" H 4700 2600 50  0001 C CNN
+AR Path="/6174477C/6572958A/65833E38" Ref="#PWR0161"  Part="1"
+F 0 "#PWR0161" H 4700 2600 50  0001 C CNN
 F 1 "GND" H 4705 2677 50  0000 C CNN
 F 2 "" H 4700 2850 50  0001 C CNN
@@
 AR Path="/6174477C/6572958C/65833E59" Ref="#PWR?"  Part="1"
 AR Path="/6174477C/6577909A/65833E59" Ref="#PWR?"  Part="1"
-AR Path="/6174477C/6572958A/65833E59" Ref="#PWR0156"  Part="1"
-F 0 "#PWR0156" H 4200 5300 50  0001 C CNN
+AR Path="/6174477C/6572958A/65833E59" Ref="#PWR0160"  Part="1"
+F 0 "#PWR0160" H 4200 5300 50  0001 C CNN
 F 1 "GND" H 4205 5377 50  0000 C CNN
 F 2 "" H 4200 5550 50  0001 C CNN
@@
 AR Path="/6174477C/6572958C/6391667E" Ref="#PWR?"  Part="1"
 AR Path="/6174477C/6577909A/6391667E" Ref="#PWR?"  Part="1"
-AR Path="/6174477C/6572958A/6391667E" Ref="#PWR0162"  Part="1"
-F 0 "#PWR0162" H 8400 3100 50  0001 C CNN
+AR Path="/6174477C/6572958A/6391667E" Ref="#PWR0166"  Part="1"
+F 0 "#PWR0166" H 8400 3100 50  0001 C CNN
 F 1 "GND" H 8405 3177 50  0000 C CNN
 F 2 "" H 8400 3350 50  0001 C CNN
@@
 AR Path="/6174477C/6572958C/65833DCC" Ref="#PWR?"  Part="1"
 AR Path="/6174477C/6577909A/65833DCC" Ref="#PWR?"  Part="1"
-AR Path="/6174477C/6572958A/65833DCC" Ref="#PWR0158"  Part="1"
-F 0 "#PWR0158" H 6100 5800 50  0001 C CNN
+AR Path="/6174477C/6572958A/65833DCC" Ref="#PWR0162"  Part="1"
+F 0 "#PWR0162" H 6100 5800 50  0001 C CNN
 F 1 "GND" H 6105 5877 50  0000 C CNN
 F 2 "" H 6100 6050 50  0001 C CNN
