File: ykts-payload/ykts-mcu-node6.sch (KiCad schematic (older format))
At the start: 12 parts

Commit message: Update nodes
Parts:
- D11: renamed from D?; value NODE0_STATUSLED -> NODE6_STATUSLED
- gave numbers to parts that had none: 11
Connections:
- net NODE0_PWR renamed NODE6_PWR
- net NODE0_RESET renamed NODE6_RESET
- net NODE0_RX renamed NODE6_RX
- net NODE0_TX renamed NODE6_TX
Other:
- note added: "MCU Node 6"
- note removed: "MCU Node 0"
