File: ykts-payload/ykts-mcu-node6.sch (KiCad schematic (older format))
At the start: 12 parts, among them J11 AVR-ISP-6, SW6 ADG802BRT, U19 ATmega328PB-MU, Y8 8 MHz

Commit message: Fixed annotations & sheet ordering
Parts:
- renumbered C48 to C52, C49 to C53, C50 to C54, C51 to C55, D11 to D15, J11 to J14, R74 to R87, R75 to R88, R76 to R89, SW6 to SW7, U19 to U20, Y8 to Y9

Commit message: Revision A2
Added debug power
Basic ESD protection on UART
MCP Reset from MCU
Parts:
- renumbered D15 to D14, J14 to J15, R87 to R91, R88 to R92, R89 to R93
Changed lines of the file:
@@
 $Descr A4 11693 8268
 encoding utf-8
-Sheet 8 18
+Sheet 9 18
 Title "YktSat Payload Module"
-Date "2021-10-02"
-Rev "A1"
+Date "2021-10-03"
+Rev "A2"
 Comp "Sakha Aerospace Systems, LLC"
 Comment1 ""
@@
 AR Path="/6174477C/63801AEE/638383B3" Ref="#PWR?"  Part="1"
 AR Path="/6174477C/638385B8/638383B3" Ref="#PWR?"  Part="1"
-AR Path="/6174477C/638385BA/638383B3" Ref="#PWR0149"  Part="1"
+AR Path="/6174477C/638385BA/638383B3" Ref="#PWR0151"  Part="1"
 AR Path="/6174477C/638DF127/638383B3" Ref="#PWR?"  Part="1"
-F 0 "#PWR0149" H 3500 2600 50  0001 C CNN
+F 0 "#PWR0151" H 3500 2600 50  0001 C CNN
 F 1 "GND" H 3505 2677 50  0000 C CNN
 F 2 "" H 3500 2850 50  0001 C CNN
@@
 AR Path="/6174477C/63801AEE/63916C81" Ref="#PWR?"  Part="1"
 AR Path="/6174477C/638385B8/63916C81" Ref="#PWR?"  Part="1"
-AR Path="/6174477C/638385BA/63916C81" Ref="#PWR0157"  Part="1"
+AR Path="/6174477C/638385BA/63916C81" Ref="#PWR0159"  Part="1"
 AR Path="/6174477C/638DF127/63916C81" Ref="#PWR?"  Part="1"
-F 0 "#PWR0157" H 8400 4450 50  0001 C CNN
+F 0 "#PWR0159" H 8400 4450 50  0001 C CNN
 F 1 "GND" H 8405 4527 50  0000 C CNN
 F 2 "" H 8400 4700 50  0001 C CNN
@@
 AR Path="/6174477C/63801AEE/6386EE35" Ref="#PWR?"  Part="1"
 AR Path="/6174477C/638385B8/6386EE35" Ref="#PWR?"  Part="1"
-AR Path="/6174477C/638385BA/6386EE35" Ref="#PWR0153"  Part="1"
+AR Path="/6174477C/638385BA/6386EE35" Ref="#PWR0155"  Part="1"
 AR Path="/6174477C/638DF127/6386EE35" Ref="#PWR?"  Part="1"
-F 0 "#PWR0153" H 8000 4450 50  0001 C CNN
+F 0 "#PWR0155" H 8000 4450 50  0001 C CNN
 F 1 "GND" H 8005 4527 50  0000 C CNN
 F 2 "" H 8000 4700 50  0001 C CNN
@@
 AR Path="/6174477C/63801AEE/6386F140" Ref="#PWR?"  Part="1"
 AR Path="/6174477C/638385B8/6386F140" Ref="#PWR?"  Part="1"
-AR Path="/6174477C/638385BA/6386F140" Ref="#PWR0154"  Part="1"
+AR Path="/6174477C/638385BA/6386F140" Ref="#PWR0156"  Part="1"
 AR Path="/6174477C/638DF127/6386F140" Ref="#PWR?"  Part="1"
-F 0 "#PWR0154" H 8200 3950 50  0001 C CNN
+F 0 "#PWR0156" H 8200 3950 50  0001 C CNN
 F 1 "GND" H 8205 4027 50  0000 C CNN
 F 2 "" H 8200 4200 50  0001 C CNN
@@
 AR Path="/6174477C/63801AEE/63916C8B" Ref="#PWR?"  Part="1"
 AR Path="/6174477C/638385B8/63916C8B" Ref="#PWR?"  Part="1"
-AR Path="/6174477C/638385BA/63916C8B" Ref="#PWR0155"  Part="1"
+AR Path="/6174477C/638385BA/63916C8B" Ref="#PWR0157"  Part="1"
 AR Path="/6174477C/638DF127/63916C8B" Ref="#PWR?"  Part="1"
-F 0 "#PWR0155" H 8200 4150 50  0001 C CNN
+F 0 "#PWR0157" H 8200 4150 50  0001 C CNN
 F 1 "GND" H 8205 4227 50  0000 C CNN
 F 2 "" H 8200 4400 50  0001 C CNN
@@
 AR Path="/6174477C/63801AEE/63916C8E" Ref="R?"  Part="1"
 AR Path="/6174477C/638385B8/63916C8E" Ref="R?"  Part="1"
-AR Path="/6174477C/638385BA/63916C8E" Ref="R87"  Part="1"
+AR Path="/6174477C/638385BA/63916C8E" Ref="R91"  Part="1"
 AR Path="/6174477C/638DF127/63916C8E" Ref="R?"  Part="1"
-F 0 "R87" V 6754 4400 50  0000 C CNN
+F 0 "R91" V 6754 4400 50  0000 C CNN
 F 1 "20K" V 6845 4400 50  0000 C CNN
 F 2 "Resistor_SMD:R_0402_1005Metric" H 6950 4400 50  0001 C CNN
@@
 AR Path="/6174477C/63801AEE/63916C8C" Ref="#PWR?"  Part="1"
 AR Path="/6174477C/638385B8/63916C8C" Ref="#PWR?"  Part="1"
-AR Path="/6174477C/638385BA/63916C8C" Ref="#PWR0148"  Part="1"
+AR Path="/6174477C/638385BA/63916C8C" Ref="#PWR0150"  Part="1"
 AR Path="/6174477C/638DF127/63916C8C" Ref="#PWR?"  Part="1"
-F 0 "#PWR0148" H 3500 1650 50  0001 C CNN
+F 0 "#PWR0150" H 3500 1650 50  0001 C CNN
 F 1 "+5V_A" H 3515 1973 50  0000 C CNN
 F 2 "" H 3500 1800 50  0001 C CNN
@@
 AR Path="/6174477C/63801AEE/63916C8F" Ref="#PWR?"  Part="1"
 AR Path="/6174477C/638385B8/63916C8F" Ref="#PWR?"  Part="1"
-AR Path="/6174477C/638385BA/63916C8F" Ref="#PWR0151"  Part="1"
+AR Path="/6174477C/638385BA/63916C8F" Ref="#PWR0153"  Part="1"
 AR Path="/6174477C/638DF127/63916C8F" Ref="#PWR?"  Part="1"
-F 0 "#PWR0151" H 4550 2600 50  0001 C CNN
+F 0 "#PWR0153" H 4550 2600 50  0001 C CNN
 F 1 "GND" H 4555 2677 50  0000 C CNN
 F 2 "" H 4550 2850 50  0001 C CNN
@@
 AR Path="/6174477C/63801AEE/6386F138" Ref="R?"  Part="1"
 AR Path="/6174477C/638385B8/6386F138" Ref="R?"  Part="1"
-AR Path="/6174477C/638385BA/6386F138" Ref="R88"  Part="1"
+AR Path="/6174477C/638385BA/6386F138" Ref="R92"  Part="1"
 AR Path="/6174477C/638DF127/6386F138" Ref="R?"  Part="1"
-F 0 "R88" V 8004 3950 50  0000 C CNN
+F 0 "R92" V 8004 3950 50  0000 C CNN
 F 1 "1M" V 8095 3950 50  0000 C CNN
 F 2 "Resistor_SMD:R_0402_1005Metric" H 8200 3950 50  0001 C CNN
@@
 AR Path="/6174477C/63801AEE/6386F139" Ref="J?"  Part="1"
 AR Path="/6174477C/638385B8/6386F139" Ref="J?"  Part="1"
-AR Path="/6174477C/638385BA/6386F139" Ref="J14"  Part="1"
+AR Path="/6174477C/638385BA/6386F139" Ref="J15"  Part="1"
 AR Path="/6174477C/638DF127/6386F139" Ref="J?"  Part="1"
-F 0 "J14" H 3770 5146 50  0000 R CNN
+F 0 "J15" H 3770 5146 50  0000 R CNN
 F 1 "AVR-ISP-6" H 3770 5055 50  0000 R CNN
 F 2 "Connector_PinHeader_2.54mm:PinHeader_2x03_P2.54mm_Vertical" V 3850 5100 50  0001 C CNN
@@
 AR Path="/6174477C/63801AEE/6386F13A" Ref="#PWR?"  Part="1"
 AR Path="/6174477C/638385B8/6386F13A" Ref="#PWR?"  Part="1"
-AR Path="/6174477C/638385BA/6386F13A" Ref="#PWR0150"  Part="1"
+AR Path="/6174477C/638385BA/6386F13A" Ref="#PWR0152"  Part="1"
 AR Path="/6174477C/638DF127/6386F13A" Ref="#PWR?"  Part="1"
-F 0 "#PWR0150" H 4200 5300 50  0001 C CNN
+F 0 "#PWR0152" H 4200 5300 50  0001 C CNN
 F 1 "GND" H 4205 5377 50  0000 C CNN
 F 2 "" H 4200 5550 50  0001 C CNN
@@
 AR Path="/6174477C/63801AEE/6386F149" Ref="D?"  Part="1"
 AR Path="/6174477C/638385B8/6386F149" Ref="D?"  Part="1"
-AR Path="/6174477C/638385BA/6386F149" Ref="D15"  Part="1"
+AR Path="/6174477C/638385BA/6386F149" Ref="D14"  Part="1"
 AR Path="/6174477C/638DF127/6386F149" Ref="D?"  Part="1"
-F 0 "D15" V 8439 2682 50  0000 R CNN
+F 0 "D14" V 8439 2682 50  0000 R CNN
 F 1 "NODE6_STATUSLED" V 8348 2682 50  0000 R CNN
 F 2 "LED_SMD:LED_0402_1005Metric" H 8400 2800 50  0001 C CNN
@@
 AR Path="/6174477C/63801AEE/63916C83" Ref="R?"  Part="1"
 AR Path="/6174477C/638385B8/63916C83" Ref="R?"  Part="1"
-AR Path="/6174477C/638385BA/63916C83" Ref="R89"  Part="1"
+AR Path="/6174477C/638385BA/63916C83" Ref="R93"  Part="1"
 AR Path="/6174477C/638DF127/63916C83" Ref="R?"  Part="1"
-F 0 "R89" V 8204 3150 50  0000 C CNN
+F 0 "R93" V 8204 3150 50  0000 C CNN
 F 1 "1K" V 8295 3150 50  0000 C CNN
 F 2 "Resistor_SMD:R_0402_1005Metric" H 8400 3150 50  0001 C CNN
@@
 AR Path="/6174477C/63801AEE/6386EE41" Ref="#PWR?"  Part="1"
 AR Path="/6174477C/638385B8/6386EE41" Ref="#PWR?"  Part="1"
-AR Path="/6174477C/638385BA/6386EE41" Ref="#PWR0156"  Part="1"
+AR Path="/6174477C/638385BA/6386EE41" Ref="#PWR0158"  Part="1"
 AR Path="/6174477C/638DF127/6386EE41" Ref="#PWR?"  Part="1"
-F 0 "#PWR0156" H 8400 3100 50  0001 C CNN
+F 0 "#PWR0158" H 8400 3100 50  0001 C CNN
 F 1 "GND" H 8405 3177 50  0000 C CNN
 F 2 "" H 8400 3350 50  0001 C CNN
@@
 AR Path="/6174477C/63801AEE/6386F143" Ref="#PWR?"  Part="1"
 AR Path="/6174477C/638385B8/6386F143" Ref="#PWR?"  Part="1"
-AR Path="/6174477C/638385BA/6386F143" Ref="#PWR0152"  Part="1"
+AR Path="/6174477C/638385BA/6386F143" Ref="#PWR0154"  Part="1"
 AR Path="/6174477C/638DF127/6386F143" Ref="#PWR?"  Part="1"
-F 0 "#PWR0152" H 6100 5800 50  0001 C CNN
+F 0 "#PWR0154" H 6100 5800 50  0001 C CNN
 F 1 "GND" H 6105 5877 50  0000 C CNN
 F 2 "" H 6100 6050 50  0001 C CNN

Commit message: Fix git
Connections:
- net +5V_A: no longer C52.1, C53.1, D14.2 (A), R91.2, U20.18 (AVCC), U20.20 (AREF), U20.4 (VCC)
- net at SW7.1 (D): now also C52.1, C53.1, D14.2 (A), R91.2, U20.18 (AVCC), U20.20 (AREF), U20.4 (VCC)

Commit message: Change node ISP connector footprint
Parts:
- J15: footprint Connector_PinHeader_2.54mm:PinHeader_2x03_P2.54mm_Vertical -> Connector_PinHeader_1.27mm:PinHeader_2x03_P1.27mm_Vertical_SMD
Changed lines of the file:
@@
 F 0 "J15" H 3770 5146 50  0000 R CNN
 F 1 "AVR-ISP-6" H 3770 5055 50  0000 R CNN
-F 2 "Connector_PinHeader_2.54mm:PinHeader_2x03_P2.54mm_Vertical" V 3850 5100 50  0001 C CNN
+F 2 "Connector_PinHeader_1.27mm:PinHeader_2x03_P1.27mm_Vertical_SMD" V 3850 5100 50  0001 C CNN
 F 3 " ~" H 2825 4500 50  0001 C CNN
 	1    4100 5050

Commit message: Revision B0
Added second supervisor, mega2560 -> mega128a
Parts:
- renumbered C52 to C63, C53 to C64, C54 to C65, C55 to C66, D14 to D16, J15 to J19, R91 to R69, R92 to R70, R93 to R71, U20 to U18, Y9 to Y11

Commit message: Revision B2
Hierarchal sheets for nodes
Partial PCB layout
Parts:
- renumbered C63 to C65, C64 to C66, C65 to C67, C66 to C68, U18 to U20
Changed lines of the file:
@@
 Sheet 9 18
 Title "YktSat Payload Module"
-Date "2021-10-22"
-Rev "B0"
+Date "2021-10-26"
+Rev "B1"
 Comp "Sakha Aerospace Systems, LLC"
 Comment1 ""
@@
 AR Path="/6174477C/656DAE2A/65833EE9" Ref="U?"  Part="1"
 AR Path="/6174477C/65729588/65833EE9" Ref="U?"  Part="1"
-AR Path="/6174477C/6572958C/65833EE9" Ref="U18"  Part="1"
+AR Path="/6174477C/6572958C/65833EE9" Ref="U20"  Part="1"
 AR Path="/6174477C/6577909A/65833EE9" Ref="U?"  Part="1"
-F 0 "U18" H 6100 2711 50  0000 C CNN
+F 0 "U20" H 6100 2711 50  0000 C CNN
 F 1 "ATmega328PB-MU" H 6100 2620 50  0000 C CNN
 F 2 "Package_DFN_QFN:QFN-32-1EP_5x5mm_P0.5mm_EP3.1x3.1mm" H 6100 4300 50  0001 C CIN
@@
 AR Path="/6174477C/656DAE2A/65833DBC" Ref="C?"  Part="1"
 AR Path="/6174477C/65729588/65833DBC" Ref="C?"  Part="1"
-AR Path="/6174477C/6572958C/65833DBC" Ref="C63"  Part="1"
+AR Path="/6174477C/6572958C/65833DBC" Ref="C65"  Part="1"
 AR Path="/6174477C/6577909A/65833DBC" Ref="C?"  Part="1"
-F 0 "C63" H 4442 2646 50  0000 L CNN
+F 0 "C65" H 4442 2646 50  0000 L CNN
 F 1 "1uF" H 4442 2555 50  0000 L CNN
 F 2 "Capacitor_SMD:C_0603_1608Metric" H 4350 2600 50  0001 C CNN
@@
 AR Path="/6174477C/656DAE2A/65833EDB" Ref="C?"  Part="1"
 AR Path="/6174477C/65729588/65833EDB" Ref="C?"  Part="1"
-AR Path="/6174477C/6572958C/65833EDB" Ref="C64"  Part="1"
+AR Path="/6174477C/6572958C/65833EDB" Ref="C66"  Part="1"
 AR Path="/6174477C/6577909A/65833EDB" Ref="C?"  Part="1"
-F 0 "C64" H 4792 2646 50  0000 L CNN
+F 0 "C66" H 4792 2646 50  0000 L CNN
 F 1 "100nF" H 4792 2555 50  0000 L CNN
 F 2 "Capacitor_SMD:C_0402_1005Metric" H 4700 2600 50  0001 C CNN
@@
 AR Path="/6174477C/656DAE2A/65833DDF" Ref="#PWR?"  Part="1"
 AR Path="/6174477C/65729588/65833DDF" Ref="#PWR?"  Part="1"
-AR Path="/6174477C/6572958C/65833DDF" Ref="#PWR0165"  Part="1"
+AR Path="/6174477C/6572958C/65833DDF" Ref="#PWR0169"  Part="1"
 AR Path="/6174477C/6577909A/65833DDF" Ref="#PWR?"  Part="1"
-F 0 "#PWR0165" H 3500 2600 50  0001 C CNN
+F 0 "#PWR0169" H 3500 2600 50  0001 C CNN
 F 1 "GND" H 3505 2677 50  0000 C CNN
 F 2 "" H 3500 2850 50  0001 C CNN
@@
 AR Path="/6174477C/656DAE2A/65833DEF" Ref="C?"  Part="1"
 AR Path="/6174477C/65729588/65833DEF" Ref="C?"  Part="1"
-AR Path="/6174477C/6572958C/65833DEF" Ref="C66"  Part="1"
+AR Path="/6174477C/6572958C/65833DEF" Ref="C68"  Part="1"
 AR Path="/6174477C/6577909A/65833DEF" Ref="C?"  Part="1"
-F 0 "C66" H 8100 4600 50  0000 L CNN
+F 0 "C68" H 8100 4600 50  0000 L CNN
 F 1 "22pF" H 8100 4500 50  0000 L CNN
 F 2 "Capacitor_SMD:C_0402_1005Metric" H 8400 4550 50  0001 C CNN
@@
 AR Path="/6174477C/656DAE2A/65833E9D" Ref="C?"  Part="1"
 AR Path="/6174477C/65729588/65833E9D" Ref="C?"  Part="1"
-AR Path="/6174477C/6572958C/65833E9D" Ref="C65"  Part="1"
+AR Path="/6174477C/6572958C/65833E9D" Ref="C67"  Part="1"
 AR Path="/6174477C/6577909A/65833E9D" Ref="C?"  Part="1"
-F 0 "C65" H 8100 4600 50  0000 L CNN
+F 0 "C67" H 8100 4600 50  0000 L CNN
 F 1 "22pF" H 8100 4500 50  0000 L CNN
 F 2 "Capacitor_SMD:C_0402_1005Metric" H 8000 4550 50  0001 C CNN
@@
 AR Path="/6174477C/656DAE2A/65833EA6" Ref="#PWR?"  Part="1"
 AR Path="/6174477C/65729588/65833EA6" Ref="#PWR?"  Part="1"
-AR Path="/6174477C/6572958C/65833EA6" Ref="#PWR0173"  Part="1"
+AR Path="/6174477C/6572958C/65833EA6" Ref="#PWR0177"  Part="1"
 AR Path="/6174477C/6577909A/65833EA6" Ref="#PWR?"  Part="1"
-F 0 "#PWR0173" H 8400 4450 50  0001 C CNN
+F 0 "#PWR0177" H 8400 4450 50  0001 C CNN
 F 1 "GND" H 8405 4527 50  0000 C CNN
 F 2 "" H 8400 4700 50  0001 C CNN
@@
 AR Path="/6174477C/656DAE2A/65833EBA" Ref="#PWR?"  Part="1"
 AR Path="/6174477C/65729588/65833EBA" Ref="#PWR?"  Part="1"
-AR Path="/6174477C/6572958C/65833EBA" Ref="#PWR0169"  Part="1"
+AR Path="/6174477C/6572958C/65833EBA" Ref="#PWR0173"  Part="1"
 AR Path="/6174477C/6577909A/65833EBA" Ref="#PWR?"  Part="1"
-F 0 "#PWR0169" H 8000 4450 50  0001 C CNN
+F 0 "#PWR0173" H 8000 4450 50  0001 C CNN
 F 1 "GND" H 8005 4527 50  0000 C CNN
 F 2 "" H 8000 4700 50  0001 C CNN
@@
 AR Path="/6174477C/656DAE2A/6386EE37" Ref="#PWR?"  Part="1"
 AR Path="/6174477C/65729588/6386EE37" Ref="#PWR?"  Part="1"
-AR Path="/6174477C/6572958C/6386EE37" Ref="#PWR0170"  Part="1"
+AR Path="/6174477C/6572958C/6386EE37" Ref="#PWR0174"  Part="1"
 AR Path="/6174477C/6577909A/6386EE37" Ref="#PWR?"  Part="1"
-F 0 "#PWR0170" H 8200 3950 50  0001 C CNN
+F 0 "#PWR0174" H 8200 3950 50  0001 C CNN
 F 1 "GND" H 8205 4027 50  0000 C CNN
 F 2 "" H 8200 4200 50  0001 C CNN
@@
 AR Path="/6174477C/656DAE2A/65833E10" Ref="#PWR?"  Part="1"
 AR Path="/6174477C/65729588/65833E10" Ref="#PWR?"  Part="1"
-AR Path="/6174477C/6572958C/65833E10" Ref="#PWR0171"  Part="1"
+AR Path="/6174477C/6572958C/65833E10" Ref="#PWR0175"  Part="1"
 AR Path="/6174477C/6577909A/65833E10" Ref="#PWR?"  Part="1"
-F 0 "#PWR0171" H 8200 4150 50  0001 C CNN
+F 0 "#PWR0175" H 8200 4150 50  0001 C CNN
 F 1 "GND" H 8205 4227 50  0000 C CNN
 F 2 "" H 8200 4400 50  0001 C CNN
@@
 AR Path="/6174477C/656DAE2A/65833E21" Ref="#PWR?"  Part="1"
 AR Path="/6174477C/65729588/65833E21" Ref="#PWR?"  Part="1"
-AR Path="/6174477C/6572958C/65833E21" Ref="#PWR0164"  Part="1"
+AR Path="/6174477C/6572958C/65833E21" Ref="#PWR0168"  Part="1"
 AR Path="/6174477C/6577909A/65833E21" Ref="#PWR?"  Part="1"
-F 0 "#PWR0164" H 3500 1650 50  0001 C CNN
+F 0 "#PWR0168" H 3500 1650 50  0001 C CNN
 F 1 "+5V_A" H 3515 1973 50  0000 C CNN
 F 2 "" H 3500 1800 50  0001 C CNN
@@
 AR Path="/6174477C/656DAE2A/65833E30" Ref="#PWR?"  Part="1"
 AR Path="/6174477C/65729588/65833E30" Ref="#PWR?"  Part="1"
-AR Path="/6174477C/6572958C/65833E30" Ref="#PWR0167"  Part="1"
+AR Path="/6174477C/6572958C/65833E30" Ref="#PWR0171"  Part="1"
 AR Path="/6174477C/6577909A/65833E30" Ref="#PWR?"  Part="1"
-F 0 "#PWR0167" H 4700 2600 50  0001 C CNN
+F 0 "#PWR0171" H 4700 2600 50  0001 C CNN
 F 1 "GND" H 4705 2677 50  0000 C CNN
 F 2 "" H 4700 2850 50  0001 C CNN
@@
 AR Path="/6174477C/656DAE2A/65833E62" Ref="#PWR?"  Part="1"
 AR Path="/6174477C/65729588/65833E62" Ref="#PWR?"  Part="1"
-AR Path="/6174477C/6572958C/65833E62" Ref="#PWR0166"  Part="1"
+AR Path="/6174477C/6572958C/65833E62" Ref="#PWR0170"  Part="1"
 AR Path="/6174477C/6577909A/65833E62" Ref="#PWR?"  Part="1"
-F 0 "#PWR0166" H 4200 5300 50  0001 C CNN
+F 0 "#PWR0170" H 4200 5300 50  0001 C CNN
 F 1 "GND" H 4205 5377 50  0000 C CNN
 F 2 "" H 4200 5550 50  0001 C CNN
@@
 AR Path="/6174477C/656DAE2A/65833EF6" Ref="#PWR?"  Part="1"
 AR Path="/6174477C/65729588/65833EF6" Ref="#PWR?"  Part="1"
-AR Path="/6174477C/6572958C/65833EF6" Ref="#PWR0172"  Part="1"
+AR Path="/6174477C/6572958C/65833EF6" Ref="#PWR0176"  Part="1"
 AR Path="/6174477C/6577909A/65833EF6" Ref="#PWR?"  Part="1"
-F 0 "#PWR0172" H 8400 3100 50  0001 C CNN
+F 0 "#PWR0176" H 8400 3100 50  0001 C CNN
 F 1 "GND" H 8405 3177 50  0000 C CNN
 F 2 "" H 8400 3350 50  0001 C CNN
@@
 AR Path="/6174477C/656DAE2A/65833DCB" Ref="#PWR?"  Part="1"
 AR Path="/6174477C/65729588/65833DCB" Ref="#PWR?"  Part="1"
-AR Path="/6174477C/6572958C/65833DCB" Ref="#PWR0168"  Part="1"
+AR Path="/6174477C/6572958C/65833DCB" Ref="#PWR0172"  Part="1"
 AR Path="/6174477C/6577909A/65833DCB" Ref="#PWR?"  Part="1"
-F 0 "#PWR0168" H 6100 5800 50  0001 C CNN
+F 0 "#PWR0172" H 6100 5800 50  0001 C CNN
 F 1 "GND" H 6105 5877 50  0000 C CNN
 F 2 "" H 6100 6050 50  0001 C CNN
