File: ykts-payload/ykts-mcu-node7.sch (KiCad schematic (older format))
At the start: 12 parts

Commit message: Update nodes
Parts:
- removed C?: 22pF, Capacitor_SMD:C_0402_1005Metric, symbol Device:C_Small
- removed R?: 20K, Resistor_SMD:R_0402_1005Metric, symbol Device:R_Small
- removed R?: 1K, Resistor_SMD:R_0402_1005Metric, symbol Device:R_Small
- removed Y?: 8 MHz, Crystal:Crystal_SMD_2520-4Pin_2.5x2.0mm, symbol Device:Crystal_GND24_Small
- added C55: 22pF, Capacitor_SMD:C_0402_1005Metric, symbol Device:C_Small
- added R77: 20K, Resistor_SMD:R_0402_1005Metric, symbol Device:R_Small
- added R79: 1K, Resistor_SMD:R_0402_1005Metric, symbol Device:R_Small
- added Y9: 8 MHz, Crystal:Crystal_SMD_2520-4Pin_2.5x2.0mm, symbol Device:Crystal_GND24_Small
- D12: renamed from D?; value NODE0_STATUSLED -> NODE7_STATUSLED
- gave numbers to parts that had none: 7
Connections:
- net +5V_A: now also R77.2
- net GND: now also C55.2, R79.1, Y9.2, Y9.4
- net at C54.1, R78.2, U20.8 (XTAL2/PB7): now also Y9.3
- net at R78.1, U20.7 (XTAL1/PB6): now also C55.1, Y9.1
- net at D12.1 (K): now also R79.2
- net NODE0_PWR renamed NODE7_PWR
- net NODE0_RESET renamed NODE7_RESET
- net NODE7_RESET: now also R77.1
- net NODE0_RX renamed NODE7_RX
- net NODE0_TX renamed NODE7_TX
Other:
- note added: "MCU Node 7"
- note removed: "MCU Node 0"
