File: ykts-payload/ykts-mcu-node7.sch (KiCad schematic (older format))
At the start: 12 parts, among them J12 AVR-ISP-6, SW7 ADG802BRT, U20 ATmega328PB-MU, Y9 8 MHz

Commit message: Fixed annotations & sheet ordering
Parts:
- renumbered C52 to C56, C53 to C57, C54 to C58, C55 to C59, D12 to D16, J12 to J15, R77 to R90, R78 to R91, R79 to R92, SW7 to SW8, U20 to U21, Y9 to Y10

Commit message: Revision A2
Added debug power
Basic ESD protection on UART
MCP Reset from MCU
Parts:
- renumbered D16 to D15, J15 to J16, R90 to R94, R91 to R95, R92 to R96
Changed lines of the file:
@@
 $Descr A4 11693 8268
 encoding utf-8
-Sheet 9 18
+Sheet 10 18
 Title "YktSat Payload Module"
-Date "2021-10-02"
-Rev "A1"
+Date "2021-10-03"
+Rev "A2"
 Comp "Sakha Aerospace Systems, LLC"
 Comment1 ""
@@
 AR Path="/6174477C/637CB186/6375CF10" Ref="#PWR?"  Part="1"
 AR Path="/6174477C/63801AF0/6375CF10" Ref="#PWR?"  Part="1"
-AR Path="/6174477C/638385BC/6375CF10" Ref="#PWR0159"  Part="1"
+AR Path="/6174477C/638385BC/6375CF10" Ref="#PWR0161"  Part="1"
 AR Path="/6174477C/638DF129/6375CF10" Ref="#PWR?"  Part="1"
-F 0 "#PWR0159" H 3500 2600 50  0001 C CNN
+F 0 "#PWR0161" H 3500 2600 50  0001 C CNN
 F 1 "GND" H 3505 2677 50  0000 C CNN
 F 2 "" H 3500 2850 50  0001 C CNN
@@
 AR Path="/6174477C/637CB186/63760B09" Ref="#PWR?"  Part="1"
 AR Path="/6174477C/63801AF0/63760B09" Ref="#PWR?"  Part="1"
-AR Path="/6174477C/638385BC/63760B09" Ref="#PWR0167"  Part="1"
+AR Path="/6174477C/638385BC/63760B09" Ref="#PWR0169"  Part="1"
 AR Path="/6174477C/638DF129/63760B09" Ref="#PWR?"  Part="1"
-F 0 "#PWR0167" H 8400 4450 50  0001 C CNN
+F 0 "#PWR0169" H 8400 4450 50  0001 C CNN
 F 1 "GND" H 8405 4527 50  0000 C CNN
 F 2 "" H 8400 4700 50  0001 C CNN
@@
 AR Path="/6174477C/637CB186/63760B0F" Ref="#PWR?"  Part="1"
 AR Path="/6174477C/63801AF0/63760B0F" Ref="#PWR?"  Part="1"
-AR Path="/6174477C/638385BC/63760B0F" Ref="#PWR0163"  Part="1"
+AR Path="/6174477C/638385BC/63760B0F" Ref="#PWR0165"  Part="1"
 AR Path="/6174477C/638DF129/63760B0F" Ref="#PWR?"  Part="1"
-F 0 "#PWR0163" H 8000 4450 50  0001 C CNN
+F 0 "#PWR0165" H 8000 4450 50  0001 C CNN
 F 1 "GND" H 8005 4527 50  0000 C CNN
 F 2 "" H 8000 4700 50  0001 C CNN
@@
 AR Path="/6174477C/637CB186/639B62C5" Ref="#PWR?"  Part="1"
 AR Path="/6174477C/63801AF0/639B62C5" Ref="#PWR?"  Part="1"
-AR Path="/6174477C/638385BC/639B62C5" Ref="#PWR0164"  Part="1"
+AR Path="/6174477C/638385BC/639B62C5" Ref="#PWR0166"  Part="1"
 AR Path="/6174477C/638DF129/639B62C5" Ref="#PWR?"  Part="1"
-F 0 "#PWR0164" H 8200 3950 50  0001 C CNN
+F 0 "#PWR0166" H 8200 3950 50  0001 C CNN
 F 1 "GND" H 8205 4027 50  0000 C CNN
 F 2 "" H 8200 4200 50  0001 C CNN
@@
 AR Path="/6174477C/637CB186/639B62C6" Ref="#PWR?"  Part="1"
 AR Path="/6174477C/63801AF0/639B62C6" Ref="#PWR?"  Part="1"
-AR Path="/6174477C/638385BC/639B62C6" Ref="#PWR0165"  Part="1"
+AR Path="/6174477C/638385BC/639B62C6" Ref="#PWR0167"  Part="1"
 AR Path="/6174477C/638DF129/639B62C6" Ref="#PWR?"  Part="1"
-F 0 "#PWR0165" H 8200 4150 50  0001 C CNN
+F 0 "#PWR0167" H 8200 4150 50  0001 C CNN
 F 1 "GND" H 8205 4227 50  0000 C CNN
 F 2 "" H 8200 4400 50  0001 C CNN
@@
 AR Path="/6174477C/637CB186/639B62C8" Ref="R?"  Part="1"
 AR Path="/6174477C/63801AF0/639B62C8" Ref="R?"  Part="1"
-AR Path="/6174477C/638385BC/639B62C8" Ref="R90"  Part="1"
+AR Path="/6174477C/638385BC/639B62C8" Ref="R94"  Part="1"
 AR Path="/6174477C/638DF129/639B62C8" Ref="R?"  Part="1"
-F 0 "R90" V 6754 4400 50  0000 C CNN
+F 0 "R94" V 6754 4400 50  0000 C CNN
 F 1 "20K" V 6845 4400 50  0000 C CNN
 F 2 "Resistor_SMD:R_0402_1005Metric" H 6950 4400 50  0001 C CNN
@@
 AR Path="/6174477C/637CB186/639B62CD" Ref="#PWR?"  Part="1"
 AR Path="/6174477C/63801AF0/639B62CD" Ref="#PWR?"  Part="1"
-AR Path="/6174477C/638385BC/639B62CD" Ref="#PWR0158"  Part="1"
+AR Path="/6174477C/638385BC/639B62CD" Ref="#PWR0160"  Part="1"
 AR Path="/6174477C/638DF129/639B62CD" Ref="#PWR?"  Part="1"
-F 0 "#PWR0158" H 3500 1650 50  0001 C CNN
+F 0 "#PWR0160" H 3500 1650 50  0001 C CNN
 F 1 "+5V_A" H 3515 1973 50  0000 C CNN
 F 2 "" H 3500 1800 50  0001 C CNN
@@
 AR Path="/6174477C/637CB186/63776BAF" Ref="#PWR?"  Part="1"
 AR Path="/6174477C/63801AF0/63776BAF" Ref="#PWR?"  Part="1"
-AR Path="/6174477C/638385BC/63776BAF" Ref="#PWR0161"  Part="1"
+AR Path="/6174477C/638385BC/63776BAF" Ref="#PWR0163"  Part="1"
 AR Path="/6174477C/638DF129/63776BAF" Ref="#PWR?"  Part="1"
-F 0 "#PWR0161" H 4550 2600 50  0001 C CNN
+F 0 "#PWR0163" H 4550 2600 50  0001 C CNN
 F 1 "GND" H 4555 2677 50  0000 C CNN
 F 2 "" H 4550 2850 50  0001 C CNN
@@
 AR Path="/6174477C/637CB186/6386EE3C" Ref="R?"  Part="1"
 AR Path="/6174477C/63801AF0/6386EE3C" Ref="R?"  Part="1"
-AR Path="/6174477C/638385BC/6386EE3C" Ref="R91"  Part="1"
+AR Path="/6174477C/638385BC/6386EE3C" Ref="R95"  Part="1"
 AR Path="/6174477C/638DF129/6386EE3C" Ref="R?"  Part="1"
-F 0 "R91" V 8004 3950 50  0000 C CNN
+F 0 "R95" V 8004 3950 50  0000 C CNN
 F 1 "1M" V 8095 3950 50  0000 C CNN
 F 2 "Resistor_SMD:R_0402_1005Metric" H 8200 3950 50  0001 C CNN
@@
 AR Path="/6174477C/637CB186/6386EE3D" Ref="J?"  Part="1"
 AR Path="/6174477C/63801AF0/6386EE3D" Ref="J?"  Part="1"
-AR Path="/6174477C/638385BC/6386EE3D" Ref="J15"  Part="1"
+AR Path="/6174477C/638385BC/6386EE3D" Ref="J16"  Part="1"
 AR Path="/6174477C/638DF129/6386EE3D" Ref="J?"  Part="1"
-F 0 "J15" H 3770 5146 50  0000 R CNN
+F 0 "J16" H 3770 5146 50  0000 R CNN
 F 1 "AVR-ISP-6" H 3770 5055 50  0000 R CNN
 F 2 "Connector_PinHeader_2.54mm:PinHeader_2x03_P2.54mm_Vertical" V 3850 5100 50  0001 C CNN
@@
 AR Path="/6174477C/637CB186/6386EE3E" Ref="#PWR?"  Part="1"
 AR Path="/6174477C/63801AF0/6386EE3E" Ref="#PWR?"  Part="1"
-AR Path="/6174477C/638385BC/6386EE3E" Ref="#PWR0160"  Part="1"
+AR Path="/6174477C/638385BC/6386EE3E" Ref="#PWR0162"  Part="1"
 AR Path="/6174477C/638DF129/6386EE3E" Ref="#PWR?"  Part="1"
-F 0 "#PWR0160" H 4200 5300 50  0001 C CNN
+F 0 "#PWR0162" H 4200 5300 50  0001 C CNN
 F 1 "GND" H 4205 5377 50  0000 C CNN
 F 2 "" H 4200 5550 50  0001 C CNN
@@
 AR Path="/6174477C/637CB186/6391656D" Ref="D?"  Part="1"
 AR Path="/6174477C/63801AF0/6391656D" Ref="D?"  Part="1"
-AR Path="/6174477C/638385BC/6391656D" Ref="D16"  Part="1"
+AR Path="/6174477C/638385BC/6391656D" Ref="D15"  Part="1"
 AR Path="/6174477C/638DF129/6391656D" Ref="D?"  Part="1"
-F 0 "D16" V 8439 2682 50  0000 R CNN
+F 0 "D15" V 8439 2682 50  0000 R CNN
 F 1 "NODE7_STATUSLED" V 8348 2682 50  0000 R CNN
 F 2 "LED_SMD:LED_0402_1005Metric" H 8400 2800 50  0001 C CNN
@@
 AR Path="/6174477C/637CB186/639B62CA" Ref="R?"  Part="1"
 AR Path="/6174477C/63801AF0/639B62CA" Ref="R?"  Part="1"
-AR Path="/6174477C/638385BC/639B62CA" Ref="R92"  Part="1"
+AR Path="/6174477C/638385BC/639B62CA" Ref="R96"  Part="1"
 AR Path="/6174477C/638DF129/639B62CA" Ref="R?"  Part="1"
-F 0 "R92" V 8204 3150 50  0000 C CNN
+F 0 "R96" V 8204 3150 50  0000 C CNN
 F 1 "1K" V 8295 3150 50  0000 C CNN
 F 2 "Resistor_SMD:R_0402_1005Metric" H 8400 3150 50  0001 C CNN
@@
 AR Path="/6174477C/637CB186/637997DF" Ref="#PWR?"  Part="1"
 AR Path="/6174477C/63801AF0/637997DF" Ref="#PWR?"  Part="1"
-AR Path="/6174477C/638385BC/637997DF" Ref="#PWR0166"  Part="1"
+AR Path="/6174477C/638385BC/637997DF" Ref="#PWR0168"  Part="1"
 AR Path="/6174477C/638DF129/637997DF" Ref="#PWR?"  Part="1"
-F 0 "#PWR0166" H 8400 3100 50  0001 C CNN
+F 0 "#PWR0168" H 8400 3100 50  0001 C CNN
 F 1 "GND" H 8405 3177 50  0000 C CNN
 F 2 "" H 8400 3350 50  0001 C CNN
@@
 AR Path="/6174477C/637CB186/63916578" Ref="#PWR?"  Part="1"
 AR Path="/6174477C/63801AF0/63916578" Ref="#PWR?"  Part="1"
-AR Path="/6174477C/638385BC/63916578" Ref="#PWR0162"  Part="1"
+AR Path="/6174477C/638385BC/63916578" Ref="#PWR0164"  Part="1"
 AR Path="/6174477C/638DF129/63916578" Ref="#PWR?"  Part="1"
-F 0 "#PWR0162" H 6100 5800 50  0001 C CNN
+F 0 "#PWR0164" H 6100 5800 50  0001 C CNN
 F 1 "GND" H 6105 5877 50  0000 C CNN
 F 2 "" H 6100 6050 50  0001 C CNN

Commit message: Fix git
Connections:
- net +5V_A: no longer C56.1, C57.1, D15.2 (A), R94.2, U21.18 (AVCC), U21.20 (AREF), U21.4 (VCC)
- net at SW8.1 (D): now also C56.1, C57.1, D15.2 (A), R94.2, U21.18 (AVCC), U21.20 (AREF), U21.4 (VCC)

Commit message: Change node ISP connector footprint
Parts:
- J16: footprint Connector_PinHeader_2.54mm:PinHeader_2x03_P2.54mm_Vertical -> Connector_PinHeader_1.27mm:PinHeader_2x03_P1.27mm_Vertical_SMD
Changed lines of the file:
@@
 F 0 "J16" H 3770 5146 50  0000 R CNN
 F 1 "AVR-ISP-6" H 3770 5055 50  0000 R CNN
-F 2 "Connector_PinHeader_2.54mm:PinHeader_2x03_P2.54mm_Vertical" V 3850 5100 50  0001 C CNN
+F 2 "Connector_PinHeader_1.27mm:PinHeader_2x03_P1.27mm_Vertical_SMD" V 3850 5100 50  0001 C CNN
 F 3 " ~" H 2825 4500 50  0001 C CNN
 	1    4100 5050

Commit message: Revision B0
Added second supervisor, mega2560 -> mega128a
Parts:
- renumbered C56 to C67, C57 to C68, C58 to C69, C59 to C70, D15 to D17, J16 to J20, R94 to R72, R95 to R73, R96 to R74, U21 to U19, Y10 to Y12
Changed lines of the file:
@@
 Sheet 10 18
 Title "YktSat Payload Module"
-Date "2021-10-03"
-Rev "A3"
+Date "2021-10-22"
+Rev "B0"
 Comp "Sakha Aerospace Systems, LLC"
 Comment1 ""
@@
 AR Path="/6174477C/6572958C/65833EEA" Ref="U?"  Part="1"
 AR Path="/6174477C/6577909A/65833EEA" Ref="U?"  Part="1"
-AR Path="/6174477C/6572958E/65833EEA" Ref="U21"  Part="1"
-F 0 "U21" H 6100 2711 50  0000 C CNN
+AR Path="/6174477C/6572958E/65833EEA" Ref="U19"  Part="1"
+F 0 "U19" H 6100 2711 50  0000 C CNN
 F 1 "ATmega328PB-MU" H 6100 2620 50  0000 C CNN
 F 2 "Package_DFN_QFN:QFN-32-1EP_5x5mm_P0.5mm_EP3.1x3.1mm" H 6100 4300 50  0001 C CIN
@@
 AR Path="/6174477C/6572958C/65833DBB" Ref="C?"  Part="1"
 AR Path="/6174477C/6577909A/65833DBB" Ref="C?"  Part="1"
-AR Path="/6174477C/6572958E/65833DBB" Ref="C56"  Part="1"
-F 0 "C56" H 4442 2646 50  0000 L CNN
+AR Path="/6174477C/6572958E/65833DBB" Ref="C67"  Part="1"
+F 0 "C67" H 4442 2646 50  0000 L CNN
 F 1 "1uF" H 4442 2555 50  0000 L CNN
 F 2 "Capacitor_SMD:C_0603_1608Metric" H 4350 2600 50  0001 C CNN
@@
 AR Path="/6174477C/6572958C/65833ED7" Ref="C?"  Part="1"
 AR Path="/6174477C/6577909A/65833ED7" Ref="C?"  Part="1"
-AR Path="/6174477C/6572958E/65833ED7" Ref="C57"  Part="1"
-F 0 "C57" H 4792 2646 50  0000 L CNN
+AR Path="/6174477C/6572958E/65833ED7" Ref="C68"  Part="1"
+F 0 "C68" H 4792 2646 50  0000 L CNN
 F 1 "100nF" H 4792 2555 50  0000 L CNN
 F 2 "Capacitor_SMD:C_0402_1005Metric" H 4700 2600 50  0001 C CNN
@@
 AR Path="/6174477C/6572958C/65833DE2" Ref="#PWR?"  Part="1"
 AR Path="/6174477C/6577909A/65833DE2" Ref="#PWR?"  Part="1"
-AR Path="/6174477C/6572958E/65833DE2" Ref="#PWR0161"  Part="1"
-F 0 "#PWR0161" H 3500 2600 50  0001 C CNN
+AR Path="/6174477C/6572958E/65833DE2" Ref="#PWR0175"  Part="1"
+F 0 "#PWR0175" H 3500 2600 50  0001 C CNN
 F 1 "GND" H 3505 2677 50  0000 C CNN
 F 2 "" H 3500 2850 50  0001 C CNN
@@
 AR Path="/6174477C/6572958C/65833DF3" Ref="C?"  Part="1"
 AR Path="/6174477C/6577909A/65833DF3" Ref="C?"  Part="1"
-AR Path="/6174477C/6572958E/65833DF3" Ref="C59"  Part="1"
-F 0 "C59" H 8100 4600 50  0000 L CNN
+AR Path="/6174477C/6572958E/65833DF3" Ref="C70"  Part="1"
+F 0 "C70" H 8100 4600 50  0000 L CNN
 F 1 "22pF" H 8100 4500 50  0000 L CNN
 F 2 "Capacitor_SMD:C_0402_1005Metric" H 8400 4550 50  0001 C CNN
@@
 AR Path="/6174477C/6572958C/65833E9E" Ref="C?"  Part="1"
 AR Path="/6174477C/6577909A/65833E9E" Ref="C?"  Part="1"
-AR Path="/6174477C/6572958E/65833E9E" Ref="C58"  Part="1"
-F 0 "C58" H 8100 4600 50  0000 L CNN
+AR Path="/6174477C/6572958E/65833E9E" Ref="C69"  Part="1"
+F 0 "C69" H 8100 4600 50  0000 L CNN
 F 1 "22pF" H 8100 4500 50  0000 L CNN
 F 2 "Capacitor_SMD:C_0402_1005Metric" H 8000 4550 50  0001 C CNN
@@
 AR Path="/6174477C/6572958C/65833EAE" Ref="#PWR?"  Part="1"
 AR Path="/6174477C/6577909A/65833EAE" Ref="#PWR?"  Part="1"
-AR Path="/6174477C/6572958E/65833EAE" Ref="#PWR0169"  Part="1"
-F 0 "#PWR0169" H 8400 4450 50  0001 C CNN
+AR Path="/6174477C/6572958E/65833EAE" Ref="#PWR0183"  Part="1"
+F 0 "#PWR0183" H 8400 4450 50  0001 C CNN
 F 1 "GND" H 8405 4527 50  0000 C CNN
 F 2 "" H 8400 4700 50  0001 C CNN
@@
 AR Path="/6174477C/6572958C/65833EB8" Ref="#PWR?"  Part="1"
 AR Path="/6174477C/6577909A/65833EB8" Ref="#PWR?"  Part="1"
-AR Path="/6174477C/6572958E/65833EB8" Ref="#PWR0165"  Part="1"
-F 0 "#PWR0165" H 8000 4450 50  0001 C CNN
+AR Path="/6174477C/6572958E/65833EB8" Ref="#PWR0179"  Part="1"
+F 0 "#PWR0179" H 8000 4450 50  0001 C CNN
 F 1 "GND" H 8005 4527 50  0000 C CNN
 F 2 "" H 8000 4700 50  0001 C CNN
@@
 AR Path="/6174477C/6572958C/65833EC9" Ref="Y?"  Part="1"
 AR Path="/6174477C/6577909A/65833EC9" Ref="Y?"  Part="1"
-AR Path="/6174477C/6572958E/65833EC9" Ref="Y10"  Part="1"
-F 0 "Y10" H 8450 4350 50  0000 L CNN
+AR Path="/6174477C/6572958E/65833EC9" Ref="Y12"  Part="1"
+F 0 "Y12" H 8450 4350 50  0000 L CNN
 F 1 "8 MHz" H 8450 4250 50  0000 L CNN
 F 2 "Crystal:Crystal_SMD_2520-4Pin_2.5x2.0mm" H 8200 4300 50  0001 C CNN
@@
 AR Path="/6174477C/6572958C/65833DFF" Ref="#PWR?"  Part="1"
 AR Path="/6174477C/6577909A/65833DFF" Ref="#PWR?"  Part="1"
-AR Path="/6174477C/6572958E/65833DFF" Ref="#PWR0166"  Part="1"
-F 0 "#PWR0166" H 8200 3950 50  0001 C CNN
+AR Path="/6174477C/6572958E/65833DFF" Ref="#PWR0180"  Part="1"
+F 0 "#PWR0180" H 8200 3950 50  0001 C CNN
 F 1 "GND" H 8205 4027 50  0000 C CNN
 F 2 "" H 8200 4200 50  0001 C CNN
@@
 AR Path="/6174477C/6572958C/65833E11" Ref="#PWR?"  Part="1"
 AR Path="/6174477C/6577909A/65833E11" Ref="#PWR?"  Part="1"
-AR Path="/6174477C/6572958E/65833E11" Ref="#PWR0167"  Part="1"
-F 0 "#PWR0167" H 8200 4150 50  0001 C CNN
+AR Path="/6174477C/6572958E/65833E11" Ref="#PWR0181"  Part="1"
+F 0 "#PWR0181" H 8200 4150 50  0001 C CNN
 F 1 "GND" H 8205 4227 50  0000 C CNN
 F 2 "" H 8200 4400 50  0001 C CNN
@@
 AR Path="/6174477C/6572958C/65833DDA" Ref="R?"  Part="1"
 AR Path="/6174477C/6577909A/65833DDA" Ref="R?"  Part="1"
-AR Path="/6174477C/6572958E/65833DDA" Ref="R94"  Part="1"
-F 0 "R94" V 6754 4400 50  0000 C CNN
+AR Path="/6174477C/6572958E/65833DDA" Ref="R72"  Part="1"
+F 0 "R72" V 6754 4400 50  0000 C CNN
 F 1 "20K" V 6845 4400 50  0000 C CNN
 F 2 "Resistor_SMD:R_0402_1005Metric" H 6950 4400 50  0001 C CNN
@@
 AR Path="/6174477C/6572958C/65833E22" Ref="#PWR?"  Part="1"
 AR Path="/6174477C/6577909A/65833E22" Ref="#PWR?"  Part="1"
-AR Path="/6174477C/6572958E/65833E22" Ref="#PWR0160"  Part="1"
-F 0 "#PWR0160" H 3500 1650 50  0001 C CNN
+AR Path="/6174477C/6572958E/65833E22" Ref="#PWR0174"  Part="1"
+F 0 "#PWR0174" H 3500 1650 50  0001 C CNN
 F 1 "+5V_A" H 3515 1973 50  0000 C CNN
 F 2 "" H 3500 1800 50  0001 C CNN
@@
 AR Path="/6174477C/6572958C/65833E2A" Ref="#PWR?"  Part="1"
 AR Path="/6174477C/6577909A/65833E2A" Ref="#PWR?"  Part="1"
-AR Path="/6174477C/6572958E/65833E2A" Ref="#PWR0163"  Part="1"
-F 0 "#PWR0163" H 4700 2600 50  0001 C CNN
+AR Path="/6174477C/6572958E/65833E2A" Ref="#PWR0177"  Part="1"
+F 0 "#PWR0177" H 4700 2600 50  0001 C CNN
 F 1 "GND" H 4705 2677 50  0000 C CNN
 F 2 "" H 4700 2850 50  0001 C CNN
@@
 AR Path="/6174477C/6572958C/65833E3F" Ref="R?"  Part="1"
 AR Path="/6174477C/6577909A/65833E3F" Ref="R?"  Part="1"
-AR Path="/6174477C/6572958E/65833E3F" Ref="R95"  Part="1"
-F 0 "R95" V 8004 3950 50  0000 C CNN
+AR Path="/6174477C/6572958E/65833E3F" Ref="R73"  Part="1"
+F 0 "R73" V 8004 3950 50  0000 C CNN
 F 1 "1M" V 8095 3950 50  0000 C CNN
 F 2 "Resistor_SMD:R_0402_1005Metric" H 8200 3950 50  0001 C CNN
@@
 AR Path="/6174477C/6572958C/65833E52" Ref="J?"  Part="1"
 AR Path="/6174477C/6577909A/65833E52" Ref="J?"  Part="1"
-AR Path="/6174477C/6572958E/65833E52" Ref="J16"  Part="1"
-F 0 "J16" H 3770 5146 50  0000 R CNN
+AR Path="/6174477C/6572958E/65833E52" Ref="J20"  Part="1"
+F 0 "J20" H 3770 5146 50  0000 R CNN
 F 1 "AVR-ISP-6" H 3770 5055 50  0000 R CNN
 F 2 "Connector_PinHeader_1.27mm:PinHeader_2x03_P1.27mm_Vertical_SMD" V 3850 5100 50  0001 C CNN
@@
 AR Path="/6174477C/6572958C/65833E61" Ref="#PWR?"  Part="1"
 AR Path="/6174477C/6577909A/65833E61" Ref="#PWR?"  Part="1"
-AR Path="/6174477C/6572958E/65833E61" Ref="#PWR0162"  Part="1"
-F 0 "#PWR0162" H 4200 5300 50  0001 C CNN
+AR Path="/6174477C/6572958E/65833E61" Ref="#PWR0176"  Part="1"
+F 0 "#PWR0176" H 4200 5300 50  0001 C CNN
 F 1 "GND" H 4205 5377 50  0000 C CNN
 F 2 "" H 4200 5550 50  0001 C CNN
@@
 AR Path="/6174477C/6572958C/65833E74" Ref="D?"  Part="1"
 AR Path="/6174477C/6577909A/65833E74" Ref="D?"  Part="1"
-AR Path="/6174477C/6572958E/65833E74" Ref="D15"  Part="1"
-F 0 "D15" V 8439 2682 50  0000 R CNN
+AR Path="/6174477C/6572958E/65833E74" Ref="D17"  Part="1"
+F 0 "D17" V 8439 2682 50  0000 R CNN
 F 1 "NODE7_STATUSLED" V 8348 2682 50  0000 R CNN
 F 2 "LED_SMD:LED_0402_1005Metric" H 8400 2800 50  0001 C CNN
@@
 AR Path="/6174477C/6572958C/65833E77" Ref="R?"  Part="1"
 AR Path="/6174477C/6577909A/65833E77" Ref="R?"  Part="1"
-AR Path="/6174477C/6572958E/65833E77" Ref="R96"  Part="1"
-F 0 "R96" V 8204 3150 50  0000 C CNN
+AR Path="/6174477C/6572958E/65833E77" Ref="R74"  Part="1"
+F 0 "R74" V 8204 3150 50  0000 C CNN
 F 1 "1K" V 8295 3150 50  0000 C CNN
 F 2 "Resistor_SMD:R_0402_1005Metric" H 8400 3150 50  0001 C CNN
@@
 AR Path="/6174477C/6572958C/65833EF7" Ref="#PWR?"  Part="1"
 AR Path="/6174477C/6577909A/65833EF7" Ref="#PWR?"  Part="1"
-AR Path="/6174477C/6572958E/65833EF7" Ref="#PWR0168"  Part="1"
-F 0 "#PWR0168" H 8400 3100 50  0001 C CNN
+AR Path="/6174477C/6572958E/65833EF7" Ref="#PWR0182"  Part="1"
+F 0 "#PWR0182" H 8400 3100 50  0001 C CNN
 F 1 "GND" H 8405 3177 50  0000 C CNN
 F 2 "" H 8400 3350 50  0001 C CNN
@@
 AR Path="/6174477C/6572958C/65833DCA" Ref="#PWR?"  Part="1"
 AR Path="/6174477C/6577909A/65833DCA" Ref="#PWR?"  Part="1"
-AR Path="/6174477C/6572958E/65833DCA" Ref="#PWR0164"  Part="1"
-F 0 "#PWR0164" H 6100 5800 50  0001 C CNN
+AR Path="/6174477C/6572958E/65833DCA" Ref="#PWR0178"  Part="1"
+F 0 "#PWR0178" H 6100 5800 50  0001 C CNN
 F 1 "GND" H 6105 5877 50  0000 C CNN
 F 2 "" H 6100 6050 50  0001 C CNN
