File: ykts-payload/ykts-mcu-node7.sch (KiCad schematic (older format))
At the start: 12 parts, among them J20 AVR-ISP-6, SW8 ADG802BRT, U19 ATmega328PB-MU, Y12 8 MHz

Commit message: Revision B2
Hierarchal sheets for nodes
Partial PCB layout
Parts:
- renumbered C67 to C69, C68 to C70, C69 to C71, C70 to C72, U19 to U21
Changed lines of the file:
@@
 Sheet 10 18
 Title "YktSat Payload Module"
-Date "2021-10-22"
-Rev "B0"
+Date "2021-10-26"
+Rev "B1"
 Comp "Sakha Aerospace Systems, LLC"
 Comment1 ""
@@
 AR Path="/6174477C/6572958C/65833EEA" Ref="U?"  Part="1"
 AR Path="/6174477C/6577909A/65833EEA" Ref="U?"  Part="1"
-AR Path="/6174477C/6572958E/65833EEA" Ref="U19"  Part="1"
-F 0 "U19" H 6100 2711 50  0000 C CNN
+AR Path="/6174477C/6572958E/65833EEA" Ref="U21"  Part="1"
+F 0 "U21" H 6100 2711 50  0000 C CNN
 F 1 "ATmega328PB-MU" H 6100 2620 50  0000 C CNN
 F 2 "Package_DFN_QFN:QFN-32-1EP_5x5mm_P0.5mm_EP3.1x3.1mm" H 6100 4300 50  0001 C CIN
@@
 AR Path="/6174477C/6572958C/65833DBB" Ref="C?"  Part="1"
 AR Path="/6174477C/6577909A/65833DBB" Ref="C?"  Part="1"
-AR Path="/6174477C/6572958E/65833DBB" Ref="C67"  Part="1"
-F 0 "C67" H 4442 2646 50  0000 L CNN
+AR Path="/6174477C/6572958E/65833DBB" Ref="C69"  Part="1"
+F 0 "C69" H 4442 2646 50  0000 L CNN
 F 1 "1uF" H 4442 2555 50  0000 L CNN
 F 2 "Capacitor_SMD:C_0603_1608Metric" H 4350 2600 50  0001 C CNN
@@
 AR Path="/6174477C/6572958C/65833ED7" Ref="C?"  Part="1"
 AR Path="/6174477C/6577909A/65833ED7" Ref="C?"  Part="1"
-AR Path="/6174477C/6572958E/65833ED7" Ref="C68"  Part="1"
-F 0 "C68" H 4792 2646 50  0000 L CNN
+AR Path="/6174477C/6572958E/65833ED7" Ref="C70"  Part="1"
+F 0 "C70" H 4792 2646 50  0000 L CNN
 F 1 "100nF" H 4792 2555 50  0000 L CNN
 F 2 "Capacitor_SMD:C_0402_1005Metric" H 4700 2600 50  0001 C CNN
@@
 AR Path="/6174477C/6572958C/65833DE2" Ref="#PWR?"  Part="1"
 AR Path="/6174477C/6577909A/65833DE2" Ref="#PWR?"  Part="1"
-AR Path="/6174477C/6572958E/65833DE2" Ref="#PWR0175"  Part="1"
-F 0 "#PWR0175" H 3500 2600 50  0001 C CNN
+AR Path="/6174477C/6572958E/65833DE2" Ref="#PWR0179"  Part="1"
+F 0 "#PWR0179" H 3500 2600 50  0001 C CNN
 F 1 "GND" H 3505 2677 50  0000 C CNN
 F 2 "" H 3500 2850 50  0001 C CNN
@@
 AR Path="/6174477C/6572958C/65833DF3" Ref="C?"  Part="1"
 AR Path="/6174477C/6577909A/65833DF3" Ref="C?"  Part="1"
-AR Path="/6174477C/6572958E/65833DF3" Ref="C70"  Part="1"
-F 0 "C70" H 8100 4600 50  0000 L CNN
+AR Path="/6174477C/6572958E/65833DF3" Ref="C72"  Part="1"
+F 0 "C72" H 8100 4600 50  0000 L CNN
 F 1 "22pF" H 8100 4500 50  0000 L CNN
 F 2 "Capacitor_SMD:C_0402_1005Metric" H 8400 4550 50  0001 C CNN
@@
 AR Path="/6174477C/6572958C/65833E9E" Ref="C?"  Part="1"
 AR Path="/6174477C/6577909A/65833E9E" Ref="C?"  Part="1"
-AR Path="/6174477C/6572958E/65833E9E" Ref="C69"  Part="1"
-F 0 "C69" H 8100 4600 50  0000 L CNN
+AR Path="/6174477C/6572958E/65833E9E" Ref="C71"  Part="1"
+F 0 "C71" H 8100 4600 50  0000 L CNN
 F 1 "22pF" H 8100 4500 50  0000 L CNN
 F 2 "Capacitor_SMD:C_0402_1005Metric" H 8000 4550 50  0001 C CNN
@@
 AR Path="/6174477C/6572958C/65833EAE" Ref="#PWR?"  Part="1"
 AR Path="/6174477C/6577909A/65833EAE" Ref="#PWR?"  Part="1"
-AR Path="/6174477C/6572958E/65833EAE" Ref="#PWR0183"  Part="1"
-F 0 "#PWR0183" H 8400 4450 50  0001 C CNN
+AR Path="/6174477C/6572958E/65833EAE" Ref="#PWR0187"  Part="1"
+F 0 "#PWR0187" H 8400 4450 50  0001 C CNN
 F 1 "GND" H 8405 4527 50  0000 C CNN
 F 2 "" H 8400 4700 50  0001 C CNN
@@
 AR Path="/6174477C/6572958C/65833EB8" Ref="#PWR?"  Part="1"
 AR Path="/6174477C/6577909A/65833EB8" Ref="#PWR?"  Part="1"
-AR Path="/6174477C/6572958E/65833EB8" Ref="#PWR0179"  Part="1"
-F 0 "#PWR0179" H 8000 4450 50  0001 C CNN
+AR Path="/6174477C/6572958E/65833EB8" Ref="#PWR0183"  Part="1"
+F 0 "#PWR0183" H 8000 4450 50  0001 C CNN
 F 1 "GND" H 8005 4527 50  0000 C CNN
 F 2 "" H 8000 4700 50  0001 C CNN
@@
 AR Path="/6174477C/6572958C/65833DFF" Ref="#PWR?"  Part="1"
 AR Path="/6174477C/6577909A/65833DFF" Ref="#PWR?"  Part="1"
-AR Path="/6174477C/6572958E/65833DFF" Ref="#PWR0180"  Part="1"
-F 0 "#PWR0180" H 8200 3950 50  0001 C CNN
+AR Path="/6174477C/6572958E/65833DFF" Ref="#PWR0184"  Part="1"
+F 0 "#PWR0184" H 8200 3950 50  0001 C CNN
 F 1 "GND" H 8205 4027 50  0000 C CNN
 F 2 "" H 8200 4200 50  0001 C CNN
@@
 AR Path="/6174477C/6572958C/65833E11" Ref="#PWR?"  Part="1"
 AR Path="/6174477C/6577909A/65833E11" Ref="#PWR?"  Part="1"
-AR Path="/6174477C/6572958E/65833E11" Ref="#PWR0181"  Part="1"
-F 0 "#PWR0181" H 8200 4150 50  0001 C CNN
+AR Path="/6174477C/6572958E/65833E11" Ref="#PWR0185"  Part="1"
+F 0 "#PWR0185" H 8200 4150 50  0001 C CNN
 F 1 "GND" H 8205 4227 50  0000 C CNN
 F 2 "" H 8200 4400 50  0001 C CNN
@@
 AR Path="/6174477C/6572958C/65833E22" Ref="#PWR?"  Part="1"
 AR Path="/6174477C/6577909A/65833E22" Ref="#PWR?"  Part="1"
-AR Path="/6174477C/6572958E/65833E22" Ref="#PWR0174"  Part="1"
-F 0 "#PWR0174" H 3500 1650 50  0001 C CNN
+AR Path="/6174477C/6572958E/65833E22" Ref="#PWR0178"  Part="1"
+F 0 "#PWR0178" H 3500 1650 50  0001 C CNN
 F 1 "+5V_A" H 3515 1973 50  0000 C CNN
 F 2 "" H 3500 1800 50  0001 C CNN
@@
 AR Path="/6174477C/6572958C/65833E2A" Ref="#PWR?"  Part="1"
 AR Path="/6174477C/6577909A/65833E2A" Ref="#PWR?"  Part="1"
-AR Path="/6174477C/6572958E/65833E2A" Ref="#PWR0177"  Part="1"
-F 0 "#PWR0177" H 4700 2600 50  0001 C CNN
+AR Path="/6174477C/6572958E/65833E2A" Ref="#PWR0181"  Part="1"
+F 0 "#PWR0181" H 4700 2600 50  0001 C CNN
 F 1 "GND" H 4705 2677 50  0000 C CNN
 F 2 "" H 4700 2850 50  0001 C CNN
@@
 AR Path="/6174477C/6572958C/65833E61" Ref="#PWR?"  Part="1"
 AR Path="/6174477C/6577909A/65833E61" Ref="#PWR?"  Part="1"
-AR Path="/6174477C/6572958E/65833E61" Ref="#PWR0176"  Part="1"
-F 0 "#PWR0176" H 4200 5300 50  0001 C CNN
+AR Path="/6174477C/6572958E/65833E61" Ref="#PWR0180"  Part="1"
+F 0 "#PWR0180" H 4200 5300 50  0001 C CNN
 F 1 "GND" H 4205 5377 50  0000 C CNN
 F 2 "" H 4200 5550 50  0001 C CNN
@@
 AR Path="/6174477C/6572958C/65833EF7" Ref="#PWR?"  Part="1"
 AR Path="/6174477C/6577909A/65833EF7" Ref="#PWR?"  Part="1"
-AR Path="/6174477C/6572958E/65833EF7" Ref="#PWR0182"  Part="1"
-F 0 "#PWR0182" H 8400 3100 50  0001 C CNN
+AR Path="/6174477C/6572958E/65833EF7" Ref="#PWR0186"  Part="1"
+F 0 "#PWR0186" H 8400 3100 50  0001 C CNN
 F 1 "GND" H 8405 3177 50  0000 C CNN
 F 2 "" H 8400 3350 50  0001 C CNN
@@
 AR Path="/6174477C/6572958C/65833DCA" Ref="#PWR?"  Part="1"
 AR Path="/6174477C/6577909A/65833DCA" Ref="#PWR?"  Part="1"
-AR Path="/6174477C/6572958E/65833DCA" Ref="#PWR0178"  Part="1"
-F 0 "#PWR0178" H 6100 5800 50  0001 C CNN
+AR Path="/6174477C/6572958E/65833DCA" Ref="#PWR0182"  Part="1"
+F 0 "#PWR0182" H 6100 5800 50  0001 C CNN
 F 1 "GND" H 6105 5877 50  0000 C CNN
 F 2 "" H 6100 6050 50  0001 C CNN
