File: ykts-payload/ykts-mcu-node9.sch (KiCad schematic (older format))
At the start: 12 parts

Commit message: Update nodes
Parts:
- D14: renamed from D?; value NODE0_STATUSLED -> NODE9_STATUSLED
- gave numbers to parts that had none: 11
Connections:
- net NODE0_PWR renamed NODE9_PWR
- net NODE0_RESET renamed NODE9_RESET
- net NODE0_RX renamed NODE9_RX
- net NODE0_TX renamed NODE9_TX
Other:
- note added: "MCU Node 9"
- note removed: "MCU Node 0"
