File: ykts-payload/ykts-mcu-node9.sch (KiCad schematic (older format))
At the start: 12 parts, among them J14 AVR-ISP-6, SW9 ADG802BRT, U22 ATmega328PB-MU, Y11 8 MHz

Commit message: Fixed annotations & sheet ordering
Parts:
- renumbered C60 to C64, C61 to C65, C62 to C66, C63 to C67, D14 to D18, J14 to J17, R83 to R96, R84 to R97, R85 to R98, SW9 to SW10, U22 to U23, Y11 to Y12

Commit message: Revision A2
Added debug power
Basic ESD protection on UART
MCP Reset from MCU
Parts:
- renumbered D18 to D17, J17 to J18, R96 to R100, R97 to R101, R98 to R102
Changed lines of the file:
@@
 $Descr A4 11693 8268
 encoding utf-8
-Sheet 11 18
+Sheet 12 18
 Title "YktSat Payload Module"
-Date "2021-10-02"
-Rev "A1"
+Date "2021-10-03"
+Rev "A2"
 Comp "Sakha Aerospace Systems, LLC"
 Comment1 ""
@@
 AR Path="/6174477C/638385B8/6386F03B" Ref="#PWR?"  Part="1"
 AR Path="/6174477C/638385BA/6386F03B" Ref="#PWR?"  Part="1"
-AR Path="/6174477C/638DF11D/6386F03B" Ref="#PWR0179"  Part="1"
+AR Path="/6174477C/638DF11D/6386F03B" Ref="#PWR0181"  Part="1"
 AR Path="/6174477C/638DF11F/6386F03B" Ref="#PWR?"  Part="1"
-F 0 "#PWR0179" H 3500 2600 50  0001 C CNN
+F 0 "#PWR0181" H 3500 2600 50  0001 C CNN
 F 1 "GND" H 3505 2677 50  0000 C CNN
 F 2 "" H 3500 2850 50  0001 C CNN
@@
 AR Path="/6174477C/638385B8/6386F042" Ref="#PWR?"  Part="1"
 AR Path="/6174477C/638385BA/6386F042" Ref="#PWR?"  Part="1"
-AR Path="/6174477C/638DF11D/6386F042" Ref="#PWR0187"  Part="1"
+AR Path="/6174477C/638DF11D/6386F042" Ref="#PWR0189"  Part="1"
 AR Path="/6174477C/638DF11F/6386F042" Ref="#PWR?"  Part="1"
-F 0 "#PWR0187" H 8400 4450 50  0001 C CNN
+F 0 "#PWR0189" H 8400 4450 50  0001 C CNN
 F 1 "GND" H 8405 4527 50  0000 C CNN
 F 2 "" H 8400 4700 50  0001 C CNN
@@
 AR Path="/6174477C/638385B8/6386F043" Ref="#PWR?"  Part="1"
 AR Path="/6174477C/638385BA/6386F043" Ref="#PWR?"  Part="1"
-AR Path="/6174477C/638DF11D/6386F043" Ref="#PWR0183"  Part="1"
+AR Path="/6174477C/638DF11D/6386F043" Ref="#PWR0185"  Part="1"
 AR Path="/6174477C/638DF11F/6386F043" Ref="#PWR?"  Part="1"
-F 0 "#PWR0183" H 8000 4450 50  0001 C CNN
+F 0 "#PWR0185" H 8000 4450 50  0001 C CNN
 F 1 "GND" H 8005 4527 50  0000 C CNN
 F 2 "" H 8000 4700 50  0001 C CNN
@@
 AR Path="/6174477C/638385B8/6386F03D" Ref="#PWR?"  Part="1"
 AR Path="/6174477C/638385BA/6386F03D" Ref="#PWR?"  Part="1"
-AR Path="/6174477C/638DF11D/6386F03D" Ref="#PWR0184"  Part="1"
+AR Path="/6174477C/638DF11D/6386F03D" Ref="#PWR0186"  Part="1"
 AR Path="/6174477C/638DF11F/6386F03D" Ref="#PWR?"  Part="1"
-F 0 "#PWR0184" H 8200 3950 50  0001 C CNN
+F 0 "#PWR0186" H 8200 3950 50  0001 C CNN
 F 1 "GND" H 8205 4027 50  0000 C CNN
 F 2 "" H 8200 4200 50  0001 C CNN
@@
 AR Path="/6174477C/638385B8/638383BA" Ref="#PWR?"  Part="1"
 AR Path="/6174477C/638385BA/638383BA" Ref="#PWR?"  Part="1"
-AR Path="/6174477C/638DF11D/638383BA" Ref="#PWR0185"  Part="1"
+AR Path="/6174477C/638DF11D/638383BA" Ref="#PWR0187"  Part="1"
 AR Path="/6174477C/638DF11F/638383BA" Ref="#PWR?"  Part="1"
-F 0 "#PWR0185" H 8200 4150 50  0001 C CNN
+F 0 "#PWR0187" H 8200 4150 50  0001 C CNN
 F 1 "GND" H 8205 4227 50  0000 C CNN
 F 2 "" H 8200 4400 50  0001 C CNN
@@
 AR Path="/6174477C/638385B8/63916872" Ref="R?"  Part="1"
 AR Path="/6174477C/638385BA/63916872" Ref="R?"  Part="1"
-AR Path="/6174477C/638DF11D/63916872" Ref="R96"  Part="1"
+AR Path="/6174477C/638DF11D/63916872" Ref="R100"  Part="1"
 AR Path="/6174477C/638DF11F/63916872" Ref="R?"  Part="1"
-F 0 "R96" V 6754 4400 50  0000 C CNN
+F 0 "R100" V 6754 4400 50  0000 C CNN
 F 1 "20K" V 6845 4400 50  0000 C CNN
 F 2 "Resistor_SMD:R_0402_1005Metric" H 6950 4400 50  0001 C CNN
@@
 AR Path="/6174477C/638385B8/6391677B" Ref="#PWR?"  Part="1"
 AR Path="/6174477C/638385BA/6391677B" Ref="#PWR?"  Part="1"
-AR Path="/6174477C/638DF11D/6391677B" Ref="#PWR0178"  Part="1"
+AR Path="/6174477C/638DF11D/6391677B" Ref="#PWR0180"  Part="1"
 AR Path="/6174477C/638DF11F/6391677B" Ref="#PWR?"  Part="1"
-F 0 "#PWR0178" H 3500 1650 50  0001 C CNN
+F 0 "#PWR0180" H 3500 1650 50  0001 C CNN
 F 1 "+5V_A" H 3515 1973 50  0000 C CNN
 F 2 "" H 3500 1800 50  0001 C CNN
@@
 AR Path="/6174477C/638385B8/6386F045" Ref="#PWR?"  Part="1"
 AR Path="/6174477C/638385BA/6386F045" Ref="#PWR?"  Part="1"
-AR Path="/6174477C/638DF11D/6386F045" Ref="#PWR0181"  Part="1"
+AR Path="/6174477C/638DF11D/6386F045" Ref="#PWR0183"  Part="1"
 AR Path="/6174477C/638DF11F/6386F045" Ref="#PWR?"  Part="1"
-F 0 "#PWR0181" H 4550 2600 50  0001 C CNN
+F 0 "#PWR0183" H 4550 2600 50  0001 C CNN
 F 1 "GND" H 4555 2677 50  0000 C CNN
 F 2 "" H 4550 2850 50  0001 C CNN
@@
 AR Path="/6174477C/638385B8/63916772" Ref="R?"  Part="1"
 AR Path="/6174477C/638385BA/63916772" Ref="R?"  Part="1"
-AR Path="/6174477C/638DF11D/63916772" Ref="R97"  Part="1"
+AR Path="/6174477C/638DF11D/63916772" Ref="R101"  Part="1"
 AR Path="/6174477C/638DF11F/63916772" Ref="R?"  Part="1"
-F 0 "R97" V 8004 3950 50  0000 C CNN
+F 0 "R101" V 8004 3950 50  0000 C CNN
 F 1 "1M" V 8095 3950 50  0000 C CNN
 F 2 "Resistor_SMD:R_0402_1005Metric" H 8200 3950 50  0001 C CNN
@@
 AR Path="/6174477C/638385B8/63916773" Ref="J?"  Part="1"
 AR Path="/6174477C/638385BA/63916773" Ref="J?"  Part="1"
-AR Path="/6174477C/638DF11D/63916773" Ref="J17"  Part="1"
+AR Path="/6174477C/638DF11D/63916773" Ref="J18"  Part="1"
 AR Path="/6174477C/638DF11F/63916773" Ref="J?"  Part="1"
-F 0 "J17" H 3770 5146 50  0000 R CNN
+F 0 "J18" H 3770 5146 50  0000 R CNN
 F 1 "AVR-ISP-6" H 3770 5055 50  0000 R CNN
 F 2 "Connector_PinHeader_2.54mm:PinHeader_2x03_P2.54mm_Vertical" V 3850 5100 50  0001 C CNN
@@
 AR Path="/6174477C/638385B8/63916774" Ref="#PWR?"  Part="1"
 AR Path="/6174477C/638385BA/63916774" Ref="#PWR?"  Part="1"
-AR Path="/6174477C/638DF11D/63916774" Ref="#PWR0180"  Part="1"
+AR Path="/6174477C/638DF11D/63916774" Ref="#PWR0182"  Part="1"
 AR Path="/6174477C/638DF11F/63916774" Ref="#PWR?"  Part="1"
-F 0 "#PWR0180" H 4200 5300 50  0001 C CNN
+F 0 "#PWR0182" H 4200 5300 50  0001 C CNN
 F 1 "GND" H 4205 5377 50  0000 C CNN
 F 2 "" H 4200 5550 50  0001 C CNN
@@
 AR Path="/6174477C/638385B8/63916770" Ref="D?"  Part="1"
 AR Path="/6174477C/638385BA/63916770" Ref="D?"  Part="1"
-AR Path="/6174477C/638DF11D/63916770" Ref="D18"  Part="1"
+AR Path="/6174477C/638DF11D/63916770" Ref="D17"  Part="1"
 AR Path="/6174477C/638DF11F/63916770" Ref="D?"  Part="1"
-F 0 "D18" V 8439 2682 50  0000 R CNN
+F 0 "D17" V 8439 2682 50  0000 R CNN
 F 1 "NODE9_STATUSLED" V 8348 2682 50  0000 R CNN
 F 2 "LED_SMD:LED_0402_1005Metric" H 8400 2800 50  0001 C CNN
@@
 AR Path="/6174477C/638385B8/6391677F" Ref="R?"  Part="1"
 AR Path="/6174477C/638385BA/6391677F" Ref="R?"  Part="1"
-AR Path="/6174477C/638DF11D/6391677F" Ref="R98"  Part="1"
+AR Path="/6174477C/638DF11D/6391677F" Ref="R102"  Part="1"
 AR Path="/6174477C/638DF11F/6391677F" Ref="R?"  Part="1"
-F 0 "R98" V 8204 3150 50  0000 C CNN
+F 0 "R102" V 8204 3150 50  0000 C CNN
 F 1 "1K" V 8295 3150 50  0000 C CNN
 F 2 "Resistor_SMD:R_0402_1005Metric" H 8400 3150 50  0001 C CNN
@@
 AR Path="/6174477C/638385B8/63916883" Ref="#PWR?"  Part="1"
 AR Path="/6174477C/638385BA/63916883" Ref="#PWR?"  Part="1"
-AR Path="/6174477C/638DF11D/63916883" Ref="#PWR0186"  Part="1"
+AR Path="/6174477C/638DF11D/63916883" Ref="#PWR0188"  Part="1"
 AR Path="/6174477C/638DF11F/63916883" Ref="#PWR?"  Part="1"
-F 0 "#PWR0186" H 8400 3100 50  0001 C CNN
+F 0 "#PWR0188" H 8400 3100 50  0001 C CNN
 F 1 "GND" H 8405 3177 50  0000 C CNN
 F 2 "" H 8400 3350 50  0001 C CNN
@@
 AR Path="/6174477C/638385B8/6391676E" Ref="#PWR?"  Part="1"
 AR Path="/6174477C/638385BA/6391676E" Ref="#PWR?"  Part="1"
-AR Path="/6174477C/638DF11D/6391676E" Ref="#PWR0182"  Part="1"
+AR Path="/6174477C/638DF11D/6391676E" Ref="#PWR0184"  Part="1"
 AR Path="/6174477C/638DF11F/6391676E" Ref="#PWR?"  Part="1"
-F 0 "#PWR0182" H 6100 5800 50  0001 C CNN
+F 0 "#PWR0184" H 6100 5800 50  0001 C CNN
 F 1 "GND" H 6105 5877 50  0000 C CNN
 F 2 "" H 6100 6050 50  0001 C CNN

Commit message: Fix git
Connections:
- net +5V_A: no longer C64.1, C65.1, D17.2 (A), R100.2, U23.18 (AVCC), U23.20 (AREF), U23.4 (VCC)
- net at SW10.1 (D): now also C64.1, C65.1, D17.2 (A), R100.2, U23.18 (AVCC), U23.20 (AREF), U23.4 (VCC)
