File: ykts-payload/ykts-mcu-node2.sch (KiCad schematic (older format))
At the start: 12 parts

Commit message: Update nodes
Parts:
- removed C? (x2): 22pF, Capacitor_SMD:C_0402_1005Metric, symbol Device:C_Small
- removed C?: 100nF, Capacitor_SMD:C_0402_1005Metric, symbol Device:C_Small
- removed U?: ATmega328PB-MU, Package_DFN_QFN:QFN-32-1EP_5x5mm_P0.5mm_EP3.1x3.1mm, symbol MCU_Microchip_ATmega:ATmega328PB-MU
- added C89: 100nF, Capacitor_SMD:C_0402_1005Metric, symbol Device:C_Small
- added C90, C91: 22pF, Capacitor_SMD:C_0402_1005Metric, symbol Device:C_Small
- added U29: ATmega328PB-MU, Package_DFN_QFN:QFN-32-1EP_5x5mm_P0.5mm_EP3.1x3.1mm, symbol MCU_Microchip_ATmega:ATmega328PB-MU
- D21: renamed from D?; value NODE1_STATUSLED -> NODE2_STATUSLED
- gave numbers to parts that had none: 7
Connections:
- net +5V_A: now also C89.1, U29.18 (AVCC), U29.20 (AREF), U29.4 (VCC)
- net GND: now also C89.2, C90.2, C91.2, U29.21 (GND), U29.33 (GND), U29.5 (GND)
- net ISP_MISO: now also U29.16 (PB4)
- net ISP_MOSI: now also U29.15 (PB3)
- net ISP_SCK: now also U29.17 (PB5)
- net at R105.1, Y18.1: now also C91.1, U29.7 (XTAL1/PB6)
- net at R105.2, Y18.3: now also C90.1, U29.8 (XTAL2/PB7)
- net NODE1_PWR renamed NODE2_PWR
- net NODE1_RESET renamed NODE2_RESET
- net NODE2_RESET: now also U29.29 (~RESET~/PC6)
- new net NODE2_RX: U29.31 (PD1)
- new net NODE2_TX: U29.30 (PD0)
Other:
- note added: "MCU Node 2"
- note removed: "MCU Node 1"

Commit message: Fixed annotations & sheet ordering
Parts:
- renumbered C88 to C36, C89 to C37, C90 to C38, C91 to C39, D21 to D11, J21 to J10, R104 to R75, R105 to R76, R106 to R77, SW16 to SW3, U29 to U16, Y18 to Y5

Commit message: Revision A2
Added debug power
Basic ESD protection on UART
MCP Reset from MCU
Parts:
- renumbered D11 to D10, J10 to J11, R75 to R79, R76 to R80, R77 to R81

Commit message: Fix git
Connections:
- net +5V_A: no longer C36.1, C37.1, D10.2 (A), R79.2, U16.18 (AVCC), U16.20 (AREF), U16.4 (VCC)
- net at SW3.1 (D): now also C36.1, C37.1, D10.2 (A), R79.2, U16.18 (AVCC), U16.20 (AREF), U16.4 (VCC)

Commit message: Change node ISP connector footprint
Parts:
- J11: footprint Connector_PinHeader_2.54mm:PinHeader_2x03_P2.54mm_Vertical -> Connector_PinHeader_1.27mm:PinHeader_2x03_P1.27mm_Vertical_SMD
Changed lines of the file:
@@
 F 0 "J11" H 3770 5146 50  0000 R CNN
 F 1 "AVR-ISP-6" H 3770 5055 50  0000 R CNN
-F 2 "Connector_PinHeader_2.54mm:PinHeader_2x03_P2.54mm_Vertical" V 3850 5100 50  0001 C CNN
+F 2 "Connector_PinHeader_1.27mm:PinHeader_2x03_P1.27mm_Vertical_SMD" V 3850 5100 50  0001 C CNN
 F 3 " ~" H 2825 4500 50  0001 C CNN
 	1    4100 5050

Commit message: Revision B0
Added second supervisor, mega2560 -> mega128a
Parts:
- renumbered C36 to C47, C37 to C48, C38 to C49, C39 to C50, D10 to D12, J11 to J15, R79 to R57, R80 to R58, R81 to R59, U16 to U14, Y5 to Y7
