File: ykts-payload/ykts-mcu-node0.sch (KiCad schematic (older format))
At the start: 12 parts

Commit message: Update nodes
Parts:
- gave numbers to parts that had none: 12

Commit message: Fixed annotations & sheet ordering
Parts:
- renumbered C19 to C28, C23 to C29, C24 to C30, C25 to C31, D6 to D9, J6 to J8, R59 to R69, R60 to R70, R61 to R71

Commit message: Revision A2
Added debug power
Basic ESD protection on UART
MCP Reset from MCU
Parts:
- renumbered D9 to D8, J8 to J9, R69 to R73, R70 to R74, R71 to R75
Changed lines of the file:
@@
 Sheet 3 18
 Title "YktSat Payload Module"
-Date "2021-10-02"
-Rev "A1"
+Date "2021-10-03"
+Rev "A2"
 Comp "Sakha Aerospace Systems, LLC"
 Comment1 ""
@@
 P 3500 2850
 AR Path="/6174477C/6386EE31" Ref="#PWR?"  Part="1"
-AR Path="/6174477C/637564E2/6386EE31" Ref="#PWR089"  Part="1"
+AR Path="/6174477C/637564E2/6386EE31" Ref="#PWR091"  Part="1"
 AR Path="/6174477C/637CB186/6386EE31" Ref="#PWR?"  Part="1"
 AR Path="/6174477C/63801AEE/6386EE31" Ref="#PWR?"  Part="1"
 AR Path="/6174477C/638385B6/6386EE31" Ref="#PWR?"  Part="1"
 AR Path="/6174477C/638DF11B/6386EE31" Ref="#PWR?"  Part="1"
-F 0 "#PWR089" H 3500 2600 50  0001 C CNN
+F 0 "#PWR091" H 3500 2600 50  0001 C CNN
 F 1 "GND" H 3505 2677 50  0000 C CNN
 F 2 "" H 3500 2850 50  0001 C CNN
@@
 P 8400 4700
 AR Path="/6174477C/6391666D" Ref="#PWR?"  Part="1"
-AR Path="/6174477C/637564E2/6391666D" Ref="#PWR097"  Part="1"
+AR Path="/6174477C/637564E2/6391666D" Ref="#PWR099"  Part="1"
 AR Path="/6174477C/637CB186/6391666D" Ref="#PWR?"  Part="1"
 AR Path="/6174477C/63801AEE/6391666D" Ref="#PWR?"  Part="1"
 AR Path="/6174477C/638385B6/6391666D" Ref="#PWR?"  Part="1"
 AR Path="/6174477C/638DF11B/6391666D" Ref="#PWR?"  Part="1"
-F 0 "#PWR097" H 8400 4450 50  0001 C CNN
+F 0 "#PWR099" H 8400 4450 50  0001 C CNN
 F 1 "GND" H 8405 4527 50  0000 C CNN
 F 2 "" H 8400 4700 50  0001 C CNN
@@
 P 8000 4700
 AR Path="/6174477C/6391666E" Ref="#PWR?"  Part="1"
-AR Path="/6174477C/637564E2/6391666E" Ref="#PWR093"  Part="1"
+AR Path="/6174477C/637564E2/6391666E" Ref="#PWR095"  Part="1"
 AR Path="/6174477C/637CB186/6391666E" Ref="#PWR?"  Part="1"
 AR Path="/6174477C/63801AEE/6391666E" Ref="#PWR?"  Part="1"
 AR Path="/6174477C/638385B6/6391666E" Ref="#PWR?"  Part="1"
 AR Path="/6174477C/638DF11B/6391666E" Ref="#PWR?"  Part="1"
-F 0 "#PWR093" H 8000 4450 50  0001 C CNN
+F 0 "#PWR095" H 8000 4450 50  0001 C CNN
 F 1 "GND" H 8005 4527 50  0000 C CNN
 F 2 "" H 8000 4700 50  0001 C CNN
@@
 P 8200 4200
 AR Path="/6174477C/6386EE37" Ref="#PWR?"  Part="1"
-AR Path="/6174477C/637564E2/6386EE37" Ref="#PWR094"  Part="1"
+AR Path="/6174477C/637564E2/6386EE37" Ref="#PWR096"  Part="1"
 AR Path="/6174477C/637CB186/6386EE37" Ref="#PWR?"  Part="1"
 AR Path="/6174477C/63801AEE/6386EE37" Ref="#PWR?"  Part="1"
 AR Path="/6174477C/638385B6/6386EE37" Ref="#PWR?"  Part="1"
 AR Path="/6174477C/638DF11B/6386EE37" Ref="#PWR?"  Part="1"
-F 0 "#PWR094" H 8200 3950 50  0001 C CNN
+F 0 "#PWR096" H 8200 3950 50  0001 C CNN
 F 1 "GND" H 8205 4027 50  0000 C CNN
 F 2 "" H 8200 4200 50  0001 C CNN
@@
 P 8200 4400
 AR Path="/6174477C/6386EE38" Ref="#PWR?"  Part="1"
-AR Path="/6174477C/637564E2/6386EE38" Ref="#PWR095"  Part="1"
+AR Path="/6174477C/637564E2/6386EE38" Ref="#PWR097"  Part="1"
 AR Path="/6174477C/637CB186/6386EE38" Ref="#PWR?"  Part="1"
 AR Path="/6174477C/63801AEE/6386EE38" Ref="#PWR?"  Part="1"
 AR Path="/6174477C/638385B6/6386EE38" Ref="#PWR?"  Part="1"
 AR Path="/6174477C/638DF11B/6386EE38" Ref="#PWR?"  Part="1"
-F 0 "#PWR095" H 8200 4150 50  0001 C CNN
+F 0 "#PWR097" H 8200 4150 50  0001 C CNN
 F 1 "GND" H 8205 4227 50  0000 C CNN
 F 2 "" H 8200 4400 50  0001 C CNN
@@
 AR Path="/638383BB" Ref="R?"  Part="1"
 AR Path="/6174477C/638383BB" Ref="R?"  Part="1"
-AR Path="/6174477C/637564E2/638383BB" Ref="R69"  Part="1"
+AR Path="/6174477C/637564E2/638383BB" Ref="R73"  Part="1"
 AR Path="/6174477C/637CB186/638383BB" Ref="R?"  Part="1"
 AR Path="/6174477C/63801AEE/638383BB" Ref="R?"  Part="1"
 AR Path="/6174477C/638385B6/638383BB" Ref="R?"  Part="1"
 AR Path="/6174477C/638DF11B/638383BB" Ref="R?"  Part="1"
-F 0 "R69" V 6754 4400 50  0000 C CNN
+F 0 "R73" V 6754 4400 50  0000 C CNN
 F 1 "20K" V 6845 4400 50  0000 C CNN
 F 2 "Resistor_SMD:R_0402_1005Metric" H 6950 4400 50  0001 C CNN
@@
 NODE0_TX
 $Comp
-L yktsat-common:+5V_A #PWR088
+L yktsat-common:+5V_A #PWR090
 U 1 1 6386EE3A
 P 3500 1800
-AR Path="/6174477C/637564E2/6386EE3A" Ref="#PWR088"  Part="1"
+AR Path="/6174477C/637564E2/6386EE3A" Ref="#PWR090"  Part="1"
 AR Path="/6174477C/637CB186/6386EE3A" Ref="#PWR?"  Part="1"
 AR Path="/6174477C/63801AEE/6386EE3A" Ref="#PWR?"  Part="1"
 AR Path="/6174477C/638385B6/6386EE3A" Ref="#PWR?"  Part="1"
 AR Path="/6174477C/638DF11B/6386EE3A" Ref="#PWR?"  Part="1"
-F 0 "#PWR088" H 3500 1650 50  0001 C CNN
+F 0 "#PWR090" H 3500 1650 50  0001 C CNN
 F 1 "+5V_A" H 3515 1973 50  0000 C CNN
 F 2 "" H 3500 1800 50  0001 C CNN
@@
 P 4550 2850
 AR Path="/6174477C/6386EF3F" Ref="#PWR?"  Part="1"
-AR Path="/6174477C/637564E2/6386EF3F" Ref="#PWR091"  Part="1"
+AR Path="/6174477C/637564E2/6386EF3F" Ref="#PWR093"  Part="1"
 AR Path="/6174477C/637CB186/6386EF3F" Ref="#PWR?"  Part="1"
 AR Path="/6174477C/63801AEE/6386EF3F" Ref="#PWR?"  Part="1"
 AR Path="/6174477C/638385B6/6386EF3F" Ref="#PWR?"  Part="1"
 AR Path="/6174477C/638DF11B/6386EF3F" Ref="#PWR?"  Part="1"
-F 0 "#PWR091" H 4550 2600 50  0001 C CNN
+F 0 "#PWR093" H 4550 2600 50  0001 C CNN
 F 1 "GND" H 4555 2677 50  0000 C CNN
 F 2 "" H 4550 2850 50  0001 C CNN
@@
 AR Path="/6386EF40" Ref="R?"  Part="1"
 AR Path="/6174477C/6386EF40" Ref="R?"  Part="1"
-AR Path="/6174477C/637564E2/6386EF40" Ref="R70"  Part="1"
+AR Path="/6174477C/637564E2/6386EF40" Ref="R74"  Part="1"
 AR Path="/6174477C/637CB186/6386EF40" Ref="R?"  Part="1"
 AR Path="/6174477C/63801AEE/6386EF40" Ref="R?"  Part="1"
 AR Path="/6174477C/638385B6/6386EF40" Ref="R?"  Part="1"
 AR Path="/6174477C/638DF11B/6386EF40" Ref="R?"  Part="1"
-F 0 "R70" V 8004 3950 50  0000 C CNN
+F 0 "R74" V 8004 3950 50  0000 C CNN
 F 1 "1M" V 8095 3950 50  0000 C CNN
 F 2 "Resistor_SMD:R_0402_1005Metric" H 8200 3950 50  0001 C CNN
@@
 P 4100 5050
 AR Path="/6174477C/6386EF41" Ref="J?"  Part="1"
-AR Path="/6174477C/637564E2/6386EF41" Ref="J8"  Part="1"
+AR Path="/6174477C/637564E2/6386EF41" Ref="J9"  Part="1"
 AR Path="/6174477C/637CB186/6386EF41" Ref="J?"  Part="1"
 AR Path="/6174477C/63801AEE/6386EF41" Ref="J?"  Part="1"
 AR Path="/6174477C/638385B6/6386EF41" Ref="J?"  Part="1"
 AR Path="/6174477C/638DF11B/6386EF41" Ref="J?"  Part="1"
-F 0 "J8" H 3770 5146 50  0000 R CNN
+F 0 "J9" H 3770 5146 50  0000 R CNN
 F 1 "AVR-ISP-6" H 3770 5055 50  0000 R CNN
 F 2 "Connector_PinHeader_2.54mm:PinHeader_2x03_P2.54mm_Vertical" V 3850 5100 50  0001 C CNN
@@
 P 4200 5550
 AR Path="/6174477C/6386EF42" Ref="#PWR?"  Part="1"
-AR Path="/6174477C/637564E2/6386EF42" Ref="#PWR090"  Part="1"
+AR Path="/6174477C/637564E2/6386EF42" Ref="#PWR092"  Part="1"
 AR Path="/6174477C/637CB186/6386EF42" Ref="#PWR?"  Part="1"
 AR Path="/6174477C/63801AEE/6386EF42" Ref="#PWR?"  Part="1"
 AR Path="/6174477C/638385B6/6386EF42" Ref="#PWR?"  Part="1"
 AR Path="/6174477C/638DF11B/6386EF42" Ref="#PWR?"  Part="1"
-F 0 "#PWR090" H 4200 5300 50  0001 C CNN
+F 0 "#PWR092" H 4200 5300 50  0001 C CNN
 F 1 "GND" H 4205 5377 50  0000 C CNN
 F 2 "" H 4200 5550 50  0001 C CNN
@@
 	5400 2450 6100 2450
 $Comp
-L Device:LED D9
+L Device:LED D8
 U 1 1 6386EF43
 P 8400 2800
-AR Path="/6174477C/637564E2/6386EF43" Ref="D9"  Part="1"
+AR Path="/6174477C/637564E2/6386EF43" Ref="D8"  Part="1"
 AR Path="/6174477C/637CB186/6386EF43" Ref="D?"  Part="1"
 AR Path="/6174477C/63801AEE/6386EF43" Ref="D?"  Part="1"
 AR Path="/6174477C/638385B6/6386EF43" Ref="D?"  Part="1"
 AR Path="/6174477C/638DF11B/6386EF43" Ref="D?"  Part="1"
-F 0 "D9" V 8439 2682 50  0000 R CNN
+F 0 "D8" V 8439 2682 50  0000 R CNN
 F 1 "NODE0_STATUSLED" V 8348 2682 50  0000 R CNN
 F 2 "LED_SMD:LED_0402_1005Metric" H 8400 2800 50  0001 C CNN
@@
 AR Path="/6386EF44" Ref="R?"  Part="1"
 AR Path="/6174477C/6386EF44" Ref="R?"  Part="1"
-AR Path="/6174477C/637564E2/6386EF44" Ref="R71"  Part="1"
+AR Path="/6174477C/637564E2/6386EF44" Ref="R75"  Part="1"
 AR Path="/6174477C/637CB186/6386EF44" Ref="R?"  Part="1"
 AR Path="/6174477C/63801AEE/6386EF44" Ref="R?"  Part="1"
 AR Path="/6174477C/638385B6/6386EF44" Ref="R?"  Part="1"
 AR Path="/6174477C/638DF11B/6386EF44" Ref="R?"  Part="1"
-F 0 "R71" V 8204 3150 50  0000 C CNN
+F 0 "R75" V 8204 3150 50  0000 C CNN
 F 1 "1K" V 8295 3150 50  0000 C CNN
 F 2 "Resistor_SMD:R_0402_1005Metric" H 8400 3150 50  0001 C CNN
@@
 P 8400 3350
 AR Path="/6174477C/6391667E" Ref="#PWR?"  Part="1"
-AR Path="/6174477C/637564E2/6391667E" Ref="#PWR096"  Part="1"
+AR Path="/6174477C/637564E2/6391667E" Ref="#PWR098"  Part="1"
 AR Path="/6174477C/637CB186/6391667E" Ref="#PWR?"  Part="1"
 AR Path="/6174477C/63801AEE/6391667E" Ref="#PWR?"  Part="1"
 AR Path="/6174477C/638385B6/6391667E" Ref="#PWR?"  Part="1"
 AR Path="/6174477C/638DF11B/6391667E" Ref="#PWR?"  Part="1"
-F 0 "#PWR096" H 8400 3100 50  0001 C CNN
+F 0 "#PWR098" H 8400 3100 50  0001 C CNN
 F 1 "GND" H 8405 3177 50  0000 C CNN
 F 2 "" H 8400 3350 50  0001 C CNN
@@
 P 6100 6050
 AR Path="/6174477C/6379A741" Ref="#PWR?"  Part="1"
-AR Path="/6174477C/637564E2/6379A741" Ref="#PWR092"  Part="1"
+AR Path="/6174477C/637564E2/6379A741" Ref="#PWR094"  Part="1"
 AR Path="/6174477C/637CB186/6379A741" Ref="#PWR?"  Part="1"
 AR Path="/6174477C/63801AEE/6379A741" Ref="#PWR?"  Part="1"
 AR Path="/6174477C/638385B6/6379A741" Ref="#PWR?"  Part="1"
 AR Path="/6174477C/638DF11B/6379A741" Ref="#PWR?"  Part="1"
-F 0 "#PWR092" H 6100 5800 50  0001 C CNN
+F 0 "#PWR094" H 6100 5800 50  0001 C CNN
 F 1 "GND" H 6105 5877 50  0000 C CNN
 F 2 "" H 6100 6050 50  0001 C CNN

Commit message: Fix git
Connections:
- net +5V_A: no longer C28.1, C29.1, D8.2 (A), R73.2, U14.18 (AVCC), U14.20 (AREF), U14.4 (VCC)
- net at SW1.1 (D): now also C28.1, C29.1, D8.2 (A), R73.2, U14.18 (AVCC), U14.20 (AREF), U14.4 (VCC)

Commit message: Change node ISP connector footprint
Parts:
- J9: footprint Connector_PinHeader_2.54mm:PinHeader_2x03_P2.54mm_Vertical -> Connector_PinHeader_1.27mm:PinHeader_2x03_P1.27mm_Vertical_SMD
Changed lines of the file:
@@
 F 0 "J9" H 3770 5146 50  0000 R CNN
 F 1 "AVR-ISP-6" H 3770 5055 50  0000 R CNN
-F 2 "Connector_PinHeader_2.54mm:PinHeader_2x03_P2.54mm_Vertical" V 3850 5100 50  0001 C CNN
+F 2 "Connector_PinHeader_1.27mm:PinHeader_2x03_P1.27mm_Vertical_SMD" V 3850 5100 50  0001 C CNN
 F 3 " ~" H 2825 4500 50  0001 C CNN
 	1    4100 5050

Commit message: Revision B0
Added second supervisor, mega2560 -> mega128a
Parts:
- renumbered C28 to C39, C29 to C40, C30 to C41, C31 to C42, D8 to D10, J9 to J13, R73 to R51, R74 to R52, R75 to R53, U14 to U12, Y3 to Y5

Commit message: Revision B2
Hierarchal sheets for nodes
Partial PCB layout
Parts:
- renumbered C39 to C41, C40 to C42, C41 to C43, C42 to C44, U12 to U14
Changed lines of the file:
@@
 Sheet 3 18
 Title "YktSat Payload Module"
-Date "2021-10-22"
-Rev "B0"
+Date "2021-10-26"
+Rev "B1"
 Comp "Sakha Aerospace Systems, LLC"
 Comment1 ""
@@
 $EndDescr
 $Comp
-L MCU_Microchip_ATmega:ATmega328PB-MU U12
+L MCU_Microchip_ATmega:ATmega328PB-MU U14
 U 1 1 65833EE1
 P 6100 4300
-AR Path="/6174477C/637564E2/65833EE1" Ref="U12"  Part="1"
+AR Path="/6174477C/637564E2/65833EE1" Ref="U14"  Part="1"
 AR Path="/6174477C/637CB186/65833EE1" Ref="U?"  Part="1"
 AR Path="/6174477C/63801AEE/65833EE1" Ref="U?"  Part="1"
@@
 AR Path="/6174477C/6572958C/65833EE1" Ref="U?"  Part="1"
 AR Path="/6174477C/6577909A/65833EE1" Ref="U?"  Part="1"
-F 0 "U12" H 6100 2711 50  0000 C CNN
+F 0 "U14" H 6100 2711 50  0000 C CNN
 F 1 "ATmega328PB-MU" H 6100 2620 50  0000 C CNN
 F 2 "Package_DFN_QFN:QFN-32-1EP_5x5mm_P0.5mm_EP3.1x3.1mm" H 6100 4300 50  0001 C CIN
@@
 P 4350 2600
 AR Path="/6174477C/65833DB4" Ref="C?"  Part="1"
-AR Path="/6174477C/637564E2/65833DB4" Ref="C39"  Part="1"
+AR Path="/6174477C/637564E2/65833DB4" Ref="C41"  Part="1"
 AR Path="/6174477C/637CB186/65833DB4" Ref="C?"  Part="1"
 AR Path="/6174477C/63801AEE/65833DB4" Ref="C?"  Part="1"
@@
 AR Path="/6174477C/6572958C/65833DB4" Ref="C?"  Part="1"
 AR Path="/6174477C/6577909A/65833DB4" Ref="C?"  Part="1"
-F 0 "C39" H 4442 2646 50  0000 L CNN
+F 0 "C41" H 4442 2646 50  0000 L CNN
 F 1 "1uF" H 4442 2555 50  0000 L CNN
 F 2 "Capacitor_SMD:C_0603_1608Metric" H 4350 2600 50  0001 C CNN
@@
 P 4700 2600
 AR Path="/6174477C/65833ED8" Ref="C?"  Part="1"
-AR Path="/6174477C/637564E2/65833ED8" Ref="C40"  Part="1"
+AR Path="/6174477C/637564E2/65833ED8" Ref="C42"  Part="1"
 AR Path="/6174477C/637CB186/65833ED8" Ref="C?"  Part="1"
 AR Path="/6174477C/63801AEE/65833ED8" Ref="C?"  Part="1"
@@
 AR Path="/6174477C/6572958C/65833ED8" Ref="C?"  Part="1"
 AR Path="/6174477C/6577909A/65833ED8" Ref="C?"  Part="1"
-F 0 "C40" H 4792 2646 50  0000 L CNN
+F 0 "C42" H 4792 2646 50  0000 L CNN
 F 1 "100nF" H 4792 2555 50  0000 L CNN
 F 2 "Capacitor_SMD:C_0402_1005Metric" H 4700 2600 50  0001 C CNN
@@
 P 3500 2850
 AR Path="/6174477C/65833DE5" Ref="#PWR?"  Part="1"
-AR Path="/6174477C/637564E2/65833DE5" Ref="#PWR0105"  Part="1"
+AR Path="/6174477C/637564E2/65833DE5" Ref="#PWR0109"  Part="1"
 AR Path="/6174477C/637CB186/65833DE5" Ref="#PWR?"  Part="1"
 AR Path="/6174477C/63801AEE/65833DE5" Ref="#PWR?"  Part="1"
@@
 AR Path="/6174477C/6572958C/65833DE5" Ref="#PWR?"  Part="1"
 AR Path="/6174477C/6577909A/65833DE5" Ref="#PWR?"  Part="1"
-F 0 "#PWR0105" H 3500 2600 50  0001 C CNN
+F 0 "#PWR0109" H 3500 2600 50  0001 C CNN
 F 1 "GND" H 3505 2677 50  0000 C CNN
 F 2 "" H 3500 2850 50  0001 C CNN
@@
 P 8400 4550
 AR Path="/6174477C/65833DF0" Ref="C?"  Part="1"
-AR Path="/6174477C/637564E2/65833DF0" Ref="C42"  Part="1"
+AR Path="/6174477C/637564E2/65833DF0" Ref="C44"  Part="1"
 AR Path="/6174477C/637CB186/65833DF0" Ref="C?"  Part="1"
 AR Path="/6174477C/63801AEE/65833DF0" Ref="C?"  Part="1"
@@
 AR Path="/6174477C/6572958C/65833DF0" Ref="C?"  Part="1"
 AR Path="/6174477C/6577909A/65833DF0" Ref="C?"  Part="1"
-F 0 "C42" H 8100 4600 50  0000 L CNN
+F 0 "C44" H 8100 4600 50  0000 L CNN
 F 1 "22pF" H 8100 4500 50  0000 L CNN
 F 2 "Capacitor_SMD:C_0402_1005Metric" H 8400 4550 50  0001 C CNN
@@
 P 8000 4550
 AR Path="/6174477C/65833E95" Ref="C?"  Part="1"
-AR Path="/6174477C/637564E2/65833E95" Ref="C41"  Part="1"
+AR Path="/6174477C/637564E2/65833E95" Ref="C43"  Part="1"
 AR Path="/6174477C/637CB186/65833E95" Ref="C?"  Part="1"
 AR Path="/6174477C/63801AEE/65833E95" Ref="C?"  Part="1"
@@
 AR Path="/6174477C/6572958C/65833E95" Ref="C?"  Part="1"
 AR Path="/6174477C/6577909A/65833E95" Ref="C?"  Part="1"
-F 0 "C41" H 8100 4600 50  0000 L CNN
+F 0 "C43" H 8100 4600 50  0000 L CNN
 F 1 "22pF" H 8100 4500 50  0000 L CNN
 F 2 "Capacitor_SMD:C_0402_1005Metric" H 8000 4550 50  0001 C CNN
@@
 P 8400 4700
 AR Path="/6174477C/65833EB0" Ref="#PWR?"  Part="1"
-AR Path="/6174477C/637564E2/65833EB0" Ref="#PWR0113"  Part="1"
+AR Path="/6174477C/637564E2/65833EB0" Ref="#PWR0117"  Part="1"
 AR Path="/6174477C/637CB186/65833EB0" Ref="#PWR?"  Part="1"
 AR Path="/6174477C/63801AEE/65833EB0" Ref="#PWR?"  Part="1"
@@
 AR Path="/6174477C/6572958C/65833EB0" Ref="#PWR?"  Part="1"
 AR Path="/6174477C/6577909A/65833EB0" Ref="#PWR?"  Part="1"
-F 0 "#PWR0113" H 8400 4450 50  0001 C CNN
+F 0 "#PWR0117" H 8400 4450 50  0001 C CNN
 F 1 "GND" H 8405 4527 50  0000 C CNN
 F 2 "" H 8400 4700 50  0001 C CNN
@@
 P 8000 4700
 AR Path="/6174477C/65833EBB" Ref="#PWR?"  Part="1"
-AR Path="/6174477C/637564E2/65833EBB" Ref="#PWR0109"  Part="1"
+AR Path="/6174477C/637564E2/65833EBB" Ref="#PWR0113"  Part="1"
 AR Path="/6174477C/637CB186/65833EBB" Ref="#PWR?"  Part="1"
 AR Path="/6174477C/63801AEE/65833EBB" Ref="#PWR?"  Part="1"
@@
 AR Path="/6174477C/6572958C/65833EBB" Ref="#PWR?"  Part="1"
 AR Path="/6174477C/6577909A/65833EBB" Ref="#PWR?"  Part="1"
-F 0 "#PWR0109" H 8000 4450 50  0001 C CNN
+F 0 "#PWR0113" H 8000 4450 50  0001 C CNN
 F 1 "GND" H 8005 4527 50  0000 C CNN
 F 2 "" H 8000 4700 50  0001 C CNN
@@
 P 8200 4200
 AR Path="/6174477C/65833E09" Ref="#PWR?"  Part="1"
-AR Path="/6174477C/637564E2/65833E09" Ref="#PWR0110"  Part="1"
+AR Path="/6174477C/637564E2/65833E09" Ref="#PWR0114"  Part="1"
 AR Path="/6174477C/637CB186/65833E09" Ref="#PWR?"  Part="1"
 AR Path="/6174477C/63801AEE/65833E09" Ref="#PWR?"  Part="1"
@@
 AR Path="/6174477C/6572958C/65833E09" Ref="#PWR?"  Part="1"
 AR Path="/6174477C/6577909A/65833E09" Ref="#PWR?"  Part="1"
-F 0 "#PWR0110" H 8200 3950 50  0001 C CNN
+F 0 "#PWR0114" H 8200 3950 50  0001 C CNN
 F 1 "GND" H 8205 4027 50  0000 C CNN
 F 2 "" H 8200 4200 50  0001 C CNN
@@
 P 8200 4400
 AR Path="/6174477C/6386EE38" Ref="#PWR?"  Part="1"
-AR Path="/6174477C/637564E2/6386EE38" Ref="#PWR0111"  Part="1"
+AR Path="/6174477C/637564E2/6386EE38" Ref="#PWR0115"  Part="1"
 AR Path="/6174477C/637CB186/6386EE38" Ref="#PWR?"  Part="1"
 AR Path="/6174477C/63801AEE/6386EE38" Ref="#PWR?"  Part="1"
@@
 AR Path="/6174477C/6572958C/6386EE38" Ref="#PWR?"  Part="1"
 AR Path="/6174477C/6577909A/6386EE38" Ref="#PWR?"  Part="1"
-F 0 "#PWR0111" H 8200 4150 50  0001 C CNN
+F 0 "#PWR0115" H 8200 4150 50  0001 C CNN
 F 1 "GND" H 8205 4227 50  0000 C CNN
 F 2 "" H 8200 4400 50  0001 C CNN
@@
 NODE0_TX
 $Comp
-L yktsat-common:+5V_A #PWR0104
+L yktsat-common:+5V_A #PWR0108
 U 1 1 65833E25
 P 3500 1800
-AR Path="/6174477C/637564E2/65833E25" Ref="#PWR0104"  Part="1"
+AR Path="/6174477C/637564E2/65833E25" Ref="#PWR0108"  Part="1"
 AR Path="/6174477C/637CB186/65833E25" Ref="#PWR?"  Part="1"
 AR Path="/6174477C/63801AEE/65833E25" Ref="#PWR?"  Part="1"
@@
 AR Path="/6174477C/6572958C/65833E25" Ref="#PWR?"  Part="1"
 AR Path="/6174477C/6577909A/65833E25" Ref="#PWR?"  Part="1"
-F 0 "#PWR0104" H 3500 1650 50  0001 C CNN
+F 0 "#PWR0108" H 3500 1650 50  0001 C CNN
 F 1 "+5V_A" H 3515 1973 50  0000 C CNN
 F 2 "" H 3500 1800 50  0001 C CNN
@@
 P 4700 2850
 AR Path="/6174477C/65833E2E" Ref="#PWR?"  Part="1"
-AR Path="/6174477C/637564E2/65833E2E" Ref="#PWR0107"  Part="1"
+AR Path="/6174477C/637564E2/65833E2E" Ref="#PWR0111"  Part="1"
 AR Path="/6174477C/637CB186/65833E2E" Ref="#PWR?"  Part="1"
 AR Path="/6174477C/63801AEE/65833E2E" Ref="#PWR?"  Part="1"
@@
 AR Path="/6174477C/6572958C/65833E2E" Ref="#PWR?"  Part="1"
 AR Path="/6174477C/6577909A/65833E2E" Ref="#PWR?"  Part="1"
-F 0 "#PWR0107" H 4700 2600 50  0001 C CNN
+F 0 "#PWR0111" H 4700 2600 50  0001 C CNN
 F 1 "GND" H 4705 2677 50  0000 C CNN
 F 2 "" H 4700 2850 50  0001 C CNN
@@
 P 4200 5550
 AR Path="/6174477C/65833E5D" Ref="#PWR?"  Part="1"
-AR Path="/6174477C/637564E2/65833E5D" Ref="#PWR0106"  Part="1"
+AR Path="/6174477C/637564E2/65833E5D" Ref="#PWR0110"  Part="1"
 AR Path="/6174477C/637CB186/65833E5D" Ref="#PWR?"  Part="1"
 AR Path="/6174477C/63801AEE/65833E5D" Ref="#PWR?"  Part="1"
@@
 AR Path="/6174477C/6572958C/65833E5D" Ref="#PWR?"  Part="1"
 AR Path="/6174477C/6577909A/65833E5D" Ref="#PWR?"  Part="1"
-F 0 "#PWR0106" H 4200 5300 50  0001 C CNN
+F 0 "#PWR0110" H 4200 5300 50  0001 C CNN
 F 1 "GND" H 4205 5377 50  0000 C CNN
 F 2 "" H 4200 5550 50  0001 C CNN
@@
 P 8400 3350
 AR Path="/6174477C/65833EEF" Ref="#PWR?"  Part="1"
-AR Path="/6174477C/637564E2/65833EEF" Ref="#PWR0112"  Part="1"
+AR Path="/6174477C/637564E2/65833EEF" Ref="#PWR0116"  Part="1"
 AR Path="/6174477C/637CB186/65833EEF" Ref="#PWR?"  Part="1"
 AR Path="/6174477C/63801AEE/65833EEF" Ref="#PWR?"  Part="1"
@@
 AR Path="/6174477C/6572958C/65833EEF" Ref="#PWR?"  Part="1"
 AR Path="/6174477C/6577909A/65833EEF" Ref="#PWR?"  Part="1"
-F 0 "#PWR0112" H 8400 3100 50  0001 C CNN
+F 0 "#PWR0116" H 8400 3100 50  0001 C CNN
 F 1 "GND" H 8405 3177 50  0000 C CNN
 F 2 "" H 8400 3350 50  0001 C CNN
@@
 P 6100 6050
 AR Path="/6174477C/65833DC5" Ref="#PWR?"  Part="1"
-AR Path="/6174477C/637564E2/65833DC5" Ref="#PWR0108"  Part="1"
+AR Path="/6174477C/637564E2/65833DC5" Ref="#PWR0112"  Part="1"
 AR Path="/6174477C/637CB186/65833DC5" Ref="#PWR?"  Part="1"
 AR Path="/6174477C/63801AEE/65833DC5" Ref="#PWR?"  Part="1"
@@
 AR Path="/6174477C/6572958C/65833DC5" Ref="#PWR?"  Part="1"
 AR Path="/6174477C/6577909A/65833DC5" Ref="#PWR?"  Part="1"
-F 0 "#PWR0108" H 6100 5800 50  0001 C CNN
+F 0 "#PWR0112" H 6100 5800 50  0001 C CNN
 F 1 "GND" H 6105 5877 50  0000 C CNN
 F 2 "" H 6100 6050 50  0001 C CNN
