File: ykts-payload/ykts-mcu-node1.sch (KiCad schematic (older format))
At the start: 12 parts, among them J7 AVR-ISP-6, SW2 ADG802BRT, U15 ATmega328PB-MU, Y4 8 MHz

Commit message: Fixed annotations & sheet ordering
Parts:
- renumbered C26 to C32, C27 to C33, C28 to C34, C29 to C35, D7 to D10, J7 to J9, R62 to R72, R63 to R73, R64 to R74

Commit message: Revision A2
Added debug power
Basic ESD protection on UART
MCP Reset from MCU
Parts:
- renumbered D10 to D9, J9 to J10, R72 to R76, R73 to R77, R74 to R78
Changed lines of the file:
@@
 Sheet 4 18
 Title "YktSat Payload Module"
-Date "2021-10-02"
-Rev "A1"
+Date "2021-10-03"
+Rev "A2"
 Comp "Sakha Aerospace Systems, LLC"
 Comment1 ""
@@
 AR Path="/6174477C/639BAF4E" Ref="#PWR?"  Part="1"
 AR Path="/6174477C/637564E2/639BAF4E" Ref="#PWR?"  Part="1"
-AR Path="/6174477C/637CB186/639BAF4E" Ref="#PWR099"  Part="1"
+AR Path="/6174477C/637CB186/639BAF4E" Ref="#PWR0101"  Part="1"
 AR Path="/6174477C/63801AF0/639BAF4E" Ref="#PWR?"  Part="1"
 AR Path="/6174477C/63801AEE/639BAF4E" Ref="#PWR?"  Part="1"
@@
 AR Path="/6174477C/638DF11D/639BAF4E" Ref="#PWR?"  Part="1"
 AR Path="/6174477C/638DF11F/639BAF4E" Ref="#PWR?"  Part="1"
-F 0 "#PWR099" H 3500 2600 50  0001 C CNN
+F 0 "#PWR0101" H 3500 2600 50  0001 C CNN
 F 1 "GND" H 3505 2677 50  0000 C CNN
 F 2 "" H 3500 2850 50  0001 C CNN
@@
 AR Path="/6174477C/639BAF51" Ref="#PWR?"  Part="1"
 AR Path="/6174477C/637564E2/639BAF51" Ref="#PWR?"  Part="1"
-AR Path="/6174477C/637CB186/639BAF51" Ref="#PWR0107"  Part="1"
+AR Path="/6174477C/637CB186/639BAF51" Ref="#PWR0109"  Part="1"
 AR Path="/6174477C/63801AF0/639BAF51" Ref="#PWR?"  Part="1"
 AR Path="/6174477C/63801AEE/639BAF51" Ref="#PWR?"  Part="1"
@@
 AR Path="/6174477C/638DF11D/639BAF51" Ref="#PWR?"  Part="1"
 AR Path="/6174477C/638DF11F/639BAF51" Ref="#PWR?"  Part="1"
-F 0 "#PWR0107" H 8400 4450 50  0001 C CNN
+F 0 "#PWR0109" H 8400 4450 50  0001 C CNN
 F 1 "GND" H 8405 4527 50  0000 C CNN
 F 2 "" H 8400 4700 50  0001 C CNN
@@
 AR Path="/6174477C/639BAF52" Ref="#PWR?"  Part="1"
 AR Path="/6174477C/637564E2/639BAF52" Ref="#PWR?"  Part="1"
-AR Path="/6174477C/637CB186/639BAF52" Ref="#PWR0103"  Part="1"
+AR Path="/6174477C/637CB186/639BAF52" Ref="#PWR0105"  Part="1"
 AR Path="/6174477C/63801AF0/639BAF52" Ref="#PWR?"  Part="1"
 AR Path="/6174477C/63801AEE/639BAF52" Ref="#PWR?"  Part="1"
@@
 AR Path="/6174477C/638DF11D/639BAF52" Ref="#PWR?"  Part="1"
 AR Path="/6174477C/638DF11F/639BAF52" Ref="#PWR?"  Part="1"
-F 0 "#PWR0103" H 8000 4450 50  0001 C CNN
+F 0 "#PWR0105" H 8000 4450 50  0001 C CNN
 F 1 "GND" H 8005 4527 50  0000 C CNN
 F 2 "" H 8000 4700 50  0001 C CNN
@@
 AR Path="/6174477C/6391677A" Ref="#PWR?"  Part="1"
 AR Path="/6174477C/637564E2/6391677A" Ref="#PWR?"  Part="1"
-AR Path="/6174477C/637CB186/6391677A" Ref="#PWR0104"  Part="1"
+AR Path="/6174477C/637CB186/6391677A" Ref="#PWR0106"  Part="1"
 AR Path="/6174477C/63801AF0/6391677A" Ref="#PWR?"  Part="1"
 AR Path="/6174477C/63801AEE/6391677A" Ref="#PWR?"  Part="1"
@@
 AR Path="/6174477C/638DF11D/6391677A" Ref="#PWR?"  Part="1"
 AR Path="/6174477C/638DF11F/6391677A" Ref="#PWR?"  Part="1"
-F 0 "#PWR0104" H 8200 3950 50  0001 C CNN
+F 0 "#PWR0106" H 8200 3950 50  0001 C CNN
 F 1 "GND" H 8205 4027 50  0000 C CNN
 F 2 "" H 8200 4200 50  0001 C CNN
@@
 AR Path="/6174477C/6391676D" Ref="#PWR?"  Part="1"
 AR Path="/6174477C/637564E2/6391676D" Ref="#PWR?"  Part="1"
-AR Path="/6174477C/637CB186/6391676D" Ref="#PWR0105"  Part="1"
+AR Path="/6174477C/637CB186/6391676D" Ref="#PWR0107"  Part="1"
 AR Path="/6174477C/63801AF0/6391676D" Ref="#PWR?"  Part="1"
 AR Path="/6174477C/63801AEE/6391676D" Ref="#PWR?"  Part="1"
@@
 AR Path="/6174477C/638DF11D/6391676D" Ref="#PWR?"  Part="1"
 AR Path="/6174477C/638DF11F/6391676D" Ref="#PWR?"  Part="1"
-F 0 "#PWR0105" H 8200 4150 50  0001 C CNN
+F 0 "#PWR0107" H 8200 4150 50  0001 C CNN
 F 1 "GND" H 8205 4227 50  0000 C CNN
 F 2 "" H 8200 4400 50  0001 C CNN
@@
 AR Path="/6174477C/639BAF4C" Ref="R?"  Part="1"
 AR Path="/6174477C/637564E2/639BAF4C" Ref="R?"  Part="1"
-AR Path="/6174477C/637CB186/639BAF4C" Ref="R72"  Part="1"
+AR Path="/6174477C/637CB186/639BAF4C" Ref="R76"  Part="1"
 AR Path="/6174477C/63801AF0/639BAF4C" Ref="R?"  Part="1"
 AR Path="/6174477C/63801AEE/639BAF4C" Ref="R?"  Part="1"
@@
 AR Path="/6174477C/638DF11D/639BAF4C" Ref="R?"  Part="1"
 AR Path="/6174477C/638DF11F/639BAF4C" Ref="R?"  Part="1"
-F 0 "R72" V 6754 4400 50  0000 C CNN
+F 0 "R76" V 6754 4400 50  0000 C CNN
 F 1 "20K" V 6845 4400 50  0000 C CNN
 F 2 "Resistor_SMD:R_0402_1005Metric" H 6950 4400 50  0001 C CNN
@@
 P 3500 1800
 AR Path="/6174477C/637564E2/6391687E" Ref="#PWR?"  Part="1"
-AR Path="/6174477C/637CB186/6391687E" Ref="#PWR098"  Part="1"
+AR Path="/6174477C/637CB186/6391687E" Ref="#PWR0100"  Part="1"
 AR Path="/6174477C/63801AF0/6391687E" Ref="#PWR?"  Part="1"
 AR Path="/6174477C/63801AEE/6391687E" Ref="#PWR?"  Part="1"
@@
 AR Path="/6174477C/638DF11D/6391687E" Ref="#PWR?"  Part="1"
 AR Path="/6174477C/638DF11F/6391687E" Ref="#PWR?"  Part="1"
-F 0 "#PWR098" H 3500 1650 50  0001 C CNN
+F 0 "#PWR0100" H 3500 1650 50  0001 C CNN
 F 1 "+5V_A" H 3515 1973 50  0000 C CNN
 F 2 "" H 3500 1800 50  0001 C CNN
@@
 AR Path="/6174477C/639BAF53" Ref="#PWR?"  Part="1"
 AR Path="/6174477C/637564E2/639BAF53" Ref="#PWR?"  Part="1"
-AR Path="/6174477C/637CB186/639BAF53" Ref="#PWR0101"  Part="1"
+AR Path="/6174477C/637CB186/639BAF53" Ref="#PWR0103"  Part="1"
 AR Path="/6174477C/63801AF0/639BAF53" Ref="#PWR?"  Part="1"
 AR Path="/6174477C/63801AEE/639BAF53" Ref="#PWR?"  Part="1"
@@
 AR Path="/6174477C/638DF11D/639BAF53" Ref="#PWR?"  Part="1"
 AR Path="/6174477C/638DF11F/639BAF53" Ref="#PWR?"  Part="1"
-F 0 "#PWR0101" H 4550 2600 50  0001 C CNN
+F 0 "#PWR0103" H 4550 2600 50  0001 C CNN
 F 1 "GND" H 4555 2677 50  0000 C CNN
 F 2 "" H 4550 2850 50  0001 C CNN
@@
 AR Path="/6174477C/639BAF44" Ref="R?"  Part="1"
 AR Path="/6174477C/637564E2/639BAF44" Ref="R?"  Part="1"
-AR Path="/6174477C/637CB186/639BAF44" Ref="R73"  Part="1"
+AR Path="/6174477C/637CB186/639BAF44" Ref="R77"  Part="1"
 AR Path="/6174477C/63801AF0/639BAF44" Ref="R?"  Part="1"
 AR Path="/6174477C/63801AEE/639BAF44" Ref="R?"  Part="1"
@@
 AR Path="/6174477C/638DF11D/639BAF44" Ref="R?"  Part="1"
 AR Path="/6174477C/638DF11F/639BAF44" Ref="R?"  Part="1"
-F 0 "R73" V 8004 3950 50  0000 C CNN
+F 0 "R77" V 8004 3950 50  0000 C CNN
 F 1 "1M" V 8095 3950 50  0000 C CNN
 F 2 "Resistor_SMD:R_0402_1005Metric" H 8200 3950 50  0001 C CNN
@@
 AR Path="/6174477C/639BAF45" Ref="J?"  Part="1"
 AR Path="/6174477C/637564E2/639BAF45" Ref="J?"  Part="1"
-AR Path="/6174477C/637CB186/639BAF45" Ref="J9"  Part="1"
+AR Path="/6174477C/637CB186/639BAF45" Ref="J10"  Part="1"
 AR Path="/6174477C/63801AF0/639BAF45" Ref="J?"  Part="1"
 AR Path="/6174477C/63801AEE/639BAF45" Ref="J?"  Part="1"
@@
 AR Path="/6174477C/638DF11D/639BAF45" Ref="J?"  Part="1"
 AR Path="/6174477C/638DF11F/639BAF45" Ref="J?"  Part="1"
-F 0 "J9" H 3770 5146 50  0000 R CNN
+F 0 "J10" H 3770 5146 50  0000 R CNN
 F 1 "AVR-ISP-6" H 3770 5055 50  0000 R CNN
 F 2 "Connector_PinHeader_2.54mm:PinHeader_2x03_P2.54mm_Vertical" V 3850 5100 50  0001 C CNN
@@
 AR Path="/6174477C/6386F037" Ref="#PWR?"  Part="1"
 AR Path="/6174477C/637564E2/6386F037" Ref="#PWR?"  Part="1"
-AR Path="/6174477C/637CB186/6386F037" Ref="#PWR0100"  Part="1"
+AR Path="/6174477C/637CB186/6386F037" Ref="#PWR0102"  Part="1"
 AR Path="/6174477C/63801AF0/6386F037" Ref="#PWR?"  Part="1"
 AR Path="/6174477C/63801AEE/6386F037" Ref="#PWR?"  Part="1"
@@
 AR Path="/6174477C/638DF11D/6386F037" Ref="#PWR?"  Part="1"
 AR Path="/6174477C/638DF11F/6386F037" Ref="#PWR?"  Part="1"
-F 0 "#PWR0100" H 4200 5300 50  0001 C CNN
+F 0 "#PWR0102" H 4200 5300 50  0001 C CNN
 F 1 "GND" H 4205 5377 50  0000 C CNN
 F 2 "" H 4200 5550 50  0001 C CNN
@@
 P 8400 2800
 AR Path="/6174477C/637564E2/639BAF55" Ref="D?"  Part="1"
-AR Path="/6174477C/637CB186/639BAF55" Ref="D10"  Part="1"
+AR Path="/6174477C/637CB186/639BAF55" Ref="D9"  Part="1"
 AR Path="/6174477C/63801AF0/639BAF55" Ref="D?"  Part="1"
 AR Path="/6174477C/63801AEE/639BAF55" Ref="D?"  Part="1"
@@
 AR Path="/6174477C/638DF11D/639BAF55" Ref="D?"  Part="1"
 AR Path="/6174477C/638DF11F/639BAF55" Ref="D?"  Part="1"
-F 0 "D10" V 8439 2682 50  0000 R CNN
+F 0 "D9" V 8439 2682 50  0000 R CNN
 F 1 "NODE1_STATUSLED" V 8348 2682 50  0000 R CNN
 F 2 "LED_SMD:LED_0402_1005Metric" H 8400 2800 50  0001 C CNN
@@
 AR Path="/6174477C/639BAF58" Ref="R?"  Part="1"
 AR Path="/6174477C/637564E2/639BAF58" Ref="R?"  Part="1"
-AR Path="/6174477C/637CB186/639BAF58" Ref="R74"  Part="1"
+AR Path="/6174477C/637CB186/639BAF58" Ref="R78"  Part="1"
 AR Path="/6174477C/63801AF0/639BAF58" Ref="R?"  Part="1"
 AR Path="/6174477C/63801AEE/639BAF58" Ref="R?"  Part="1"
@@
 AR Path="/6174477C/638DF11D/639BAF58" Ref="R?"  Part="1"
 AR Path="/6174477C/638DF11F/639BAF58" Ref="R?"  Part="1"
-F 0 "R74" V 8204 3150 50  0000 C CNN
+F 0 "R78" V 8204 3150 50  0000 C CNN
 F 1 "1K" V 8295 3150 50  0000 C CNN
 F 2 "Resistor_SMD:R_0402_1005Metric" H 8400 3150 50  0001 C CNN
@@
 AR Path="/6174477C/639BAF54" Ref="#PWR?"  Part="1"
 AR Path="/6174477C/637564E2/639BAF54" Ref="#PWR?"  Part="1"
-AR Path="/6174477C/637CB186/639BAF54" Ref="#PWR0106"  Part="1"
+AR Path="/6174477C/637CB186/639BAF54" Ref="#PWR0108"  Part="1"
 AR Path="/6174477C/63801AF0/639BAF54" Ref="#PWR?"  Part="1"
 AR Path="/6174477C/63801AEE/639BAF54" Ref="#PWR?"  Part="1"
@@
 AR Path="/6174477C/638DF11D/639BAF54" Ref="#PWR?"  Part="1"
 AR Path="/6174477C/638DF11F/639BAF54" Ref="#PWR?"  Part="1"
-F 0 "#PWR0106" H 8400 3100 50  0001 C CNN
+F 0 "#PWR0108" H 8400 3100 50  0001 C CNN
 F 1 "GND" H 8405 3177 50  0000 C CNN
 F 2 "" H 8400 3350 50  0001 C CNN
@@
 AR Path="/6174477C/639BAF43" Ref="#PWR?"  Part="1"
 AR Path="/6174477C/637564E2/639BAF43" Ref="#PWR?"  Part="1"
-AR Path="/6174477C/637CB186/639BAF43" Ref="#PWR0102"  Part="1"
+AR Path="/6174477C/637CB186/639BAF43" Ref="#PWR0104"  Part="1"
 AR Path="/6174477C/63801AF0/639BAF43" Ref="#PWR?"  Part="1"
 AR Path="/6174477C/63801AEE/639BAF43" Ref="#PWR?"  Part="1"
@@
 AR Path="/6174477C/638DF11D/639BAF43" Ref="#PWR?"  Part="1"
 AR Path="/6174477C/638DF11F/639BAF43" Ref="#PWR?"  Part="1"
-F 0 "#PWR0102" H 6100 5800 50  0001 C CNN
+F 0 "#PWR0104" H 6100 5800 50  0001 C CNN
 F 1 "GND" H 6105 5877 50  0000 C CNN
 F 2 "" H 6100 6050 50  0001 C CNN

Commit message: Fix git
Connections:
- net +5V_A: no longer C32.1, C33.1, D9.2 (A), R76.2, U15.18 (AVCC), U15.20 (AREF), U15.4 (VCC)
- net at SW2.1 (D): now also C32.1, C33.1, D9.2 (A), R76.2, U15.18 (AVCC), U15.20 (AREF), U15.4 (VCC)

Commit message: Change node ISP connector footprint
Parts:
- J10: footprint Connector_PinHeader_2.54mm:PinHeader_2x03_P2.54mm_Vertical -> Connector_PinHeader_1.27mm:PinHeader_2x03_P1.27mm_Vertical_SMD
Changed lines of the file:
@@
 F 0 "J10" H 3770 5146 50  0000 R CNN
 F 1 "AVR-ISP-6" H 3770 5055 50  0000 R CNN
-F 2 "Connector_PinHeader_2.54mm:PinHeader_2x03_P2.54mm_Vertical" V 3850 5100 50  0001 C CNN
+F 2 "Connector_PinHeader_1.27mm:PinHeader_2x03_P1.27mm_Vertical_SMD" V 3850 5100 50  0001 C CNN
 F 3 " ~" H 2825 4500 50  0001 C CNN
 	1    4100 5050

Commit message: Revision B0
Added second supervisor, mega2560 -> mega128a
Parts:
- renumbered C32 to C43, C33 to C44, C34 to C45, C35 to C46, D9 to D11, J10 to J14, R76 to R54, R77 to R55, R78 to R56, U15 to U13, Y4 to Y6

Commit message: Revision B2
Hierarchal sheets for nodes
Partial PCB layout
Parts:
- renumbered C43 to C45, C44 to C46, C45 to C47, C46 to C48, U13 to U15
Changed lines of the file:
@@
 Sheet 4 18
 Title "YktSat Payload Module"
-Date "2021-10-22"
-Rev "B0"
+Date "2021-10-26"
+Rev "B1"
 Comp "Sakha Aerospace Systems, LLC"
 Comment1 ""
@@
 AR Path="/6174477C/638385B6/65833EE3" Ref="U?"  Part="1"
 AR Path="/6174477C/638DF11B/65833EE3" Ref="U?"  Part="1"
-AR Path="/6174477C/6568C69E/65833EE3" Ref="U13"  Part="1"
+AR Path="/6174477C/6568C69E/65833EE3" Ref="U15"  Part="1"
 AR Path="/6174477C/656DAE2A/65833EE3" Ref="U?"  Part="1"
 AR Path="/6174477C/65729588/65833EE3" Ref="U?"  Part="1"
 AR Path="/6174477C/6572958C/65833EE3" Ref="U?"  Part="1"
 AR Path="/6174477C/6577909A/65833EE3" Ref="U?"  Part="1"
-F 0 "U13" H 6100 2711 50  0000 C CNN
+F 0 "U15" H 6100 2711 50  0000 C CNN
 F 1 "ATmega328PB-MU" H 6100 2620 50  0000 C CNN
 F 2 "Package_DFN_QFN:QFN-32-1EP_5x5mm_P0.5mm_EP3.1x3.1mm" H 6100 4300 50  0001 C CIN
@@
 AR Path="/6174477C/638385B6/65833DB3" Ref="C?"  Part="1"
 AR Path="/6174477C/638DF11B/65833DB3" Ref="C?"  Part="1"
-AR Path="/6174477C/6568C69E/65833DB3" Ref="C43"  Part="1"
+AR Path="/6174477C/6568C69E/65833DB3" Ref="C45"  Part="1"
 AR Path="/6174477C/656DAE2A/65833DB3" Ref="C?"  Part="1"
 AR Path="/6174477C/65729588/65833DB3" Ref="C?"  Part="1"
 AR Path="/6174477C/6572958C/65833DB3" Ref="C?"  Part="1"
 AR Path="/6174477C/6577909A/65833DB3" Ref="C?"  Part="1"
-F 0 "C43" H 4442 2646 50  0000 L CNN
+F 0 "C45" H 4442 2646 50  0000 L CNN
 F 1 "1uF" H 4442 2555 50  0000 L CNN
 F 2 "Capacitor_SMD:C_0603_1608Metric" H 4350 2600 50  0001 C CNN
@@
 AR Path="/6174477C/638385B6/65833EDC" Ref="C?"  Part="1"
 AR Path="/6174477C/638DF11B/65833EDC" Ref="C?"  Part="1"
-AR Path="/6174477C/6568C69E/65833EDC" Ref="C44"  Part="1"
+AR Path="/6174477C/6568C69E/65833EDC" Ref="C46"  Part="1"
 AR Path="/6174477C/656DAE2A/65833EDC" Ref="C?"  Part="1"
 AR Path="/6174477C/65729588/65833EDC" Ref="C?"  Part="1"
 AR Path="/6174477C/6572958C/65833EDC" Ref="C?"  Part="1"
 AR Path="/6174477C/6577909A/65833EDC" Ref="C?"  Part="1"
-F 0 "C44" H 4792 2646 50  0000 L CNN
+F 0 "C46" H 4792 2646 50  0000 L CNN
 F 1 "100nF" H 4792 2555 50  0000 L CNN
 F 2 "Capacitor_SMD:C_0402_1005Metric" H 4700 2600 50  0001 C CNN
@@
 AR Path="/6174477C/638385B6/65833DE0" Ref="#PWR?"  Part="1"
 AR Path="/6174477C/638DF11B/65833DE0" Ref="#PWR?"  Part="1"
-AR Path="/6174477C/6568C69E/65833DE0" Ref="#PWR0115"  Part="1"
+AR Path="/6174477C/6568C69E/65833DE0" Ref="#PWR0119"  Part="1"
 AR Path="/6174477C/656DAE2A/65833DE0" Ref="#PWR?"  Part="1"
 AR Path="/6174477C/65729588/65833DE0" Ref="#PWR?"  Part="1"
 AR Path="/6174477C/6572958C/65833DE0" Ref="#PWR?"  Part="1"
 AR Path="/6174477C/6577909A/65833DE0" Ref="#PWR?"  Part="1"
-F 0 "#PWR0115" H 3500 2600 50  0001 C CNN
+F 0 "#PWR0119" H 3500 2600 50  0001 C CNN
 F 1 "GND" H 3505 2677 50  0000 C CNN
 F 2 "" H 3500 2850 50  0001 C CNN
@@
 AR Path="/6174477C/638385B6/65833DF6" Ref="C?"  Part="1"
 AR Path="/6174477C/638DF11B/65833DF6" Ref="C?"  Part="1"
-AR Path="/6174477C/6568C69E/65833DF6" Ref="C46"  Part="1"
+AR Path="/6174477C/6568C69E/65833DF6" Ref="C48"  Part="1"
 AR Path="/6174477C/656DAE2A/65833DF6" Ref="C?"  Part="1"
 AR Path="/6174477C/65729588/65833DF6" Ref="C?"  Part="1"
 AR Path="/6174477C/6572958C/65833DF6" Ref="C?"  Part="1"
 AR Path="/6174477C/6577909A/65833DF6" Ref="C?"  Part="1"
-F 0 "C46" H 8100 4600 50  0000 L CNN
+F 0 "C48" H 8100 4600 50  0000 L CNN
 F 1 "22pF" H 8100 4500 50  0000 L CNN
 F 2 "Capacitor_SMD:C_0402_1005Metric" H 8400 4550 50  0001 C CNN
@@
 AR Path="/6174477C/638385B6/65833EA0" Ref="C?"  Part="1"
 AR Path="/6174477C/638DF11B/65833EA0" Ref="C?"  Part="1"
-AR Path="/6174477C/6568C69E/65833EA0" Ref="C45"  Part="1"
+AR Path="/6174477C/6568C69E/65833EA0" Ref="C47"  Part="1"
 AR Path="/6174477C/656DAE2A/65833EA0" Ref="C?"  Part="1"
 AR Path="/6174477C/65729588/65833EA0" Ref="C?"  Part="1"
 AR Path="/6174477C/6572958C/65833EA0" Ref="C?"  Part="1"
 AR Path="/6174477C/6577909A/65833EA0" Ref="C?"  Part="1"
-F 0 "C45" H 8100 4600 50  0000 L CNN
+F 0 "C47" H 8100 4600 50  0000 L CNN
 F 1 "22pF" H 8100 4500 50  0000 L CNN
 F 2 "Capacitor_SMD:C_0402_1005Metric" H 8000 4550 50  0001 C CNN
@@
 AR Path="/6174477C/638385B6/65833EAA" Ref="#PWR?"  Part="1"
 AR Path="/6174477C/638DF11B/65833EAA" Ref="#PWR?"  Part="1"
-AR Path="/6174477C/6568C69E/65833EAA" Ref="#PWR0123"  Part="1"
+AR Path="/6174477C/6568C69E/65833EAA" Ref="#PWR0127"  Part="1"
 AR Path="/6174477C/656DAE2A/65833EAA" Ref="#PWR?"  Part="1"
 AR Path="/6174477C/65729588/65833EAA" Ref="#PWR?"  Part="1"
 AR Path="/6174477C/6572958C/65833EAA" Ref="#PWR?"  Part="1"
 AR Path="/6174477C/6577909A/65833EAA" Ref="#PWR?"  Part="1"
-F 0 "#PWR0123" H 8400 4450 50  0001 C CNN
+F 0 "#PWR0127" H 8400 4450 50  0001 C CNN
 F 1 "GND" H 8405 4527 50  0000 C CNN
 F 2 "" H 8400 4700 50  0001 C CNN
@@
 AR Path="/6174477C/638385B6/65833EB7" Ref="#PWR?"  Part="1"
 AR Path="/6174477C/638DF11B/65833EB7" Ref="#PWR?"  Part="1"
-AR Path="/6174477C/6568C69E/65833EB7" Ref="#PWR0119"  Part="1"
+AR Path="/6174477C/6568C69E/65833EB7" Ref="#PWR0123"  Part="1"
 AR Path="/6174477C/656DAE2A/65833EB7" Ref="#PWR?"  Part="1"
 AR Path="/6174477C/65729588/65833EB7" Ref="#PWR?"  Part="1"
 AR Path="/6174477C/6572958C/65833EB7" Ref="#PWR?"  Part="1"
 AR Path="/6174477C/6577909A/65833EB7" Ref="#PWR?"  Part="1"
-F 0 "#PWR0119" H 8000 4450 50  0001 C CNN
+F 0 "#PWR0123" H 8000 4450 50  0001 C CNN
 F 1 "GND" H 8005 4527 50  0000 C CNN
 F 2 "" H 8000 4700 50  0001 C CNN
@@
 AR Path="/6174477C/638385B6/65833E01" Ref="#PWR?"  Part="1"
 AR Path="/6174477C/638DF11B/65833E01" Ref="#PWR?"  Part="1"
-AR Path="/6174477C/6568C69E/65833E01" Ref="#PWR0120"  Part="1"
+AR Path="/6174477C/6568C69E/65833E01" Ref="#PWR0124"  Part="1"
 AR Path="/6174477C/656DAE2A/65833E01" Ref="#PWR?"  Part="1"
 AR Path="/6174477C/65729588/65833E01" Ref="#PWR?"  Part="1"
 AR Path="/6174477C/6572958C/65833E01" Ref="#PWR?"  Part="1"
 AR Path="/6174477C/6577909A/65833E01" Ref="#PWR?"  Part="1"
-F 0 "#PWR0120" H 8200 3950 50  0001 C CNN
+F 0 "#PWR0124" H 8200 3950 50  0001 C CNN
 F 1 "GND" H 8205 4027 50  0000 C CNN
 F 2 "" H 8200 4200 50  0001 C CNN
@@
 AR Path="/6174477C/638385B6/65833E0D" Ref="#PWR?"  Part="1"
 AR Path="/6174477C/638DF11B/65833E0D" Ref="#PWR?"  Part="1"
-AR Path="/6174477C/6568C69E/65833E0D" Ref="#PWR0121"  Part="1"
+AR Path="/6174477C/6568C69E/65833E0D" Ref="#PWR0125"  Part="1"
 AR Path="/6174477C/656DAE2A/65833E0D" Ref="#PWR?"  Part="1"
 AR Path="/6174477C/65729588/65833E0D" Ref="#PWR?"  Part="1"
 AR Path="/6174477C/6572958C/65833E0D" Ref="#PWR?"  Part="1"
 AR Path="/6174477C/6577909A/65833E0D" Ref="#PWR?"  Part="1"
-F 0 "#PWR0121" H 8200 4150 50  0001 C CNN
+F 0 "#PWR0125" H 8200 4150 50  0001 C CNN
 F 1 "GND" H 8205 4227 50  0000 C CNN
 F 2 "" H 8200 4400 50  0001 C CNN
@@
 AR Path="/6174477C/638385B6/65833E29" Ref="#PWR?"  Part="1"
 AR Path="/6174477C/638DF11B/65833E29" Ref="#PWR?"  Part="1"
-AR Path="/6174477C/6568C69E/65833E29" Ref="#PWR0114"  Part="1"
+AR Path="/6174477C/6568C69E/65833E29" Ref="#PWR0118"  Part="1"
 AR Path="/6174477C/656DAE2A/65833E29" Ref="#PWR?"  Part="1"
 AR Path="/6174477C/65729588/65833E29" Ref="#PWR?"  Part="1"
 AR Path="/6174477C/6572958C/65833E29" Ref="#PWR?"  Part="1"
 AR Path="/6174477C/6577909A/65833E29" Ref="#PWR?"  Part="1"
-F 0 "#PWR0114" H 3500 1650 50  0001 C CNN
+F 0 "#PWR0118" H 3500 1650 50  0001 C CNN
 F 1 "+5V_A" H 3515 1973 50  0000 C CNN
 F 2 "" H 3500 1800 50  0001 C CNN
@@
 AR Path="/6174477C/638385B6/6386EF3F" Ref="#PWR?"  Part="1"
 AR Path="/6174477C/638DF11B/6386EF3F" Ref="#PWR?"  Part="1"
-AR Path="/6174477C/6568C69E/6386EF3F" Ref="#PWR0117"  Part="1"
+AR Path="/6174477C/6568C69E/6386EF3F" Ref="#PWR0121"  Part="1"
 AR Path="/6174477C/656DAE2A/6386EF3F" Ref="#PWR?"  Part="1"
 AR Path="/6174477C/65729588/6386EF3F" Ref="#PWR?"  Part="1"
 AR Path="/6174477C/6572958C/6386EF3F" Ref="#PWR?"  Part="1"
 AR Path="/6174477C/6577909A/6386EF3F" Ref="#PWR?"  Part="1"
-F 0 "#PWR0117" H 4700 2600 50  0001 C CNN
+F 0 "#PWR0121" H 4700 2600 50  0001 C CNN
 F 1 "GND" H 4705 2677 50  0000 C CNN
 F 2 "" H 4700 2850 50  0001 C CNN
@@
 AR Path="/6174477C/638385B6/65833E65" Ref="#PWR?"  Part="1"
 AR Path="/6174477C/638DF11B/65833E65" Ref="#PWR?"  Part="1"
-AR Path="/6174477C/6568C69E/65833E65" Ref="#PWR0116"  Part="1"
+AR Path="/6174477C/6568C69E/65833E65" Ref="#PWR0120"  Part="1"
 AR Path="/6174477C/656DAE2A/65833E65" Ref="#PWR?"  Part="1"
 AR Path="/6174477C/65729588/65833E65" Ref="#PWR?"  Part="1"
 AR Path="/6174477C/6572958C/65833E65" Ref="#PWR?"  Part="1"
 AR Path="/6174477C/6577909A/65833E65" Ref="#PWR?"  Part="1"
-F 0 "#PWR0116" H 4200 5300 50  0001 C CNN
+F 0 "#PWR0120" H 4200 5300 50  0001 C CNN
 F 1 "GND" H 4205 5377 50  0000 C CNN
 F 2 "" H 4200 5550 50  0001 C CNN
@@
 AR Path="/6174477C/638385B6/65833EF2" Ref="#PWR?"  Part="1"
 AR Path="/6174477C/638DF11B/65833EF2" Ref="#PWR?"  Part="1"
-AR Path="/6174477C/6568C69E/65833EF2" Ref="#PWR0122"  Part="1"
+AR Path="/6174477C/6568C69E/65833EF2" Ref="#PWR0126"  Part="1"
 AR Path="/6174477C/656DAE2A/65833EF2" Ref="#PWR?"  Part="1"
 AR Path="/6174477C/65729588/65833EF2" Ref="#PWR?"  Part="1"
 AR Path="/6174477C/6572958C/65833EF2" Ref="#PWR?"  Part="1"
 AR Path="/6174477C/6577909A/65833EF2" Ref="#PWR?"  Part="1"
-F 0 "#PWR0122" H 8400 3100 50  0001 C CNN
+F 0 "#PWR0126" H 8400 3100 50  0001 C CNN
 F 1 "GND" H 8405 3177 50  0000 C CNN
 F 2 "" H 8400 3350 50  0001 C CNN
@@
 AR Path="/6174477C/638385B6/65833DC2" Ref="#PWR?"  Part="1"
 AR Path="/6174477C/638DF11B/65833DC2" Ref="#PWR?"  Part="1"
-AR Path="/6174477C/6568C69E/65833DC2" Ref="#PWR0118"  Part="1"
+AR Path="/6174477C/6568C69E/65833DC2" Ref="#PWR0122"  Part="1"
 AR Path="/6174477C/656DAE2A/65833DC2" Ref="#PWR?"  Part="1"
 AR Path="/6174477C/65729588/65833DC2" Ref="#PWR?"  Part="1"
 AR Path="/6174477C/6572958C/65833DC2" Ref="#PWR?"  Part="1"
 AR Path="/6174477C/6577909A/65833DC2" Ref="#PWR?"  Part="1"
-F 0 "#PWR0118" H 6100 5800 50  0001 C CNN
+F 0 "#PWR0122" H 6100 5800 50  0001 C CNN
 F 1 "GND" H 6105 5877 50  0000 C CNN
 F 2 "" H 6100 6050 50  0001 C CNN
