File: ykts-payload/ykts-mcu-node11.sch (KiCad schematic (older format))
At the start: 12 parts

Commit message: Update nodes
Parts:
- D16: renamed from D?; value NODE0_STATUSLED -> NODE11_STATUSLED
- gave numbers to parts that had none: 11
Connections:
- net NODE0_PWR renamed NODE11_PWR
- net NODE0_RESET renamed NODE11_RESET
- net NODE0_RX renamed NODE11_RX
- net NODE0_TX renamed NODE11_TX
Other:
- note added: "MCU Node 11"
- note removed: "MCU Node 0"
Changed lines of the file:
@@
 AR Path="/6174477C/63801AF0/6386EE2D" Ref="U?"  Part="1"
 AR Path="/6174477C/638385BC/6386EE2D" Ref="U?"  Part="1"
-AR Path="/6174477C/638DF121/6386EE2D" Ref="U?"  Part="1"
-F 0 "U?" H 6100 2711 50  0000 C CNN
+AR Path="/6174477C/638DF121/6386EE2D" Ref="U24"  Part="1"
+F 0 "U24" H 6100 2711 50  0000 C CNN
 F 1 "ATmega328PB-MU" H 6100 2620 50  0000 C CNN
 F 2 "Package_DFN_QFN:QFN-32-1EP_5x5mm_P0.5mm_EP3.1x3.1mm" H 6100 4300 50  0001 C CIN
@@
 AR Path="/6174477C/63801AF0/6391697F" Ref="SW?"  Part="1"
 AR Path="/6174477C/638385BC/6391697F" Ref="SW?"  Part="1"
-AR Path="/6174477C/638DF121/6391697F" Ref="SW?"  Part="1"
-F 0 "SW?" H 3500 2631 50  0000 C CNN
+AR Path="/6174477C/638DF121/6391697F" Ref="SW11"  Part="1"
+F 0 "SW11" H 3500 2631 50  0000 C CNN
 F 1 "ADG802BRT" H 3500 2540 50  0000 C CNN
 F 2 "Package_TO_SOT_SMD:SOT-23-6" H 3500 2500 50  0001 C CNN
@@
 AR Path="/6174477C/63801AF0/63916572" Ref="C?"  Part="1"
 AR Path="/6174477C/638385BC/63916572" Ref="C?"  Part="1"
-AR Path="/6174477C/638DF121/63916572" Ref="C?"  Part="1"
-F 0 "C?" H 4292 2646 50  0000 L CNN
+AR Path="/6174477C/638DF121/63916572" Ref="C68"  Part="1"
+F 0 "C68" H 4292 2646 50  0000 L CNN
 F 1 "1uF" H 4292 2555 50  0000 L CNN
 F 2 "Capacitor_SMD:C_0603_1608Metric" H 4200 2600 50  0001 C CNN
@@
 AR Path="/6174477C/63801AF0/63916573" Ref="C?"  Part="1"
 AR Path="/6174477C/638385BC/63916573" Ref="C?"  Part="1"
-AR Path="/6174477C/638DF121/63916573" Ref="C?"  Part="1"
-F 0 "C?" H 4642 2646 50  0000 L CNN
+AR Path="/6174477C/638DF121/63916573" Ref="C69"  Part="1"
+F 0 "C69" H 4642 2646 50  0000 L CNN
 F 1 "100nF" H 4642 2555 50  0000 L CNN
 F 2 "Capacitor_SMD:C_0402_1005Metric" H 4550 2600 50  0001 C CNN
@@
 AR Path="/6174477C/63801AF0/63916979" Ref="#PWR?"  Part="1"
 AR Path="/6174477C/638385BC/63916979" Ref="#PWR?"  Part="1"
-AR Path="/6174477C/638DF121/63916979" Ref="#PWR?"  Part="1"
-F 0 "#PWR?" H 3500 2600 50  0001 C CNN
+AR Path="/6174477C/638DF121/63916979" Ref="#PWR0257"  Part="1"
+F 0 "#PWR0257" H 3500 2600 50  0001 C CNN
 F 1 "GND" H 3505 2677 50  0000 C CNN
 F 2 "" H 3500 2850 50  0001 C CNN
@@
 AR Path="/6174477C/63801AF0/63760AF5" Ref="C?"  Part="1"
 AR Path="/6174477C/638385BC/63760AF5" Ref="C?"  Part="1"
-AR Path="/6174477C/638DF121/63760AF5" Ref="C?"  Part="1"
-F 0 "C?" H 8100 4600 50  0000 L CNN
+AR Path="/6174477C/638DF121/63760AF5" Ref="C71"  Part="1"
+F 0 "C71" H 8100 4600 50  0000 L CNN
 F 1 "22pF" H 8100 4500 50  0000 L CNN
 F 2 "Capacitor_SMD:C_0402_1005Metric" H 8400 4550 50  0001 C CNN
@@
 AR Path="/6174477C/63801AF0/6391697A" Ref="C?"  Part="1"
 AR Path="/6174477C/638385BC/6391697A" Ref="C?"  Part="1"
-AR Path="/6174477C/638DF121/6391697A" Ref="C?"  Part="1"
-F 0 "C?" H 8100 4600 50  0000 L CNN
+AR Path="/6174477C/638DF121/6391697A" Ref="C70"  Part="1"
+F 0 "C70" H 8100 4600 50  0000 L CNN
 F 1 "22pF" H 8100 4500 50  0000 L CNN
 F 2 "Capacitor_SMD:C_0402_1005Metric" H 8000 4550 50  0001 C CNN
@@
 AR Path="/6174477C/63801AF0/6391697B" Ref="#PWR?"  Part="1"
 AR Path="/6174477C/638385BC/6391697B" Ref="#PWR?"  Part="1"
-AR Path="/6174477C/638DF121/6391697B" Ref="#PWR?"  Part="1"
-F 0 "#PWR?" H 8400 4450 50  0001 C CNN
+AR Path="/6174477C/638DF121/6391697B" Ref="#PWR0258"  Part="1"
+F 0 "#PWR0258" H 8400 4450 50  0001 C CNN
 F 1 "GND" H 8405 4527 50  0000 C CNN
 F 2 "" H 8400 4700 50  0001 C CNN
@@
 AR Path="/6174477C/63801AF0/6391656A" Ref="#PWR?"  Part="1"
 AR Path="/6174477C/638385BC/6391656A" Ref="#PWR?"  Part="1"
-AR Path="/6174477C/638DF121/6391656A" Ref="#PWR?"  Part="1"
-F 0 "#PWR?" H 8000 4450 50  0001 C CNN
+AR Path="/6174477C/638DF121/6391656A" Ref="#PWR0259"  Part="1"
+F 0 "#PWR0259" H 8000 4450 50  0001 C CNN
 F 1 "GND" H 8005 4527 50  0000 C CNN
 F 2 "" H 8000 4700 50  0001 C CNN
@@
 	8400 4700 8400 4650
 Text Label 7050 4600 0    50   ~ 0
-NODE0_RESET
+NODE11_RESET
 $Comp
 L Device:Crystal_GND24_Small Y?
@@
 AR Path="/6174477C/63801AF0/63916574" Ref="Y?"  Part="1"
 AR Path="/6174477C/638385BC/63916574" Ref="Y?"  Part="1"
-AR Path="/6174477C/638DF121/63916574" Ref="Y?"  Part="1"
-F 0 "Y?" H 8450 4350 50  0000 L CNN
+AR Path="/6174477C/638DF121/63916574" Ref="Y13"  Part="1"
+F 0 "Y13" H 8450 4350 50  0000 L CNN
 F 1 "8 MHz" H 8450 4250 50  0000 L CNN
 F 2 "Crystal:Crystal_SMD_2520-4Pin_2.5x2.0mm" H 8200 4300 50  0001 C CNN
@@
 AR Path="/6174477C/63801AF0/63916579" Ref="#PWR?"  Part="1"
 AR Path="/6174477C/638385BC/63916579" Ref="#PWR?"  Part="1"
-AR Path="/6174477C/638DF121/63916579" Ref="#PWR?"  Part="1"
-F 0 "#PWR?" H 8200 3950 50  0001 C CNN
+AR Path="/6174477C/638DF121/63916579" Ref="#PWR0260"  Part="1"
+F 0 "#PWR0260" H 8200 3950 50  0001 C CNN
 F 1 "GND" H 8205 4027 50  0000 C CNN
 F 2 "" H 8200 4200 50  0001 C CNN
@@
 AR Path="/6174477C/63801AF0/6391657A" Ref="#PWR?"  Part="1"
 AR Path="/6174477C/638385BC/6391657A" Ref="#PWR?"  Part="1"
-AR Path="/6174477C/638DF121/6391657A" Ref="#PWR?"  Part="1"
-F 0 "#PWR?" H 8200 4150 50  0001 C CNN
+AR Path="/6174477C/638DF121/6391657A" Ref="#PWR0261"  Part="1"
+F 0 "#PWR0261" H 8200 4150 50  0001 C CNN
 F 1 "GND" H 8205 4227 50  0000 C CNN
 F 2 "" H 8200 4400 50  0001 C CNN
@@
 AR Path="/6174477C/63801AF0/63916973" Ref="R?"  Part="1"
 AR Path="/6174477C/638385BC/63916973" Ref="R?"  Part="1"
-AR Path="/6174477C/638DF121/63916973" Ref="R?"  Part="1"
-F 0 "R?" V 6754 4400 50  0000 C CNN
+AR Path="/6174477C/638DF121/63916973" Ref="R89"  Part="1"
+F 0 "R89" V 6754 4400 50  0000 C CNN
 F 1 "20K" V 6845 4400 50  0000 C CNN
 F 2 "Resistor_SMD:R_0402_1005Metric" H 6950 4400 50  0001 C CNN
@@
 $EndComp
 Text GLabel 2700 2450 0    50   Input ~ 0
-NODE0_PWR
+NODE11_PWR
 Text GLabel 3900 3650 0    50   Input ~ 0
-NODE0_RESET
+NODE11_RESET
 Text GLabel 3900 3750 0    50   Input ~ 0
-NODE0_RX
+NODE11_RX
 Text GLabel 3900 3850 0    50   Input ~ 0
-NODE0_TX
+NODE11_TX
 $Comp
 L yktsat-common:+5V_A #PWR?
@@
 AR Path="/6174477C/63801AF0/63916978" Ref="#PWR?"  Part="1"
 AR Path="/6174477C/638385BC/63916978" Ref="#PWR?"  Part="1"
-AR Path="/6174477C/638DF121/63916978" Ref="#PWR?"  Part="1"
-F 0 "#PWR?" H 3500 1650 50  0001 C CNN
+AR Path="/6174477C/638DF121/63916978" Ref="#PWR0262"  Part="1"
+F 0 "#PWR0262" H 3500 1650 50  0001 C CNN
 F 1 "+5V_A" H 3515 1973 50  0000 C CNN
 F 2 "" H 3500 1800 50  0001 C CNN
@@
 AR Path="/6174477C/63801AF0/6391656C" Ref="#PWR?"  Part="1"
 AR Path="/6174477C/638385BC/6391656C" Ref="#PWR?"  Part="1"
-AR Path="/6174477C/638DF121/6391656C" Ref="#PWR?"  Part="1"
-F 0 "#PWR?" H 4550 2600 50  0001 C CNN
+AR Path="/6174477C/638DF121/6391656C" Ref="#PWR0263"  Part="1"
+F 0 "#PWR0263" H 4550 2600 50  0001 C CNN
 F 1 "GND" H 4555 2677 50  0000 C CNN
 F 2 "" H 4550 2850 50  0001 C CNN
@@
 AR Path="/6174477C/63801AF0/63916575" Ref="R?"  Part="1"
 AR Path="/6174477C/638385BC/63916575" Ref="R?"  Part="1"
-AR Path="/6174477C/638DF121/63916575" Ref="R?"  Part="1"
-F 0 "R?" V 8004 3950 50  0000 C CNN
+AR Path="/6174477C/638DF121/63916575" Ref="R90"  Part="1"
+F 0 "R90" V 8004 3950 50  0000 C CNN
 F 1 "1M" V 8095 3950 50  0000 C CNN
 F 2 "Resistor_SMD:R_0402_1005Metric" H 8200 3950 50  0001 C CNN
@@
 AR Path="/6174477C/63801AF0/63916576" Ref="J?"  Part="1"
 AR Path="/6174477C/638385BC/63916576" Ref="J?"  Part="1"
-AR Path="/6174477C/638DF121/63916576" Ref="J?"  Part="1"
-F 0 "J?" H 3770 5146 50  0000 R CNN
+AR Path="/6174477C/638DF121/63916576" Ref="J16"  Part="1"
+F 0 "J16" H 3770 5146 50  0000 R CNN
 F 1 "AVR-ISP-6" H 3770 5055 50  0000 R CNN
 F 2 "Connector_PinHeader_2.54mm:PinHeader_2x03_P2.54mm_Vertical" V 3850 5100 50  0001 C CNN
@@
 AR Path="/6174477C/63801AF0/63916985" Ref="#PWR?"  Part="1"
 AR Path="/6174477C/638385BC/63916985" Ref="#PWR?"  Part="1"
-AR Path="/6174477C/638DF121/63916985" Ref="#PWR?"  Part="1"
-F 0 "#PWR?" H 4200 5300 50  0001 C CNN
+AR Path="/6174477C/638DF121/63916985" Ref="#PWR0264"  Part="1"
+F 0 "#PWR0264" H 4200 5300 50  0001 C CNN
 F 1 "GND" H 4205 5377 50  0000 C CNN
 F 2 "" H 4200 5550 50  0001 C CNN
@@
 AR Path="/6174477C/63801AF0/63916974" Ref="D?"  Part="1"
 AR Path="/6174477C/638385BC/63916974" Ref="D?"  Part="1"
-AR Path="/6174477C/638DF121/63916974" Ref="D?"  Part="1"
-F 0 "D?" V 8439 2682 50  0000 R CNN
-F 1 "NODE0_STATUSLED" V 8348 2682 50  0000 R CNN
+AR Path="/6174477C/638DF121/63916974" Ref="D16"  Part="1"
+F 0 "D16" V 8439 2682 50  0000 R CNN
+F 1 "NODE11_STATUSLED" V 8348 2682 50  0000 R CNN
 F 2 "LED_SMD:LED_0402_1005Metric" H 8400 2800 50  0001 C CNN
 F 3 "~" H 8400 2800 50  0001 C CNN
@@
 AR Path="/6174477C/63801AF0/63797BAD" Ref="R?"  Part="1"
 AR Path="/6174477C/638385BC/63797BAD" Ref="R?"  Part="1"
-AR Path="/6174477C/638DF121/63797BAD" Ref="R?"  Part="1"
-F 0 "R?" V 8204 3150 50  0000 C CNN
+AR Path="/6174477C/638DF121/63797BAD" Ref="R91"  Part="1"
+F 0 "R91" V 8204 3150 50  0000 C CNN
 F 1 "1K" V 8295 3150 50  0000 C CNN
 F 2 "Resistor_SMD:R_0402_1005Metric" H 8400 3150 50  0001 C CNN
@@
 AR Path="/6174477C/63801AF0/6391697E" Ref="#PWR?"  Part="1"
 AR Path="/6174477C/638385BC/6391697E" Ref="#PWR?"  Part="1"
-AR Path="/6174477C/638DF121/6391697E" Ref="#PWR?"  Part="1"
-F 0 "#PWR?" H 8400 3100 50  0001 C CNN
+AR Path="/6174477C/638DF121/6391697E" Ref="#PWR0265"  Part="1"
+F 0 "#PWR0265" H 8400 3100 50  0001 C CNN
 F 1 "GND" H 8405 3177 50  0000 C CNN
 F 2 "" H 8400 3350 50  0001 C CNN
@@
 AR Path="/6174477C/63801AF0/63916977" Ref="#PWR?"  Part="1"
 AR Path="/6174477C/638385BC/63916977" Ref="#PWR?"  Part="1"
-AR Path="/6174477C/638DF121/63916977" Ref="#PWR?"  Part="1"
-F 0 "#PWR?" H 6100 5800 50  0001 C CNN
+AR Path="/6174477C/638DF121/63916977" Ref="#PWR0266"  Part="1"
+F 0 "#PWR0266" H 6100 5800 50  0001 C CNN
 F 1 "GND" H 6105 5877 50  0000 C CNN
 F 2 "" H 6100 6050 50  0001 C CNN
@@
 	4200 3750 3900 3750
 Text Label 4200 3650 0    50   ~ 0
-NODE0_RESET
+NODE11_RESET
 Wire Wire Line
 	4200 3650 3900 3650
 Text Notes 5700 950  0    100  ~ 0
-MCU Node 0
+MCU Node 11
 Wire Wire Line
 	2700 2450 3100 2450
@@
 ISP_RESET
 Text Label 4200 3550 0    50   ~ 0
-NODE0_RESET
+NODE11_RESET
 Wire Wire Line
 	4200 3550 3900 3550
