File: ykts-payload/ykts-mcu-node11.sch (KiCad schematic (older format))
At the start: 12 parts, among them J24 AVR-ISP-6, SW12 ADG802BRT, U23 ATmega328PB-MU, Y16 8 MHz

Commit message: Revision B2
Hierarchal sheets for nodes
Partial PCB layout
Parts:
- renumbered C83 to C85, C84 to C86, C85 to C87, C86 to C88, U23 to U25
Changed lines of the file:
@@
 Sheet 14 18
 Title "YktSat Payload Module"
-Date "2021-10-22"
-Rev "B0"
+Date "2021-10-26"
+Rev "B1"
 Comp "Sakha Aerospace Systems, LLC"
 Comment1 ""
@@
 AR Path="/6174477C/6572958C/65833EE6" Ref="U?"  Part="1"
 AR Path="/6174477C/6577909A/65833EE6" Ref="U?"  Part="1"
-AR Path="/6174477C/657790A0/65833EE6" Ref="U23"  Part="1"
-F 0 "U23" H 6100 2711 50  0000 C CNN
+AR Path="/6174477C/657790A0/65833EE6" Ref="U25"  Part="1"
+F 0 "U25" H 6100 2711 50  0000 C CNN
 F 1 "ATmega328PB-MU" H 6100 2620 50  0000 C CNN
 F 2 "Package_DFN_QFN:QFN-32-1EP_5x5mm_P0.5mm_EP3.1x3.1mm" H 6100 4300 50  0001 C CIN
@@
 AR Path="/6174477C/6572958C/65833DB7" Ref="C?"  Part="1"
 AR Path="/6174477C/6577909A/65833DB7" Ref="C?"  Part="1"
-AR Path="/6174477C/657790A0/65833DB7" Ref="C83"  Part="1"
-F 0 "C83" H 4442 2646 50  0000 L CNN
+AR Path="/6174477C/657790A0/65833DB7" Ref="C85"  Part="1"
+F 0 "C85" H 4442 2646 50  0000 L CNN
 F 1 "1uF" H 4442 2555 50  0000 L CNN
 F 2 "Capacitor_SMD:C_0603_1608Metric" H 4350 2600 50  0001 C CNN
@@
 AR Path="/6174477C/6572958C/65833ED1" Ref="C?"  Part="1"
 AR Path="/6174477C/6577909A/65833ED1" Ref="C?"  Part="1"
-AR Path="/6174477C/657790A0/65833ED1" Ref="C84"  Part="1"
-F 0 "C84" H 4792 2646 50  0000 L CNN
+AR Path="/6174477C/657790A0/65833ED1" Ref="C86"  Part="1"
+F 0 "C86" H 4792 2646 50  0000 L CNN
 F 1 "100nF" H 4792 2555 50  0000 L CNN
 F 2 "Capacitor_SMD:C_0402_1005Metric" H 4700 2600 50  0001 C CNN
@@
 AR Path="/6174477C/6572958C/65833DE6" Ref="#PWR?"  Part="1"
 AR Path="/6174477C/6577909A/65833DE6" Ref="#PWR?"  Part="1"
-AR Path="/6174477C/657790A0/65833DE6" Ref="#PWR0215"  Part="1"
-F 0 "#PWR0215" H 3500 2600 50  0001 C CNN
+AR Path="/6174477C/657790A0/65833DE6" Ref="#PWR0219"  Part="1"
+F 0 "#PWR0219" H 3500 2600 50  0001 C CNN
 F 1 "GND" H 3505 2677 50  0000 C CNN
 F 2 "" H 3500 2850 50  0001 C CNN
@@
 AR Path="/6174477C/6572958C/65833DF8" Ref="C?"  Part="1"
 AR Path="/6174477C/6577909A/65833DF8" Ref="C?"  Part="1"
-AR Path="/6174477C/657790A0/65833DF8" Ref="C86"  Part="1"
-F 0 "C86" H 8100 4600 50  0000 L CNN
+AR Path="/6174477C/657790A0/65833DF8" Ref="C88"  Part="1"
+F 0 "C88" H 8100 4600 50  0000 L CNN
 F 1 "22pF" H 8100 4500 50  0000 L CNN
 F 2 "Capacitor_SMD:C_0402_1005Metric" H 8400 4550 50  0001 C CNN
@@
 AR Path="/6174477C/6572958C/65833E97" Ref="C?"  Part="1"
 AR Path="/6174477C/6577909A/65833E97" Ref="C?"  Part="1"
-AR Path="/6174477C/657790A0/65833E97" Ref="C85"  Part="1"
-F 0 "C85" H 8100 4600 50  0000 L CNN
+AR Path="/6174477C/657790A0/65833E97" Ref="C87"  Part="1"
+F 0 "C87" H 8100 4600 50  0000 L CNN
 F 1 "22pF" H 8100 4500 50  0000 L CNN
 F 2 "Capacitor_SMD:C_0402_1005Metric" H 8000 4550 50  0001 C CNN
@@
 AR Path="/6174477C/6572958C/65833EAD" Ref="#PWR?"  Part="1"
 AR Path="/6174477C/6577909A/65833EAD" Ref="#PWR?"  Part="1"
-AR Path="/6174477C/657790A0/65833EAD" Ref="#PWR0223"  Part="1"
-F 0 "#PWR0223" H 8400 4450 50  0001 C CNN
+AR Path="/6174477C/657790A0/65833EAD" Ref="#PWR0227"  Part="1"
+F 0 "#PWR0227" H 8400 4450 50  0001 C CNN
 F 1 "GND" H 8405 4527 50  0000 C CNN
 F 2 "" H 8400 4700 50  0001 C CNN
@@
 AR Path="/6174477C/6572958C/65833EB2" Ref="#PWR?"  Part="1"
 AR Path="/6174477C/6577909A/65833EB2" Ref="#PWR?"  Part="1"
-AR Path="/6174477C/657790A0/65833EB2" Ref="#PWR0219"  Part="1"
-F 0 "#PWR0219" H 8000 4450 50  0001 C CNN
+AR Path="/6174477C/657790A0/65833EB2" Ref="#PWR0223"  Part="1"
+F 0 "#PWR0223" H 8000 4450 50  0001 C CNN
 F 1 "GND" H 8005 4527 50  0000 C CNN
 F 2 "" H 8000 4700 50  0001 C CNN
@@
 AR Path="/6174477C/6572958C/65833E02" Ref="#PWR?"  Part="1"
 AR Path="/6174477C/6577909A/65833E02" Ref="#PWR?"  Part="1"
-AR Path="/6174477C/657790A0/65833E02" Ref="#PWR0220"  Part="1"
-F 0 "#PWR0220" H 8200 3950 50  0001 C CNN
+AR Path="/6174477C/657790A0/65833E02" Ref="#PWR0224"  Part="1"
+F 0 "#PWR0224" H 8200 3950 50  0001 C CNN
 F 1 "GND" H 8205 4027 50  0000 C CNN
 F 2 "" H 8200 4200 50  0001 C CNN
@@
 AR Path="/6174477C/6572958C/65833E16" Ref="#PWR?"  Part="1"
 AR Path="/6174477C/6577909A/65833E16" Ref="#PWR?"  Part="1"
-AR Path="/6174477C/657790A0/65833E16" Ref="#PWR0221"  Part="1"
-F 0 "#PWR0221" H 8200 4150 50  0001 C CNN
+AR Path="/6174477C/657790A0/65833E16" Ref="#PWR0225"  Part="1"
+F 0 "#PWR0225" H 8200 4150 50  0001 C CNN
 F 1 "GND" H 8205 4227 50  0000 C CNN
 F 2 "" H 8200 4400 50  0001 C CNN
@@
 AR Path="/6174477C/6572958C/65833E26" Ref="#PWR?"  Part="1"
 AR Path="/6174477C/6577909A/65833E26" Ref="#PWR?"  Part="1"
-AR Path="/6174477C/657790A0/65833E26" Ref="#PWR0214"  Part="1"
-F 0 "#PWR0214" H 3500 1650 50  0001 C CNN
+AR Path="/6174477C/657790A0/65833E26" Ref="#PWR0218"  Part="1"
+F 0 "#PWR0218" H 3500 1650 50  0001 C CNN
 F 1 "+5V_A" H 3515 1973 50  0000 C CNN
 F 2 "" H 3500 1800 50  0001 C CNN
@@
 AR Path="/6174477C/6572958C/65833E36" Ref="#PWR?"  Part="1"
 AR Path="/6174477C/6577909A/65833E36" Ref="#PWR?"  Part="1"
-AR Path="/6174477C/657790A0/65833E36" Ref="#PWR0217"  Part="1"
-F 0 "#PWR0217" H 4700 2600 50  0001 C CNN
+AR Path="/6174477C/657790A0/65833E36" Ref="#PWR0221"  Part="1"
+F 0 "#PWR0221" H 4700 2600 50  0001 C CNN
 F 1 "GND" H 4705 2677 50  0000 C CNN
 F 2 "" H 4700 2850 50  0001 C CNN
@@
 AR Path="/6174477C/6572958C/65833E5E" Ref="#PWR?"  Part="1"
 AR Path="/6174477C/6577909A/65833E5E" Ref="#PWR?"  Part="1"
-AR Path="/6174477C/657790A0/65833E5E" Ref="#PWR0216"  Part="1"
-F 0 "#PWR0216" H 4200 5300 50  0001 C CNN
+AR Path="/6174477C/657790A0/65833E5E" Ref="#PWR0220"  Part="1"
+F 0 "#PWR0220" H 4200 5300 50  0001 C CNN
 F 1 "GND" H 4205 5377 50  0000 C CNN
 F 2 "" H 4200 5550 50  0001 C CNN
@@
 AR Path="/6174477C/6572958C/65833EFA" Ref="#PWR?"  Part="1"
 AR Path="/6174477C/6577909A/65833EFA" Ref="#PWR?"  Part="1"
-AR Path="/6174477C/657790A0/65833EFA" Ref="#PWR0222"  Part="1"
-F 0 "#PWR0222" H 8400 3100 50  0001 C CNN
+AR Path="/6174477C/657790A0/65833EFA" Ref="#PWR0226"  Part="1"
+F 0 "#PWR0226" H 8400 3100 50  0001 C CNN
 F 1 "GND" H 8405 3177 50  0000 C CNN
 F 2 "" H 8400 3350 50  0001 C CNN
@@
 AR Path="/6174477C/6572958C/65833DC4" Ref="#PWR?"  Part="1"
 AR Path="/6174477C/6577909A/65833DC4" Ref="#PWR?"  Part="1"
-AR Path="/6174477C/657790A0/65833DC4" Ref="#PWR0218"  Part="1"
-F 0 "#PWR0218" H 6100 5800 50  0001 C CNN
+AR Path="/6174477C/657790A0/65833DC4" Ref="#PWR0222"  Part="1"
+F 0 "#PWR0222" H 6100 5800 50  0001 C CNN
 F 1 "GND" H 6105 5877 50  0000 C CNN
 F 2 "" H 6100 6050 50  0001 C CNN
