File: ykts-payload/ykts-mcu-node13.sch (KiCad schematic (older format))
At the start: 12 parts, among them J26 AVR-ISP-6, SW14 ADG802BRT, U25 ATmega328PB-MU, Y18 8 MHz

Commit message: Revision B2
Hierarchal sheets for nodes
Partial PCB layout
Parts:
- renumbered C91 to C93, C92 to C94, C93 to C95, C94 to C96, U25 to U27
Changed lines of the file:
@@
 Sheet 16 18
 Title "YktSat Payload Module"
-Date "2021-10-22"
-Rev "B0"
+Date "2021-10-26"
+Rev "B1"
 Comp "Sakha Aerospace Systems, LLC"
 Comment1 ""
@@
 AR Path="/6174477C/6572958C/65833EDE" Ref="U?"  Part="1"
 AR Path="/6174477C/6577909A/65833EDE" Ref="U?"  Part="1"
-AR Path="/6174477C/657790A4/65833EDE" Ref="U25"  Part="1"
-F 0 "U25" H 6100 2711 50  0000 C CNN
+AR Path="/6174477C/657790A4/65833EDE" Ref="U27"  Part="1"
+F 0 "U27" H 6100 2711 50  0000 C CNN
 F 1 "ATmega328PB-MU" H 6100 2620 50  0000 C CNN
 F 2 "Package_DFN_QFN:QFN-32-1EP_5x5mm_P0.5mm_EP3.1x3.1mm" H 6100 4300 50  0001 C CIN
@@
 AR Path="/6174477C/6572958C/65833DBF" Ref="C?"  Part="1"
 AR Path="/6174477C/6577909A/65833DBF" Ref="C?"  Part="1"
-AR Path="/6174477C/657790A4/65833DBF" Ref="C91"  Part="1"
-F 0 "C91" H 4442 2646 50  0000 L CNN
+AR Path="/6174477C/657790A4/65833DBF" Ref="C93"  Part="1"
+F 0 "C93" H 4442 2646 50  0000 L CNN
 F 1 "1uF" H 4442 2555 50  0000 L CNN
 F 2 "Capacitor_SMD:C_0603_1608Metric" H 4350 2600 50  0001 C CNN
@@
 AR Path="/6174477C/6572958C/65833ED2" Ref="C?"  Part="1"
 AR Path="/6174477C/6577909A/65833ED2" Ref="C?"  Part="1"
-AR Path="/6174477C/657790A4/65833ED2" Ref="C92"  Part="1"
-F 0 "C92" H 4792 2646 50  0000 L CNN
+AR Path="/6174477C/657790A4/65833ED2" Ref="C94"  Part="1"
+F 0 "C94" H 4792 2646 50  0000 L CNN
 F 1 "100nF" H 4792 2555 50  0000 L CNN
 F 2 "Capacitor_SMD:C_0402_1005Metric" H 4700 2600 50  0001 C CNN
@@
 AR Path="/6174477C/6572958C/65833DEA" Ref="#PWR?"  Part="1"
 AR Path="/6174477C/6577909A/65833DEA" Ref="#PWR?"  Part="1"
-AR Path="/6174477C/657790A4/65833DEA" Ref="#PWR0235"  Part="1"
-F 0 "#PWR0235" H 3500 2600 50  0001 C CNN
+AR Path="/6174477C/657790A4/65833DEA" Ref="#PWR0239"  Part="1"
+F 0 "#PWR0239" H 3500 2600 50  0001 C CNN
 F 1 "GND" H 3505 2677 50  0000 C CNN
 F 2 "" H 3500 2850 50  0001 C CNN
@@
 AR Path="/6174477C/6572958C/65833DFC" Ref="C?"  Part="1"
 AR Path="/6174477C/6577909A/65833DFC" Ref="C?"  Part="1"
-AR Path="/6174477C/657790A4/65833DFC" Ref="C94"  Part="1"
-F 0 "C94" H 8100 4600 50  0000 L CNN
+AR Path="/6174477C/657790A4/65833DFC" Ref="C96"  Part="1"
+F 0 "C96" H 8100 4600 50  0000 L CNN
 F 1 "22pF" H 8100 4500 50  0000 L CNN
 F 2 "Capacitor_SMD:C_0402_1005Metric" H 8400 4550 50  0001 C CNN
@@
 AR Path="/6174477C/6572958C/65833EA1" Ref="C?"  Part="1"
 AR Path="/6174477C/6577909A/65833EA1" Ref="C?"  Part="1"
-AR Path="/6174477C/657790A4/65833EA1" Ref="C93"  Part="1"
-F 0 "C93" H 8100 4600 50  0000 L CNN
+AR Path="/6174477C/657790A4/65833EA1" Ref="C95"  Part="1"
+F 0 "C95" H 8100 4600 50  0000 L CNN
 F 1 "22pF" H 8100 4500 50  0000 L CNN
 F 2 "Capacitor_SMD:C_0402_1005Metric" H 8000 4550 50  0001 C CNN
@@
 AR Path="/6174477C/6572958C/65833EAF" Ref="#PWR?"  Part="1"
 AR Path="/6174477C/6577909A/65833EAF" Ref="#PWR?"  Part="1"
-AR Path="/6174477C/657790A4/65833EAF" Ref="#PWR0243"  Part="1"
-F 0 "#PWR0243" H 8400 4450 50  0001 C CNN
+AR Path="/6174477C/657790A4/65833EAF" Ref="#PWR0247"  Part="1"
+F 0 "#PWR0247" H 8400 4450 50  0001 C CNN
 F 1 "GND" H 8405 4527 50  0000 C CNN
 F 2 "" H 8400 4700 50  0001 C CNN
@@
 AR Path="/6174477C/6572958C/6391666E" Ref="#PWR?"  Part="1"
 AR Path="/6174477C/6577909A/6391666E" Ref="#PWR?"  Part="1"
-AR Path="/6174477C/657790A4/6391666E" Ref="#PWR0239"  Part="1"
-F 0 "#PWR0239" H 8000 4450 50  0001 C CNN
+AR Path="/6174477C/657790A4/6391666E" Ref="#PWR0243"  Part="1"
+F 0 "#PWR0243" H 8000 4450 50  0001 C CNN
 F 1 "GND" H 8005 4527 50  0000 C CNN
 F 2 "" H 8000 4700 50  0001 C CNN
@@
 AR Path="/6174477C/6572958C/65833E0A" Ref="#PWR?"  Part="1"
 AR Path="/6174477C/6577909A/65833E0A" Ref="#PWR?"  Part="1"
-AR Path="/6174477C/657790A4/65833E0A" Ref="#PWR0240"  Part="1"
-F 0 "#PWR0240" H 8200 3950 50  0001 C CNN
+AR Path="/6174477C/657790A4/65833E0A" Ref="#PWR0244"  Part="1"
+F 0 "#PWR0244" H 8200 3950 50  0001 C CNN
 F 1 "GND" H 8205 4027 50  0000 C CNN
 F 2 "" H 8200 4200 50  0001 C CNN
@@
 AR Path="/6174477C/6572958C/65833E19" Ref="#PWR?"  Part="1"
 AR Path="/6174477C/6577909A/65833E19" Ref="#PWR?"  Part="1"
-AR Path="/6174477C/657790A4/65833E19" Ref="#PWR0241"  Part="1"
-F 0 "#PWR0241" H 8200 4150 50  0001 C CNN
+AR Path="/6174477C/657790A4/65833E19" Ref="#PWR0245"  Part="1"
+F 0 "#PWR0245" H 8200 4150 50  0001 C CNN
 F 1 "GND" H 8205 4227 50  0000 C CNN
 F 2 "" H 8200 4400 50  0001 C CNN
@@
 AR Path="/6174477C/6572958C/65833E28" Ref="#PWR?"  Part="1"
 AR Path="/6174477C/6577909A/65833E28" Ref="#PWR?"  Part="1"
-AR Path="/6174477C/657790A4/65833E28" Ref="#PWR0234"  Part="1"
-F 0 "#PWR0234" H 3500 1650 50  0001 C CNN
+AR Path="/6174477C/657790A4/65833E28" Ref="#PWR0238"  Part="1"
+F 0 "#PWR0238" H 3500 1650 50  0001 C CNN
 F 1 "+5V_A" H 3515 1973 50  0000 C CNN
 F 2 "" H 3500 1800 50  0001 C CNN
@@
 AR Path="/6174477C/6572958C/65833E32" Ref="#PWR?"  Part="1"
 AR Path="/6174477C/6577909A/65833E32" Ref="#PWR?"  Part="1"
-AR Path="/6174477C/657790A4/65833E32" Ref="#PWR0237"  Part="1"
-F 0 "#PWR0237" H 4700 2600 50  0001 C CNN
+AR Path="/6174477C/657790A4/65833E32" Ref="#PWR0241"  Part="1"
+F 0 "#PWR0241" H 4700 2600 50  0001 C CNN
 F 1 "GND" H 4705 2677 50  0000 C CNN
 F 2 "" H 4700 2850 50  0001 C CNN
@@
 AR Path="/6174477C/6572958C/65833E60" Ref="#PWR?"  Part="1"
 AR Path="/6174477C/6577909A/65833E60" Ref="#PWR?"  Part="1"
-AR Path="/6174477C/657790A4/65833E60" Ref="#PWR0236"  Part="1"
-F 0 "#PWR0236" H 4200 5300 50  0001 C CNN
+AR Path="/6174477C/657790A4/65833E60" Ref="#PWR0240"  Part="1"
+F 0 "#PWR0240" H 4200 5300 50  0001 C CNN
 F 1 "GND" H 4205 5377 50  0000 C CNN
 F 2 "" H 4200 5550 50  0001 C CNN
@@
 AR Path="/6174477C/6572958C/65833EF8" Ref="#PWR?"  Part="1"
 AR Path="/6174477C/6577909A/65833EF8" Ref="#PWR?"  Part="1"
-AR Path="/6174477C/657790A4/65833EF8" Ref="#PWR0242"  Part="1"
-F 0 "#PWR0242" H 8400 3100 50  0001 C CNN
+AR Path="/6174477C/657790A4/65833EF8" Ref="#PWR0246"  Part="1"
+F 0 "#PWR0246" H 8400 3100 50  0001 C CNN
 F 1 "GND" H 8405 3177 50  0000 C CNN
 F 2 "" H 8400 3350 50  0001 C CNN
@@
 AR Path="/6174477C/6572958C/65833DC6" Ref="#PWR?"  Part="1"
 AR Path="/6174477C/6577909A/65833DC6" Ref="#PWR?"  Part="1"
-AR Path="/6174477C/657790A4/65833DC6" Ref="#PWR0238"  Part="1"
-F 0 "#PWR0238" H 6100 5800 50  0001 C CNN
+AR Path="/6174477C/657790A4/65833DC6" Ref="#PWR0242"  Part="1"
+F 0 "#PWR0242" H 6100 5800 50  0001 C CNN
 F 1 "GND" H 6105 5877 50  0000 C CNN
 F 2 "" H 6100 6050 50  0001 C CNN
