File: ykts-payload/ykts-mcu-node8.sch (KiCad schematic (older format))
At the start: 12 parts

Commit message: Update nodes
Parts:
- D13: renamed from D?; value NODE0_STATUSLED -> NODE8_STATUSLED
- gave numbers to parts that had none: 11
Connections:
- net NODE0_PWR renamed NODE8_PWR
- net NODE0_RESET renamed NODE8_RESET
- net NODE0_RX renamed NODE8_RX
- net NODE0_TX renamed NODE8_TX
Other:
- note added: "MCU Node 8"
- note removed: "MCU Node 0"

Commit message: Fixed annotations & sheet ordering
Parts:
- renumbered C56 to C60, C57 to C61, C58 to C62, C59 to C63, D13 to D17, J13 to J16, R80 to R93, R81 to R94, R82 to R95, SW8 to SW9, U21 to U22, Y10 to Y11
Changed lines of the file:
@@
 Sheet 10 18
 Title "YktSat Payload Module"
-Date "2021-09-30"
-Rev "A0"
+Date "2021-10-02"
+Rev "A1"
 Comp "Sakha Aerospace Systems, LLC"
 Comment1 ""
@@
 AR Path="/6174477C/63801AEE/6386EF39" Ref="U?"  Part="1"
 AR Path="/6174477C/638385B6/6386EF39" Ref="U?"  Part="1"
-AR Path="/6174477C/638DF11B/6386EF39" Ref="U21"  Part="1"
-F 0 "U21" H 6100 2711 50  0000 C CNN
+AR Path="/6174477C/638DF11B/6386EF39" Ref="U22"  Part="1"
+F 0 "U22" H 6100 2711 50  0000 C CNN
 F 1 "ATmega328PB-MU" H 6100 2620 50  0000 C CNN
 F 2 "Package_DFN_QFN:QFN-32-1EP_5x5mm_P0.5mm_EP3.1x3.1mm" H 6100 4300 50  0001 C CIN
@@
 AR Path="/6174477C/63801AEE/6375A038" Ref="SW?"  Part="1"
 AR Path="/6174477C/638385B6/6375A038" Ref="SW?"  Part="1"
-AR Path="/6174477C/638DF11B/6375A038" Ref="SW8"  Part="1"
-F 0 "SW8" H 3500 2631 50  0000 C CNN
+AR Path="/6174477C/638DF11B/6375A038" Ref="SW9"  Part="1"
+F 0 "SW9" H 3500 2631 50  0000 C CNN
 F 1 "ADG802BRT" H 3500 2540 50  0000 C CNN
 F 2 "Package_TO_SOT_SMD:SOT-23-6" H 3500 2500 50  0001 C CNN
@@
 AR Path="/6174477C/63801AEE/6391666A" Ref="C?"  Part="1"
 AR Path="/6174477C/638385B6/6391666A" Ref="C?"  Part="1"
-AR Path="/6174477C/638DF11B/6391666A" Ref="C56"  Part="1"
-F 0 "C56" H 4292 2646 50  0000 L CNN
+AR Path="/6174477C/638DF11B/6391666A" Ref="C60"  Part="1"
+F 0 "C60" H 4292 2646 50  0000 L CNN
 F 1 "1uF" H 4292 2555 50  0000 L CNN
 F 2 "Capacitor_SMD:C_0603_1608Metric" H 4200 2600 50  0001 C CNN
@@
 AR Path="/6174477C/63801AEE/6386EF32" Ref="C?"  Part="1"
 AR Path="/6174477C/638385B6/6386EF32" Ref="C?"  Part="1"
-AR Path="/6174477C/638DF11B/6386EF32" Ref="C57"  Part="1"
-F 0 "C57" H 4642 2646 50  0000 L CNN
+AR Path="/6174477C/638DF11B/6386EF32" Ref="C61"  Part="1"
+F 0 "C61" H 4642 2646 50  0000 L CNN
 F 1 "100nF" H 4642 2555 50  0000 L CNN
 F 2 "Capacitor_SMD:C_0402_1005Metric" H 4550 2600 50  0001 C CNN
@@
 AR Path="/6174477C/63801AEE/63916671" Ref="#PWR?"  Part="1"
 AR Path="/6174477C/638385B6/63916671" Ref="#PWR?"  Part="1"
-AR Path="/6174477C/638DF11B/63916671" Ref="#PWR0227"  Part="1"
-F 0 "#PWR0227" H 3500 2600 50  0001 C CNN
+AR Path="/6174477C/638DF11B/63916671" Ref="#PWR0169"  Part="1"
+F 0 "#PWR0169" H 3500 2600 50  0001 C CNN
 F 1 "GND" H 3505 2677 50  0000 C CNN
 F 2 "" H 3500 2850 50  0001 C CNN
@@
 AR Path="/6174477C/63801AEE/63916672" Ref="C?"  Part="1"
 AR Path="/6174477C/638385B6/63916672" Ref="C?"  Part="1"
-AR Path="/6174477C/638DF11B/63916672" Ref="C59"  Part="1"
-F 0 "C59" H 8100 4600 50  0000 L CNN
+AR Path="/6174477C/638DF11B/63916672" Ref="C63"  Part="1"
+F 0 "C63" H 8100 4600 50  0000 L CNN
 F 1 "22pF" H 8100 4500 50  0000 L CNN
 F 2 "Capacitor_SMD:C_0402_1005Metric" H 8400 4550 50  0001 C CNN
@@
 AR Path="/6174477C/63801AEE/638383B5" Ref="C?"  Part="1"
 AR Path="/6174477C/638385B6/638383B5" Ref="C?"  Part="1"
-AR Path="/6174477C/638DF11B/638383B5" Ref="C58"  Part="1"
-F 0 "C58" H 8100 4600 50  0000 L CNN
+AR Path="/6174477C/638DF11B/638383B5" Ref="C62"  Part="1"
+F 0 "C62" H 8100 4600 50  0000 L CNN
 F 1 "22pF" H 8100 4500 50  0000 L CNN
 F 2 "Capacitor_SMD:C_0402_1005Metric" H 8000 4550 50  0001 C CNN
@@
 AR Path="/6174477C/63801AEE/638383B6" Ref="#PWR?"  Part="1"
 AR Path="/6174477C/638385B6/638383B6" Ref="#PWR?"  Part="1"
-AR Path="/6174477C/638DF11B/638383B6" Ref="#PWR0228"  Part="1"
-F 0 "#PWR0228" H 8400 4450 50  0001 C CNN
+AR Path="/6174477C/638DF11B/638383B6" Ref="#PWR0177"  Part="1"
+F 0 "#PWR0177" H 8400 4450 50  0001 C CNN
 F 1 "GND" H 8405 4527 50  0000 C CNN
 F 2 "" H 8400 4700 50  0001 C CNN
@@
 AR Path="/6174477C/63801AEE/638383B7" Ref="#PWR?"  Part="1"
 AR Path="/6174477C/638385B6/638383B7" Ref="#PWR?"  Part="1"
-AR Path="/6174477C/638DF11B/638383B7" Ref="#PWR0229"  Part="1"
-F 0 "#PWR0229" H 8000 4450 50  0001 C CNN
+AR Path="/6174477C/638DF11B/638383B7" Ref="#PWR0173"  Part="1"
+F 0 "#PWR0173" H 8000 4450 50  0001 C CNN
 F 1 "GND" H 8005 4527 50  0000 C CNN
 F 2 "" H 8000 4700 50  0001 C CNN
@@
 AR Path="/6174477C/63801AEE/638383B8" Ref="Y?"  Part="1"
 AR Path="/6174477C/638385B6/638383B8" Ref="Y?"  Part="1"
-AR Path="/6174477C/638DF11B/638383B8" Ref="Y10"  Part="1"
-F 0 "Y10" H 8450 4350 50  0000 L CNN
+AR Path="/6174477C/638DF11B/638383B8" Ref="Y11"  Part="1"
+F 0 "Y11" H 8450 4350 50  0000 L CNN
 F 1 "8 MHz" H 8450 4250 50  0000 L CNN
 F 2 "Crystal:Crystal_SMD_2520-4Pin_2.5x2.0mm" H 8200 4300 50  0001 C CNN
@@
 AR Path="/6174477C/63801AEE/63916673" Ref="#PWR?"  Part="1"
 AR Path="/6174477C/638385B6/63916673" Ref="#PWR?"  Part="1"
-AR Path="/6174477C/638DF11B/63916673" Ref="#PWR0230"  Part="1"
-F 0 "#PWR0230" H 8200 3950 50  0001 C CNN
+AR Path="/6174477C/638DF11B/63916673" Ref="#PWR0174"  Part="1"
+F 0 "#PWR0174" H 8200 3950 50  0001 C CNN
 F 1 "GND" H 8205 4027 50  0000 C CNN
 F 2 "" H 8200 4200 50  0001 C CNN
@@
 AR Path="/6174477C/63801AEE/63916674" Ref="#PWR?"  Part="1"
 AR Path="/6174477C/638385B6/63916674" Ref="#PWR?"  Part="1"
-AR Path="/6174477C/638DF11B/63916674" Ref="#PWR0231"  Part="1"
-F 0 "#PWR0231" H 8200 4150 50  0001 C CNN
+AR Path="/6174477C/638DF11B/63916674" Ref="#PWR0175"  Part="1"
+F 0 "#PWR0175" H 8200 4150 50  0001 C CNN
 F 1 "GND" H 8205 4227 50  0000 C CNN
 F 2 "" H 8200 4400 50  0001 C CNN
@@
 AR Path="/6174477C/63801AEE/63916670" Ref="R?"  Part="1"
 AR Path="/6174477C/638385B6/63916670" Ref="R?"  Part="1"
-AR Path="/6174477C/638DF11B/63916670" Ref="R80"  Part="1"
-F 0 "R80" V 6754 4400 50  0000 C CNN
+AR Path="/6174477C/638DF11B/63916670" Ref="R93"  Part="1"
+F 0 "R93" V 6754 4400 50  0000 C CNN
 F 1 "20K" V 6845 4400 50  0000 C CNN
 F 2 "Resistor_SMD:R_0402_1005Metric" H 6950 4400 50  0001 C CNN
@@
 AR Path="/6174477C/63801AEE/63916675" Ref="#PWR?"  Part="1"
 AR Path="/6174477C/638385B6/63916675" Ref="#PWR?"  Part="1"
-AR Path="/6174477C/638DF11B/63916675" Ref="#PWR0232"  Part="1"
-F 0 "#PWR0232" H 3500 1650 50  0001 C CNN
+AR Path="/6174477C/638DF11B/63916675" Ref="#PWR0168"  Part="1"
+F 0 "#PWR0168" H 3500 1650 50  0001 C CNN
 F 1 "+5V_A" H 3515 1973 50  0000 C CNN
 F 2 "" H 3500 1800 50  0001 C CNN
@@
 AR Path="/6174477C/63801AEE/63916678" Ref="#PWR?"  Part="1"
 AR Path="/6174477C/638385B6/63916678" Ref="#PWR?"  Part="1"
-AR Path="/6174477C/638DF11B/63916678" Ref="#PWR0233"  Part="1"
-F 0 "#PWR0233" H 4550 2600 50  0001 C CNN
+AR Path="/6174477C/638DF11B/63916678" Ref="#PWR0171"  Part="1"
+F 0 "#PWR0171" H 4550 2600 50  0001 C CNN
 F 1 "GND" H 4555 2677 50  0000 C CNN
 F 2 "" H 4550 2850 50  0001 C CNN
@@
 AR Path="/6174477C/63801AEE/63916679" Ref="R?"  Part="1"
 AR Path="/6174477C/638385B6/63916679" Ref="R?"  Part="1"
-AR Path="/6174477C/638DF11B/63916679" Ref="R81"  Part="1"
-F 0 "R81" V 8004 3950 50  0000 C CNN
+AR Path="/6174477C/638DF11B/63916679" Ref="R94"  Part="1"
+F 0 "R94" V 8004 3950 50  0000 C CNN
 F 1 "1M" V 8095 3950 50  0000 C CNN
 F 2 "Resistor_SMD:R_0402_1005Metric" H 8200 3950 50  0001 C CNN
@@
 AR Path="/6174477C/63801AEE/6391667A" Ref="J?"  Part="1"
 AR Path="/6174477C/638385B6/6391667A" Ref="J?"  Part="1"
-AR Path="/6174477C/638DF11B/6391667A" Ref="J13"  Part="1"
-F 0 "J13" H 3770 5146 50  0000 R CNN
+AR Path="/6174477C/638DF11B/6391667A" Ref="J16"  Part="1"
+F 0 "J16" H 3770 5146 50  0000 R CNN
 F 1 "AVR-ISP-6" H 3770 5055 50  0000 R CNN
 F 2 "Connector_PinHeader_2.54mm:PinHeader_2x03_P2.54mm_Vertical" V 3850 5100 50  0001 C CNN
@@
 AR Path="/6174477C/63801AEE/6391667B" Ref="#PWR?"  Part="1"
 AR Path="/6174477C/638385B6/6391667B" Ref="#PWR?"  Part="1"
-AR Path="/6174477C/638DF11B/6391667B" Ref="#PWR0234"  Part="1"
-F 0 "#PWR0234" H 4200 5300 50  0001 C CNN
+AR Path="/6174477C/638DF11B/6391667B" Ref="#PWR0170"  Part="1"
+F 0 "#PWR0170" H 4200 5300 50  0001 C CNN
 F 1 "GND" H 4205 5377 50  0000 C CNN
 F 2 "" H 4200 5550 50  0001 C CNN
@@
 AR Path="/6174477C/63801AEE/6391667C" Ref="D?"  Part="1"
 AR Path="/6174477C/638385B6/6391667C" Ref="D?"  Part="1"
-AR Path="/6174477C/638DF11B/6391667C" Ref="D13"  Part="1"
-F 0 "D13" V 8439 2682 50  0000 R CNN
+AR Path="/6174477C/638DF11B/6391667C" Ref="D17"  Part="1"
+F 0 "D17" V 8439 2682 50  0000 R CNN
 F 1 "NODE8_STATUSLED" V 8348 2682 50  0000 R CNN
 F 2 "LED_SMD:LED_0402_1005Metric" H 8400 2800 50  0001 C CNN
@@
 AR Path="/6174477C/63801AEE/6391667D" Ref="R?"  Part="1"
 AR Path="/6174477C/638385B6/6391667D" Ref="R?"  Part="1"
-AR Path="/6174477C/638DF11B/6391667D" Ref="R82"  Part="1"
-F 0 "R82" V 8204 3150 50  0000 C CNN
+AR Path="/6174477C/638DF11B/6391667D" Ref="R95"  Part="1"
+F 0 "R95" V 8204 3150 50  0000 C CNN
 F 1 "1K" V 8295 3150 50  0000 C CNN
 F 2 "Resistor_SMD:R_0402_1005Metric" H 8400 3150 50  0001 C CNN
@@
 AR Path="/6174477C/63801AEE/6386EF45" Ref="#PWR?"  Part="1"
 AR Path="/6174477C/638385B6/6386EF45" Ref="#PWR?"  Part="1"
-AR Path="/6174477C/638DF11B/6386EF45" Ref="#PWR0235"  Part="1"
-F 0 "#PWR0235" H 8400 3100 50  0001 C CNN
+AR Path="/6174477C/638DF11B/6386EF45" Ref="#PWR0176"  Part="1"
+F 0 "#PWR0176" H 8400 3100 50  0001 C CNN
 F 1 "GND" H 8405 3177 50  0000 C CNN
 F 2 "" H 8400 3350 50  0001 C CNN
@@
 AR Path="/6174477C/63801AEE/6391666B" Ref="#PWR?"  Part="1"
 AR Path="/6174477C/638385B6/6391666B" Ref="#PWR?"  Part="1"
-AR Path="/6174477C/638DF11B/6391666B" Ref="#PWR0236"  Part="1"
-F 0 "#PWR0236" H 6100 5800 50  0001 C CNN
+AR Path="/6174477C/638DF11B/6391666B" Ref="#PWR0172"  Part="1"
+F 0 "#PWR0172" H 6100 5800 50  0001 C CNN
 F 1 "GND" H 6105 5877 50  0000 C CNN
 F 2 "" H 6100 6050 50  0001 C CNN

Commit message: Revision A2
Added debug power
Basic ESD protection on UART
MCP Reset from MCU
Parts:
- renumbered D17 to D16, J16 to J17, R93 to R97, R94 to R98, R95 to R99
Changed lines of the file:
@@
 $Descr A4 11693 8268
 encoding utf-8
-Sheet 10 18
+Sheet 11 18
 Title "YktSat Payload Module"
-Date "2021-10-02"
-Rev "A1"
+Date "2021-10-03"
+Rev "A2"
 Comp "Sakha Aerospace Systems, LLC"
 Comment1 ""
@@
 AR Path="/6174477C/63801AEE/63916671" Ref="#PWR?"  Part="1"
 AR Path="/6174477C/638385B6/63916671" Ref="#PWR?"  Part="1"
-AR Path="/6174477C/638DF11B/63916671" Ref="#PWR0169"  Part="1"
-F 0 "#PWR0169" H 3500 2600 50  0001 C CNN
+AR Path="/6174477C/638DF11B/63916671" Ref="#PWR0171"  Part="1"
+F 0 "#PWR0171" H 3500 2600 50  0001 C CNN
 F 1 "GND" H 3505 2677 50  0000 C CNN
 F 2 "" H 3500 2850 50  0001 C CNN
@@
 AR Path="/6174477C/63801AEE/638383B6" Ref="#PWR?"  Part="1"
 AR Path="/6174477C/638385B6/638383B6" Ref="#PWR?"  Part="1"
-AR Path="/6174477C/638DF11B/638383B6" Ref="#PWR0177"  Part="1"
-F 0 "#PWR0177" H 8400 4450 50  0001 C CNN
+AR Path="/6174477C/638DF11B/638383B6" Ref="#PWR0179"  Part="1"
+F 0 "#PWR0179" H 8400 4450 50  0001 C CNN
 F 1 "GND" H 8405 4527 50  0000 C CNN
 F 2 "" H 8400 4700 50  0001 C CNN
@@
 AR Path="/6174477C/63801AEE/638383B7" Ref="#PWR?"  Part="1"
 AR Path="/6174477C/638385B6/638383B7" Ref="#PWR?"  Part="1"
-AR Path="/6174477C/638DF11B/638383B7" Ref="#PWR0173"  Part="1"
-F 0 "#PWR0173" H 8000 4450 50  0001 C CNN
+AR Path="/6174477C/638DF11B/638383B7" Ref="#PWR0175"  Part="1"
+F 0 "#PWR0175" H 8000 4450 50  0001 C CNN
 F 1 "GND" H 8005 4527 50  0000 C CNN
 F 2 "" H 8000 4700 50  0001 C CNN
@@
 AR Path="/6174477C/63801AEE/63916673" Ref="#PWR?"  Part="1"
 AR Path="/6174477C/638385B6/63916673" Ref="#PWR?"  Part="1"
-AR Path="/6174477C/638DF11B/63916673" Ref="#PWR0174"  Part="1"
-F 0 "#PWR0174" H 8200 3950 50  0001 C CNN
+AR Path="/6174477C/638DF11B/63916673" Ref="#PWR0176"  Part="1"
+F 0 "#PWR0176" H 8200 3950 50  0001 C CNN
 F 1 "GND" H 8205 4027 50  0000 C CNN
 F 2 "" H 8200 4200 50  0001 C CNN
@@
 AR Path="/6174477C/63801AEE/63916674" Ref="#PWR?"  Part="1"
 AR Path="/6174477C/638385B6/63916674" Ref="#PWR?"  Part="1"
-AR Path="/6174477C/638DF11B/63916674" Ref="#PWR0175"  Part="1"
-F 0 "#PWR0175" H 8200 4150 50  0001 C CNN
+AR Path="/6174477C/638DF11B/63916674" Ref="#PWR0177"  Part="1"
+F 0 "#PWR0177" H 8200 4150 50  0001 C CNN
 F 1 "GND" H 8205 4227 50  0000 C CNN
 F 2 "" H 8200 4400 50  0001 C CNN
@@
 AR Path="/6174477C/63801AEE/63916670" Ref="R?"  Part="1"
 AR Path="/6174477C/638385B6/63916670" Ref="R?"  Part="1"
-AR Path="/6174477C/638DF11B/63916670" Ref="R93"  Part="1"
-F 0 "R93" V 6754 4400 50  0000 C CNN
+AR Path="/6174477C/638DF11B/63916670" Ref="R97"  Part="1"
+F 0 "R97" V 6754 4400 50  0000 C CNN
 F 1 "20K" V 6845 4400 50  0000 C CNN
 F 2 "Resistor_SMD:R_0402_1005Metric" H 6950 4400 50  0001 C CNN
@@
 AR Path="/6174477C/63801AEE/63916675" Ref="#PWR?"  Part="1"
 AR Path="/6174477C/638385B6/63916675" Ref="#PWR?"  Part="1"
-AR Path="/6174477C/638DF11B/63916675" Ref="#PWR0168"  Part="1"
-F 0 "#PWR0168" H 3500 1650 50  0001 C CNN
+AR Path="/6174477C/638DF11B/63916675" Ref="#PWR0170"  Part="1"
+F 0 "#PWR0170" H 3500 1650 50  0001 C CNN
 F 1 "+5V_A" H 3515 1973 50  0000 C CNN
 F 2 "" H 3500 1800 50  0001 C CNN
@@
 AR Path="/6174477C/63801AEE/63916678" Ref="#PWR?"  Part="1"
 AR Path="/6174477C/638385B6/63916678" Ref="#PWR?"  Part="1"
-AR Path="/6174477C/638DF11B/63916678" Ref="#PWR0171"  Part="1"
-F 0 "#PWR0171" H 4550 2600 50  0001 C CNN
+AR Path="/6174477C/638DF11B/63916678" Ref="#PWR0173"  Part="1"
+F 0 "#PWR0173" H 4550 2600 50  0001 C CNN
 F 1 "GND" H 4555 2677 50  0000 C CNN
 F 2 "" H 4550 2850 50  0001 C CNN
@@
 AR Path="/6174477C/63801AEE/63916679" Ref="R?"  Part="1"
 AR Path="/6174477C/638385B6/63916679" Ref="R?"  Part="1"
-AR Path="/6174477C/638DF11B/63916679" Ref="R94"  Part="1"
-F 0 "R94" V 8004 3950 50  0000 C CNN
+AR Path="/6174477C/638DF11B/63916679" Ref="R98"  Part="1"
+F 0 "R98" V 8004 3950 50  0000 C CNN
 F 1 "1M" V 8095 3950 50  0000 C CNN
 F 2 "Resistor_SMD:R_0402_1005Metric" H 8200 3950 50  0001 C CNN
@@
 AR Path="/6174477C/63801AEE/6391667A" Ref="J?"  Part="1"
 AR Path="/6174477C/638385B6/6391667A" Ref="J?"  Part="1"
-AR Path="/6174477C/638DF11B/6391667A" Ref="J16"  Part="1"
-F 0 "J16" H 3770 5146 50  0000 R CNN
+AR Path="/6174477C/638DF11B/6391667A" Ref="J17"  Part="1"
+F 0 "J17" H 3770 5146 50  0000 R CNN
 F 1 "AVR-ISP-6" H 3770 5055 50  0000 R CNN
 F 2 "Connector_PinHeader_2.54mm:PinHeader_2x03_P2.54mm_Vertical" V 3850 5100 50  0001 C CNN
@@
 AR Path="/6174477C/63801AEE/6391667B" Ref="#PWR?"  Part="1"
 AR Path="/6174477C/638385B6/6391667B" Ref="#PWR?"  Part="1"
-AR Path="/6174477C/638DF11B/6391667B" Ref="#PWR0170"  Part="1"
-F 0 "#PWR0170" H 4200 5300 50  0001 C CNN
+AR Path="/6174477C/638DF11B/6391667B" Ref="#PWR0172"  Part="1"
+F 0 "#PWR0172" H 4200 5300 50  0001 C CNN
 F 1 "GND" H 4205 5377 50  0000 C CNN
 F 2 "" H 4200 5550 50  0001 C CNN
@@
 AR Path="/6174477C/63801AEE/6391667C" Ref="D?"  Part="1"
 AR Path="/6174477C/638385B6/6391667C" Ref="D?"  Part="1"
-AR Path="/6174477C/638DF11B/6391667C" Ref="D17"  Part="1"
-F 0 "D17" V 8439 2682 50  0000 R CNN
+AR Path="/6174477C/638DF11B/6391667C" Ref="D16"  Part="1"
+F 0 "D16" V 8439 2682 50  0000 R CNN
 F 1 "NODE8_STATUSLED" V 8348 2682 50  0000 R CNN
 F 2 "LED_SMD:LED_0402_1005Metric" H 8400 2800 50  0001 C CNN
@@
 AR Path="/6174477C/63801AEE/6391667D" Ref="R?"  Part="1"
 AR Path="/6174477C/638385B6/6391667D" Ref="R?"  Part="1"
-AR Path="/6174477C/638DF11B/6391667D" Ref="R95"  Part="1"
-F 0 "R95" V 8204 3150 50  0000 C CNN
+AR Path="/6174477C/638DF11B/6391667D" Ref="R99"  Part="1"
+F 0 "R99" V 8204 3150 50  0000 C CNN
 F 1 "1K" V 8295 3150 50  0000 C CNN
 F 2 "Resistor_SMD:R_0402_1005Metric" H 8400 3150 50  0001 C CNN
@@
 AR Path="/6174477C/63801AEE/6386EF45" Ref="#PWR?"  Part="1"
 AR Path="/6174477C/638385B6/6386EF45" Ref="#PWR?"  Part="1"
-AR Path="/6174477C/638DF11B/6386EF45" Ref="#PWR0176"  Part="1"
-F 0 "#PWR0176" H 8400 3100 50  0001 C CNN
+AR Path="/6174477C/638DF11B/6386EF45" Ref="#PWR0178"  Part="1"
+F 0 "#PWR0178" H 8400 3100 50  0001 C CNN
 F 1 "GND" H 8405 3177 50  0000 C CNN
 F 2 "" H 8400 3350 50  0001 C CNN
@@
 AR Path="/6174477C/63801AEE/6391666B" Ref="#PWR?"  Part="1"
 AR Path="/6174477C/638385B6/6391666B" Ref="#PWR?"  Part="1"
-AR Path="/6174477C/638DF11B/6391666B" Ref="#PWR0172"  Part="1"
-F 0 "#PWR0172" H 6100 5800 50  0001 C CNN
+AR Path="/6174477C/638DF11B/6391666B" Ref="#PWR0174"  Part="1"
+F 0 "#PWR0174" H 6100 5800 50  0001 C CNN
 F 1 "GND" H 6105 5877 50  0000 C CNN
 F 2 "" H 6100 6050 50  0001 C CNN

Commit message: Fix git
Connections:
- net +5V_A: no longer C60.1, C61.1, D16.2 (A), R97.2, U22.18 (AVCC), U22.20 (AREF), U22.4 (VCC)
- net at SW9.1 (D): now also C60.1, C61.1, D16.2 (A), R97.2, U22.18 (AVCC), U22.20 (AREF), U22.4 (VCC)

Commit message: Change node ISP connector footprint
Parts:
- J17: footprint Connector_PinHeader_2.54mm:PinHeader_2x03_P2.54mm_Vertical -> Connector_PinHeader_1.27mm:PinHeader_2x03_P1.27mm_Vertical_SMD
Changed lines of the file:
@@
 F 0 "J17" H 3770 5146 50  0000 R CNN
 F 1 "AVR-ISP-6" H 3770 5055 50  0000 R CNN
-F 2 "Connector_PinHeader_2.54mm:PinHeader_2x03_P2.54mm_Vertical" V 3850 5100 50  0001 C CNN
+F 2 "Connector_PinHeader_1.27mm:PinHeader_2x03_P1.27mm_Vertical_SMD" V 3850 5100 50  0001 C CNN
 F 3 " ~" H 2825 4500 50  0001 C CNN
 	1    4100 5050
