File: ykts-payload/ykts-mcu-node8.sch (KiCad schematic (older format))
At the start: 12 parts, among them J17 AVR-ISP-6, SW9 ADG802BRT, U22 ATmega328PB-MU, Y11 8 MHz

Commit message: Revision B0
Added second supervisor, mega2560 -> mega128a
Parts:
- renumbered C60 to C71, C61 to C72, C62 to C73, C63 to C74, D16 to D18, J17 to J21, R97 to R75, R98 to R76, R99 to R77, U22 to U20, Y11 to Y13
Changed lines of the file:
@@
 Sheet 11 18
 Title "YktSat Payload Module"
-Date "2021-10-03"
-Rev "A3"
+Date "2021-10-22"
+Rev "B0"
 Comp "Sakha Aerospace Systems, LLC"
 Comment1 ""
@@
 AR Path="/6174477C/65729588/63916677" Ref="U?"  Part="1"
 AR Path="/6174477C/6572958C/63916677" Ref="U?"  Part="1"
-AR Path="/6174477C/6577909A/63916677" Ref="U22"  Part="1"
-F 0 "U22" H 6100 2711 50  0000 C CNN
+AR Path="/6174477C/6577909A/63916677" Ref="U20"  Part="1"
+F 0 "U20" H 6100 2711 50  0000 C CNN
 F 1 "ATmega328PB-MU" H 6100 2620 50  0000 C CNN
 F 2 "Package_DFN_QFN:QFN-32-1EP_5x5mm_P0.5mm_EP3.1x3.1mm" H 6100 4300 50  0001 C CIN
@@
 AR Path="/6174477C/65729588/65833DB9" Ref="C?"  Part="1"
 AR Path="/6174477C/6572958C/65833DB9" Ref="C?"  Part="1"
-AR Path="/6174477C/6577909A/65833DB9" Ref="C60"  Part="1"
-F 0 "C60" H 4442 2646 50  0000 L CNN
+AR Path="/6174477C/6577909A/65833DB9" Ref="C71"  Part="1"
+F 0 "C71" H 4442 2646 50  0000 L CNN
 F 1 "1uF" H 4442 2555 50  0000 L CNN
 F 2 "Capacitor_SMD:C_0603_1608Metric" H 4350 2600 50  0001 C CNN
@@
 AR Path="/6174477C/65729588/65833ED9" Ref="C?"  Part="1"
 AR Path="/6174477C/6572958C/65833ED9" Ref="C?"  Part="1"
-AR Path="/6174477C/6577909A/65833ED9" Ref="C61"  Part="1"
-F 0 "C61" H 4792 2646 50  0000 L CNN
+AR Path="/6174477C/6577909A/65833ED9" Ref="C72"  Part="1"
+F 0 "C72" H 4792 2646 50  0000 L CNN
 F 1 "100nF" H 4792 2555 50  0000 L CNN
 F 2 "Capacitor_SMD:C_0402_1005Metric" H 4700 2600 50  0001 C CNN
@@
 AR Path="/6174477C/65729588/65833DE1" Ref="#PWR?"  Part="1"
 AR Path="/6174477C/6572958C/65833DE1" Ref="#PWR?"  Part="1"
-AR Path="/6174477C/6577909A/65833DE1" Ref="#PWR0171"  Part="1"
-F 0 "#PWR0171" H 3500 2600 50  0001 C CNN
+AR Path="/6174477C/6577909A/65833DE1" Ref="#PWR0185"  Part="1"
+F 0 "#PWR0185" H 3500 2600 50  0001 C CNN
 F 1 "GND" H 3505 2677 50  0000 C CNN
 F 2 "" H 3500 2850 50  0001 C CNN
@@
 AR Path="/6174477C/65729588/65833DEE" Ref="C?"  Part="1"
 AR Path="/6174477C/6572958C/65833DEE" Ref="C?"  Part="1"
-AR Path="/6174477C/6577909A/65833DEE" Ref="C63"  Part="1"
-F 0 "C63" H 8100 4600 50  0000 L CNN
+AR Path="/6174477C/6577909A/65833DEE" Ref="C74"  Part="1"
+F 0 "C74" H 8100 4600 50  0000 L CNN
 F 1 "22pF" H 8100 4500 50  0000 L CNN
 F 2 "Capacitor_SMD:C_0402_1005Metric" H 8400 4550 50  0001 C CNN
@@
 AR Path="/6174477C/65729588/65833E96" Ref="C?"  Part="1"
 AR Path="/6174477C/6572958C/65833E96" Ref="C?"  Part="1"
-AR Path="/6174477C/6577909A/65833E96" Ref="C62"  Part="1"
-F 0 "C62" H 8100 4600 50  0000 L CNN
+AR Path="/6174477C/6577909A/65833E96" Ref="C73"  Part="1"
+F 0 "C73" H 8100 4600 50  0000 L CNN
 F 1 "22pF" H 8100 4500 50  0000 L CNN
 F 2 "Capacitor_SMD:C_0402_1005Metric" H 8000 4550 50  0001 C CNN
@@
 AR Path="/6174477C/65729588/65833EAC" Ref="#PWR?"  Part="1"
 AR Path="/6174477C/6572958C/65833EAC" Ref="#PWR?"  Part="1"
-AR Path="/6174477C/6577909A/65833EAC" Ref="#PWR0179"  Part="1"
-F 0 "#PWR0179" H 8400 4450 50  0001 C CNN
+AR Path="/6174477C/6577909A/65833EAC" Ref="#PWR0193"  Part="1"
+F 0 "#PWR0193" H 8400 4450 50  0001 C CNN
 F 1 "GND" H 8405 4527 50  0000 C CNN
 F 2 "" H 8400 4700 50  0001 C CNN
@@
 AR Path="/6174477C/65729588/65833EBC" Ref="#PWR?"  Part="1"
 AR Path="/6174477C/6572958C/65833EBC" Ref="#PWR?"  Part="1"
-AR Path="/6174477C/6577909A/65833EBC" Ref="#PWR0175"  Part="1"
-F 0 "#PWR0175" H 8000 4450 50  0001 C CNN
+AR Path="/6174477C/6577909A/65833EBC" Ref="#PWR0189"  Part="1"
+F 0 "#PWR0189" H 8000 4450 50  0001 C CNN
 F 1 "GND" H 8005 4527 50  0000 C CNN
 F 2 "" H 8000 4700 50  0001 C CNN
@@
 AR Path="/6174477C/65729588/65833ECE" Ref="Y?"  Part="1"
 AR Path="/6174477C/6572958C/65833ECE" Ref="Y?"  Part="1"
-AR Path="/6174477C/6577909A/65833ECE" Ref="Y11"  Part="1"
-F 0 "Y11" H 8450 4350 50  0000 L CNN
+AR Path="/6174477C/6577909A/65833ECE" Ref="Y13"  Part="1"
+F 0 "Y13" H 8450 4350 50  0000 L CNN
 F 1 "8 MHz" H 8450 4250 50  0000 L CNN
 F 2 "Crystal:Crystal_SMD_2520-4Pin_2.5x2.0mm" H 8200 4300 50  0001 C CNN
@@
 AR Path="/6174477C/65729588/65833E08" Ref="#PWR?"  Part="1"
 AR Path="/6174477C/6572958C/65833E08" Ref="#PWR?"  Part="1"
-AR Path="/6174477C/6577909A/65833E08" Ref="#PWR0176"  Part="1"
-F 0 "#PWR0176" H 8200 3950 50  0001 C CNN
+AR Path="/6174477C/6577909A/65833E08" Ref="#PWR0190"  Part="1"
+F 0 "#PWR0190" H 8200 3950 50  0001 C CNN
 F 1 "GND" H 8205 4027 50  0000 C CNN
 F 2 "" H 8200 4200 50  0001 C CNN
@@
 AR Path="/6174477C/65729588/65833E18" Ref="#PWR?"  Part="1"
 AR Path="/6174477C/6572958C/65833E18" Ref="#PWR?"  Part="1"
-AR Path="/6174477C/6577909A/65833E18" Ref="#PWR0177"  Part="1"
-F 0 "#PWR0177" H 8200 4150 50  0001 C CNN
+AR Path="/6174477C/6577909A/65833E18" Ref="#PWR0191"  Part="1"
+F 0 "#PWR0191" H 8200 4150 50  0001 C CNN
 F 1 "GND" H 8205 4227 50  0000 C CNN
 F 2 "" H 8200 4400 50  0001 C CNN
@@
 AR Path="/6174477C/65729588/65833DDE" Ref="R?"  Part="1"
 AR Path="/6174477C/6572958C/65833DDE" Ref="R?"  Part="1"
-AR Path="/6174477C/6577909A/65833DDE" Ref="R97"  Part="1"
-F 0 "R97" V 6754 4400 50  0000 C CNN
+AR Path="/6174477C/6577909A/65833DDE" Ref="R75"  Part="1"
+F 0 "R75" V 6754 4400 50  0000 C CNN
 F 1 "20K" V 6845 4400 50  0000 C CNN
 F 2 "Resistor_SMD:R_0402_1005Metric" H 6950 4400 50  0001 C CNN
@@
 AR Path="/6174477C/65729588/65833E24" Ref="#PWR?"  Part="1"
 AR Path="/6174477C/6572958C/65833E24" Ref="#PWR?"  Part="1"
-AR Path="/6174477C/6577909A/65833E24" Ref="#PWR0170"  Part="1"
-F 0 "#PWR0170" H 3500 1650 50  0001 C CNN
+AR Path="/6174477C/6577909A/65833E24" Ref="#PWR0184"  Part="1"
+F 0 "#PWR0184" H 3500 1650 50  0001 C CNN
 F 1 "+5V_A" H 3515 1973 50  0000 C CNN
 F 2 "" H 3500 1800 50  0001 C CNN
@@
 AR Path="/6174477C/65729588/65833E2B" Ref="#PWR?"  Part="1"
 AR Path="/6174477C/6572958C/65833E2B" Ref="#PWR?"  Part="1"
-AR Path="/6174477C/6577909A/65833E2B" Ref="#PWR0173"  Part="1"
-F 0 "#PWR0173" H 4700 2600 50  0001 C CNN
+AR Path="/6174477C/6577909A/65833E2B" Ref="#PWR0187"  Part="1"
+F 0 "#PWR0187" H 4700 2600 50  0001 C CNN
 F 1 "GND" H 4705 2677 50  0000 C CNN
 F 2 "" H 4700 2850 50  0001 C CNN
@@
 AR Path="/6174477C/65729588/65833E3E" Ref="R?"  Part="1"
 AR Path="/6174477C/6572958C/65833E3E" Ref="R?"  Part="1"
-AR Path="/6174477C/6577909A/65833E3E" Ref="R98"  Part="1"
-F 0 "R98" V 8004 3950 50  0000 C CNN
+AR Path="/6174477C/6577909A/65833E3E" Ref="R76"  Part="1"
+F 0 "R76" V 8004 3950 50  0000 C CNN
 F 1 "1M" V 8095 3950 50  0000 C CNN
 F 2 "Resistor_SMD:R_0402_1005Metric" H 8200 3950 50  0001 C CNN
@@
 AR Path="/6174477C/65729588/65833E56" Ref="J?"  Part="1"
 AR Path="/6174477C/6572958C/65833E56" Ref="J?"  Part="1"
-AR Path="/6174477C/6577909A/65833E56" Ref="J17"  Part="1"
-F 0 "J17" H 3770 5146 50  0000 R CNN
+AR Path="/6174477C/6577909A/65833E56" Ref="J21"  Part="1"
+F 0 "J21" H 3770 5146 50  0000 R CNN
 F 1 "AVR-ISP-6" H 3770 5055 50  0000 R CNN
 F 2 "Connector_PinHeader_1.27mm:PinHeader_2x03_P1.27mm_Vertical_SMD" V 3850 5100 50  0001 C CNN
@@
 AR Path="/6174477C/65729588/65833E5C" Ref="#PWR?"  Part="1"
 AR Path="/6174477C/6572958C/65833E5C" Ref="#PWR?"  Part="1"
-AR Path="/6174477C/6577909A/65833E5C" Ref="#PWR0172"  Part="1"
-F 0 "#PWR0172" H 4200 5300 50  0001 C CNN
+AR Path="/6174477C/6577909A/65833E5C" Ref="#PWR0186"  Part="1"
+F 0 "#PWR0186" H 4200 5300 50  0001 C CNN
 F 1 "GND" H 4205 5377 50  0000 C CNN
 F 2 "" H 4200 5550 50  0001 C CNN
@@
 AR Path="/6174477C/65729588/65833E6D" Ref="D?"  Part="1"
 AR Path="/6174477C/6572958C/65833E6D" Ref="D?"  Part="1"
-AR Path="/6174477C/6577909A/65833E6D" Ref="D16"  Part="1"
-F 0 "D16" V 8439 2682 50  0000 R CNN
+AR Path="/6174477C/6577909A/65833E6D" Ref="D18"  Part="1"
+F 0 "D18" V 8439 2682 50  0000 R CNN
 F 1 "NODE8_STATUSLED" V 8348 2682 50  0000 R CNN
 F 2 "LED_SMD:LED_0402_1005Metric" H 8400 2800 50  0001 C CNN
@@
 AR Path="/6174477C/65729588/65833E7C" Ref="R?"  Part="1"
 AR Path="/6174477C/6572958C/65833E7C" Ref="R?"  Part="1"
-AR Path="/6174477C/6577909A/65833E7C" Ref="R99"  Part="1"
-F 0 "R99" V 8204 3150 50  0000 C CNN
+AR Path="/6174477C/6577909A/65833E7C" Ref="R77"  Part="1"
+F 0 "R77" V 8204 3150 50  0000 C CNN
 F 1 "1K" V 8295 3150 50  0000 C CNN
 F 2 "Resistor_SMD:R_0402_1005Metric" H 8400 3150 50  0001 C CNN
@@
 AR Path="/6174477C/65729588/65833EF4" Ref="#PWR?"  Part="1"
 AR Path="/6174477C/6572958C/65833EF4" Ref="#PWR?"  Part="1"
-AR Path="/6174477C/6577909A/65833EF4" Ref="#PWR0178"  Part="1"
-F 0 "#PWR0178" H 8400 3100 50  0001 C CNN
+AR Path="/6174477C/6577909A/65833EF4" Ref="#PWR0192"  Part="1"
+F 0 "#PWR0192" H 8400 3100 50  0001 C CNN
 F 1 "GND" H 8405 3177 50  0000 C CNN
 F 2 "" H 8400 3350 50  0001 C CNN
@@
 AR Path="/6174477C/65729588/65833DC9" Ref="#PWR?"  Part="1"
 AR Path="/6174477C/6572958C/65833DC9" Ref="#PWR?"  Part="1"
-AR Path="/6174477C/6577909A/65833DC9" Ref="#PWR0174"  Part="1"
-F 0 "#PWR0174" H 6100 5800 50  0001 C CNN
+AR Path="/6174477C/6577909A/65833DC9" Ref="#PWR0188"  Part="1"
+F 0 "#PWR0188" H 6100 5800 50  0001 C CNN
 F 1 "GND" H 6105 5877 50  0000 C CNN
 F 2 "" H 6100 6050 50  0001 C CNN

Commit message: Revision B2
Hierarchal sheets for nodes
Partial PCB layout
Parts:
- renumbered C71 to C73, C72 to C74, C73 to C75, C74 to C76, U20 to U22
Changed lines of the file:
@@
 Sheet 11 18
 Title "YktSat Payload Module"
-Date "2021-10-22"
-Rev "B0"
+Date "2021-10-26"
+Rev "B1"
 Comp "Sakha Aerospace Systems, LLC"
 Comment1 ""
@@
 AR Path="/6174477C/65729588/63916677" Ref="U?"  Part="1"
 AR Path="/6174477C/6572958C/63916677" Ref="U?"  Part="1"
-AR Path="/6174477C/6577909A/63916677" Ref="U20"  Part="1"
-F 0 "U20" H 6100 2711 50  0000 C CNN
+AR Path="/6174477C/6577909A/63916677" Ref="U22"  Part="1"
+F 0 "U22" H 6100 2711 50  0000 C CNN
 F 1 "ATmega328PB-MU" H 6100 2620 50  0000 C CNN
 F 2 "Package_DFN_QFN:QFN-32-1EP_5x5mm_P0.5mm_EP3.1x3.1mm" H 6100 4300 50  0001 C CIN
@@
 AR Path="/6174477C/65729588/65833DB9" Ref="C?"  Part="1"
 AR Path="/6174477C/6572958C/65833DB9" Ref="C?"  Part="1"
-AR Path="/6174477C/6577909A/65833DB9" Ref="C71"  Part="1"
-F 0 "C71" H 4442 2646 50  0000 L CNN
+AR Path="/6174477C/6577909A/65833DB9" Ref="C73"  Part="1"
+F 0 "C73" H 4442 2646 50  0000 L CNN
 F 1 "1uF" H 4442 2555 50  0000 L CNN
 F 2 "Capacitor_SMD:C_0603_1608Metric" H 4350 2600 50  0001 C CNN
@@
 AR Path="/6174477C/65729588/65833ED9" Ref="C?"  Part="1"
 AR Path="/6174477C/6572958C/65833ED9" Ref="C?"  Part="1"
-AR Path="/6174477C/6577909A/65833ED9" Ref="C72"  Part="1"
-F 0 "C72" H 4792 2646 50  0000 L CNN
+AR Path="/6174477C/6577909A/65833ED9" Ref="C74"  Part="1"
+F 0 "C74" H 4792 2646 50  0000 L CNN
 F 1 "100nF" H 4792 2555 50  0000 L CNN
 F 2 "Capacitor_SMD:C_0402_1005Metric" H 4700 2600 50  0001 C CNN
@@
 AR Path="/6174477C/65729588/65833DE1" Ref="#PWR?"  Part="1"
 AR Path="/6174477C/6572958C/65833DE1" Ref="#PWR?"  Part="1"
-AR Path="/6174477C/6577909A/65833DE1" Ref="#PWR0185"  Part="1"
-F 0 "#PWR0185" H 3500 2600 50  0001 C CNN
+AR Path="/6174477C/6577909A/65833DE1" Ref="#PWR0189"  Part="1"
+F 0 "#PWR0189" H 3500 2600 50  0001 C CNN
 F 1 "GND" H 3505 2677 50  0000 C CNN
 F 2 "" H 3500 2850 50  0001 C CNN
@@
 AR Path="/6174477C/65729588/65833DEE" Ref="C?"  Part="1"
 AR Path="/6174477C/6572958C/65833DEE" Ref="C?"  Part="1"
-AR Path="/6174477C/6577909A/65833DEE" Ref="C74"  Part="1"
-F 0 "C74" H 8100 4600 50  0000 L CNN
+AR Path="/6174477C/6577909A/65833DEE" Ref="C76"  Part="1"
+F 0 "C76" H 8100 4600 50  0000 L CNN
 F 1 "22pF" H 8100 4500 50  0000 L CNN
 F 2 "Capacitor_SMD:C_0402_1005Metric" H 8400 4550 50  0001 C CNN
@@
 AR Path="/6174477C/65729588/65833E96" Ref="C?"  Part="1"
 AR Path="/6174477C/6572958C/65833E96" Ref="C?"  Part="1"
-AR Path="/6174477C/6577909A/65833E96" Ref="C73"  Part="1"
-F 0 "C73" H 8100 4600 50  0000 L CNN
+AR Path="/6174477C/6577909A/65833E96" Ref="C75"  Part="1"
+F 0 "C75" H 8100 4600 50  0000 L CNN
 F 1 "22pF" H 8100 4500 50  0000 L CNN
 F 2 "Capacitor_SMD:C_0402_1005Metric" H 8000 4550 50  0001 C CNN
@@
 AR Path="/6174477C/65729588/65833EAC" Ref="#PWR?"  Part="1"
 AR Path="/6174477C/6572958C/65833EAC" Ref="#PWR?"  Part="1"
-AR Path="/6174477C/6577909A/65833EAC" Ref="#PWR0193"  Part="1"
-F 0 "#PWR0193" H 8400 4450 50  0001 C CNN
+AR Path="/6174477C/6577909A/65833EAC" Ref="#PWR0197"  Part="1"
+F 0 "#PWR0197" H 8400 4450 50  0001 C CNN
 F 1 "GND" H 8405 4527 50  0000 C CNN
 F 2 "" H 8400 4700 50  0001 C CNN
@@
 AR Path="/6174477C/65729588/65833EBC" Ref="#PWR?"  Part="1"
 AR Path="/6174477C/6572958C/65833EBC" Ref="#PWR?"  Part="1"
-AR Path="/6174477C/6577909A/65833EBC" Ref="#PWR0189"  Part="1"
-F 0 "#PWR0189" H 8000 4450 50  0001 C CNN
+AR Path="/6174477C/6577909A/65833EBC" Ref="#PWR0193"  Part="1"
+F 0 "#PWR0193" H 8000 4450 50  0001 C CNN
 F 1 "GND" H 8005 4527 50  0000 C CNN
 F 2 "" H 8000 4700 50  0001 C CNN
@@
 AR Path="/6174477C/65729588/65833E08" Ref="#PWR?"  Part="1"
 AR Path="/6174477C/6572958C/65833E08" Ref="#PWR?"  Part="1"
-AR Path="/6174477C/6577909A/65833E08" Ref="#PWR0190"  Part="1"
-F 0 "#PWR0190" H 8200 3950 50  0001 C CNN
+AR Path="/6174477C/6577909A/65833E08" Ref="#PWR0194"  Part="1"
+F 0 "#PWR0194" H 8200 3950 50  0001 C CNN
 F 1 "GND" H 8205 4027 50  0000 C CNN
 F 2 "" H 8200 4200 50  0001 C CNN
@@
 AR Path="/6174477C/65729588/65833E18" Ref="#PWR?"  Part="1"
 AR Path="/6174477C/6572958C/65833E18" Ref="#PWR?"  Part="1"
-AR Path="/6174477C/6577909A/65833E18" Ref="#PWR0191"  Part="1"
-F 0 "#PWR0191" H 8200 4150 50  0001 C CNN
+AR Path="/6174477C/6577909A/65833E18" Ref="#PWR0195"  Part="1"
+F 0 "#PWR0195" H 8200 4150 50  0001 C CNN
 F 1 "GND" H 8205 4227 50  0000 C CNN
 F 2 "" H 8200 4400 50  0001 C CNN
@@
 AR Path="/6174477C/65729588/65833E24" Ref="#PWR?"  Part="1"
 AR Path="/6174477C/6572958C/65833E24" Ref="#PWR?"  Part="1"
-AR Path="/6174477C/6577909A/65833E24" Ref="#PWR0184"  Part="1"
-F 0 "#PWR0184" H 3500 1650 50  0001 C CNN
+AR Path="/6174477C/6577909A/65833E24" Ref="#PWR0188"  Part="1"
+F 0 "#PWR0188" H 3500 1650 50  0001 C CNN
 F 1 "+5V_A" H 3515 1973 50  0000 C CNN
 F 2 "" H 3500 1800 50  0001 C CNN
@@
 AR Path="/6174477C/65729588/65833E2B" Ref="#PWR?"  Part="1"
 AR Path="/6174477C/6572958C/65833E2B" Ref="#PWR?"  Part="1"
-AR Path="/6174477C/6577909A/65833E2B" Ref="#PWR0187"  Part="1"
-F 0 "#PWR0187" H 4700 2600 50  0001 C CNN
+AR Path="/6174477C/6577909A/65833E2B" Ref="#PWR0191"  Part="1"
+F 0 "#PWR0191" H 4700 2600 50  0001 C CNN
 F 1 "GND" H 4705 2677 50  0000 C CNN
 F 2 "" H 4700 2850 50  0001 C CNN
@@
 AR Path="/6174477C/65729588/65833E5C" Ref="#PWR?"  Part="1"
 AR Path="/6174477C/6572958C/65833E5C" Ref="#PWR?"  Part="1"
-AR Path="/6174477C/6577909A/65833E5C" Ref="#PWR0186"  Part="1"
-F 0 "#PWR0186" H 4200 5300 50  0001 C CNN
+AR Path="/6174477C/6577909A/65833E5C" Ref="#PWR0190"  Part="1"
+F 0 "#PWR0190" H 4200 5300 50  0001 C CNN
 F 1 "GND" H 4205 5377 50  0000 C CNN
 F 2 "" H 4200 5550 50  0001 C CNN
@@
 AR Path="/6174477C/65729588/65833EF4" Ref="#PWR?"  Part="1"
 AR Path="/6174477C/6572958C/65833EF4" Ref="#PWR?"  Part="1"
-AR Path="/6174477C/6577909A/65833EF4" Ref="#PWR0192"  Part="1"
-F 0 "#PWR0192" H 8400 3100 50  0001 C CNN
+AR Path="/6174477C/6577909A/65833EF4" Ref="#PWR0196"  Part="1"
+F 0 "#PWR0196" H 8400 3100 50  0001 C CNN
 F 1 "GND" H 8405 3177 50  0000 C CNN
 F 2 "" H 8400 3350 50  0001 C CNN
@@
 AR Path="/6174477C/65729588/65833DC9" Ref="#PWR?"  Part="1"
 AR Path="/6174477C/6572958C/65833DC9" Ref="#PWR?"  Part="1"
-AR Path="/6174477C/6577909A/65833DC9" Ref="#PWR0188"  Part="1"
-F 0 "#PWR0188" H 6100 5800 50  0001 C CNN
+AR Path="/6174477C/6577909A/65833DC9" Ref="#PWR0192"  Part="1"
+F 0 "#PWR0192" H 6100 5800 50  0001 C CNN
 F 1 "GND" H 6105 5877 50  0000 C CNN
 F 2 "" H 6100 6050 50  0001 C CNN
