File: ykts-payload/ykts-payload.sch (KiCad schematic (older format))
At the start: 43 parts, among them U2 MCP2515-xST, U3 TJA1051T-3, U6 INA3221AIRGVR, Y2 12MHz

Commit message: Sync changes
Parts:
- gave numbers to parts that had none: 19
- renumbered C5 to C6, C6 to C8, C7 to C9

Commit message: Add nodes
Connections:
- net SPI0_MISO: no longer R10.2, R6.1
- net SPI0_MOSI: no longer R4.1, R8.2
- net SPI0_SCK: no longer R5.1, R9.2
- new net SPI1_MISO: R10.2, R6.1
- new net SPI1_MOSI: R4.1, R8.2
- new net SPI1_SCK: R5.1, R9.2
Other:
- note added: "TODO:\nReset control from MCU"
Changed lines of the file:
@@
 $Descr A4 11693 8268
 encoding utf-8
-Sheet 1 3
+Sheet 1 18
 Title "YktSat Payload Module"
 Date "2021-09-30"
@@
 NoConn ~ 8850 5450
 Text GLabel 7450 5350 0    50   Input ~ 0
-SPI0_MISO
+SPI1_MISO
 $Comp
 L Device:R_Small R9
@@
 	8900 5350 9050 5350
 Text GLabel 7450 5150 0    50   Input ~ 0
-SPI0_SCK
+SPI1_SCK
 Wire Wire Line
 	8900 5150 9050 5150
 Text GLabel 7450 4950 0    50   Input ~ 0
-SPI0_MOSI
+SPI1_MOSI
 Wire Wire Line
 	8900 4950 9050 4950
@@
 F1 "ykts-payload-mcu.sch" 50
 $EndSheet
-$Sheet
-S 2000 8750 1650 550
-U 619FBF62
-F0 "Sheet619FBF61" 50
-F1 "file619FBF61.sch" 50
-$EndSheet
+Text Notes 6700 3500 0    50   ~ 0
+TODO:\nReset control from MCU
 $EndSCHEMATC

Commit message: Schematic mostly complete
Parts:
- removed C10: 100nF, Capacitor_SMD:C_0603_1608Metric, symbol Device:C_Small
- removed C5: 10uF, Capacitor_SMD:C_0603_1608Metric, symbol Device:C_Small
- removed C7: 22uF, Capacitor_SMD:C_0603_1608Metric, symbol Device:C_Small
- removed J2: Micro_SD_Card, symbol Connector:Micro_SD_Card
- removed R10, R7, R8, R9: 4.7K, Resistor_SMD:R_0402_1005Metric, symbol Device:R_Small
- removed R3, R4, R5, R6: 10K, Resistor_SMD:R_0402_1005Metric, symbol Device:R_Small
- removed U1: AMS1117-3.3, Package_TO_SOT_SMD:SOT-223-3_TabPin2, symbol Regulator_Linear:AMS1117-3.3
- added D? (x3): LED, LED_SMD:LED_0402_1005Metric, symbol Device:LED
- added Q? (x3): KIA3415, Package_TO_SOT_SMD:SOT-23, symbol Device:Q_PMOS_GSD
- added R? (x6): 1K, Resistor_SMD:R_0402_1005Metric, symbol Device:R_Small
- added R? (x3): 10K, Resistor_SMD:R_0402_1005Metric, symbol Device:R_Small
Connections:
- net +5V: now also Q?.2 (S), R?.1
- net +5V_A: now also R22.1, U6.14 (IN-2), D?.2 (A), Q?.2 (S), Q?.3 (D), R?.1; no longer R23.1, U6.11 (IN-1)
- net +5V_B: now also R23.1, U6.11 (IN-1), D?.2 (A), Q?.2 (S), Q?.3 (D), R?.1; no longer R22.1, U6.14 (IN-2)
- net GND: now also R?.2, R?.2, R?.2
- new net: Q?.1 (G), R?.1, R?.2 (x3)
- new net: D?.1 (K), R?.1 (x3)
- new net +5V_GEIGER: D?.2 (A), Q?.3 (D)
- new net MOSFET_5VA: R?.2
- new net MOSFET_5VB: R?.2
- new net MOSFET_GEIGER: R?.2
- no-connect marks 2 -> 0
Other:
- note added: "P-channel MOSFETs\nSOT-23 package\n1A MAX"
- note added: "Power Switches"
- note removed: "SD Card"

Commit message: Fixed annotations & sheet ordering
Parts:
- U3: footprint Package_SO:SOIC-8_3.9x4.9mm_P1.27mm -> Package_SON:HVSON-8-1EP_3x3mm_P0.65mm_EP1.6x2.4mm
- gave numbers to parts that had none: 15
- renumbered C16 to C1, C9 to C10, C17 to C2, C18 to C3, C1 to C4, C2 to C5, C3 to C6, C4 to C7, C6 to C8, C8 to C9, D1 to D3, D2 to D5, D3 to D6, R19 to R1, R20 to R2, R21 to R3, R22 to R4, R23 to R5, R1 to R7, R2 to R9, U6 to U1, Y2 to Y1

Commit message: Revision A2
Added debug power
Basic ESD protection on UART
MCP Reset from MCU
Parts:
- removed D3: Generic, Diode_SMD:D_SOD-323, symbol Device:D_Small
- added J2: DBG_PWR, Connector_PinHeader_2.54mm:PinHeader_1x03_P2.54mm_Vertical, symbol Connector:Conn_01x03_Male
- C8: footprint Capacitor_SMD:C_0603_1608Metric -> Capacitor_SMD:C_0402_1005Metric
- R9: value 1K -> 10K
- renumbered D4 to D3, D5 to D4, D6 to D5
Connections:
- net +5V: now also J2.2 (Pin_2)
- net GND: now also J2.1 (Pin_1), J2.3 (Pin_3)
- net MCP_RESET: now reaches C8.1, R7.1, R9.2
Other:
- note added: "Debug power"
- note removed: "TODO:\nReset control from MCU"
Changed lines of the file:
@@
 Sheet 1 18
 Title "YktSat Payload Module"
-Date "2021-10-02"
-Rev "A1"
+Date "2021-10-03"
+Rev "A2"
 Comp "Sakha Aerospace Systems, LLC"
 Comment1 ""
@@
 	6250 4150 6250 4250
 $Comp
-L power:GND #PWR018
+L power:GND #PWR019
 U 1 1 6194D8B3
 P 6250 4250
-AR Path="/6194D8B3" Ref="#PWR018"  Part="1"
+AR Path="/6194D8B3" Ref="#PWR019"  Part="1"
 AR Path="/5E6C4D56/6194D8B3" Ref="#PWR?"  Part="1"
-F 0 "#PWR018" H 6250 4000 50  0001 C CNN
+F 0 "#PWR019" H 6250 4000 50  0001 C CNN
 F 1 "GND" H 6255 4077 50  0000 C CNN
 F 2 "" H 6250 4250 50  0001 C CNN
@@
 	1    0    0    -1
 $EndComp
-Wire Wire Line
-	6550 3850 6250 3850
-Wire Wire Line
-	6550 3750 6550 3850
-Connection ~ 6400 3450
-Wire Wire Line
-	6550 3450 6550 3550
-Wire Wire Line
-	6400 3450 6550 3450
-Wire Wire Line
-	6250 3450 6250 3550
-Wire Wire Line
-	6400 3450 6250 3450
-Wire Wire Line
-	6400 3400 6400 3450
-$Comp
-L power:+5V #PWR019
+$Comp
+L power:+5V #PWR018
 U 1 1 61956076
-P 6400 3400
-AR Path="/61956076" Ref="#PWR019"  Part="1"
+P 6250 3450
+AR Path="/61956076" Ref="#PWR018"  Part="1"
 AR Path="/5E6C4D56/61956076" Ref="#PWR?"  Part="1"
-F 0 "#PWR019" H 6400 3250 50  0001 C CNN
-F 1 "+5V" H 6415 3573 50  0000 C CNN
-F 2 "" H 6400 3400 50  0001 C CNN
-F 3 "" H 6400 3400 50  0001 C CNN
-	1    6400 3400
-	1    0    0    -1
-$EndComp
-$Comp
-L Device:D_Small D3
-U 1 1 6194D8B4
-P 6550 3650
-AR Path="/6194D8B4" Ref="D3"  Part="1"
-AR Path="/5E6C4D56/6194D8B4" Ref="D?"  Part="1"
-F 0 "D3" V 6504 3718 50  0000 L CNN
-F 1 "Generic" V 6595 3718 50  0000 L CNN
-F 2 "Diode_SMD:D_SOD-323" V 6550 3650 50  0001 C CNN
-F 3 "~" V 6550 3650 50  0001 C CNN
-	1    6550 3650
-	0    1    1    0
+F 0 "#PWR018" H 6250 3300 50  0001 C CNN
+F 1 "+5V" H 6265 3623 50  0000 C CNN
+F 2 "" H 6250 3450 50  0001 C CNN
+F 3 "" H 6250 3450 50  0001 C CNN
+	1    6250 3450
+	1    0    0    -1
 $EndComp
 Wire Wire Line
@@
 F 0 "C8" H 6342 4096 50  0000 L CNN
 F 1 "100nF" H 6342 4005 50  0000 L CNN
-F 2 "Capacitor_SMD:C_0603_1608Metric" H 6250 4050 50  0001 C CNN
+F 2 "Capacitor_SMD:C_0402_1005Metric" H 6250 4050 50  0001 C CNN
 F 3 "~" H 6250 4050 50  0001 C CNN
 	1    6250 4050
@@
 AR Path="/5E6C4D56/61956077" Ref="R?"  Part="1"
 F 0 "R9" H 6309 3696 50  0000 L CNN
-F 1 "1K" H 6309 3605 50  0000 L CNN
+F 1 "10K" H 6309 3605 50  0000 L CNN
 F 2 "Resistor_SMD:R_0402_1005Metric" H 6250 3650 50  0001 C CNN
 F 3 "~" H 6250 3650 50  0001 C CNN
@@
 	4850 3400 4850 3450
 $Comp
-L power:GND #PWR023
+L power:GND #PWR025
 U 1 1 61956078
 P 6950 2700
-AR Path="/61956078" Ref="#PWR023"  Part="1"
+AR Path="/61956078" Ref="#PWR025"  Part="1"
 AR Path="/5E6C4D56/61956078" Ref="#PWR?"  Part="1"
-F 0 "#PWR023" H 6950 2450 50  0001 C CNN
+F 0 "#PWR025" H 6950 2450 50  0001 C CNN
 F 1 "GND" H 6955 2527 50  0000 C CNN
 F 2 "" H 6950 2700 50  0001 C CNN
@@
 	7200 1500 7200 1550
 $Comp
-L power:GND #PWR025
+L power:GND #PWR027
 U 1 1 6194D8BA
 P 7400 1600
-AR Path="/6194D8BA" Ref="#PWR025"  Part="1"
+AR Path="/6194D8BA" Ref="#PWR027"  Part="1"
 AR Path="/5E6C4D56/6194D8BA" Ref="#PWR?"  Part="1"
-F 0 "#PWR025" H 7400 1350 50  0001 C CNN
+F 0 "#PWR027" H 7400 1350 50  0001 C CNN
 F 1 "GND" H 7405 1427 50  0000 C CNN
 F 2 "" H 7400 1600 50  0001 C CNN
@@
 $EndComp
 $Comp
-L power:+5V #PWR022
+L power:+5V #PWR024
 U 1 1 6195607C
 P 6950 1100
-AR Path="/6195607C" Ref="#PWR022"  Part="1"
+AR Path="/6195607C" Ref="#PWR024"  Part="1"
 AR Path="/5E6C4D56/6195607C" Ref="#PWR?"  Part="1"
-F 0 "#PWR022" H 6950 950 50  0001 C CNN
+F 0 "#PWR024" H 6950 950 50  0001 C CNN
 F 1 "+5V" H 6965 1273 50  0000 C CNN
 F 2 "" H 6950 1100 50  0001 C CNN
@@
 $EndComp
 $Comp
-L power:GND #PWR026
+L power:GND #PWR028
 U 1 1 6159FC12
 P 7950 2800
-AR Path="/6159FC12" Ref="#PWR026"  Part="1"
+AR Path="/6159FC12" Ref="#PWR028"  Part="1"
 AR Path="/5E6C4D56/6159FC12" Ref="#PWR?"  Part="1"
-F 0 "#PWR026" H 7950 2550 50  0001 C CNN
+F 0 "#PWR028" H 7950 2550 50  0001 C CNN
 F 1 "GND" H 7955 2627 50  0000 C CNN
 F 2 "" H 7950 2800 50  0001 C CNN
@@
 	8150 2300 8300 2300
 $Comp
-L Device:D_TVS D5
+L Device:D_TVS D4
 U 1 1 615B1EE7
 P 9650 2550
-F 0 "D5" V 9604 2630 50  0000 L CNN
+F 0 "D4" V 9604 2630 50  0000 L CNN
 F 1 "TVS1" V 9695 2630 50  0000 L CNN
 F 2 "Diode_SMD:D_SOD-323" H 9650 2550 50  0001 C CNN
@@
 $EndComp
 $Comp
-L power:GND #PWR029
+L power:GND #PWR031
 U 1 1 615B61EC
 P 9850 2800
-AR Path="/615B61EC" Ref="#PWR029"  Part="1"
+AR Path="/615B61EC" Ref="#PWR031"  Part="1"
 AR Path="/5E6C4D56/615B61EC" Ref="#PWR?"  Part="1"
-F 0 "#PWR029" H 9850 2550 50  0001 C CNN
+F 0 "#PWR031" H 9850 2550 50  0001 C CNN
 F 1 "GND" H 9855 2627 50  0000 C CNN
 F 2 "" H 9850 2800 50  0001 C CNN
@@
 $EndComp
 $Comp
-L power:GND #PWR028
+L power:GND #PWR030
 U 1 1 615CC5F6
 P 9000 2800
-AR Path="/615CC5F6" Ref="#PWR028"  Part="1"
+AR Path="/615CC5F6" Ref="#PWR030"  Part="1"
 AR Path="/5E6C4D56/615CC5F6" Ref="#PWR?"  Part="1"
-F 0 "#PWR028" H 9000 2550 50  0001 C CNN
+F 0 "#PWR030" H 9000 2550 50  0001 C CNN
 F 1 "GND" H 9005 2627 50  0000 C CNN
 F 2 "" H 9000 2800 50  0001 C CNN
@@
 CAN protection
 $Comp
-L Device:D_TVS D6
+L Device:D_TVS D5
 U 1 1 615B2F1D
 P 10050 2550
-F 0 "D6" V 10004 2630 50  0000 L CNN
+F 0 "D5" V 10004 2630 50  0000 L CNN
 F 1 "TVS2" V 10095 2630 50  0000 L CNN
 F 2 "Diode_SMD:D_SOD-323" H 10050 2550 50  0001 C CNN
@@
 F1 "ykts-payload-mcu.sch" 50
 $EndSheet
-Text Notes 6700 3500 0    50   ~ 0
-TODO:\nReset control from MCU
 $Bitmap
 Pos 10350 6850
@@
 P 10450 6200
 AR Path="/63A0A7B5/642B62F8" Ref="#PWR?"  Part="1"
-AR Path="/642B62F8" Ref="#PWR030"  Part="1"
-F 0 "#PWR030" H 10450 6050 50  0001 C CNN
+AR Path="/642B62F8" Ref="#PWR032"  Part="1"
+F 0 "#PWR032" H 10450 6050 50  0001 C CNN
 F 1 "+5V_B" H 10465 6373 50  0000 C CNN
 F 2 "" H 10450 6200 50  0001 C CNN
@@
 P 8850 4700
 AR Path="/63A0A7B5/642B62FE" Ref="#PWR?"  Part="1"
-AR Path="/642B62FE" Ref="#PWR027"  Part="1"
-F 0 "#PWR027" H 8850 4550 50  0001 C CNN
+AR Path="/642B62FE" Ref="#PWR029"  Part="1"
+F 0 "#PWR029" H 8850 4550 50  0001 C CNN
 F 1 "+5V" H 8865 4873 50  0000 C CNN
 F 2 "" H 8850 4700 50  0001 C CNN
@@
 P 7350 6200
 AR Path="/63A0A7B5/642B6304" Ref="#PWR?"  Part="1"
-AR Path="/642B6304" Ref="#PWR024"  Part="1"
-F 0 "#PWR024" H 7350 6050 50  0001 C CNN
+AR Path="/642B6304" Ref="#PWR026"  Part="1"
+F 0 "#PWR026" H 7350 6050 50  0001 C CNN
 F 1 "+5V_A" H 7365 6373 50  0000 C CNN
 F 2 "" H 7350 6200 50  0001 C CNN
@@
 $EndComp
 $Comp
-L Device:LED D4
+L Device:LED D3
 U 1 1 64E4294A
 P 6550 6900
-F 0 "D4" V 6589 6782 50  0000 R CNN
+F 0 "D3" V 6589 6782 50  0000 R CNN
 F 1 "LED" V 6498 6782 50  0000 R CNN
 F 2 "LED_SMD:LED_0402_1005Metric" H 6550 6900 50  0001 C CNN
@@
 	6150 7450 6150 7350
 $Comp
-L power:GND #PWR021
+L power:GND #PWR023
 U 1 1 64E7FBF8
 P 6550 7450
-F 0 "#PWR021" H 6550 7200 50  0001 C CNN
+F 0 "#PWR023" H 6550 7200 50  0001 C CNN
 F 1 "GND" H 6555 7277 50  0000 C CNN
 F 2 "" H 6550 7450 50  0001 C CNN
@@
 P 6550 6650
 AR Path="/63A0A7B5/64E8C16F" Ref="#PWR?"  Part="1"
-AR Path="/64E8C16F" Ref="#PWR020"  Part="1"
-F 0 "#PWR020" H 6550 6500 50  0001 C CNN
+AR Path="/64E8C16F" Ref="#PWR022"  Part="1"
+F 0 "#PWR022" H 6550 6500 50  0001 C CNN
 F 1 "+5V_A" H 6565 6823 50  0000 C CNN
 F 2 "" H 6550 6650 50  0001 C CNN
@@
 Wire Wire Line
 	6550 6650 6550 6750
+$Comp
+L Connector:Conn_01x03_Male J2
+U 1 1 654AE64C
+P 5900 5150
+F 0 "J2" H 6008 5431 50  0000 C CNN
+F 1 "DBG_PWR" H 6008 5340 50  0000 C CNN
+F 2 "Connector_PinHeader_2.54mm:PinHeader_1x03_P2.54mm_Vertical" H 5900 5150 50  0001 C CNN
+F 3 "~" H 5900 5150 50  0001 C CNN
+	1    5900 5150
+	1    0    0    -1
+$EndComp
+$Comp
+L power:+5V #PWR?
+U 1 1 654AF5A4
+P 6400 5150
+AR Path="/63A0A7B5/654AF5A4" Ref="#PWR?"  Part="1"
+AR Path="/654AF5A4" Ref="#PWR021"  Part="1"
+F 0 "#PWR021" H 6400 5000 50  0001 C CNN
+F 1 "+5V" H 6415 5323 50  0000 C CNN
+F 2 "" H 6400 5150 50  0001 C CNN
+F 3 "" H 6400 5150 50  0001 C CNN
+	1    6400 5150
+	-1   0    0    -1
+$EndComp
+Wire Wire Line
+	6100 5150 6400 5150
+$Comp
+L power:GND #PWR020
+U 1 1 654BC7CC
+P 6250 5350
+F 0 "#PWR020" H 6250 5100 50  0001 C CNN
+F 1 "GND" H 6255 5177 50  0000 C CNN
+F 2 "" H 6250 5350 50  0001 C CNN
+F 3 "" H 6250 5350 50  0001 C CNN
+	1    6250 5350
+	1    0    0    -1
+$EndComp
+Wire Wire Line
+	6250 5250 6250 5050
+Wire Wire Line
+	6250 5050 6100 5050
+Wire Wire Line
+	6100 5250 6250 5250
+Wire Wire Line
+	6250 5250 6250 5350
+Connection ~ 6250 5250
+Text Notes 5900 4750 0    50   ~ 0
+Debug power
+Text GLabel 6500 3850 2    50   Input ~ 0
+MCP_RESET
+Wire Wire Line
+	6250 3850 6500 3850
+Wire Wire Line
+	6250 3450 6250 3550
 $EndSCHEMATC

Commit message: Revision B0
Added second supervisor, mega2560 -> mega128a
Parts:
- removed C1: 10nF, Capacitor_SMD:C_0402_1005Metric, symbol Device:C_Small
- removed C2: 100nF, Capacitor_SMD:C_0603_1608Metric, symbol Device:C_Small
- removed C3: 10uF, Capacitor_Tantalum_SMD:CP_EIA-3216-10_Kemet-I, symbol Device:CP1_Small
- removed D1: LED, LED_SMD:LED_0402_1005Metric, symbol Device:LED
- removed Q1: KIA3415, Package_TO_SOT_SMD:SOT-23, symbol Device:Q_PMOS_GSD
- removed R1, R5: 0.1, Resistor_SMD:R_2512_6332Metric, symbol Device:R_Small
- removed R13, R6: 1K, Resistor_SMD:R_0402_1005Metric, symbol Device:R_Small
- removed R14, R3: 10K, Resistor_SMD:R_0402_1005Metric, symbol Device:R_Small
- removed U1: INA3221AIRGVR, Package_DFN_QFN:QFN-16-1EP_4x4mm_P0.65mm_EP2.1x2.1mm, symbol yktsat-common:INA3221AIRGVR
- added C10: 100nF, Capacitor_SMD:C_0402_1005Metric, symbol Device:C_Small
- added C12, C6: 100nF, Capacitor_SMD:C_0603_1608Metric, symbol Device:C_Small
- added C14, C8: 22uF, Capacitor_Tantalum_SMD:CP_EIA-3216-10_Kemet-I, symbol Device:CP1_Small
- added C3, C4: 22pF, Capacitor_SMD:C_0402_1005Metric, symbol Device:C_Small
- added CH2, CH4, CL2, CL4: 50pF, Capacitor_SMD:C_0402_1005Metric, symbol Device:C_Small
- added D4: TVS1, Diode_SMD:D_SOD-323, symbol Device:D_TVS
- added D6: TVS2, Diode_SMD:D_SOD-323, symbol Device:D_TVS
- added FL2: DLW21SN921SK2, Inductor_SMD:L_CommonModeChoke_Coilcraft_0805USB, symbol Device:EMI_Filter_CommonMode
- added Q3: KIA3415, Package_TO_SOT_SMD:SOT-23, symbol Device:Q_PMOS_GSD
- added R7: 1K, Resistor_SMD:R_0402_1005Metric, symbol Device:R_Small
- added R8: 10K, Resistor_SMD:R_0402_1005Metric, symbol Device:R_Small
- added U2: MCP2515-xST, Package_SO:TSSOP-20_4.4x6.5mm_P0.65mm, symbol Interface_CAN_LIN:MCP2515-xST
- added U4: TJA1051T-3, Package_SON:HVSON-8-1EP_3x3mm_P0.65mm_EP1.6x2.4mm, symbol Interface_CAN_LIN:TJA1051T-3
- added Y2: 12MHz, Crystal:Crystal_SMD_5032-4Pin_5.0x3.2mm, symbol Device:Crystal_GND24_Small
- R2: value 10K -> 1K
- R4: value 0.1 -> 10K; footprint Resistor_SMD:R_2512_6332Metric -> Resistor_SMD:R_0402_1005Metric
- renumbered C4 to C1, C9 to C11, C10 to C13, C5 to C2, C6 to C5, C8 to C9, CH2 to CH3, CL2 to CL3, D3 to D1, D4 to D3, Q3 to Q1, R15 to R1, R9 to R11, R16 to R3, R11 to R5, R8 to R6, R7 to R9, U2 to U1
Connections:
- net +5V: now also Q1.2 (S), R12.1, R3.1, R4.1, C12.1, C14.1, C6.1, C8.1, Q3.2 (S), R8.1, U2.20 (VDD), U4.3 (VCC), U4.5 (VIO); no longer R4.2
- net +5V_A: now also Q1.3 (D); no longer R12.1, R4.1
- net +5V_B: now also Q2.3 (D); no longer Q1.2 (S), Q1.3 (D), R3.1
- net +5V_GEIGER: now also Q3.3 (D); no longer Q2.3 (D)
- net CAN1-H: now also CH4.1, D4.1 (A1), FL2.2
- net CAN1-L: now also CL4.1, D6.1 (A1), FL2.4
- net GND: now also C10.2, C12.2, C14.2, C3.2, C4.2, C6.2, C8.2, CH2.2, CH4.2, CL2.2, CL4.2, D4.2 (A2), D6.2 (A2), U2.10 (VSS), U4.2 (GND), U4.8 (S), Y2.2, Y2.4; no longer R2.2
- net MOSFET_5VB: now also R2.2; no longer R10.2
- net MOSFET_GEIGER: now also R7.2
- net at R2.1: now also Q2.1 (G), R4.2
- net S1_MCP_RESET: now reaches R10.1, R12.2
- net S1_MCP_RESET: now also C10.1
- net MCP_CS renamed S0_MCP_CS
- net MCP_INT renamed S0_MCP_INT
- net MCP_RESET renamed S0_MCP_RESET
- net MCP_RX0BF renamed S0_MCP_RX0BF
- net MCP_RX1BF renamed S0_MCP_RX1BF
- net MCP_TX0RTS renamed S0_MCP_TX0RTS
- net MCP_TX1RTS: no longer names the net of U1.5 (~TX1RTS)
- net MCP_TX2RTS: no longer names the net of U1.7 (~TX2RTS)
- net SPI0_MISO renamed S0_SPI0_MISO
- net SPI0_MOSI renamed S0_SPI0_MOSI
- net SPI0_SCK renamed S0_SPI0_SCK
- new net: R10.2, U2.19 (~RESET)
- new net: C3.1, U2.8 (OSC2), Y2.3
- new net: C4.1, U2.9 (OSC1), Y2.1
- new net: U2.1 (TXCAN), U4.4 (RXD)
- new net: U2.2 (RXCAN), U4.1 (TXD)
- new net: CL2.1, FL2.3, U4.6 (CANL)
- new net: CH2.1, FL2.1, U4.7 (CANH)
- new net: Q3.1 (G), R7.1, R8.2
- new net S1_MCP_CS: U2.18 (~CS)
- new net S1_MCP_INT: U2.13 (~INT)
- new net S1_MCP_RX0BF: U2.12 (~RX0BF)
- new net S1_MCP_RX1BF: U2.11 (~RX1BF)
- new net S1_MCP_TX0RTS: U2.4 (~TX0RTS)
- new net S1_SPI0_MISO: U2.17 (SO)
- new net S1_SPI0_MOSI: U2.16 (SI)
- new net S1_SPI0_SCK: U2.14 (SCK)
- no-connect marks 0 -> 4
Other:
- note added: "CANBUS Controllers"
- note added: "Geiger power"
- note added: "Node Group0 S0"
- note added: "Node Group1 S1"
- note added: "P-channel MOSFET\nSOT-23 package\n1A MAX"
- note added: "Power Control"
- note added: "Power LEDs"
- note removed: "CANBUS Controller"
- note removed: "Current Sensor"
- note removed: "Power Switches"
- moved on the sheet: C1, C11, C13, C2, C5, C7, C9, CH1, CH3, CL1, CL3, D1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

Commit message: Revision B2
Hierarchal sheets for nodes
Partial PCB layout
Parts:
- removed C13, C14: 22uF, Capacitor_Tantalum_SMD:CP_EIA-3216-10_Kemet-I, symbol Device:CP1_Small
- removed Q1, Q2: KIA3415, Package_TO_SOT_SMD:SOT-23, symbol Device:Q_PMOS_GSD
- removed R3, R4: 10K, Resistor_SMD:R_0402_1005Metric, symbol Device:R_Small
- added C1, C2: 100nF, Capacitor_SMD:C_0402_1005Metric, symbol Device:C_Small
- added R_CSA1, R_CSB1: 0.1, Resistor_SMD:R_2010_5025Metric, symbol Device:R_Small
- added U1, U2: MAX4372FEUK, Package_TO_SOT_SMD:SOT-23-5, symbol yktsat-common:MAX4372FEUK
- R1, R2: value 1K -> 1M
- Y1, Y2: footprint Crystal:Crystal_SMD_5032-4Pin_5.0x3.2mm -> Crystal:Crystal_SMD_3225-4Pin_3.2x2.5mm
- renumbered C8 to C10, C9 to C11, C10 to C12, C11 to C13, C12 to C14, C1 to C3, C2 to C4, C3 to C5, C4 to C6, C5 to C7, C6 to C8, C7 to C9, Q3 to Q1, R12 to R10, R5 to R3, R6 to R4, R7 to R5, R8 to R6, R9 to R7, R10 to R8, R11 to R9, U1 to U3, U2 to U4, U3 to U5, U4 to U6
Connections:
- net MOSFET_5VA is gone; now on an unnamed net: R1.2
- net MOSFET_5VB is gone; now on an unnamed net: R2.2
- net +5V: now also C1.1, C2.1, R_CSA1.2, R_CSB1.2, U1.3 (VCC), U1.4 (RS+), U2.3 (VCC), U2.4 (RS+)
- net +5V_A: now also R_CSA1.1, U1.5 (RS-)
- net +5V_B: now also R_CSB1.1, U2.5 (RS-)
- net GND: now also C1.2, C2.2, U1.1 (GND), U2.1 (GND)
- net at C4.1, U3.9 (OSC1), Y1.1: now also R1.1
- net at C6.1, U4.9 (OSC1), Y2.1: now also R2.1
- new net CS_5VA: U1.2 (OUT)
- new net CS_5VB: U2.2 (OUT)
Other:
- note added: "Current Sensors"
- note removed: "Note:\nConnect XTAL 2-4 directly to\nVSS, not to the polygon"
- note removed: "P-channel MOSFETs\nSOT-23 package\n1A MAX"
- note removed: "Power Control"
- moved on the sheet: C10, C12, C13, C14, C5, C6, C8, CH2, CH4, CL2, CL4, D4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
