File: ykts-payload/ykts-payload.sch (KiCad schematic (older format))
At the start: 59 parts, among them J1 PC/104 Connector, J2 DBG_PWR, Q1 PMV65XP, Q2 PMV65XP, Q3 PMV65XP, U1 MAX4372FEUK, U2 MAX4372FEUK, U3 MCP2515-xST, U4 MCP2515-xST, U5 TJA1051T-3, U6 TJA1051T-3, Y1 12MHz, Y2 12MHz

Commit message: Hierarchal sheet rework
Parts:
- removed C1, C11, C12, C2: 100nF, Capacitor_SMD:C_0402_1005Metric, symbol Device:C_Small
- removed C10, C9: 22uF, Capacitor_Tantalum_SMD:CP_EIA-3216-10_Kemet-I, symbol Device:CP1_Small
- removed C13, C14, C7, C8: 100nF, Capacitor_SMD:C_0603_1608Metric, symbol Device:C_Small
- removed C3, C4, C5, C6: 22pF, Capacitor_SMD:C_0402_1005Metric, symbol Device:C_Small
- removed CH1, CH2, CH3, CH4, CL1, CL2, CL3, CL4: 50pF, Capacitor_SMD:C_0402_1005Metric, symbol Device:C_Small
- removed D2: LED, LED_SMD:LED_0402_1005Metric, symbol Device:LED
- removed D3, D4: TVS1, Diode_SMD:D_SOD-323, symbol Device:D_TVS
- removed D5, D6: TVS2, Diode_SMD:D_SOD-323, symbol Device:D_TVS
- removed FL1, FL2: DLW21SN921SK2, Inductor_SMD:L_CommonModeChoke_Coilcraft_0805USB, symbol Device:EMI_Filter_CommonMode
- removed Q1, Q2: PMV65XP, symbol Device:Q_PMOS_GDS
- removed R10, R48, R50, R9: 10K, Resistor_SMD:R_0402_1005Metric, symbol Device:R_Small
- removed R47, R49: 1K, Resistor_SMD:R_0402_1005Metric, symbol Device:R_Small
- removed R_CSA1, R_CSB1: 0.1, Resistor_SMD:R_2010_5025Metric, symbol Device:R_Small
- removed U1, U2: MAX4372FEUK, Package_TO_SOT_SMD:SOT-23-5, symbol yktsat-common:MAX4372FEUK
- removed U3, U4: MCP2515-xST, Package_SO:TSSOP-20_4.4x6.5mm_P0.65mm, symbol Interface_CAN_LIN:MCP2515-xST
- removed U5, U6: TJA1051T-3, Package_SON:HVSON-8-1EP_3x3mm_P0.65mm_EP1.6x2.4mm, symbol Interface_CAN_LIN:TJA1051T-3
- removed Y1, Y2: 12MHz, Crystal:Crystal_SMD_3225-4Pin_3.2x2.5mm, symbol Device:Crystal_GND24_Small
- added H1, H2, H3, H4: CubeSat Mount / M3, MountingHole:MountingHole_3.2mm_M3_ISO7380_Pad, symbol Mechanical:MountingHole_Pad
- added H5, H6, H7, H8: GeigerBoard Mount / M2, MountingHole:MountingHole_2.2mm_M2_Pad, symbol Mechanical:MountingHole_Pad
- added J2: GeigerBoard, Connector_PinHeader_1.27mm:PinHeader_1x07_P1.27mm_Vertical, symbol Connector:Conn_01x07_Female
- added J4: Solar_Temp, Connector_PinHeader_1.27mm:PinHeader_1x03_P1.27mm_Vertical, symbol Connector:Conn_01x03_Female
- added J5: Sensor_Ext, Connector_PinHeader_1.27mm:PinHeader_1x04_P1.27mm_Vertical, symbol Connector:Conn_01x04_Female
- added N1, N10, N11, N12, N13, N14, N15, N16, N2, N3, N4, N5, N6, N7, N8, N9: YKTS-MCU-NODE, ykts-mcu-node:YktSat_MCU_node, symbol yktsat-common:YKTS-MCU-NODE
- added R5: 1K, Resistor_SMD:R_0402_1005Metric, symbol Device:R_Small
- added R6: 4.7K, Resistor_SMD:R_0402_1005Metric, symbol Device:R_Small
- D1: value LED -> LED_PWON
- Q1: renamed from Q3; footprint (none) -> Package_TO_SOT_SMD:SOT-23
- R1, R2: footprint Resistor_SMD:R_0402_1005Metric -> Resistor_SMD:R_0603_1608Metric
- R3, R4: value 1K -> 1M; footprint Resistor_SMD:R_0402_1005Metric -> Resistor_SMD:R_0603_1608Metric
- R7, R8: value 1K -> 4.7K
- renumbered J2 to J1, J1 to J3, R6 to R10, R5 to R9
Connections:
- net PCH4 is gone; now on net +5V: J3.a9 (Pin_a9), J3.b9 (Pin_b9)
- net S1_MCP_RESET is gone; now on net +5V_A: R8.1
- net +5V: now also D1.2 (A), R7.2, R6.1
- net +5V_A: now also J4.2 (Pin_2), J5.1 (Pin_1), N1.6 (VCC), N1.7 (VCC), N10.6 (VCC), N10.7 (VCC), N11.6 (VCC), N11.7 (VCC), N12.6 (VCC), N12.7 (VCC), N13.6 (VCC), N13.7 (VCC), N14.6 (VCC), N14.7 (VCC), N15.6 (VCC), N15.7 (VCC), N16.6 (VCC), N16.7 (VCC), N2.6 (VCC), N2.7 (VCC), N3.6 (VCC), N3.7 (VCC), N4.6 (VCC), N4.7 (VCC), N5.6 (VCC), N5.7 (VCC), N6.6 (VCC), N6.7 (VCC), N7.6 (VCC), N7.7 (VCC), N8.6 (VCC), N8.7 (VCC), N9.6 (VCC), N9.7 (VCC); no longer D1.2 (A)
- net +5V_GEIGER: now also J2.4 (Pin_4)
- net GND: now also R1.2, R2.2, H5.1, H6.1, H7.1, H8.1, J2.1 (Pin_1), J2.7 (Pin_7), J4.1 (Pin_1), J5.3 (Pin_3), N1.5 (GND), N1.8 (GND), N10.5 (GND), N10.8 (GND), N11.5 (GND), N11.8 (GND), N12.5 (GND), N12.8 (GND), N13.5 (GND), N13.8 (GND), N14.5 (GND), N14.8 (GND), N15.5 (GND), N15.8 (GND), N16.5 (GND), N16.8 (GND), N2.5 (GND), N2.8 (GND), N3.5 (GND), N3.8 (GND), N4.5 (GND), N4.8 (GND), N5.5 (GND), N5.8 (GND), N6.5 (GND), N6.8 (GND), N7.5 (GND), N7.8 (GND), N8.5 (GND), N8.8 (GND), N9.5 (GND), N9.8 (GND), R5.1
- net at R1.1: now also H1.1
- net at R2.1: now also H2.1
- net 1WIRE: now reaches R8.2
- net 1WIRE: now also J4.3 (Pin_3)
- net at R4.1: now also H4.1
- net at D1.1 (K): now also R5.2; no longer R3.1
- net CAN1-H renamed CANH
- net CAN1-L renamed CANL
- net S0_MCP_RESET renamed I2C_SDA
- net I2C_SDA: now also J2.2 (Pin_2), J5.4 (Pin_4)
- new net: H3.1, R3.1
- new net GEIGER_EN: J2.5 (Pin_5)
- new net I2C_SCL: J2.6 (Pin_6), J5.2 (Pin_2), R6.2
- new net N0_PWR: N1.1 (PWEN)
- new net N0_RST: N1.4 (~RST)
- new net N0_RX: N1.3 (RX)
- new net N0_TX: N1.2 (TX)
- new net N10_PWR: N11.1 (PWEN)
- new net N10_RST: N11.4 (~RST)
- new net N10_RX: N11.3 (RX)
- new net N10_TX: N11.2 (TX)
- new net N11_PWR: N12.1 (PWEN)
- new net N11_RST: N12.4 (~RST)
- new net N11_RX: N12.3 (RX)
- new net N11_TX: N12.2 (TX)
- new net N12_PWR: N13.1 (PWEN)
- new net N12_RST: N13.4 (~RST)
- new net N12_RX: N13.3 (RX)
- new net N12_TX: N13.2 (TX)
- new net N13_PWR: N14.1 (PWEN)
- new net N13_RST: N14.4 (~RST)
- new net N13_RX: N14.3 (RX)
- new net N13_TX: N14.2 (TX)
- new net N14_PWR: N15.1 (PWEN)
- new net N14_RST: N15.4 (~RST)
- new net N14_RX: N15.3 (RX)
- new net N14_TX: N15.2 (TX)
- new net N15_PWR: N16.1 (PWEN)
- new net N15_RST: N16.4 (~RST)
- new net N15_RX: N16.3 (RX)
- new net N15_TX: N16.2 (TX)
- new net N1_PWR: N2.1 (PWEN)
- new net N1_RST: N2.4 (~RST)
- new net N1_RX: N2.3 (RX)
- new net N1_TX: N2.2 (TX)
- new net N2_PWR: N3.1 (PWEN)
- new net N2_RST: N3.4 (~RST)
- new net N2_RX: N3.3 (RX)
- new net N2_TX: N3.2 (TX)
- new net N3_PWR: N4.1 (PWEN)
- new net N3_RST: N4.4 (~RST)
- new net N3_RX: N4.3 (RX)
- new net N3_TX: N4.2 (TX)
- new net N4_PWR: N5.1 (PWEN)
- new net N4_RST: N5.4 (~RST)
- new net N4_RX: N5.3 (RX)
- new net N4_TX: N5.2 (TX)
- new net N5_PWR: N6.1 (PWEN)
- new net N5_RST: N6.4 (~RST)
- new net N5_RX: N6.3 (RX)
- new net N5_TX: N6.2 (TX)
- new net N6_PWR: N7.1 (PWEN)
- new net N6_RST: N7.4 (~RST)
- new net N6_RX: N7.3 (RX)
- new net N6_TX: N7.2 (TX)
- new net N7_PWR: N8.1 (PWEN)
- new net N7_RST: N8.4 (~RST)
- new net N7_RX: N8.3 (RX)
- new net N7_TX: N8.2 (TX)
- new net N8_PWR: N9.1 (PWEN)
- new net N8_RST: N9.4 (~RST)
- new net N8_RX: N9.3 (RX)
- new net N8_TX: N9.2 (TX)
- new net N9_PWR: N10.1 (PWEN)
- new net N9_RST: N10.4 (~RST)
- new net N9_RX: N10.3 (RX)
- new net N9_TX: N10.2 (TX)
- no-connect marks 4 -> 3
Other:
- note added: "Auxilary\nDevices"
- note added: "Debug Power"
- note added: "Geiger board,\nDS18B20 sensors"
- note added: "Mounting Holes"
- note added: "Node Group 0"
- note added: "Node Group 1"
- note added: "Nodes 0-7\nTop side"
- note added: "Nodes 8-15\nBottom side"
- note removed: "CAN protection"
- note removed: "CANBUS Controllers"
- note removed: "Current Sensors"
- note removed: "Debug power"
- note removed: "Node Group0 S0"
- note removed: "Node Group1 S1"
- note removed: "P-channel MOSFETs\nSOT-23 package\n1A MAX, NO"
- note removed: "Power LEDs"
- note removed: "TVS Diodes:\nSD12_323"
- moved on the sheet: J1, J3, Q1, R10, R9
