File: ykts-payload/ykts-mcu-node.sch (KiCad schematic (older format))
At the start: 13 parts, among them J15 AVR-ISP-6, SW3 ADG802BRT, U16 ATmega328PB-MU, Y7 8 MHz

Commit message: Revision C0
Basic OC protection on 5V_A & 5V_B
SD Card -> SPI Flash
MCU Node boards
Parts:
- renumbered C49 to C39, C50 to C40, C51 to C41, C52 to C42, D12 to D10, J15 to J9, R57 to R47, R99 to R48, R58 to R49, R59 to R50, SW3 to SW1, U16 to U17, Y7 to Y5
