File: ykts-payload/ykts-payload-mcu.sch (KiCad schematic (older format))
At the start: 77 parts, among them J3 AVR-JTAG-10, J4 AVR-ISP-6, J5 Conn_01x03_Male, U10 PCA9534BS3,118, U11 PCA9534BS3,118, U12 PCA9534BS3,118, U13 PCA9534BS3,118, U4 ATmega2560-16AU, U5 74HC4051BQ,115, U7 74HC4051BQ,115, U8 74HC4051BQ,115, U9 74HC4051BQ,115, Y1 8 MHz

Commit message: Schematic mostly complete
Parts:
- added C?: 10uF, Capacitor_SMD:C_0603_1608Metric, symbol Device:C_Small
- added C?: 22uF, Capacitor_SMD:C_0603_1608Metric, symbol Device:C_Small
- added C?: 100nF, Capacitor_SMD:C_0603_1608Metric, symbol Device:C_Small
- added H? (x4): GeigerBoard Mount / M2, MountingHole:MountingHole_2.2mm_M2_Pad, symbol Mechanical:MountingHole_Pad
- added J?: Micro_SD_Card, symbol Connector:Micro_SD_Card
- added J?: Conn_01x07_Female, symbol Connector:Conn_01x07_Female
- added J?: Conn_01x03_Female, symbol Connector:Conn_01x03_Female
- added R? (x5): 4.7K, Resistor_SMD:R_0402_1005Metric, symbol Device:R_Small
- added R? (x4): 10K, Resistor_SMD:R_0402_1005Metric, symbol Device:R_Small
- added U?: AMS1117-3.3, Package_TO_SOT_SMD:SOT-89-3, symbol Regulator_Linear:AMS1117-3.3
- H1, H2, H3, H4: value MountingHole_Pad -> CubeSat Mount / M3
Connections:
- net +5V: now also C?.1, J?.2 (Pin_2), R?.1, U?.3 (VI)
- net 1WIRE: now also J?.3 (Pin_3), R?.2
- net GND: now also C?.2, C?.2, C?.2, H?.1, H?.1, H?.1, H?.1, J?.1 (Pin_1), J?.1 (Pin_1), J?.7 (Pin_7), J?.9 (SHIELD), R?.2, R?.2, R?.2, R?.2, U?.1 (GND)
- net SD_CS: now also R?.1, R?.2
- net SPI1_MISO: now also R?.1, R?.2
- net SPI1_MOSI: now also R?.1, R?.2
- net SPI1_SCK: now also R?.1, R?.2
- net UART2_RX: now also J?.6 (Pin_6)
- net UART2_TX: now also J?.2 (Pin_2)
- net GEIGER_EN: now reaches U4.74 (PA4)
- net GEIGER_EN: now also J?.5 (Pin_5)
- net MOSFET_GEIGER: now reaches U4.76 (PA2)
- net MOSFET_5VB: now reaches U4.77 (PA1)
- net MOSFET_5VA: now reaches U4.78 (PA0)
- new net: J?.2 (DAT3/CD), R?.1
- new net: J?.3 (CMD), R?.1
- new net: J?.5 (CLK), R?.1
- new net: J?.7 (DAT0), R?.1
- new net +3V3: C?.1, C?.1, J?.4 (VDD), J?.6 (VSS), U?.2 (VO)
- new net +5V_GEIGER: J?.4 (Pin_4)
- no-connect marks 7 -> 10
Other:
- note added: "Auxilary\nDevices"
- note added: "Bus Connections"
- note added: "Geiger board,\nDS18B20 sensors"
- note added: "SD Card"
- note added: "TODO:\nESD Protection"
- note added: "TODO:\nUART ESD Protection"
- note removed: "Approved:"
- note removed: "Verified:"
- moved on the sheet: C11, C12, C13, C14, C15, C20, C21, C22, C31, C32, C33, C34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

Commit message: Fixed annotations & sheet ordering
Parts:
- gave numbers to parts that had none: 20
- renumbered C12 to C11, C13 to C12, C22 to C13, C32 to C14, C20 to C15, C11 to C16, C21 to C17, C31 to C18, C33 to C19, C34 to C21, C35 to C23, C36 to C24, C14 to C26, C15 to C27, D4 to D7, D5 to D8, J3 to J2, J4 to J6, J5 to J7, L5 to L1, R15 to R17, R16 to R18, R17 to R19, R18 to R20, R24 to R21, R25 to R22, R26 to R23, R27 to R24, R28 to R25, R29 to R26, R30 to R27, R31 to R28, R32 to R29, R33 to R30, R34 to R31, R35 to R32, R36 to R34, R38 to R43, R39 to R44, R40 to R45, R41 to R46, R37 to R47, R42 to R48, R43 to R49, R44 to R50, R45 to R51, R46 to R52, R47 to R53, R48 to R54, R11 to R55, R12 to R56, R49 to R57, R50 to R58, R51 to R59, R13 to R60, R14 to R61, R52 to R62, R53 to R63, R54 to R64, R55 to R65, R56 to R66, R57 to R67, R58 to R68, U7 to U10, U8 to U11, U9 to U12, U11 to U4, U12 to U5, U4 to U6, U10 to U8, U5 to U9, Y1 to Y2

Commit message: Revision A2
Added debug power
Basic ESD protection on UART
MCP Reset from MCU
Parts:
- added R35, R36, R45, R46: 1K, Resistor_SMD:R_0402_1005Metric, symbol Device:R_Small
- renumbered D7 to D6, D8 to D7, J2 to J3, J3 to J4, J4 to J5, J5 to J6, J6 to J7, J7 to J8, R35 to R37, R36 to R38, R37 to R39, R38 to R40, R39 to R41, R40 to R42, R41 to R43, R42 to R44, R43 to R47, R44 to R48, R45 to R49, R46 to R50, R47 to R51, R48 to R52, R49 to R53, R50 to R54, R51 to R55, R52 to R56, R53 to R57, R54 to R58, R55 to R59, R56 to R60, R57 to R61, R58 to R62, R59 to R63, R60 to R64, R61 to R65, R62 to R66, R63 to R67, R64 to R68, R65 to R69, R66 to R70, R67 to R71, R68 to R72
Connections:
- net DBG_RX: now also R45.1; no longer U6.2 (PE0)
- net DBG_TX: now also R46.2; no longer U6.3 (PE1)
- net UART2_RX: now also R35.2; no longer U6.12 (PH0)
- net UART2_TX: now also R36.1; no longer U6.13 (PH1)
- net MCP_RESET: now reaches U6.71 (PA7)
- new net: R35.1, U6.12 (PH0)
- new net: R36.2, U6.13 (PH1)
- new net: R45.2, U6.2 (PE0)
- new net: R46.1, U6.3 (PE1)
Other:
- note removed: "TODO:\nESD Protection"
- note removed: "TODO:\nUART ESD Protection"

Commit message: Fix git
Changed lines of the file:
@@
 Title "YktSat Payload Module"
 Date "2021-10-03"
-Rev "A2"
+Rev "A3"
 Comp "Sakha Aerospace Systems, LLC"
 Comment1 "Approved by:"
@@
 F1 "ykts-mcu-node0.sch" 50
 $EndSheet
-$Sheet
-S 2200 12600 1500 500
-U 637CB186
-F0 "MCU Node1" 50
-F1 "ykts-mcu-node1.sch" 50
-$EndSheet
-$Sheet
-S 500  13500 1500 500
-U 63801AEE
-F0 "MCU Node2" 50
-F1 "ykts-mcu-node2.sch" 50
-$EndSheet
-$Sheet
-S 2200 13500 1500 500
-U 63801AF0
-F0 "MCU Node3" 50
-F1 "ykts-mcu-node3.sch" 50
-$EndSheet
-$Sheet
-S 500  14350 1500 500
-U 638385B6
-F0 "MCU Node4" 50
-F1 "ykts-mcu-node4.sch" 50
-$EndSheet
-$Sheet
-S 2200 14350 1500 500
-U 638385B8
-F0 "MCU Node5" 50
-F1 "ykts-mcu-node5.sch" 50
-$EndSheet
-$Sheet
-S 500  15250 1500 500
-U 638385BA
-F0 "MCU Node6" 50
-F1 "ykts-mcu-node6.sch" 50
-$EndSheet
-$Sheet
-S 2200 15250 1500 500
-U 638385BC
-F0 "MCU Node7" 50
-F1 "ykts-mcu-node7.sch" 50
-$EndSheet
 Wire Notes Line
 	350  12400 350  16000
@@
 Text Notes 5250 12300 0    100  ~ 0
 Power Channel B nodes
-$Sheet
-S 4550 12600 1500 500
-U 638DF11B
-F0 "MCU Node8" 50
-F1 "ykts-mcu-node8.sch" 50
-$EndSheet
-$Sheet
-S 6250 12600 1500 500
-U 638DF11D
-F0 "MCU Node9" 50
-F1 "ykts-mcu-node9.sch" 50
-$EndSheet
-$Sheet
-S 4550 13500 1500 500
-U 638DF11F
-F0 "MCU Node10" 50
-F1 "ykts-mcu-node10.sch" 50
-$EndSheet
-$Sheet
-S 6250 13500 1500 500
-U 638DF121
-F0 "MCU Node11" 50
-F1 "ykts-mcu-node11.sch" 50
-$EndSheet
-$Sheet
-S 4550 14350 1500 500
-U 638DF123
-F0 "MCU Node12" 50
-F1 "ykts-mcu-node12.sch" 50
-$EndSheet
-$Sheet
-S 6250 14350 1500 500
-U 638DF125
-F0 "MCU Node13" 50
-F1 "ykts-mcu-node13.sch" 50
-$EndSheet
-$Sheet
-S 4550 15250 1500 500
-U 638DF127
-F0 "MCU Node14" 50
-F1 "ykts-mcu-node14.sch" 50
-$EndSheet
-$Sheet
-S 6250 15250 1500 500
-U 638DF129
-F0 "MCU Node15" 50
-F1 "ykts-mcu-node15.sch" 50
-$EndSheet
 $Bitmap
 Pos 15150 10250
@@
 Wire Wire Line
 	8250 2700 7900 2700
+$Sheet
+S 2200 12600 1500 500
+U 6568C69E
+F0 "MCU Node1" 50
+F1 "ykts-mcu-node1.sch" 50
+$EndSheet
+$Sheet
+S 500  13350 1500 500
+U 656DAE2A
+F0 "MCU Node2" 50
+F1 "ykts-mcu-node2.sch" 50
+$EndSheet
+$Sheet
+S 2200 13350 1500 500
+U 656DAE2C
+F0 "MCU Node3" 50
+F1 "ykts-mcu-node3.sch" 50
+$EndSheet
+$Sheet
+S 500  14100 1500 500
+U 65729588
+F0 "MCU Node4" 50
+F1 "ykts-mcu-node4.sch" 50
+$EndSheet
+$Sheet
+S 2200 14100 1500 500
+U 6572958A
+F0 "MCU Node5" 50
+F1 "ykts-mcu-node5.sch" 50
+$EndSheet
+$Sheet
+S 500  14850 1500 500
+U 6572958C
+F0 "MCU Node6" 50
+F1 "ykts-mcu-node6.sch" 50
+$EndSheet
+$Sheet
+S 2200 14850 1500 500
+U 6572958E
+F0 "MCU Node7" 50
+F1 "ykts-mcu-node7.sch" 50
+$EndSheet
+$Sheet
+S 4550 12600 1500 500
+U 6577909A
+F0 "MCU Node8" 50
+F1 "ykts-mcu-node8.sch" 50
+$EndSheet
+$Sheet
+S 6250 12600 1500 500
+U 6577909C
+F0 "MCU Node9" 50
+F1 "ykts-mcu-node9.sch" 50
+$EndSheet
+$Sheet
+S 4550 13350 1500 500
+U 6577909E
+F0 "MCU Node10" 50
+F1 "ykts-mcu-node10.sch" 50
+$EndSheet
+$Sheet
+S 6250 13350 1500 500
+U 657790A0
+F0 "MCU Node11" 50
+F1 "ykts-mcu-node11.sch" 50
+$EndSheet
+$Sheet
+S 4550 14100 1500 500
+U 657790A2
+F0 "MCU Node12" 50
+F1 "ykts-mcu-node12.sch" 50
+$EndSheet
+$Sheet
+S 6250 14100 1500 500
+U 657790A4
+F0 "MCU Node13" 50
+F1 "ykts-mcu-node13.sch" 50
+$EndSheet
+$Sheet
+S 4550 14850 1500 500
+U 657790A6
+F0 "MCU Node14" 50
+F1 "ykts-mcu-node14.sch" 50
+$EndSheet
+$Sheet
+S 6250 14850 1500 500
+U 657790A8
+F0 "MCU Node15" 50
+F1 "ykts-mcu-node15.sch" 50
+$EndSheet
 $EndSCHEMATC

Commit message: Update PCB
Parts:
- added R?: 1K, Resistor_SMD:R_0402_1005Metric, symbol Device:R_Small
Connections:
- net GEIGER_EN: now also R?.2; no longer U6.74 (PA4)
- new net: R?.1, U6.74 (PA4)
Changed lines of the file:
@@
 $EndComp
-Wire Wire Line
-	1350 5400 1750 5400
 Wire Wire Line
 	1750 5200 1950 5200
@@
 	950  5400 950  5300
 Connection ~ 950  5300
-$Comp
-L Device:R_Small R?
-U 1 1 617C444E
-P 1950 5600
-AR Path="/617C444E" Ref="R?"  Part="1"
-AR Path="/6174477C/617C444E" Ref="R32"  Part="1"
-F 0 "R32" V 1754 5600 50  0000 C CNN
-F 1 "10K" V 1845 5600 50  0000 C CNN
-F 2 "Resistor_SMD:R_0402_1005Metric" H 1950 5600 50  0001 C CNN
-F 3 "~" H 1950 5600 50  0001 C CNN
-	1    1950 5600
-	-1   0    0    1
-$EndComp
-$Comp
-L Device:R_Small R?
-U 1 1 617C4454
-P 1850 5800
-AR Path="/617C4454" Ref="R?"  Part="1"
-AR Path="/6174477C/617C4454" Ref="R28"  Part="1"
-F 0 "R28" V 1654 5800 50  0000 C CNN
-F 1 "10K" V 1745 5800 50  0000 C CNN
-F 2 "Resistor_SMD:R_0402_1005Metric" H 1850 5800 50  0001 C CNN
-F 3 "~" H 1850 5800 50  0001 C CNN
-	1    1850 5800
-	-1   0    0    1
-$EndComp
-$Comp
-L Device:R_Small R?
-U 1 1 617C445A
-P 1750 6000
-AR Path="/617C445A" Ref="R?"  Part="1"
-AR Path="/6174477C/617C445A" Ref="R24"  Part="1"
-F 0 "R24" V 1554 6000 50  0000 C CNN
-F 1 "10K" V 1645 6000 50  0000 C CNN
-F 2 "Resistor_SMD:R_0402_1005Metric" H 1750 6000 50  0001 C CNN
-F 3 "~" H 1750 6000 50  0001 C CNN
-	1    1750 6000
-	-1   0    0    1
-$EndComp
 Wire Wire Line
 	2450 5700 2450 6150
-Wire Wire Line
-	1750 6100 1750 6150
 Connection ~ 2450 6150
 Wire Wire Line
 	2450 6150 2450 6200
-Wire Wire Line
-	1850 5900 1850 6150
-Wire Wire Line
-	1750 6150 1850 6150
-Connection ~ 1850 6150
-Wire Wire Line
-	1950 5700 1950 6150
-Wire Wire Line
-	1850 6150 1950 6150
-Connection ~ 1950 6150
-Wire Wire Line
-	1950 6150 2450 6150
-Wire Wire Line
-	1950 5500 1950 5200
 Connection ~ 1950 5200
 Wire Wire Line
 	1950 5200 2050 5200
-Wire Wire Line
-	1850 5700 1850 5300
-Wire Wire Line
-	1550 5300 1850 5300
-Connection ~ 1850 5300
-Wire Wire Line
-	1850 5300 2050 5300
-Wire Wire Line
-	1750 5900 1750 5400
-Connection ~ 1750 5400
-Wire Wire Line
-	1750 5400 2050 5400
 NoConn ~ 2050 4900
 Text GLabel 3150 4700 2    50   Input ~ 0
@@
 Wire Wire Line
 	4200 9250 4050 9250
-Text Label 8250 2400 0    50   ~ 0
+Text Label 8550 2400 0    50   ~ 0
 GEIGER_EN
-Wire Wire Line
-	8250 2400 7900 2400
 Text Label 4350 9450 0    50   ~ 0
 GEIGER_EN
@@
 F1 "ykts-mcu-node15.sch" 50
 $EndSheet
+Wire Wire Line
+	1950 5500 1950 5200
+Wire Wire Line
+	1750 6100 1750 6150
+Wire Wire Line
+	1750 6150 1850 6150
+Connection ~ 1850 6150
+Wire Wire Line
+	1850 5900 1850 6150
+Wire Wire Line
+	1950 6150 2450 6150
+Wire Wire Line
+	1850 6150 1950 6150
+Connection ~ 1950 6150
+Wire Wire Line
+	1950 5700 1950 6150
+Wire Wire Line
+	1850 5300 2050 5300
+Wire Wire Line
+	1550 5300 1850 5300
+Connection ~ 1850 5300
+Wire Wire Line
+	1850 5700 1850 5300
+Wire Wire Line
+	1750 5400 2050 5400
+Wire Wire Line
+	1350 5400 1750 5400
+Connection ~ 1750 5400
+Wire Wire Line
+	1750 5900 1750 5400
+$Comp
+L Device:R_Small R?
+U 1 1 617C444E
+P 1950 5600
+AR Path="/617C444E" Ref="R?"  Part="1"
+AR Path="/6174477C/617C444E" Ref="R32"  Part="1"
+F 0 "R32" V 1754 5600 50  0000 C CNN
+F 1 "10K" V 1845 5600 50  0000 C CNN
+F 2 "Resistor_SMD:R_0402_1005Metric" H 1950 5600 50  0001 C CNN
+F 3 "~" H 1950 5600 50  0001 C CNN
+	1    1950 5600
+	-1   0    0    1
+$EndComp
+$Comp
+L Device:R_Small R?
+U 1 1 617C4454
+P 1850 5800
+AR Path="/617C4454" Ref="R?"  Part="1"
+AR Path="/6174477C/617C4454" Ref="R28"  Part="1"
+F 0 "R28" V 1654 5800 50  0000 C CNN
+F 1 "10K" V 1745 5800 50  0000 C CNN
+F 2 "Resistor_SMD:R_0402_1005Metric" H 1850 5800 50  0001 C CNN
+F 3 "~" H 1850 5800 50  0001 C CNN
+	1    1850 5800
+	-1   0    0    1
+$EndComp
+$Comp
+L Device:R_Small R?
+U 1 1 617C445A
+P 1750 6000
+AR Path="/617C445A" Ref="R?"  Part="1"
+AR Path="/6174477C/617C445A" Ref="R24"  Part="1"
+F 0 "R24" V 1554 6000 50  0000 C CNN
+F 1 "10K" V 1645 6000 50  0000 C CNN
+F 2 "Resistor_SMD:R_0402_1005Metric" H 1750 6000 50  0001 C CNN
+F 3 "~" H 1750 6000 50  0001 C CNN
+	1    1750 6000
+	-1   0    0    1
+$EndComp
+$Comp
+L Device:R_Small R?
+U 1 1 65A83E0A
+P 8400 2400
+AR Path="/65A83E0A" Ref="R?"  Part="1"
+AR Path="/6174477C/65A83E0A" Ref="R?"  Part="1"
+F 0 "R?" V 8204 2400 50  0000 C CNN
+F 1 "1K" V 8295 2400 50  0000 C CNN
+F 2 "Resistor_SMD:R_0402_1005Metric" H 8400 2400 50  0001 C CNN
+F 3 "~" H 8400 2400 50  0001 C CNN
+	1    8400 2400
+	0    -1   -1   0
+$EndComp
+Wire Wire Line
+	7900 2400 8300 2400
+Wire Wire Line
+	8500 2400 8550 2400
 $EndSCHEMATC

Commit message: Revision B0
Added second supervisor, mega2560 -> mega128a
Parts:
- removed C11, C12, C26, C27: 100nF, Capacitor_SMD:C_0402_1005Metric, symbol Device:C_Small
- removed R18, R19, R20, R21, R22, R51, R52, R53, R61, R62, R63: JMP, Resistor_SMD:R_0402_1005Metric, symbol Device:R_Small
- removed R23, R25, R26, R27, R28, R32, R54, R55, R56, R57, R58, R66, R67, R68, R69, R70: 10K, Resistor_SMD:R_0402_1005Metric, symbol Device:R_Small
- removed U13, U4, U5, U8: PCA9534BS3,118, Package_DFN_QFN:HVQFN-16-1EP_3x3mm_P0.5mm_EP1.5x1.5mm, symbol yktsat-common:PCA9534BS3,118
- removed U6: ATmega2560-16AU, Package_QFP:TQFP-100_14x14mm_P0.5mm, symbol MCU_Microchip_ATmega:ATmega2560-16AU
- added C15, C17: 22pF, Capacitor_SMD:C_0402_1005Metric, symbol Device:C_Small
- added C16, C18, C19, C20, C21, C23: 100nF, Capacitor_SMD:C_0402_1005Metric, symbol Device:C_Small
- added C24, C25: 22uF, Capacitor_Tantalum_SMD:CP_EIA-3216-10_Kemet-I, symbol Device:CP1_Small
- added C35: 100nF, Capacitor_SMD:C_0603_1608Metric, symbol Device:C_Small
- added D9: LED_STATUS, LED_SMD:LED_0402_1005Metric, symbol Device:LED
- added J10: Conn_01x03_Male, Connector_PinHeader_2.54mm:PinHeader_1x03_P2.54mm_Vertical, symbol Connector:Conn_01x03_Male
- added J12: AVR-ISP-6, Connector_PinHeader_2.54mm:PinHeader_2x03_P2.54mm_Vertical, symbol Connector:AVR-ISP-6
- added J6: Micro_SD_Card, symbol Connector:Micro_SD_Card
- added J8: AVR-JTAG-10, Connector_PinHeader_2.54mm:PinHeader_2x05_P2.54mm_Vertical, symbol Connector:AVR-JTAG-10
- added L1: Ferrite, Inductor_SMD:L_1206_3216Metric, symbol Device:L_Small
- added R13: 20K, Resistor_SMD:R_0402_1005Metric, symbol Device:R_Small
- added R14, R15, R50: 1K, Resistor_SMD:R_0402_1005Metric, symbol Device:R_Small
- added R16, R37, R38: 4.7K, Resistor_SMD:R_0402_1005Metric, symbol Device:R_Small
- added R34: 10K, Resistor_SMD:R_0402_1005Metric, symbol Device:R_Small
- added U5, U7: ATmega128A-AU, Package_QFP:TQFP-64_14x14mm_P0.8mm, symbol MCU_Microchip_ATmega:ATmega128A-AU
- added Y3: 8 MHz, Crystal:Crystal_SMD_5032-4Pin_5.0x3.2mm, symbol Device:Crystal_GND24_Small
- R17: value JMP -> 4.7K
- R24: value 10K -> 1K
- R35, R36: value 1K -> 4.7K
- gave numbers to parts that had none: 1
- renumbered C20 to C22, C22 to C26, C13 to C27, C15 to C28, C25 to C29, C14 to C30, C17 to C31, C16 to C32, C18 to C33, C19 to C34, C21 to C36, C23 to C37, C24 to C38, D6 to D7, D7 to D8, J7 to J11, J4 to J3, J6 to J4, J3 to J7, J8 to J9, L1 to L2, R41 to R18, R42 to R19, R43 to R20, R44 to R21, R40 to R22, R39 to R23, R33 to R25, R38 to R26, R37 to R27, R34 to R28, R45 to R32, R46 to R33, R47 to R40, R48 to R41, R49 to R42, R50 to R43, R59 to R44, R60 to R45, R64 to R46, R65 to R47, R71 to R48, R72 to R49, U11 to U10, U12 to U11, U7 to U6, U9 to U8, U10 to U9, Y2 to Y4
Connections:
- net SPI0_MOSI is gone; now on net S0_SPI0_MOSI: J11.4 (MOSI)
- net +3V3: now also C35.1, J6.4 (VDD), J6.6 (VSS)
- net +5V: now also C16.1, C18.1, C20.1, C21.1, C24.1, C25.1, J8.4 (VREF), L1.1, R13.2, R16.1, U5.21 (VCC), U5.52 (VCC), U7.21 (VCC), U7.52 (VCC); no longer R29.2, R31.2
- net 1WIRE: now also U5.17 (PB7), U7.17 (PB7)
- net GEIGER_EN: now also R24.2
- net GND: now also R29.2, R30.2, R31.2, C15.2, C16.2, C17.2, C18.2, C19.2, C20.2, C21.2, C23.2, C24.2, C25.2, C35.2, J10.2 (Pin_2), J12.6 (GND), J6.9 (SHIELD), J8.10 (GND), J8.2 (GND), R34.2, R50.1, U5.22 (GND), U5.53 (GND), U5.63 (GND), U7.22 (GND), U7.53 (GND), U7.63 (GND), Y3.2, Y3.4; no longer R24.1, R30.1
- net MOSFET_5VA: now also U7.18 (PG3)
- net MOSFET_5VB: now also U5.18 (PG3)
- net MOSFET_GEIGER: now also U5.19 (PG4), U7.19 (PG4)
- net NODE0_PWR: now also U7.35 (PC0)
- net NODE0_RESET: now also U7.51 (PA0)
- net NODE10_PWR: now also U5.37 (PC2)
- net NODE10_RESET: now also U5.49 (PA2)
- net NODE11_PWR: now also U5.38 (PC3)
- net NODE11_RESET: now also U5.48 (PA3)
- net NODE12_PWR: now also U5.39 (PC4)
- net NODE12_RESET: now also U5.47 (PA4)
- net NODE13_PWR: now also U5.40 (PC5)
- net NODE13_RESET: now also U5.46 (PA5)
- net NODE14_PWR: now also U5.41 (PC6)
- net NODE14_RESET: now also U5.45 (PA6)
- net NODE15_PWR: now also U5.42 (PC7)
- net NODE15_RESET: now also U5.44 (PA7)
- net NODE1_PWR: now also U7.36 (PC1)
- net NODE1_RESET: now also U7.50 (PA1)
- net NODE2_PWR: now also U7.37 (PC2)
- net NODE2_RESET: now also U7.49 (PA2)
- net NODE3_PWR: now also U7.38 (PC3)
- net NODE3_RESET: now also U7.48 (PA3)
- net NODE4_PWR: now also U7.39 (PC4)
- net NODE4_RESET: now also U7.47 (PA4)
- net NODE5_PWR: now also U7.40 (PC5)
- net NODE5_RESET: now also U7.46 (PA5)
- net NODE6_PWR: now also U7.41 (PC6)
- net NODE6_RESET: now also U7.45 (PA6)
- net NODE7_PWR: now also U7.42 (PC7)
- net NODE7_RESET: now also U7.44 (PA7)
- net NODE8_PWR: now also U5.35 (PC0)
- net NODE8_RESET: now also U5.51 (PA0)
- net NODE9_PWR: now also U5.36 (PC1)
- net NODE9_RESET: now also U5.50 (PA1)
- net at C27.1, Y4.1: now also U7.24 (XTAL1)
- net at C30.1, Y4.3: now also U7.23 (XTAL2)
- net at C36.1, L2.2: now also U7.64 (AVCC)
- net I2C_SDA: now reaches R17.1
- net I2C_SDA: now also J3.2 (Pin_2), U5.26 (PD1), U7.26 (PD1)
- net at R35.1: now also J6.2 (DAT3/CD)
- net S0_SPI0_MOSI: now reaches R36.2
- net S0_SPI0_MOSI: now also R30.1, U7.12 (PB2)
- net at R32.2: now also U7.2 (PE0)
- net at R33.1: now also U7.3 (PE1)
- net at R39.1: now also U7.32 (PD7)
- net at C32.1: now also U7.62 (AREF)
- net DBG_RX renamed S0_DBG_RX
- net DBG_TX renamed S0_DBG_TX
- net I2C0_SDA renamed S0_SD_CS
- net S0_SD_CS: now also R35.2, U7.29 (PD4); no longer R31.1
- net ISP_RESET renamed S0_ISP_RESET
- net S0_ISP_RESET: now also U7.20 (~RESET)
- net JTAG_TCK renamed S0_JTAG_TCK
- net S0_JTAG_TCK: now also U7.57 (PF4)
- net JTAG_TDI renamed S0_JTAG_TDI
- net S0_JTAG_TDI: now also U7.54 (PF7)
- net JTAG_TDO renamed S0_JTAG_TDO
- net S0_JTAG_TDO: now also U7.55 (PF6)
- net JTAG_TMS renamed S0_JTAG_TMS
- net S0_JTAG_TMS: now also U7.56 (PF5)
- net LED_ST renamed S0_LED_ST
- net S0_LED_ST: now also U7.31 (PD6)
- net SD_CS renamed S1_SD_CS
- net S1_SD_CS: now also U5.29 (PD4)
- net SPI0_MISO renamed S0_SPI0_MISO
- net S0_SPI0_MISO: now also R34.1, R38.2, U7.13 (PB3)
- net SPI0_SCK renamed S0_SPI0_SCK
- net S0_SPI0_SCK: now also R31.1, R37.2, U7.11 (PB1)
- net SPI1_MISO renamed S1_SPI0_MISO
- net S1_SPI0_MISO: now also J12.1 (MISO), U5.13 (PB3)
- net SPI1_MOSI renamed S1_SPI0_MOSI
- net S1_SPI0_MOSI: now also J12.4 (MOSI), U5.12 (PB2)
- net SPI1_SCK renamed S1_SPI0_SCK
- net S1_SPI0_SCK: now also J12.3 (SCK), U5.11 (PB1)
- net UART1_MUX0_A0 renamed S0_UART1_MUX0_A0
- net S0_UART1_MUX0_A0: now also U7.14 (PB4)
- net UART1_MUX0_A1 renamed S0_UART1_MUX0_A1
- net S0_UART1_MUX0_A1: now also U7.15 (PB5)
- net UART1_MUX0_A2 renamed S0_UART1_MUX0_A2
- net S0_UART1_MUX0_A2: now also U7.16 (PB6)
- net UART1_MUX1_A0 renamed S1_UART1_MUX1_A0
- net S1_UART1_MUX1_A0: now also U5.14 (PB4)
- net UART1_MUX1_A1 renamed S1_UART1_MUX1_A1
- net S1_UART1_MUX1_A1: now also U5.15 (PB5)
- net UART1_MUX1_A2 renamed S1_UART1_MUX1_A2
- net S1_UART1_MUX1_A2: now also U5.16 (PB6)
- net UART1_RX renamed S0_UART1_RX
- net S0_UART1_RX: now also U7.27 (PD2); no longer U9.3 (A)
- net UART1_TX renamed S0_UART1_TX
- net S0_UART1_TX: now also U7.28 (PD3); no longer U11.3 (A)
- net UART2_RX renamed I2C_SCL
- net I2C_SCL: now also R16.2, U5.25 (PD0), U7.25 (PD0); no longer R35.2
- net UART2_TX: no longer names the net of R36.1
- net UART2_TX: now also J6.3 (CMD); no longer J3.2 (Pin_2)
- new net: C15.1, U5.24 (XTAL1), Y3.1
- new net: C17.1, U5.23 (XTAL2), Y3.3
- new net: C23.1, L1.2, U5.64 (AVCC)
- new net: C19.1, U5.62 (AREF)
- new net: R14.2, U5.2 (PE0)
- new net: R15.1, U5.3 (PE1)
- new net: R24.1, U5.32 (PD7)
- new net: J6.5 (CLK), R37.1
- new net: J6.7 (DAT0), R38.1
- new net: D9.1 (K), R50.2
- new net S0_MCP_CS: U7.30 (PD5)
- new net S0_MCP_INT: U7.9 (PE7)
- new net S0_MCP_RESET: U7.43 (PG2)
- new net S0_MCP_RX0BF: U7.7 (PE5)
- new net S0_MCP_RX1BF: U7.6 (PE4)
- new net S0_MCP_TX0RTS: U7.8 (PE6)
- new net S1_DBG_RX: J10.1 (Pin_1), R14.1
- new net S1_DBG_TX: J10.3 (Pin_3), R15.2
- new net S1_ISP_RESET: J12.5 (~RST), J8.6 (~SRST), R13.1, U5.20 (~RESET)
- new net S1_JTAG_TCK: J8.1 (TCK), U5.57 (PF4)
- new net S1_JTAG_TDI: J8.9 (TDI), U5.54 (PF7)
- new net S1_JTAG_TDO: J8.3 (TDO), U5.55 (PF6)
- new net S1_JTAG_TMS: J8.5 (TMS), U5.56 (PF5)
- new net S1_LED_ST: D9.2 (A), U5.31 (PD6)
- new net S1_MCP_CS: U5.30 (PD5)
- new net S1_MCP_INT: U5.9 (PE7)
- new net S1_MCP_RESET: U5.43 (PG2)
- new net S1_MCP_RX0BF: U5.7 (PE5)
- new net S1_MCP_RX1BF: U5.6 (PE4)
- new net S1_MCP_TX0RTS: U5.8 (PE6)
- new net S1_UART1_RX: U5.27 (PD2), U9.3 (A)
- new net S1_UART1_TX: U11.3 (A), U5.28 (PD3)
- no-connect marks 10 -> 11
Other:
- note added: "Global\nBus \nConnections"
- note added: "Main MCUs"
- note added: "Status LEDs"
- note added: "Supervisor 0 SD"
- note added: "Supervisor 1 SD"
- note removed: "Bus Connections"
- note removed: "Main MCU"
- note removed: "Node Power Control"
- note removed: "Node Reset Control"
- note removed: "SD Card"
- moved on the sheet: C22, C26, C27, C28, C29, C30, C31, C32, C33, C34, C36, C37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

Commit message: Revision B2
Hierarchal sheets for nodes
Partial PCB layout
Parts:
- added R12, R31: 1M, Resistor_SMD:R_0402_1005Metric, symbol Device:R_Small
- J3: footprint (none) -> Connector_PinHeader_1.27mm:PinHeader_1x07_P1.27mm_Vertical
- J4, J6: footprint (none) -> Connector_Card:microSD_HC_Wuerth_693072010801
- J5: footprint (none) -> Connector_PinHeader_1.27mm:PinHeader_1x03_P1.27mm_Vertical
- renumbered C15 to C17, C16 to C18, C17 to C19, C18 to C20, C19 to C21, C20 to C22, C21 to C23, C22 to C24, C23 to C25, C24 to C26, C25 to C27, C26 to C28, C27 to C29, C28 to C30, C29 to C31, C30 to C32, C31 to C33, C32 to C34, C33 to C35, C34 to C36, C35 to C37, C36 to C38, C37 to C39, C38 to C40, R13 to R11, R14 to R13, R15 to R14, R16 to R15, R17 to R16, R18 to R17, R19 to R18, R20 to R19, R21 to R20, R22 to R21, R23 to R22, R24 to R23, R25 to R24, R26 to R25, R27 to R26, R28 to R27, R29 to R28, R30 to R29, R31 to R30, U8 to U10, U9 to U11, U10 to U12, U11 to U13, U5 to U7, U6 to U8, U7 to U9
Connections:
- net at C29.1, U9.24 (XTAL1), Y4.1: now also R31.1
- net at C32.1, U9.23 (XTAL2), Y4.3: now also R31.2
- net CS_5VA: now reaches U9.61 (PF0)
- net at C17.1, U7.24 (XTAL1), Y3.1: now also R12.1
- net at C19.1, U7.23 (XTAL2), Y3.3: now also R12.2
- net CS_5VB: now reaches U7.61 (PF0)
- net MOSFET_5VB: no longer names the net of U7.18 (PG3)
