File: ykts-payload/ykts-payload-mcu.sch (KiCad schematic (older format))
At the start: 96 parts, among them J10 Conn_01x03_Male, J11 AVR-ISP-6, J12 AVR-ISP-6, J3 Conn_01x07_Female, J4 Micro_SD_Card, J5 Conn_01x03_Female, J6 Micro_SD_Card, J7 AVR-JTAG-10, J8 AVR-JTAG-10, J9 Conn_01x03_Male, U10 74HC4051BQ,115, U11 74HC4051BQ,115, U12 74HC4051BQ,115, U13 74HC4051BQ,115, U7 ATmega128A-AU, U8 AMS1117-3.3, U9 ATmega128A-AU, Y3 8 MHz, Y4 8 MHz

Commit message: Revision C0
Basic OC protection on 5V_A & 5V_B
SD Card -> SPI Flash
MCU Node boards
Parts:
- removed C24, C37: 100nF, Capacitor_SMD:C_0603_1608Metric, symbol Device:C_Small
- removed J11, J12: AVR-ISP-6, Connector_PinHeader_2.54mm:PinHeader_2x03_P2.54mm_Vertical, symbol Connector:AVR-ISP-6
- removed J4, J6: Micro_SD_Card, Connector_Card:microSD_HC_Wuerth_693072010801, symbol Connector:Micro_SD_Card
- removed J7, J8: AVR-JTAG-10, Connector_PinHeader_2.54mm:PinHeader_2x05_P2.54mm_Vertical, symbol Connector:AVR-JTAG-10
- removed R19, R35, R36, R37, R38: 4.7K, Resistor_SMD:R_0402_1005Metric, symbol Device:R_Small
- removed R22, R34: 10K, Resistor_SMD:R_0402_1005Metric, symbol Device:R_Small
- added C35: 22uF, Capacitor_SMD:C_0603_1608Metric, symbol Device:C_Small
- added C38: 10uF, Capacitor_SMD:C_0603_1608Metric, symbol Device:C_Small
- added J25: Sensor_Ext, symbol Connector:Conn_01x04_Female
- added J4, J6: Conn_02x03_Odd_Even, Connector_PinHeader_2.54mm:PinHeader_2x03_P2.54mm_Vertical, symbol Connector_Generic:Conn_02x03_Odd_Even
- added N1, N10, N11, N12, N13, N14, N15, N16, N2, N3, N4, N5, N6, N7, N8, N9: YKTS-MCU-NODE, symbol yktsat-common:YKTS-MCU-NODE
- added R26, R27: 10K, Resistor_SMD:R_0402_1005Metric, symbol Device:R_Small
- added R31: 4.7K, Resistor_SMD:R_0402_1005Metric, symbol Device:R_Small
- added U10, U8: AT25DF161-SF-T, Package_SO:SO-8_3.9x4.9mm_P1.27mm, symbol yktsat-common:AT25DF161-SF-T
- added U12: AMS1117-3.3, Package_TO_SOT_SMD:SOT-89-3, symbol Regulator_Linear:AMS1117-3.3
- J3: value Conn_01x07_Female -> GeigerBoard
- J5: value Conn_01x03_Female -> Solar_Temp
- R29, R30: value 10K -> 4.7K
- renumbered C17 to C15, C28 to C16, C18 to C17, C19 to C18, C20 to C19, C21 to C20, C31 to C21, C25 to C24, C26 to C25, C27 to C26, C29 to C27, C30 to C28, C32 to C29, C33 to C30, C34 to C31, C35 to C32, C36 to C33, C38 to C34, C39 to C36, C40 to C37, J9 to J7, J10 to J8, R20 to R19, R23 to R20, R24 to R22, R25 to R23, R26 to R24, R27 to R25, R31 to R32, R32 to R33, R33 to R34, R39 to R35, R40 to R36, R41 to R37, R42 to R38, R43 to R39, R44 to R40, R45 to R41, R46 to R42, R47 to R43, R48 to R44, R49 to R45, R50 to R46, U9 to U11, U10 to U13, U11 to U14, U12 to U15, U13 to U16, U8 to U7, U7 to U9
Connections:
- net +5V: no longer C16.1, C17.1, C19.1, C22.1, C23.1, C25.1, C26.1, C28.1, C30.1, C32.1, C33.1, C36.1, C37.1, D7.2 (A), J5.2 (Pin_2), L1.1, L2.1, R11.2, R22.1, R25.2, R40.1, R41.1, R42.1, R43.1, U11.21 (VCC), U11.52 (VCC), U13.16 (VCC), U14.16 (VCC), U15.16 (VCC), U16.16 (VCC), U7.3 (VI), U9.21 (VCC), U9.52 (VCC)
- net GND: now also C35.2, C38.2, J25.3 (Pin_3), J4.6 (Pin_6), J6.6 (Pin_6), N1.5 (GND), N1.8 (GND), N10.5 (GND), N10.8 (GND), N11.5 (GND), N11.8 (GND), N12.5 (GND), N12.8 (GND), N13.5 (GND), N13.8 (GND), N14.5 (GND), N14.8 (GND), N15.5 (GND), N15.8 (GND), N16.5 (GND), N16.8 (GND), N2.5 (GND), N2.8 (GND), N3.5 (GND), N3.8 (GND), N4.5 (GND), N4.8 (GND), N5.5 (GND), N5.8 (GND), N6.5 (GND), N6.8 (GND), N7.5 (GND), N7.8 (GND), N8.5 (GND), N8.8 (GND), N9.5 (GND), N9.8 (GND), R26.2, R27.2, U10.4 (GND), U12.1 (GND), U8.4 (GND); no longer R29.2, R30.2
- net I2C_SCL: now also J25.2 (Pin_2)
- net I2C_SDA: now also J25.4 (Pin_4)
- net NODE0_PWR: now also N1.1 (PWEN)
- net NODE0_RESET: now also N1.4 (~RST)
- net NODE0_RX: now also N1.2 (RX)
- net NODE0_TX: now also N1.3 (TX)
- net NODE10_PWR: now also N11.1 (PWEN)
- net NODE10_RESET: now also N11.4 (~RST)
- net NODE10_RX: now also N11.2 (RX)
- net NODE10_TX: now also N11.3 (TX)
- net NODE11_PWR: now also N12.1 (PWEN)
- net NODE11_RESET: now also N12.4 (~RST)
- net NODE11_RX: now also N12.2 (RX)
- net NODE11_TX: now also N12.3 (TX)
- net NODE12_PWR: now also N13.1 (PWEN)
- net NODE12_RESET: now also N13.4 (~RST)
- net NODE12_RX: now also N13.2 (RX)
- net NODE12_TX: now also N13.3 (TX)
- net NODE13_PWR: now also N14.1 (PWEN)
- net NODE13_RESET: now also N14.4 (~RST)
- net NODE13_RX: now also N14.2 (RX)
- net NODE13_TX: now also N14.3 (TX)
- net NODE14_PWR: now also N15.1 (PWEN)
- net NODE14_RESET: now also N15.4 (~RST)
- net NODE14_RX: now also N15.2 (RX)
- net NODE14_TX: now also N15.3 (TX)
- net NODE15_PWR: now also N16.1 (PWEN)
- net NODE15_RESET: now also N16.4 (~RST)
- net NODE15_RX: now also N16.2 (RX)
- net NODE15_TX: now also N16.3 (TX)
- net NODE1_PWR: now also N2.1 (PWEN)
- net NODE1_RESET: now also N2.4 (~RST)
- net NODE1_RX: now also N2.2 (RX)
- net NODE1_TX: now also N2.3 (TX)
- net NODE2_PWR: now also N3.1 (PWEN)
- net NODE2_RESET: now also N3.4 (~RST)
- net NODE2_RX: now also N3.2 (RX)
- net NODE2_TX: now also N3.3 (TX)
- net NODE3_PWR: now also N4.1 (PWEN)
- net NODE3_RESET: now also N4.4 (~RST)
- net NODE3_RX: now also N4.2 (RX)
- net NODE3_TX: now also N4.3 (TX)
- net NODE4_PWR: now also N5.1 (PWEN)
- net NODE4_RESET: now also N5.4 (~RST)
- net NODE4_RX: now also N5.2 (RX)
- net NODE4_TX: now also N5.3 (TX)
- net NODE5_PWR: now also N6.1 (PWEN)
- net NODE5_RESET: now also N6.4 (~RST)
- net NODE5_RX: now also N6.2 (RX)
- net NODE5_TX: now also N6.3 (TX)
- net NODE6_PWR: now also N7.1 (PWEN)
- net NODE6_RESET: now also N7.4 (~RST)
- net NODE6_RX: now also N7.2 (RX)
- net NODE6_TX: now also N7.3 (TX)
- net NODE7_PWR: now also N8.1 (PWEN)
- net NODE7_RESET: now also N8.4 (~RST)
- net NODE7_RX: now also N8.2 (RX)
- net NODE7_TX: now also N8.3 (TX)
- net NODE8_PWR: now also N9.1 (PWEN)
- net NODE8_RESET: now also N9.4 (~RST)
- net NODE8_RX: now also N9.2 (RX)
- net NODE8_TX: now also N9.3 (TX)
- net NODE9_PWR: now also N10.1 (PWEN)
- net NODE9_RESET: now also N10.4 (~RST)
- net NODE9_RX: now also N10.2 (RX)
- net NODE9_TX: now also N10.3 (TX)
- net S0_ISP_RESET: now also J6.5 (Pin_5)
- net S0_SD_CS: now also R31.2
- net S0_SPI0_MISO: now also J6.1 (Pin_1), U10.2 (SO/IO1)
- net S0_SPI0_MOSI: now also R30.2, J6.4 (Pin_4), R27.1; no longer R29.1
- net S0_SPI0_SCK: now also R29.2, J6.3 (Pin_3), R26.1; no longer R30.1
- net S1_ISP_RESET: now also J4.5 (Pin_5)
- net S1_SD_CS: now also R19.2, R21.1; no longer R17.2, R24.1
- net S1_SPI0_MISO: now also J4.1 (Pin_1), U8.2 (SO/IO1); no longer R19.2, R21.1
- net S1_SPI0_MOSI: now also J4.4 (Pin_4)
- net S1_SPI0_SCK: now also R17.2, R24.1, J4.3 (Pin_3)
- net at R17.1: now also U8.6 (SCK)
- net at R18.1: now also U8.5 (SI/IO0)
- net at R19.1: now also U8.1 (~CS)
- net +3V3: no longer names the net of C21.1, U7.2 (VO)
- net +3V3: now also U8.3 (~WP~), U8.7 (~HOLD~), U8.8 (VCC)
- new net: C35.1, U10.3 (~WP~), U10.7 (~HOLD~), U10.8 (VCC), U12.2 (VO)
- new net: R31.1, U10.1 (~CS)
- new net: R30.1, U10.5 (SI/IO0)
- new net: R29.1, U10.6 (SCK)
- new net +5V_A: C28.1, C30.1, C32.1, C33.1, C36.1, C37.1, C38.1, D7.2 (A), J25.1 (Pin_1), J5.2 (Pin_2), L2.1, N1.6 (VCC), N1.7 (VCC), N10.6 (VCC), N10.7 (VCC), N11.6 (VCC), N11.7 (VCC), N12.6 (VCC), N12.7 (VCC), N13.6 (VCC), N13.7 (VCC), N14.6 (VCC), N14.7 (VCC), N15.6 (VCC), N15.7 (VCC), N16.6 (VCC), N16.7 (VCC), N2.6 (VCC), N2.7 (VCC), N3.6 (VCC), N3.7 (VCC), N4.6 (VCC), N4.7 (VCC), N5.6 (VCC), N5.7 (VCC), N6.6 (VCC), N6.7 (VCC), N7.6 (VCC), N7.7 (VCC), N8.6 (VCC), N8.7 (VCC), N9.6 (VCC), N9.7 (VCC), R22.1, R25.2, R40.1, R42.1, U11.21 (VCC), U11.52 (VCC), U12.3 (VI), U13.16 (VCC), U15.16 (VCC)
- new net +5V_B: C16.1, C17.1, C19.1, C22.1, C23.1, C25.1, C26.1, L1.1, R11.2, R41.1, R43.1, U14.16 (VCC), U16.16 (VCC), U7.3 (VI), U9.21 (VCC), U9.52 (VCC)
- no-connect marks 11 -> 3
Other:
- note added: "MCU Nodes"
- note added: "Supervisor 0 Flash"
- note added: "Supervisor 1 Flash"
- note removed: "AVR ISP6"
- note removed: "AVR JTAG"
- note removed: "Power Channel B nodes"
- note removed: "Supervisor 0 SD"
- note removed: "Supervisor 1 SD"
- moved on the sheet: C15, C16, C17, C18, C19, C20, C21, C22, C23, C24, C25, C26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
