File: ykts-payload/ykts-payload.kicad_pcb (KiCad board)
At the start: 2 copper layers, 79 parts, among them J1 PC/104 Connector, U1 AMS1117-3.3, U10 PCA9534BS3,118, U11 PCA9534BS3,118, U12 PCA9534BS3,118, U13 PCA9534BS3,118, U14 ATmega328PB-MU, U15 ATmega328PB-MU, U16 ATmega328PB-MU, U17 ATmega328PB-MU, U18 ATmega328PB-MU, U19 ATmega328PB-MU, U2 MCP2515-xST, U20 ATmega328PB-MU, U21 ATmega328PB-MU, U22 ATmega328PB-MU, U23 ATmega328PB-MU, U24 ATmega328PB-MU, U25 ATmega328PB-MU, U26 ATmega328PB-MU, U27 ATmega328PB-MU, U28 ATmega328PB-MU, U29 ATmega328PB-MU, U3 TJA1051T-3, U4 ATmega2560-16AU, U5 74HC4051BQ,115, U6 INA3221AIRGVR, U7 74HC4051BQ,115, U8 74HC4051BQ,115, U9 74HC4051BQ,115, Y1 8 MHz, Y2 12MHz

Commit message: Update PCB
Parts:
- removed L5: Ferrite, Inductor_SMD:L_1206_3216Metric
- added C12: 100nF, Capacitor_SMD:C_0402_1005Metric, F.Cu at (72.5, 136.6)
- added C13: 22pF, Capacitor_SMD:C_0402_1005Metric, F.Cu at (65.4, 142.6)
- added C14: 22pF, Capacitor_SMD:C_0402_1005Metric, F.Cu at (78.4, 130.4)
- added C15: 100nF, Capacitor_SMD:C_0402_1005Metric, F.Cu at (65.4, 144.6)
- added C19: 100nF, Capacitor_SMD:C_0402_1005Metric, F.Cu at (61.6, 145.9)
- added C23: 22uF, Capacitor_Tantalum_SMD:CP_EIA-3216-10_Kemet-I, F.Cu at (60.0, 129.1)
- added C24: 22uF, Capacitor_Tantalum_SMD:CP_EIA-3216-10_Kemet-I, F.Cu at (69.8, 121.6)
- added C25: 22uF, Capacitor_SMD:C_0603_1608Metric, F.Cu at (79.0, 115.5)
- added C26: 100nF, Capacitor_SMD:C_0402_1005Metric, F.Cu at (113.5, 119.4)
- added C27: 100nF, Capacitor_SMD:C_0402_1005Metric, F.Cu at (68.3, 142.6)
- added C28: 1uF, Capacitor_SMD:C_0603_1608Metric, F.Cu at (240.3, 48.1)
- added C29: 100nF, Capacitor_SMD:C_0402_1005Metric, F.Cu at (243.8, 49.8)
- added C30: 22pF, Capacitor_SMD:C_0402_1005Metric, F.Cu at (237.3, 53.0)
- added C37: 100nF, Capacitor_SMD:C_0402_1005Metric, F.Cu at (215.8, 65.4)
- added C38: 22pF, Capacitor_SMD:C_0402_1005Metric, F.Cu at (212.8, 68.1)
- added C39: 22pF, Capacitor_SMD:C_0402_1005Metric, F.Cu at (219.3, 64.9)
- added C40: 1uF, Capacitor_SMD:C_0603_1608Metric, F.Cu at (274.6, 81.4)
- added C41: 100nF, Capacitor_SMD:C_0402_1005Metric, F.Cu at (278.0, 83.2)
- added C42: 22pF, Capacitor_SMD:C_0402_1005Metric, F.Cu at (271.6, 86.4)
- added C43: 22pF, Capacitor_SMD:C_0402_1005Metric, F.Cu at (274.5, 83.7)
- added C44: 1uF, Capacitor_SMD:C_0603_1608Metric, F.Cu at (191.4, 78.2)
- added C45: 100nF, Capacitor_SMD:C_0402_1005Metric, F.Cu at (191.3, 80.5)
- added C46: 22pF, Capacitor_SMD:C_0402_1005Metric, F.Cu at (194.8, 79.9)
- added C47: 22pF, Capacitor_SMD:C_0402_1005Metric, F.Cu at (188.4, 83.2)
- added C48: 1uF, Capacitor_SMD:C_0603_1608Metric, F.Cu at (240.3, 33.0)
- added C49: 100nF, Capacitor_SMD:C_0402_1005Metric, F.Cu at (240.2, 35.2)
- added C50: 22pF, Capacitor_SMD:C_0402_1005Metric, F.Cu at (237.3, 38.0)
- added C51: 22pF, Capacitor_SMD:C_0402_1005Metric, F.Cu at (243.8, 34.7)
- added C52: 1uF, Capacitor_SMD:C_0603_1608Metric, F.Cu at (250.1, 96.5)
- added C53: 100nF, Capacitor_SMD:C_0402_1005Metric, F.Cu at (250.0, 98.7)
- added C54: 22pF, Capacitor_SMD:C_0402_1005Metric, F.Cu at (247.1, 101.5)
- added C55: 22pF, Capacitor_SMD:C_0402_1005Metric, F.Cu at (253.6, 98.2)
- added C56: 1uF, Capacitor_SMD:C_0603_1608Metric, F.Cu at (215.9, 48.1)
- added C57: 100nF, Capacitor_SMD:C_0402_1005Metric, F.Cu at (219.3, 49.8)
- added C58: 22pF, Capacitor_SMD:C_0402_1005Metric, F.Cu at (212.8, 53.0)
- added C59: 22pF, Capacitor_SMD:C_0402_1005Metric, F.Cu at (215.8, 50.3)
- added C60: 1uF, Capacitor_SMD:C_0603_1608Metric, F.Cu at (225.7, 111.6)
- added C61: 100nF, Capacitor_SMD:C_0402_1005Metric, F.Cu at (225.6, 113.8)
- added C62: 22pF, Capacitor_SMD:C_0402_1005Metric, F.Cu at (222.7, 116.5)
- added C63: 22pF, Capacitor_SMD:C_0402_1005Metric, F.Cu at (229.1, 113.3)
- added C64: 1uF, Capacitor_SMD:C_0603_1608Metric, F.Cu at (191.4, 63.1)
- added C65: 100nF, Capacitor_SMD:C_0402_1005Metric, F.Cu at (191.3, 65.4)
- added C66: 22pF, Capacitor_SMD:C_0402_1005Metric, F.Cu at (188.4, 68.1)
- added C67: 22pF, Capacitor_SMD:C_0402_1005Metric, F.Cu at (194.8, 64.9)
- added C68: 1uF, Capacitor_SMD:C_0603_1608Metric, F.Cu at (250.1, 81.4)
- added C69: 100nF, Capacitor_SMD:C_0402_1005Metric, F.Cu at (253.6, 83.2)
- added C70: 22pF, Capacitor_SMD:C_0402_1005Metric, F.Cu at (247.1, 86.4)
- added C71: 22pF, Capacitor_SMD:C_0402_1005Metric, F.Cu at (250.0, 83.7)
- added C72: 1uF, Capacitor_SMD:C_0603_1608Metric, F.Cu at (215.9, 33.0)
- added C73: 100nF, Capacitor_SMD:C_0402_1005Metric, F.Cu at (219.3, 34.7)
- added C74: 22pF, Capacitor_SMD:C_0402_1005Metric, F.Cu at (212.8, 38.0)
- added C75: 22pF, Capacitor_SMD:C_0402_1005Metric, F.Cu at (215.8, 35.2)
- added C76: 1uF, Capacitor_SMD:C_0603_1608Metric, F.Cu at (225.7, 96.5)
- added C77: 100nF, Capacitor_SMD:C_0402_1005Metric, F.Cu at (229.1, 98.2)
- added C78: 22pF, Capacitor_SMD:C_0402_1005Metric, F.Cu at (222.7, 101.5)
- added C79: 22pF, Capacitor_SMD:C_0402_1005Metric, F.Cu at (225.6, 98.7)
- added C80: 1uF, Capacitor_SMD:C_0603_1608Metric, F.Cu at (191.4, 48.1)
- added C81: 100nF, Capacitor_SMD:C_0402_1005Metric, F.Cu at (194.8, 49.8)
- added C82: 22pF, Capacitor_SMD:C_0402_1005Metric, F.Cu at (188.4, 53.0)
- added C83: 22pF, Capacitor_SMD:C_0402_1005Metric, F.Cu at (191.3, 50.3)
- added C84: 1uF, Capacitor_SMD:C_0603_1608Metric, F.Cu at (225.7, 81.4)
- added C85: 100nF, Capacitor_SMD:C_0402_1005Metric, F.Cu at (225.6, 83.7)
- added C86: 22pF, Capacitor_SMD:C_0402_1005Metric, F.Cu at (222.7, 86.4)
- added C87: 22pF, Capacitor_SMD:C_0402_1005Metric, F.Cu at (229.1, 83.2)
- added C88: 1uF, Capacitor_SMD:C_0603_1608Metric, F.Cu at (191.4, 33.0)
- added C89: 100nF, Capacitor_SMD:C_0402_1005Metric, F.Cu at (188.4, 38.0)
- added C90: 22pF, Capacitor_SMD:C_0402_1005Metric, F.Cu at (191.3, 35.2)
- added C91: 22pF, Capacitor_SMD:C_0402_1005Metric, F.Cu at (194.8, 34.7)
- added D10: NODE2_STATUSLED, LED_SMD:LED_0402_1005Metric, F.Cu at (201.1, 68.5)
- added D11: NODE3_STATUSLED, LED_SMD:LED_0402_1005Metric, F.Cu at (259.8, 86.8)
- added D12: NODE4_STATUSLED, LED_SMD:LED_0402_1005Metric, F.Cu at (176.6, 83.6)
- added D13: NODE5_STATUSLED, LED_SMD:LED_0402_1005Metric, F.Cu at (225.5, 38.4)
- added D14: NODE6_STATUSLED, LED_SMD:LED_0402_1005Metric, F.Cu at (235.3, 101.9)
- added D15: NODE7_STATUSLED, LED_SMD:LED_0402_1005Metric, F.Cu at (201.1, 53.5)
- added D16: NODE8_STATUSLED, LED_SMD:LED_0402_1005Metric, F.Cu at (210.9, 117.0)
- added D17: NODE9_STATUSLED, LED_SMD:LED_0402_1005Metric, F.Cu at (176.6, 68.5)
- added D18: NODE10_STATUSLED, LED_SMD:LED_0402_1005Metric, F.Cu at (235.3, 86.8)
- added D19: NODE11_STATUSLED, LED_SMD:LED_0402_1005Metric, F.Cu at (201.1, 38.4)
- added D20: NODE12_STATUSLED, LED_SMD:LED_0402_1005Metric, F.Cu at (210.9, 101.9)
- added D21: NODE13_STATUSLED, LED_SMD:LED_0402_1005Metric, F.Cu at (176.6, 53.5)
- added D22: NODE14_STATUSLED, LED_SMD:LED_0402_1005Metric, F.Cu at (210.9, 86.8)
- added D23: NODE15_STATUSLED, LED_SMD:LED_0402_1005Metric, F.Cu at (176.6, 38.4)
- added D4: TVS1, Diode_SMD:D_SOD-323, F.Cu at (94.1, 32.3)
- added D5: TVS2, Diode_SMD:D_SOD-323, F.Cu at (94.1, 35.3)
- added D6: LED_PWON, LED_SMD:LED_0402_1005Metric, F.Cu at (68.5, 126.7)
- added D7: LED_STATUS, LED_SMD:LED_0402_1005Metric, F.Cu at (57.6, 137.0)
- added D8: NODE0_STATUSLED, LED_SMD:LED_0402_1005Metric, F.Cu at (225.5, 53.5)
- added D9: NODE1_STATUSLED, LED_SMD:LED_0402_1005Metric, F.Cu at (235.3, 117.0)
- added H1: CubeSat Mount / M3, MountingHole:MountingHole_3.2mm_M3_ISO7380_Pad, F.Cu at (57.3, 117.8)
- added H2: CubeSat Mount / M3, MountingHole:MountingHole_3.2mm_M3_ISO7380_Pad, F.Cu at (34.3, 136.2)
- added H3: CubeSat Mount / M3, MountingHole:MountingHole_3.2mm_M3_ISO7380_Pad, F.Cu at (41.6, 136.2)
- added H4: CubeSat Mount / M3, MountingHole:MountingHole_3.2mm_M3_ISO7380_Pad, F.Cu at (45.5, 127.5)
- added H5: GeigerBoard Mount / M2, MountingHole:MountingHole_2.2mm_M2_Pad, F.Cu at (54.1, 130.5)
- added H6: GeigerBoard Mount / M2, MountingHole:MountingHole_2.2mm_M2_Pad, F.Cu at (48.2, 134.2)
- added H7: GeigerBoard Mount / M2, MountingHole:MountingHole_2.2mm_M2_Pad, F.Cu at (40.3, 142.8)
- added H8: GeigerBoard Mount / M2, MountingHole:MountingHole_2.2mm_M2_Pad, F.Cu at (63.9, 117.2)
- added J10: AVR-ISP-6, Connector_PinHeader_2.54mm:PinHeader_2x03_P2.54mm_Vertical, F.Cu at (236.0, 108.6)
- added J11: AVR-ISP-6, Connector_PinHeader_2.54mm:PinHeader_2x03_P2.54mm_Vertical, F.Cu at (201.7, 60.2)
- added J12: AVR-ISP-6, Connector_PinHeader_2.54mm:PinHeader_2x03_P2.54mm_Vertical, F.Cu at (260.4, 78.5)
- added J13: AVR-ISP-6, Connector_PinHeader_2.54mm:PinHeader_2x03_P2.54mm_Vertical, F.Cu at (177.2, 75.2)
- added J14: AVR-ISP-6, Connector_PinHeader_2.54mm:PinHeader_2x03_P2.54mm_Vertical, F.Cu at (226.2, 30.0)
- added J15: AVR-ISP-6, Connector_PinHeader_2.54mm:PinHeader_2x03_P2.54mm_Vertical, F.Cu at (236.0, 93.5)
- added J16: AVR-ISP-6, Connector_PinHeader_2.54mm:PinHeader_2x03_P2.54mm_Vertical, F.Cu at (201.7, 45.1)
- added J17: AVR-ISP-6, Connector_PinHeader_2.54mm:PinHeader_2x03_P2.54mm_Vertical, F.Cu at (211.5, 108.6)
- added J18: AVR-ISP-6, Connector_PinHeader_2.54mm:PinHeader_2x03_P2.54mm_Vertical, F.Cu at (177.2, 60.2)
- added J19: AVR-ISP-6, Connector_PinHeader_2.54mm:PinHeader_2x03_P2.54mm_Vertical, F.Cu at (236.0, 78.5)
- added J2: DBG_PWR, Connector_PinHeader_2.54mm:PinHeader_1x03_P2.54mm_Vertical, F.Cu at (33.0, 30.0)
- added J20: AVR-ISP-6, Connector_PinHeader_2.54mm:PinHeader_2x03_P2.54mm_Vertical, F.Cu at (201.7, 30.0)
- added J21: AVR-ISP-6, Connector_PinHeader_2.54mm:PinHeader_2x03_P2.54mm_Vertical, F.Cu at (211.5, 93.5)
- added J22: AVR-ISP-6, Connector_PinHeader_2.54mm:PinHeader_2x03_P2.54mm_Vertical, F.Cu at (177.2, 45.1)
- added J23: AVR-ISP-6, Connector_PinHeader_2.54mm:PinHeader_2x03_P2.54mm_Vertical, F.Cu at (211.5, 78.5)
- added J24: AVR-ISP-6, Connector_PinHeader_2.54mm:PinHeader_2x03_P2.54mm_Vertical, F.Cu at (177.2, 30.0)
- added J3: AVR-JTAG-10, Connector_PinHeader_2.54mm:PinHeader_2x05_P2.54mm_Vertical, F.Cu at (25.8, 134.9)
- added J7: AVR-ISP-6, Connector_PinHeader_2.54mm:PinHeader_2x03_P2.54mm_Vertical, F.Cu at (44.2, 116.5)
- added J8: Conn_01x03_Male, Connector_PinHeader_2.54mm:PinHeader_1x03_P2.54mm_Vertical, F.Cu at (51.4, 116.5)
- added J9: AVR-ISP-6, Connector_PinHeader_2.54mm:PinHeader_2x03_P2.54mm_Vertical, F.Cu at (226.2, 45.1)
- added L1: Ferrite, Inductor_SMD:L_1206_3216Metric, F.Cu at (33.6, 146.4)
- added Q1: KIA3415, Package_TO_SOT_SMD:SOT-23, F.Cu at (89.7, 33.1)
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Connections:
- C1 pad 1: Net-(C1-Pad1) -> +5V
- C10 pad 1: +3V3 -> +5V
- C11 pad 1: Net-(C11-Pad1) -> +5V
- C16 pad 1: +5V -> Net-(C16-Pad1)
- C2 pad 1: Net-(C2-Pad1) -> +5V
- C20 pad 1: +5V -> +3V3
- C21 pad 1: +5V -> Net-(C21-Pad1)
- C22 pad 1: Net-(C22-Pad1) -> +5V
- C31 pad 1: +5V -> Net-(C31-Pad1)
- C33 pad 1: +5V -> Net-(C32-Pad1)
- C35 pad 1: +5V -> Net-(C35-Pad1)
- C36 pad 1: +5V -> Net-(C36-Pad1)
- C4 pad 1: +5V -> Net-(C4-Pad1)
- C5 pad 1: +5V -> Net-(C5-Pad1)
- C6 pad 1: Net-(C6-Pad1) -> +5V
- C7 pad 1: +3V3 -> +5V
- C8 pad 1: +5V -> MCP_RESET
- D1 pad 1: +5V -> Net-(D1-Pad1)
- D1 pad 2: Net-(C6-Pad1) -> +5V_GEIGER
- D2 pad 1: /CAN1-H -> Net-(D2-Pad1)
- D2 pad 2: GND -> +5V_B
- D3 pad 1: /CAN1-L -> Net-(D3-Pad1)
- D3 pad 2: GND -> +5V_A
- R1 pad 1: Net-(C6-Pad1) -> /PCH4
- R1 pad 2: Net-(R1-Pad2) -> +5V
- R10 pad 2: SPI0_MISO -> MOSFET_5VB
- R19 pad 1: /PCH4 -> Net-(R19-Pad1)
- R2 pad 1: +5V -> Net-(R2-Pad1)
- R2 pad 2: Net-(C6-Pad1) -> GND
- R20 pad 2: GND -> +5V
- R21 pad 2: /PV -> +5V
- R22 pad 1: +5V_B -> Net-(R22-Pad1)
- R23 pad 1: +5V_A -> GND
- R23 pad 2: +5V -> Net-(R17-Pad1)
- R3 pad 1: SD_CS -> Net-(R3-Pad1)
- R3 pad 2: GND -> /PV
- R4 pad 1: SPI0_MOSI -> +5V_A
- R4 pad 2: GND -> +5V
- R5 pad 1: SPI0_SCK -> +5V_B
- R5 pad 2: GND -> +5V
- R6 pad 1: SPI0_MISO -> Net-(D1-Pad1)
- R7 pad 1: Net-(J2-Pad2) -> MCP_RESET
- R7 pad 2: SD_CS -> Net-(R7-Pad2)
- R8 pad 1: Net-(J2-Pad3) -> Net-(D2-Pad1)
- R8 pad 2: SPI0_MOSI -> GND
- R9 pad 1: Net-(J2-Pad5) -> +5V
- R9 pad 2: SPI0_SCK -> MCP_RESET
- U1 pad 1: GND -> +5V
- U1 pad 2: +3V3 -> /PCH4
- U1 pad 3: +5V -> GND
- U10 pad 1: Net-(U10-Pad1) -> NODE12_RX
- U10 pad 10: Net-(U10-Pad10) -> /Payload MCU/UART1_MUX1_A1
- U10 pad 11: Net-(U10-Pad11) -> /Payload MCU/UART1_MUX1_A0
- U10 pad 12: Net-(U10-Pad12) -> NODE11_RX
- U10 pad 13: Net-(U10-Pad13) -> NODE8_RX
- U10 pad 14: Net-(U10-Pad14) -> NODE9_RX
- U10 pad 15: Net-(U10-Pad15) -> NODE10_RX
- U10 pad 16: Net-(U10-Pad16) -> +5V
- U10 pad 2: Net-(U10-Pad2) -> NODE14_RX
- U10 pad 3: Net-(U10-Pad3) -> /Payload MCU/UART1_RX
- U10 pad 4: Net-(U10-Pad4) -> NODE15_RX
- U10 pad 5: Net-(U10-Pad5) -> NODE13_RX
- U10 pad 7: Net-(U10-Pad7) -> +5V
- U10 pad 8: Net-(U10-Pad8) -> GND
- U10 pad 9: Net-(U10-Pad9) -> /Payload MCU/UART1_MUX1_A2
- U11 pad 1: Net-(U11-Pad1) -> NODE4_TX
- U11 pad 10: Net-(U11-Pad10) -> /Payload MCU/UART1_MUX0_A1
- U11 pad 11: Net-(U11-Pad11) -> /Payload MCU/UART1_MUX0_A0
- U11 pad 12: Net-(U11-Pad12) -> NODE3_TX
- U11 pad 13: Net-(U11-Pad13) -> NODE0_TX
- U11 pad 14: Net-(U11-Pad14) -> NODE1_TX
- U11 pad 15: Net-(U11-Pad15) -> NODE2_TX
- U11 pad 16: Net-(U11-Pad16) -> +5V
- U11 pad 2: Net-(U11-Pad2) -> NODE6_TX
- U11 pad 3: Net-(U11-Pad3) -> /Payload MCU/UART1_TX
- U11 pad 4: Net-(U11-Pad4) -> NODE7_TX
- U11 pad 5: Net-(U11-Pad5) -> NODE5_TX
- U11 pad 7: Net-(U11-Pad7) -> +5V
- U11 pad 8: Net-(U11-Pad8) -> GND
- U11 pad 9: Net-(U11-Pad9) -> /Payload MCU/UART1_MUX0_A2
- U12 pad 1: Net-(U12-Pad1) -> NODE12_TX
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Other:
- copper layers 2 -> 4

Commit message: PC/104 Outline
Parts:
- J10, J11, J12, J13, J14, J15, J16, J17, J18, J19, J20, J21, J22, J23, J24, J9: footprint Connector_PinHeader_2.54mm:PinHeader_2x03_P2.54mm_Vertical -> Connector_PinHeader_1.27mm:PinHeader_2x03_P1.27mm_Vertical_SMD
- moved J1 183.1 mm to (172.1, 143.5), turned to 180 degrees
- moved H2 162.0 mm to (179.7, 64.8)
- moved H1 125.3 mm to (179.7, 144.8)
- moved U6 108.0 mm to (140.3, 131.4)
- moved H6 94.7 mm to (124.5, 78.1)
- moved H3 85.6 mm to (94.0, 68.6)
- moved C13 79.4 mm to (139.7, 114.7)
- moved C15 79.4 mm to (139.7, 116.6)
- moved C24 79.4 mm to (144.1, 93.7)
- moved D6 79.4 mm to (142.8, 98.7)
- moved R33 79.4 mm to (137.7, 110.0)
- moved R34 79.4 mm to (133.1, 117.0)
- moved R39 79.4 mm to (145.7, 98.2)
- moved R41 79.4 mm to (156.7, 87.3)
- moved R44 79.4 mm to (156.7, 89.3)
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- renumbered R101 to R100, R102 to R101, R103 to R102, R104 to R103, R105 to R104, R106 to R105, R107 to R106, R108 to R107, R109 to R108, R110 to R109, R111 to R110, R112 to R111, R113 to R112, R114 to R113, R115 to R114, R116 to R115, R117 to R116, R118 to R117, R119 to R118, R120 to R119, R121 to R120, R47 to R121, R48 to R47, R49 to R48, R50 to R49, R51 to R50, R52 to R51, R53 to R52, R54 to R53, R55 to R54, R56 to R55, R57 to R56, R58 to R57, R59 to R58, R60 to R59, R61 to R60, R62 to R61, R63 to R62, R64 to R63, R65 to R64, R66 to R65, R67 to R66, R68 to R67, R69 to R68, R70 to R69, R71 to R70, R72 to R71, R73 to R72, R74 to R73, R75 to R74, R76 to R75, R77 to R76, R78 to R77, R79 to R78, R80 to R79, R81 to R80, R82 to R81, R83 to R82, R84 to R83, R85 to R84, R86 to R85, R87 to R86, R88 to R87, R89 to R88, R90 to R89, R91 to R90, R92 to R91, R93 to R92, R94 to R93, R95 to R94, R96 to R95, R97 to R96, R98 to R97, R99 to R98, R100 to R99
Other:
- board outline added: 95.9 x 90.2 mm

Commit message: Revision B2
Hierarchal sheets for nodes
Partial PCB layout
Parts:
- removed the J7 at (118.5, 88.6)
- removed Q2, Q3: KIA3415, Package_TO_SOT_SMD:SOT-23
- removed R115, R118: 20K, Resistor_SMD:R_0402_1005Metric
- removed R116, R119: 1M, Resistor_SMD:R_0402_1005Metric
- removed R117, R120, R121: 1K, Resistor_SMD:R_0402_1005Metric
- added C100: 100nF, Capacitor_SMD:C_0402_1005Metric, F.Cu at (380.5, 79.2)
- added C101: 22pF, Capacitor_SMD:C_0402_1005Metric, F.Cu at (374.9, 82.2)
- added C102: 22pF, Capacitor_SMD:C_0402_1005Metric, F.Cu at (377.2, 80.2)
- added C92: 100nF, Capacitor_SMD:C_0402_1005Metric, F.Cu at (380.5, 64.5)
- added C93: 22pF, Capacitor_SMD:C_0402_1005Metric, F.Cu at (374.9, 67.5)
- added C94: 22pF, Capacitor_SMD:C_0402_1005Metric, F.Cu at (377.2, 65.5)
- added C95: 1uF, Capacitor_SMD:C_0603_1608Metric, F.Cu at (367.1, 91.4)
- added C96: 100nF, Capacitor_SMD:C_0402_1005Metric, F.Cu at (356.7, 93.9)
- added C97: 22pF, Capacitor_SMD:C_0402_1005Metric, F.Cu at (351.1, 97.0)
- added C98: 22pF, Capacitor_SMD:C_0402_1005Metric, F.Cu at (353.4, 94.9)
- added C99: 1uF, Capacitor_SMD:C_0603_1608Metric, F.Cu at (390.9, 76.7)
- added CH3: 50pF, Capacitor_SMD:C_0402_1005Metric, F.Cu at (58.3, 51.8)
- added CH4: 50pF, Capacitor_SMD:C_0402_1005Metric, F.Cu at (307.5, 178.8)
- added CL3: 50pF, Capacitor_SMD:C_0402_1005Metric, F.Cu at (58.3, 47.2)
- added CL4: 50pF, Capacitor_SMD:C_0402_1005Metric, F.Cu at (307.5, 183.4)
- added D24: NODE_STATUSLED, LED_SMD:LED_0402_1005Metric, F.Cu at (355.4, 93.9)
- added D25: NODE_STATUSLED, LED_SMD:LED_0402_1005Metric, F.Cu at (379.2, 79.2)
- added FL2: DLW21SN921SK2, Inductor_SMD:L_CommonModeChoke_Coilcraft_0805USB, F.Cu at (309.0, 181.1)
- added J25: AVR-ISP-6, Connector_PinHeader_1.27mm:PinHeader_2x03_P1.27mm_Vertical_SMD, F.Cu at (361.7, 86.1)
- added J26: AVR-ISP-6, Connector_PinHeader_1.27mm:PinHeader_2x03_P1.27mm_Vertical_SMD, F.Cu at (385.6, 71.3)
- added J27: AVR-ISP-6, Connector_PinHeader_1.27mm:PinHeader_2x03_P1.27mm_Vertical_SMD, F.Cu at (361.7, 100.8)
- added J28: AVR-ISP-6, Connector_PinHeader_1.27mm:PinHeader_2x03_P1.27mm_Vertical_SMD, F.Cu at (385.6, 86.1)
- added J3: Conn_01x07_Female, Connector_PinHeader_1.27mm:PinHeader_1x07_P1.27mm_Vertical, F.Cu at (118.3, -34.0)
- added J4: Micro_SD_Card, Connector_Card:microSD_HC_Wuerth_693072010801, F.Cu at (47.1, 64.5)
- added J5: Conn_01x03_Female, Connector_PinHeader_1.27mm:PinHeader_1x03_P1.27mm_Vertical, F.Cu at (152.7, -44.9)
- added J6: Micro_SD_Card, Connector_Card:microSD_HC_Wuerth_693072010801, F.Cu at (124.8, -44.7)
- added L2: Ferrite, Inductor_SMD:L_1206_3216Metric, F.Cu at (133.9, -28.0)
- added R_CSA1: 0.1, Resistor_SMD:R_2010_5025Metric, F.Cu at (342.8, 179.8)
- added R_CSB1: 0.1, Resistor_SMD:R_2010_5025Metric, F.Cu at (342.8, 175.6)
- added Y19: 8 MHz, Crystal:Crystal_SMD_2520-4Pin_2.5x2.0mm, F.Cu at (353.4, 97.0)
- added Y20: 8 MHz, Crystal:Crystal_SMD_2520-4Pin_2.5x2.0mm, F.Cu at (377.2, 82.2)
- C1: value 10nF -> 100nF
- C13, C14: value 22pF -> 100nF; footprint Capacitor_SMD:C_0402_1005Metric -> Capacitor_SMD:C_0603_1608Metric
- C15, C49: value 100nF -> 1uF; footprint Capacitor_SMD:C_0402_1005Metric -> Capacitor_SMD:C_0603_1608Metric
- C17, C19, C29, C41, C45, C53, C57, C61, C65, C69, C73, C77, C81, C85, C89: value 100nF -> 22pF
- C2, C20: footprint Capacitor_SMD:C_0603_1608Metric -> Capacitor_SMD:C_0402_1005Metric
- C22: value 10uF -> 100nF; footprint Capacitor_SMD:C_0603_1608Metric -> Capacitor_SMD:C_0402_1005Metric
- C23: value 22uF -> 100nF; footprint Capacitor_Tantalum_SMD:CP_EIA-3216-10_Kemet-I -> Capacitor_SMD:C_0402_1005Metric
- C24, C7: value 22uF -> 100nF; footprint Capacitor_Tantalum_SMD:CP_EIA-3216-10_Kemet-I -> Capacitor_SMD:C_0603_1608Metric
- C25: value 22uF -> 100nF; footprint Capacitor_SMD:C_0603_1608Metric -> Capacitor_SMD:C_0402_1005Metric
- C26, C27: value 100nF -> 22uF; footprint Capacitor_SMD:C_0402_1005Metric -> Capacitor_Tantalum_SMD:CP_EIA-3216-10_Kemet-I
- C28: value 1uF -> 10uF
- C3: value 10uF -> 22pF; footprint Capacitor_Tantalum_SMD:CP_EIA-3216-10_Kemet-I -> Capacitor_SMD:C_0402_1005Metric
- C30, C34, C35, C38, C50: value 22pF -> 100nF
- C31: value 22pF -> 22uF; footprint Capacitor_SMD:C_0402_1005Metric -> Capacitor_SMD:C_0603_1608Metric
- C32, C52: value 1uF -> 22pF; footprint Capacitor_SMD:C_0603_1608Metric -> Capacitor_SMD:C_0402_1005Metric
- C36, C44, C48, C56, C60, C64, C68, C72, C76, C80, C84, C88: value 1uF -> 100nF; footprint Capacitor_SMD:C_0603_1608Metric -> Capacitor_SMD:C_0402_1005Metric
- C37, C8: footprint Capacitor_SMD:C_0402_1005Metric -> Capacitor_SMD:C_0603_1608Metric
- C39: value 22pF -> 22uF; footprint Capacitor_SMD:C_0402_1005Metric -> Capacitor_Tantalum_SMD:CP_EIA-3216-10_Kemet-I
- C40: value 1uF -> 22uF; footprint Capacitor_SMD:C_0603_1608Metric -> Capacitor_Tantalum_SMD:CP_EIA-3216-10_Kemet-I
- C43, C47, C55, C59, C63, C67, C71, C75, C79, C83, C87, C91: value 22pF -> 1uF; footprint Capacitor_SMD:C_0402_1005Metric -> Capacitor_SMD:C_0603_1608Metric
- C6: value 100nF -> 22pF; footprint Capacitor_SMD:C_0603_1608Metric -> Capacitor_SMD:C_0402_1005Metric
- C9: value 100nF -> 22uF; footprint Capacitor_SMD:C_0603_1608Metric -> Capacitor_Tantalum_SMD:CP_EIA-3216-10_Kemet-I
- D10: value NODE2_STATUSLED -> NODE_STATUSLED
- D11: value NODE3_STATUSLED -> NODE_STATUSLED
- D12: value NODE4_STATUSLED -> NODE_STATUSLED
- D13: value NODE5_STATUSLED -> NODE_STATUSLED
- D14: value NODE6_STATUSLED -> NODE_STATUSLED
- D15: value NODE7_STATUSLED -> NODE_STATUSLED
- D16: value NODE8_STATUSLED -> NODE_STATUSLED
- D17: value NODE9_STATUSLED -> NODE_STATUSLED
- D18: value NODE10_STATUSLED -> NODE_STATUSLED
- D19: value NODE11_STATUSLED -> NODE_STATUSLED
- D20: value NODE12_STATUSLED -> NODE_STATUSLED
- D21: value NODE13_STATUSLED -> NODE_STATUSLED
- D22: value NODE14_STATUSLED -> NODE_STATUSLED
- D23: value NODE15_STATUSLED -> NODE_STATUSLED
- D3: value LED -> TVS1; footprint LED_SMD:LED_0402_1005Metric -> Diode_SMD:D_SOD-323
- D6: value LED_PWON -> TVS2; footprint LED_SMD:LED_0402_1005Metric -> Diode_SMD:D_SOD-323
- D7: value LED_STATUS -> LED_PWON
- D8: value NODE0_STATUSLED -> LED_STATUS
- D9: value NODE1_STATUSLED -> LED_STATUS
- J10, J9: value AVR-ISP-6 -> Conn_01x03_Male; footprint Connector_PinHeader_1.27mm:PinHeader_2x03_P1.27mm_Vertical_SMD -> Connector_PinHeader_2.54mm:PinHeader_1x03_P2.54mm_Vertical
- J11, J12: footprint Connector_PinHeader_1.27mm:PinHeader_2x03_P1.27mm_Vertical_SMD -> Connector_PinHeader_2.54mm:PinHeader_2x03_P2.54mm_Vertical
- J8: value Conn_01x03_Male -> AVR-JTAG-10; footprint Connector_PinHeader_2.54mm:PinHeader_1x03_P2.54mm_Vertical -> Connector_PinHeader_2.54mm:PinHeader_2x05_P2.54mm_Vertical
- R1: value 0.1 -> 1M; footprint Resistor_SMD:R_2512_6332Metric -> Resistor_SMD:R_0402_1005Metric
- R10, R6: value 1K -> 10K
- R100, R103, R106, R109, R112: value 20K -> 0R; footprint Resistor_SMD:R_0402_1005Metric -> Resistor_SMD:R_0603_1608Metric
- R101, R104, R107, R110, R113: value 1M -> 0R; footprint Resistor_SMD:R_0402_1005Metric -> Resistor_SMD:R_0603_1608Metric
- R102, R105, R108, R111, R114, R99: value 1K -> 0R; footprint Resistor_SMD:R_0402_1005Metric -> Resistor_SMD:R_0603_1608Metric
- R11, R72, R75, R78, R81, R84, R87, R90, R93, R96: value 1K -> 20K
- R12, R2, R31, R55, R58, R67, R70: value 10K -> 1M
- R14, R23, R3, R32, R39, R56, R68: value 10K -> 1K
- R15, R35, R36: value 1K -> 4.7K
- R16, R24, R37, R38: value 10K -> 4.7K
- R17, R18, R19, R20: value JMP -> 4.7K
- R21, R22: value JMP -> 10K
- R27, R54, R57, R66, R69: value 10K -> 20K
- R33: value 4.7K -> 1K
- R34: value 20K -> 10K
- R4, R5: value 0.1 -> 1K; footprint Resistor_SMD:R_2512_6332Metric -> Resistor_SMD:R_0402_1005Metric
- R40: value 10K -> 1M; footprint Resistor_SMD:R_0402_1005Metric -> Resistor_SMD:R_0603_1608Metric
- R41, R42, R43: value 4.7K -> 1M; footprint Resistor_SMD:R_0402_1005Metric -> Resistor_SMD:R_0603_1608Metric
- R44: value 4.7K -> 33K
- R45, R46: value 1K -> 33K
- R47: value 1M -> 33K; footprint Resistor_SMD:R_0603_1608Metric -> Resistor_SMD:R_0402_1005Metric
- R48, R49, R50: value 1M -> 1K; footprint Resistor_SMD:R_0603_1608Metric -> Resistor_SMD:R_0402_1005Metric
- R51, R63: value JMP -> 20K
- R52, R61: value JMP -> 1M
- R53, R62: value JMP -> 1K
- R59, R65: value 33K -> 1K
- R60: value 33K -> 20K
- R64: value 33K -> 1M
- R73, R76, R79, R82, R85, R88, R91, R94, R97: value 20K -> 1M
- R74, R77, R80, R83, R86, R89, R92, R95, R98: value 1M -> 1K
- U1: value INA3221AIRGVR -> MAX4372FEUK; footprint Package_DFN_QFN:QFN-16-1EP_4x4mm_P0.65mm_EP2.1x2.1mm -> Package_TO_SOT_SMD:SOT-23-5
- U13: value PCA9534BS3,118 -> 74HC4051BQ,115; footprint Package_DFN_QFN:HVQFN-16-1EP_3x3mm_P0.5mm_EP1.5x1.5mm -> 74hc4051:QFN50P250X350X100-17N-D
- U2: value MCP2515-xST -> MAX4372FEUK; footprint Package_SO:TSSOP-20_4.4x6.5mm_P0.65mm -> Package_TO_SOT_SMD:SOT-23-5
- U3: value TJA1051T-3 -> MCP2515-xST; footprint Package_SON:HVSON-8-1EP_3x3mm_P0.65mm_EP1.6x2.4mm -> Package_SO:TSSOP-20_4.4x6.5mm_P0.65mm
- U4: value PCA9534BS3,118 -> MCP2515-xST; footprint Package_DFN_QFN:HVQFN-16-1EP_3x3mm_P0.5mm_EP1.5x1.5mm -> Package_SO:TSSOP-20_4.4x6.5mm_P0.65mm
- U5: value PCA9534BS3,118 -> TJA1051T-3; footprint Package_DFN_QFN:HVQFN-16-1EP_3x3mm_P0.5mm_EP1.5x1.5mm -> Package_SON:HVSON-8-1EP_3x3mm_P0.65mm_EP1.6x2.4mm
- U6: value ATmega2560-16AU -> TJA1051T-3; footprint Package_QFP:TQFP-100_14x14mm_P0.5mm -> Package_SON:HVSON-8-1EP_3x3mm_P0.65mm_EP1.6x2.4mm
- U7: value AMS1117-3.3 -> ATmega128A-AU; footprint Package_TO_SOT_SMD:SOT-89-3 -> Package_QFP:TQFP-64_14x14mm_P0.8mm
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- renumbered J3 to J7
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Connections:
- C11 pad 1: +5V -> S0_MCP_RESET
- C12 pad 1: +5V -> S1_MCP_RESET
- C13 pad 1: Net-(C13-Pad1) -> +5V
- C14 pad 1: Net-(C14-Pad1) -> +5V
- C15 pad 1: +5V -> +5V_A
- C17 pad 1: +5V -> Net-(C17-Pad1)
- C19 pad 1: +5V -> Net-(C19-Pad1)
- C20 pad 1: +3V3 -> +5V
- C24 pad 1: +5V -> +3V3
- C25 pad 1: +3V3 -> Net-(C25-Pad1)
- C28 pad 1: Net-(C28-Pad1) -> +5V
- C29 pad 1: Net-(C28-Pad1) -> Net-(C29-Pad1)
- C3 pad 1: +5V -> Net-(C3-Pad1)
- C30 pad 1: Net-(C30-Pad1) -> +5V
- C31 pad 1: Net-(C31-Pad1) -> +3V3
- C33 pad 1: Net-(C32-Pad1) -> +5V
- C35 pad 1: Net-(C35-Pad1) -> +5V
- C36 pad 1: Net-(C36-Pad1) -> +5V
- C37 pad 1: Net-(C36-Pad1) -> +3V3
- C39 pad 1: Net-(C39-Pad1) -> +5V
- C40 pad 1: Net-(C40-Pad1) -> +5V
- C41 pad 1: Net-(C40-Pad1) -> Net-(C41-Pad1)
- C43 pad 1: Net-(C43-Pad1) -> +5V_A
- C45 pad 1: Net-(C44-Pad1) -> Net-(C45-Pad1)
- C47 pad 1: Net-(C47-Pad1) -> +5V_A
- C49 pad 1: Net-(C48-Pad1) -> +5V_A
- C53 pad 1: Net-(C52-Pad1) -> Net-(C53-Pad1)
- C55 pad 1: Net-(C55-Pad1) -> +5V_A
- C57 pad 1: Net-(C56-Pad1) -> Net-(C57-Pad1)
- C59 pad 1: Net-(C59-Pad1) -> +5V_A
- C6 pad 1: +5V -> Net-(C6-Pad1)
- C61 pad 1: Net-(C60-Pad1) -> Net-(C61-Pad1)
- C63 pad 1: Net-(C63-Pad1) -> +5V_A
- C65 pad 1: Net-(C64-Pad1) -> Net-(C65-Pad1)
- C67 pad 1: Net-(C67-Pad1) -> +5V_A
- C69 pad 1: Net-(C68-Pad1) -> Net-(C69-Pad1)
- C71 pad 1: Net-(C71-Pad1) -> +5V_A
- C73 pad 1: Net-(C72-Pad1) -> Net-(C73-Pad1)
- C75 pad 1: Net-(C75-Pad1) -> +5V_A
- C77 pad 1: Net-(C76-Pad1) -> Net-(C77-Pad1)
- C79 pad 1: Net-(C79-Pad1) -> +5V_A
- C8 pad 1: MCP_RESET -> +5V
- C81 pad 1: Net-(C80-Pad1) -> Net-(C81-Pad1)
- C83 pad 1: Net-(C83-Pad1) -> +5V_A
- C85 pad 1: Net-(C84-Pad1) -> Net-(C85-Pad1)
- C87 pad 1: Net-(C87-Pad1) -> +5V_A
- C89 pad 1: Net-(C88-Pad1) -> Net-(C89-Pad1)
- C91 pad 1: Net-(C91-Pad1) -> +5V_A
- CH2 pad 1: /CAN1-H -> Net-(CH2-Pad1)
- CL2 pad 1: /CAN1-L -> Net-(CL2-Pad1)
- D1 pad 2: +5V_GEIGER -> +5V_A
- D10 pad 2: Net-(C36-Pad1) -> Net-(C16-Pad1)
- D11 pad 2: Net-(C40-Pad1) -> Net-(C44-Pad1)
- D12 pad 2: Net-(C44-Pad1) -> Net-(C50-Pad1)
- D14 pad 2: Net-(C52-Pad1) -> Net-(C56-Pad1)
- D15 pad 2: Net-(C56-Pad1) -> Net-(C60-Pad1)
- D16 pad 2: Net-(C60-Pad1) -> Net-(C64-Pad1)
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Routing:
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- added copper zone on F.Cu, net Net-(C100-Pad1)
- added copper zone on F.Cu, net Net-(C16-Pad1)
- added copper zone on F.Cu, net Net-(C44-Pad1)
- added copper zone on F.Cu, net Net-(C48-Pad1)
- added copper zone on F.Cu, net Net-(C50-Pad1)
- added copper zone on F.Cu, net Net-(C56-Pad1)
- added copper zone on F.Cu, net Net-(C60-Pad1)
- added copper zone on F.Cu, net Net-(C64-Pad1)
- added copper zone on F.Cu, net Net-(C68-Pad1)
- added copper zone on F.Cu, net Net-(C72-Pad1)
- added copper zone on F.Cu, net Net-(C76-Pad1)
- added copper zone on F.Cu, net Net-(C80-Pad1)
- added copper zone on F.Cu, net Net-(C84-Pad1)
- added copper zone on F.Cu, net Net-(C88-Pad1)
- added copper zone on F.Cu, net Net-(C92-Pad1)
- added copper zone on F.Cu, net Net-(C96-Pad1)
Other:
- net class Default: via_dia 0.8 -> 0.6; via_drill 0.4 -> 0.3
- net class Power added: clearance 0.3, trace_width 0.35, via_dia 0.8, via_drill 0.4

Commit message: Merge with github repo
Update naming scheme for older boards
Prepare for merge
Parts:
- removed C100, C44, C48, C50, C56, C60, C64, C68, C72, C76, C80, C84, C88, C92, C96: 100nF, Capacitor_SMD:C_0402_1005Metric
- removed C101, C102, C41, C42, C45, C46, C51, C52, C53, C54, C57, C58, C61, C62, C65, C66, C69, C70, C73, C74, C77, C78, C81, C82, C85, C86, C89, C90, C93, C94, C97, C98: 22pF, Capacitor_SMD:C_0402_1005Metric
- removed C39, C40: 22uF, Capacitor_Tantalum_SMD:CP_EIA-3216-10_Kemet-I
- removed C43, C47, C49, C55, C59, C63, C67, C71, C75, C79, C83, C87, C91, C95, C99: 1uF, Capacitor_SMD:C_0603_1608Metric
- removed D10, D11, D12, D13, D14, D15, D16, D17, D18, D19, D20, D21, D22, D23, D24, D25: NODE_STATUSLED, LED_SMD:LED_0402_1005Metric
- removed J10: Conn_01x03_Male, Connector_PinHeader_2.54mm:PinHeader_1x03_P2.54mm_Vertical
- removed J11, J12: AVR-ISP-6, Connector_PinHeader_2.54mm:PinHeader_2x03_P2.54mm_Vertical
- removed J13, J14, J15, J16, J17, J18, J19, J20, J21, J22, J23, J24, J25, J26, J27, J28: AVR-ISP-6, Connector_PinHeader_1.27mm:PinHeader_2x03_P1.27mm_Vertical_SMD
- removed the J7 at (209.9, -52.6)
- removed R100, R101, R102, R103, R104, R105, R106, R107, R108, R109, R110, R111, R112, R113, R114, R99: 0R, Resistor_SMD:R_0603_1608Metric
- removed R47: 33K, Resistor_SMD:R_0402_1005Metric
- removed R48, R49, R50, R53, R56, R59, R62, R65, R68, R71, R74, R77, R80, R83, R86, R89, R92, R95, R98: 1K, Resistor_SMD:R_0402_1005Metric
- removed R51, R54, R57, R60, R63, R66, R69, R72, R75, R78, R81, R84, R87, R90, R93, R96: 20K, Resistor_SMD:R_0402_1005Metric
- removed R52, R55, R58, R61, R64, R67, R70, R73, R76, R79, R82, R85, R88, R91, R94, R97: 1M, Resistor_SMD:R_0402_1005Metric
- removed SW1, SW10, SW11, SW12, SW13, SW14, SW15, SW16, SW2, SW3, SW4, SW5, SW6, SW7, SW8, SW9: ADG802BRT, Package_TO_SOT_SMD:SOT-23-6
- removed U17, U18, U19, U20, U21, U22, U23, U24, U25, U26, U27, U28, U29: ATmega328PB-MU, Package_DFN_QFN:QFN-32-1EP_5x5mm_P0.5mm_EP3.1x3.1mm
- removed Y10, Y11, Y12, Y13, Y14, Y15, Y16, Y17, Y18, Y19, Y20, Y5, Y6, Y7, Y8, Y9: 8 MHz, Crystal:Crystal_SMD_2520-4Pin_2.5x2.0mm
- added F1: Polyfuse, Resistor_SMD:R_0805_2012Metric, F.Cu at (500.3, 112.8)
- added F2: Polyfuse, Resistor_SMD:R_0805_2012Metric, F.Cu at (500.3, 115.8)
- C15: value 1uF -> 22pF; footprint Capacitor_SMD:C_0603_1608Metric -> Capacitor_SMD:C_0402_1005Metric
- C16, C38: value 100nF -> 10uF; footprint Capacitor_SMD:C_0402_1005Metric -> Capacitor_SMD:C_0603_1608Metric
- C17, C19, C32: value 22pF -> 100nF
- C18: value 100nF -> 22pF
- C21, C35: value 100nF -> 22uF; footprint Capacitor_SMD:C_0402_1005Metric -> Capacitor_SMD:C_0603_1608Metric
- C24: footprint Capacitor_SMD:C_0603_1608Metric -> Capacitor_SMD:C_0402_1005Metric
- C25, C36: value 100nF -> 22uF; footprint Capacitor_SMD:C_0402_1005Metric -> Capacitor_Tantalum_SMD:CP_EIA-3216-10_Kemet-I
- C27: value 22uF -> 22pF; footprint Capacitor_Tantalum_SMD:CP_EIA-3216-10_Kemet-I -> Capacitor_SMD:C_0402_1005Metric
- C28: value 10uF -> 100nF; footprint Capacitor_SMD:C_0603_1608Metric -> Capacitor_SMD:C_0402_1005Metric
- C31: value 22uF -> 100nF; footprint Capacitor_SMD:C_0603_1608Metric -> Capacitor_SMD:C_0402_1005Metric
- C37: value 100nF -> 22uF; footprint Capacitor_SMD:C_0603_1608Metric -> Capacitor_Tantalum_SMD:CP_EIA-3216-10_Kemet-I
- J3: value Conn_01x07_Female -> GeigerBoard
- J4, J6: value Micro_SD_Card -> Conn_02x03_Odd_Even; footprint Connector_Card:microSD_HC_Wuerth_693072010801 -> Connector_PinHeader_2.54mm:PinHeader_2x03_P2.54mm_Vertical
- J5: value Conn_01x03_Female -> Solar_Temp
- J8: value AVR-JTAG-10 -> Conn_01x03_Male; footprint Connector_PinHeader_2.54mm:PinHeader_2x05_P2.54mm_Vertical -> Connector_PinHeader_2.54mm:PinHeader_1x03_P2.54mm_Vertical
- R20, R35: value 4.7K -> 1K
- R22, R29, R30: value 10K -> 4.7K
- R23: value 1K -> 10K
- R24: value 4.7K -> 10K
- R25: value 10K -> 20K
- R27: value 20K -> 10K
- R31: value 1M -> 4.7K
- R32: value 1K -> 1M
- R34: value 10K -> 1K
- R36, R37, R38: value 4.7K -> 1M; footprint Resistor_SMD:R_0402_1005Metric -> Resistor_SMD:R_0603_1608Metric
- R39: value 1K -> 1M; footprint Resistor_SMD:R_0402_1005Metric -> Resistor_SMD:R_0603_1608Metric
- R40, R41, R42, R43: value 1M -> 33K; footprint Resistor_SMD:R_0603_1608Metric -> Resistor_SMD:R_0402_1005Metric
- R44, R45, R46: value 33K -> 1K
- U10: value 74HC4051BQ,115 -> AT25DF161-SF-T; footprint 74hc4051:QFN50P250X350X100-17N-D -> Package_SO:SO-8_3.9x4.9mm_P1.27mm
- U11: value 74HC4051BQ,115 -> ATmega128A-AU; footprint 74hc4051:QFN50P250X350X100-17N-D -> Package_QFP:TQFP-64_14x14mm_P0.8mm
- U12: value 74HC4051BQ,115 -> AMS1117-3.3; footprint 74hc4051:QFN50P250X350X100-17N-D -> Package_TO_SOT_SMD:SOT-89-3
- U14, U15, U16: value ATmega328PB-MU -> 74HC4051BQ,115; footprint Package_DFN_QFN:QFN-32-1EP_5x5mm_P0.5mm_EP3.1x3.1mm -> 74hc4051:QFN50P250X350X100-17N-D
- U7: value ATmega128A-AU -> AMS1117-3.3; footprint Package_QFP:TQFP-64_14x14mm_P0.8mm -> Package_TO_SOT_SMD:SOT-89-3
- U8: value AMS1117-3.3 -> AT25DF161-SF-T; footprint Package_TO_SOT_SMD:SOT-89-3 -> Package_SO:SO-8_3.9x4.9mm_P1.27mm
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- renumbered J9 to J7
Connections:
- C1 pad 1: +5V -> +5V_A
- C10 pad 1: +5V -> +5V_A
- C13 pad 1: +5V -> +5V_A
- C14 pad 1: +5V -> +5V_A
- C15 pad 1: +5V_A -> Net-(C15-Pad1)
- C16 pad 1: Net-(C16-Pad1) -> +5V_A
- C17 pad 1: Net-(C17-Pad1) -> +5V_A
- C18 pad 1: +5V -> Net-(C18-Pad1)
- C19 pad 1: Net-(C19-Pad1) -> +5V_A
- C2 pad 1: +5V -> +5V_A
- C20 pad 1: +5V -> Net-(C20-Pad1)
- C22 pad 1: +5V -> +5V_A
- C23 pad 1: +5V -> +5V_A
- C24 pad 1: +3V3 -> Net-(C24-Pad1)
- C25 pad 1: Net-(C25-Pad1) -> +5V_A
- C26 pad 1: +5V -> +5V_A
- C27 pad 1: +5V -> Net-(C27-Pad1)
- C28 pad 1: +5V -> +5V_A
- C30 pad 1: +5V -> +5V_A
- C31 pad 1: +3V3 -> Net-(C31-Pad1)
- C32 pad 1: Net-(C32-Pad1) -> +5V_A
- C33 pad 1: +5V -> +5V_A
- C35 pad 1: +5V -> Net-(C35-Pad1)
- C36 pad 1: +5V -> +5V_A
- C37 pad 1: +3V3 -> +5V_A
- C38 pad 1: Net-(C38-Pad1) -> +5V_A
- C7 pad 1: +5V -> +5V_A
- C8 pad 1: +5V -> +5V_A
- C9 pad 1: +5V -> +5V_A
- D2 pad 2: +5V_B -> +5V_A
- D7 pad 2: +5V -> +5V_A
- J4 pad 1: (no net) -> S1_SPI0_MISO
- J4 pad 2: Net-(J4-Pad2) -> (no net)
- J4 pad 3: Net-(J4-Pad3) -> S1_SPI0_SCK
- J4 pad 4: +3V3 -> S1_SPI0_MOSI
- J4 pad 5: Net-(J4-Pad5) -> /Payload MCU/S1_ISP_RESET
- J4 pad 6: +3V3 -> GND
- J5 pad 2: +5V -> +5V_A
- J6 pad 1: (no net) -> S0_SPI0_MISO
- J6 pad 2: Net-(J6-Pad2) -> (no net)
- J6 pad 3: Net-(J6-Pad3) -> S0_SPI0_SCK
- J6 pad 4: +3V3 -> S0_SPI0_MOSI
- J6 pad 5: Net-(J6-Pad5) -> /Payload MCU/S0_ISP_RESET
- J6 pad 6: +3V3 -> GND
- J8 pad 1: /Payload MCU/S1_JTAG_TCK -> /Payload MCU/S1_DBG_RX
- J8 pad 3: /Payload MCU/S1_JTAG_TDO -> /Payload MCU/S1_DBG_TX
- L1 pad 1: +5V -> +5V_A
- L1 pad 2: Net-(C25-Pad1) -> Net-(C24-Pad1)
- L2 pad 1: +5V -> +5V_A
- L2 pad 2: Net-(C38-Pad1) -> Net-(C34-Pad1)
- R10 pad 1: +5V -> +5V_A
- R11 pad 2: +5V -> +5V_A
- R12 pad 1: Net-(C17-Pad1) -> Net-(C15-Pad1)
- R12 pad 2: Net-(C19-Pad1) -> Net-(C18-Pad1)
- R17 pad 1: Net-(J4-Pad2) -> Net-(R17-Pad1)
- R17 pad 2: /Payload MCU/S1_SD_CS -> S1_SPI0_SCK
- R18 pad 1: Net-(J4-Pad3) -> Net-(R18-Pad1)
- R19 pad 1: Net-(J4-Pad5) -> Net-(R19-Pad1)
- R19 pad 2: S1_SPI0_SCK -> /Payload MCU/S1_SD_CS
- R20 pad 1: Net-(J4-Pad7) -> Net-(R20-Pad1)
- R20 pad 2: S1_SPI0_MISO -> /Payload MCU/GEIGER_EN
- R21 pad 1: S1_SPI0_MISO -> /Payload MCU/S1_SD_CS
- R22 pad 1: S1_SPI0_SCK -> +5V_A
- R22 pad 2: GND -> 1WIRE
- R23 pad 1: Net-(R23-Pad1) -> S1_SPI0_MOSI
- R23 pad 2: /Payload MCU/GEIGER_EN -> GND
- R24 pad 1: +5V -> S1_SPI0_SCK
- R24 pad 2: 1WIRE -> GND
- R25 pad 1: S1_SPI0_MOSI -> /Payload MCU/S0_ISP_RESET
- R25 pad 2: GND -> +5V_A
- R26 pad 1: /Payload MCU/S1_SD_CS -> S0_SPI0_SCK
- R27 pad 1: /Payload MCU/S0_ISP_RESET -> S0_SPI0_MOSI
- R27 pad 2: +5V -> GND
- R29 pad 1: S0_SPI0_MOSI -> Net-(R29-Pad1)
- R29 pad 2: GND -> S0_SPI0_SCK
- R30 pad 1: S0_SPI0_SCK -> Net-(R30-Pad1)
- R30 pad 2: GND -> S0_SPI0_MOSI
- R31 pad 1: Net-(C29-Pad1) -> Net-(R31-Pad1)
- R31 pad 2: Net-(C32-Pad1) -> /Payload MCU/S0_SD_CS
- R32 pad 1: /Payload MCU/S0_DBG_RX -> Net-(C27-Pad1)
- R32 pad 2: Net-(R32-Pad2) -> Net-(C29-Pad1)
- R33 pad 1: Net-(R33-Pad1) -> /Payload MCU/S0_DBG_RX
- R33 pad 2: /Payload MCU/S0_DBG_TX -> Net-(R33-Pad2)
- R34 pad 1: S0_SPI0_MISO -> Net-(R34-Pad1)
- R34 pad 2: GND -> /Payload MCU/S0_DBG_TX
- R35 pad 1: Net-(J6-Pad2) -> Net-(R35-Pad1)
- R35 pad 2: /Payload MCU/S0_SD_CS -> /Payload MCU/GEIGER_EN
- R36 pad 1: Net-(J6-Pad3) -> Net-(H1-Pad1)
- R36 pad 2: S0_SPI0_MOSI -> GND
- R37 pad 1: Net-(J6-Pad5) -> Net-(H2-Pad1)
- R37 pad 2: S0_SPI0_SCK -> GND
- R38 pad 1: Net-(J6-Pad7) -> Net-(H3-Pad1)
- R38 pad 2: S0_SPI0_MISO -> GND
- R39 pad 1: Net-(R39-Pad1) -> Net-(H4-Pad1)
- R39 pad 2: /Payload MCU/GEIGER_EN -> GND
- R40 pad 1: Net-(H1-Pad1) -> +5V_A
- R40 pad 2: GND -> Net-(R40-Pad2)
- R41 pad 1: Net-(H2-Pad1) -> +5V_A
- R41 pad 2: GND -> Net-(R41-Pad2)
- R42 pad 1: Net-(H3-Pad1) -> +5V_A
- R42 pad 2: GND -> Net-(R42-Pad2)
- R43 pad 1: Net-(H4-Pad1) -> +5V_A
- R43 pad 2: GND -> Net-(R43-Pad2)
- R44 pad 1: +5V -> GND
- R44 pad 2: Net-(R44-Pad2) -> Net-(D7-Pad1)
- R45 pad 1: +5V -> GND
- R45 pad 2: Net-(R45-Pad2) -> Net-(D8-Pad1)
- R46 pad 1: +5V -> GND
- R46 pad 2: Net-(R46-Pad2) -> Net-(D9-Pad1)
- R9 pad 1: +5V -> +5V_A
- R_CSA1 pad 2: +5V -> Net-(F1-Pad2)
- R_CSB1 pad 1: +5V_B -> +5V_A
- R_CSB1 pad 2: +5V -> Net-(F2-Pad2)
- U1 pad 3: +5V -> +5V_A
- U1 pad 4: +5V -> Net-(F1-Pad2)
- U10 pad 1: NODE4_RX -> Net-(R31-Pad1)
- U10 pad 2: NODE6_RX -> S0_SPI0_MISO
- U10 pad 3: /Payload MCU/S0_UART1_RX -> Net-(C35-Pad1)
- U10 pad 4: NODE7_RX -> GND
- U10 pad 5: NODE5_RX -> Net-(R30-Pad1)
- U10 pad 6: Net-(R44-Pad2) -> Net-(R29-Pad1)
- U10 pad 7: +5V -> Net-(C35-Pad1)
- U10 pad 8: GND -> Net-(C35-Pad1)
- U11 pad 1: NODE12_RX -> (no net)
- U11 pad 10: /Payload MCU/S1_UART1_MUX1_A1 -> (no net)
- U11 pad 11: /Payload MCU/S1_UART1_MUX1_A0 -> S0_SPI0_SCK
- U11 pad 12: NODE11_RX -> S0_SPI0_MOSI
- U11 pad 13: NODE8_RX -> S0_SPI0_MISO
- U11 pad 14: NODE9_RX -> /Payload MCU/S0_UART1_MUX0_A0
- U11 pad 15: NODE10_RX -> /Payload MCU/S0_UART1_MUX0_A1
- U11 pad 16: +5V -> /Payload MCU/S0_UART1_MUX0_A2
- U11 pad 17: (no net) -> 1WIRE
- U11 pad 2: NODE14_RX -> Net-(R33-Pad2)
- U11 pad 3: /Payload MCU/S1_UART1_RX -> Net-(R34-Pad1)
- U11 pad 4: NODE15_RX -> (no net)
- U11 pad 5: NODE13_RX -> (no net)
- U11 pad 6: Net-(R45-Pad2) -> S0_MCP_RX1BF
- U11 pad 7: +5V -> S0_MCP_RX0BF
- U11 pad 8: GND -> S0_MCP_TX0RTS
- U11 pad 9: /Payload MCU/S1_UART1_MUX1_A2 -> S0_MCP_INT
- U12 pad 1: NODE4_TX -> GND
- U12 pad 2: NODE6_TX -> Net-(C35-Pad1)
- U12 pad 3: /Payload MCU/S0_UART1_TX -> +5V_A
- U13 pad 1: NODE12_TX -> (no net)
- U13 pad 10: /Payload MCU/S1_UART1_MUX1_A1 -> /Payload MCU/S0_UART1_MUX0_A1
- U13 pad 11: /Payload MCU/S1_UART1_MUX1_A0 -> /Payload MCU/S0_UART1_MUX0_A0
- U13 pad 12: NODE11_TX -> (no net)
- U13 pad 13: NODE8_TX -> (no net)
- U13 pad 14: NODE9_TX -> (no net)
- U13 pad 15: NODE10_TX -> (no net)
- U13 pad 16: +5V -> +5V_A
- U13 pad 2: NODE14_TX -> (no net)
- U13 pad 3: /Payload MCU/S1_UART1_TX -> /Payload MCU/S0_UART1_RX
- U13 pad 4: NODE15_TX -> (no net)
- U13 pad 5: NODE13_TX -> (no net)
- U13 pad 6: Net-(R47-Pad2) -> Net-(R40-Pad2)
- U13 pad 9: /Payload MCU/S1_UART1_MUX1_A2 -> /Payload MCU/S0_UART1_MUX0_A2
- U14 pad 10: (no net) -> /Payload MCU/S1_UART1_MUX1_A1
- U14 pad 11: (no net) -> /Payload MCU/S1_UART1_MUX1_A0
- U14 pad 15: /Payload MCU/MCU Node1/ISP_MOSI -> (no net)
- U14 pad 16: /Payload MCU/MCU Node1/ISP_MISO -> +5V_A
- U14 pad 17: Net-(R100-Pad1) -> (no net)
- U14 pad 3: (no net) -> /Payload MCU/S1_UART1_RX
- U14 pad 4: Net-(C16-Pad1) -> (no net)
- U14 pad 5: GND -> (no net)
- U14 pad 6: (no net) -> Net-(R41-Pad2)
- U14 pad 7: Net-(C42-Pad1) -> +5V
- U14 pad 8: Net-(C41-Pad1) -> GND
- U14 pad 9: (no net) -> /Payload MCU/S1_UART1_MUX1_A2
- U15 pad 10: (no net) -> /Payload MCU/S0_UART1_MUX0_A1
- U15 pad 11: (no net) -> /Payload MCU/S0_UART1_MUX0_A0
- U15 pad 15: /Payload MCU/MCU Node2/ISP_MOSI -> (no net)
- U15 pad 16: /Payload MCU/MCU Node2/ISP_MISO -> +5V_A
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Routing:
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- removed copper zone on F.Cu, net Net-(C100-Pad1)
- removed copper zone on F.Cu, net Net-(C16-Pad1)
- removed copper zone on F.Cu, net Net-(C44-Pad1)
- removed copper zone on F.Cu, net Net-(C48-Pad1)
- removed copper zone on F.Cu, net Net-(C50-Pad1)
- removed copper zone on F.Cu, net Net-(C56-Pad1)
- removed copper zone on F.Cu, net Net-(C60-Pad1)
- removed copper zone on F.Cu, net Net-(C64-Pad1)
- removed copper zone on F.Cu, net Net-(C68-Pad1)
- removed copper zone on F.Cu, net Net-(C72-Pad1)
- removed copper zone on F.Cu, net Net-(C76-Pad1)
- removed copper zone on F.Cu, net Net-(C80-Pad1)
- removed copper zone on F.Cu, net Net-(C84-Pad1)
- removed copper zone on F.Cu, net Net-(C88-Pad1)
- removed copper zone on F.Cu, net Net-(C92-Pad1)
- removed copper zone on F.Cu, net Net-(C96-Pad1)
