File: ykts-payload/ykts-payload.kicad_pcb (KiCad board)
At the start: 4 copper layers, 95.9 x 90.2 mm, 146 parts, among them J1 PC/104 Connector, J2 DBG_PWR, J3 GeigerBoard, J4 Conn_02x03_Odd_Even, J5 Solar_Temp, J6 Conn_02x03_Odd_Even, J7 Conn_01x03_Male, J8 Conn_01x03_Male, Q1 KIA3415, U1 MAX4372FEUK, U10 AT25DF161-SF-T, U11 ATmega128A-AU, U12 AMS1117-3.3, U13 74HC4051BQ,115, U14 74HC4051BQ,115, U15 74HC4051BQ,115, U16 74HC4051BQ,115, U2 MAX4372FEUK, U3 MCP2515-xST, U4 MCP2515-xST, U5 TJA1051T-3, U6 TJA1051T-3, U7 AMS1117-3.3, U8 AT25DF161-SF-T, U9 ATmega128A-AU, Y1 12MHz, Y2 12MHz, Y3 8 MHz, Y4 8 MHz

Commit message: Hierarchal sheet rework
Parts:
- removed C31, C32, C33, C34: 100nF, Capacitor_SMD:C_0402_1005Metric
- removed C35: 22uF, Capacitor_SMD:C_0603_1608Metric
- removed C36, C37: 22uF, Capacitor_Tantalum_SMD:CP_EIA-3216-10_Kemet-I
- removed C38: 10uF, Capacitor_SMD:C_0603_1608Metric
- removed F1, F2: Polyfuse, Resistor_SMD:R_0805_2012Metric
- removed the J2 at (238.6, -23.9)
- removed the R27 at (431.7, 124.8)
- removed the R28 at (423.0, 129.7)
- removed the R29 at (428.6, 124.3)
- removed the R30 at (407.9, 144.7)
- removed the R5 at (366.9, 179.3)
- removed the R6 at (360.7, 180.5)
- removed R_CSA1: 0.1, Resistor_SMD:R_2010_5025Metric
- removed the U5 at (319.9, 158.0)
- added J1: DBG_PWR, Connector_PinHeader_2.54mm:PinHeader_1x03_P2.54mm_Vertical, F.Cu at (302.5, -63.6)
- added J9: Conn_01x03_Male, Connector_PinHeader_2.54mm:PinHeader_1x03_P2.54mm_Vertical, F.Cu at (256.6, -13.6)
- added N1: YKTS-MCU-NODE, ykts-mcu-node:YktSat_MCU_node, F.Cu at (134.4, 117.1)
- added N10: YKTS-MCU-NODE, ykts-mcu-node:YktSat_MCU_node, F.Cu at (237.7, -49.7)
- added N11: YKTS-MCU-NODE, ykts-mcu-node:YktSat_MCU_node, F.Cu at (259.1, -65.1)
- added N12: YKTS-MCU-NODE, ykts-mcu-node:YktSat_MCU_node, F.Cu at (237.7, -34.4)
- added N13: YKTS-MCU-NODE, ykts-mcu-node:YktSat_MCU_node, F.Cu at (259.1, -49.7)
- added N14: YKTS-MCU-NODE, ykts-mcu-node:YktSat_MCU_node, F.Cu at (280.5, -65.1)
- added N15: YKTS-MCU-NODE, ykts-mcu-node:YktSat_MCU_node, F.Cu at (259.1, -34.4)
- added N16: YKTS-MCU-NODE, ykts-mcu-node:YktSat_MCU_node, F.Cu at (280.5, -49.7)
- added N2: YKTS-MCU-NODE, ykts-mcu-node:YktSat_MCU_node, F.Cu at (117.6, 109.5)
- added N3: YKTS-MCU-NODE, ykts-mcu-node:YktSat_MCU_node, F.Cu at (101.1, 109.5)
- added N4: YKTS-MCU-NODE, ykts-mcu-node:YktSat_MCU_node, F.Cu at (150.9, 117.1)
- added N5: YKTS-MCU-NODE, ykts-mcu-node:YktSat_MCU_node, F.Cu at (114.9, 123.2)
- added N6: YKTS-MCU-NODE, ykts-mcu-node:YktSat_MCU_node, F.Cu at (164.5, 123.2)
- added N7: YKTS-MCU-NODE, ykts-mcu-node:YktSat_MCU_node, F.Cu at (131.4, 123.2)
- added N8: YKTS-MCU-NODE, ykts-mcu-node:YktSat_MCU_node, F.Cu at (148.0, 123.2)
- added N9: YKTS-MCU-NODE, ykts-mcu-node:YktSat_MCU_node, F.Cu at (237.7, -65.1)
- added Q2: PMV65XP, Package_TO_SOT_SMD:SOT-23, F.Cu at (208.0, 93.4)
- added Q3: PMV65XP, Package_TO_SOT_SMD:SOT-23, F.Cu at (229.4, 59.9)
- added R10: 10K, Resistor_SMD:R_0402_1005Metric, F.Cu at (217.6, 82.7)
- added R36: 1K, Resistor_SMD:R_0402_1005Metric, F.Cu at (267.1, -8.96)
- added R44: 10K, Resistor_SMD:R_0402_1005Metric, F.Cu at (326.7, -46.6)
- added R45: 1K, Resistor_SMD:R_0402_1005Metric, F.Cu at (323.8, -47.0)
- added R46: 1M, Resistor_SMD:R_0402_1005Metric, F.Cu at (329.6, -56.8)
- added R47: 1K, Resistor_SMD:R_0402_1005Metric, F.Cu at (326.7, -56.8)
- added R48: 10K, Resistor_SMD:R_0402_1005Metric, F.Cu at (323.8, -56.8)
- added R49: 33K, Resistor_SMD:R_0402_1005Metric, F.Cu at (304.3, -14.9)
- added R50: 33K, Resistor_SMD:R_0402_1005Metric, F.Cu at (354.4, -64.9)
- added R9: 1K, Resistor_SMD:R_0402_1005Metric, F.Cu at (217.6, 80.7)
- added R_CSB2: 0.1, Resistor_SMD:R_1210_3225Metric, F.Cu at (325.1, -50.1)
- added U9: ATmega128A-AU, Package_QFP:TQFP-64_14x14mm_P0.8mm, F.Cu at (245.1, -6.71)
- C1, C11, C17, C2: value 100nF -> 22pF
- C10, C25, C26: value 22uF -> 22pF; footprint Capacitor_Tantalum_SMD:CP_EIA-3216-10_Kemet-I -> Capacitor_SMD:C_0402_1005Metric
- C12, C30: footprint Capacitor_SMD:C_0402_1005Metric -> Capacitor_SMD:C_0603_1608Metric
- C13: value 100nF -> 22uF; footprint Capacitor_SMD:C_0603_1608Metric -> Capacitor_Tantalum_SMD:CP_EIA-3216-10_Kemet-I
- C14: footprint Capacitor_SMD:C_0603_1608Metric -> Capacitor_SMD:C_0402_1005Metric
- C15, C27: value 22pF -> 100nF; footprint Capacitor_SMD:C_0402_1005Metric -> Capacitor_SMD:C_0603_1608Metric
- C16: value 10uF -> 22pF; footprint Capacitor_SMD:C_0603_1608Metric -> Capacitor_SMD:C_0402_1005Metric
- C18, C29, C3, C4, C5: value 22pF -> 100nF
- C21: footprint Capacitor_SMD:C_0603_1608Metric -> Capacitor_Tantalum_SMD:CP_EIA-3216-10_Kemet-I
- C22: value 100nF -> 10uF; footprint Capacitor_SMD:C_0402_1005Metric -> Capacitor_SMD:C_0603_1608Metric
- C23: value 100nF -> 22uF; footprint Capacitor_SMD:C_0402_1005Metric -> Capacitor_SMD:C_0603_1608Metric
- C28: value 100nF -> 22uF; footprint Capacitor_SMD:C_0402_1005Metric -> Capacitor_Tantalum_SMD:CP_EIA-3216-10_Kemet-I
- C6: value 22pF -> 22uF; footprint Capacitor_SMD:C_0402_1005Metric -> Capacitor_Tantalum_SMD:CP_EIA-3216-10_Kemet-I
- C7: value 100nF -> 10uF
- C8: value 100nF -> 22uF
- C9: value 22uF -> 100nF; footprint Capacitor_Tantalum_SMD:CP_EIA-3216-10_Kemet-I -> Capacitor_SMD:C_0402_1005Metric
- D1: value LED -> LED_PWON
- D2: value LED -> LED_STATUS
- D3: value TVS1 -> LED; footprint Diode_SMD:D_SOD-323 -> LED_SMD:LED_0402_1005Metric
- D6: value TVS2 -> LED_STATUS; footprint Diode_SMD:D_SOD-323 -> LED_SMD:LED_0402_1005Metric
- D7: value LED_PWON -> LED
- D8: value LED_STATUS -> TVS1; footprint LED_SMD:LED_0402_1005Metric -> Diode_SMD:D_SOD-323
- D9: value LED_STATUS -> TVS2; footprint LED_SMD:LED_0402_1005Metric -> Diode_SMD:D_SOD-323
- J4: value Conn_02x03_Odd_Even -> Solar_Temp; footprint Connector_PinHeader_2.54mm:PinHeader_2x03_P2.54mm_Vertical -> Connector_PinHeader_1.27mm:PinHeader_1x03_P1.27mm_Vertical
- J5: value Solar_Temp -> Sensor_Ext; footprint Connector_PinHeader_1.27mm:PinHeader_1x03_P1.27mm_Vertical -> Connector_PinHeader_1.27mm:PinHeader_1x04_P1.27mm_Vertical
- J6: footprint Connector_PinHeader_2.54mm:PinHeader_2x03_P2.54mm_Vertical -> Connector_PinHeader_1.27mm:PinHeader_2x03_P1.27mm_Vertical_SMD
- J8: value Conn_01x03_Male -> Conn_02x03_Odd_Even; footprint Connector_PinHeader_2.54mm:PinHeader_1x03_P2.54mm_Vertical -> Connector_PinHeader_1.27mm:PinHeader_2x03_P1.27mm_Vertical_SMD
- Q1: value KIA3415 -> PMV65XP
- R1, R2: footprint Resistor_SMD:R_0402_1005Metric -> Resistor_SMD:R_0603_1608Metric
- R15, R16: value 4.7K -> 1K
- R17, R18, R19: value 4.7K -> 10K
- R20: value 1K -> 4.7K
- R21: value 10K -> 4.7K
- R23: value 10K -> 1K
- R25: value 20K -> 1K
- R26: value 10K -> 33K
- R27: renamed from R36; value 1M -> 33K; footprint Resistor_SMD:R_0603_1608Metric -> Resistor_SMD:R_0402_1005Metric
- R28: renamed from R44; value 1K -> 1M
- R3, R4: value 1K -> 1M; footprint Resistor_SMD:R_0402_1005Metric -> Resistor_SMD:R_0603_1608Metric
- R30: renamed from R46; value 1K -> 10K
- R31: value 4.7K -> 20K
- R37, R38, R39: value 1M -> 10K; footprint Resistor_SMD:R_0603_1608Metric -> Resistor_SMD:R_0402_1005Metric
- R40, R41, R42: value 33K -> 4.7K
- R43: value 33K -> 1K
- R6: renamed from R8; value 1K -> 4.7K
- R7: renamed from R9; value 10K -> 4.7K
- R8: renamed from R10; value 10K -> 4.7K
- R_CSB1: footprint Resistor_SMD:R_2010_5025Metric -> Resistor_SMD:R_1210_3225Metric
- U1: value MAX4372FEUK -> ATmega128A-AU; footprint Package_TO_SOT_SMD:SOT-23-5 -> Package_QFP:TQFP-64_14x14mm_P0.8mm
- U10: value AT25DF161-SF-T -> AMS1117-3.3; footprint Package_SO:SO-8_3.9x4.9mm_P1.27mm -> Package_TO_SOT_SMD:SOT-89-3
- U11: value ATmega128A-AU -> AT25DF161-SF-T; footprint Package_QFP:TQFP-64_14x14mm_P0.8mm -> Package_SO:SO-8_3.9x4.9mm_P1.27mm
- U12: value AMS1117-3.3 -> MAX4372FEUK; footprint Package_TO_SOT_SMD:SOT-89-3 -> Package_TO_SOT_SMD:SOT-23-5
- U13: value 74HC4051BQ,115 -> MCP2515-xST; footprint 74hc4051:QFN50P250X350X100-17N-D -> Package_SO:TSSOP-20_4.4x6.5mm_P0.65mm
- U14: value 74HC4051BQ,115 -> MCP2551-I-SN; footprint 74hc4051:QFN50P250X350X100-17N-D -> Package_SO:SOIC-8_3.9x4.9mm_P1.27mm
- U15, U16: footprint 74hc4051:QFN50P250X350X100-17N-D -> Package_SO:TSSOP-16_4.4x5mm_P0.65mm
- U2: value MAX4372FEUK -> AMS1117-3.3; footprint Package_TO_SOT_SMD:SOT-23-5 -> Package_TO_SOT_SMD:SOT-89-3
- U3: value MCP2515-xST -> AT25DF161-SF-T; footprint Package_SO:TSSOP-20_4.4x6.5mm_P0.65mm -> Package_SO:SO-8_3.9x4.9mm_P1.27mm
- U4: value MCP2515-xST -> MAX4372FEUK; footprint Package_SO:TSSOP-20_4.4x6.5mm_P0.65mm -> Package_TO_SOT_SMD:SOT-23-5
- U5: renamed from U9; value ATmega128A-AU -> 74HC4051BQ,115; footprint Package_QFP:TQFP-64_14x14mm_P0.8mm -> Package_SO:TSSOP-16_4.4x5mm_P0.65mm
- U6: value TJA1051T-3 -> 74HC4051BQ,115; footprint Package_SON:HVSON-8-1EP_3x3mm_P0.65mm_EP1.6x2.4mm -> Package_SO:TSSOP-16_4.4x5mm_P0.65mm
- U7: value AMS1117-3.3 -> MCP2515-xST; footprint Package_TO_SOT_SMD:SOT-89-3 -> Package_SO:TSSOP-20_4.4x6.5mm_P0.65mm
- U8: value AT25DF161-SF-T -> MCP2551-I-SN; footprint Package_SO:SO-8_3.9x4.9mm_P1.27mm -> Package_SO:SOIC-8_3.9x4.9mm_P1.27mm
- Y1: value 12MHz -> 8 MHz
- Y3: footprint Crystal:Crystal_SMD_5032-4Pin_5.0x3.2mm -> Crystal:Crystal_SMD_3225-4Pin_3.2x2.5mm
- Y4: value 8 MHz -> 12MHz; footprint Crystal:Crystal_SMD_5032-4Pin_5.0x3.2mm -> Crystal:Crystal_SMD_3225-4Pin_3.2x2.5mm
- moved C24 408.9 mm to (29.8, 53.1)
- moved R11 403.3 mm to (38.5, 46.0), turned to 90 degrees
- moved L1 399.7 mm to (35.4, 41.9)
- moved C22 397.9 mm to (44.3, 49.3)
- moved C18 393.8 mm to (35.2, 57.9)
- moved C19 391.7 mm to (46.4, 47.5)
- moved R13 388.3 mm to (33.7, 63.2)
- moved R20 387.7 mm to (30.6, 66.3)
- moved R14 385.3 mm to (33.7, 65.3)
- moved C15 375.0 mm to (26.5, 55.4)
- moved C26 365.9 mm to (36.4, 37.8)
- moved Y3 357.4 mm to (37.5, 64.8)
- moved R12 355.0 mm to (73.5, 65.4), turned to 270 degrees
- moved Y4 335.2 mm to (82.9, 77.5), turned to 90 degrees
- moved J4 328.2 mm to (93.2, 43.9), turned to 180 degrees
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- renumbered J3 to J2, J1 to J3, R45 to R29, R7 to R5
Connections:
- C1 pad 1: +5V_A -> Net-(C1-Pad1)
- C10 pad 1: +5V_A -> Net-(C10-Pad1)
- C11 pad 1: S0_MCP_RESET -> Net-(C11-Pad1)
- C12 pad 1: S1_MCP_RESET -> +5V_A
- C14 pad 1: +5V_A -> /CANBUS Controller 0/MCP_RESET
- C15 pad 1: Net-(C15-Pad1) -> +5V_A
- C16 pad 1: +5V_A -> Net-(C16-Pad1)
- C17 pad 1: +5V_A -> Net-(C17-Pad1)
- C18 pad 1: Net-(C18-Pad1) -> +5V_A
- C2 pad 1: +5V_A -> Net-(C2-Pad1)
- C21 pad 1: Net-(C21-Pad1) -> +5V_A
- C23 pad 1: +5V_A -> Net-(C23-Pad1)
- C24 pad 1: Net-(C24-Pad1) -> +5V_A
- C25 pad 1: +5V_A -> Net-(C25-Pad1)
- C26 pad 1: +5V_A -> Net-(C26-Pad1)
- C27 pad 1: Net-(C27-Pad1) -> +5V_A
- C29 pad 1: Net-(C29-Pad1) -> /CANBUS Controller 1/MCP_RESET
- C3 pad 1: Net-(C3-Pad1) -> +5V_A
- C4 pad 1: Net-(C4-Pad1) -> +5V_A
- C6 pad 1: Net-(C6-Pad1) -> +5V_A
- C8 pad 1: +5V_A -> Net-(C8-Pad1)
- CH2 pad 1: Net-(CH2-Pad1) -> CANH
- CH3 pad 1: /CAN1-H -> Net-(CH3-Pad1)
- CH4 pad 1: /CAN1-H -> CANH
- CL2 pad 1: Net-(CL2-Pad1) -> CANL
- CL3 pad 1: /CAN1-L -> Net-(CL3-Pad1)
- CL4 pad 1: /CAN1-L -> CANL
- D1 pad 2: +5V_A -> +5V
- D2 pad 2: +5V_A -> Net-(D2-Pad2)
- D3 pad 1: /CAN1-H -> Net-(D3-Pad1)
- D3 pad 2: GND -> +5V_A
- D4 pad 1: /CAN1-H -> CANH
- D5 pad 1: /CAN1-L -> CANL
- D6 pad 1: /CAN1-L -> Net-(D6-Pad1)
- D6 pad 2: GND -> Net-(D6-Pad2)
- D8 pad 1: Net-(D8-Pad1) -> CANH
- D8 pad 2: /Payload MCU/S0_LED_ST -> GND
- D9 pad 1: Net-(D9-Pad1) -> CANL
- D9 pad 2: /Payload MCU/S1_LED_ST -> GND
- FL1 pad 2: /CAN1-H -> CANH
- FL1 pad 4: /CAN1-L -> CANL
- FL2 pad 1: Net-(CH2-Pad1) -> Net-(CH3-Pad1)
- FL2 pad 2: /CAN1-H -> CANH
- FL2 pad 3: Net-(CL2-Pad1) -> Net-(CL3-Pad1)
- FL2 pad 4: /CAN1-L -> CANL
- J2 pad 2: /Payload MCU/I2C_SDA -> /I2C_SDA
- J2 pad 5: /Payload MCU/GEIGER_EN -> (no net)
- J2 pad 6: /Payload MCU/I2C_SCL -> /I2C_SCL
- J4 pad 1: S1_SPI0_MISO -> GND
- J4 pad 2: (no net) -> +5V_A
- J4 pad 3: S1_SPI0_SCK -> /1WIRE
- J5 pad 1: GND -> +5V_A
- J5 pad 2: +5V_A -> /I2C_SCL
- J5 pad 3: 1WIRE -> GND
- J6 pad 1: S0_SPI0_MISO -> /CANBUS Controller 0/MISO
- J6 pad 3: S0_SPI0_SCK -> /CANBUS Controller 0/SCK
- J6 pad 4: S0_SPI0_MOSI -> /CANBUS Controller 0/MOSI
- J6 pad 5: /Payload MCU/S0_ISP_RESET -> Net-(J6-Pad5)
- J7 pad 1: /Payload MCU/S0_DBG_RX -> Net-(J7-Pad1)
- J7 pad 3: /Payload MCU/S0_DBG_TX -> Net-(J7-Pad3)
- J8 pad 1: /Payload MCU/S1_DBG_RX -> /CANBUS Controller 1/MISO
- J8 pad 2: GND -> (no net)
- J8 pad 3: /Payload MCU/S1_DBG_TX -> /CANBUS Controller 1/SCK
- L1 pad 2: Net-(C24-Pad1) -> Net-(C5-Pad1)
- L2 pad 2: Net-(C34-Pad1) -> Net-(C20-Pad1)
- Q1 pad 2: +5V -> +5V_GEIGER
- Q1 pad 3: +5V_GEIGER -> +5V
- R1 pad 1: Net-(C4-Pad1) -> Net-(H1-Pad1)
- R1 pad 2: Net-(C3-Pad1) -> GND
- R11 pad 1: /Payload MCU/S1_ISP_RESET -> Net-(J6-Pad5)
- R12 pad 1: Net-(C15-Pad1) -> Net-(C1-Pad1)
- R12 pad 2: Net-(C18-Pad1) -> Net-(C2-Pad1)
- R13 pad 1: /Payload MCU/S1_DBG_RX -> Net-(R13-Pad1)
- R13 pad 2: Net-(R13-Pad2) -> (no net)
- R14 pad 1: Net-(R14-Pad1) -> Net-(J7-Pad3)
- R14 pad 2: /Payload MCU/S1_DBG_TX -> Net-(R14-Pad2)
- R15 pad 1: +5V -> Net-(R15-Pad1)
- R15 pad 2: /Payload MCU/I2C_SCL -> Net-(J7-Pad1)
- R16 pad 1: /Payload MCU/I2C_SDA -> GND
- R16 pad 2: +5V -> Net-(D2-Pad1)
- R17 pad 1: Net-(R17-Pad1) -> /CANBUS Controller 0/SCK
- R17 pad 2: S1_SPI0_SCK -> GND
- R18 pad 1: Net-(R18-Pad1) -> /CANBUS Controller 0/MOSI
- R18 pad 2: S1_SPI0_MOSI -> GND
- R19 pad 1: Net-(R19-Pad1) -> /Payload Supervisor 0/SD_CS
- R19 pad 2: /Payload MCU/S1_SD_CS -> GND
- R2 pad 1: Net-(C6-Pad1) -> Net-(H2-Pad1)
- R2 pad 2: Net-(C5-Pad1) -> GND
- R20 pad 2: /Payload MCU/GEIGER_EN -> /CANBUS Controller 0/SCK
- R21 pad 1: /Payload MCU/S1_SD_CS -> Net-(R21-Pad1)
- R21 pad 2: GND -> /CANBUS Controller 0/MOSI
- R22 pad 1: +5V_A -> Net-(R22-Pad1)
- R22 pad 2: 1WIRE -> /Payload Supervisor 0/SD_CS
- R23 pad 1: S1_SPI0_MOSI -> Net-(Q2-Pad1)
- R23 pad 2: GND -> +5V
- R24 pad 1: S1_SPI0_SCK -> GND
- R24 pad 2: GND -> Net-(Q2-Pad1)
- R25 pad 1: /Payload MCU/S0_ISP_RESET -> Net-(D3-Pad1)
- R25 pad 2: +5V_A -> GND
- R26 pad 1: S0_SPI0_SCK -> +5V_A
- R26 pad 2: GND -> Net-(R26-Pad2)
- R27 pad 1: Net-(H1-Pad1) -> +5V_A
- R27 pad 2: GND -> Net-(R27-Pad2)
- R28 pad 1: GND -> Net-(C11-Pad1)
- R28 pad 2: Net-(D7-Pad1) -> Net-(C10-Pad1)
- R29 pad 1: GND -> /CANBUS Controller 0/MCP_RESET
- R29 pad 2: Net-(D8-Pad1) -> Net-(R29-Pad2)
- R3 pad 1: Net-(D1-Pad1) -> Net-(H3-Pad1)
- R30 pad 1: GND -> +5V_A
- R30 pad 2: Net-(D9-Pad1) -> /CANBUS Controller 0/MCP_RESET
- R31 pad 1: Net-(R31-Pad1) -> Net-(J8-Pad5)
- R31 pad 2: /Payload MCU/S0_SD_CS -> +5V_A
- R32 pad 1: Net-(C27-Pad1) -> Net-(C16-Pad1)
- R32 pad 2: Net-(C29-Pad1) -> Net-(C17-Pad1)
- R33 pad 1: /Payload MCU/S0_DBG_RX -> Net-(R33-Pad1)
- R33 pad 2: Net-(R33-Pad2) -> (no net)
- R34 pad 1: Net-(R34-Pad1) -> Net-(J9-Pad3)
- R34 pad 2: /Payload MCU/S0_DBG_TX -> Net-(R34-Pad2)
- R35 pad 2: /Payload MCU/GEIGER_EN -> Net-(J9-Pad1)
- R37 pad 1: Net-(H2-Pad1) -> /CANBUS Controller 1/SCK
- R38 pad 1: Net-(H3-Pad1) -> /CANBUS Controller 1/MOSI
- R39 pad 1: Net-(H4-Pad1) -> /Payload Supervisor 1/SD_CS
- R4 pad 1: Net-(D2-Pad1) -> Net-(H4-Pad1)
- R40 pad 1: +5V_A -> Net-(R40-Pad1)
- R40 pad 2: Net-(R40-Pad2) -> /CANBUS Controller 1/SCK
- R41 pad 1: +5V_A -> Net-(R41-Pad1)
- R41 pad 2: Net-(R41-Pad2) -> /CANBUS Controller 1/MOSI
- R42 pad 1: +5V_A -> Net-(R42-Pad1)
- R42 pad 2: Net-(R42-Pad2) -> /Payload Supervisor 1/SD_CS
- R43 pad 1: +5V_A -> Net-(Q3-Pad1)
- R43 pad 2: Net-(R43-Pad2) -> +5V
- R5 pad 1: S0_MCP_RESET -> GND
- R5 pad 2: Net-(R7-Pad2) -> Net-(D1-Pad1)
- R6 pad 1: S1_MCP_RESET -> +5V
- R6 pad 2: Net-(R8-Pad2) -> /I2C_SCL
- R7 pad 1: +5V_A -> /I2C_SDA
- R7 pad 2: S0_MCP_RESET -> +5V
- R8 pad 2: S1_MCP_RESET -> /1WIRE
- R_CSB1 pad 2: Net-(F2-Pad2) -> Net-(Q2-Pad2)
- U1 pad 1: GND -> (no net)
- U1 pad 2: CS_5VA -> Net-(R14-Pad2)
- U1 pad 3: +5V_A -> Net-(R15-Pad1)
- U1 pad 4: Net-(F1-Pad2) -> (no net)
- U1 pad 5: +5V_A -> (no net)
- U10 pad 1: Net-(R31-Pad1) -> GND
- U10 pad 2: S0_SPI0_MISO -> Net-(C23-Pad1)
- U10 pad 3: Net-(C35-Pad1) -> +5V_A
- U11 pad 1: (no net) -> Net-(R42-Pad1)
- U11 pad 2: Net-(R33-Pad2) -> /CANBUS Controller 1/MISO
- U11 pad 3: Net-(R34-Pad1) -> Net-(C23-Pad1)
- U11 pad 4: (no net) -> GND
- U11 pad 5: (no net) -> Net-(R41-Pad1)
- U11 pad 6: S0_MCP_RX1BF -> Net-(R40-Pad1)
- U11 pad 7: S0_MCP_RX0BF -> Net-(C23-Pad1)
- U11 pad 8: S0_MCP_TX0RTS -> Net-(C23-Pad1)
- U12 pad 2: Net-(C35-Pad1) -> /Payload Power Control 1/CSENSE
- U13 pad 1: (no net) -> Net-(U13-Pad1)
- U13 pad 10: /Payload MCU/S0_UART1_MUX0_A1 -> GND
- U13 pad 11: /Payload MCU/S0_UART1_MUX0_A0 -> /CANBUS Controller 1/MCP_RX1BF
- U13 pad 12: (no net) -> /CANBUS Controller 1/MCP_RX0BF
- U13 pad 13: (no net) -> /CANBUS Controller 1/MCP_INT
- U13 pad 14: (no net) -> /CANBUS Controller 1/SCK
- U13 pad 16: +5V_A -> /CANBUS Controller 1/MOSI
- U13 pad 17: (no net) -> /CANBUS Controller 1/MISO
- U13 pad 2: (no net) -> Net-(U13-Pad2)
- U13 pad 3: /Payload MCU/S0_UART1_RX -> (no net)
- U13 pad 4: (no net) -> /CANBUS Controller 1/MCP_TX0RTS
- U13 pad 6: Net-(R40-Pad2) -> (no net)
- U13 pad 7: +5V -> (no net)
- U13 pad 8: GND -> Net-(C25-Pad1)
- U13 pad 9: /Payload MCU/S0_UART1_MUX0_A2 -> Net-(C26-Pad1)
- U14 pad 1: (no net) -> Net-(U13-Pad2)
- U14 pad 2: (no net) -> GND
- U14 pad 3: /Payload MCU/S1_UART1_RX -> +5V_A
- U14 pad 4: (no net) -> Net-(U13-Pad1)
- U14 pad 5: (no net) -> +5V_A
- U14 pad 6: Net-(R41-Pad2) -> Net-(CL3-Pad1)
- U14 pad 7: +5V -> Net-(CH3-Pad1)
- U15 pad 1: (no net) -> /N12_TX
- U15 pad 10: /Payload MCU/S0_UART1_MUX0_A1 -> /Node RX MUX 1/A1
- U15 pad 11: /Payload MCU/S0_UART1_MUX0_A0 -> /Node RX MUX 1/A0
- U15 pad 12: (no net) -> /N11_TX
- U15 pad 13: (no net) -> /N10_TX
- U15 pad 14: (no net) -> /N9_TX
- U15 pad 15: (no net) -> /N8_TX
- U15 pad 2: (no net) -> /N15_TX
- U15 pad 3: /Payload MCU/S0_UART1_TX -> /Node TX MUX 1/IN
- U15 pad 4: (no net) -> /N13_TX
- U15 pad 5: (no net) -> /N14_TX
- U15 pad 6: Net-(R42-Pad2) -> Net-(R49-Pad2)
- U15 pad 7: +5V -> +5V_A
- U15 pad 9: /Payload MCU/S0_UART1_MUX0_A2 -> /Node RX MUX 1/A2
- U16 pad 1: (no net) -> /N12_RX
- U16 pad 10: /Payload MCU/S1_UART1_MUX1_A1 -> /Node RX MUX 1/A1
- U16 pad 11: /Payload MCU/S1_UART1_MUX1_A0 -> /Node RX MUX 1/A0
- U16 pad 12: (no net) -> /N11_RX
- U16 pad 13: (no net) -> /N10_RX
- U16 pad 14: (no net) -> /N9_RX
- U16 pad 15: (no net) -> /N8_RX
- U16 pad 2: (no net) -> /N15_RX
- U16 pad 3: /Payload MCU/S1_UART1_TX -> /Node RX MUX 1/IN
- U16 pad 4: (no net) -> /N13_RX
- U16 pad 5: (no net) -> /N14_RX
- U16 pad 6: Net-(R43-Pad2) -> Net-(R50-Pad2)
- U16 pad 7: +5V -> +5V_A
- U16 pad 9: /Payload MCU/S1_UART1_MUX1_A2 -> /Node RX MUX 1/A2
- U2 pad 2: CS_5VB -> Net-(C8-Pad1)
- U3 pad 1: Net-(U3-Pad1) -> Net-(R22-Pad1)
- U3 pad 2: Net-(U3-Pad2) -> /CANBUS Controller 0/MISO
- U3 pad 3: (no net) -> Net-(C8-Pad1)
- U3 pad 4: S0_MCP_TX0RTS -> GND
- U3 pad 5: (no net) -> Net-(R21-Pad1)
- U3 pad 6: (no net) -> Net-(R20-Pad1)
- U3 pad 7: (no net) -> Net-(C8-Pad1)
- U3 pad 8: Net-(C3-Pad1) -> Net-(C8-Pad1)
- U4 pad 1: Net-(U4-Pad1) -> GND
- U4 pad 2: Net-(U4-Pad2) -> /Payload Power Control 0/CSENSE
- U4 pad 3: (no net) -> +5V_A
- U4 pad 4: S1_MCP_TX0RTS -> Net-(Q2-Pad2)
- U4 pad 5: (no net) -> +5V_A
- U5 pad 1: (no net) -> /N4_RX
- U5 pad 10: (no net) -> /Node RX MUX 0/A1
- U5 pad 11: S1_SPI0_SCK -> /Node RX MUX 0/A0
- U5 pad 12: S1_SPI0_MOSI -> /N3_RX
- U5 pad 13: S1_SPI0_MISO -> /N2_RX
- U5 pad 14: /Payload MCU/S1_UART1_MUX1_A0 -> /N1_RX
- U5 pad 15: /Payload MCU/S1_UART1_MUX1_A1 -> /N0_RX
- U5 pad 16: /Payload MCU/S1_UART1_MUX1_A2 -> +5V_A
- U5 pad 2: Net-(R13-Pad2) -> /N7_RX
- U5 pad 3: Net-(R14-Pad1) -> /Node RX MUX 0/IN
- U5 pad 4: (no net) -> /N5_RX
- U5 pad 5: (no net) -> /N6_RX
- U5 pad 6: S1_MCP_RX1BF -> Net-(R26-Pad2)
- U5 pad 7: S1_MCP_RX0BF -> +5V_A
- U5 pad 8: S1_MCP_TX0RTS -> GND
- U5 pad 9: S1_MCP_INT -> /Node RX MUX 0/A2
- U6 pad 1: Net-(U4-Pad2) -> /N4_TX
- U6 pad 2: GND -> /N7_TX
- U6 pad 3: +5V_A -> /Node TX MUX 0/IN
- U6 pad 4: Net-(U4-Pad1) -> /N5_TX
- U6 pad 5: +5V_A -> /N6_TX
- U6 pad 6: Net-(CL2-Pad1) -> Net-(R27-Pad2)
- U6 pad 7: Net-(CH2-Pad1) -> +5V_A
- U6 pad 9: (no net) -> /Node RX MUX 0/A2
- U7 pad 1: GND -> Net-(U7-Pad1)
- U7 pad 2: Net-(C21-Pad1) -> Net-(U7-Pad2)
- U7 pad 3: +5V_A -> (no net)
- U8 pad 1: Net-(R19-Pad1) -> Net-(U7-Pad2)
- U8 pad 2: S1_SPI0_MISO -> GND
- U8 pad 3: Net-(C21-Pad1) -> +5V_A
- U8 pad 4: GND -> Net-(U7-Pad1)
- U8 pad 5: Net-(R18-Pad1) -> +5V_A
- U8 pad 6: Net-(R17-Pad1) -> Net-(CL1-Pad1)
- U8 pad 7: Net-(C21-Pad1) -> Net-(CH1-Pad1)
- U8 pad 8: Net-(C21-Pad1) -> GND
- Y1 pad 1: Net-(C4-Pad1) -> Net-(C1-Pad1)
- Y1 pad 3: Net-(C3-Pad1) -> Net-(C2-Pad1)
- Y2 pad 1: Net-(C6-Pad1) -> Net-(C11-Pad1)
- Y2 pad 3: Net-(C5-Pad1) -> Net-(C10-Pad1)
- Y3 pad 1: Net-(C15-Pad1) -> Net-(C16-Pad1)
- Y3 pad 3: Net-(C18-Pad1) -> Net-(C17-Pad1)
- Y4 pad 1: Net-(C27-Pad1) -> Net-(C26-Pad1)
- Y4 pad 3: Net-(C29-Pad1) -> Net-(C25-Pad1)
Routing:
- net Net-(C4-Pad1): track 18.4 -> 9.81 mm
- net Net-(C5-Pad1): track 0.00 -> 7.29 mm
- net /CAN1-H: track 8.77 -> 3.42 mm
- net /CAN1-L: track 7.44 -> 3.00 mm
- net CANH: track 0.00 -> 4.39 mm
- net CANL: track 0.00 -> 3.72 mm
- net Net-(C8-Pad1): track 0.00 -> 3.52 mm
- net +5V_A: track 9.76 -> 13.0 mm
- net Net-(D1-Pad1): track 0.00 -> 2.69 mm
- net GND: track 8.27 -> 5.91 mm, vias 4 -> 3
- net /I2C_SCL: track 0.00 -> 2.07 mm
- net Net-(R7-Pad2): track 2.07 -> 0.00 mm
- net Net-(R8-Pad2): track 2.07 -> 0.00 mm
- net Net-(C3-Pad1): track 13.4 -> 11.8 mm
- net Net-(U3-Pad1): track 6.01 -> 4.47 mm
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Other:
- outline, holes or cut-outs redrawn
