File: ykts-payload/ykts-payload.kicad_pcb (KiCad board)
At the start: 4 copper layers, 95.9 x 90.2 mm, 167 parts, among them J1 DBG_PWR, J2 GeigerBoard, J3 PC/104 Connector, J4 Solar_Temp, J5 Sensor_Ext, J6 Conn_02x03_Odd_Even, J7 Conn_01x03_Male, J8 Conn_02x03_Odd_Even, J9 Conn_01x03_Male, Q1 PMV65XP, Q2 PMV65XP, Q3 PMV65XP, Q4 RJU003N03 NMOS, Q5 RJU003N03 NMOS, Q6 RJU003N03 NMOS, Q7 RJU003N03 NMOS, U1 ATmega128A-AU, U10 AMS1117-3.3, U11 AT25DF161-SF-T, U12 MAX4372FEUK, U13 MCP2515-xST, U14 MCP2551-I-SN, U15 74HC4051BQ,115, U16 74HC4051BQ,115, U2 AMS1117-3.3, U3 AT25DF161-SF-T, U4 MAX4372FEUK, U5 74HC4051BQ,115, U6 74HC4051BQ,115, U7 MCP2515-xST, U8 MCP2551-I-SN, U9 ATmega128A-AU, Y1 8 MHz, Y2 12MHz, Y3 8 MHz, Y4 12MHz

Commit message: Bump
Parts:
- moved J5 7.11 mm to (94.5, 84.6), turned to 0 degrees
- moved R27 1.80 mm to (132.5, 109.0)
- moved U6 1.80 mm to (127.9, 110.2)
- moved C15 0.81 mm to (161.8, 89.7), turned to 90 degrees
Connections:
- U15 pad 1: /N12_TX -> /N15_TX
- U15 pad 12: /N11_TX -> /N9_TX
- U15 pad 13: /N10_TX -> /N8_TX
- U15 pad 14: /N9_TX -> /N12_TX
- U15 pad 15: /N8_TX -> /N14_TX
- U15 pad 2: /N15_TX -> /N13_TX
- U15 pad 4: /N13_TX -> /N11_TX
- U15 pad 5: /N14_TX -> /N10_TX
- U16 pad 1: /N12_RX -> /N15_RX
- U16 pad 12: /N11_RX -> /N9_RX
- U16 pad 13: /N10_RX -> /N8_RX
- U16 pad 14: /N9_RX -> /N12_RX
- U16 pad 15: /N8_RX -> /N14_RX
- U16 pad 2: /N15_RX -> /N13_RX
- U16 pad 4: /N13_RX -> /N11_RX
- U16 pad 5: /N14_RX -> /N10_RX
- U5 pad 1: /N4_RX -> /N7_RX
- U5 pad 12: /N3_RX -> /N1_RX
- U5 pad 13: /N2_RX -> /N0_RX
- U5 pad 14: /N1_RX -> /N4_RX
- U5 pad 15: /N0_RX -> /N6_RX
- U5 pad 2: /N7_RX -> /N5_RX
- U5 pad 4: /N5_RX -> /N3_RX
- U5 pad 5: /N6_RX -> /N2_RX
- U6 pad 1: /N4_TX -> /N7_TX
- U6 pad 12: /N3_TX -> /N1_TX
- U6 pad 13: /N2_TX -> /N0_TX
- U6 pad 14: /N1_TX -> /N4_TX
- U6 pad 15: /N0_TX -> /N6_TX
- U6 pad 2: /N7_TX -> /N5_TX
- U6 pad 4: /N5_TX -> /N3_TX
- U6 pad 5: /N6_TX -> /N2_TX
Routing:
- net Net-(U7-Pad2): track 0.00 -> 16.6 mm
- net Net-(U7-Pad1): track 0.00 -> 15.3 mm
- added copper zone on F.Cu, net +5V_A

Commit message: Bump board
Parts:
- removed C16, C17, C25, C26: 22pF, Capacitor_SMD:C_0402_1005Metric
- removed C18, C19, C20, C24, C27, C29, C30: 100nF, Capacitor_SMD:C_0402_1005Metric
- removed C21, C28: 22uF, Capacitor_Tantalum_SMD:CP_EIA-3216-10_Kemet-I
- removed C22: 10uF, Capacitor_SMD:C_0603_1608Metric
- removed C23: 22uF, Capacitor_SMD:C_0603_1608Metric
- removed CH3, CH4, CL3, CL4: 50pF, Capacitor_SMD:C_0402_1005Metric
- removed D1: LED_PWON, LED_SMD:LED_0402_1005Metric
- removed D3, D7: LED, LED_SMD:LED_0402_1005Metric
- removed D6: LED_STATUS, LED_SMD:LED_0402_1005Metric
- removed D8: TVS1, Diode_SMD:D_SOD-323
- removed D9: TVS2, Diode_SMD:D_SOD-323
- removed FL2: DLW21SN921SK2, Inductor_SMD:L_CommonModeChoke_Coilcraft_0805USB
- removed J8: Conn_02x03_Odd_Even, Connector_PinHeader_1.27mm:PinHeader_2x03_P1.27mm_Vertical_SMD
- removed L2: Ferrite, Inductor_SMD:L_1206_3216Metric
- removed N10, N11, N12, N13, N14, N15, N16, N9: YKTS-MCU-NODE, ykts-mcu-node:YktSat_MCU_node
- removed Q3: PMV65XP, Package_TO_SOT_SMD:SOT-23
- removed Q5, Q7: RJU003N03 NMOS, Package_TO_SOT_SMD:SOT-323_SC-70
- removed R25, R33, R34, R35, R36, R43, R45, R47, R5: 1K, Resistor_SMD:R_0402_1005Metric
- removed R31: 20K, Resistor_SMD:R_0402_1005Metric
- removed R32, R46: 1M, Resistor_SMD:R_0402_1005Metric
- removed R37, R38, R39, R44, R48, R52, R54: 10K, Resistor_SMD:R_0402_1005Metric
- removed R40, R41, R42: 4.7K, Resistor_SMD:R_0402_1005Metric
- removed R49, R50: 33K, Resistor_SMD:R_0402_1005Metric
- removed R_CSB2: 0.1, Resistor_SMD:R_1210_3225Metric
- removed U10: AMS1117-3.3, Package_TO_SOT_SMD:SOT-89-3
- removed U11: AT25DF161-SF-T, Package_SO:SO-8_3.9x4.9mm_P1.27mm
- removed U12: MAX4372FEUK, Package_TO_SOT_SMD:SOT-23-5
- removed U13: MCP2515-xST, Package_SO:TSSOP-20_4.4x6.5mm_P0.65mm
- removed U14: MCP2551-I-SN, Package_SO:SOIC-8_3.9x4.9mm_P1.27mm
- removed U15, U16: 74HC4051BQ,115, Package_SO:TSSOP-16_4.4x5mm_P0.65mm
- removed U9: ATmega128A-AU, Package_QFP:TQFP-64_14x14mm_P0.8mm
- removed Y3: 8 MHz, Crystal:Crystal_SMD_3225-4Pin_3.2x2.5mm
- removed Y4: 12MHz, Crystal:Crystal_SMD_3225-4Pin_3.2x2.5mm
- moved J1 245.8 mm to (94.6, 110.6), turned to 180 degrees
- moved R8 224.3 mm to (96.9, 123.1), turned to 90 degrees
- moved J4 221.3 mm to (94.6, 125.1)
- moved R4 216.9 mm to (94.2, 136.0), turned to 90 degrees
- moved R7 210.7 mm to (96.6, 118.1), turned to -90 degrees
- moved R6 209.4 mm to (96.6, 114.6), turned to -90 degrees
- moved R1 183.9 mm to (179.1, 139.6), turned to 90 degrees
- moved R3 171.4 mm to (94.2, 72.5), turned to -90 degrees
- moved J9 158.3 mm to (94.6, 100.3), turned to 180 degrees
- moved R2 119.4 mm to (179.1, 69.9)
- moved R14 113.3 mm to (98.2, 85.1)
- moved R15 112.3 mm to (98.2, 86.5)
- moved J6 52.7 mm to (152.7, 85.1), turned to 90 degrees
- moved J5 34.3 mm to (94.6, 118.9), turned to 180 degrees
- moved J7 27.3 mm to (94.6, 90.2)
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Connections:
- J5 pad 2: /I2C_SCL -> /SCL
- J5 pad 4: /I2C_SDA -> /SDA
- R13 pad 2: /Payload Supervisor 0/GEIGER_EN -> /GEIGER_EN
- R9 pad 2: MOSFET_GEIGER -> /GEIGER_FET
- U1 pad 19: /Payload Supervisor 0/GEIGER_FET -> /GEIGER_FET
- U1 pad 32: /Payload Supervisor 0/1WIRE -> /1WIRE
- U1 pad 39: /N0_PWR -> /N0_RST
- U1 pad 40: /N0_RST -> /N0_PWR
- U1 pad 44: /N2_PWR -> /N2_RST
- U1 pad 45: /N2_RST -> /N2_PWR
- U1 pad 46: /N3_PWR -> /N3_RST
- U1 pad 47: /N3_RST -> /N3_PWR
Routing:
- net /SCL: track 8.31 -> 226.4 mm, vias 0 -> 2
- net /SDA: track 10.1 -> 210.0 mm, vias 0 -> 4
- net +5V_A: track 37.6 -> 229.6 mm, vias 0 -> 30
- net +5V: track 1.41 -> 156.9 mm, vias 0 -> 2
- net /N6_RST: track 0.00 -> 74.5 mm
- net /N6_PWR: track 0.00 -> 72.5 mm
- net /1WIRE: track 0.00 -> 66.1 mm, vias 0 -> 1
- net /Payload Power Control 0/CSENSE: track 0.00 -> 62.8 mm, vias 0 -> 2
- net /N4_RST: track 0.00 -> 61.1 mm
- net /N4_PWR: track 0.00 -> 60.2 mm
- net /N0_RST: track 0.00 -> 58.4 mm
- net Net-(R14-Pad2): track 0.00 -> 57.9 mm, vias 0 -> 2
- net Net-(R15-Pad1): track 0.00 -> 57.8 mm, vias 0 -> 2
- net /N0_PWR: track 0.00 -> 55.9 mm
- net /N5_RST: track 0.00 -> 47.4 mm
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- added copper zone on In1.Cu, net +5V_A
- added copper zone on F.Cu, net GND
- added copper zone on In1.Cu, net GND
- removed copper zone on F.Cu, net Net-(Q3-Pad2)
Other:
- outline, holes or cut-outs redrawn

Commit message: Fix DRC on payload
Connections:
- Q4 pad 3: /SCL -> /S0_SCL
- Q6 pad 3: /SDA -> /S0_SDA
- U1 pad 25: /SCL -> /S0_SCL
- U1 pad 26: /SDA -> /S0_SDA
Routing:
- net +5V_A: track 229.6 -> 247.6 mm, vias 30 -> 31
- net /S0_SDA: track 0.00 -> 8.62 mm
- net /SDA: track 210.0 -> 201.3 mm
- net /SCL: track 226.4 -> 219.6 mm
- net /S0_SCL: track 0.00 -> 6.84 mm
- net GND: vias 75 -> 86

Commit message: Rework power supply
Parts:
- removed Q2: PMV65XP, Package_TO_SOT_SMD:SOT-23
- removed R24: 10K, Resistor_SMD:R_0402_1005Metric
- added C16: 22pF, Capacitor_SMD:C_0402_1005Metric, B.Cu at (126.2, 131.2)
- added C17: 22pF, Capacitor_SMD:C_0402_1005Metric, B.Cu at (126.2, 136.8)
- added C18: 100nF, Capacitor_SMD:C_0402_1005Metric, B.Cu at (128.7, 136.3)
- added C19: 100nF, Capacitor_SMD:C_0402_1005Metric, B.Cu at (148.7, 129.9)
- added C20: 100nF, Capacitor_SMD:C_0402_1005Metric, B.Cu at (149.6, 140.6)
- added C21: 22uF, Capacitor_Tantalum_SMD:CP_EIA-3216-10_Kemet-I, B.Cu at (150.5, 131.3)
- added C22: 10uF, Capacitor_SMD:C_0603_1608Metric, B.Cu at (116.7, 130.0)
- added C23: 22uF, Capacitor_SMD:C_0603_1608Metric, B.Cu at (119.8, 130.0)
- added C25: 22pF, Capacitor_SMD:C_0402_1005Metric, B.Cu at (165.8, 128.7)
- added C26: 22pF, Capacitor_SMD:C_0402_1005Metric, B.Cu at (165.8, 123.4)
- added C27: 100nF, Capacitor_SMD:C_0402_1005Metric, B.Cu at (156.9, 130.6)
- added C28: 22uF, Capacitor_Tantalum_SMD:CP_EIA-3216-10_Kemet-I, B.Cu at (161.7, 108.2)
- added C29: 100nF, Capacitor_SMD:C_0402_1005Metric, B.Cu at (155.4, 131.1)
- added C30: 100nF, Capacitor_SMD:C_0402_1005Metric, B.Cu at (165.3, 113.0)
- added CH3: 50pF, Capacitor_SMD:C_0402_1005Metric, B.Cu at (166.8, 103.6)
- added CH4: 50pF, Capacitor_SMD:C_0402_1005Metric, B.Cu at (163.0, 101.7)
- added CL3: 50pF, Capacitor_SMD:C_0402_1005Metric, B.Cu at (164.8, 103.6)
- added CL4: 50pF, Capacitor_SMD:C_0402_1005Metric, B.Cu at (167.8, 101.5)
- added D1: LED_PWON, LED_SMD:LED_0402_1005Metric, B.Cu at (198.4, 103.5)
- added D3: LED, LED_SMD:LED_0402_1005Metric, F.Cu at (200.3, 72.6)
- added D6: LED_STATUS, LED_SMD:LED_0402_1005Metric, B.Cu at (132.1, 142.4)
- added D8: TVS1, Diode_SMD:D_SOD-323, B.Cu at (162.4, 99.6)
- added D9: TVS2, Diode_SMD:D_SOD-323, B.Cu at (168.3, 99.6)
- added FL2: DLW21SN921SK2, Inductor_SMD:L_CommonModeChoke_Coilcraft_0805USB, B.Cu at (165.4, 101.9)
- added J8: Conn_02x03_Odd_Even, Connector_PinHeader_1.27mm:PinHeader_2x03_P1.27mm_Vertical_SMD, B.Cu at (164.0, 138.9)
- added L2: Ferrite, Inductor_SMD:L_1206_3216Metric, B.Cu at (149.6, 137.5)
- added N10: YKTS-MCU-NODE, ykts-mcu-node:YktSat_MCU_node, B.Cu at (98.9, 124.9)
- added N11: YKTS-MCU-NODE, ykts-mcu-node:YktSat_MCU_node, B.Cu at (137.0, 121.2)
- added N12: YKTS-MCU-NODE, ykts-mcu-node:YktSat_MCU_node, B.Cu at (137.0, 106.1)
- added N13: YKTS-MCU-NODE, ykts-mcu-node:YktSat_MCU_node, B.Cu at (128.1, 88.0)
- added N14: YKTS-MCU-NODE, ykts-mcu-node:YktSat_MCU_node, B.Cu at (143.2, 86.5)
- added N15: YKTS-MCU-NODE, ykts-mcu-node:YktSat_MCU_node, B.Cu at (117.6, 105.6)
- added N16: YKTS-MCU-NODE, ykts-mcu-node:YktSat_MCU_node, B.Cu at (158.1, 87.0)
- added N9: YKTS-MCU-NODE, ykts-mcu-node:YktSat_MCU_node, B.Cu at (117.7, 90.7)
- added Q5: RJU003N03 NMOS, Package_TO_SOT_SMD:SOT-323_SC-70, B.Cu at (194.9, 97.0)
- added Q7: RJU003N03 NMOS, Package_TO_SOT_SMD:SOT-323_SC-70, B.Cu at (274.2, 54.2)
- added R31: 20K, Resistor_SMD:R_0402_1005Metric, B.Cu at (129.8, 136.3)
- added R32: 1M, Resistor_SMD:R_0402_1005Metric, B.Cu at (128.7, 133.5)
- added R33: 1K, Resistor_SMD:R_0402_1005Metric, B.Cu at (129.4, 138.3)
- added R34: 1K, Resistor_SMD:R_0402_1005Metric, F.Cu at (220.5, 68.4)
- added R35: 1K, Resistor_SMD:R_0402_1005Metric, F.Cu at (223.4, 68.4)
- added R36: 1K, Resistor_SMD:R_0402_1005Metric, B.Cu at (129.9, 141.9)
- added R37: 10K, Resistor_SMD:R_0402_1005Metric, B.Cu at (117.4, 142.6)
- added R38: 10K, Resistor_SMD:R_0402_1005Metric, B.Cu at (117.4, 140.1)
- added R39: 10K, Resistor_SMD:R_0402_1005Metric, B.Cu at (121.4, 139.6)
- added R40: 4.7K, Resistor_SMD:R_0402_1005Metric, B.Cu at (117.4, 141.5)
- added R41: 4.7K, Resistor_SMD:R_0402_1005Metric, B.Cu at (117.4, 139.0)
- added R42: 4.7K, Resistor_SMD:R_0402_1005Metric, B.Cu at (120.3, 139.6)
- added R46: 1M, Resistor_SMD:R_0402_1005Metric, B.Cu at (162.2, 121.6)
- added R47: 1K, Resistor_SMD:R_0402_1005Metric, B.Cu at (157.9, 131.8)
- added R48: 10K, Resistor_SMD:R_0402_1005Metric, B.Cu at (156.9, 132.9)
- added R49: 33K, Resistor_SMD:R_0402_1005Metric, F.Cu at (200.1, 78.6)
- added R5: 1K, Resistor_SMD:R_0402_1005Metric, B.Cu at (161.0, 101.5)
- added R50: 33K, Resistor_SMD:R_0402_1005Metric, B.Cu at (196.9, 33.9)
- added R52: 10K, Resistor_SMD:R_0402_1005Metric, B.Cu at (192.3, 106.0)
- added R54: 10K, Resistor_SMD:R_0402_1005Metric, B.Cu at (192.3, 102.4)
- added U10: AMS1117-3.3, Package_TO_SOT_SMD:SOT-89-3, B.Cu at (118.9, 126.5)
- added U11: AT25DF161-SF-T, Package_SO:SO-8_3.9x4.9mm_P1.27mm, B.Cu at (118.4, 134.7)
- added U13: MCP2515-xST, Package_SO:TSSOP-20_4.4x6.5mm_P0.65mm, B.Cu at (160.3, 126.1)
- added U14: MCP2551-I-SN, Package_SO:SOIC-8_3.9x4.9mm_P1.27mm, B.Cu at (165.9, 108.1)
- added U15: 74HC4051BQ,115, Package_SO:TSSOP-16_4.4x5mm_P0.65mm, B.Cu at (127.9, 116.9)
- added U16: 74HC4051BQ,115, Package_SO:TSSOP-16_4.4x5mm_P0.65mm, B.Cu at (129.3, 105.2)
- added U9: ATmega128A-AU, Package_QFP:TQFP-64_14x14mm_P0.8mm, B.Cu at (139.3, 133.1)
- added Y3: 8 MHz, Crystal:Crystal_SMD_3225-4Pin_3.2x2.5mm, B.Cu at (126.2, 134.0)
- added Y4: 12MHz, Crystal:Crystal_SMD_3225-4Pin_3.2x2.5mm, B.Cu at (165.8, 126.1)
- moved J9 125.9 mm to (216.7, 69.7), turned to 0 degrees
- moved U4 64.7 mm to (206.7, 69.7), turned to 0 degrees
- moved C9 60.9 mm to (206.1, 73.0), turned to 0 degrees
- moved R_CSB1 58.3 mm to (201.4, 69.5)
- moved R23 53.0 mm to (203.2, 73.0)
Connections:
- net /Payload Power Control 0/CSENSE renamed /CSENSE
- net Net-(Q2-Pad2) renamed /PCH4
- C12 pad 1: +5V_A -> +5V
- C13 pad 1: +5V_A -> +5V
- C15 pad 1: +5V_A -> +5V
- C3 pad 1: +5V_A -> +5V
- C4 pad 1: +5V_A -> +5V
- C6 pad 1: +5V_A -> +5V
- C7 pad 1: +5V_A -> +5V
- C9 pad 1: +5V_A -> Net-(C9-Pad1)
- J4 pad 2: +5V_A -> +5V
- J5 pad 1: +5V_A -> +5V
- L1 pad 1: +5V_A -> +5V
- N1 pad 7: +5V_A -> +5V
- N2 pad 7: +5V_A -> +5V
- N3 pad 7: +5V_A -> +5V
- N4 pad 7: +5V_A -> +5V
- N5 pad 7: +5V_A -> +5V
- N6 pad 7: +5V_A -> +5V
- N7 pad 7: +5V_A -> +5V
- N8 pad 7: +5V_A -> +5V
- Q4 pad 2: +5V_A -> +5V
- Q6 pad 2: +5V_A -> +5V
- R11 pad 2: +5V_A -> +5V
- R23 pad 2: +5V -> GND
- R26 pad 1: +5V_A -> +5V
- R27 pad 1: +5V_A -> +5V
- R30 pad 1: +5V_A -> +5V
- R51 pad 2: +5V_A -> +5V
- R53 pad 2: +5V_A -> +5V
- R8 pad 1: +5V_A -> +5V
- R_CSB1 pad 1: +5V_A -> +5V
- U1 pad 21: +5V_A -> +5V
- U1 pad 52: +5V_A -> +5V
- U2 pad 3: +5V_A -> +5V
- U4 pad 3: +5V_A -> Net-(C9-Pad1)
- U4 pad 5: +5V_A -> +5V
- U5 pad 16: +5V_A -> +5V
- U5 pad 7: +5V_A -> +5V
- U6 pad 16: +5V_A -> +5V
- U6 pad 7: +5V_A -> +5V
- U7 pad 20: +5V_A -> +5V
- U8 pad 3: +5V_A -> +5V
- U8 pad 5: +5V_A -> +5V
Routing:
- net +5V_A: track 247.6 -> 0.00 mm, vias 31 -> 0
- net /CANBUS Controller 1/MOSI: track 0.00 -> 53.8 mm, vias 0 -> 2
- net /CANBUS Controller 1/SCK: track 0.00 -> 53.2 mm, vias 0 -> 2
- net /CANBUS Controller 1/MISO: track 0.00 -> 51.8 mm, vias 0 -> 2
- net /CSENSE: track 62.8 -> 11.7 mm, vias 2 -> 0
- net Net-(U13-Pad2): track 0.00 -> 50.8 mm, vias 0 -> 2
- net /N8_RST: track 0.00 -> 45.5 mm
- net /CANBUS Controller 1/MCP_TX0RTS: track 0.00 -> 43.8 mm, vias 0 -> 2
- net /CANBUS Controller 1/MCP_RX1BF: track 0.00 -> 34.5 mm
- net /N5_TX: track 34.2 -> 0.00 mm, vias 2 -> 0
- net /CANBUS Controller 1/CS: track 0.00 -> 33.6 mm, vias 0 -> 2
- net /CANBUS Controller 1/MCP_RESET: track 0.00 -> 33.2 mm, vias 0 -> 2
- net /Node RX MUX 1/A0: track 0.00 -> 32.4 mm, vias 0 -> 2
- net /CANBUS Controller 1/MCP_RX0BF: track 0.00 -> 31.8 mm
- net /N9_RST: track 0.00 -> 31.2 mm
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- removed copper zone on F.Cu, net +5V
- removed copper zone on F.Cu, net +5V_A
- removed copper zone on In1.Cu, net +5V_A
- removed copper zone on F.Cu, net /PCH4

Commit message: Bump
Parts:
- moved D9 1.43 mm to (167.3, 98.7), turned to -90 degrees
Routing:
- net /N8_PWR: track 0.00 -> 42.1 mm
- net /N9_RX: track 0.00 -> 37.6 mm, vias 0 -> 2
- net /N9_TX: track 0.00 -> 28.1 mm, vias 0 -> 2
- net /N8_RST: track 45.5 -> 46.4 mm

Commit message: Revision D1, board A0
Board initial release
Parts:
- removed D1: LED_PWON, LED_SMD:LED_0402_1005Metric
- removed R5: 1K, Resistor_SMD:R_0402_1005Metric
- J3: value PC/104 Connector -> Conn_02x32_Odd_Even
- R34, R35, R49: moved to B.Cu
- moved Q7 164.6 mm to (126.2, 126.2), turned to -90 degrees
- moved R35 132.7 mm to (95.2, 102.7), turned to 90 degrees
- moved R34 127.4 mm to (96.8, 98.8), turned to -90 degrees
- moved J9 125.9 mm to (94.6, 100.4), turned to 180 degrees
- moved R50 94.8 mm to (132.8, 103.8), turned to -90 degrees
- moved Q5 78.2 mm to (123.2, 128.1)
- moved R49 78.2 mm to (133.0, 118.6), turned to 90 degrees
- moved R52 71.8 mm to (123.2, 125.7), turned to 0 degrees
- moved R54 69.6 mm to (126.1, 123.8), turned to 0 degrees
- moved U4 61.9 mm to (165.4, 115.8), turned to 90 degrees
- moved R23 58.8 mm to (167.3, 119.5), turned to 180 degrees
- moved C9 57.9 mm to (167.8, 116.4), turned to 90 degrees
- moved D3 56.5 mm to (167.3, 118.4), turned to 180 degrees
- moved R_CSB1 55.5 mm to (165.4, 111.7)
- moved N14 18.4 mm to (161.5, 87.0)
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Connections:
- C9 pad 1: Net-(C9-Pad1) -> +5V
- D3 pad 2: Net-(C9-Pad1) -> +5V
- J3 pad 1: (no net) -> unconnected-(J3-Pad1)
- J3 pad 10: (no net) -> unconnected-(J3-Pad10)
- J3 pad 11: (no net) -> unconnected-(J3-Pad11)
- J3 pad 12: (no net) -> unconnected-(J3-Pad12)
- J3 pad 13: (no net) -> unconnected-(J3-Pad13)
- J3 pad 14: (no net) -> unconnected-(J3-Pad14)
- J3 pad 15: (no net) -> unconnected-(J3-Pad15)
- J3 pad 16: (no net) -> unconnected-(J3-Pad16)
- J3 pad 17: (no net) -> /PCH4
- J3 pad 18: (no net) -> /PCH4
- J3 pad 19: (no net) -> GND
- J3 pad 2: (no net) -> unconnected-(J3-Pad2)
- J3 pad 20: (no net) -> GND
- J3 pad 21: (no net) -> unconnected-(J3-Pad21)
- J3 pad 22: (no net) -> unconnected-(J3-Pad22)
- J3 pad 23: (no net) -> unconnected-(J3-Pad23)
- J3 pad 24: (no net) -> unconnected-(J3-Pad24)
- J3 pad 25: (no net) -> CANH
- J3 pad 26: (no net) -> CANL
- J3 pad 27: (no net) -> unconnected-(J3-Pad27)
- J3 pad 28: (no net) -> unconnected-(J3-Pad28)
- J3 pad 29: (no net) -> unconnected-(J3-Pad29)
- J3 pad 3: (no net) -> unconnected-(J3-Pad3)
- J3 pad 30: (no net) -> unconnected-(J3-Pad30)
- J3 pad 31: (no net) -> unconnected-(J3-Pad31)
- J3 pad 32: (no net) -> unconnected-(J3-Pad32)
- J3 pad 33: (no net) -> unconnected-(J3-Pad33)
- J3 pad 34: (no net) -> unconnected-(J3-Pad34)
- J3 pad 35: (no net) -> unconnected-(J3-Pad35)
- J3 pad 36: (no net) -> unconnected-(J3-Pad36)
- J3 pad 37: (no net) -> unconnected-(J3-Pad37)
- J3 pad 38: (no net) -> unconnected-(J3-Pad38)
- J3 pad 39: (no net) -> unconnected-(J3-Pad39)
- J3 pad 4: (no net) -> unconnected-(J3-Pad4)
- J3 pad 40: (no net) -> unconnected-(J3-Pad40)
- J3 pad 41: (no net) -> unconnected-(J3-Pad41)
- J3 pad 42: (no net) -> unconnected-(J3-Pad42)
- J3 pad 43: (no net) -> unconnected-(J3-Pad43)
- J3 pad 44: (no net) -> unconnected-(J3-Pad44)
- J3 pad 45: (no net) -> unconnected-(J3-Pad45)
- J3 pad 46: (no net) -> unconnected-(J3-Pad46)
- J3 pad 47: (no net) -> unconnected-(J3-Pad47)
- J3 pad 48: (no net) -> unconnected-(J3-Pad48)
- J3 pad 49: (no net) -> unconnected-(J3-Pad49)
- J3 pad 5: (no net) -> unconnected-(J3-Pad5)
- J3 pad 50: (no net) -> unconnected-(J3-Pad50)
- J3 pad 51: (no net) -> unconnected-(J3-Pad51)
- J3 pad 52: (no net) -> unconnected-(J3-Pad52)
- J3 pad 53: (no net) -> unconnected-(J3-Pad53)
- J3 pad 54: (no net) -> unconnected-(J3-Pad54)
- J3 pad 55: (no net) -> unconnected-(J3-Pad55)
- J3 pad 56: (no net) -> unconnected-(J3-Pad56)
- J3 pad 57: (no net) -> unconnected-(J3-Pad57)
- J3 pad 58: (no net) -> unconnected-(J3-Pad58)
- J3 pad 59: (no net) -> unconnected-(J3-Pad59)
- J3 pad 6: (no net) -> unconnected-(J3-Pad6)
- J3 pad 60: (no net) -> unconnected-(J3-Pad60)
- J3 pad 61: (no net) -> /CH_B
- J3 pad 62: (no net) -> /CH_A
- J3 pad 63: (no net) -> unconnected-(J3-Pad63)
- J3 pad 64: (no net) -> unconnected-(J3-Pad64)
- J3 pad 7: (no net) -> unconnected-(J3-Pad7)
- J3 pad 8: (no net) -> unconnected-(J3-Pad8)
- J3 pad 9: (no net) -> unconnected-(J3-Pad9)
- U15 pad 13: /N8_TX -> /N14_TX
- U15 pad 14: /N12_TX -> /N8_TX
- U15 pad 15: /N14_TX -> /N12_TX
- U16 pad 13: /N8_RX -> /N14_RX
- U16 pad 14: /N12_RX -> /N8_RX
- U16 pad 15: /N14_RX -> /N12_RX
- U4 pad 3: Net-(C9-Pad1) -> +5V
- U9 pad 37: /N14_PWR -> /N8_PWR
- U9 pad 38: /N14_RST -> /N8_RST
- U9 pad 39: /N8_RST -> /N14_RST
- U9 pad 40: /N8_PWR -> /N14_PWR
- U9 pad 41: /N12_PWR -> /N10_PWR
- U9 pad 42: /N12_RST -> /N10_RST
- U9 pad 44: /N10_RST -> /N11_RST
- U9 pad 45: /N10_PWR -> /N11_PWR
- U9 pad 46: /N11_RST -> /N12_RST
- U9 pad 47: /N11_PWR -> /N12_PWR
Routing:
- net /SCL: track 219.6 -> 441.0 mm
- net /SDA: track 201.3 -> 417.5 mm
- net /GEIGER_EN: track 17.8 -> 111.8 mm, vias 1 -> 2
- net /GEIGER_FET: track 32.8 -> 125.8 mm, vias 2 -> 4
- net Net-(R34-Pad2): track 0.00 -> 85.5 mm, vias 0 -> 2
- net Net-(R35-Pad1): track 0.00 -> 81.4 mm, vias 0 -> 2
- net /CSENSE: track 11.7 -> 91.9 mm, vias 0 -> 3
- net +5V: track 163.2 -> 232.2 mm, vias 11 -> 50
- net /N12_PWR: track 0.00 -> 59.9 mm
- net /N12_RST: track 0.00 -> 56.0 mm
- net /N13_TX: track 0.00 -> 52.5 mm, vias 0 -> 2
- net /N13_RST: track 0.00 -> 45.2 mm
- net /N15_RST: track 0.00 -> 44.5 mm
- net /N15_TX: track 0.00 -> 43.3 mm, vias 0 -> 2
- net /N15_PWR: track 0.00 -> 43.1 mm
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- added copper zone on F.Cu, net +5V
- added copper zone on In2.Cu, net +5V
- added copper zone on F.Cu, net /PCH4
- added copper zone on B.Cu, net GND
Other:
- board text added: "*"
- board text added: "*JTAG"
- board text added: "+5V"
- board text added: "CANBUS 0"
- board text added: "CANBUS 1"
- board text added: "CSENSE"
- board text added: "Designed by: ThePetrovich"
- board text added: "Flash 1"
- board text added: "GeigerBoard Mount"
- board text added: "J4 1W +5V GND"
- board text added: "J5 SDA GND SCL +5V"
- board text added: "J7 S0_RX GND S0_TX"
- board text added: "J9 S1_RX GND S1_TX"
- board text added: "MISO SCK RESET"
- board text added: "NC MOSI GND"
- board text added: "NC SI GND"
- board text added: "QC"
- board text added: "Revision A0"
- board text added: "S1 ISP"
- board text added: "SN:"
- board text added: "SO SCK RST"
- board text added: "Sakha Aerospace Systems, LLC"
- board text added: "Supervisor 1"
- board text added: "UART MUX 0"
- board text added: "UART MUX 1"
- board text added: "Verified by: nyakotronics"

Commit message: Fix RXCAN and TXCAN connection
Routing:
- net (no net): vias 2 -> 0
Changed lines of the file:
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@@
     (style (thickness 0.1) (arrow_length 1.27) (text_position_mode 0) (extension_height 0.58642) (extension_offset 0.5) keep_text_aligned)
   )
-  (via (at 189.738 90.678) (size 0.6) (drill 0.3) (layers "F.Cu" "B.Cu") (free) (net 0))
-  (via (at 74.295 113.792) (size 0.6) (drill 0.3) (layers "F.Cu" "B.Cu") (free) (net 0))
   (segment (start 145.114 79.635) (end 146.707 79.635) (width 0.25) (layer "F.Cu") (net 1))
   (segment (start 161.456 77.681) (end 161.456 78.878) (width 0.25) (layer "F.Cu") (net 1))
