File: ykts-payload/ykts-payload — копия.kicad_pcb (KiCad board)
At the start: 4 copper layers, 95.9 x 90.2 mm, 167 parts, among them J1 DBG_PWR, J2 GeigerBoard, J3 PC/104 Connector, J4 Solar_Temp, J5 Sensor_Ext, J6 Conn_02x03_Odd_Even, J7 Conn_01x03_Male, J8 Conn_02x03_Odd_Even, J9 Conn_01x03_Male, Q1 PMV65XP, Q2 PMV65XP, Q3 PMV65XP, Q4 RJU003N03 NMOS, Q5 RJU003N03 NMOS, Q6 RJU003N03 NMOS, Q7 RJU003N03 NMOS, U1 ATmega128A-AU, U10 AMS1117-3.3, U11 AT25DF161-SF-T, U12 MAX4372FEUK, U13 MCP2515-xST, U14 MCP2551-I-SN, U15 74HC4051BQ,115, U16 74HC4051BQ,115, U2 AMS1117-3.3, U3 AT25DF161-SF-T, U4 MAX4372FEUK, U5 74HC4051BQ,115, U6 74HC4051BQ,115, U7 MCP2515-xST, U8 MCP2551-I-SN, U9 ATmega128A-AU, Y1 8 MHz, Y2 12MHz, Y3 8 MHz, Y4 12MHz

Commit message: Revision D0
Parts:
- moved J4 133.8 mm to (20.1, 65.9)
- moved Q7 133.8 mm to (75.2, 74.7)
- moved R3 133.8 mm to (18.1, 79.8)
- moved R4 133.8 mm to (56.7, 61.6)
- moved R52 133.8 mm to (79.0, 85.0)
- moved R54 133.8 mm to (78.9, 73.9)
- moved Q5 133.8 mm to (70.7, 78.4)
- moved D3 106.1 mm to (260.5, 79.0)
- moved J1 106.1 mm to (225.4, 43.3)
- moved R45 106.1 mm to (236.7, 52.1)
- moved R6 106.1 mm to (202.3, 74.2)
- moved R7 106.1 mm to (202.3, 75.6)
- moved U15 106.1 mm to (190.9, 45.6)
- moved D1 106.1 mm to (211.7, 72.3)
- moved R1 106.1 mm to (210.2, 67.4)
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Connections:
- U1 pad 29: /Node RX MUX 0/A2 -> /Node RX MUX 0/A0
- U1 pad 31: /Node RX MUX 0/A0 -> /Node RX MUX 0/A2
- U9 pad 29: /Node RX MUX 1/A2 -> /Node RX MUX 1/A0
- U9 pad 31: /Node RX MUX 1/A0 -> /Node RX MUX 1/A2
Routing:
- net /Node TX MUX 0/IN: track 0.00 -> 38.4 mm, vias 0 -> 2
- net /N3_RX: track 0.00 -> 32.7 mm
- net /Node RX MUX 0/A0: track 0.00 -> 32.4 mm, vias 0 -> 2
- net /Node RX MUX 0/A1: track 0.00 -> 31.1 mm, vias 0 -> 2
- net /Node RX MUX 0/A2: track 0.00 -> 29.8 mm, vias 0 -> 2
- net /Node RX MUX 0/IN: track 0.00 -> 25.2 mm, vias 0 -> 2
- net /CANBUS Controller 0/MISO: track 27.7 -> 48.3 mm
- net /CANBUS Controller 0/SCK: track 29.4 -> 49.6 mm
- net /CANBUS Controller 0/MOSI: track 28.9 -> 48.9 mm
- net +5V_B: track 31.1 -> 49.1 mm, vias 0 -> 2
- net Net-(U7-Pad2): track 0.00 -> 16.7 mm
- net /N2_RX: track 0.00 -> 15.2 mm
- net /Payload Supervisor 0/SD_CS: track 0.00 -> 15.1 mm
- net Net-(U7-Pad1): track 0.00 -> 13.5 mm
- net Net-(CL3-Pad1): track 0.00 -> 10.2 mm
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