File: ykts-payload/ykts-payload-pwr.kicad_sch (KiCad schematic)
At the start: 8 parts, among them Q3 PMV65XP, U12 MAX4372FEUK

Commit message: Bump board
Parts:
- renumbered C24 to C9, D7 to D3, Q3 to Q2, R43 to R23, R44 to R24, R45 to R25, R_CSB2 to R_CSB1, U12 to U4
Changed lines of the file:
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@@
   (symbol (lib_id "yktsat-common:MAX4372FEUK") (at 137.16 104.14 0)
     (in_bom yes) (on_board yes)
-    (property "Reference" "U12" (id 0) (at 137.16 96.1136 0))
+    (property "Reference" "U4" (id 0) (at 137.16 96.1136 0))
     (property "Value" "MAX4372FEUK" (id 1) (at 137.16 98.425 0))
     (property "Footprint" "Package_TO_SOT_SMD:SOT-23-5" (id 2) (at 137.16 104.14 0)
@@
   (symbol (lib_id "Device:C_Small") (at 153.67 111.76 0)
     (in_bom yes) (on_board yes)
-    (property "Reference" "C24" (id 0) (at 156.0068 110.5916 0)
+    (property "Reference" "C9" (id 0) (at 156.0068 110.5916 0)
       (effects (font (size 1.27 1.27)) (justify left))
     )
@@
   (symbol (lib_id "Device:R_Small") (at 118.11 107.95 180)
     (in_bom yes) (on_board yes)
-    (property "Reference" "R_CSB2" (id 0) (at 123.0884 107.95 90))
+    (property "Reference" "R_CSB1" (id 0) (at 123.0884 107.95 90))
     (property "Value" "0.1" (id 1) (at 120.777 107.95 90))
     (property "Footprint" "Resistor_SMD:R_1210_3225Metric" (id 2) (at 118.11 107.95 0)
@@
   (symbol (lib_id "Device:R_Small") (at 106.68 85.09 180)
     (in_bom yes) (on_board yes)
-    (property "Reference" "R43" (id 0) (at 111.6584 85.09 90))
+    (property "Reference" "R23" (id 0) (at 111.6584 85.09 90))
     (property "Value" "1K" (id 1) (at 109.347 85.09 90))
     (property "Footprint" "Resistor_SMD:R_0402_1005Metric" (id 2) (at 106.68 85.09 0)
@@
   (symbol (lib_id "Device:R_Small") (at 106.68 95.25 0) (mirror x)
     (in_bom yes) (on_board yes)
-    (property "Reference" "R44" (id 0) (at 111.6584 95.25 90))
+    (property "Reference" "R24" (id 0) (at 111.6584 95.25 90))
     (property "Value" "10K" (id 1) (at 109.347 95.25 90))
     (property "Footprint" "Resistor_SMD:R_0402_1005Metric" (id 2) (at 106.68 95.25 0)
@@
   (symbol (lib_id "Device:Q_PMOS_GDS") (at 115.57 90.17 0) (mirror x)
     (in_bom yes) (on_board yes)
-    (property "Reference" "Q3" (id 0) (at 120.777 89.0016 0)
+    (property "Reference" "Q2" (id 0) (at 120.777 89.0016 0)
       (effects (font (size 1.27 1.27)) (justify left))
     )
@@
   (symbol (lib_id "Device:LED") (at 180.34 93.98 180)
     (in_bom yes) (on_board yes)
-    (property "Reference" "D7" (id 0) (at 179.3494 90.9828 90)
+    (property "Reference" "D3" (id 0) (at 179.3494 90.9828 90)
       (effects (font (size 1.27 1.27)) (justify right))
     )
@@
   (symbol (lib_id "Device:R_Small") (at 189.23 93.98 90) (mirror x)
     (in_bom yes) (on_board yes)
-    (property "Reference" "R45" (id 0) (at 189.23 89.0016 90))
+    (property "Reference" "R25" (id 0) (at 189.23 89.0016 90))
     (property "Value" "1K" (id 1) (at 189.23 91.313 90))
     (property "Footprint" "Resistor_SMD:R_0402_1005Metric" (id 2) (at 189.23 93.98 0)
