File: ykts-payload/ykts-payload-bak3.kicad_pcb (KiCad board)
At the start: 4 copper layers, 95.9 x 90.2 mm, 154 parts, among them J1 DBG_PWR, J2 GeigerBoard, J3 Conn_02x32_Odd_Even, J4 Solar_Temp, J5 Sensor_Ext, J6 Conn_02x03_Odd_Even, J7 Conn_01x03_Male, J8 Conn_02x03_Odd_Even, J9 Conn_01x03_Male, Q1 PMV65XP, Q4 RJU003N03 NMOS, Q5 RJU003N03 NMOS, Q6 RJU003N03 NMOS, Q7 RJU003N03 NMOS, U1 ATmega128A-AU, U10 AMS1117-3.3, U11 AT25DF161-SF-T, U13 MCP2515-xST, U14 MCP2551-I-SN, U15 74HC4051BQ,115, U16 74HC4051BQ,115, U2 AMS1117-3.3, U3 AT25DF161-SF-T, U4 MAX4372FEUK, U5 74HC4051BQ,115, U6 74HC4051BQ,115, U7 MCP2515-xST, U8 MCP2551-I-SN, U9 ATmega128A-AU, Y1 8 MHz, Y2 12MHz, Y3 8 MHz, Y4 12MHz

Commit message: Bump version
Connections:
- U14 pad 1: Net-(U13-Pad1) -> Net-(U13-Pad2)
- U14 pad 4: Net-(U13-Pad2) -> Net-(U13-Pad1)
- U8 pad 1: Net-(U7-Pad1) -> Net-(U7-Pad2)
- U8 pad 4: Net-(U7-Pad2) -> Net-(U7-Pad1)
Routing:
- net Net-(U13-Pad1): track 18.6 -> 15.3 mm
- net Net-(U7-Pad2): track 15.0 -> 17.6 mm
- net Net-(U7-Pad1): track 17.7 -> 15.3 mm, vias 2 -> 0
- net Net-(U13-Pad2): track 15.9 -> 17.5 mm, vias 2 -> 0
Changed lines of the file:
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@@
     (fp_line (start 1.95 -2.45) (end 1.95 2.45) (layer "F.Fab") (width 0.1))
     (pad "1" smd roundrect locked (at -2.475 -1.905 270) (size 1.95 0.6) (layers "F.Cu" "F.Paste" "F.Mask") (roundrect_rratio 0.25)
-      (net 89 "Net-(U7-Pad1)") (pinfunction "TXD") (pintype "input"))
+      (net 88 "Net-(U7-Pad2)") (pinfunction "TXD") (pintype "input"))
     (pad "2" smd roundrect locked (at -2.475 -0.635 270) (size 1.95 0.6) (layers "F.Cu" "F.Paste" "F.Mask") (roundrect_rratio 0.25)
       (net 1 "GND") (pinfunction "VSS") (pintype "power_in"))
@@
       (net 2 "+5V") (pinfunction "VDD") (pintype "power_in"))
     (pad "4" smd roundrect locked (at -2.475 1.905 270) (size 1.95 0.6) (layers "F.Cu" "F.Paste" "F.Mask") (roundrect_rratio 0.25)
-      (net 88 "Net-(U7-Pad2)") (pinfunction "RXD") (pintype "output"))
+      (net 89 "Net-(U7-Pad1)") (pinfunction "RXD") (pintype "output"))
     (pad "5" smd roundrect locked (at 2.475 1.905 270) (size 1.95 0.6) (layers "F.Cu" "F.Paste" "F.Mask") (roundrect_rratio 0.25)
       (net 2 "+5V") (pinfunction "Vref") (pintype "power_out"))
@@
     (fp_line (start -0.975 2.45) (end 1.95 2.45) (layer "B.Fab") (width 0.1))
     (pad "1" smd roundrect locked (at -2.475 1.905 90) (size 1.95 0.6) (layers "B.Cu" "B.Paste" "B.Mask") (roundrect_rratio 0.25)
-      (net 199 "Net-(U13-Pad1)") (pinfunction "TXD") (pintype "input"))
+      (net 200 "Net-(U13-Pad2)") (pinfunction "TXD") (pintype "input"))
     (pad "2" smd roundrect locked (at -2.475 0.635 90) (size 1.95 0.6) (layers "B.Cu" "B.Paste" "B.Mask") (roundrect_rratio 0.25)
       (net 1 "GND") (pinfunction "VSS") (pintype "power_in"))
@@
       (net 2 "+5V") (pinfunction "VDD") (pintype "power_in"))
     (pad "4" smd roundrect locked (at -2.475 -1.905 90) (size 1.95 0.6) (layers "B.Cu" "B.Paste" "B.Mask") (roundrect_rratio 0.25)
-      (net 200 "Net-(U13-Pad2)") (pinfunction "RXD") (pintype "output"))
+      (net 199 "Net-(U13-Pad1)") (pinfunction "RXD") (pintype "output"))
     (pad "5" smd roundrect locked (at 2.475 -1.905 90) (size 1.95 0.6) (layers "B.Cu" "B.Paste" "B.Mask") (roundrect_rratio 0.25)
       (net 2 "+5V") (pinfunction "Vref") (pintype "power_out"))
@@
   )
   (gr_line (start 113.411 142.748) (end 113.411 143.256) (layer "B.SilkS") (width 0.12))
+  (gr_line (start 121.539 143.256) (end 122.174 142.748) (layer "B.SilkS") (width 0.12))
   (gr_line (start 121.3485 137.0965) (end 121.7295 136.7155) (layer "B.SilkS") (width 0.12))
   (gr_line (start 170.688 144.907) (end 172.085 144.907) (layer "B.SilkS") (width 0.12))
@@
       (xy 170.688 96.52)
     ) (layer "B.SilkS") (width 0.12) (fill none))
-  (gr_line (start 121.539 143.256) (end 122.174 142.748) (layer "B.SilkS") (width 0.12))
   (gr_line (start 156.591 123.063) (end 156.21 122.682) (layer "B.SilkS") (width 0.12))
   (gr_line (start 168.148 112.776) (end 167.767 112.395) (layer "B.SilkS") (width 0.12))
@@
   (segment (start 154.942 72.515) (end 154.942 70.866) (width 0.25) (layer "F.Cu") (net 87))
   (segment (start 154.57 73.7185) (end 154.57 72.887) (width 0.25) (layer "F.Cu") (net 87))
-  (segment (start 158.252489 85.481489) (end 160.528 87.757) (width 0.25) (layer "F.Cu") (net 88))
-  (segment (start 154.57 80.275) (end 158.252489 83.957489) (width 0.25) (layer "F.Cu") (net 88))
-  (segment (start 154.57 79.4435) (end 154.57 80.275) (width 0.25) (layer "F.Cu") (net 88))
-  (segment (start 160.528 87.757) (end 160.528 92.013) (width 0.25) (layer "F.Cu") (net 88))
-  (segment (start 158.252489 83.957489) (end 158.252489 85.481489) (width 0.25) (layer "F.Cu") (net 88))
-  (segment (start 164.338 90.043) (end 164.338 92.013) (width 0.25) (layer "F.Cu") (net 89))
-  (segment (start 153.92 80.508178) (end 157.482911 84.071089) (width 0.25) (layer "F.Cu") (net 89))
-  (segment (start 153.92 79.4435) (end 153.92 80.508178) (width 0.25) (layer "F.Cu") (net 89))
-  (via (at 164.338 90.043) (size 0.6) (drill 0.3) (layers "F.Cu" "B.Cu") (net 89))
-  (via (at 157.482911 84.071089) (size 0.6) (drill 0.3) (layers "F.Cu" "B.Cu") (net 89))
-  (segment (start 164.338 89.667807) (end 164.338 90.043) (width 0.25) (layer "In1.Cu") (net 89))
-  (segment (start 161.285318 88.000511) (end 162.670704 88.000511) (width 0.25) (layer "In1.Cu") (net 89))
-  (segment (start 157.482911 84.071089) (end 157.482911 84.198104) (width 0.25) (layer "In1.Cu") (net 89))
-  (segment (start 157.482911 84.198104) (end 161.285318 88.000511) (width 0.25) (layer "In1.Cu") (net 89))
-  (segment (start 162.670704 88.000511) (end 164.338 89.667807) (width 0.25) (layer "In1.Cu") (net 89))
+  (segment (start 157.216229 83.174511) (end 154.57 80.528282) (width 0.25) (layer "F.Cu") (net 88))
+  (segment (start 158.866511 83.174511) (end 157.216229 83.174511) (width 0.25) (layer "F.Cu") (net 88))
+  (segment (start 164.338 88.646) (end 158.866511 83.174511) (width 0.25) (layer "F.Cu") (net 88))
+  (segment (start 164.338 92.013) (end 164.338 88.646) (width 0.25) (layer "F.Cu") (net 88))
+  (segment (start 154.57 80.528282) (end 154.57 79.4435) (width 0.25) (layer "F.Cu") (net 88))
+  (segment (start 153.92 80.514) (end 160.528 87.122) (width 0.25) (layer "F.Cu") (net 89))
+  (segment (start 160.528 87.122) (end 160.528 92.013) (width 0.25) (layer "F.Cu") (net 89))
+  (segment (start 153.92 79.4435) (end 153.92 80.514) (width 0.25) (layer "F.Cu") (net 89))
   (segment (start 129.759 72.39) (end 129.714 72.435) (width 0.25) (layer "F.Cu") (net 110))
   (segment (start 131.064 72.39) (end 129.759 72.39) (width 0.25) (layer "F.Cu") (net 110))
@@
   (segment (start 125.0265 117.8658) (end 125.714364 117.8658) (width 0.25) (layer "B.Cu") (net 187))
   (segment (start 125.714364 117.8658) (end 126.53276 117.047404) (width 0.25) (layer "B.Cu") (net 187))
-  (segment (start 157.42 121.726) (end 157.42 123.1925) (width 0.25) (layer "B.Cu") (net 199))
-  (segment (start 163.555872 118.491) (end 160.655 118.491) (width 0.25) (layer "B.Cu") (net 199))
-  (segment (start 167.838 110.623) (end 167.838 114.208872) (width 0.25) (layer "B.Cu") (net 199))
-  (segment (start 160.655 118.491) (end 157.42 121.726) (width 0.25) (layer "B.Cu") (net 199))
-  (segment (start 167.838 114.208872) (end 163.555872 118.491) (width 0.25) (layer "B.Cu") (net 199))
-  (via (at 161.544 119.126) (size 0.6) (drill 0.3) (layers "F.Cu" "B.Cu") (net 200))
-  (via (at 163.314847 117.848847) (size 0.6) (drill 0.3) (layers "F.Cu" "B.Cu") (net 200))
-  (segment (start 163.314847 117.863153) (end 162.052 119.126) (width 0.25) (layer "In2.Cu") (net 200))
-  (segment (start 162.052 119.126) (end 161.544 119.126) (width 0.25) (layer "In2.Cu") (net 200))
-  (segment (start 163.314847 117.848847) (end 163.314847 117.863153) (width 0.25) (layer "In2.Cu") (net 200))
-  (segment (start 164.028 110.623) (end 164.028 117.135694) (width 0.25) (layer "B.Cu") (net 200))
-  (segment (start 161.544 119.126) (end 160.655718 119.126) (width 0.25) (layer "B.Cu") (net 200))
-  (segment (start 158.07 121.711718) (end 158.07 123.1925) (width 0.25) (layer "B.Cu") (net 200))
-  (segment (start 164.028 117.135694) (end 163.314847 117.848847) (width 0.25) (layer "B.Cu") (net 200))
-  (segment (start 160.655718 119.126) (end 158.07 121.711718) (width 0.25) (layer "B.Cu") (net 200))
+  (segment (start 164.028 115.601089) (end 164.028 110.623) (width 0.25) (layer "B.Cu") (net 199))
+  (segment (start 157.42 123.1925) (end 157.42 122.209089) (width 0.25) (layer "B.Cu") (net 199))
+  (segment (start 157.42 122.209089) (end 164.028 115.601089) (width 0.25) (layer "B.Cu") (net 199))
+  (segment (start 167.838 110.623) (end 167.838 114.026404) (width 0.25) (layer "B.Cu") (net 200))
+  (segment (start 166.664915 115.199489) (end 165.080997 115.199489) (width 0.25) (layer "B.Cu") (net 200))
+  (segment (start 165.080997 115.199489) (end 158.07 122.210486) (width 0.25) (layer "B.Cu") (net 200))
+  (segment (start 167.838 114.026404) (end 166.664915 115.199489) (width 0.25) (layer "B.Cu") (net 200))
+  (segment (start 158.07 122.210486) (end 158.07 123.1925) (width 0.25) (layer "B.Cu") (net 200))
   (segment (start 166.304 114.724) (end 166.304 112.0685) (width 0.25) (layer "F.Cu") (net 206))
   (segment (start 166.304 112.0685) (end 166.6975 111.675) (width 0.25) (layer "F.Cu") (net 206))
