File: ykts-payload/ykts-canbus.kicad_sch (KiCad schematic)
At the start: 19 parts, among them U13 MCP2515-xST, U14 MCP2551-I-SN, Y4 12MHz

Commit message: Bump
Parts:
- renumbered C25 to C10, C26 to C11, C27 to C12, C28 to C13, C29 to C14, C30 to C15, CH3 to CH1, CH4 to CH2, CL3 to CL1, CL4 to CL2, D8 to D4, D9 to D5, FL2 to FL1, R46 to R28, R47 to R29, R48 to R30, U13 to U7, U14 to U8, Y4 to Y2
Changed lines of the file:
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@@
   (symbol (lib_id "power:GND") (at 146.05 134.62 0)
     (in_bom yes) (on_board yes)
-    (property "Reference" "#PWR0110" (id 0) (at 146.05 140.97 0)
+    (property "Reference" "#PWR083" (id 0) (at 146.05 140.97 0)
       (effects (font (size 1.27 1.27)) hide)
     )
@@
   (symbol (lib_id "Device:C_Small") (at 146.05 129.54 0)
     (in_bom yes) (on_board yes)
-    (property "Reference" "C29" (id 0) (at 148.3868 128.3716 0)
+    (property "Reference" "C14" (id 0) (at 148.3868 128.3716 0)
       (effects (font (size 1.27 1.27)) (justify left))
     )
@@
   (symbol (lib_id "Device:R_Small") (at 146.05 119.38 0)
     (in_bom yes) (on_board yes)
-    (property "Reference" "R48" (id 0) (at 147.5486 118.2116 0)
+    (property "Reference" "R30" (id 0) (at 147.5486 118.2116 0)
       (effects (font (size 1.27 1.27)) (justify left))
     )
@@
   (symbol (lib_id "Device:R_Small") (at 140.97 124.46 270)
     (in_bom yes) (on_board yes)
-    (property "Reference" "R47" (id 0) (at 140.97 119.4816 90))
+    (property "Reference" "R29" (id 0) (at 140.97 119.4816 90))
     (property "Value" "1K" (id 1) (at 140.97 121.793 90))
     (property "Footprint" "Resistor_SMD:R_0402_1005Metric" (id 2) (at 140.97 124.46 0)
@@
   (symbol (lib_id "power:GND") (at 152.4 107.95 0)
     (in_bom yes) (on_board yes)
-    (property "Reference" "#PWR0111" (id 0) (at 152.4 114.3 0)
+    (property "Reference" "#PWR084" (id 0) (at 152.4 114.3 0)
       (effects (font (size 1.27 1.27)) hide)
     )
@@
   (symbol (lib_id "power:GND") (at 99.06 127 0)
     (in_bom yes) (on_board yes)
-    (property "Reference" "#PWR0108" (id 0) (at 99.06 133.35 0)
+    (property "Reference" "#PWR081" (id 0) (at 99.06 133.35 0)
       (effects (font (size 1.27 1.27)) hide)
     )
@@
   (symbol (lib_id "power:GND") (at 165.1 83.82 0)
     (in_bom yes) (on_board yes)
-    (property "Reference" "#PWR0112" (id 0) (at 165.1 90.17 0)
+    (property "Reference" "#PWR085" (id 0) (at 165.1 90.17 0)
       (effects (font (size 1.27 1.27)) hide)
     )
@@
   (symbol (lib_id "Device:C_Small") (at 165.1 78.74 0)
     (in_bom yes) (on_board yes)
-    (property "Reference" "C30" (id 0) (at 167.4368 77.5716 0)
+    (property "Reference" "C15" (id 0) (at 167.4368 77.5716 0)
       (effects (font (size 1.27 1.27)) (justify left))
     )
@@
   (symbol (lib_id "power:GND") (at 115.57 83.82 0)
     (in_bom yes) (on_board yes)
-    (property "Reference" "#PWR0109" (id 0) (at 115.57 90.17 0)
+    (property "Reference" "#PWR082" (id 0) (at 115.57 90.17 0)
       (effects (font (size 1.27 1.27)) hide)
     )
@@
   (symbol (lib_id "Device:C_Small") (at 110.49 78.74 0)
     (in_bom yes) (on_board yes)
-    (property "Reference" "C27" (id 0) (at 112.8268 77.5716 0)
+    (property "Reference" "C12" (id 0) (at 112.8268 77.5716 0)
       (effects (font (size 1.27 1.27)) (justify left))
     )
@@
   (symbol (lib_id "Device:C_Small") (at 57.15 106.68 270)
     (in_bom yes) (on_board yes)
-    (property "Reference" "C25" (id 0) (at 58.42 100.33 0)
+    (property "Reference" "C10" (id 0) (at 58.42 100.33 0)
       (effects (font (size 1.27 1.27)) (justify left))
     )
@@
   (symbol (lib_id "Device:CP1_Small") (at 120.65 78.74 0)
     (in_bom yes) (on_board yes)
-    (property "Reference" "C28" (id 0) (at 122.9614 77.5716 0)
+    (property "Reference" "C13" (id 0) (at 122.9614 77.5716 0)
       (effects (font (size 1.27 1.27)) (justify left))
     )
@@
   (symbol (lib_id "Device:C_Small") (at 57.15 116.84 270)
     (in_bom yes) (on_board yes)
-    (property "Reference" "C26" (id 0) (at 58.42 120.65 0)
+    (property "Reference" "C11" (id 0) (at 58.42 120.65 0)
       (effects (font (size 1.27 1.27)) (justify left))
     )
@@
   (symbol (lib_id "power:GND") (at 49.53 120.65 0)
     (in_bom yes) (on_board yes)
-    (property "Reference" "#PWR0105" (id 0) (at 49.53 127 0)
+    (property "Reference" "#PWR078" (id 0) (at 49.53 127 0)
       (effects (font (size 1.27 1.27)) hide)
     )
@@
   (symbol (lib_id "Interface_CAN_LIN:MCP2515-xST") (at 99.06 105.41 0)
     (in_bom yes) (on_board yes)
-    (property "Reference" "U13" (id 0) (at 99.06 80.4926 0))
+    (property "Reference" "U7" (id 0) (at 99.06 80.4926 0))
     (property "Value" "MCP2515-xST" (id 1) (at 99.06 82.804 0))
     (property "Footprint" "Package_SO:TSSOP-20_4.4x6.5mm_P0.65mm" (id 2) (at 99.06 128.27 0)
@@
   (symbol (lib_id "Device:Crystal_GND24_Small") (at 64.77 111.76 90)
     (in_bom yes) (on_board yes)
-    (property "Reference" "Y4" (id 0) (at 63.5 105.41 0)
+    (property "Reference" "Y2" (id 0) (at 63.5 105.41 0)
       (effects (font (size 1.27 1.27)) (justify left))
     )
@@
   (symbol (lib_id "power:GND") (at 62.23 111.76 270)
     (in_bom yes) (on_board yes)
-    (property "Reference" "#PWR0106" (id 0) (at 55.88 111.76 0)
+    (property "Reference" "#PWR079" (id 0) (at 55.88 111.76 0)
       (effects (font (size 1.27 1.27)) hide)
     )
@@
   (symbol (lib_id "power:GND") (at 67.31 111.76 90)
     (in_bom yes) (on_board yes)
-    (property "Reference" "#PWR0107" (id 0) (at 73.66 111.76 0)
+    (property "Reference" "#PWR080" (id 0) (at 73.66 111.76 0)
       (effects (font (size 1.27 1.27)) hide)
     )
@@
   (symbol (lib_id "Device:EMI_Filter_CommonMode") (at 191.77 95.25 0)
     (in_bom yes) (on_board yes)
-    (property "Reference" "FL2" (id 0) (at 191.77 88.1126 0))
+    (property "Reference" "FL1" (id 0) (at 191.77 88.1126 0))
     (property "Value" "DLW21SN921SK2" (id 1) (at 191.77 90.424 0))
     (property "Footprint" "Inductor_SMD:L_CommonModeChoke_Coilcraft_0805USB" (id 2) (at 191.77 94.234 0)
@@
   (symbol (lib_id "Device:C_Small") (at 172.72 104.14 0)
     (in_bom yes) (on_board yes)
-    (property "Reference" "CH3" (id 0) (at 175.0568 102.9716 0)
+    (property "Reference" "CH1" (id 0) (at 175.0568 102.9716 0)
       (effects (font (size 1.27 1.27)) (justify left))
     )
@@
   (symbol (lib_id "Device:C_Small") (at 182.88 104.14 0)
     (in_bom yes) (on_board yes)
-    (property "Reference" "CL3" (id 0) (at 185.2168 102.9716 0)
+    (property "Reference" "CL1" (id 0) (at 185.2168 102.9716 0)
       (effects (font (size 1.27 1.27)) (justify left))
     )
@@
   (symbol (lib_id "power:GND") (at 177.8 110.49 0)
     (in_bom yes) (on_board yes)
-    (property "Reference" "#PWR0113" (id 0) (at 177.8 116.84 0)
+    (property "Reference" "#PWR086" (id 0) (at 177.8 116.84 0)
       (effects (font (size 1.27 1.27)) hide)
     )
@@
   (symbol (lib_id "Device:D_TVS") (at 220.98 104.14 270)
     (in_bom yes) (on_board yes)
-    (property "Reference" "D8" (id 0) (at 223.012 102.9716 90)
+    (property "Reference" "D4" (id 0) (at 223.012 102.9716 90)
       (effects (font (size 1.27 1.27)) (justify left))
     )
@@
   (symbol (lib_id "power:GND") (at 226.06 110.49 0)
     (in_bom yes) (on_board yes)
-    (property "Reference" "#PWR0115" (id 0) (at 226.06 116.84 0)
+    (property "Reference" "#PWR088" (id 0) (at 226.06 116.84 0)
       (effects (font (size 1.27 1.27)) hide)
     )
@@
   (symbol (lib_id "Device:C_Small") (at 199.39 104.14 0)
     (in_bom yes) (on_board yes)
-    (property "Reference" "CH4" (id 0) (at 201.7268 102.9716 0)
+    (property "Reference" "CH2" (id 0) (at 201.7268 102.9716 0)
       (effects (font (size 1.27 1.27)) (justify left))
     )
@@
   (symbol (lib_id "Device:C_Small") (at 209.55 104.14 0)
     (in_bom yes) (on_board yes)
-    (property "Reference" "CL4" (id 0) (at 211.8868 102.9716 0)
+    (property "Reference" "CL2" (id 0) (at 211.8868 102.9716 0)
       (effects (font (size 1.27 1.27)) (justify left))
     )
@@
   (symbol (lib_id "power:GND") (at 204.47 110.49 0)
     (in_bom yes) (on_board yes)
-    (property "Reference" "#PWR0114" (id 0) (at 204.47 116.84 0)
+    (property "Reference" "#PWR087" (id 0) (at 204.47 116.84 0)
       (effects (font (size 1.27 1.27)) hide)
     )
@@
   (symbol (lib_id "Device:D_TVS") (at 231.14 104.14 270)
     (in_bom yes) (on_board yes)
-    (property "Reference" "D9" (id 0) (at 233.172 102.9716 90)
+    (property "Reference" "D5" (id 0) (at 233.172 102.9716 90)
       (effects (font (size 1.27 1.27)) (justify left))
     )
@@
   (symbol (lib_id "Device:R_Small") (at 74.93 111.76 180)
     (in_bom yes) (on_board yes)
-    (property "Reference" "R46" (id 0) (at 79.9084 111.76 90))
+    (property "Reference" "R28" (id 0) (at 79.9084 111.76 90))
     (property "Value" "1M" (id 1) (at 77.597 111.76 90))
     (property "Footprint" "Resistor_SMD:R_0402_1005Metric" (id 2) (at 74.93 111.76 0)
@@
   (symbol (lib_id "Interface_CAN_LIN:MCP2551-I-SN") (at 152.4 95.25 0)
     (in_bom yes) (on_board yes)
-    (property "Reference" "U14" (id 0) (at 152.4 80.4926 0))
+    (property "Reference" "U8" (id 0) (at 152.4 80.4926 0))
     (property "Value" "MCP2551-I-SN" (id 1) (at 152.4 82.804 0))
     (property "Footprint" "Package_SO:SOIC-8_3.9x4.9mm_P1.27mm" (id 2) (at 152.4 107.95 0)

Commit message: Rework power supply
Changed lines of the file:
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@@
     (in_bom yes) (on_board yes)
     (property "Reference" "R28" (id 0) (at 79.9084 111.76 90))
-    (property "Value" "1M" (id 1) (at 77.597 111.76 90))
+    (property "Value" "1M" (id 1) (at 77.47 111.76 90))
     (property "Footprint" "Resistor_SMD:R_0402_1005Metric" (id 2) (at 74.93 111.76 0)
       (effects (font (size 1.27 1.27)) hide)

Commit message: Bump
Parts:
- renumbered C10 to C25, C11 to C26, C12 to C27, C13 to C28, C14 to C29, C15 to C30, CH1 to CH3, CH2 to CH4, CL1 to CL3, CL2 to CL4, D4 to D8, D5 to D9, FL1 to FL2, R28 to R46, R29 to R47, R30 to R48, U7 to U13, U8 to U14, Y2 to Y4
Changed lines of the file:
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@@
   (symbol (lib_id "Device:C_Small") (at 146.05 129.54 0)
     (in_bom yes) (on_board yes)
-    (property "Reference" "C14" (id 0) (at 148.3868 128.3716 0)
+    (property "Reference" "C29" (id 0) (at 148.3868 128.3716 0)
       (effects (font (size 1.27 1.27)) (justify left))
     )
@@
   (symbol (lib_id "Device:R_Small") (at 146.05 119.38 0)
     (in_bom yes) (on_board yes)
-    (property "Reference" "R30" (id 0) (at 147.5486 118.2116 0)
+    (property "Reference" "R48" (id 0) (at 147.5486 118.2116 0)
       (effects (font (size 1.27 1.27)) (justify left))
     )
@@
   (symbol (lib_id "Device:R_Small") (at 140.97 124.46 270)
     (in_bom yes) (on_board yes)
-    (property "Reference" "R29" (id 0) (at 140.97 119.4816 90))
+    (property "Reference" "R47" (id 0) (at 140.97 119.4816 90))
     (property "Value" "1K" (id 1) (at 140.97 121.793 90))
     (property "Footprint" "Resistor_SMD:R_0402_1005Metric" (id 2) (at 140.97 124.46 0)
@@
   (symbol (lib_id "Device:C_Small") (at 165.1 78.74 0)
     (in_bom yes) (on_board yes)
-    (property "Reference" "C15" (id 0) (at 167.4368 77.5716 0)
+    (property "Reference" "C30" (id 0) (at 167.4368 77.5716 0)
       (effects (font (size 1.27 1.27)) (justify left))
     )
@@
   (symbol (lib_id "Device:C_Small") (at 110.49 78.74 0)
     (in_bom yes) (on_board yes)
-    (property "Reference" "C12" (id 0) (at 112.8268 77.5716 0)
+    (property "Reference" "C27" (id 0) (at 112.8268 77.5716 0)
       (effects (font (size 1.27 1.27)) (justify left))
     )
@@
   (symbol (lib_id "Device:C_Small") (at 57.15 106.68 270)
     (in_bom yes) (on_board yes)
-    (property "Reference" "C10" (id 0) (at 58.42 100.33 0)
+    (property "Reference" "C25" (id 0) (at 58.42 100.33 0)
       (effects (font (size 1.27 1.27)) (justify left))
     )
@@
   (symbol (lib_id "Device:CP1_Small") (at 120.65 78.74 0)
     (in_bom yes) (on_board yes)
-    (property "Reference" "C13" (id 0) (at 122.9614 77.5716 0)
+    (property "Reference" "C28" (id 0) (at 122.9614 77.5716 0)
       (effects (font (size 1.27 1.27)) (justify left))
     )
@@
   (symbol (lib_id "Device:C_Small") (at 57.15 116.84 270)
     (in_bom yes) (on_board yes)
-    (property "Reference" "C11" (id 0) (at 58.42 120.65 0)
+    (property "Reference" "C26" (id 0) (at 58.42 120.65 0)
       (effects (font (size 1.27 1.27)) (justify left))
     )
@@
   (symbol (lib_id "Interface_CAN_LIN:MCP2515-xST") (at 99.06 105.41 0)
     (in_bom yes) (on_board yes)
-    (property "Reference" "U7" (id 0) (at 99.06 80.4926 0))
+    (property "Reference" "U13" (id 0) (at 99.06 80.4926 0))
     (property "Value" "MCP2515-xST" (id 1) (at 99.06 82.804 0))
     (property "Footprint" "Package_SO:TSSOP-20_4.4x6.5mm_P0.65mm" (id 2) (at 99.06 128.27 0)
@@
   (symbol (lib_id "Device:Crystal_GND24_Small") (at 64.77 111.76 90)
     (in_bom yes) (on_board yes)
-    (property "Reference" "Y2" (id 0) (at 63.5 105.41 0)
+    (property "Reference" "Y4" (id 0) (at 63.5 105.41 0)
       (effects (font (size 1.27 1.27)) (justify left))
     )
@@
   (symbol (lib_id "Device:EMI_Filter_CommonMode") (at 191.77 95.25 0)
     (in_bom yes) (on_board yes)
-    (property "Reference" "FL1" (id 0) (at 191.77 88.1126 0))
+    (property "Reference" "FL2" (id 0) (at 191.77 88.1126 0))
     (property "Value" "DLW21SN921SK2" (id 1) (at 191.77 90.424 0))
     (property "Footprint" "Inductor_SMD:L_CommonModeChoke_Coilcraft_0805USB" (id 2) (at 191.77 94.234 0)
@@
   (symbol (lib_id "Device:C_Small") (at 172.72 104.14 0)
     (in_bom yes) (on_board yes)
-    (property "Reference" "CH1" (id 0) (at 175.0568 102.9716 0)
+    (property "Reference" "CH3" (id 0) (at 175.0568 102.9716 0)
       (effects (font (size 1.27 1.27)) (justify left))
     )
@@
   (symbol (lib_id "Device:C_Small") (at 182.88 104.14 0)
     (in_bom yes) (on_board yes)
-    (property "Reference" "CL1" (id 0) (at 185.2168 102.9716 0)
+    (property "Reference" "CL3" (id 0) (at 185.2168 102.9716 0)
       (effects (font (size 1.27 1.27)) (justify left))
     )
@@
   (symbol (lib_id "Device:D_TVS") (at 220.98 104.14 270)
     (in_bom yes) (on_board yes)
-    (property "Reference" "D4" (id 0) (at 223.012 102.9716 90)
+    (property "Reference" "D8" (id 0) (at 223.012 102.9716 90)
       (effects (font (size 1.27 1.27)) (justify left))
     )
@@
   (symbol (lib_id "Device:C_Small") (at 199.39 104.14 0)
     (in_bom yes) (on_board yes)
-    (property "Reference" "CH2" (id 0) (at 201.7268 102.9716 0)
+    (property "Reference" "CH4" (id 0) (at 201.7268 102.9716 0)
       (effects (font (size 1.27 1.27)) (justify left))
     )
@@
   (symbol (lib_id "Device:C_Small") (at 209.55 104.14 0)
     (in_bom yes) (on_board yes)
-    (property "Reference" "CL2" (id 0) (at 211.8868 102.9716 0)
+    (property "Reference" "CL4" (id 0) (at 211.8868 102.9716 0)
       (effects (font (size 1.27 1.27)) (justify left))
     )
@@
   (symbol (lib_id "Device:D_TVS") (at 231.14 104.14 270)
     (in_bom yes) (on_board yes)
-    (property "Reference" "D5" (id 0) (at 233.172 102.9716 90)
+    (property "Reference" "D9" (id 0) (at 233.172 102.9716 90)
       (effects (font (size 1.27 1.27)) (justify left))
     )
@@
   (symbol (lib_id "Device:R_Small") (at 74.93 111.76 180)
     (in_bom yes) (on_board yes)
-    (property "Reference" "R28" (id 0) (at 79.9084 111.76 90))
+    (property "Reference" "R46" (id 0) (at 79.9084 111.76 90))
     (property "Value" "1M" (id 1) (at 77.47 111.76 90))
     (property "Footprint" "Resistor_SMD:R_0402_1005Metric" (id 2) (at 74.93 111.76 0)
@@
   (symbol (lib_id "Interface_CAN_LIN:MCP2551-I-SN") (at 152.4 95.25 0)
     (in_bom yes) (on_board yes)
-    (property "Reference" "U8" (id 0) (at 152.4 80.4926 0))
+    (property "Reference" "U14" (id 0) (at 152.4 80.4926 0))
     (property "Value" "MCP2551-I-SN" (id 1) (at 152.4 82.804 0))
     (property "Footprint" "Package_SO:SOIC-8_3.9x4.9mm_P1.27mm" (id 2) (at 152.4 107.95 0)

Commit message: Fix RXCAN and TXCAN connection
Parts:
- renumbered C25 to C10, C26 to C11, C27 to C12, C28 to C13, C29 to C14, C30 to C15, CH3 to CH1, CH4 to CH2, CL3 to CL1, CL4 to CL2, D8 to D4, D9 to D5, FL2 to FL1, R46 to R28, R47 to R29, R48 to R30, U13 to U7, U14 to U8, Y4 to Y2
Connections:
- net at U7.1 (TXCAN): now also U8.1 (TXD); no longer U8.4 (RXD)
- net at U7.2 (RXCAN): now also U8.4 (RXD); no longer U8.1 (TXD)

Commit message: Board revision A2
Ready for production
Added geigerboard
Parts:
- added R25, R43: 0, Resistor_SMD:R_0402_1005Metric, symbol Device:R_Small
- C28: renamed from C13; footprint Capacitor_Tantalum_SMD:CP_EIA-3216-10_Kemet-I -> Capacitor_SMD:C_0805_2012Metric; symbol Device:CP1_Small -> Device:C_Small
- renumbered C10 to C25, C11 to C26, C12 to C27, C14 to C29, C15 to C30, CH1 to CH3, CH2 to CH4, CL1 to CL3, CL2 to CL4, D4 to D8, D5 to D9, FL1 to FL2, R28 to R46, R29 to R47, R30 to R48, U7 to U13, U8 to U14, Y2 to Y4
Connections:
- net at U13.1 (TXCAN): now also R25.1; no longer U14.1 (TXD)
- net at U13.2 (RXCAN): now also R43.2; no longer U14.4 (RXD)
- new net: R25.2, U14.1 (TXD)
- new net: R43.1, U14.4 (RXD)

Commit message: Board revision A3, Schematic D3
Added 5V LDO (Fixed #15)
Added decoupling caps for mounting holes (Fixed #12)
More space for flash LDO (Fixed #1)
Removed TVS diodes from CAN bus (Fixed #3)
Parts:
- removed D8: TVS1, Diode_SMD:D_SOD-323, symbol Device:D_TVS
- removed D9: TVS2, Diode_SMD:D_SOD-323, symbol Device:D_TVS
- C13: renamed from C28; value 22uF -> 1uF; footprint Capacitor_SMD:C_0805_2012Metric -> Capacitor_SMD:C_0603_1608Metric
- renumbered C25 to C10, C26 to C11, C27 to C12, C29 to C14, C30 to C15, CH3 to CH1, CH4 to CH2, CL3 to CL1, CL4 to CL2, FL2 to FL1, R43 to R24, R46 to R28, R47 to R29, R48 to R30, R25 to R5, U13 to U7, U14 to U8, Y4 to Y2
Other:
- note removed: "TVS Diodes: SD12_323"
- moved on the sheet: C10, C11, C12, C13, C14, C15, CH1, CH2, CL1, CL2, FL1, R24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
