File: ykts-payload/ykts-payload.kicad_sch (KiCad schematic)
At the start: 49 parts, among them J1 DBG_PWR, J2 GeigerBoard, J3 PC/104 Connector, J4 Solar_Temp, J5 Sensor_Ext, Q1 PMV65XP, Q4 RJU003N03 NMOS, Q5 RJU003N03 NMOS, Q6 RJU003N03 NMOS, Q7 RJU003N03 NMOS

Commit message: Bump board
Connections:
- net I2C_SCL is gone; now on net SCL: J5.2 (Pin_2)
- net I2C_SDA is gone; now on net SDA: J5.4 (Pin_4)
- net SCL: no longer Q4.3 (D), Q5.3 (D)
- net SDA: no longer Q6.3 (D), Q7.3 (D)
- net MOSFET_GEIGER renamed GEIGER_FET
- new net S0_SCL: Q4.3 (D)
- new net S0_SDA: Q6.3 (D)
- new net S1_SCL: Q5.3 (D)
- new net S1_SDA: Q7.3 (D)

Commit message: Rework power supply
Parts:
- added C9: 100nF, Capacitor_SMD:C_0402_1005Metric, symbol Device:C_Small
- added D3: LED, LED_SMD:LED_0402_1005Metric, symbol Device:LED
- added R23: 1K, Resistor_SMD:R_0402_1005Metric, symbol Device:R_Small
- added R_CSB1: 0.1, Resistor_SMD:R_1210_3225Metric, symbol Device:R_Small
- added U4: MAX4372FEUK, Package_TO_SOT_SMD:SOT-23-5, symbol yktsat-common:MAX4372FEUK
Connections:
- net +5V_A is gone; now on net +5V: J4.2 (Pin_2), J5.1 (Pin_1), N1.7 (VCC), N2.7 (VCC), N3.7 (VCC), N4.7 (VCC), N5.7 (VCC), N6.7 (VCC), N7.7 (VCC), N8.7 (VCC), Q4.2 (G), Q6.2 (G), R51.2, R53.2, R8.1
- net +5V_B is gone; now on net +5V: N10.7 (VCC), N11.7 (VCC), N12.7 (VCC), N13.7 (VCC), N14.7 (VCC), N15.7 (VCC), N16.7 (VCC), N9.7 (VCC), Q5.2 (G), Q7.2 (G), R52.2, R54.2
- net +5V: now also R_CSB1.1, U4.5 (RS-); no longer J3.a9 (Pin_a9), J3.b9 (Pin_b9)
- net GND: now also C9.2, R23.2, U4.1 (GND)
- new net: C9.1, D3.2 (A), U4.3 (VCC)
- new net: D3.1 (K), R23.1
- new net CSENSE: U4.2 (OUT)
- new net PCH4: J3.a9 (Pin_a9), J3.b9 (Pin_b9), R_CSB1.2, U4.4 (RS+)
Other:
- removed sheet Payload Power Control 0
- removed sheet Payload Power Control 1

Commit message: Revision D1, board A0
Board initial release
Parts:
- removed D1: LED_PWON, LED_SMD:LED_0402_1005Metric, symbol Device:LED
- removed J3: PC/104 Connector, Connector_PinSocket_2.54mm:PinSocket_2x32_P2.54mm_Vertical, symbol Connector_Generic:Conn_02x32_Row_Letter_First
- removed R5: 1K, Resistor_SMD:R_0402_1005Metric, symbol Device:R_Small
- added J111: PC/104 Connector, symbol Connector_Generic:Conn_02x32_Row_Letter_First
- added J3: Conn_02x32_Odd_Even, Connector_PinHeader_2.54mm:PinHeader_2x32_P2.54mm_Vertical, symbol Connector_Generic:Conn_02x32_Odd_Even
Connections:
- net +5V: now also C9.1, D3.2 (A), U4.3 (VCC)
- net CANH: now also J3.25 (Pin_25)
- net CANL: now also J3.26 (Pin_26)
- net CH_A: now also J3.62 (Pin_62)
- net CH_B: now also J3.61 (Pin_61)
- net GND: now also J3.19 (Pin_19), J3.20 (Pin_20)
- net PCH4: now also J3.17 (Pin_17), J3.18 (Pin_18)
- no-connect marks 3 -> 59
Other:
- moved on the sheet: J1

Commit message: Fix RXCAN and TXCAN connection
Other:
- note added: "Note: Row B = odd Row A = even"
- moved on the sheet: J111, J3

Commit message: Board revision A2
Ready for production
Added geigerboard
Parts:
- removed Q4, Q5, Q6, Q7: RJU003N03 NMOS, Package_TO_SOT_SMD:SOT-323_SC-70, symbol Device:Q_NMOS_SGD
- removed R51, R52, R53, R54: 10K, Resistor_SMD:R_0402_1005Metric, symbol Device:R_Small
- added H9: GeigerBoard Mount / M2, MountingHole:MountingHole_2.2mm_M2_Pad, symbol Mechanical:MountingHole_Pad
Connections:
- net CANH: now also J3.26 (Pin_26); no longer J3.25 (Pin_25)
- net CANL: now also J3.25 (Pin_25); no longer J3.26 (Pin_26)
- net CH_A: now also J3.61 (Pin_61); no longer J3.62 (Pin_62)
- net CH_B: now also J3.62 (Pin_62); no longer J3.61 (Pin_61)
- net GND: now also H9.1
Other:
- note added: "Note: Row A = odd Row B = even"
- note removed: "Note: Row B = odd Row A = even"
- moved on the sheet: C9, D3, H1, H2, H3, H4, H5, H6, H7, H8, R1, R2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

Commit message: Board revision A3, Schematic D3
Added 5V LDO (Fixed #15)
Added decoupling caps for mounting holes (Fixed #12)
More space for flash LDO (Fixed #1)
Removed TVS diodes from CAN bus (Fixed #3)
Parts:
- added C? (x4): 10nF 1000V, Capacitor_SMD:C_0603_1608Metric, symbol Device:C_Small
- added C? (x2): 100nF, Capacitor_SMD:C_0402_1005Metric, symbol Device:C_Small
- added C? (x2): 1uF, Capacitor_SMD:C_0603_1608Metric, symbol Device:C_Small
- added U? (x2): AMS1117-5.0, Package_TO_SOT_SMD:SOT-223-3_TabPin2, symbol Regulator_Linear:AMS1117-5.0
- R1, R2, R3, R4: value 1M -> 10M
- R6, R7: value 4.7K -> 30K
Connections:
- net GND: now also C?.1, C?.1, C?.1, C?.1, C?.2, C?.2, C?.2, C?.2, U?.1 (GND), U?.1 (GND)
- net PCH4: now also C?.1, C?.1, U?.3 (VI), U?.3 (VI); no longer R_CSB1.2, U4.4 (RS+)
- net at H1.1, R1.1: now also C?.2
- net at H2.1, R2.1: now also C?.2
- net at H3.1, R3.1: now also C?.2
- net at H4.1, R4.1: now also C?.2
- new net: C?.1, C?.1, R_CSB1.2, U4.4 (RS+), U?.2 (VO), U?.2 (VO)
Other:
- note added: "PCH4: 6.5 - 8.5 V"
- moved on the sheet: C9, D3, H1, H2, H3, H4, H5, H6, H7, H8, H9, N1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
