File: ykts-payload/ykts-payload.kicad_sch (KiCad schematic)
At the start: 53 parts, among them J1 DBG_PWR, J111 PC/104 Connector, J2 GeigerBoard, J3 Conn_02x32_Odd_Even, J4 Solar_Temp, J5 Sensor_Ext, Q1 PMV65XP, U12 AMS1117-5.0, U4 MAX4372FEUK

Commit message: Board revision A5, schematic E0
Fixed #16
Fixed #17
Revamped schematic
Parts:
- added R26, R27, R44, R45: 33K, Resistor_SMD:R_0402_1005Metric, symbol Device:R_Small
- added U15, U16, U5, U6: 74HC4051BQ,115, Package_SO:TSSOP-16_4.4x5mm_P0.65mm, symbol yktsat-common:74HC4051BQ,115
Connections:
- net +5V: now also R26.1, R27.2, R44.1, R45.2, U15.16 (VCC), U15.7 (VEE), U16.16 (VCC), U16.7 (VEE), U5.16 (VCC), U5.7 (VEE), U6.16 (VCC), U6.7 (VEE)
- net GND: now also U15.8 (GND), U16.8 (GND), U5.8 (GND), U6.8 (GND)
- net N0_RX: now also U6.13 (A0)
- net N0_TX: now also U5.13 (A0)
- net N10_RX: now also U16.5 (A5)
- net N10_TX: now also U15.5 (A5)
- net N11_RX: now also U16.4 (A7)
- net N11_TX: now also U15.4 (A7)
- net N12_RX: now also U16.15 (A2)
- net N12_TX: now also U15.15 (A2)
- net N13_RX: now also U16.2 (A6)
- net N13_TX: now also U15.2 (A6)
- net N14_RX: now also U16.13 (A0)
- net N14_TX: now also U15.13 (A0)
- net N15_RX: now also U16.1 (A4)
- net N15_TX: now also U15.1 (A4)
- net N1_RX: now also U6.12 (A3)
- net N1_TX: now also U5.12 (A3)
- net N2_RX: now also U6.5 (A5)
- net N2_TX: now also U5.5 (A5)
- net N3_RX: now also U6.4 (A7)
- net N3_TX: now also U5.4 (A7)
- net N4_RX: now also U6.14 (A1)
- net N4_TX: now also U5.14 (A1)
- net N5_RX: now also U6.2 (A6)
- net N5_TX: now also U5.2 (A6)
- net N6_RX: now also U6.15 (A2)
- net N6_TX: now also U5.15 (A2)
- net N7_RX: now also U6.1 (A4)
- net N7_TX: now also U5.1 (A4)
- net N8_RX: now also U16.14 (A1)
- net N8_TX: now also U15.14 (A1)
- net N9_RX: now also U16.12 (A3)
- net N9_TX: now also U15.12 (A3)
- new net: R27.1, U6.6 (~{E})
- new net: R45.1, U16.6 (~{E})
- new net: R44.2, U15.6 (~{E})
- new net: R26.2, U5.6 (~{E})
- new net Payload Supervisor 0/MUX_A0: U5.11 (S0), U6.11 (S0)
- new net Payload Supervisor 0/MUX_A1: U5.10 (S1), U6.10 (S1)
- new net Payload Supervisor 0/MUX_A2: U5.9 (S2), U6.9 (S2)
- new net Payload Supervisor 0/RX1: U5.3 (A)
- new net Payload Supervisor 0/TX1: U6.3 (A)
- new net Payload Supervisor 1/MUX_A0: U15.9 (S2), U16.9 (S2)
- new net Payload Supervisor 1/MUX_A1: U15.10 (S1), U16.10 (S1)
- new net Payload Supervisor 1/MUX_A2: U15.11 (S0), U16.11 (S0)
- new net Payload Supervisor 1/RX1: U15.3 (A)
- new net Payload Supervisor 1/TX1: U16.3 (A)
Other:
- removed sheet Node RX MUX 0
- removed sheet Node RX MUX 1
- removed sheet Node TX MUX 0
- removed sheet Node TX MUX 1

Commit message: Schematic revision E1
Cleanup
Parts:
- H1, H2, H3, H4: value CubeSat Mount / M3 -> Chasis / M3
- H5, H6, H7, H8, H9: value GeigerBoard Mount / M2 -> Geiger / M2
Other:
- note added: "5V PCH4 Regulator"
- note added: "Node Group 0 - Nodes 0-7, Top side"
- note added: "Node Group 1 - Nodes 8-16, Bottom side"
- note added: "Supervisor / CAN 0"
- note added: "Supervisor / CAN 1"
- note added: "UART MUX 0"
- note added: "UART MUX 1"
- note removed: "Node Group 0"
- note removed: "Node Group 1"
- note removed: "Nodes 0-7 Top side"
- note removed: "Nodes 8-15 Bottom side"
- moved on the sheet: C24, C31, C32, C33, C34, C36, C9, D3, H1, H2, H3, H4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

Commit message: Sync with remote
Connections:
- net Payload Supervisor 0/MUX_A0: now also U5.9 (S2), U6.9 (S2); no longer U5.11 (S0), U6.11 (S0)
- net Payload Supervisor 0/MUX_A2: now also U5.11 (S0), U6.11 (S0); no longer U5.9 (S2), U6.9 (S2)
- net Payload Supervisor 1/MUX_A0: now also U15.11 (S0), U16.11 (S0); no longer U15.9 (S2), U16.9 (S2)
- net Payload Supervisor 1/MUX_A2: now also U15.9 (S2), U16.9 (S2); no longer U15.11 (S0), U16.11 (S0)
Other:
- note added: "0"
- note added: "1"
- note added: "10"
- note added: "11"
- note added: "12"
- note added: "13"
- note added: "14"
- note added: "15"
- note added: "2"
- note added: "3"
- note added: "4"
- note added: "5"
- note added: "6"
- note added: "7"
- note added: "8"
- note added: "9"
- note added: "MCU Pin"
- note added: "MUX Pin"
- note added: "MUX pin mappings"
- note added: "NOTE: TX/RX are swapped here"
- note added: "Node #"
- note added: "Node pin mappings"
- note added: "PA0"
- note added: "PA1"
- note added: "PA2"
- note added: "PA3"
- note added: "PA4"
- note added: "PA5"
- note added: "PA6"
- note added: "PA7"
- note added: "PC0"
- note added: "PC1"
- note added: "PC2"
- note added: "PC3"
- note added: "PC4"
- note added: "PC5"
- note added: "PC6"
- note added: "PC7"
- note added: "PD4"
- note added: "PD5"
- note added: "PD6"
- note added: "PWR"
- note added: "Reset"
- note added: "S0 (A0)"
- note added: "S1 (A1)"
- note added: "S2 (A2)"
- moved on the sheet: D3, J1, J111, R23, R26, R27, R44, R45
