File: ykts-payload/ykts-payload-mux.kicad_sch (KiCad schematic)
At the start: 2 parts, among them U6 74HC4051BQ,115

Commit message: Rework power supply
Parts:
- renumbered R27 to R49, U6 to U15
Changed lines of the file:
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@@
   (symbol (lib_id "Device:R_Small") (at 137.16 88.9 0)
     (in_bom yes) (on_board yes)
-    (property "Reference" "R27" (id 0) (at 132.1816 88.9 90))
+    (property "Reference" "R49" (id 0) (at 132.1816 88.9 90))
     (property "Value" "33K" (id 1) (at 134.493 88.9 90))
     (property "Footprint" "Resistor_SMD:R_0402_1005Metric" (id 2) (at 137.16 88.9 0)
@@
   (symbol (lib_id "yktsat-common:74HC4051BQ,115") (at 149.86 104.14 0)
     (in_bom yes) (on_board yes)
-    (property "Reference" "U6" (id 0) (at 151.13 86.8426 0))
+    (property "Reference" "U15" (id 0) (at 151.13 86.8426 0))
     (property "Value" "74HC4051BQ,115" (id 1) (at 151.13 89.154 0))
     (property "Footprint" "Package_SO:TSSOP-16_4.4x5mm_P0.65mm" (id 2) (at 149.86 114.3 0)

Commit message: Fix RXCAN and TXCAN connection
Parts:
- renumbered R49 to R27, U15 to U6
Changed lines of the file:
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@@
   (symbol (lib_id "Device:R_Small") (at 137.16 88.9 0)
     (in_bom yes) (on_board yes)
-    (property "Reference" "R49" (id 0) (at 132.1816 88.9 90))
+    (property "Reference" "R27" (id 0) (at 132.1816 88.9 90))
     (property "Value" "33K" (id 1) (at 134.493 88.9 90))
     (property "Footprint" "Resistor_SMD:R_0402_1005Metric" (id 2) (at 137.16 88.9 0)
@@
   (symbol (lib_id "yktsat-common:74HC4051BQ,115") (at 149.86 104.14 0)
     (in_bom yes) (on_board yes)
-    (property "Reference" "U15" (id 0) (at 151.13 86.8426 0))
+    (property "Reference" "U6" (id 0) (at 151.13 86.8426 0))
     (property "Value" "74HC4051BQ,115" (id 1) (at 151.13 89.154 0))
     (property "Footprint" "Package_SO:TSSOP-16_4.4x5mm_P0.65mm" (id 2) (at 149.86 114.3 0)

Commit message: Board revision A2
Ready for production
Added geigerboard
Parts:
- renumbered R27 to R49, U6 to U15
Changed lines of the file:
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@@
   (title_block
     (title "YktSat Payload Module")
-    (date "2021-12-07")
-    (rev "D1")
+    (date "2021-12-18")
+    (rev "D2")
     (company "Sakha Aerospace Systems, LLC")
+    (comment 2 "Designed by: ThePetrovich")
   )
   (junction (at 137.16 82.55) (diameter 0) (color 0 0 0 0)
@@
   (symbol (lib_id "Device:R_Small") (at 137.16 88.9 0)
     (in_bom yes) (on_board yes)
-    (property "Reference" "R27" (id 0) (at 132.1816 88.9 90))
+    (property "Reference" "R49" (id 0) (at 132.1816 88.9 90))
     (property "Value" "33K" (id 1) (at 134.493 88.9 90))
     (property "Footprint" "Resistor_SMD:R_0402_1005Metric" (id 2) (at 137.16 88.9 0)
@@
   (symbol (lib_id "yktsat-common:74HC4051BQ,115") (at 149.86 104.14 0)
     (in_bom yes) (on_board yes)
-    (property "Reference" "U6" (id 0) (at 151.13 86.8426 0))
+    (property "Reference" "U15" (id 0) (at 151.13 86.8426 0))
     (property "Value" "74HC4051BQ,115" (id 1) (at 151.13 89.154 0))
     (property "Footprint" "Package_SO:TSSOP-16_4.4x5mm_P0.65mm" (id 2) (at 149.86 114.3 0)

Commit message: Board revision A3, Schematic D3
Added 5V LDO (Fixed #15)
Added decoupling caps for mounting holes (Fixed #12)
More space for flash LDO (Fixed #1)
Removed TVS diodes from CAN bus (Fixed #3)
Parts:
- renumbered R49 to R27, U15 to U6
Changed lines of the file:
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@@
   (title_block
     (title "YktSat Payload Module")
-    (date "2021-12-18")
-    (rev "D2")
+    (date "2022-01-28")
+    (rev "D3")
     (company "Sakha Aerospace Systems, LLC")
     (comment 2 "Designed by: ThePetrovich")
@@
   (symbol (lib_id "Device:R_Small") (at 137.16 88.9 0)
     (in_bom yes) (on_board yes)
-    (property "Reference" "R49" (id 0) (at 132.1816 88.9 90))
+    (property "Reference" "R27" (id 0) (at 132.1816 88.9 90))
     (property "Value" "33K" (id 1) (at 134.493 88.9 90))
     (property "Footprint" "Resistor_SMD:R_0402_1005Metric" (id 2) (at 137.16 88.9 0)
@@
   (symbol (lib_id "yktsat-common:74HC4051BQ,115") (at 149.86 104.14 0)
     (in_bom yes) (on_board yes)
-    (property "Reference" "U15" (id 0) (at 151.13 86.8426 0))
+    (property "Reference" "U6" (id 0) (at 151.13 86.8426 0))
     (property "Value" "74HC4051BQ,115" (id 1) (at 151.13 89.154 0))
     (property "Footprint" "Package_SO:TSSOP-16_4.4x5mm_P0.65mm" (id 2) (at 149.86 114.3 0)
@@
   (symbol (lib_id "power:GND") (at 149.86 123.19 0)
     (in_bom yes) (on_board yes)
-    (property "Reference" "#PWR0116" (id 0) (at 149.86 129.54 0)
+    (property "Reference" "#PWR077" (id 0) (at 149.86 129.54 0)
       (effects (font (size 1.27 1.27)) hide)
     )

Commit message: Changed flash LDO to L78L33
Parts:
- renumbered R27 to R49, U6 to U15
Changed lines of the file:
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@@
   (symbol (lib_id "Device:R_Small") (at 137.16 88.9 0)
     (in_bom yes) (on_board yes)
-    (property "Reference" "R27" (id 0) (at 132.1816 88.9 90))
+    (property "Reference" "R49" (id 0) (at 132.1816 88.9 90))
     (property "Value" "33K" (id 1) (at 134.493 88.9 90))
     (property "Footprint" "Resistor_SMD:R_0402_1005Metric" (id 2) (at 137.16 88.9 0)
@@
   (symbol (lib_id "yktsat-common:74HC4051BQ,115") (at 149.86 104.14 0)
     (in_bom yes) (on_board yes)
-    (property "Reference" "U6" (id 0) (at 151.13 86.8426 0))
+    (property "Reference" "U15" (id 0) (at 151.13 86.8426 0))
     (property "Value" "74HC4051BQ,115" (id 1) (at 151.13 89.154 0))
     (property "Footprint" "Package_SO:TSSOP-16_4.4x5mm_P0.65mm" (id 2) (at 149.86 114.3 0)
@@
   (symbol (lib_id "power:GND") (at 149.86 123.19 0)
     (in_bom yes) (on_board yes)
-    (property "Reference" "#PWR077" (id 0) (at 149.86 129.54 0)
+    (property "Reference" "#PWR0116" (id 0) (at 149.86 129.54 0)
       (effects (font (size 1.27 1.27)) hide)
     )
