File: ykts-payload/ykts-payload-supervisor-flash.kicad_sch (KiCad schematic)
At the start: 10 parts, among them U10 AMS1117-3.3, U11 AT25DF161-SF-T

Commit message: Fix RXCAN and TXCAN connection
Parts:
- renumbered C22 to C7, C23 to C8, R37 to R17, R38 to R18, R39 to R19, R40 to R20, R41 to R21, R42 to R22, U10 to U2, U11 to U3
Changed lines of the file:
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@@
   (symbol (lib_id "power:GND") (at 132.08 125.73 0)
     (in_bom yes) (on_board yes)
-    (property "Reference" "#PWR0100" (id 0) (at 132.08 132.08 0)
+    (property "Reference" "#PWR071" (id 0) (at 132.08 132.08 0)
       (effects (font (size 1.27 1.27)) hide)
     )
@@
   (symbol (lib_id "Device:R_Small") (at 137.16 119.38 0)
     (in_bom yes) (on_board yes)
-    (property "Reference" "R39" (id 0) (at 138.6586 118.2116 0)
+    (property "Reference" "R19" (id 0) (at 138.6586 118.2116 0)
       (effects (font (size 1.27 1.27)) (justify left))
     )
@@
   (symbol (lib_id "Device:R_Small") (at 132.08 114.3 0)
     (in_bom yes) (on_board yes)
-    (property "Reference" "R38" (id 0) (at 133.5786 113.1316 0)
+    (property "Reference" "R18" (id 0) (at 133.5786 113.1316 0)
       (effects (font (size 1.27 1.27)) (justify left))
     )
@@
   (symbol (lib_id "Device:C_Small") (at 143.51 80.01 0) (mirror y)
     (in_bom yes) (on_board yes)
-    (property "Reference" "C23" (id 0) (at 141.1732 78.8416 0)
+    (property "Reference" "C8" (id 0) (at 141.1732 78.8416 0)
       (effects (font (size 1.27 1.27)) (justify left))
     )
@@
   (symbol (lib_id "yktsat-common:AT25DF161-SF-T") (at 165.1 101.6 0)
     (in_bom yes) (on_board yes)
-    (property "Reference" "U11" (id 0) (at 154.94 87.63 0))
+    (property "Reference" "U3" (id 0) (at 154.94 87.63 0))
     (property "Value" "AT25DF161-SF-T" (id 1) (at 154.94 90.17 0))
     (property "Footprint" "Package_SO:SO-8_3.9x4.9mm_P1.27mm" (id 2) (at 160.02 116.84 0)
@@
   (symbol (lib_id "Device:R_Small") (at 143.51 96.52 270)
     (in_bom yes) (on_board yes)
-    (property "Reference" "R40" (id 0) (at 139.7 97.79 90))
+    (property "Reference" "R20" (id 0) (at 139.7 97.79 90))
     (property "Value" "4.7K" (id 1) (at 147.32 97.79 90)
       (effects (font (size 0.9906 0.9906)))
@@
   (symbol (lib_id "Device:R_Small") (at 143.51 99.06 270)
     (in_bom yes) (on_board yes)
-    (property "Reference" "R41" (id 0) (at 139.7 100.33 90))
+    (property "Reference" "R21" (id 0) (at 139.7 100.33 90))
     (property "Value" "4.7K" (id 1) (at 147.32 100.33 90)
       (effects (font (size 0.9906 0.9906)))
@@
   (symbol (lib_id "Regulator_Linear:AMS1117-3.3") (at 132.08 74.93 0)
     (in_bom yes) (on_board yes)
-    (property "Reference" "U10" (id 0) (at 132.08 68.7832 0))
+    (property "Reference" "U2" (id 0) (at 132.08 68.7832 0))
     (property "Value" "AMS1117-3.3" (id 1) (at 132.08 71.0946 0))
     (property "Footprint" "Package_TO_SOT_SMD:SOT-89-3" (id 2) (at 132.08 69.85 0)
@@
   (symbol (lib_id "Device:R_Small") (at 127 109.22 0)
     (in_bom yes) (on_board yes)
-    (property "Reference" "R37" (id 0) (at 128.4986 108.0516 0)
+    (property "Reference" "R17" (id 0) (at 128.4986 108.0516 0)
       (effects (font (size 1.27 1.27)) (justify left))
     )
@@
   (symbol (lib_id "power:GND") (at 165.1 116.84 0)
     (in_bom yes) (on_board yes)
-    (property "Reference" "#PWR0101" (id 0) (at 165.1 123.19 0)
+    (property "Reference" "#PWR072" (id 0) (at 165.1 123.19 0)
       (effects (font (size 1.27 1.27)) hide)
     )
@@
   (symbol (lib_id "power:GND") (at 132.08 85.09 0)
     (in_bom yes) (on_board yes)
-    (property "Reference" "#PWR099" (id 0) (at 132.08 91.44 0)
+    (property "Reference" "#PWR070" (id 0) (at 132.08 91.44 0)
       (effects (font (size 1.27 1.27)) hide)
     )
@@
   (symbol (lib_id "Device:R_Small") (at 143.51 104.14 270)
     (in_bom yes) (on_board yes)
-    (property "Reference" "R42" (id 0) (at 139.7 105.41 90))
+    (property "Reference" "R22" (id 0) (at 139.7 105.41 90))
     (property "Value" "4.7K" (id 1) (at 147.32 105.41 90)
       (effects (font (size 0.9906 0.9906)))
@@
   (symbol (lib_id "Device:C_Small") (at 121.92 80.01 0) (mirror y)
     (in_bom yes) (on_board yes)
-    (property "Reference" "C22" (id 0) (at 119.5832 78.8416 0)
+    (property "Reference" "C7" (id 0) (at 119.5832 78.8416 0)
       (effects (font (size 1.27 1.27)) (justify left))
     )

Commit message: Board revision A2
Ready for production
Added geigerboard
Parts:
- renumbered C7 to C22, C8 to C23, R17 to R37, R18 to R38, R19 to R39, R20 to R40, R21 to R41, R22 to R42, U2 to U10, U3 to U11
Changed lines of the file:
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@@
   (title_block
     (title "YktSat Payload Module")
-    (date "2021-12-07")
-    (rev "D1")
+    (date "2021-12-18")
+    (rev "D2")
     (company "Sakha Aerospace Systems, LLC")
+    (comment 2 "Designed by: ThePetrovich")
   )
   (junction (at 165.1 86.36) (diameter 0) (color 0 0 0 0)
@@
   (symbol (lib_id "power:GND") (at 132.08 125.73 0)
     (in_bom yes) (on_board yes)
-    (property "Reference" "#PWR071" (id 0) (at 132.08 132.08 0)
+    (property "Reference" "#PWR0100" (id 0) (at 132.08 132.08 0)
       (effects (font (size 1.27 1.27)) hide)
     )
@@
   (symbol (lib_id "Device:R_Small") (at 137.16 119.38 0)
     (in_bom yes) (on_board yes)
-    (property "Reference" "R19" (id 0) (at 138.6586 118.2116 0)
+    (property "Reference" "R39" (id 0) (at 138.6586 118.2116 0)
       (effects (font (size 1.27 1.27)) (justify left))
     )
@@
   (symbol (lib_id "Device:R_Small") (at 132.08 114.3 0)
     (in_bom yes) (on_board yes)
-    (property "Reference" "R18" (id 0) (at 133.5786 113.1316 0)
+    (property "Reference" "R38" (id 0) (at 133.5786 113.1316 0)
       (effects (font (size 1.27 1.27)) (justify left))
     )
@@
   (symbol (lib_id "Device:C_Small") (at 143.51 80.01 0) (mirror y)
     (in_bom yes) (on_board yes)
-    (property "Reference" "C8" (id 0) (at 141.1732 78.8416 0)
+    (property "Reference" "C23" (id 0) (at 141.1732 78.8416 0)
       (effects (font (size 1.27 1.27)) (justify left))
     )
@@
   (symbol (lib_id "yktsat-common:AT25DF161-SF-T") (at 165.1 101.6 0)
     (in_bom yes) (on_board yes)
-    (property "Reference" "U3" (id 0) (at 154.94 87.63 0))
+    (property "Reference" "U11" (id 0) (at 154.94 87.63 0))
     (property "Value" "AT25DF161-SF-T" (id 1) (at 154.94 90.17 0))
     (property "Footprint" "Package_SO:SO-8_3.9x4.9mm_P1.27mm" (id 2) (at 160.02 116.84 0)
@@
   (symbol (lib_id "Device:R_Small") (at 143.51 96.52 270)
     (in_bom yes) (on_board yes)
-    (property "Reference" "R20" (id 0) (at 139.7 97.79 90))
+    (property "Reference" "R40" (id 0) (at 139.7 97.79 90))
     (property "Value" "4.7K" (id 1) (at 147.32 97.79 90)
       (effects (font (size 0.9906 0.9906)))
@@
   (symbol (lib_id "Device:R_Small") (at 143.51 99.06 270)
     (in_bom yes) (on_board yes)
-    (property "Reference" "R21" (id 0) (at 139.7 100.33 90))
+    (property "Reference" "R41" (id 0) (at 139.7 100.33 90))
     (property "Value" "4.7K" (id 1) (at 147.32 100.33 90)
       (effects (font (size 0.9906 0.9906)))
@@
   (symbol (lib_id "Regulator_Linear:AMS1117-3.3") (at 132.08 74.93 0)
     (in_bom yes) (on_board yes)
-    (property "Reference" "U2" (id 0) (at 132.08 68.7832 0))
+    (property "Reference" "U10" (id 0) (at 132.08 68.7832 0))
     (property "Value" "AMS1117-3.3" (id 1) (at 132.08 71.0946 0))
     (property "Footprint" "Package_TO_SOT_SMD:SOT-89-3" (id 2) (at 132.08 69.85 0)
@@
   (symbol (lib_id "Device:R_Small") (at 127 109.22 0)
     (in_bom yes) (on_board yes)
-    (property "Reference" "R17" (id 0) (at 128.4986 108.0516 0)
+    (property "Reference" "R37" (id 0) (at 128.4986 108.0516 0)
       (effects (font (size 1.27 1.27)) (justify left))
     )
@@
   (symbol (lib_id "power:GND") (at 165.1 116.84 0)
     (in_bom yes) (on_board yes)
-    (property "Reference" "#PWR072" (id 0) (at 165.1 123.19 0)
+    (property "Reference" "#PWR0101" (id 0) (at 165.1 123.19 0)
       (effects (font (size 1.27 1.27)) hide)
     )
@@
   (symbol (lib_id "power:GND") (at 132.08 85.09 0)
     (in_bom yes) (on_board yes)
-    (property "Reference" "#PWR070" (id 0) (at 132.08 91.44 0)
+    (property "Reference" "#PWR099" (id 0) (at 132.08 91.44 0)
       (effects (font (size 1.27 1.27)) hide)
     )
@@
   (symbol (lib_id "Device:R_Small") (at 143.51 104.14 270)
     (in_bom yes) (on_board yes)
-    (property "Reference" "R22" (id 0) (at 139.7 105.41 90))
+    (property "Reference" "R42" (id 0) (at 139.7 105.41 90))
     (property "Value" "4.7K" (id 1) (at 147.32 105.41 90)
       (effects (font (size 0.9906 0.9906)))
@@
   (symbol (lib_id "Device:C_Small") (at 121.92 80.01 0) (mirror y)
     (in_bom yes) (on_board yes)
-    (property "Reference" "C7" (id 0) (at 119.5832 78.8416 0)
-      (effects (font (size 1.27 1.27)) (justify left))
-    )
+    (property "Reference" "C22" (id 0) (at 119.5832 78.8416 0)
+      (effects (font (size 1.27 1.27)) (justify left))
+    )

Commit message: Changed flash LDO to L78L33
Parts:
- removed U10: AMS1117-3.3, Package_TO_SOT_SMD:SOT-89-3, symbol Regulator_Linear:AMS1117-3.3
- added U?: L78L33_SOT89, Package_TO_SOT_SMD:SOT-89-3, symbol Regulator_Linear:L78L33_SOT89
Connections:
- net 5V: now also U?.3 (IN)
- net GND: now also U?.2 (GND)
- net at C23.1, U11.3 (~{WP}), U11.7 (~{HOLD})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: now also U?.1 (OUT)
Changed lines of the file:
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@@
     (pin "2")
-  )
-  (symbol (lib_id "Regulator_Linear:AMS1117-3.3") (at 132.08 74.93 0)
-    (in_bom yes) (on_board yes)
-    (property "Reference" "U10" (id 0) (at 132.08 68.7832 0))
-    (property "Value" "AMS1117-3.3" (id 1) (at 132.08 71.0946 0))
-    (property "Footprint" "Package_TO_SOT_SMD:SOT-89-3" (id 2) (at 132.08 69.85 0)
-      (effects (font (size 1.27 1.27)) hide)
-    )
-    (property "Datasheet" "http://www.advanced-monolithic.com/pdf/ds1117.pdf" (id 3) (at 134.62 81.28 0)
-      (effects (font (size 1.27 1.27)) hide)
-    )
-    (pin "1")
-    (pin "2")
-    (pin "3")
   )
   (symbol (lib_id "Device:R_Small") (at 127 109.22 0)
@@
     (pin "2")
   )
+  (symbol (lib_id "Regulator_Linear:L78L33_SOT89") (at 132.08 74.93 0)
+    (in_bom yes) (on_board yes) (fields_autoplaced)
+    (property "Reference" "U?" (id 0) (at 132.08 69.0585 0))
+    (property "Value" "L78L33_SOT89" (id 1) (at 132.08 71.8336 0))
+    (property "Footprint" "Package_TO_SOT_SMD:SOT-89-3" (id 2) (at 132.08 69.85 0)
+      (effects (font (size 1.27 1.27) italic) hide)
+    )
+    (property "Datasheet" "http://www.st.com/content/ccc/resource/technical/document/datasheet/15/55/e5/aa/23/5b/43/fd/CD00000446.pdf/files/CD00000446.pdf/jcr:content/translations/en.CD00000446.pdf" (id 3) (at 132.08 76.2 0)
+      (effects (font (size 1.27 1.27)) hide)
+    )
+    (pin "1")
+    (pin "2")
+    (pin "3")
+  )
   (symbol (lib_id "power:GND") (at 165.1 116.84 0)
