File: ykts-payload/ykts-payload-supervisor.kicad_sch (KiCad schematic)
At the start: 18 parts, among them J6 Conn_02x03_Odd_Even, J7 Conn_01x03_Male, U1 ATmega128A-AU, Y1 8 MHz

Commit message: Board revision A5, schematic E0
Fixed #16
Fixed #17
Revamped schematic
Parts:
- added C7: 10uF, Capacitor_SMD:C_0603_1608Metric, symbol Device:C_Small
- added C8: 22uF, Capacitor_SMD:C_0603_1608Metric, symbol Device:C_Small
- added R17, R18, R19: 10K, Resistor_SMD:R_0402_1005Metric, symbol Device:R_Small
- added R20, R21, R22: 4.7K, Resistor_SMD:R_0402_1005Metric, symbol Device:R_Small
- added U2: L78L33_SOT89, Package_TO_SOT_SMD:SOT-89-3, symbol Regulator_Linear:L78L33_SOT89
- added U3: AT25DF161-SF-T, Package_SO:SO-8_5.3x6.2mm_P1.27mm, symbol yktsat-common:AT25DF161-SF-T
Connections:
- net 5V: now also C7.1, U2.3 (IN)
- net GND: now also C7.2, C8.2, R17.2, R18.2, R19.2, U2.2 (GND), U3.4 (GND)
- net MISO: now also U3.2 (SO/IO1)
- net MOSI: now also R21.2
- net SCK: now also R20.2
- net SD_CS: now also R22.2
- new net: R19.1, R22.1, U3.1 (~{CS})
- new net: C8.1, U2.1 (OUT), U3.3 (~{WP}), U3.7 (~{HOLD}), U3.8 (VCC)
- new net: R18.1, R21.1, U3.5 (SI/IO0)
- new net: R17.1, R20.1, U3.6 (SCK)
Other:
- removed sheet Payload Supervisor Flash
- note added: "SPI Flash"
- moved on the sheet: C5

Commit message: Schematic revision E1
Cleanup
Parts:
- J6: value Conn_02x03_Odd_Even -> AVR ISP
- J7: value Conn_01x03_Male -> DBG_UART
Other:
- moved on the sheet: C1, C2, C3, C4, C5, C6, C7, C8, D2, J6, J7, L1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

Commit message: Sync with remote
Parts:
- renumbered C1 to C16, C2 to C17, C3 to C18, C4 to C19, C5 to C20, C6 to C21, C7 to C22, C8 to C23, D2 to D6, J6 to J8, J7 to J9, L1 to L2, R11 to R31, R12 to R32, R13 to R33, R14 to R34, R15 to R35, R16 to R36, R17 to R37, R18 to R38, R19 to R39, R20 to R40, R21 to R41, R22 to R42, U2 to U10, U3 to U11, U1 to U9, Y1 to Y3
Connections:
- net MUX_A0: now also U9.29 (PD4); no longer U9.31 (PD6)
- net MUX_A2: now also U9.31 (PD6); no longer U9.29 (PD4)
- net NODE0_PWR: now also U9.50 (PA1); no longer U9.40 (PC5)
- net NODE0_RST: now also U9.51 (PA0); no longer U9.39 (PC4)
- net NODE1_PWR: now also U9.48 (PA3); no longer U9.41 (PC6)
- net NODE1_RST: now also U9.49 (PA2); no longer U9.42 (PC7)
- net NODE2_PWR: now also U9.47 (PA4); no longer U9.45 (PA6)
- net NODE2_RST: now also U9.46 (PA5); no longer U9.44 (PA7)
- net NODE3_PWR: now also U9.45 (PA6); no longer U9.47 (PA4)
- net NODE3_RST: now also U9.44 (PA7); no longer U9.46 (PA5)
- net NODE5_PWR: now also U9.37 (PC2); no longer U9.50 (PA1)
- net NODE5_RST: now also U9.38 (PC3); no longer U9.51 (PA0)
- net NODE6_PWR: now also U9.40 (PC5); no longer U9.37 (PC2)
- net NODE6_RST: now also U9.39 (PC4); no longer U9.38 (PC3)
- net NODE7_PWR: now also U9.41 (PC6); no longer U9.48 (PA3)
- net NODE7_RST: now also U9.42 (PC7); no longer U9.49 (PA2)
Other:
- note added: "3V3_FLASH"
- moved on the sheet: C22, C23, R37, R38, R39, R40, R41, R42, U10, U11
