File: ykts-mcu-node/ykts-mcu-node.sch (KiCad schematic (older format))
At the start: 22 parts, among them J1 PWEN, J2 RX, J3 TX, J4 ~RST, J5 GND, J6 VCC, J7 VCC, J8 GND, SW1 ADG802BRT, U1 ATmega328PB-MU, Y1 8 MHz

Commit message: Hierarchal sheet rework
Parts:
- removed R3: 1M, Resistor_SMD:R_0402_1005Metric, symbol Device:R_Small
- J1, J4, J5, J6, J7, J8: footprint ykts-mcu-node:CastellatedHole_0.6mm -> ykts-mcu-node:CastellatedHole_1.0mm
- J2: value RX -> TX; footprint ykts-mcu-node:CastellatedHole_0.6mm -> ykts-mcu-node:CastellatedHole_1.0mm
- J3: value TX -> RX; footprint ykts-mcu-node:CastellatedHole_0.6mm -> ykts-mcu-node:CastellatedHole_1.0mm
- Y1: footprint Crystal:Crystal_SMD_2520-4Pin_2.5x2.0mm -> Crystal:Crystal_SMD_3225-4Pin_3.2x2.5mm
Other:
- moved on the sheet: J2, J3
