File: ykts-mcu-node/ykts-mcu-node.kicad_pcb (KiCad board)
At the start: 2 copper layers, 16.8 x 13.5 mm, 22 parts, among them J1 PWEN, J2 RX, J3 TX, J4 ~RST, J5 GND, J6 VCC, J7 VCC, J8 GND, SW1 ADG802BRT, U1 ATmega328PB-MU, Y1 8 MHz

Commit message: Hierarchal sheet rework
Parts:
- removed R3: 1M, Resistor_SMD:R_0402_1005Metric
- J1, J4, J5, J6, J7, J8: footprint ykts-mcu-node:CastellatedHole_0.6mm -> ykts-mcu-node:CastellatedHole_1.0mm
- J2: value RX -> TX; footprint ykts-mcu-node:CastellatedHole_0.6mm -> ykts-mcu-node:CastellatedHole_1.0mm
- J3: value TX -> RX; footprint ykts-mcu-node:CastellatedHole_0.6mm -> ykts-mcu-node:CastellatedHole_1.0mm
- Y1: footprint Crystal:Crystal_SMD_2520-4Pin_2.5x2.0mm -> Crystal:Crystal_SMD_3225-4Pin_3.2x2.5mm
- moved D1 2.09 mm to (115.6, 85.3)
- moved C1 2.09 mm to (116.1, 79.8)
- moved R4 2.09 mm to (116.6, 86.6)
- moved SW1 2.09 mm to (116.1, 82.8)
- moved J1 1.14 mm to (102.1, 87.4)
- moved J2 1.05 mm to (102.1, 84.8)
- moved J4 1.05 mm to (102.1, 79.8)
- moved J3 1.02 mm to (102.1, 82.3)
- moved TP1 0.92 mm to (113.0, 81.3)
- moved TP2 0.92 mm to (113.0, 83.6)
- moved TP3 0.92 mm to (113.0, 79.0)
- moved C3 0.85 mm to (113.3, 87.8)
- moved R1 0.72 mm to (104.6, 82.0)
- moved U1 0.72 mm to (108.6, 82.5)
- moved C2 0.68 mm to (108.8, 78.5)
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Connections:
- SW1 pad 5: Net-(SW1-Pad5) -> (no net)
- U1 pad 1: Net-(U1-Pad1) -> (no net)
- U1 pad 10: Net-(U1-Pad10) -> (no net)
- U1 pad 11: Net-(U1-Pad11) -> (no net)
- U1 pad 12: Net-(U1-Pad12) -> (no net)
- U1 pad 13: Net-(U1-Pad13) -> (no net)
- U1 pad 14: Net-(U1-Pad14) -> (no net)
- U1 pad 19: Net-(U1-Pad19) -> (no net)
- U1 pad 2: Net-(U1-Pad2) -> (no net)
- U1 pad 22: Net-(U1-Pad22) -> (no net)
- U1 pad 23: Net-(U1-Pad23) -> (no net)
- U1 pad 24: Net-(U1-Pad24) -> (no net)
- U1 pad 25: Net-(U1-Pad25) -> (no net)
- U1 pad 26: Net-(U1-Pad26) -> (no net)
- U1 pad 27: Net-(U1-Pad27) -> (no net)
- U1 pad 28: Net-(U1-Pad28) -> (no net)
- U1 pad 3: Net-(U1-Pad3) -> (no net)
- U1 pad 32: Net-(U1-Pad32) -> (no net)
- U1 pad 6: Net-(U1-Pad6) -> (no net)
- U1 pad 9: Net-(U1-Pad9) -> (no net)
Routing:
- net Net-(C2-Pad1): track 33.2 -> 31.0 mm
- net +5V: track 12.4 -> 13.9 mm
- net /ISP_MOSI: track 4.97 -> 3.74 mm
- net /ISP_RESET: track 4.80 -> 5.87 mm
- net Net-(C4-Pad1): track 7.87 -> 6.83 mm
- net /ISP_MISO: track 3.23 -> 2.25 mm
- net /UART0_RX: track 3.36 -> 3.98 mm
- net GND: track 11.1 -> 10.7 mm, vias 7 -> 10
Other:
- board size 16.8 x 13.5 mm -> 17.8 x 13.7 mm
- board text removed: "SCK"
- board text removed: "SI"
- board text removed: "SO"

Commit message: Revision D0
Parts:
- added Q1: RJU003N03 NMOS, Package_TO_SOT_SMD:SOT-323_SC-70, F.Cu at (116.6, 88.1)
- added Q2: RJU003N03 NMOS, Package_TO_SOT_SMD:SOT-323_SC-70, F.Cu at (112.8, 88.1)
- added R2: 10K, Resistor_SMD:R_0402_1005Metric, F.Cu at (115.8, 86.1)
- added R3: 10K, Resistor_SMD:R_0402_1005Metric, F.Cu at (112.0, 86.1)
- J1: value PWEN -> TX
- J2: value TX -> RX
- J3: value RX -> ~RST
- J4: value ~RST -> PWEN
- J5: value GND -> SDA
- J6: value VCC -> SCL
- moved C3 3.33 mm to (110.0, 87.3)
- moved C4 3.30 mm to (104.4, 87.8)
- moved Y1 3.30 mm to (107.2, 87.8)
- moved R4 1.93 mm to (117.3, 84.8), turned to 90 degrees
- moved C1 1.05 mm to (116.3, 78.7)
- moved SW1 1.05 mm to (116.3, 81.8)
- moved D1 1.02 mm to (115.6, 84.3)
- moved R1 0.76 mm to (103.9, 82.0)
- moved C2 0.32 mm to (108.8, 78.2)
- moved TP1 0.32 mm to (113.0, 81.0)
- moved TP2 0.32 mm to (113.0, 83.2)
- moved TP3 0.32 mm to (113.0, 78.7)
- moved U1 0.32 mm to (108.6, 82.2)
Connections:
- J1 pad 1: Net-(J1-Pad1) -> /UART0_TX
- J2 pad 1: /UART0_TX -> /UART0_RX
- J3 pad 1: /UART0_RX -> /ISP_RESET
- J4 pad 1: /ISP_RESET -> /PWEN
- J5 pad 1: GND -> /SDA
- J6 pad 1: +5V -> /SCL
- SW1 pad 4: Net-(J1-Pad1) -> /PWEN
- SW1 pad 5: (no net) -> unconnected-(SW1-Pad5)
- U1 pad 1: (no net) -> unconnected-(U1-Pad1)
- U1 pad 10: (no net) -> unconnected-(U1-Pad10)
- U1 pad 11: (no net) -> unconnected-(U1-Pad11)
- U1 pad 12: (no net) -> unconnected-(U1-Pad12)
- U1 pad 13: (no net) -> unconnected-(U1-Pad13)
- U1 pad 14: (no net) -> unconnected-(U1-Pad14)
- U1 pad 19: (no net) -> unconnected-(U1-Pad19)
- U1 pad 2: (no net) -> unconnected-(U1-Pad2)
- U1 pad 22: (no net) -> unconnected-(U1-Pad22)
- U1 pad 23: (no net) -> unconnected-(U1-Pad23)
- U1 pad 24: (no net) -> unconnected-(U1-Pad24)
- U1 pad 25: (no net) -> unconnected-(U1-Pad25)
- U1 pad 26: (no net) -> unconnected-(U1-Pad26)
- U1 pad 27: (no net) -> Net-(Q1-Pad1)
- U1 pad 28: (no net) -> Net-(Q2-Pad1)
- U1 pad 3: (no net) -> unconnected-(U1-Pad3)
- U1 pad 32: (no net) -> unconnected-(U1-Pad32)
- U1 pad 6: (no net) -> unconnected-(U1-Pad6)
- U1 pad 9: (no net) -> unconnected-(U1-Pad9)
Routing:
- net Net-(J1-Pad1): track 17.9 -> 0.00 mm, vias 1 -> 0
- net Net-(Q1-Pad1): track 0.00 -> 16.8 mm, vias 0 -> 2
- net /PWEN: track 0.00 -> 16.7 mm, vias 0 -> 2
- net Net-(Q2-Pad1): track 0.00 -> 15.0 mm, vias 0 -> 2
- net Net-(C2-Pad1): track 31.0 -> 45.5 mm
- net /SCL: track 0.00 -> 7.52 mm
- net +5V: track 13.9 -> 11.3 mm
- net /UART0_TX: track 4.05 -> 6.30 mm
- net Net-(C4-Pad1): track 6.83 -> 9.05 mm
- net /SDA: track 0.00 -> 2.19 mm
- net /ISP_RESET: track 5.87 -> 3.75 mm
- net GND: track 10.7 -> 11.0 mm, vias 10 -> 15
Other:
- net class Default removed
- board text added: "SCL"
- board text added: "SDA"
- board text added: "~{RST}"
- board text removed: "~RST"

Commit message: MCU Node silkscreen improvements
Fixes #7
Parts:
- moved C3 0.09 mm to (110.0, 87.2)
Other:
- board text added: "SCK SI SO"
- board text added: "YKTSAT-1 MCU Node Revision A1"

Commit message: Sync with remote
Routing:
- net Net-(C2-Pad1): track 45.7 -> 45.1 mm
Other:
- board text added: "0,2000 мм / 0,0000 мм"
- board text added: "0,3000 мм"
- board text added: "0,6000 мм"
- board text added: "17,8300 мм x 13,7660 мм"
- board text added: "2"
- board text added: "None"
- board text added: "Габариты платы:"
- board text added: "Да"
- board text added: "Количество слоёв меди:"
- board text added: "Контроль импеданса:"
- board text added: "Краевой соединитель:"
- board text added: "Метал. торцы:"
- board text added: "Мин. дорожка/зазор:"
- board text added: "Мин. сверло:"
- board text added: "Нет"
- board text added: "Периферийные полу-отверстия:"
- board text added: "Покрытие меди:"
- board text added: "Толщина платы:"
- board text added: "ХАРАКТЕРИСТИКИ ПЛАТЫ"
Changed lines of the file:
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@@
     (effects (font (size 1 1) (thickness 0.15)))
+  )
+  (gr_text "Количество слоёв меди: " (at 169.238857 24.695) (layer "Dwgs.User")
+    (effects (font (size 1.5 1.5) (thickness 0.2)) (justify left top))
+  )
+  (gr_text "17,8300 мм x 13,7660 мм" (at 209.296 29.21) (layer "Dwgs.User")
+    (effects (font (size 1.5 1.5) (thickness 0.2)) (justify left top))
+  )
+  (gr_text "None" (at 209.296 38.24) (layer "Dwgs.User")
+    (effects (font (size 1.5 1.5) (thickness 0.2)) (justify left top))
+  )
+  (gr_text "0,6000 мм" (at 269.124571 24.695) (layer "Dwgs.User")
+    (effects (font (size 1.5 1.5) (thickness 0.2)) (justify left top))
+  )
+  (gr_text "Нет" (at 269.124571 38.24) (layer "Dwgs.User")
+    (effects (font (size 1.5 1.5) (thickness 0.2)) (justify left top))
+  )
+  (gr_text "Толщина платы: " (at 241.638857 24.695) (layer "Dwgs.User")
+    (effects (font (size 1.5 1.5) (thickness 0.2)) (justify left top))
+  )
+  (gr_text "0,3000 мм" (at 269.124571 33.725) (layer "Dwgs.User")
+    (effects (font (size 1.5 1.5) (thickness 0.2)) (justify left top))
+  )
+  (gr_text "Метал. торцы: " (at 241.638857 42.755) (layer "Dwgs.User")
+    (effects (font (size 1.5 1.5) (thickness 0.2)) (justify left top))
+  )
+  (gr_text "Мин. сверло: " (at 241.638857 33.725) (layer "Dwgs.User")
+    (effects (font (size 1.5 1.5) (thickness 0.2)) (justify left top))
+  )
+  (gr_text "" (at 241.638857 29.21) (layer "Dwgs.User")
+    (effects (font (size 1.5 1.5) (thickness 0.2)) (justify left top))
+  )
+  (gr_text "Краевой соединитель: " (at 169.238857 47.27) (layer "Dwgs.User")
+    (effects (font (size 1.5 1.5) (thickness 0.2)) (justify left top))
+  )
+  (gr_text "Покрытие меди: " (at 169.238857 38.24) (layer "Dwgs.User")
+    (effects (font (size 1.5 1.5) (thickness 0.2)) (justify left top))
+  )
+  (gr_text "Контроль импеданса: " (at 241.638857 38.24) (layer "Dwgs.User")
+    (effects (font (size 1.5 1.5) (thickness 0.2)) (justify left top))
+  )
+  (gr_text "Нет" (at 269.124571 42.755) (layer "Dwgs.User")
+    (effects (font (size 1.5 1.5) (thickness 0.2)) (justify left top))
+  )
+  (gr_text "2" (at 209.296 24.695) (layer "Dwgs.User")
+    (effects (font (size 1.5 1.5) (thickness 0.2)) (justify left top))
+  )
+  (gr_text "Габариты платы: " (at 169.238857 29.21) (layer "Dwgs.User")
+    (effects (font (size 1.5 1.5) (thickness 0.2)) (justify left top))
+  )
+  (gr_text "Мин. дорожка/зазор: " (at 169.238857 33.725) (layer "Dwgs.User")
+    (effects (font (size 1.5 1.5) (thickness 0.2)) (justify left top))
+  )
+  (gr_text "" (at 269.124571 29.21) (layer "Dwgs.User")
+    (effects (font (size 1.5 1.5) (thickness 0.2)) (justify left top))
+  )
+  (gr_text "ХАРАКТЕРИСТИКИ ПЛАТЫ" (at 168.488857 18.525) (layer "Dwgs.User")
+    (effects (font (size 2 2) (thickness 0.4)) (justify left top))
+  )
+  (gr_text "Нет" (at 209.296 47.27) (layer "Dwgs.User")
+    (effects (font (size 1.5 1.5) (thickness 0.2)) (justify left top))
+  )
+  (gr_text "Да" (at 209.296 42.755) (layer "Dwgs.User")
+    (effects (font (size 1.5 1.5) (thickness 0.2)) (justify left top))
+  )
+  (gr_text "0,2000 мм / 0,0000 мм" (at 209.296 33.725) (layer "Dwgs.User")
+    (effects (font (size 1.5 1.5) (thickness 0.2)) (justify left top))
+  )
+  (gr_text "Периферийные полу-отверстия: " (at 169.238857 42.755) (layer "Dwgs.User")
+    (effects (font (size 1.5 1.5) (thickness 0.2)) (justify left top))
   )
   (dimension (type aligned) (layer "Dwgs.User")
@@
   (segment (start 109.0676 78.8924) (end 109.5248 78.8924) (width 0.2) (layer "F.Cu") (net 3))
   (segment (start 109.601 77.532) (end 109.319 77.814) (width 0.25) (layer "F.Cu") (net 3))
+  (segment (start 112.524 84.33) (end 112.522 84.328) (width 0.25) (layer "F.Cu") (net 3))
   (segment (start 109.06199 77.55699) (end 106.84701 77.55699) (width 0.2) (layer "F.Cu") (net 3))
   (segment (start 113.792 84.328) (end 115.085 84.328) (width 0.25) (layer "F.Cu") (net 3))
@@
   (segment (start 115.085 84.351) (end 116.334 85.6) (width 0.25) (layer "F.Cu") (net 3))
   (segment (start 112.38 88.788) (end 112.790989 88.377011) (width 0.25) (layer "F.Cu") (net 3))
-  (segment (start 112.524 86.106) (end 112.524 85.596) (width 0.25) (layer "F.Cu") (net 3))
   (segment (start 115.586 88.788) (end 113.201978 88.788) (width 0.25) (layer "F.Cu") (net 3))
   (segment (start 114.731999 78.725999) (end 113.538 77.532) (width 0.25) (layer "F.Cu") (net 3))
@@
   (segment (start 112.524 88.110022) (end 112.524 86.106) (width 0.25) (layer "F.Cu") (net 3))
   (segment (start 115.382 84.031) (end 115.085 84.328) (width 0.25) (layer "F.Cu") (net 3))
-  (segment (start 112.524 85.596) (end 113.792 84.328) (width 0.25) (layer "F.Cu") (net 3))
   (segment (start 111.5975 84.328) (end 113.792 84.328) (width 0.25) (layer "F.Cu") (net 3))
   (segment (start 109.319 78.167) (end 109.319 77.814) (width 0.25) (layer "F.Cu") (net 3))
@@
   (segment (start 109.5248 78.8924) (end 109.812 79.1796) (width 0.2) (layer "F.Cu") (net 3))
   (segment (start 108.812 79.148) (end 109.0676 78.8924) (width 0.2) (layer "F.Cu") (net 3))
+  (segment (start 112.524 86.106) (end 112.524 84.33) (width 0.25) (layer "F.Cu") (net 3))
   (via (at 111.252 84.6735) (size 0.6) (drill 0.35) (layers "F.Cu" "B.Cu") (net 3))
   (via (at 106.68 85.598) (size 0.6) (drill 0.35) (layers "F.Cu" "B.Cu") (net 3))
@@
     )
   )
+  (group "group-boardCharacteristics" (id 165f4d8d-26a9-4cf2-a8d6-9936cd983be4)
+    (members
+      06665bf8-cef1-4e75-8d5b-1537b3c1b090
+      178ae27e-edb9-4ffb-bd13-c0a6dd659606
+      1a22eb2d-f625-4371-a918-ff1b97dc8219
+      25c663ff-96b6-4263-a06e-d1829409cf73
+      291935ec-f8ff-41f0-8717-e68b8af7b8c1
+      34ce7009-187e-4541-a14e-708b3a2903d9
+      35fb7c56-dc85-43f7-b954-81b8040a8500
+      49a65079-57a9-46fc-8711-1d7f2cab8dbf
+      4e677390-a246-4ca0-954c-746e0870f88f
+      637e9edf-ffed-49a2-8408-fa110c9a4c79
+      6ae963fb-e34f-4e11-9adf-78839a5b2ef1
+      6ff9bb63-d6fd-4e32-bb60-7ac65509c2e9
+      73ee7e03-97a8-4121-b568-c25f3934a935
+      87ba184f-bff5-4989-8217-6af375cc3dd8
+      9fdca5c2-1fbd-4774-a9c3-8795a40c206d
+      a0d52767-051a-423c-a600-928281f27952
+      aa8663be-9516-4b07-84d2-4c4d668b8596
+      b456cffc-d9d7-4c91-91f2-36ec9a65dd1b
+      d32956af-146b-4a09-a053-d9d64b8dd86d
+      d45d1afe-78e6-4045-862c-b274469da903
+      d767f2ff-12ec-4778-96cb-3fdd7a473d60
+      dfcef016-1bf5-4158-8a79-72d38a522877
+      f674b8e7-203d-419e-988a-58e0f9ae4fad
+    )
+  )
