File: ykts-geigerboard/ykts-detector-mcu.kicad_sch (KiCad schematic)
At the start: 16 parts

Commit message: Sync with remote
Parts:
- R19, R21: renamed from R?; value 10K -> 33K
- gave numbers to parts that had none: 14
Connections:
- net +3V3: now also Q1.2 (G), Q2.2 (G), R19.2, R21.2
- net DET_IN_OUT: now reaches U7.19 (ADC6)
Other:
- note added: "Notes: 1. This schematic is not finished yet 2. DET_IN_TRIG signal is ~10 uSec 3. Mega328p ADC: - Sample & Hold 1.25 uSec - Full 10-bit sample time: 50 uSec @ 250 kHz ADC clock - Full 8-bit sample time: 10 uSec @ 2 MHz ADC clock - fast mode 4. Mega328p interrupt response time: 4 cycles + ~16 cycles ISR preamble - ~3 uSec until ADC conversion starts 5. Potentially replaceable with Mega4809 for 0.5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"
- title: (none) -> Detector MCU
- moved on the sheet: C18, C19, C20, C21, C22, C23, D3, L2, Q1, Q2, R18, R19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
