File: ykts-geigerboard/ykts-detector-psu.kicad_sch (KiCad schematic)
At the start: 0 parts

Commit message: Sync with remote
Parts:
- added C24: 1uF, Capacitor_SMD:C_0805_2012Metric, symbol Device:C_Small
- added C25: 100nF, Capacitor_SMD:C_0402_1005Metric, symbol Device:C_Small
- added C26: 2.2uF, Capacitor_SMD:C_0805_2012Metric, symbol Device:C_Small
- added C27: 4.7uF, Capacitor_SMD:C_0805_2012Metric, symbol Device:C_Small
- added C28: 220, Capacitor_SMD:C_0402_1005Metric, symbol Device:C_Small
- added C29, C30: 1000, Capacitor_SMD:C_0402_1005Metric, symbol Device:C_Small
- added C31, C32, C33, C34: 10nF, Capacitor_SMD:C_0402_1005Metric, symbol Device:C_Small
- added C35: 22uF 35V, Capacitor_Tantalum_SMD:CP_EIA-3216-10_Kemet-I, symbol Device:CP1_Small
- added D4: MBR0520LT, Diode_SMD:D_SOD-123, symbol Device:D
- added L3, L4: 10uH, Inductor_SMD:L_1812_4532Metric, symbol Device:L
- added R23: 10K, Resistor_SMD:R_0402_1005Metric, symbol Device:R_Small
- added R24: 13.3K, Resistor_SMD:R_0402_1005Metric, symbol Device:R_Small
- added R25: 270K, Resistor_SMD:R_0402_1005Metric, symbol Device:R_Small
- added R26: 100, Resistor_SMD:R_0603_1608Metric, symbol Device:R_Small
- added R27: 1K, Resistor_SMD:R_0603_1608Metric, symbol Device:R_Small
- added RV1: 33K, Potentiometer_SMD:Potentiometer_Bourns_3224J_Horizontal, symbol Device:R_POT_Small
- added U8: TPS2041B, Package_TO_SOT_SMD:SOT-23-5, symbol Power_Management:TPS2041B
- added U9: LM2733YMF, Package_TO_SOT_SMD:SOT-23-5, symbol Regulator_Switching:LM2733YMF
Connections:
- new net: C28.1, R24.1, R25.2, U9.3 (FB)
- new net: C27.1, C28.2, D4.1 (K), L4.1, R24.2
- new net: C29.1, C30.2, L4.2, R26.2
- new net: C31.1, C32.2, R26.1, R27.2
- new net: C25.2, C26.1, L3.1, U8.1 (OUT), U9.4 (EN), U9.5 (VIN)
- new net: R25.1, RV1.1, RV1.2
- new net: D4.2 (A), L3.2, U9.1 (SW)
- new net +5V: C24.1, U8.5 (IN)
- new net GEIGER_EN: R23.2, U8.4 (~{EN})
- new net GND: C24.2, C25.1, C26.2, C27.2, C29.2, C30.1, C31.2, C32.1, C33.2, C34.1, C35.2, R23.1, RV1.3, U8.2 (GND), U9.2 (GND)
- new net HV_OUT: C33.1, C34.2, C35.1, R27.1
- no-connect marks 0 -> 1
Other:
- note added: "28V Power Supply"
- note added: "Original shcematic by: @jar_ohty - KBRadar https://habr.com/ru/post/456878/"
- note added: "Output: 28V DC"
- title: (none) -> SiPM HV PSU
