File: ykts-geigerboard/ykts-geigerboard.kicad_pcb (KiCad board)
At the start: 2 copper layers, 79.8 x 81.5 mm, 21 parts, among them J1 Conn_01x07_Female, Q1 RJU003N03 NMOS, Q2 RJU003N03 NMOS, SW1 ADG802BRT, U1 ATmega328PB-MU, Y1 8 MHz

Commit message: SiPM analog detector schematic
Parts:
- added H7: MountingHole_Pad, MountingHole:MountingHole_3.2mm_M3_ISO7380_Pad, F.Cu at (99.7, 67.3)
- added J2: Conn_01x05_Female, Connector_Molex:Molex_PicoBlade_53048-0510_1x05_P1.25mm_Horizontal, F.Cu at (108.5, 101.4)
- added J3: Conn_01x05_Female, Connector_Molex:Molex_PicoBlade_53048-0510_1x05_P1.25mm_Horizontal, F.Cu at (108.8, 85.9)
- added J4: Conn_01x05_Female, Connector_Molex:Molex_PicoBlade_53048-0510_1x05_P1.25mm_Horizontal, F.Cu at (151.8, 134.7)
- added J5: Conn_01x05_Female, Connector_Molex:Molex_PicoBlade_53048-0510_1x05_P1.25mm_Horizontal, F.Cu at (135.5, 134.7)
- added J6: Conn_01x05_Female, Connector_Molex:Molex_PicoBlade_53048-0510_1x05_P1.25mm_Horizontal, F.Cu at (108.8, 117.4)
- added J7: Conn_01x05_Female, Connector_Molex:Molex_PicoBlade_53048-0510_1x05_P1.25mm_Horizontal, F.Cu at (119.0, 134.7)
- added U2: LMV7239M5, Package_TO_SOT_SMD:SOT-23-5, F.Cu at (161.0, 72.1)
- added U3: TS5A3166DBVR, Package_TO_SOT_SMD:SOT-23-5, F.Cu at (146.4, 82.8)
- added U4: AD8606ARZ, Package_SO:SOIC-8_3.9x4.9mm_P1.27mm, F.Cu at (152.3, 72.9)
- added U5: LMC555xM, Package_SO:SOIC-8_3.9x4.9mm_P1.27mm, F.Cu at (157.0, 82.4)
Other:
- board size 79.8 x 81.5 mm -> 79.9 x 83.8 mm

Commit message: Sync with remote
Parts:
- removed H5, H7: MountingHole_Pad, MountingHole:MountingHole_3.2mm_M3_ISO7380_Pad
- removed H6: MountingHole_Pad, MountingHole:MountingHole_2.2mm_M2_Pad
- removed J4, J5, J7: Conn_01x05_Female, Connector_Molex:Molex_PicoBlade_53048-0510_1x05_P1.25mm_Horizontal
- added J6: Conn_01x05_Female, Connector_Molex:Molex_PicoBlade_53048-0510_1x05_P1.25mm_Horizontal, B.Cu at (119.8, 102.8)
- added J6: Conn_01x05_Female, Connector_Molex:Molex_PicoBlade_53048-0510_1x05_P1.25mm_Horizontal, B.Cu at (131.4, 69.8)
- added J6: Conn_01x05_Female, Connector_Molex:Molex_PicoBlade_53048-0510_1x05_P1.25mm_Horizontal, B.Cu at (132.0, 111.9)
- J2, J3, J6, U2, U3, U4, U5: moved to B.Cu
- moved J3 59.6 mm to (162.4, 111.9), turned to 180 degrees
- moved J2 49.4 mm to (146.5, 69.8), turned to 0 degrees
- moved J6 38.4 mm to (146.8, 111.9), turned to 180 degrees
- moved U3 20.9 mm to (165.9, 75.2), turned to 180 degrees
- moved R4 18.8 mm to (144.3, 78.4), turned to -90 degrees
- moved D1 18.1 mm to (144.3, 80.9), turned to 90 degrees
- moved U4 14.2 mm to (162.1, 83.2), turned to 180 degrees
- moved U5 11.6 mm to (162.2, 92.8), turned to 180 degrees
- moved C2 7.16 mm to (139.1, 83.6)
- moved C4 7.16 mm to (127.6, 78.5)
- moved R1 7.16 mm to (127.9, 80.8)
- moved R2 7.16 mm to (131.7, 85.9)
- moved R3 7.16 mm to (127.9, 84.3)
- moved SW1 7.16 mm to (139.8, 86.4)
- moved Y1 7.16 mm to (139.0, 80.3)
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Other:
- board size 79.9 x 83.8 mm -> 59.8 x 52.5 mm
- board text added: "0,2000 мм / 0,0000 мм"
- board text added: "0,3000 мм"
- board text added: "1,6000 мм"
- board text added: "2"
- board text added: "59,9251 мм x 52,5542 мм"
- board text added: "None"
- board text added: "Габариты платы:"
- board text added: "Количество слоёв меди:"
- board text added: "Контроль импеданса:"
- board text added: "Краевой соединитель:"
- board text added: "Метал. торцы:"
- board text added: "Мин. дорожка/зазор:"
- board text added: "Мин. сверло:"
- board text added: "Нет"
- board text added: "Периферийные полу-отверстия:"
- board text added: "Покрытие меди:"
- board text added: "Толщина платы:"
- board text added: "ХАРАКТЕРИСТИКИ ПЛАТЫ"
