File: ykts-geigerboard/ykts-geigerboard.kicad_sch (KiCad schematic)
At the start: 21 parts, among them J1 Conn_01x07_Female, Q1 RJU003N03 NMOS, Q2 RJU003N03 NMOS, SW1 ADG802BRT, U1 ATmega328PB-MU, Y1 8 MHz

Commit message: SiPM analog detector schematic
Parts:
- removed C1: 1uF, Capacitor_SMD:C_0603_1608Metric, symbol Device:C_Small
- removed C2: 100nF, Capacitor_SMD:C_0402_1005Metric, symbol Device:C_Small
- removed C3, C4: 22pF, Capacitor_SMD:C_0402_1005Metric, symbol Device:C_Small
- removed D1: NODE_STATUSLED, LED_SMD:LED_0402_1005Metric, symbol Device:LED
- removed Q1, Q2: RJU003N03 NMOS, Package_TO_SOT_SMD:SOT-323_SC-70, symbol Device:Q_NMOS_SGD
- removed R1: 20K, Resistor_SMD:R_0402_1005Metric, symbol Device:R_Small
- removed R2, R3: 10K, Resistor_SMD:R_0402_1005Metric, symbol Device:R_Small
- removed R4: 1K, Resistor_SMD:R_0402_1005Metric, symbol Device:R_Small
- removed SW1: ADG802BRT, Package_TO_SOT_SMD:SOT-23-6, symbol yktsat-common:ADG802BRT
- removed U1: ATmega328PB-MU, Package_DFN_QFN:QFN-32-1EP_5x5mm_P0.5mm_EP3.1x3.1mm, symbol MCU_Microchip_ATmega:ATmega328PB-MU
- removed Y1: 8 MHz, Crystal:Crystal_SMD_3225-4Pin_3.2x2.5mm, symbol Device:Crystal_GND24_Small
- added H7: MountingHole_Pad, MountingHole:MountingHole_3.2mm_M3_ISO7380_Pad, symbol Mechanical:MountingHole_Pad
Other:
- added sheet Auxilary MCU (ykts-aux-mcu.kicad_sch)
- added sheet Detector MCU (ykts-detector-mcu.kicad_sch)
- added sheet HV PSU (ykts-detector-psu.kicad_sch)
- added sheet Light Sensors (ykts-light-sensors.kicad_sch)
- added sheet SiPM (ykts-sipm.kicad_sch)
- note removed: "Power input"
- moved on the sheet: H1, H2, H3, H4, H5, H6, J1

Commit message: Sync with remote
Other:
- sheet SiPM ports: added TRIG; removed none
