File: ykts-geigerboard/ykts-sipm.kicad_sch (KiCad schematic)
At the start: 30 parts, among them J2 DETECTOR, U1 NC7SVU04P5X, U2 LMV7239M5, U3 TS5A3166DBVR, U4 AD8606ARZ, U5 LMC555xM

Commit message: Sync with remote
Connections:
- net TRIG: now reaches U2.4, U5.2 (TR)
Other:
- note added: "Original shcematic by: @jar_ohty - KBRadar https://habr.com/ru/post/456878/"
- note removed: "Original shcematic by: @jar_ohty https://habr.com/ru/post/456878/"
- title: (none) -> SiPM analog in
Changed lines of the file:
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@@
 (kicad_sch (version 20211123) (generator eeschema)
   (paper "A4")
+  (title_block
+    (title "SiPM analog in")
+    (date "2022-03-26")
+    (rev "A0")
+  )
   (junction (at 102.87 72.39) (diameter 0) (color 0 0 0 0)
   )
@@
   (junction (at 171.45 123.19) (diameter 0) (color 0 0 0 0)
   )
+  (junction (at 156.21 69.85) (diameter 0) (color 0 0 0 0)
+  )
   (junction (at 186.69 53.34) (diameter 0) (color 0 0 0 0)
   )
@@
     (stroke (width 0) (type default) (color 0 0 0 0))
   )
+  (wire (pts (xy 156.21 69.85) (xy 173.99 69.85))
+    (stroke (width 0) (type default) (color 0 0 0 0))
+  )
   (wire (pts (xy 158.75 123.19) (xy 171.45 123.19))
     (stroke (width 0) (type default) (color 0 0 0 0))
@@
     (stroke (width 0) (type default) (color 0 0 0 0))
   )
+  (wire (pts (xy 156.21 97.155) (xy 156.21 69.85))
+    (stroke (width 0) (type default) (color 0 0 0 0))
+  )
   (wire (pts (xy 67.31 64.77) (xy 71.12 64.77))
     (stroke (width 0) (type default) (color 0 0 0 0))
@@
     (stroke (width 0) (type default) (color 0 0 0 0))
   )
-  (wire (pts (xy 144.78 69.85) (xy 173.99 69.85))
+  (wire (pts (xy 144.78 69.85) (xy 156.21 69.85))
     (stroke (width 0) (type default) (color 0 0 0 0))
   )
@@
     (stroke (width 0) (type default) (color 0 0 0 0))
   )
+  (wire (pts (xy 233.68 97.155) (xy 156.21 97.155))
+    (stroke (width 0) (type default) (color 0 0 0 0))
+  )
   (wire (pts (xy 96.52 83.82) (xy 102.87 83.82))
     (stroke (width 0) (type default) (color 0 0 0 0))
@@
     (stroke (width 0) (type default) (color 0 0 0 0))
   )
-  (text "Detector" (at 140.97 27.94 0)
+  (text "Detector" (at 142.24 31.75 0)
     (effects (font (size 2.54 2.54)) (justify left bottom))
   )
@@
     (effects (font (size 1.27 1.27)) (justify left bottom))
   )
-  (text "Original shcematic by:\n@jar_ohty\nhttps://habr.com/ru/post/456878/"
+  (text "Original shcematic by:\n@jar_ohty - KBRadar\nhttps://habr.com/ru/post/456878/"
     (at 180.34 176.53 0)
     (effects (font (size 1.27 1.27)) (justify left bottom))
@@
     (effects (font (size 1.27 1.27)) (justify left))
   )
+  (hierarchical_label "TRIG" (shape output) (at 233.68 97.155 0)
+    (effects (font (size 1.27 1.27)) (justify left))
+  )
